Commit message: adapt launch file to new packages names

File: cob_defs/ros/defs/arm.urdf (robot description, URDF)
Before this commit: robot arm, 8 links, 7 joints
Links:
- link link_arm0: geometry collision mesh filename=package://cob_defs/common/files/meshes/arm0.stl; visual mesh filename=package://cob_defs/common/files/meshes/arm0.stl
- link link_arm1: geometry collision mesh filename=package://cob_defs/common/files/meshes/arm1.stl; visual mesh filename=package://cob_defs/common/files/meshes/arm1.stl
- link link_arm2: geometry collision mesh filename=package://cob_defs/common/files/meshes/arm2.stl; visual mesh filename=package://cob_defs/common/files/meshes/arm2.stl
- link link_arm3: geometry collision mesh filename=package://cob_defs/common/files/meshes/arm3.stl; visual mesh filename=package://cob_defs/common/files/meshes/arm3.stl
- link link_arm4: geometry collision mesh filename=package://cob_defs/common/files/meshes/arm4.stl; visual mesh filename=package://cob_defs/common/files/meshes/arm4.stl
- link link_arm5: geometry collision mesh filename=package://cob_defs/common/files/meshes/arm5.stl; visual mesh filename=package://cob_defs/common/files/meshes/arm5.stl
- link link_arm6: geometry collision mesh filename=package://cob_defs/common/files/meshes/arm6.stl; visual mesh filename=package://cob_defs/common/files/meshes/arm6.stl
- link link_arm7: geometry collision mesh filename=package://cob_defs/common/files/meshes/arm7.stl; visual mesh filename=package://cob_defs/common/files/meshes/arm7.stl

File: cob_defs/ros/defs/sdh.urdf (robot description, URDF)
Before this commit: robot sdh, 10 links, 9 joints
Links:
- link link_finger11: geometry collision mesh filename=package://cob_defs/common/files/meshes/knuckle.stl; visual mesh filename=package://cob_defs/common/files/meshes/knuckle.stl
- link link_finger12: geometry collision mesh filename=package://cob_defs/common/files/meshes/finger.stl; visual mesh filename=package://cob_defs/common/files/meshes/finger.stl
- link link_finger13: geometry collision mesh filename=package://cob_defs/common/files/meshes/finger_tip.stl; visual mesh filename=package://cob_defs/common/files/meshes/finger_tip.stl
- link link_finger21: geometry collision mesh filename=package://cob_defs/common/files/meshes/knuckle.stl; visual mesh filename=package://cob_defs/common/files/meshes/knuckle.stl
- link link_finger22: geometry collision mesh filename=package://cob_defs/common/files/meshes/finger.stl; visual mesh filename=package://cob_defs/common/files/meshes/finger.stl
- link link_finger23: geometry collision mesh filename=package://cob_defs/common/files/meshes/finger_tip.stl; visual mesh filename=package://cob_defs/common/files/meshes/finger_tip.stl
- link link_palm: geometry collision mesh filename=package://cob_defs/common/files/meshes/palm.stl; visual mesh filename=package://cob_defs/common/files/meshes/palm.stl
- link link_thumb1: geometry collision mesh filename=package://cob_defs/common/files/meshes/knuckle.stl; visual mesh filename=package://cob_defs/common/files/meshes/knuckle.stl
- link link_thumb2: geometry collision mesh filename=package://cob_defs/common/files/meshes/finger.stl; visual mesh filename=package://cob_defs/common/files/meshes/finger.stl
- link link_thumb3: geometry collision mesh filename=package://cob_defs/common/files/meshes/finger_tip.stl; visual mesh filename=package://cob_defs/common/files/meshes/finger_tip.stl

File: cob_defs/ros/defs/torso.urdf (robot description, URDF)
Before this commit: robot torso, 19 links, 18 joints
Links:
- link link_head: geometry collision mesh filename=package://cob_defs/common/files/meshes/head.stl; visual mesh filename=package://cob_defs/common/files/meshes/head.stl
- link link_head_cover: geometry collision mesh filename=package://cob_defs/common/files/meshes/head_cover.stl; visual mesh filename=package://cob_defs/common/files/meshes/head_cover.stl
- link link_neck: geometry collision mesh filename=package://cob_defs/common/files/meshes/neck.stl; visual mesh filename=package://cob_defs/common/files/meshes/neck.stl
- link link_platform: geometry collision mesh filename=package://cob_defs/common/files/meshes/platform.stl; visual mesh filename=package://cob_defs/common/files/meshes/platform.stl
- link link_tray: geometry collision mesh filename=package://cob_defs/common/files/meshes/tray.stl; visual mesh filename=package://cob_defs/common/files/meshes/tray.stl

File: cob_defs/ros/robots/arm.urdf.xacro (robot description, xacro)
@@ -1,16 +1,16 @@
 <?xml version="1.0"?>
-<robot name="cob3_sdh"
+<robot name="cob_arm"
 	xmlns:sensor="http://playerstage.sourceforge.net/gazebo/xmlschema/#sensor"
 	xmlns:controller="http://playerstage.sourceforge.net/gazebo/xmlschema/#controller"
 	xmlns:interface="http://playerstage.sourceforge.net/gazebo/xmlschema/#interface">
 	<!-- include gazebo defs-->
-	<include filename="$(find cob3_defs)/ros/defs/gazebo.urdf" />
+	<include filename="$(find cob_defs)/ros/defs/gazebo.urdf" />
 	<!-- create joint to world -->
-	<joint name="joint_world_palm" type="fixed">
-		<origin xyz="0 0 0" rpy="0 0 0" />
+	<joint name="joint_world_arm0" type="fixed">
+		<origin xyz="0 0 0" rpy="3.1415926 0 0" />
 		<parent link="world"/>
-		<child link="link_palm"/>
+		<child link="link_arm0"/>
 	</joint>
-	<!-- include sdh defs-->
-	<include filename="$(find cob3_defs)/ros/defs/sdh.urdf" />
+	<!-- include arm defs-->
+	<include filename="$(find cob_defs)/ros/defs/arm.urdf" />
 </robot>

File: cob_defs/ros/robots/cob3.urdf.xacro (robot description, xacro)
@@ -5,5 +5,5 @@
 	xmlns:interface="http://playerstage.sourceforge.net/gazebo/xmlschema/#interface">
 	<!-- include gazebo defs-->
-	<include filename="$(find cob3_defs)/ros/defs/gazebo.urdf" />
+	<include filename="$(find cob_defs)/ros/defs/gazebo.urdf" />
 	<!-- create joint to world -->
 	<joint name="joint_world_platform" type="fixed">
@@ -13,9 +13,9 @@
 	</joint>
 	<!-- include torso defs-->
-	<include filename="$(find cob3_defs)/ros/defs/torso.urdf" />
+	<include filename="$(find cob_defs)/ros/defs/torso.urdf" />
 	<!-- include sensor defs-->
-	<include filename="$(find cob3_defs)/ros/defs/torso_sensors.urdf" />
+	<include filename="$(find cob_defs)/ros/defs/torso_sensors.urdf" />
 	<!-- include arm defs-->
-	<include filename="$(find cob3_defs)/ros/defs/arm.urdf" />
+	<include filename="$(find cob_defs)/ros/defs/arm.urdf" />
 	<joint name="joint_platform_arm0" type="fixed">
 		<origin xyz="0.040 -0.005 0.83637" rpy="3.1415926 0.7854 -1.8326" /> <!-- TODO: put in real transformation from platform to arm0-->
@@ -24,5 +24,5 @@
 	</joint>
 	<!-- include sdh defs-->
-	<include filename="$(find cob3_defs)/ros/defs/sdh.urdf" />
+	<include filename="$(find cob_defs)/ros/defs/sdh.urdf" />
   	<joint name="joint_arm7_palm" type="fixed">
 		<origin xyz="0 0 -0.1126" rpy="0 0 0" />

File: cob_defs/ros/robots/cob3_torso_arm_sdh.urdf.xacro (robot description, xacro)
@@ -5,5 +5,5 @@
 	xmlns:interface="http://playerstage.sourceforge.net/gazebo/xmlschema/#interface">
 	<!-- include gazebo defs-->
-	<include filename="$(find cob3_defs)/ros/defs/gazebo.urdf" />
+	<include filename="$(find cob_defs)/ros/defs/gazebo.urdf" />
 	<!-- create joint to world -->
 	<joint name="joint_world_torso" type="fixed">
@@ -13,5 +13,5 @@
 	</joint>
 	<!-- include torso defs-->
-	<include filename="$(find cob3_defs)/ros/defs/torso.urdf" />
+	<include filename="$(find cob_defs)/ros/defs/torso.urdf" />
 	<joint name="joint_basePlate_torso" type="fixed">
 		<origin xyz="0 0 0.1126" rpy="0 0 0" />
@@ -20,5 +20,5 @@
 	</joint>
 	<!-- include arm defs-->
-	<include filename="$(find cob3_defs)/ros/defs/arm.urdf" />
+	<include filename="$(find cob_defs)/ros/defs/arm.urdf" />
 	<joint name="joint_torso_arm0" type="fixed">
 		<origin xyz="-0.1 0 0.3" rpy="0.5 0 0" />
@@ -27,5 +27,5 @@
 	</joint>
 	<!-- include sdh defs-->
-	<include filename="$(find cob3_defs)/ros/defs/sdh.urdf" />
+	<include filename="$(find cob_defs)/ros/defs/sdh.urdf" />
   	<joint name="joint_arm7_palm" type="fixed">
 		<origin xyz="0 0 0.1126" rpy="0 0 0" />

File: cob_defs/ros/robots/sdh.urdf.xacro (robot description, xacro)
@@ -1,16 +1,16 @@
 <?xml version="1.0"?>
-<robot name="cob3_arm"
+<robot name="cob_sdh"
 	xmlns:sensor="http://playerstage.sourceforge.net/gazebo/xmlschema/#sensor"
 	xmlns:controller="http://playerstage.sourceforge.net/gazebo/xmlschema/#controller"
 	xmlns:interface="http://playerstage.sourceforge.net/gazebo/xmlschema/#interface">
 	<!-- include gazebo defs-->
-	<include filename="$(find cob3_defs)/ros/defs/gazebo.urdf" />
+	<include filename="$(find cob_defs)/ros/defs/gazebo.urdf" />
 	<!-- create joint to world -->
-	<joint name="joint_world_arm0" type="fixed">
-		<origin xyz="0 0 0" rpy="3.1415926 0 0" />
+	<joint name="joint_world_palm" type="fixed">
+		<origin xyz="0 0 0" rpy="0 0 0" />
 		<parent link="world"/>
-		<child link="link_arm0"/>
+		<child link="link_palm"/>
 	</joint>
-	<!-- include arm defs-->
-	<include filename="$(find cob3_defs)/ros/defs/arm.urdf" />
+	<!-- include sdh defs-->
+	<include filename="$(find cob_defs)/ros/defs/sdh.urdf" />
 </robot>

File: cob_defs/ros/robots/torso.urdf.xacro (robot description, xacro)
@@ -1,9 +1,9 @@
 <?xml version="1.0"?>
-<robot name="cob3_torso"
+<robot name="cob_torso"
 	xmlns:sensor="http://playerstage.sourceforge.net/gazebo/xmlschema/#sensor"
 	xmlns:controller="http://playerstage.sourceforge.net/gazebo/xmlschema/#controller"
 	xmlns:interface="http://playerstage.sourceforge.net/gazebo/xmlschema/#interface">
 	<!-- include gazebo defs-->
-	<include filename="$(find cob3_defs)/ros/defs/gazebo.urdf" />
+	<include filename="$(find cob_defs)/ros/defs/gazebo.urdf" />
 	<!-- create joint to world -->
 	<joint name="joint_world_platform" type="fixed">
@@ -13,6 +13,6 @@
 	</joint>
 	<!-- include torso defs-->
-	<include filename="$(find cob3_defs)/ros/defs/torso.urdf" />
+	<include filename="$(find cob_defs)/ros/defs/torso.urdf" />
 	<!-- include sensor defs-->
-	<include filename="$(find cob3_defs)/ros/defs/torso_sensors.urdf" />
+	<include filename="$(find cob_defs)/ros/defs/torso_sensors.urdf" />
 </robot>
