Commit message: changed cob3_defs to cob_def in xacro, launch and urdf files

File: cob_defs/ros/defs/platform.urdf (robot description, URDF)
Before this commit: robot torso, 9 links, 8 joints
Links:
- link link_platform: geometry collision mesh filename=package://cob_defs/common/files/meshes/platform.stl; visual mesh filename=package://cob_defs/common/files/meshes/platform.stl

File: cob_defs/ros/defs/pr2base.urdf.xacro (robot description, xacro)
@@ -3,6 +3,6 @@
        xmlns:controller="http://playerstage.sourceforge.net/gazebo/xmlschema/#controller"
        xmlns:interface="http://playerstage.sourceforge.net/gazebo/xmlschema/#interface">
-  <include filename="$(find cob3_defs)/ros/defs/pr2base_gazebo.xacro" />
-  <include filename="$(find cob3_defs)/ros/defs/pr2base_transmission.xacro" />
+  <include filename="$(find cob_defs)/ros/defs/pr2base_gazebo.xacro" />
+  <include filename="$(find cob_defs)/ros/defs/pr2base_transmission.xacro" />
   <property name="M_PI" value="3.1415926535897931" />
   <property name="caster_wheel_offset_y" value="0.049" /> <!-- from function spreadsheet -->
@@ -116,5 +116,5 @@
         <origin xyz="0 0 0" rpy="0 0 0" />
         <geometry>
-          <mesh filename="package://cob3_defs/common/files/meshes/platform.stl"/>
+          <mesh filename="package://cob_defs/common/files/meshes/platform.stl"/>
         </geometry>
         <material name="Green" />
@@ -169,5 +169,5 @@
 			<origin xyz="0 0 0" rpy="0 0 0" />
 			<geometry>
-				<mesh filename="package://cob3_defs/common/files/meshes/neck.stl" />
+				<mesh filename="package://cob_defs/common/files/meshes/neck.stl" />
 			</geometry>
 		</visual>
@@ -175,5 +175,5 @@
 			<origin xyz="0 0 0" rpy="0 0 0" />
 			<geometry>
-				<mesh filename="package://cob3_defs/common/files/meshes/neck.stl"/>
+				<mesh filename="package://cob_defs/common/files/meshes/neck.stl"/>
 			</geometry>
 		</collision>
@@ -192,5 +192,5 @@
 			<origin xyz="0 0 0" rpy="0 0 0" />
 			<geometry>
-				<mesh filename="package://cob3_defs/common/files/meshes/head.stl" />
+				<mesh filename="package://cob_defs/common/files/meshes/head.stl" />
 			</geometry>
 		</visual>
@@ -198,5 +198,5 @@
 			<origin xyz="0 0 0" rpy="0 0 0" />
 			<geometry>
-				<mesh filename="package://cob3_defs/common/files/meshes/head.stl"/>
+				<mesh filename="package://cob_defs/common/files/meshes/head.stl"/>
 			</geometry>
 		</collision>

File: cob_defs/ros/robots/cob3_arm.urdf.xacro (robot description, xacro)
@@ -5,5 +5,5 @@
 	xmlns:interface="http://playerstage.sourceforge.net/gazebo/xmlschema/#interface">
 	<!-- include gazebo defs-->
-	<include filename="$(find cob3_defs)/ros/defs/gazebo.urdf" />
+	<include filename="$(find cob_defs)/ros/defs/gazebo.urdf" />
 	<!-- create joint to world -->
 	<joint name="joint_world_arm0" type="fixed">
@@ -13,4 +13,4 @@
 	</joint>
 	<!-- include arm defs-->
-	<include filename="$(find cob3_defs)/ros/defs/arm.urdf" />
+	<include filename="$(find cob_defs)/ros/defs/arm.urdf" />
 </robot>

File: cob_defs/ros/robots/cob3_platform.urdf.xacro (robot description, xacro)
@@ -5,5 +5,5 @@
 	xmlns:interface="http://playerstage.sourceforge.net/gazebo/xmlschema/#interface">
 	<!-- include gazebo defs-->
-	<include filename="$(find cob3_defs)/ros/defs/gazebo.urdf" />
+	<include filename="$(find cob_defs)/ros/defs/gazebo.urdf" />
 	<!-- create joint to world -->
 <!--	<joint name="joint_world_platform" type="floating">
@@ -14,4 +14,4 @@
 -->
 	<!-- include torso defs-->
-	<include filename="$(find cob3_defs)/ros/defs/platform.urdf" />
+	<include filename="$(find cob_defs)/ros/defs/platform.urdf" />
 </robot>

File: cob_defs/ros/robots/cob3_pr2base.urdf.xacro (robot description, xacro)
@@ -5,6 +5,6 @@
 	<!--  <include filename="$(find pr2_defs)/defs/head/head_defs.urdf.xacro" />
 	<include filename="$(find pr2_defs)/defs/body/body_defs.urdf.xacro" /> -->
-	<include filename="$(find cob3_defs)/ros/defs/pr2base.urdf.xacro" />
-	<include filename="$(find cob3_defs)/ros/defs/gazebo.urdf" />
+	<include filename="$(find cob_defs)/ros/defs/pr2base.urdf.xacro" />
+	<include filename="$(find cob_defs)/ros/defs/gazebo.urdf" />
 	<include filename="$(find pr2_defs)/defs/materials.urdf.xacro" />
 	<pr2_base name="base"/>

File: cob_defs/ros/robots/cob3_sdh.urdf.xacro (robot description, xacro)
@@ -5,5 +5,5 @@
 	xmlns:interface="http://playerstage.sourceforge.net/gazebo/xmlschema/#interface">
 	<!-- include gazebo defs-->
-	<include filename="$(find cob3_defs)/ros/defs/gazebo.urdf" />
+	<include filename="$(find cob_defs)/ros/defs/gazebo.urdf" />
 	<!-- create joint to world -->
 	<joint name="joint_world_palm" type="fixed">
@@ -13,4 +13,4 @@
 	</joint>
 	<!-- include sdh defs-->
-	<include filename="$(find cob3_defs)/ros/defs/sdh.urdf" />
+	<include filename="$(find cob_defs)/ros/defs/sdh.urdf" />
 </robot>

File: cob_defs/ros/robots/cob3_torso.urdf.xacro (robot description, xacro)
@@ -5,5 +5,5 @@
 	xmlns:interface="http://playerstage.sourceforge.net/gazebo/xmlschema/#interface">
 	<!-- include gazebo defs-->
-	<include filename="$(find cob3_defs)/ros/defs/gazebo.urdf" />
+	<include filename="$(find cob_defs)/ros/defs/gazebo.urdf" />
 	<!-- create joint to world -->
 	<joint name="joint_world_platform" type="fixed">
@@ -13,6 +13,6 @@
 	</joint>
 	<!-- include torso defs-->
-	<include filename="$(find cob3_defs)/ros/defs/torso.urdf" />
+	<include filename="$(find cob_defs)/ros/defs/torso.urdf" />
 	<!-- include sensor defs-->
-	<include filename="$(find cob3_defs)/ros/defs/torso_sensors.urdf" />
+	<include filename="$(find cob_defs)/ros/defs/torso_sensors.urdf" />
 </robot>
