Commit message: desire update

File: desire_description/ros/urdf/base_v0/base.urdf.xacro (robot description, xacro)
@@ -59,5 +59,5 @@
         <origin xyz="0 0 0" rpy="0 0 0" />
         <geometry>
-          <mesh filename="package://desire_description/ros/meshes/base_v0/pr2_wheel.stl" />
+          <mesh filename="package://cob_description/ros/meshes/base_v0/pr2_wheel.stl" />
         </geometry>
         <material name="Wheel_${suffix}" />
@@ -96,5 +96,5 @@
         <origin xyz="0 0 0" rpy="0 0 0" />
         <geometry>
-          <mesh filename="package://desire_description/ros/meshes/base_v0/caster.stl" />
+          <mesh filename="$(find cob_description)/ros/meshes/base_v0/caster.stl" />
         </geometry>
         <material name="Green" />
@@ -134,5 +134,5 @@
         <!-- modify here for test-->
         <geometry>
-          <mesh filename="package://desire_defs/common/files/meshes/platform.stl"/>
+          <mesh filename="$(find desire_description)/ros/meshes/base_v0/base.stl"/>
         </geometry>
         <material name="Grey"/>

File: desire_description/ros/urdf/head_v0/head.transmission.xacro (robot description, xacro)
@@ -5,12 +5,12 @@
        xmlns:xacro="http://ros.org/wiki/xacro">
 	<xacro:macro name="desire_head_transmission_v0" params="name">
-		<transmission name="${name}_axis1_trans" type="pr2_mechanism_model/SimpleTransmission">
-			<actuator name="${name}_axis1_motor"/>
-			<joint name="${name}_axis1_joint"/>
+		<transmission name="${name}_pan_trans" type="pr2_mechanism_model/SimpleTransmission">
+			<actuator name="${name}_pan_motor"/>
+			<joint name="${name}_pan_joint"/>
 			<mechanicalReduction>1</mechanicalReduction>
 		</transmission>
-		<transmission name="${name}_axis2_trans" type="pr2_mechanism_model/SimpleTransmission">
-			<actuator name="${name}_axis2_motor"/>
-			<joint name="${name}_axis2_joint"/>
+		<transmission name="${name}_tilt_trans" type="pr2_mechanism_model/SimpleTransmission">
+			<actuator name="${name}_tilt_motor"/>
+			<joint name="${name}_tilt_joint"/>
 			<mechanicalReduction>1</mechanicalReduction>
 		</transmission>

File: desire_description/ros/urdf/head_v0/head.urdf.xacro (robot description, xacro)
@@ -6,13 +6,12 @@
 	<include filename="$(find desire_description)/ros/urdf/head_v0/head.gazebo.xacro" />
 	<include filename="$(find desire_description)/ros/urdf/head_v0/head.transmission.xacro" />
-	<include filename="$(find desire_description)/ros/urdf/sensors/cameraone.urdf.xacro" />
-	<include filename="$(find desire_description)/ros/urdf/sensors/tof.urdf.xacro" />
-	<include filename="$(find desire_description)/ros/urdf/sensors/hokuyo_SR400_laser.urdf.xacro" />
+	<include filename="$(find cob_description)/ros/urdf/sensors/cameraone.urdf.xacro" />
+	<include filename="$(find cob_description)/ros/urdf/sensors/tof.urdf.xacro" />
 	<xacro:macro name="desire_head_v0" params="name parent *origin">
 		<!-- joint between base_link and head_axis_link -->
-		<joint name="${name}_axis1_joint" type="revolute">
+		<joint name="${name}_pan_joint" type="revolute">
 			<insert_block name="origin" />
 			<parent link="${parent}"/>
-			<child link="${name}_axis1_link"/>
+			<child link="${name}_pan_link"/>
 			<axis xyz="0 0 1" />
 			<dynamics damping="0.1" />
@@ -20,5 +19,5 @@
 			<limit effort="100" lower="-3.2" upper="0.1" velocity="0.5"/>
 		</joint>
-		<link name="${name}_axis1_link">
+		<link name="${name}_pan_link">
 			<inertial>
 				<origin xyz="0 0 0" rpy="0 0 0"/>
@@ -40,14 +39,14 @@
 			</collision>
 		</link>
-		<joint name="${name}_axis2_joint" type="revolute">
-			<insert_block name="origin" />
-			<parent link="${name}_axis1_link"/>
-			<child link="${name}_axis2_link"/>
-			<axis xyz="1 0 0" />
+		<joint name="${name}_tilt_joint" type="revolute">
+			<origin xyz="0 0 0" rpy="1.5708 0 0"/>
+			<parent link="${name}_pan_link"/>
+			<child link="${name}_tilt_link"/>
+			<axis xyz="0 0 1" />
 			<dynamics damping="0.1" />
 			<calibration rising="${head_axis_ref}" falling="${head_axis_ref}"/>
 			<limit effort="100" lower="-3.2" upper="0.1" velocity="0.5"/>
 		</joint>
-		<link name="${name}_axis2_link">
+		<link name="${name}_tilt_link">
 			<inertial>
 				<origin xyz="0 0 0" rpy="0 0 0"/>
@@ -70,15 +69,15 @@
 		</link>
 		<!-- right camera -->
-		<xacro:desire_cameraone_v0 name="${name}_color_camera_r" parent="${name}_axis2_link">
+		<xacro:cob_cameraone_v0 name="${name}_color_camera_r" parent="${name}_tilt_link">
 			<origin xyz="${cam_r_x} ${cam_r_y} ${cam_r_z-0.06}" rpy="${cam_r_roll} ${cam_r_pitch+1.5708} ${cam_r_yaw+3.14159}" />
-		</xacro:desire_cameraone_v0>
+		</xacro:cob_cameraone_v0>
 		<!-- left camera -->
-		<xacro:desire_cameraone_v0 name="${name}_color_camera_l" parent="${name}_axis2_link">
+		<xacro:cob_cameraone_v0 name="${name}_color_camera_l" parent="${name}_tilt_link">
 			<origin xyz="${cam_l_x-0.12} ${cam_l_y} ${cam_l_z}" rpy="${cam_l_roll} ${cam_l_pitch} ${cam_l_yaw}" />
-		</xacro:desire_cameraone_v0>
+		</xacro:cob_cameraone_v0>
 		<!-- tof -->
-		<xacro:desire_tof_v0 name="${name}_tof" parent="${name}_axis2_link">
+		<xacro:cob_tof_v0 name="${name}_tof" parent="${name}_tilt_link">
 			<origin xyz="${tof_x-0.06} ${tof_y} ${tof_z}" rpy="${tof_roll} ${tof_pitch} ${tof_yaw}" />
-		</xacro:desire_tof_v0>
+		</xacro:cob_tof_v0>
 		<!-- extensions -->
 		<xacro:desire_head_gazebo_v0 name="${name}" />

File: desire_description/ros/urdf/torso_v0/torso.urdf.xacro (robot description, xacro)
@@ -15,19 +15,19 @@
 		<link name="${name}_lower_link">
 			<inertial>
-				<origin xyz="0 0 0.2155" rpy="0 0 0"/>
+				<origin xyz="0 0 0" rpy="0 0 0"/>
 				<mass value="1.0"/>
 				<inertia ixx="0.200549" ixy="0.001322" ixz="-0.000000" iyy="0.123664" iyz="-0.000000" izz="0.104101" />
 			</inertial>
 			<visual>
-				<origin xyz="0 0 0.2155" rpy="0 0 0" />
+				<origin xyz="0 0 0" rpy="0 0 0" />
 				<geometry>
-					<box size="0.433 0.512 0.431"/>
+					<box size="0.01 0.01 0.01"/>
 				</geometry>
 				<material name="Blue" />
 			</visual>
 			<collision>
-				<origin xyz="0 0 0.2155" rpy="0 0 0" />
+				<origin xyz="0 0 0.0" rpy="0 0 0" />
 				<geometry>
-					<box size="0.433 0.512 0.431"/>
+					<box size="0.01 0.01 0.01"/>
 				</geometry>
 			</collision>
@@ -35,5 +35,5 @@
 		<!-- joint between torso_lower_link and torso_middle_link -->
 		<joint name="${name}_middle_joint" type="fixed">
-			<origin xyz="0 0 0.2155" rpy="0 0 0" />
+			<origin xyz="0 0 0" rpy="0 0 0" />
 			<parent link="${name}_lower_link"/>
 			<child link="${name}_middle_link"/>
@@ -48,12 +48,12 @@
 				<origin xyz="0 0 0.2155" rpy="0 0 0" />
 				<geometry>
-					<box size="0.433 0.512 0.431"/>
+				<mesh filename="$(find desire_description)/ros/meshes/head_v0/head.stl"/>
 				</geometry>
 				<material name="Red" />
 			</visual>
 			<collision>
-				<origin xyz="0 0 0.2155" rpy="0 0 0" />
+				<origin xyz="0 0 0" rpy="0 0 0" />
 				<geometry>
-					<box size="0.433 0.512 0.431"/>
+				<mesh filename="$(find desire_description)/ros/meshes/head_v0/head.stl"/>
 				</geometry>
 			</collision>

Commit message: restructure urdf files and launch files for simulation

File: desire_description/ros/urdf/base_v0/base.urdf.xacro (robot description, xacro)
@@ -134,7 +134,7 @@
         <!-- modify here for test-->
         <geometry>
-          <mesh filename="$(find desire_description)/ros/meshes/base_v0/base.stl"/>
-        </geometry>
-        <material name="Grey"/>
+          <mesh filename="package://desire_description/ros/meshes/base_v0/base.stl"/>
+        </geometry>
+        <material name="Green"/>
       </visual>
       <collision>

File: desire_description/ros/urdf/head_v0/head.urdf.xacro (robot description, xacro)
@@ -57,5 +57,5 @@
 				<origin xyz="0 0 0" rpy="0 0 0" />
 				<geometry>
-					<box size="0.01 0.01 0.12"/>
+					<mesh filename="package://desire_description/ros/meshes/head_v0/head.stl"/>
 				</geometry>
 				<material name="Green" />
@@ -64,5 +64,5 @@
 				<origin xyz="0 0 0" rpy="0 0 0" />
 				<geometry>
-					<box size="0.01 0.01 0.12"/>
+					<mesh filename="package://desire_description/ros/meshes/head_v0/head.stl"/>
 				</geometry>
 			</collision>
