Commit message: head calibration for desire, robot modules in configuration file

File: desire_description/ros/calibration/desire.urdf.xacro (robot description, xacro)
@@ -3,18 +3,8 @@
 	<!-- common properties -->
 	<property name="M_PI" value="3.1415926535897931" />
-	<!-- torso reference positions -->
-	<property name="torso_lower_ref" value="-0.5470" />
-	<property name="torso_middle_ref" value="0.0247" />
-	<!-- head camera axis reference position -->
-	<property name="head_axis_ref" value="-3.14" />
-	<!-- arm reference positions -->
-	<property name="arm_1_ref" value="-2.8761" />
-	<property name="arm_2_ref" value="-0.1687" />
-	<property name="arm_3_ref" value="-0.0274" />
-	<property name="arm_4_ref" value="-1.7193" />
-	<property name="arm_5_ref" value="0.0342" />
-	<property name="arm_6_ref" value="-1.6959" />
-	<property name="arm_7_ref" value="1.8707" />
-	<!-- arm reference positions -->
+	<!-- head reference positions -->
+	<property name="head_pan_ref" value="0.55" />
+	<property name="head_tilt_ref" value="0.0" />
+	<!-- arm right reference positions -->
 	<property name="arm_1_ref" value="-2.8761" />
 	<property name="arm_2_ref" value="-0.1687" />

File: desire_description/ros/urdf/head_v0/head.urdf.xacro (robot description, xacro)
@@ -16,6 +16,6 @@
 			<axis xyz="0 0 1" />
 			<dynamics damping="0.1" />
-			<calibration rising="${head_axis_ref}" falling="${head_axis_ref}"/>
-			<limit effort="100" lower="-3.2" upper="0.1" velocity="0.5"/>
+			<calibration rising="${head_pan_ref}" falling="${head_pan_ref}"/>
+			<limit effort="100" lower="-0.7" upper="0.7" velocity="0.5"/>
 		</joint>
 		<link name="${name}_pan_link">
@@ -45,6 +45,6 @@
 			<axis xyz="0 0 1" />
 			<dynamics damping="0.1" />
-			<calibration rising="${head_axis_ref}" falling="${head_axis_ref}"/>
-			<limit effort="100" lower="-3.2" upper="0.1" velocity="0.5"/>
+			<calibration rising="${head_tilt_ref}" falling="${head_tilt_ref}"/>
+			<limit effort="100" lower="-0.25" upper="1.6" velocity="0.5"/>
 		</joint>
 		<link name="${name}_tilt_link">
