Commit message: sensors correct assuming y axis of head up

File: desire_description/ros/urdf/head_v0/head.urdf.xacro (robot description, xacro)
@@ -40,5 +40,5 @@
 		</link>
 		<joint name="${name}_tilt_joint" type="revolute">
-			<origin xyz="0 0 0" rpy="1.5708 0 0"/>
+			<origin xyz="0 0 0" rpy="-1.5708 0 0"/>
 			<parent link="${name}_pan_link"/>
 			<child link="${name}_tilt_link"/>
@@ -70,12 +70,13 @@
 		<!-- right camera -->
 		<xacro:cob_cameraone_v0 name="${name}_color_camera_r" parent="${name}_tilt_link">
-			<origin xyz="${cam_r_x} ${cam_r_y} ${cam_r_z-0.06}" rpy="${cam_r_roll} ${cam_r_pitch+1.5708} ${cam_r_yaw+3.14159}" />
+			<!--origin xyz="${cam_r_x} ${cam_r_y} ${cam_r_z-0.06}" rpy="${cam_r_roll} ${cam_r_pitch+1.5708} ${cam_r_yaw+3.14159}" /-->
+<origin xyz="${cam_r_x} ${cam_r_y} ${cam_r_z+0.06}" rpy="${cam_r_roll+3.14159} ${cam_r_pitch-1.5708} ${cam_r_yaw}" />
 		</xacro:cob_cameraone_v0>
 		<!-- left camera -->
-		<xacro:cob_cameraone_v0 name="${name}_color_camera_l" parent="${name}_tilt_link">
+		<xacro:cob_cameraone_v0 name="${name}_color_camera_l" parent="${name}_color_camera_r_link">
 			<origin xyz="${cam_l_x-0.12} ${cam_l_y} ${cam_l_z}" rpy="${cam_l_roll} ${cam_l_pitch} ${cam_l_yaw}" />
 		</xacro:cob_cameraone_v0>
 		<!-- tof -->
-		<xacro:cob_tof_v0 name="${name}_tof" parent="${name}_tilt_link">
+		<xacro:cob_tof_v0 name="${name}_tof" parent="${name}_color_camera_r_link">
 			<origin xyz="${tof_x-0.06} ${tof_y} ${tof_z}" rpy="${tof_roll} ${tof_pitch} ${tof_yaw}" />
 		</xacro:cob_tof_v0>

Commit message: corrected axes and wheel hubs

File: desire_description/ros/urdf/head_v0/head.urdf.xacro (robot description, xacro)
@@ -40,5 +40,5 @@
 		</link>
 		<joint name="${name}_tilt_joint" type="revolute">
-			<origin xyz="0 0 0" rpy="-1.5708 0 0"/>
+			<origin xyz="0 0 0" rpy="1.5708 0 0"/>
 			<parent link="${name}_pan_link"/>
 			<child link="${name}_tilt_link"/>
@@ -70,6 +70,6 @@
 		<!-- right camera -->
 		<xacro:cob_cameraone_v0 name="${name}_color_camera_r" parent="${name}_tilt_link">
-			<!--origin xyz="${cam_r_x} ${cam_r_y} ${cam_r_z-0.06}" rpy="${cam_r_roll} ${cam_r_pitch+1.5708} ${cam_r_yaw+3.14159}" /-->
-<origin xyz="${cam_r_x} ${cam_r_y} ${cam_r_z+0.06}" rpy="${cam_r_roll+3.14159} ${cam_r_pitch-1.5708} ${cam_r_yaw}" />
+			<!--origin xyz="${cam_r_x} ${cam_r_y} ${cam_r_z-0.06}" rpy="${cam_r_roll} ${cam_r_pitch+1.5708} ${cam_r_yaw+3.14159}"{cam_r_roll-3.14159} /-->
+<origin xyz="${cam_r_x} ${cam_r_y} ${cam_r_z-0.06}" rpy="${cam_r_roll} ${cam_r_pitch+1.5708} ${cam_r_yaw}" />
 		</xacro:cob_cameraone_v0>
 		<!-- left camera -->

Commit message: updated position limits from desire head

File: desire_description/ros/urdf/head_v0/head.urdf.xacro (robot description, xacro)
@@ -46,5 +46,5 @@
 			<dynamics damping="0.1" />
 			<calibration rising="${head_tilt_ref}" falling="${head_tilt_ref}"/>
-			<limit effort="100" lower="-0.25" upper="1.6" velocity="0.5"/>
+			<limit effort="100" lower="-0.25" upper="0.35" velocity="0.5"/>
 		</joint>
 		<link name="${name}_tilt_link">
