Commit message: added calib values for cam to neck

File: cob_description/ros/calibration/cob3-3.urdf.xacro (robot description, xacro)
@@ -21,10 +21,10 @@
 	<!-- camera calibration properties -->
 	<!-- hand eye calibration -->
-	<property name="cam_l_x" value="0" />
-	<property name="cam_l_y" value="0" />
-	<property name="cam_l_z" value="0" />
-	<property name="cam_l_roll" value="0" />
-	<property name="cam_l_pitch" value="0" />
-	<property name="cam_l_yaw" value="0" />
+	<property name="cam_l_x" value="-0.11572" />
+	<property name="cam_l_y" value="0.0285" />
+	<property name="cam_l_z" value="0.0112" />
+	<property name="cam_l_roll" value="-0.00158" />
+	<property name="cam_l_pitch" value="-0.00389" />
+	<property name="cam_l_yaw" value="0.00852" />
 	<!-- right to left calibration -->
 	<property name="cam_r_x" value="-0.00008029" />

File: cob_description/ros/urdf/head_v0/head.urdf.xacro (robot description, xacro)
@@ -42,13 +42,13 @@
 		<!-- left camera -->
 		<xacro:cob_prosilica_v0 name="${name}_color_camera_l" ros_topic="stereo/left" parent="${name}_axis_link">
-			<origin xyz="${cam_l_x} ${cam_l_y} ${cam_l_z-0.06}" rpy="${cam_l_roll} ${cam_l_pitch+1.5708} ${cam_l_yaw+3.14159}" />
+			<origin xyz="${cam_l_x} ${cam_l_y} ${cam_l_z+0.06}" rpy="${cam_l_roll} ${cam_l_pitch+1.5708} ${cam_l_yaw+3.14159}" />
 		</xacro:cob_prosilica_v0>
 		<!-- right camera -->
 		<xacro:cob_prosilica_v0 name="${name}_color_camera_r" ros_topic="stereo/right" parent="${name}_color_camera_l_link">
-			<origin xyz="${cam_r_x-0.12} ${cam_r_y} ${cam_r_z}" rpy="${cam_r_roll} ${cam_r_pitch} ${cam_r_yaw}" />
+			<origin xyz="${cam_r_x+0.12} ${cam_r_y} ${cam_r_z}" rpy="${cam_r_roll} ${cam_r_pitch} ${cam_r_yaw}" />
 		</xacro:cob_prosilica_v0>
 		<!-- cam3d -->
 		<xacro:cob_kinect_v0 name="${name}_cam3d" ros_topic="cam3d/depth/points1" parent="${name}_color_camera_l_link">
-			<origin xyz="${cam3d_x-0.06} ${cam3d_y} ${cam3d_z}" rpy="${cam3d_roll} ${cam3d_pitch} ${cam3d_yaw}" />
+			<origin xyz="${cam3d_x+0.06} ${cam3d_y} ${cam3d_z}" rpy="${cam3d_roll} ${cam3d_pitch} ${cam3d_yaw}" />
 		</xacro:cob_kinect_v0>
 		<!-- extensions -->
