Commit message: fixed bug with xyz values

File: cob_description/ros/urdf/head_v3/head.urdf.xacro (robot description, xacro)
@@ -42,5 +42,5 @@
 		<!-- left camera -->
 		<xacro:cob_prosilica_v0 name="${name}_color_camera_l" ros_topic="stereo/left" parent="${name}_axis_link">
-			<origin xyz="${cam_l_x} ${cam_l_y} ${cam_l_z}-0.06" rpy="${cam_l_roll} ${cam_l_pitch}-1.5708 ${cam_l_yaw}" />
+			<origin xyz="${cam_l_x} ${cam_l_y} ${cam_l_z-0.06}" rpy="${cam_l_roll} ${cam_l_pitch-1.5708} ${cam_l_yaw}" />
 		</xacro:cob_prosilica_v0>
 		<!-- right camera -->
