Commit message: fix collision problem with floor: lift collision base_footprint

File: cob_description/robots/cob3-3.urdf.xacro (robot description, xacro)
@@ -7,21 +7,21 @@
   <!-- The following included files set up definitions of parts of the robot body -->
   <!-- misc common stuff? -->
-  <include filename="$(find cob_description)/ros/urdf/common.xacro" />
+  <include filename="$(find cob_description)/urdf/common.xacro" />
   <!-- calibration -->
-  <include filename="$(find cob_description)/ros/calibration/cob3-3.urdf.xacro" />
+  <include filename="$(find cob_description)/calibration/cob3-3.urdf.xacro" />
   <!-- base -->
-  <include filename="$(find cob_description)/ros/urdf/base_v1/base.urdf.xacro" />	<!-- new version; platform_controller and platform_navigation not yet working -->
+  <include filename="$(find cob_description)/urdf/base/base.urdf.xacro" />	<!-- new version; platform_controller and platform_navigation not yet working -->
   <!-- torso -->
-  <include filename="$(find cob_description)/ros/urdf/torso_v1/torso.urdf.xacro" />
+  <include filename="$(find cob_description)/urdf/torso_v1/torso.urdf.xacro" />
   <!-- head -->
-  <include filename="$(find cob_description)/ros/urdf/head_v3/head.urdf.xacro" />
+  <include filename="$(find cob_description)/urdf/head_v3/head.urdf.xacro" />
   <!-- arm -->
-  <include filename="$(find cob_description)/ros/urdf/lbr_v0/lbr.urdf.xacro" />
+  <include filename="$(find cob_description)/urdf/lbr/lbr.urdf.xacro" />
   <!-- sdh -->
-  <include filename="$(find cob_description)/ros/urdf/sdh_v0/sdh.urdf.xacro" />
+  <include filename="$(find schunk_description)/urdf/sdh/sdh.urdf.xacro" />
   <!-- generic simulator_gazebo plugins for starting mechanism control, ros time, ros battery -->
-  <include filename="$(find cob_description)/ros/gazebo/gazebo.urdf.xacro" />
+  <include filename="$(find cob_description)/gazebo/gazebo.urdf.xacro" />
   <!-- materials for visualization -->
-  <include filename="$(find cob_description)/ros/urdf/materials.urdf.xacro" />
+  <include filename="$(find cob_description)/urdf/materials.urdf.xacro" />
   <!-- Now we can start using the macros included above to define the actual cob -->
   <!-- The first use of a macro.  This one was defined in base.urdf.xacro above.
@@ -32,5 +32,5 @@
        the origin block defines where the component is w.r.t its parent (in this case the parent
        is the world frame). For more, see http://www.ros.org/wiki/xacro -->
-  <xacro:cob_base_v1 name="base"/>	<!--with new collision_model, but no platform_controller available yet-->
+  <xacro:cob_base name="base"/>	<!--with new collision_model, but no platform_controller available yet-->
   <xacro:cob_torso_v1 name="torso" parent="base_link">
     <origin xyz="0.155 0 0.892" rpy="1.5708 0 0" />

File: cob_description/urdf/base/base.urdf.xacro (robot description, xacro)
@@ -168,5 +168,5 @@
       </visual>
       <collision>
-        <origin xyz="0 0 0" rpy="0 0 0" />
+        <origin xyz="0 0 0.1" rpy="0 0 0" />
         <geometry>
           <box size="0.001 0.001 0.001" />
