Commit message: restructured icob_description

File: icob_description/urdf/base_icob/base_icob.urdf.xacro (robot description, xacro)
@@ -4,9 +4,12 @@
        xmlns:interface="http://playerstage.sourceforge.net/gazebo/xmlschema/#interface"
        xmlns:xacro="http://ros.org/wiki/xacro">
-  <include filename="$(find cob_description)/ros/urdf/base_v0/base.gazebo.xacro" />
-  <include filename="$(find cob_description)/ros/urdf/base_v0/base.transmission.xacro" />
-  <include filename="$(find cob_description)/ros/urdf/sensors/kinect.urdf.xacro" />
+  <!-- fxm: this is the base.urdf.xacro for icob from old repository structure, why did it use base_v0 although it was named base_v1?	-->
+  <!--include filename="$(find cob_description)/urdf/base_v0/base.gazebo.xacro" />
+  <include filename="$(find cob_description)/urdf/base_v0/base.transmission.xacro" /-->
+  <include filename="$(find icob_description)/urdf/base_icob/base_icob.gazebo.xacro" />
+  <include filename="$(find icob_description)/urdf/base_icob/base_icob.transmission.xacro" />
   <!-- modify here for test -->
-  <include filename="$(find cob_description)/ros/urdf/sensors/sick_s300_laser.urdf.xacro"/>
+  <!--  <include filename="$(find cob_description)/ros/urdf/sensors/kinect.urdf.xacro" />		-->
+  <include filename="$(find cob_description)/urdf/sensors/sick_s300_laser.urdf.xacro"/>
   <!-- DATA SOURCES -->
   <!-- all link offsets, CG, limits are obtained from Function Engineering spreadsheet 090224_link_data.xls unless stated otherwise -->
@@ -41,5 +44,5 @@
   <!--           wheel                                      -->
   <!--                                                      -->
-  <xacro:macro name="cob_wheel_v0" params="suffix parent reflect">
+  <xacro:macro name="cob_wheel" params="suffix parent reflect">
     <joint name="${parent}_${suffix}_wheel_joint" type="continuous">
       <axis xyz="0 1 0" />
@@ -74,9 +77,9 @@
     </link>
     <!-- extensions -->
-    <xacro:cob_wheel_gazebo_v0 parent="${parent}" suffix="${suffix}" />
-    <xacro:cob_wheel_transmission_v0 parent="${parent}" suffix="${suffix}" reflect="${reflect}" />
+    <xacro:cob_wheel_gazebo parent="${parent}" suffix="${suffix}" />
+    <xacro:cob_wheel_transmission parent="${parent}" suffix="${suffix}" reflect="${reflect}" />
   </xacro:macro>
   <!-- Macro for Caster hub only -->
-  <xacro:macro name="cob_caster_hub_v0" params="suffix parent *origin ref_position" >
+  <xacro:macro name="cob_caster_hub" params="suffix parent *origin ref_position" >
     <joint name="${suffix}_rotation_joint" type="continuous">
       <axis xyz="0 0 1" />
@@ -114,19 +117,19 @@
     </link>
     <!-- extensions -->
-    <xacro:cob_caster_transmission_v0 suffix="${suffix}" />
-  </xacro:macro>
-  <xacro:macro name="cob_caster_v0" params="suffix parent *origin ref_position">
-    <xacro:cob_caster_hub_v0 parent="${parent}" suffix="${suffix}_caster"
+    <xacro:cob_caster_transmission suffix="${suffix}" />
+  </xacro:macro>
+  <xacro:macro name="cob_caster" params="suffix parent *origin ref_position">
+    <xacro:cob_caster_hub parent="${parent}" suffix="${suffix}_caster"
                              ref_position="${ref_position}" >
       <insert_block name="origin" />
-    </xacro:cob_caster_hub_v0>
+    </xacro:cob_caster_hub>
     <!-- wheel macros -->
     <!--xacro:cob_wheel_v0 parent="${suffix}_caster" suffix="l" reflect="1" /--> <!--### modified by jie ###-->
-    <xacro:cob_wheel_v0 parent="${suffix}_caster" suffix="r" reflect="-1" />
+    <xacro:cob_wheel parent="${suffix}_caster" suffix="r" reflect="-1" />
     <!-- extensions -->
-    <xacro:cob_caster_gazebo_v0 suffix="${suffix}" />
+    <xacro:cob_caster_gazebo suffix="${suffix}" />
   </xacro:macro>
   <!-- The xacro macro xacro:cob_base contains: base, casters and wheels -->
-  <xacro:macro name="icob_base_v1" params="name">
+  <xacro:macro name="base_icob" params="name">
   <link name="${name}_link">
       <inertial>
@@ -139,5 +142,5 @@
         <origin xyz="0 0 0.045" rpy="${M_PI/2} 0 0" />
         <geometry>
-          <mesh filename="package://icob_description/ros/meshes/base_v1/base.stl"/>
+          <mesh filename="package://icob_description/meshes/base_icob/base_icob.stl"/>
           <!--box size="${base_size_x} ${base_size_y} ${base_collision_size_z}" /-->
         </geometry>
@@ -148,5 +151,5 @@
         <geometry>
 		  <!--box size="0.001 0.001 0.001" /-->
-	      <mesh filename="package://icob_description/ros/meshes/base_v1/base.stlb"/>
+	      <mesh filename="package://icob_description/meshes/base_icob/base_icob.stlb"/>
           <!--box size="${base_size_x} ${base_size_y} ${base_collision_size_z}" /-->
         </geometry>
@@ -185,30 +188,26 @@
     <!--modify here for test: front,base and top lasers -->
     <!-- base laser front -->
-    <xacro:sick_s300_laser_v0 name="${name}_laser_front" parent="${name}" ros_topic="scan_front_raw" update_rate="10" min_angle="-2.3562" max_angle="2.3562" >
+    <xacro:sick_s300_laser name="${name}_laser_front" parent="${name}" ros_topic="scan_front_raw" update_rate="10" min_angle="-2.3562" max_angle="2.3562" >
       <origin xyz="${base_laser_x} ${-base_laser_y} ${base_laser_z}" rpy="0 0 ${-M_PI/4}" />
-    </xacro:sick_s300_laser_v0>
+    </xacro:sick_s300_laser>
     <!-- base laser back -->
-    <xacro:sick_s300_laser_v0 name="${name}_laser_rear" parent="${name}" ros_topic="scan_rear_raw" update_rate="10" min_angle="-2.3562" max_angle="2.3562" >
+    <xacro:sick_s300_laser name="${name}_laser_rear" parent="${name}" ros_topic="scan_rear_raw" update_rate="10" min_angle="-2.3562" max_angle="2.3562" >
       <origin xyz="${-base_laser_x} ${base_laser_y} ${base_laser_z}" rpy="0 0 ${3*M_PI/4}" />
-    </xacro:sick_s300_laser_v0>
+    </xacro:sick_s300_laser>
     <!-- all four caster macros -->
-    <xacro:cob_caster_v0 suffix="fl" parent="${name}_link" ref_position="${cal_caster_fl - M_PI/4}" >
+    <xacro:cob_caster suffix="fl" parent="${name}_link" ref_position="${cal_caster_fl - M_PI/4}" >
       <origin xyz="${caster_offset_x} ${caster_offset_y2} ${caster_offset_z}" rpy="0 0 0" />
-    </xacro:cob_caster_v0>
-    <xacro:cob_caster_v0 suffix="fr" parent="${name}_link" ref_position="${cal_caster_fr - M_PI/4}" >
+    </xacro:cob_caster>
+    <xacro:cob_caster suffix="fr" parent="${name}_link" ref_position="${cal_caster_fr - M_PI/4}" >
       <origin xyz="${caster_offset_x} ${-caster_offset_y1} ${caster_offset_z}" rpy="0 0 0" />
-    </xacro:cob_caster_v0>
-    <xacro:cob_caster_v0 suffix="bl" parent="${name}_link" ref_position="${cal_caster_bl - M_PI / 4 + M_PI}" >
+    </xacro:cob_caster>
+    <xacro:cob_caster suffix="bl" parent="${name}_link" ref_position="${cal_caster_bl - M_PI / 4 + M_PI}" >
       <origin xyz="${-caster_offset_x} ${caster_offset_y1} ${caster_offset_z}" rpy="0 0 0" />
-    </xacro:cob_caster_v0>
-    <xacro:cob_caster_v0 suffix="br" parent="${name}_link" ref_position="${cal_caster_br - M_PI / 4 + M_PI}"  >
+    </xacro:cob_caster>
+    <xacro:cob_caster suffix="br" parent="${name}_link" ref_position="${cal_caster_br - M_PI / 4 + M_PI}"  >
       <origin xyz="${-caster_offset_x} ${-caster_offset_y2} ${caster_offset_z}" rpy="0 0 0" />
-    </xacro:cob_caster_v0>
-<!-- cam3d -->
-   <xacro:cob_kinect_v0 name="${name}_cam3d" ros_topic="cam3d/depth" parent="${name}_link">
-                        <origin xyz="0.51 0.12 0.27" rpy="-1.57 0 -1.57" />
-                </xacro:cob_kinect_v0>
+    </xacro:cob_caster>
     <!-- gazebo extensions -->
-    <xacro:cob_base_gazebo_v0 name="${name}" />
+    <xacro:cob_base_gazebo name="${name}" />
   </xacro:macro>
 </robot>
