Commit message: fix icob urdf

File: icob_description/urdf/base/base.urdf.xacro (robot description, xacro)
@@ -4,9 +4,9 @@
        xmlns:interface="http://playerstage.sourceforge.net/gazebo/xmlschema/#interface"
        xmlns:xacro="http://ros.org/wiki/xacro">
-  <include filename="$(find cob_description)/ros/urdf/base_v0/base.gazebo.xacro" />
-  <include filename="$(find cob_description)/ros/urdf/base_v0/base.transmission.xacro" />
-  <include filename="$(find cob_description)/ros/urdf/sensors/kinect.urdf.xacro" />
-  <!-- modify here for test -->
-  <include filename="$(find cob_description)/ros/urdf/sensors/sick_s300_laser.urdf.xacro"/>
+  <include filename="$(find cob_description)/urdf/base/base.gazebo.xacro" />
+  <include filename="$(find cob_description)/urdf/base/base.transmission.xacro" />
+  <!-- sensors -->
+  <include filename="$(find cob_description)/urdf/sensors/kinect.urdf.xacro" />
+  <include filename="$(find cob_description)/urdf/sensors/sick_s300_laser.urdf.xacro"/>
   <!-- DATA SOURCES -->
   <!-- all link offsets, CG, limits are obtained from Function Engineering spreadsheet 090224_link_data.xls unless stated otherwise -->
@@ -41,5 +41,5 @@
   <!--           wheel                                      -->
   <!--                                                      -->
-  <xacro:macro name="cob_wheel_v0" params="suffix parent reflect">
+  <xacro:macro name="cob_wheel" params="suffix parent reflect">
     <joint name="${parent}_${suffix}_wheel_joint" type="continuous">
       <axis xyz="0 1 0" />
@@ -61,5 +61,4 @@
         <origin xyz="0 0 0" rpy="${M_PI/2} 0 0" />
         <geometry>
-          <!--mesh filename="package://cob_description/ros/meshes/base_v0/pr2_wheel.stl" /-->
           <cylinder radius="${wheel_radius}" length="${wheel_length}" />
         </geometry>
@@ -74,9 +73,9 @@
     </link>
     <!-- extensions -->
-    <xacro:cob_wheel_gazebo_v0 parent="${parent}" suffix="${suffix}" />
-    <xacro:cob_wheel_transmission_v0 parent="${parent}" suffix="${suffix}" reflect="${reflect}" />
+    <xacro:cob_wheel_gazebo parent="${parent}" suffix="${suffix}" />
+    <xacro:cob_wheel_transmission parent="${parent}" suffix="${suffix}" reflect="${reflect}" />
   </xacro:macro>
   <!-- Macro for Caster hub only -->
-  <xacro:macro name="cob_caster_hub_v0" params="suffix parent *origin ref_position" >
+  <xacro:macro name="cob_caster_hub" params="suffix parent *origin ref_position" >
     <joint name="${suffix}_rotation_joint" type="continuous">
       <axis xyz="0 0 1" />
@@ -100,5 +99,5 @@
 		<origin xyz="0 0 0.002" rpy="0.0 0.0 0.0" />
         <geometry>
-          <!--mesh filename="package://cob_description/ros/meshes/base_v0/caster.stl" /-->  <!--modified by jie-->
+          <!--mesh filename="package://cob_description/meshes/base/caster.stl" /-->  <!--modified by jie-->
           <!--box size="0.192 0.164 0.013" /-->
 		  <box size="0.001 0.001 0.001" />
@@ -114,30 +113,30 @@
     </link>
     <!-- extensions -->
-    <xacro:cob_caster_transmission_v0 suffix="${suffix}" />
-  </xacro:macro>
-  <xacro:macro name="cob_caster_v0" params="suffix parent *origin ref_position">
-    <xacro:cob_caster_hub_v0 parent="${parent}" suffix="${suffix}_caster"
+    <xacro:cob_caster_transmission suffix="${suffix}" />
+  </xacro:macro>
+  <xacro:macro name="cob_caster" params="suffix parent *origin ref_position">
+    <xacro:cob_caster_hub parent="${parent}" suffix="${suffix}_caster"
                              ref_position="${ref_position}" >
       <insert_block name="origin" />
-    </xacro:cob_caster_hub_v0>
+    </xacro:cob_caster_hub>
     <!-- wheel macros -->
-    <!--xacro:cob_wheel_v0 parent="${suffix}_caster" suffix="l" reflect="1" /--> <!--### modified by jie ###-->
-    <xacro:cob_wheel_v0 parent="${suffix}_caster" suffix="r" reflect="-1" />
+    <!--xacro:cob_wheel parent="${suffix}_caster" suffix="l" reflect="1" /--> <!--### modified by jie ###-->
+    <xacro:cob_wheel parent="${suffix}_caster" suffix="r" reflect="-1" />
     <!-- extensions -->
-    <xacro:cob_caster_gazebo_v0 suffix="${suffix}" />
+    <xacro:cob_caster_gazebo suffix="${suffix}" />
   </xacro:macro>
   <!-- The xacro macro xacro:cob_base contains: base, casters and wheels -->
-  <xacro:macro name="icob_base_v1" params="name">
+  <xacro:macro name="icob_base" params="name">
   <link name="${name}_link">
       <inertial>
         <mass value="${base_mass}" />
-        <origin xyz="${base_cg_x} ${base_cg_y} ${base_cg_z}" />
+        <origin xyz="0 0 0" />
         <inertia ixx="5.652232699207" ixy="-0.009719934438" ixz="1.293988226423"
                  iyy="5.669473158652" iyz="-0.007379583694" izz="3.683196351726" />
       </inertial>
       <visual>
-        <origin xyz="0 0 0.045" rpy="${M_PI/2} 0 0" />
-        <geometry>
-          <mesh filename="package://icob_description/ros/meshes/base_v1/base.stl"/>
+        <origin xyz="0 0 0.045" rpy="${M_PI/2} 0 0" />  <!--TODO: fix this in stl orientation not in urdf -->
+        <geometry>
+          <mesh filename="package://icob_description/meshes/base/base.stl"/>
           <!--box size="${base_size_x} ${base_size_y} ${base_collision_size_z}" /-->
         </geometry>
@@ -145,8 +144,8 @@
       </visual>
       <collision>
-        <origin xyz="0 0 0.045" rpy="${M_PI/2} 0 0" />
+        <origin xyz="0 0 0.045" rpy="${M_PI/2} 0 0" />  <!--TODO: fix this in stl orientation not in urdf -->
         <geometry>
 		  <!--box size="0.001 0.001 0.001" /-->
-	      <mesh filename="package://icob_description/ros/meshes/base_v1/base.stlb"/>
+	      <mesh filename="package://icob_description/meshes/base/base.stlb"/>
           <!--box size="${base_size_x} ${base_size_y} ${base_collision_size_z}" /-->
         </geometry>
@@ -170,7 +169,5 @@
       </visual>
       <collision>
-        <!-- represent base collision with a simple rectangular model, positioned by base_size_z s.t. top
-             surface of the collision box matches the top surface of the PR2 base -->
-        <origin xyz="0 0 ${0.051+base_collision_size_z/2}" rpy="0 0 0" />
+        <origin xyz="0 0 0.1" rpy="0 0 0" />
         <geometry>
           <box size="0.001 0.001 0.001" />
@@ -188,27 +185,27 @@
       <origin xyz="${base_laser_x} ${-base_laser_y} ${base_laser_z}" rpy="0 0 ${-M_PI/4}" />
     </xacro:sick_s300_laser_v0>
-    <!-- base laser back -->
+    <!-- base laser rear -->
     <xacro:sick_s300_laser_v0 name="${name}_laser_rear" parent="${name}" ros_topic="scan_rear_raw" update_rate="10" min_angle="-2.3562" max_angle="2.3562" >
       <origin xyz="${-base_laser_x} ${base_laser_y} ${base_laser_z}" rpy="0 0 ${3*M_PI/4}" />
     </xacro:sick_s300_laser_v0>
     <!-- all four caster macros -->
-    <xacro:cob_caster_v0 suffix="fl" parent="${name}_link" ref_position="${cal_caster_fl - M_PI/4}" >
+    <xacro:cob_caster suffix="fl" parent="${name}_link" ref_position="${cal_caster_fl - M_PI/4}" >
       <origin xyz="${caster_offset_x} ${caster_offset_y2} ${caster_offset_z}" rpy="0 0 0" />
-    </xacro:cob_caster_v0>
-    <xacro:cob_caster_v0 suffix="fr" parent="${name}_link" ref_position="${cal_caster_fr - M_PI/4}" >
+    </xacro:cob_caster>
+    <xacro:cob_caster suffix="fr" parent="${name}_link" ref_position="${cal_caster_fr - M_PI/4}" >
       <origin xyz="${caster_offset_x} ${-caster_offset_y1} ${caster_offset_z}" rpy="0 0 0" />
-    </xacro:cob_caster_v0>
-    <xacro:cob_caster_v0 suffix="bl" parent="${name}_link" ref_position="${cal_caster_bl - M_PI / 4 + M_PI}" >
+    </xacro:cob_caster>
+    <xacro:cob_caster suffix="bl" parent="${name}_link" ref_position="${cal_caster_bl - M_PI / 4 + M_PI}" >
       <origin xyz="${-caster_offset_x} ${caster_offset_y1} ${caster_offset_z}" rpy="0 0 0" />
-    </xacro:cob_caster_v0>
-    <xacro:cob_caster_v0 suffix="br" parent="${name}_link" ref_position="${cal_caster_br - M_PI / 4 + M_PI}"  >
+    </xacro:cob_caster>
+    <xacro:cob_caster suffix="br" parent="${name}_link" ref_position="${cal_caster_br - M_PI / 4 + M_PI}"  >
       <origin xyz="${-caster_offset_x} ${-caster_offset_y2} ${caster_offset_z}" rpy="0 0 0" />
-    </xacro:cob_caster_v0>
-<!-- cam3d -->
-   <xacro:cob_kinect_v0 name="${name}_cam3d" ros_topic="cam3d/depth" parent="${name}_link">
-                        <origin xyz="0.51 0.12 0.27" rpy="-1.57 0 -1.57" />
-                </xacro:cob_kinect_v0>
+    </xacro:cob_caster>
+   <!-- cam3d -->
+   <xacro:cob_kinect_v0 name="${name}_cam3d" ros_topic="cam3d" parent="${name}_link">
+      <origin xyz="0.51 0.12 0.27" rpy="-1.57 0 -1.57" />
+   </xacro:cob_kinect_v0>
     <!-- gazebo extensions -->
-    <xacro:cob_base_gazebo_v0 name="${name}" />
+    <xacro:cob_base_gazebo name="${name}" />
   </xacro:macro>
 </robot>
