Commit message: urdf structure change: tray can be calibrated now

File: cob_description/urdf/torso_v0/torso.gazebo.xacro (robot description, xacro)
@@ -5,8 +5,4 @@
        xmlns:xacro="http://ros.org/wiki/xacro">
 	<xacro:macro name="cob_torso_gazebo_v0" params="name">
-		<gazebo reference="${name}_tray_link">
-			<material>Gazebo/Green</material>
-			<turnGravityOff>false</turnGravityOff>
-		</gazebo>
 		<gazebo reference="${name}_lower_neck_pan_link">
 			<material>Gazebo/Blue</material>

File: cob_description/urdf/torso_v0/torso.transmission.xacro (robot description, xacro)
@@ -5,9 +5,4 @@
        xmlns:xacro="http://ros.org/wiki/xacro">
 	<xacro:macro name="cob_torso_transmission_v0" params="name">
-		<transmission name="${name}_tray_trans" type="pr2_mechanism_model/SimpleTransmission">
-			<actuator name="${name}_tray_motor"/>
-			<joint name="${name}_tray_joint"/>
-			<mechanicalReduction>1</mechanicalReduction>
-		</transmission>
 		<transmission name="${name}_lower_neck_pan_trans" type="pr2_mechanism_model/SimpleTransmission">
 			<actuator name="${name}_lower_neck_pan_motor"/>

File: cob_description/urdf/torso_v0/torso.urdf.xacro (robot description, xacro)
@@ -7,34 +7,4 @@
 	<include filename="$(find cob_description)/urdf/torso_v0/torso.transmission.xacro" />
 	<xacro:macro name="cob_torso_v0" params="name parent *origin">
-		<!-- joint between base_link and torso_tray_link -->
-		<joint name="${name}_tray_joint" type="revolute">
-			<origin xyz="0.2406 0.1900 0.7320" rpy="2.3561 0 0" />
-			<parent link="${parent}"/>
-			<child link="${name}_tray_link"/>
-			<axis xyz="0 0 1" />
-			<calibration rising="${torso_tray_ref}"/>
-			<dynamics damping="5.0" friction="0.5"/>
-			<limit effort="100" lower="-3.31612" upper="0.2" velocity="5"/>
-		</joint>
-		<link name="${name}_tray_link">
-			<inertial>
-				<origin xyz="0 0 0" rpy="0 0 0"/>
-				<mass value="0.1"/>
-				<inertia ixx="0.01" ixy="0" ixz="0" iyy="0.01" iyz="0" izz="0.01" />
-			</inertial>
-			<visual>
-				<origin xyz="0 0 0" rpy="0 0 0" />
-				<geometry>
-					<mesh filename="package://cob_description/meshes/torso_v0/tray.stl" />
-				</geometry>
-				<material name="Green" />
-			</visual>
-			<collision>
-				<origin xyz="0 0 0" rpy="0 0 0" />
-				<geometry>
-					<mesh filename="package://cob_description/meshes/torso_v0/tray_collision.stlb" />
-				</geometry>
-			</collision>
-		</link>
 		<!-- joint between base_link and torso_lower_neck_pan_link -->
 		<joint name="${name}_lower_neck_pan_joint" type="revolute">

File: cob_description/urdf/torso_v1/torso.gazebo.xacro (robot description, xacro)
@@ -5,8 +5,4 @@
        xmlns:xacro="http://ros.org/wiki/xacro">
 	<xacro:macro name="cob_torso_gazebo_v1" params="name">
-		<gazebo reference="${name}_tray_link">
-			<material>Gazebo/Green</material>
-			<turnGravityOff>false</turnGravityOff>
-		</gazebo>
 		<gazebo reference="${name}_lower_neck_tilt_link">
 			<material>Gazebo/Red</material>

File: cob_description/urdf/torso_v1/torso.transmission.xacro (robot description, xacro)
@@ -5,9 +5,4 @@
        xmlns:xacro="http://ros.org/wiki/xacro">
 	<xacro:macro name="cob_torso_transmission_v1" params="name">
-		<transmission name="${name}_tray_trans" type="pr2_mechanism_model/SimpleTransmission">
-			<actuator name="${name}_tray_motor"/>
-			<joint name="${name}_tray_joint"/>
-			<mechanicalReduction>1</mechanicalReduction>
-		</transmission>
 		<transmission name="${name}_lower_neck_tilt_trans" type="pr2_mechanism_model/SimpleTransmission">
 			<actuator name="${name}_lower_neck_tilt_motor"/>

File: cob_description/urdf/torso_v1/torso.urdf.xacro (robot description, xacro)
@@ -7,34 +7,4 @@
 	<include filename="$(find cob_description)/urdf/torso_v1/torso.transmission.xacro" />
 	<xacro:macro name="cob_torso_v1" params="name parent *origin">
-		<!-- joint between base_link and torso_tray_link -->
-		<joint name="${name}_tray_joint" type="revolute">
-			<origin xyz="0.2406 0.1900 0.7320" rpy="2.3561 0 0" />
-			<parent link="${parent}"/>
-			<child link="${name}_tray_link"/>
-			<axis xyz="0 0 1" />
-			<calibration rising="${torso_tray_ref}"/>
-			<dynamics damping="5.0" friction="0.5"/>
-			<limit effort="100" lower="-3.31612" upper="0.2" velocity="5"/>
-		</joint>
-		<link name="${name}_tray_link">
-			<inertial>
-				<origin xyz="0 0 0" rpy="0 0 0"/>
-				<mass value="0.1"/>
-				<inertia ixx="0.01" ixy="0" ixz="0" iyy="0.01" iyz="0" izz="0.01" />
-			</inertial>
-			<visual>
-				<origin xyz="0 0 0" rpy="0 0 0" />
-				<geometry>
-					<mesh filename="package://cob_description/meshes/torso_v0/tray.stl" />
-				</geometry>
-				<material name="Green" />
-			</visual>
-			<collision>
-				<origin xyz="0 0 0" rpy="0 0 0" />
-				<geometry>
-					<mesh filename="package://cob_description/meshes/torso_v0/tray_collision.stlb" />
-				</geometry>
-			</collision>
-		</link>
 		<!-- joint between base_link and torso_lower_neck_tilt_link -->
 		<joint name="${name}_lower_neck_tilt_joint" type="revolute">
