Commit message: read correct torso stl

File: cob_description/urdf/torso_v0/torso.urdf.xacro (robot description, xacro)
@@ -56,5 +56,5 @@
 				<origin xyz="0 0 0" rpy="0 0 0" />
 				<geometry>
-					<mesh filename="package://cob_description/meshes/torso_v0/lower_neck.stl" />
+					<mesh filename="package://cob_description/meshes/torso/lower_neck.stl" />
 				</geometry>
 				<material name="Red" />
@@ -63,5 +63,5 @@
 				<origin xyz="0 0 0" rpy="0 0 0" />
 				<geometry>
-					<mesh filename="package://cob_description/meshes/torso_v0/lower_neck_collision.stlb" />
+					<mesh filename="package://cob_description/meshes/torso/lower_neck_collision.stlb" />
 				</geometry>
 			</collision>
@@ -116,5 +116,5 @@
 				<origin xyz="0 0 0" rpy="0 0 0" />
 				<geometry>
-					<mesh filename="package://cob_description/meshes/torso_v0/upper_neck.stl" />
+					<mesh filename="package://cob_description/meshes/torso/upper_neck.stl" />
 				</geometry>
 				<material name="Grey" />
@@ -123,5 +123,5 @@
 				<origin xyz="0 0 0" rpy="0 0 0" />
 				<geometry>
-					<mesh filename="package://cob_description/meshes/torso_v0/upper_neck_collision.stlb" />
+					<mesh filename="package://cob_description/meshes/torso/upper_neck_collision.stlb" />
 				</geometry>
 			</collision>
@@ -142,5 +142,5 @@
 				<origin xyz="0 0 0" rpy="0 0 0" />
 				<geometry>
-					<mesh filename="package://cob_description/meshes/torso_v0/head_cover.stl" />
+					<mesh filename="package://cob_description/meshes/torso/head_cover.stl" />
 				</geometry>
 				<material name="Blue" />
@@ -149,5 +149,5 @@
 				<origin xyz="0 0 0" rpy="0 0 0" />
 				<geometry>
-					<mesh filename="package://cob_description/meshes/torso_v0/head_cover_collision.stlb" />
+					<mesh filename="package://cob_description/meshes/torso/head_cover_collision.stlb" />
 				</geometry>
 			</collision>

File: cob_description/urdf/torso_v1/torso.urdf.xacro (robot description, xacro)
@@ -26,5 +26,5 @@
 				<origin xyz="0 0 0" rpy="3.14 0 0" />
 				<geometry>
-					<mesh filename="package://cob_description/meshes/torso_v0/lower_neck.stl" />
+					<mesh filename="package://cob_description/meshes/torso/lower_neck.stl" />
 				</geometry>
 				<material name="Red" />
@@ -33,5 +33,5 @@
 				<origin xyz="0 0 0" rpy="3.14 0 0" />
 				<geometry>
-					<mesh filename="package://cob_description/meshes/torso_v0/lower_neck_collision.stlb" />
+					<mesh filename="package://cob_description/meshes/torso/lower_neck_collision.stlb" />
 				</geometry>
 			</collision>
@@ -86,5 +86,5 @@
 				<origin xyz="0 0 0" rpy="3.1415926 0 0" />
 				<geometry>
-					<mesh filename="package://cob_description/meshes/torso_v0/upper_neck.stl" />
+					<mesh filename="package://cob_description/meshes/torso/upper_neck.stl" />
 				</geometry>
 				<material name="Grey" />
@@ -93,5 +93,5 @@
 				<origin xyz="0 0 0" rpy="3.1415926 0 0" />
 				<geometry>
-					<mesh filename="package://cob_description/meshes/torso_v0/upper_neck_collision.stlb" />
+					<mesh filename="package://cob_description/meshes/torso/upper_neck_collision.stlb" />
 				</geometry>
 			</collision>
@@ -112,5 +112,5 @@
 				<origin xyz="0 0 0" rpy="0 0 0" />
 				<geometry>
-					<mesh filename="package://cob_description/meshes/torso_v0/head_cover.stl" />
+					<mesh filename="package://cob_description/meshes/torso/head_cover.stl" />
 				</geometry>
 				<material name="Blue" />
@@ -119,5 +119,5 @@
 				<origin xyz="0 0 0" rpy="0 0 0" />
 				<geometry>
-					<mesh filename="package://cob_description/meshes/torso_v0/head_cover_collision.stlb" />
+					<mesh filename="package://cob_description/meshes/torso/head_cover_collision.stlb" />
 				</geometry>
 			</collision>

Commit message: limit torso pan and tilt joints

File: cob_description/urdf/torso_v0/torso.urdf.xacro (robot description, xacro)
@@ -15,5 +15,5 @@
 			<calibration rising="${torso_lower_neck_pan_ref}"/>
 			<dynamics damping="25.0" friction="10.0"/>
-			<limit effort="24" lower="-${2*M_PI}" upper="${2*M_PI}" velocity="0.5"/>
+			<limit effort="24" lower="-0.2" upper="0.2" velocity="0.5"/>
 		</joint>
 		<link name="${name}_lower_neck_pan_link">
@@ -45,5 +45,5 @@
 			<dynamics damping="25.0" friction="10.0"/>
 			<calibration rising="${torso_lower_neck_tilt_ref}"/>
-			<limit effort="46" lower="-1.5" upper="1.5" velocity="0.5"/>
+			<limit effort="46" lower="-0.4" upper="0.4" velocity="0.5"/>
 		</joint>
 		<link name="${name}_lower_neck_tilt_link">
@@ -75,5 +75,5 @@
 			<dynamics damping="25.0" friction="10.0"/>
 			<calibration rising="${torso_upper_neck_pan_ref}"/>
-			<limit effort="4" lower="-${2*M_PI}" upper="${2*M_PI}" velocity="0.5"/>
+			<limit effort="4" lower="-0.2" upper="0.2" velocity="0.5"/>
 		</joint>
 		<link name="${name}_upper_neck_pan_link">
@@ -105,5 +105,5 @@
 			<dynamics damping="25.0" friction="10.0"/>
 			<calibration rising="${torso_upper_neck_tilt_ref}"/>
-			<limit effort="24" lower="-1.5" upper="1.5" velocity="0.5"/>
+			<limit effort="24" lower="-0.4" upper="0.4" velocity="0.5"/>
 		</joint>
 		<link name="${name}_upper_neck_tilt_link">

File: cob_description/urdf/torso_v1/torso.urdf.xacro (robot description, xacro)
@@ -15,5 +15,5 @@
 			<dynamics damping="25.0" friction="10.0"/>
 			<calibration rising="${torso_lower_neck_tilt_ref}"/>
-			<limit effort="41.4" lower="-${2*M_PI}" upper="${2*M_PI}" velocity="0.5"/>
+			<limit effort="41.4" lower="-0.25" upper="0.25" velocity="0.5"/>
 		</joint>
 		<link name="${name}_lower_neck_tilt_link">
@@ -45,5 +45,5 @@
 			<dynamics damping="25.0" friction="10.0"/>
 			<calibration rising="${torso_pan_ref}"/>
-			<limit effort="41.4" lower="-${2*M_PI}" upper="${2*M_PI}" velocity="0.5"/>
+			<limit effort="41.4" lower="-0.2" upper="0.2" velocity="0.5"/>
 		</joint>
 		<link name="${name}_pan_link">
@@ -75,5 +75,5 @@
 			<dynamics damping="25.0" friction="10.0"/>
 			<calibration rising="${torso_upper_neck_tilt_ref}"/>
-			<limit effort="41.4" lower="-${2*M_PI}" upper="${2*M_PI}" velocity="0.5"/>
+			<limit effort="41.4" lower="-0.4" upper="0.4" velocity="0.5"/>
 		</joint>
 		<link name="${name}_upper_neck_tilt_link">

Commit message: increased torso_v0 limits for the initialization of cob3-1

File: cob_description/urdf/torso_v0/torso.urdf.xacro (robot description, xacro)
@@ -15,5 +15,5 @@
 			<calibration rising="${torso_lower_neck_pan_ref}"/>
 			<dynamics damping="25.0" friction="10.0"/>
-			<limit effort="24" lower="-0.2" upper="0.2" velocity="0.5"/>
+			<limit effort="24" lower="-1.0" upper="1.0" velocity="0.5"/>
 		</joint>
 		<link name="${name}_lower_neck_pan_link">
@@ -75,5 +75,5 @@
 			<dynamics damping="25.0" friction="10.0"/>
 			<calibration rising="${torso_upper_neck_pan_ref}"/>
-			<limit effort="4" lower="-0.2" upper="0.2" velocity="0.5"/>
+			<limit effort="4" lower="-1.0" upper="1.0" velocity="0.5"/>
 		</joint>
 		<link name="${name}_upper_neck_pan_link">

Commit message: unified torso frames

File: cob_description/urdf/torso_v0/torso.urdf.xacro (robot description, xacro)
@@ -7,8 +7,21 @@
 	<include filename="$(find cob_description)/urdf/torso_v0/torso.transmission.xacro" />
 	<xacro:macro name="cob_torso_v0" params="name parent *origin">
+		<!-- joint between base_link and torso_base_link -->
+		<joint name="${name}_base_joint" type="fixed" >
+			<insert_block name="origin" />
+			<parent link="${parent}" />
+			<child link="${name}_base_link" />
+		</joint>
+		<link name="${name}_base_link">
+			<inertial>
+				<origin xyz="0 0 0" rpy="0 0 0"/>
+				<mass value="0.01"/>
+				<inertia ixx="1" ixy="0" ixz="0" iyy="1" iyz="0" izz="1" />
+			</inertial>
+		</link>
 		<!-- joint between base_link and torso_lower_neck_pan_link -->
 		<joint name="${name}_lower_neck_pan_joint" type="revolute">
-			<insert_block name="origin" />
-			<parent link="${parent}"/>
+			<origin xyz="0 0 0" rpy="0 0 0" />
+			<parent link="${name}_base_link"/>
 			<child link="${name}_lower_neck_pan_link"/>
 			<axis xyz="0 0 1" />

File: cob_description/urdf/torso_v1/torso.urdf.xacro (robot description, xacro)
@@ -19,17 +19,4 @@
 				<inertia ixx="1" ixy="0" ixz="0" iyy="1" iyz="0" izz="1" />
 			</inertial>
-			<visual>
-				<origin xyz="0 0 -0.00" rpy="0 0 0" />
-				<geometry>
-					<cylinder radius="0" length="0"/>
-				</geometry>
-                <material name="IPA/DarkGrey" />
-			</visual>
-			<collision>
-				<origin xyz="0 0 0" rpy="0 0 0" />
-				<geometry>
-					<box size="0 0 0"/>
-				</geometry>
-			</collision>
 		</link>
 		<!-- joint between base_link and torso_lower_neck_tilt_link -->

Commit message: fixed torso joint limits

File: cob_description/urdf/torso_v0/torso.urdf.xacro (robot description, xacro)
@@ -28,5 +28,5 @@
 			<calibration rising="${torso_lower_neck_pan_ref}"/>
 			<dynamics damping="25.0" friction="10.0"/>
-			<limit effort="24" lower="-1.0" upper="1.0" velocity="0.5"/>
+			<limit effort="24" lower="-0.1" upper="0.1" velocity="0.5"/>
 		</joint>
 		<link name="${name}_lower_neck_pan_link">
@@ -58,5 +58,5 @@
 			<dynamics damping="25.0" friction="10.0"/>
 			<calibration rising="${torso_lower_neck_tilt_ref}"/>
-			<limit effort="46" lower="-0.4" upper="0.4" velocity="0.5"/>
+			<limit effort="46" lower="-0.25" upper="0.25" velocity="0.5"/>
 		</joint>
 		<link name="${name}_lower_neck_tilt_link">
@@ -88,5 +88,5 @@
 			<dynamics damping="25.0" friction="10.0"/>
 			<calibration rising="${torso_upper_neck_pan_ref}"/>
-			<limit effort="4" lower="-1.0" upper="1.0" velocity="0.5"/>
+			<limit effort="4" lower="-0.2" upper="0.2" velocity="0.5"/>
 		</joint>
 		<link name="${name}_upper_neck_pan_link">
@@ -118,5 +118,5 @@
 			<dynamics damping="25.0" friction="10.0"/>
 			<calibration rising="${torso_upper_neck_tilt_ref}"/>
-			<limit effort="24" lower="-0.4" upper="0.4" velocity="0.5"/>
+			<limit effort="24" lower="-0.3" upper="0.3" velocity="0.5"/>
 		</joint>
 		<link name="${name}_upper_neck_tilt_link">

Commit message: optimize effort and joint limits + use visual mesh as collision for upper neck to give arem some more space

File: cob_description/urdf/torso_v0/torso.urdf.xacro (robot description, xacro)
@@ -25,5 +25,5 @@
       <calibration rising="${torso_lower_neck_pan_ref}"/>
       <dynamics damping="25.0" friction="10.0"/>
-      <limit effort="24" lower="-0.1" upper="0.1" velocity="0.5"/>
+      <limit effort="200" lower="-0.1" upper="0.1" velocity="0.5"/>
     </joint>
     <link name="${name}_lower_neck_pan_link">
@@ -55,5 +55,5 @@
       <dynamics damping="25.0" friction="10.0"/>
       <calibration rising="${torso_lower_neck_tilt_ref}"/>
-      <limit effort="46" lower="-0.25" upper="0.25" velocity="0.5"/>
+      <limit effort="200" lower="-0.26" upper="0.25" velocity="0.5"/>
     </joint>
     <link name="${name}_lower_neck_tilt_link">
@@ -85,5 +85,5 @@
       <dynamics damping="25.0" friction="10.0"/>
       <calibration rising="${torso_upper_neck_pan_ref}"/>
-      <limit effort="4" lower="-0.2" upper="0.2" velocity="0.5"/>
+      <limit effort="200" lower="-0.2" upper="0.2" velocity="0.5"/>
     </joint>
     <link name="${name}_upper_neck_pan_link">
@@ -115,5 +115,5 @@
       <dynamics damping="25.0" friction="10.0"/>
       <calibration rising="${torso_upper_neck_tilt_ref}"/>
-      <limit effort="24" lower="-0.3" upper="0.3" velocity="0.5"/>
+      <limit effort="200" lower="-0.21" upper="0.3" velocity="0.5"/>
     </joint>
     <link name="${name}_upper_neck_tilt_link">
@@ -133,5 +133,6 @@
         <origin xyz="0 0 0" rpy="0 0 0" />
         <geometry>
-          <mesh filename="package://cob_description/meshes/torso/upper_neck_collision.stl" />
+          <!--mesh filename="package://cob_description/meshes/torso/upper_neck_collision.stl" /-->
+          <mesh filename="package://cob_description/meshes/torso/upper_neck.stl" />
         </geometry>
       </collision>

File: cob_description/urdf/torso_v1/torso.urdf.xacro (robot description, xacro)
@@ -16,4 +16,6 @@
         <inertia ixx="1" ixy="0" ixz="0" iyy="1" iyz="0" izz="1" />
       </inertial>
+      <!--xacro:box_inertial x="0.01" y="0.01" z="0.01" mass="0.01" /-->
+      <!--xacro:default_inertial/-->
     </link>
     <!-- joint between base_link and torso_lower_neck_tilt_link -->
@@ -25,5 +27,6 @@
       <dynamics damping="25.0" friction="10.0"/>
       <calibration rising="${torso_lower_neck_tilt_ref}"/>
-      <limit effort="41.4" lower="-0.25" upper="0.25" velocity="0.5"/>
+      <limit effort="200.0" lower="-0.25" upper="0.21" velocity="0.5"/>
+      <!--safety_controller k_position="20" k_velocity="50" soft_lower_limit="${-0.25 + 0.01}" soft_upper_limit="${0.25 - 0.01}" /-->
     </joint>
     <link name="${name}_lower_neck_tilt_link">
@@ -33,4 +36,6 @@
         <inertia ixx="0.171118" ixy="0.002544" ixz="-0.000000" iyy="0.083077" iyz="0.000000" izz="0.120948" />
       </inertial>
+      <!--xacro:box_inertial x="0.197825" y="0.410127" z="0.418714" mass="6.209720" /-->   <!-- x,y,z values from bounding box -->
+      <!--xacro:default_inertial/-->
       <visual>
         <origin xyz="0 0 0" rpy="${M_PI} 0 0" />
@@ -55,5 +60,6 @@
       <dynamics damping="25.0" friction="10.0"/>
       <calibration rising="${torso_pan_ref}"/>
-      <limit effort="41.4" lower="-0.2" upper="0.2" velocity="0.5"/>
+      <limit effort="200.0" lower="-0.2" upper="0.2" velocity="0.5"/>
+      <!--safety_controller k_position="20" k_velocity="50" soft_lower_limit="${-0.2 + 0.01}" soft_upper_limit="${0.2 - 0.01}" /-->
     </joint>
     <link name="${name}_pan_link">
@@ -63,4 +69,6 @@
         <inertia ixx="0.200549" ixy="0.001322" ixz="-0.000000" iyy="0.123664" iyz="-0.000000" izz="0.104101" />
       </inertial>
+      <!--xacro:box_inertial x="0.01" y="0.01" z="0.01" mass="0.01" /-->
+      <!--xacro:default_inertial/-->
     </link>
     <!-- joint between torso_pan_link and torso_upper_neck_tilt_link -->
@@ -72,5 +80,6 @@
       <dynamics damping="25.0" friction="10.0"/>
       <calibration rising="${torso_upper_neck_tilt_ref}"/>
-      <limit effort="41.4" lower="-0.4" upper="0.4" velocity="0.5"/>
+      <limit effort="200.0" lower="-0.4" upper="0.36" velocity="0.5"/>
+      <!--safety_controller k_position="20" k_velocity="50" soft_lower_limit="${-0.4 + 0.01}" soft_upper_limit="${0.4 - 0.01}" /-->
     </joint>
     <link name="${name}_upper_neck_tilt_link">
@@ -80,4 +89,6 @@
         <inertia ixx="0.01" ixy="0" ixz="0" iyy="0.01" iyz="0" izz="0.01" />
       </inertial>
+      <!--xacro:box_inertial x="0.188249" y="0.359198" z="0.413754" mass="6.209720" /-->   <!-- x,y,z values from bounding box -->
+      <!--xacro:default_inertial/-->
       <visual>
         <origin xyz="0 0 0" rpy="${M_PI} 0 0" />
@@ -90,5 +101,6 @@
         <origin xyz="0 0 0" rpy="${M_PI} 0 0" />
         <geometry>
-          <mesh filename="package://cob_description/meshes/torso/upper_neck_collision.stl" />
+          <!--mesh filename="package://cob_description/meshes/torso/upper_neck_collision.stl" /-->
+          <mesh filename="package://cob_description/meshes/torso/upper_neck.stl" />
         </geometry>
       </collision>
@@ -106,4 +118,6 @@
         <inertia ixx="0.01" ixy="0" ixz="0" iyy="0.01" iyz="0" izz="0.01" />
       </inertial>
+      <!--xacro:box_inertial x="0.192076" y="0.264614" z="0.269999" mass="6.209720" /-->   <!-- x,y,z values from bounding box -->
+      <!--xacro:default_inertial/-->
       <visual>
         <origin xyz="0 0 0" rpy="0 0 0" />
