Commit message: Update desire_description

File: cob_description/urdf/sensors/tof.urdf.xacro (robot description, xacro)
@@ -5,5 +5,5 @@
        xmlns:xacro="http://playerstage.sourceforge.net/gazebo/xmlschema/#interface"
        name="LaserBlock">
-  <include filename="$(find cob_description)/ros/urdf/sensors/tof.gazebo.xacro" />
+  <include filename="$(find cob_description)/urdf/sensors/tof.gazebo.xacro" />
   <xacro:macro name="cob_tof_v0" params="name parent *origin ros_topic">
     <joint name="${name}_joint" type="fixed">

File: desire_description/urdf/base_desire/base.urdf.xacro (robot description, xacro)
@@ -4,12 +4,13 @@
        xmlns:interface="http://playerstage.sourceforge.net/gazebo/xmlschema/#interface"
        xmlns:xacro="http://ros.org/wiki/xacro">
-  <include filename="$(find desire_description)/ros/urdf/base_v0/base.gazebo.xacro" />
-  <include filename="$(find desire_description)/ros/urdf/base_v0/base.transmission.xacro" />
+  <include filename="$(find desire_description)/urdf/base_desire/base.gazebo.xacro" />
+  <include filename="$(find desire_description)/urdf/base_desire/base.transmission.xacro" />
   <!-- modify here for test -->
-  <include filename="$(find cob_description)/ros/urdf/sensors/sick_s300_laser.urdf.xacro"/>
+  <include filename="$(find cob_description)/urdf/sensors/sick_s300_laser.urdf.xacro"/>
   <!-- DATA SOURCES -->
   <!-- all link offsets, CG, limits are obtained from Function Engineering spreadsheet 090224_link_data.xls unless stated otherwise -->
   <!-- all link geometry sizes are obtained from Function provided CAD model unless stated otherwise -->
   <!-- all simplified collision geometry are hand approximated from CAD model, sometimes from respective bounding boxes -->
+  <property name="M_PI" value="3.1415926535897931" />
   <property name="caster_offset_x" value="0.235" />  <!--modify here-->
   <property name="caster_offset_y" value="0.185" />
@@ -58,5 +59,5 @@
         <origin xyz="0 0 0" rpy="0 0 0" />
         <geometry>
-          <mesh filename="package://cob_description/ros/meshes/base_v0/pr2_wheel.stl" />
+          <mesh filename="package://cob_description/meshes/base/pr2_wheel.stl" />
         </geometry>
         <material name="Wheel_${suffix}" />
@@ -95,5 +96,5 @@
         <origin xyz="0 0 0" rpy="0 0 0" />
         <geometry>
-          <mesh filename="$(find cob_description)/ros/meshes/base_v0/caster.stl" />
+          <mesh filename="$(find cob_description)/meshes/base/caster.stl" />
         </geometry>
         <material name="Green" />
@@ -121,5 +122,6 @@
   </xacro:macro>
   <!-- The xacro macro xacro:desire_base contains: base, casters and wheels -->
-  <xacro:macro name="desire_base_v0" params="name">
+  <!--xacro:macro name="desire_base_v0" params="name"-->
+  <xacro:macro name="desire_base" params="name">
   <link name="${name}_link">
       <inertial>
@@ -133,5 +135,5 @@
         <!-- modify here for test-->
         <geometry>
-          <mesh filename="package://desire_description/ros/meshes/base_v0/base.stl"/>
+          <mesh filename="package://desire_description/meshes/base_desire/base.stl"/>
         </geometry>
         <material name="Green"/>

File: desire_description/urdf/head_desire/head.gazebo.xacro (robot description, xacro)
@@ -4,11 +4,11 @@
        xmlns:interface="http://playerstage.sourceforge.net/gazebo/xmlschema/#interface"
        xmlns:xacro="http://ros.org/wiki/xacro">
-	<xacro:macro name="desire_head_gazebo_v0" params="name">
+	<xacro:macro name="head_desire_gazebo_v0" params="name">
 		<gazebo reference="${name}_axis1_link">
-			<material>Gazebo/Green</material>
+			<material>Gazebo/Blue</material>
 			<turnGravityOff>false</turnGravityOff>
 		</gazebo>
 		<gazebo reference="${name}_axis2_link">
-			<material>Gazebo/Green</material>
+			<material>Gazebo/Blue</material>
 			<turnGravityOff>false</turnGravityOff>
 		</gazebo>

File: desire_description/urdf/head_desire/head.transmission.xacro (robot description, xacro)
@@ -4,5 +4,5 @@
        xmlns:interface="http://playerstage.sourceforge.net/gazebo/xmlschema/#interface"
        xmlns:xacro="http://ros.org/wiki/xacro">
-	<xacro:macro name="desire_head_transmission_v0" params="name">
+	<xacro:macro name="head_desire_transmission_v0" params="name">
 		<transmission name="${name}_pan_trans" type="pr2_mechanism_model/SimpleTransmission">
 			<actuator name="${name}_pan_motor"/>

File: desire_description/urdf/head_desire/head.urdf.xacro (robot description, xacro)
@@ -4,9 +4,9 @@
        xmlns:interface="http://playerstage.sourceforge.net/gazebo/xmlschema/#interface"
        xmlns:xacro="http://ros.org/wiki/xacro">
-	<include filename="$(find desire_description)/ros/urdf/head_v0/head.gazebo.xacro" />
-	<include filename="$(find desire_description)/ros/urdf/head_v0/head.transmission.xacro" />
-	<include filename="$(find cob_description)/ros/urdf/sensors/prosilica.urdf.xacro" />
-	<include filename="$(find cob_description)/ros/urdf/sensors/tof.urdf.xacro" />
-	<xacro:macro name="desire_head_v0" params="name parent *origin">
+	<include filename="$(find desire_description)/urdf/head_desire/head.gazebo.xacro" />
+	<include filename="$(find desire_description)/urdf/head_desire/head.transmission.xacro" />
+	<include filename="$(find cob_description)/urdf/sensors/prosilica.urdf.xacro" />
+	<!--include filename="$(find cob_description)/urdf/sensors/tof.urdf.xacro" /-->
+	<xacro:macro name="head_desire" params="name parent *origin">
 		<!-- joint between base_link and head_axis_link -->
 		<joint name="${name}_pan_joint" type="revolute">
@@ -17,5 +17,5 @@
 			<dynamics damping="0.1" />
 			<calibration rising="${head_pan_ref}" falling="${head_pan_ref}"/>
-			<limit effort="100" lower="-0.7" upper="0.7" velocity="0.5"/>
+			<limit effort="100" lower="-1.4" upper="1.4" velocity="0.5"/>
 		</joint>
 		<link name="${name}_pan_link">
@@ -30,5 +30,5 @@
 					<box size="0.01 0.01 0.12"/>
 				</geometry>
-				<material name="Green" />
+				<material name="Blue" />
 			</visual>
 			<collision>
@@ -40,5 +40,5 @@
 		</link>
 		<joint name="${name}_tilt_joint" type="revolute">
-			<origin xyz="0 0 0" rpy="${M_PI/2} 0 0"/>
+			<origin xyz="0 0 0" rpy="1.5708 0 0"/>
 			<parent link="${name}_pan_link"/>
 			<child link="${name}_tilt_link"/>
@@ -57,12 +57,12 @@
 				<origin xyz="0 0 0" rpy="0 0 0" />
 				<geometry>
-					<mesh filename="package://desire_description/ros/meshes/head_v0/head.stl"/>
+					<mesh filename="package://desire_description/meshes/head_desire/head.stl"/>
 				</geometry>
-				<material name="Green" />
+				<material name="Blue" />
 			</visual>
 			<collision>
 				<origin xyz="0 0 0" rpy="0 0 0" />
 				<geometry>
-					<mesh filename="package://desire_description/ros/meshes/head_v0/head.stl"/>
+					<mesh filename="package://desire_description/meshes/head_desire/head.stl"/>
 				</geometry>
 			</collision>
@@ -70,6 +70,6 @@
 		<!-- right camera -->
 		<xacro:cob_prosilica_v0 name="${name}_color_camera_r" ros_topic="stereo/right"  parent="${name}_tilt_link">
-			<!--origin xyz="${cam_r_x} ${cam_r_y} ${cam_r_z-0.06}" rpy="${cam_r_roll} ${cam_r_pitch+M_PI/2} ${cam_r_yaw+M_PI}"{cam_r_roll-M_PI} /-->
-<origin xyz="${cam_r_x} ${cam_r_y} ${cam_r_z-0.06}" rpy="${cam_r_roll} ${cam_r_pitch+M_PI/2} ${cam_r_yaw}" />
+			<!--origin xyz="${cam_r_x} ${cam_r_y} ${cam_r_z-0.06}" rpy="${cam_r_roll} ${cam_r_pitch+1.5708} ${cam_r_yaw+3.14159}"{cam_r_roll-3.14159} /-->
+<origin xyz="${cam_r_x} ${cam_r_y} ${cam_r_z-0.06}" rpy="${cam_r_roll} ${cam_r_pitch+1.5708} ${cam_r_yaw}" />
 		</xacro:cob_prosilica_v0>
 		<!-- left camera -->
@@ -82,6 +82,6 @@
 		</xacro:cob_tof_v0>
 		<!-- extensions -->
-		<xacro:desire_head_gazebo_v0 name="${name}" />
-		<xacro:desire_head_transmission_v0 name="${name}" />
+		<xacro:head_desire_gazebo_v0 name="${name}" />
+		<xacro:head_desire_transmission_v0 name="${name}" />
 	</xacro:macro>
 </robot>
