Commit message: added colored collada model for sick s300 scanner

File: cob_description/urdf/sensors/sick_s300_laser.gazebo.xacro (robot description, xacro)
@@ -27,5 +27,5 @@
         </controller:gazebo_ros_laser>
       </sensor:ray>
-      <material value="IPA/LightGrey" />
+      <!--material value="IPA/LightGrey" /-->
     </gazebo>
   </xacro:macro>

Commit message: gazebo needs a new link for the topic, if we use the origin of the scanner (the center), the topic detects only the collision model

File: cob_description/urdf/sensors/sick_s300_laser.gazebo.xacro (robot description, xacro)
@@ -2,5 +2,5 @@
 <robot xmlns:xacro="http://www.ros.org/wiki/xacro">
   <xacro:macro name="sick_s300_laser_gazebo_v0" params="name ros_topic update_rate min_angle max_angle">
-    <gazebo reference="${name}_link">
+    <gazebo reference="${name}_gazebo_topic_link">
       <sensor name="${name}" type="ray">
         <always_on>true</always_on>

File: cob_description/urdf/sensors/sick_s300_laser.urdf.xacro (robot description, xacro)
@@ -30,4 +30,10 @@
       </collision>
     </link>
+    <joint name="${name}_gazebo_topic_joint" type="fixed">
+      <origin xyz="0.05 0 0" rpy="0 0 0"/>
+      <parent link="${name}_link"/>
+      <child link="${name}_gazebo_topic_link"/>
+    </joint>
+    <link name="${name}_gazebo_topic_link"/>
     <!-- gazebo extensions -->
     <xacro:sick_s300_laser_gazebo_v0 name="${name}" ros_topic="${ros_topic}" update_rate="${update_rate}" min_angle="${min_angle}" max_angle="${max_angle}" />

Commit message: new sick_s300 collision model

File: cob_description/urdf/sensors/sick_s300_laser.gazebo.xacro (robot description, xacro)
@@ -2,5 +2,5 @@
 <robot xmlns:xacro="http://www.ros.org/wiki/xacro">
   <xacro:macro name="sick_s300_laser_gazebo_v0" params="name ros_topic update_rate min_angle max_angle">
-    <gazebo reference="${name}_gazebo_topic_link">
+    <gazebo reference="${name}_link">
       <sensor name="${name}" type="ray">
         <always_on>true</always_on>

File: cob_description/urdf/sensors/sick_s300_laser.urdf.xacro (robot description, xacro)
@@ -26,14 +26,8 @@
         <origin xyz="0 0 0" rpy="0 0 0" />
         <geometry>
-          <cylinder radius="${cylinder_radius}" length="${cylinder_length}" />
+          <mesh filename="package://cob_description/meshes/sensors/sick_s300_laser_collision.stl"/>
         </geometry>
       </collision>
     </link>
-    <joint name="${name}_gazebo_topic_joint" type="fixed">
-      <origin xyz="0.05 0 0" rpy="0 0 0"/>
-      <parent link="${name}_link"/>
-      <child link="${name}_gazebo_topic_link"/>
-    </joint>
-    <link name="${name}_gazebo_topic_link"/>
     <!-- gazebo extensions -->
     <xacro:sick_s300_laser_gazebo_v0 name="${name}" ros_topic="${ros_topic}" update_rate="${update_rate}" min_angle="${min_angle}" max_angle="${max_angle}" />
