Commit message: the realsense publishes already the frames, it is a bug

File: cob_description/urdf/sensors/realsense.urdf.xacro (robot description, xacro)
@@ -27,5 +27,5 @@
       </collision>
     </link>
-    <joint name="${name}_rgb_joint" type="fixed">
+    <!--joint name="${name}_rgb_joint" type="fixed">
       <origin xyz="0.0088 -0.1034 0.0483" rpy="0 0 0"/>
       <parent link="${name}_link"/>
@@ -50,5 +50,5 @@
       <child link="${name}_depth_optical_frame" />
     </joint>
-    <link name="${name}_depth_optical_frame"/>
+    <link name="${name}_depth_optical_frame"/-->
     <!-- extensions -->
     <xacro:realsense_gazebo name="${name}" ros_topic="${ros_topic}" />

Commit message: remove static tf frames

File: cob_description/urdf/sensors/realsense.urdf.xacro (robot description, xacro)
@@ -27,28 +27,4 @@
       </collision>
     </link>
-    <!--joint name="${name}_rgb_joint" type="fixed">
-      <origin xyz="0.0088 -0.1034 0.0483" rpy="0 0 0"/>
-      <parent link="${name}_link"/>
-      <child link="${name}_rgb_frame" />
-    </joint>
-    <link name="${name}_rgb_frame"/>
-    <joint name="${name}_rgb_optical_joint" type="fixed">
-      <origin xyz="0 0 0" rpy="${-M_PI/2} 0 ${-M_PI/2}" />
-      <parent link="${name}_rgb_frame" />
-      <child link="${name}_rgb_optical_frame" />
-    </joint>
-    <link name="${name}_rgb_optical_frame"/>
-    <joint name="${name}_depth_joint" type="fixed">
-      <origin xyz="0 0.0274 0" rpy="0 0 0" />
-      <parent link="${name}_rgb_frame" />
-      <child link="${name}_depth_frame" />
-    </joint>
-    <link name="${name}_depth_frame"/>
-    <joint name="${name}_depth_optical_joint" type="fixed">
-      <origin xyz="0 0 0" rpy="${-M_PI/2} 0 ${-M_PI/2}" />
-      <parent link="${name}_depth_frame" />
-      <child link="${name}_depth_optical_frame" />
-    </joint>
-    <link name="${name}_depth_optical_frame"/-->
     <!-- extensions -->
     <xacro:realsense_gazebo name="${name}" ros_topic="${ros_topic}" />
