Commit message: depth joint for kinect implemented

File: cob_description/urdf/sensors/kinect.urdf.xacro (robot description, xacro)
@@ -37,4 +37,10 @@
     </joint>
     <link name="${name}_frame"/>
+    <joint name="${name}_frame_depth_joint" type="fixed">
+      <origin xyz="-0.02 0 0" rpy="0 0 0" />
+      <parent link="${name}_link"/>
+      <child link="${name}_depth_link"/>
+    </joint>
+    <link name="${name}_depth_link"/>
     <!-- extensions -->
     <xacro:cob_kinect_gazebo_v0 name="${name}" ros_topic="${ros_topic}" />

Commit message: Revert "depth joint for kinect implemented"
This reverts commit f3449462cd05a5efc8f47252e28366d6a495acb2.

File: cob_description/urdf/sensors/kinect.urdf.xacro (robot description, xacro)
@@ -37,10 +37,4 @@
     </joint>
     <link name="${name}_frame"/>
-    <joint name="${name}_frame_depth_joint" type="fixed">
-      <origin xyz="-0.02 0 0" rpy="0 0 0" />
-      <parent link="${name}_link"/>
-      <child link="${name}_depth_link"/>
-    </joint>
-    <link name="${name}_depth_link"/>
     <!-- extensions -->
     <xacro:cob_kinect_gazebo_v0 name="${name}" ros_topic="${ros_topic}" />

Commit message: visual and collision geometry of cameras are now not colliding with head_cover anymore

File: cob_description/urdf/sensors/kinect.urdf.xacro (robot description, xacro)
@@ -15,14 +15,14 @@
       </inertial>
       <visual>
-        <origin xyz="0 0 0.015" rpy="0 0 0" />
+        <origin xyz="0 0 -0.03" rpy="0 0 0" />
         <geometry>
-          <box size="0.02 0.02 0.075"/>
+          <box size="0.06 0.02 0.02"/>
         </geometry>
         <material name="IPA/LightGrey" />
       </visual>
       <collision>
-        <origin xyz="0 0 0.015" rpy="0 0 0" />
+        <origin xyz="0 0 -0.03" rpy="0 0 0" />
         <geometry>
-           <box size="0.02 0.02 0.075"/>
+           <box size="0.06 0.02 0.02"/>
         </geometry>
       </collision>

File: cob_description/urdf/sensors/prosilica.urdf.xacro (robot description, xacro)
@@ -16,14 +16,14 @@
       </inertial>
       <visual>
-        <origin xyz="0 0 0.015" rpy="0 0 0" />
+        <origin xyz="0 0 0" rpy="0 0 0" />
         <geometry>
-          <cylinder radius="0.01" length="0.075"/>
+          <cylinder radius="0.01" length="0.03"/>
         </geometry>
         <material name="IPA/LightGrey" />
       </visual>
       <collision>
-        <origin xyz="0 0 0.015" rpy="0 0 0" />
+        <origin xyz="0 0 0" rpy="0 0 0" />
         <geometry>
-          <cylinder radius="0.01" length="0.075"/>
+          <cylinder radius="0.01" length="0.03"/>
         </geometry>
       </collision>

Commit message: use asus xtion default values

File: cob_description/urdf/sensors/kinect.urdf.xacro (robot description, xacro)
@@ -2,5 +2,5 @@
 <root xmlns:xacro="http://www.ros.org/wiki/xacro">
   <xacro:include filename="$(find cob_description)/urdf/sensors/kinect.gazebo.xacro" />
-  <xacro:macro name="cob_kinect_v0" params="name parent *origin ros_topic">
+  <xacro:macro name="cob_kinect_v0" params="name parent *origin ros_topic update_rate:=20 data_skip:=0 height:=480 width:=640">
     <joint name="${name}_joint" type="fixed">
       <xacro:insert_block name="origin" />
@@ -33,5 +33,9 @@
     <link name="${name}_frame"/>
     <!-- extensions -->
-    <xacro:cob_kinect_gazebo_v0 name="${name}" ros_topic="${ros_topic}" />
+    <xacro:cob_kinect_gazebo_v0 name="${name}" ros_topic="${ros_topic}"
+    									       update_rate="${update_rate}"
+    									       data_skip="${data_skip}"
+									           height="${height}"
+									           width="${width}"/>
   </xacro:macro>
 </root>
