Commit message: unique macro name for zr300

File: cob_description/urdf/sensors/realsense_zr300.gazebo.xacro (robot description, xacro)
@@ -2,5 +2,5 @@
 <robot xmlns:xacro="http://www.ros.org/wiki/xacro">
   <!-- use default values of realsense_camera/r200_nodelet_rgbd -->
-  <xacro:macro name="realsense_gazebo" params="name ros_topic
+  <xacro:macro name="realsense_zr300_gazebo" params="name ros_topic
                                                depth_fps:=30.0 depth_height:=480 depth_width:=640
                                                color_fps:=30.0 color_height:=480 color_width:=640" >
@@ -17,6 +17,6 @@
           </image>
           <clip>
-            <near>0.2</near>
-            <far>3.5</far>
+            <near>0.55</near>
+            <far>2.8</far>
           </clip>
           <noise>
@@ -35,6 +35,6 @@
           <depthImageTopicName>depth_registered/image_raw</depthImageTopicName>
           <depthImageCameraInfoTopicName>depth_registered/camera_info</depthImageCameraInfoTopicName>
-          <pointCloudCutoff>0.5</pointCloudCutoff>
-          <pointCloudCutoffMax>5.0</pointCloudCutoffMax>
+          <pointCloudCutoff>0.55</pointCloudCutoff>
+          <pointCloudCutoffMax>2.8</pointCloudCutoffMax>
           <distortionK1>0.0</distortionK1>
           <distortionK2>0.0</distortionK2>
@@ -48,4 +48,5 @@
         </plugin>
       </sensor>
+      <!-- ToDo: add plugins for IMU, Fisheye, IR -->
       <material>IPA/LightGrey</material>
     </gazebo>

File: cob_description/urdf/sensors/realsense_zr300.urdf.xacro (robot description, xacro)
@@ -28,5 +28,5 @@
     </link>
     <!-- extensions -->
-    <xacro:realsense_gazebo name="${name}" ros_topic="${ros_topic}" />
+    <xacro:realsense_zr300_gazebo name="${name}" ros_topic="${ros_topic}" />
   </xacro:macro>
 </robot>
