Commit message: update gazebo tags for sensor plugins

File: cob_description/urdf/sensors/kinect.gazebo.xacro (robot description, xacro)
@@ -1,47 +1,51 @@
 <?xml version="1.0"?>
 <root xmlns:xacro="http://www.ros.org/wiki/xacro">
-<xacro:macro name="cob_kinect_gazebo_v0" params="name ros_topic">
-  <gazebo reference="${name}_frame">
-  <sensor type="depth" name="${name}_frame_sensor">
-    <always_on>true</always_on>
-    <update_rate>20.0</update_rate>
-    <camera>
-      <horizontal_fov>${62.0*M_PI/180.0}</horizontal_fov>
-      <image>
-        <format>R8G8B8</format>
-        <width>640</width>
-        <height>480</height>
-      </image>
-      <clip>
-        <near>0.1</near>
-        <far>100</far>
-      </clip>
-    </camera>
-    <plugin name="${name}_controller" filename="libgazebo_ros_openni_kinect.so">
-      <alwaysOn>true</alwaysOn>
-      <updateRate>20.0</updateRate>
-      <cameraName>${ros_topic}</cameraName>
-      <frameName>${name}_link</frameName>
-      <imageTopicName>rgb/image_raw</imageTopicName>
-      <depthImageTopicName>depth/image_raw</depthImageTopicName>
-      <pointCloudTopicName>depth_registered/points</pointCloudTopicName>
-      <cameraInfoTopicName>rgb/camera_info</cameraInfoTopicName>
-      <depthImageCameraInfoTopicName>depth_registered/camera_info</depthImageCameraInfoTopicName>
-      <pointCloudCutoff>0.5</pointCloudCutoff>
-      <baseline>0.2</baseline>
-      <hackBaseline>0.0</hackBaseline>
-      <distortionK1>0.0</distortionK1>
-      <distortionK2>0.0</distortionK2>
-      <distortionK3>0.0</distortionK3>
-      <distortionT1>0.0</distortionT1>
-      <distortionT2>0.0</distortionT2>
-      <CxPrime>0.0</CxPrime>
-      <Cx>0.0</Cx>
-      <Cy>0.0</Cy>
-      <focalLength>0.0</focalLength>
-    </plugin>
-  </sensor>
-    <material>IPA/LightGrey</material>
-  </gazebo>
-</xacro:macro>
+  <xacro:macro name="cob_kinect_gazebo_v0" params="name ros_topic">
+    <gazebo reference="${name}_frame">
+      <sensor type="depth" name="${name}_frame_sensor">
+        <always_on>true</always_on>
+        <update_rate>20.0</update_rate>
+        <camera>
+          <horizontal_fov>${62.0*M_PI/180.0}</horizontal_fov>
+          <image>
+            <format>R8G8B8</format>
+            <width>640</width>
+            <height>480</height>
+          </image>
+          <clip>
+            <near>0.1</near>
+            <far>100</far>
+          </clip>
+          <noise>
+            <type>gaussian</type>
+            <mean>0.0</mean>
+            <stddev>0.0</stddev>
+          </noise>
+        </camera>
+        <plugin name="${name}_controller" filename="libgazebo_ros_openni_kinect.so">
+          <updateRate>20.0</updateRate>
+          <cameraName>${ros_topic}</cameraName>
+          <frameName>${name}_link</frameName>
+          <imageTopicName>rgb/image_raw</imageTopicName>
+          <depthImageTopicName>depth/image_raw</depthImageTopicName>
+          <pointCloudTopicName>depth_registered/points</pointCloudTopicName>
+          <cameraInfoTopicName>rgb/camera_info</cameraInfoTopicName>
+          <depthImageCameraInfoTopicName>depth_registered/camera_info</depthImageCameraInfoTopicName>
+          <pointCloudCutoff>0.5</pointCloudCutoff>
+          <baseline>0.2</baseline>
+          <hackBaseline>0.0</hackBaseline>
+          <distortionK1>0.0</distortionK1>
+          <distortionK2>0.0</distortionK2>
+          <distortionK3>0.0</distortionK3>
+          <distortionT1>0.0</distortionT1>
+          <distortionT2>0.0</distortionT2>
+          <CxPrime>0.0</CxPrime>
+          <Cx>0.0</Cx>
+          <Cy>0.0</Cy>
+          <focalLength>0.0</focalLength>
+        </plugin>
+      </sensor>
+      <material>IPA/LightGrey</material>
+    </gazebo>
+  </xacro:macro>
 </root>

File: cob_description/urdf/sensors/phidgets_distance.gazebo.xacro (robot description, xacro)
@@ -2,36 +2,37 @@
 <robot xmlns:xacro="http://www.ros.org/wiki/xacro">
   <xacro:macro name="phidgets_distance_gazebo_v0" params="name ros_topic update_rate">
-  <gazebo reference="${name}_link">
-    <sensor name="${name}" type="ray">
-      <always_on>true</always_on>
-      <update_rate>${update_rate}</update_rate>
-      <pose>0 0 0 0 0 0</pose>
-      <visualize>false</visualize>
-      <ray>
-        <scan>
-          <horizontal>
-            <samples>10</samples>
-            <resolution>1.0</resolution>
-            <min_angle>-0.2</min_angle>
-            <max_angle>0.2</max_angle>
-          </horizontal>
-        </scan>
-        <range>
-          <min>0.01</min>    <!-- real value from sensor datasheet is 0.04m -->
-          <max>0.4</max>    <!-- real value from sensor datasheet is 0.30m -->
-          <resolution>0.005</resolution>
-        </range>
-      </ray>
-      <plugin name="gazebo_ros_${name}_controller" filename="libgazebo_ros_laser.so">
-        <gaussianNoise>0.005</gaussianNoise>
-        <alwaysOn>true</alwaysOn>
-        <updateRate>${update_rate}</updateRate>
-        <topicName>${ros_topic}</topicName>
-        <frameName>/${name}_link</frameName>
-        <hokuyoMinIntensity>101.0</hokuyoMinIntensity>
-      </plugin>
-    </sensor>
-    <material>IPA/LightGrey</material>
-  </gazebo>
+    <gazebo reference="${name}_link">
+      <sensor name="${name}" type="ray">
+        <always_on>true</always_on>
+        <update_rate>${update_rate}</update_rate>
+        <pose>0 0 0 0 0 0</pose>
+        <visualize>false</visualize>
+        <ray>
+          <scan>
+            <horizontal>
+              <samples>10</samples>
+              <resolution>1.0</resolution>
+              <min_angle>-0.2</min_angle>
+              <max_angle>0.2</max_angle>
+            </horizontal>
+          </scan>
+          <range>
+            <min>0.01</min>    <!-- real value from sensor datasheet is 0.04m -->
+            <max>0.4</max>    <!-- real value from sensor datasheet is 0.30m -->
+            <resolution>0.005</resolution>
+          </range>
+          <noise>
+            <type>gaussian</type>
+            <mean>0.0</mean>
+            <stddev>0.005</stddev>
+          </noise>
+        </ray>
+        <plugin name="gazebo_ros_${name}_controller" filename="libgazebo_ros_laser.so">
+          <topicName>${ros_topic}</topicName>
+          <frameName>/${name}_link</frameName>
+        </plugin>
+      </sensor>
+      <material>IPA/LightGrey</material>
+    </gazebo>
   </xacro:macro>
 </robot>

File: cob_description/urdf/sensors/prosilica.gazebo.xacro (robot description, xacro)
@@ -17,7 +17,11 @@
             <far>100</far>
           </clip>
+          <noise>
+            <type>gaussian</type>
+            <mean>0.0</mean>
+            <stddev>0.0</stddev>
+          </noise>
         </camera>
         <plugin name="${name}_controller" filename="libgazebo_ros_camera.so">
-          <alwaysOn>true</alwaysOn>
           <updateRate>10.0</updateRate>
           <cameraName>${name}_sensor</cameraName>
@@ -40,5 +44,4 @@
       </sensor>
       <material value="IPA/LightGrey" />
-      <turnGravityOff>true</turnGravityOff>
     </gazebo>
   </xacro:macro>

File: cob_description/urdf/sensors/softkinetic.gazebo.xacro (robot description, xacro)
@@ -1,45 +1,49 @@
 <?xml version="1.0"?>
 <robot xmlns:xacro="http://www.ros.org/wiki/xacro">
-<xacro:macro name="softkinetic_gazebo" params="name ros_topic">
-  <gazebo reference="${name}_frame">
-    <sensor type="depth" name="${name}_frame_sensor">
-      <always_on>true</always_on>
-      <update_rate>25.0</update_rate>
-      <camera>
-        <horizontal_fov>${74.0*M_PI/180.0}</horizontal_fov>
-        <image>
-          <format>R8G8B8</format>
-          <width>320</width>
-          <height>240</height>
-        </image>
-        <clip>
-          <near>0.15</near>
-          <far>1.0</far>
-        </clip>
-      </camera>
-      <plugin name="${name}_frame_controller" filename="libgazebo_ros_openni_kinect.so">
-        <alwaysOn>true</alwaysOn>
-        <updateRate>25.0</updateRate>
-        <cameraName>${ros_topic}</cameraName>
-        <imageTopicName>rgb/image_raw</imageTopicName>
-        <depthImageTopicName>depth/image_raw</depthImageTopicName>
-        <pointCloudTopicName>depth_registered/points</pointCloudTopicName>
-        <cameraInfoTopicName>rgb/camera_info</cameraInfoTopicName>
-        <depthImageCameraInfoTopicName>depth_registered/camera_info</depthImageCameraInfoTopicName>
-        <frameName>${name}_optical_frame</frameName>
-        <pointCloudCutoff>0.5</pointCloudCutoff>
-        <distortionK1>0.0</distortionK1>
-        <distortionK2>0.0</distortionK2>
-        <distortionK3>0.0</distortionK3>
-        <distortionT1>0.0</distortionT1>
-        <distortionT2>0.0</distortionT2>
-        <CxPrime>0.0</CxPrime>
-        <Cx>0.0</Cx>
-        <Cy>0.0</Cy>
-        <focalLength>0.0</focalLength>
-      </plugin>
-    </sensor>
-    <material>IPA/LightGrey</material>
-  </gazebo>
-</xacro:macro>
+  <xacro:macro name="softkinetic_gazebo" params="name ros_topic">
+    <gazebo reference="${name}_frame">
+      <sensor type="depth" name="${name}_frame_sensor">
+        <always_on>true</always_on>
+        <update_rate>25.0</update_rate>
+        <camera>
+          <horizontal_fov>${74.0*M_PI/180.0}</horizontal_fov>
+          <image>
+            <format>R8G8B8</format>
+            <width>320</width>
+            <height>240</height>
+          </image>
+          <clip>
+            <near>0.15</near>
+            <far>1.0</far>
+          </clip>
+          <noise>
+            <type>gaussian</type>
+            <mean>0.0</mean>
+            <stddev>0.0</stddev>
+          </noise>
+        </camera>
+        <plugin name="${name}_frame_controller" filename="libgazebo_ros_openni_kinect.so">
+          <updateRate>25.0</updateRate>
+          <cameraName>${ros_topic}</cameraName>
+          <imageTopicName>rgb/image_raw</imageTopicName>
+          <depthImageTopicName>depth/image_raw</depthImageTopicName>
+          <pointCloudTopicName>depth_registered/points</pointCloudTopicName>
+          <cameraInfoTopicName>rgb/camera_info</cameraInfoTopicName>
+          <depthImageCameraInfoTopicName>depth_registered/camera_info</depthImageCameraInfoTopicName>
+          <frameName>${name}_optical_frame</frameName>
+          <pointCloudCutoff>0.5</pointCloudCutoff>
+          <distortionK1>0.0</distortionK1>
+          <distortionK2>0.0</distortionK2>
+          <distortionK3>0.0</distortionK3>
+          <distortionT1>0.0</distortionT1>
+          <distortionT2>0.0</distortionT2>
+          <CxPrime>0.0</CxPrime>
+          <Cx>0.0</Cx>
+          <Cy>0.0</Cy>
+          <focalLength>0.0</focalLength>
+        </plugin>
+      </sensor>
+      <material>IPA/LightGrey</material>
+    </gazebo>
+  </xacro:macro>
 </robot>

File: cob_description/urdf/sensors/tof.gazebo.xacro (robot description, xacro)
@@ -1,44 +1,48 @@
 <?xml version="1.0"?>
 <root xmlns:xacro="http://www.ros.org/wiki/xacro">
-<!-- specs from mesa Swiss Ranger SR400001 http://www.mesa-imaging.ch/prodview4k.php -->
-<xacro:macro name="cob_tof_gazebo_v0" params="name ros_topic">
-  <gazebo reference="${name}_frame">
-  <sensor name="${name}_sensor" type="ray">
-    <always_on>true</always_on>
-    <update_rate>10</update_rate>  <!--max50Hz-->
-    <pose>0 0 0.05 0 0 0</pose>
-    <visualize>false</visualize>
-    <ray>
-      <scan>
-        <horizontal>
-          <samples>176</samples>    <!--true value 176-->
-          <resolution>1.0</resolution>
-          <min_angle>-0.38</min_angle>
-          <max_angle>0.38</max_angle>
-        </horizontal>
-        <vertical>
-          <samples>144</samples>    <!--true value 144 -->
-          <resolution>1.0</resolution>
-          <min_angle>-0.3</min_angle>
-          <max_angle>0.3</max_angle>
-        </vertical>
-      </scan>
-      <range>
-        <min>0.80</min>    <!--0.8m min calibrated range-->
-        <max>5.0</max>    <!--5.0m max calibrated range-->
-        <resolution>0.010</resolution>
-      </range>
-    </ray>
-    <plugin name="tof_controller" filename="libgazebo_ros_block_laser.so">
-      <gaussianNoise>0.005</gaussianNoise>
-      <alwaysOn>true</alwaysOn>
-      <updateRate>30</updateRate>   <!--max 50Hz, cob3 30Hz -->
-      <topicName>${ros_topic}</topicName>
-      <frameName>/${name}_frame</frameName>
-    </plugin>
-  </sensor>
-    <material value="IPA/LightGrey" />
-    <turnGravityOff>true</turnGravityOff>
-  </gazebo>
-</xacro:macro>
+  <!-- specs from mesa Swiss Ranger SR400001 http://www.mesa-imaging.ch/prodview4k.php -->
+  <xacro:macro name="cob_tof_gazebo_v0" params="name ros_topic">
+    <gazebo reference="${name}_frame">
+      <sensor name="${name}_sensor" type="ray">
+        <always_on>true</always_on>
+        <update_rate>10</update_rate>  <!--max50Hz-->
+        <pose>0 0 0.05 0 0 0</pose>
+        <visualize>false</visualize>
+        <ray>
+          <scan>
+            <horizontal>
+              <samples>176</samples>    <!--true value 176-->
+              <resolution>1.0</resolution>
+              <min_angle>-0.38</min_angle>
+              <max_angle>0.38</max_angle>
+            </horizontal>
+            <vertical>
+              <samples>144</samples>    <!--true value 144 -->
+              <resolution>1.0</resolution>
+              <min_angle>-0.3</min_angle>
+              <max_angle>0.3</max_angle>
+            </vertical>
+          </scan>
+          <range>
+            <min>0.80</min>    <!--0.8m min calibrated range-->
+            <max>5.0</max>    <!--5.0m max calibrated range-->
+            <resolution>0.010</resolution>
+          </range>
+          <noise>
+            <type>gaussian</type>
+            <mean>0.0</mean>
+            <stddev>0.005</stddev>
+          </noise>
+        </ray>
+        <plugin name="tof_controller" filename="libgazebo_ros_block_laser.so">
+          <gaussianNoise>0.005</gaussianNoise>
+          <updateRate>30</updateRate>   <!--max 50Hz, cob3 30Hz -->
+          <topicName>${ros_topic}</topicName>
+          <frameName>/${name}_frame</frameName>
+          <hokuyoMinIntensity>101</hokuyoMinIntensity>
+        </plugin>
+      </sensor>
+      <material value="IPA/LightGrey" />
+    </gazebo>
+  </xacro:macro>
 </root>

Commit message: fix coordinate frames for asus camera

File: cob_description/urdf/sensors/kinect.gazebo.xacro (robot description, xacro)
@@ -3,5 +3,5 @@
   <xacro:macro name="cob_kinect_gazebo_v0" params="name ros_topic
                                                    update_rate:=20 data_skip:=0 height:=480 width:=640">
-    <gazebo reference="${name}_frame">
+    <gazebo reference="${name}_link">
       <sensor type="depth" name="${name}_frame_sensor">
         <always_on>true</always_on>
@@ -27,5 +27,5 @@
           <updateRate>${update_rate/(data_skip+1)}</updateRate>
           <cameraName>${ros_topic}</cameraName>
-          <frameName>${name}_link</frameName>
+          <frameName>${name}_optical_frame</frameName>
           <imageTopicName>rgb/image_raw</imageTopicName>
           <cameraInfoTopicName>rgb/camera_info</cameraInfoTopicName>

File: cob_description/urdf/sensors/kinect.urdf.xacro (robot description, xacro)
@@ -26,16 +26,10 @@
       </collision>
     </link>
-    <joint name="${name}_frame_joint" type="fixed">
-      <origin xyz="0 0 0" rpy="${M_PI/2} -${M_PI/2} 0" />
-      <parent link="${name}_link"/>
-      <child link="${name}_frame"/>
-    </joint>
-    <link name="${name}_frame"/>
     <!-- extensions -->
     <xacro:cob_kinect_gazebo_v0 name="${name}" ros_topic="${ros_topic}"
-    									       update_rate="${update_rate}"
-    									       data_skip="${data_skip}"
-									           height="${height}"
-									           width="${width}"/>
+                                               update_rate="${update_rate}"
+                                               data_skip="${data_skip}"
+                                               height="${height}"
+                                               width="${width}"/>
   </xacro:macro>
 </root>
