Commit message: usb_cam default values

File: cob_description/urdf/sensors/usb_cam.gazebo.xacro (robot description, xacro)
@@ -1,14 +1,15 @@
 <?xml version="1.0"?>
 <robot xmlns:xacro="http://www.ros.org/wiki/xacro">
-  <xacro:macro name="usb_cam_gazebo" params="name ros_topic">
+  <!-- at 2048x1536 3.6hz is maximum on hw -->
+  <xacro:macro name="usb_cam_gazebo" params="name ros_topic update_rate:=3.5 height:=1536 width:=2048" >
     <gazebo reference="${name}_frame">
     <sensor type="camera" name="${name}">
-      <update_rate>5</update_rate>
+      <update_rate>${update_rate}</update_rate>
       <camera name="${name}">
-        <horizontal_fov>2.97</horizontal_fov>
+        <horizontal_fov>${170.0*M_PI/180.0}</horizontal_fov>
         <image>
-          <width>2048</width>
-          <height>1536</height>
           <format>R8G8B8</format>
+          <width>${width}</width>
+          <height>${height}</height>
         </image>
         <clip>
@@ -24,5 +25,5 @@
       <plugin name="camera_controller" filename="libgazebo_ros_camera.so">
         <alwaysOn>true</alwaysOn>
-        <updateRate>0.0</updateRate>
+        <updateRate>${update_rate}</updateRate>
         <cameraName>${ros_topic}</cameraName>
         <imageTopicName>image_raw</imageTopicName>

File: cob_description/urdf/sensors/usb_cam.urdf.xacro (robot description, xacro)
@@ -2,5 +2,5 @@
 <robot xmlns:xacro="http://www.ros.org/wiki/xacro">
   <xacro:include filename="$(find cob_description)/urdf/sensors/usb_cam.gazebo.xacro" />
-  <xacro:macro name="usb_cam" params="name parent ros_topic *origin">
+  <xacro:macro name="usb_cam" params="name parent *origin ros_topic update_rate height width">
     <joint name="${name}_joint" type="fixed">
       <xacro:insert_block name="origin" />
@@ -34,5 +34,8 @@
     <link name="${name}_frame"/>
     <!-- extensions -->
-    <xacro:usb_cam_gazebo name="${name}" ros_topic="${ros_topic}" />
+    <xacro:usb_cam_gazebo name="${name}" ros_topic="${ros_topic}"
+									     update_rate="${update_rate}"
+									     height="${height}"
+									     width="${width}"/>
   </xacro:macro>
 </robot>

Commit message: fix frames of usb_cam

File: cob_description/urdf/sensors/usb_cam.gazebo.xacro (robot description, xacro)
@@ -3,5 +3,5 @@
   <!-- at 2048x1536 3.6hz is maximum on hw -->
   <xacro:macro name="usb_cam_gazebo" params="name ros_topic update_rate:=3.5 height:=1536 width:=2048" >
-    <gazebo reference="${name}_frame">
+    <gazebo reference="${name}_optical_frame">
     <sensor type="camera" name="${name}">
       <update_rate>${update_rate}</update_rate>
@@ -29,5 +29,5 @@
         <imageTopicName>image_raw</imageTopicName>
         <cameraInfoTopicName>camera_info</cameraInfoTopicName>
-        <frameName>${name}_link</frameName>
+        <frameName>${name}_optical_frame</frameName>
         <hackBaseline>0.07</hackBaseline>
         <distortionK1>0.0</distortionK1>

File: cob_description/urdf/sensors/usb_cam.urdf.xacro (robot description, xacro)
@@ -28,14 +28,20 @@
     </link>
     <joint name="${name}_frame_joint" type="fixed">
-      <origin xyz="0 0 0" rpy="${M_PI/2} -${M_PI/2} 0" />
+      <origin xyz="0 0 0" rpy="0 0 0" />
       <parent link="${name}_link"/>
       <child link="${name}_frame"/>
     </joint>
     <link name="${name}_frame"/>
+    <joint name="${name}_optical_frame_joint" type="fixed">
+      <origin xyz="0 0 0" rpy="-${M_PI/2} 0 -${M_PI/2}" />
+      <parent link="${name}_frame"/>
+      <child link="${name}_optical_frame"/>
+    </joint>
+    <link name="${name}_optical_frame"/>
     <!-- extensions -->
     <xacro:usb_cam_gazebo name="${name}" ros_topic="${ros_topic}"
-									     update_rate="${update_rate}"
-									     height="${height}"
-									     width="${width}"/>
+                                         update_rate="${update_rate}"
+                                         height="${height}"
+                                         width="${width}"/>
   </xacro:macro>
 </robot>
