Commit message: proper mesh files for base and scanner

File: cob_description/urdf/sensors/sick_microscan3.urdf.xacro (robot description, xacro)
@@ -2,6 +2,6 @@
 <robot xmlns:xacro="http://www.ros.org/wiki/xacro">
   <xacro:include filename="$(find cob_description)/urdf/sensors/sick_microscan3.gazebo.xacro" />
-  <xacro:property name="cylinder_radius" value="0.05" />  <!--simple collision model for the laser -->
-  <xacro:property name="cylinder_length" value="0.15" />
+  <xacro:property name="cylinder_radius" value="0.056" />  <!--simple collision model for the laser -->
+  <xacro:property name="cylinder_length" value="0.150" />
   <xacro:macro name="sick_microscan3" params="name parent *origin">
     <joint name="${name}_joint" type="fixed">
@@ -17,6 +17,5 @@
         <origin xyz="0 0 0" rpy="0 0 0" />
         <geometry>
-          <mesh filename="package://cob_description/meshes/sensors/sick_s300_laser.dae"/> <!-- microscan mesh -->
-          <!--box size="0.001 0.001 0.001" /-->
+          <mesh filename="package://cob_description/meshes/sensors/sick_microscan3.stl"/>
         </geometry>
         <material name="IPA/LightGrey" />
@@ -25,5 +24,5 @@
         <origin xyz="0 0 0" rpy="0 0 0" />
         <geometry>
-          <mesh filename="package://cob_description/meshes/sensors/sick_s300_laser_collision.stl"/> <!-- microscan mesh -->
+          <mesh filename="package://cob_description/meshes/sensors/sick_microscan3_collision.stl"/>
         </geometry>
       </collision>

File: raw_description/urdf/raw4_base/base.urdf.xacro (robot description, xacro)
@@ -12,13 +12,5 @@
   <xacro:property name="caster_offset_y_fr" value="-0.190" />
   <xacro:property name="caster_offset_z" value="0.08" />
-  <!-- <xacro:property name="battery_offset_x" value="0.0" />
-  <xacro:property name="battery_offset_y" value="-0.008" />
-  <xacro:property name="battery_offset_z" value="0.065" /> -->
   <xacro:property name="base_mass" value="43.1" />
-  <!-- <xacro:property name="battery_mass" value="40" /> -->
-  <!-- <xacro:property name="battery_size_x" value="0.5" />
-  <xacro:property name="battery_size_y" value="0.148" />
-  <xacro:property name="battery_size_z" value="0.26" /> -->
-  <!-- battery macros-->
   <xacro:macro name="raw4_base" params="name">
     <link name="${name}_footprint"/>
@@ -33,8 +25,7 @@
       </xacro:box_inertial>
       <visual>
-        <origin xyz="0 0 0.25" rpy="0 0 0" />
+        <origin xyz="0 0 0" rpy="0 0 0" />
         <geometry>
-          <mesh filename="package://raw_description/meshes/raw4_base/raw4_base.dae"/>
-          <!-- <box size="1.2 0.75 0.1"/> -->
+          <mesh filename="package://raw_description/meshes/raw4_base/raw4_base.stl"/>
         </geometry>
         <material name="Grey">
@@ -43,8 +34,7 @@
       </visual>
       <collision>
-        <origin xyz="0 0 0.25" rpy="0 0 0" />
+        <origin xyz="0 0 0" rpy="0 0 0" />
         <geometry>
           <mesh filename="package://raw_description/meshes/raw4_base/raw4_base.stl"/>
-          <!-- <box size="1.2 0.75 0.1"/> -->
         </geometry>
       </collision>
@@ -63,8 +53,4 @@
       <origin xyz="${-caster_offset_x} ${caster_offset_y_br} ${caster_offset_z}" rpy="0 0 0" />
     </xacro:drive_wheel>
-    <!-- battery-->
-    <!-- <xacro:cob_batteries name="${name}_battery" parent="${name}_link">
-      <origin xyz="${-battery_offset_x} ${battery_offset_y} ${battery_offset_z}" rpy="${M_PI/2} 0 ${-M_PI/2}" />
-    </xacro:cob_batteries> -->
     <!-- gazebo extensions -->
     <xacro:base_gazebo name="${name}" />
