Commit message: fix typo

File: cob_description/urdf/sensors/sick_microscan3.gazebo.xacro (robot description, xacro)
@@ -1,5 +1,5 @@
 <?xml version="1.0"?>
 <robot xmlns:xacro="http://www.ros.org/wiki/xacro">
-  <xacro:macro name="sick_micorscan3_gazebo" params="name">
+  <xacro:macro name="sick_microscan3_gazebo" params="name">
     <gazebo reference="${name}_link">
       <sensor name="${name}" type="ray">

File: cob_description/urdf/sensors/sick_microscan3.urdf.xacro (robot description, xacro)
@@ -29,5 +29,5 @@
     </link>
     <!-- gazebo extensions -->
-    <xacro:sick_micorscan3_gazebo name="${name}"/>
+    <xacro:sick_microscan3_gazebo name="${name}"/>
   </xacro:macro>
 </robot>
