Commit message: add rplidar for gazebo

File: cob_description/urdf/sensors/rplidar.urdf.xacro (robot description, xacro)
@@ -1,6 +1,7 @@
 <?xml version="1.0"?>
 <robot xmlns:xacro="http://www.ros.org/wiki/xacro">
-  <xacro:include filename="$(find cob_description)/urdf/sensors/sick_s300_laser.gazebo.xacro" />
-  <xacro:property name="cylinder_radius" value="0.08" />  <!--simple collision model for the laser -->
+  <xacro:include filename="$(find cob_description)/urdf/sensors/rplidar.gazebo.xacro" />
+  <xacro:property name="cylinder_radius" value="0.08" />
+  <!--simple collision model for the laser -->
   <xacro:property name="cylinder_length" value="0.05" />
   <xacro:macro name="rplidar" params="name parent *origin">
@@ -17,5 +18,5 @@
         <origin xyz="0 0 0" rpy="0 0 0" />
         <geometry>
-          <mesh filename="package://cob_description/meshes/sensors/sick_s300_laser.dae"/>
+          <mesh filename="package://cob_description/meshes/sensors/rplidar.dae"/>
           <!--box size="0.001 0.001 0.001" /-->
         </geometry>
@@ -25,10 +26,10 @@
         <origin xyz="0 0 0" rpy="0 0 0" />
         <geometry>
-          <mesh filename="package://cob_description/meshes/sensors/sick_s300_laser_collision.stl"/>
+          <mesh filename="package://cob_description/meshes/sensors/rplidar.dae"/>
         </geometry>
       </collision>
     </link>
     <!-- gazebo extensions -->
-    <xacro:sick_s300_laser_gazebo_v0 name="${name}"/>
+    <xacro:rplidar_laser_gazebo name="${name}"/>
   </xacro:macro>
 </robot>
