Commit message: set valid values

File: cob_description/urdf/sensors/realsense_d435.urdf.xacro (robot description, xacro)
@@ -33,5 +33,5 @@
     <!-- extensions -->
     <!--xacro:realsense_d435_gazebo name="${name}"/-->
-    <xacro:gazebo_d435 camera_name="${name}" reference_link="${name}_link" topics_ns="${name}" depth_optical_frame="${name}_depth_optical_frame" color_optical_frame="${name}_color_optical_frame" infrared1_optical_frame="${name}_left_ir_optical_frame" infrared2_optical_frame="${name}_right_ir_optical_frame"/>
+    <xacro:gazebo_d435 camera_name="${name}" reference_link="${name}_link" topics_ns="${name}" depth_optical_frame="${name}_depth_optical_frame" color_optical_frame="${name}_color_optical_frame" infrared1_optical_frame="${name}_left_ir_optical_frame" infrared2_optical_frame="${name}_right_ir_optical_frame" depth_fps="15.0" depth_height="480" depth_width="640" color_fps="15.0" color_height="720" color_width="1280" />
   </xacro:macro>
 </robot>

File: cob_description/urdf/sensors/realsense_d435_pal.gazebo.xacro (robot description, xacro)
@@ -6,5 +6,6 @@
 -->
 <robot xmlns:xacro="http://ros.org/wiki/xacro">
-  <xacro:macro name="gazebo_d435" params="camera_name reference_link topics_ns depth_optical_frame color_optical_frame infrared1_optical_frame infrared2_optical_frame" >
+  <xacro:macro name="gazebo_d435" params="camera_name reference_link topics_ns depth_optical_frame color_optical_frame infrared1_optical_frame infrared2_optical_frame depth_fps:=15.0 depth_height:=720 depth_width:=1280
+    color_fps:=15.0 color_height:=720 color_width:=1280">
     <!-- Load parameters to model's main link-->
     <xacro:property name="deg_to_rad" value="0.01745329251994329577" />
@@ -27,6 +28,6 @@
           <horizontal_fov>${69.4*deg_to_rad}</horizontal_fov>
           <image>
-            <width>1920</width>
-            <height>1080</height>
+            <width>${color_width}</width>
+            <height>${color_height}</height>
             <format>RGB_INT8</format>
           </image>
@@ -42,5 +43,5 @@
         </camera>
         <always_on>1</always_on>
-        <update_rate>30</update_rate>
+        <update_rate>${color_fps}</update_rate>
         <visualize>1</visualize>
       </sensor>
@@ -49,6 +50,6 @@
           <horizontal_fov>${85.2*deg_to_rad}</horizontal_fov>
           <image>
-            <width>1280</width>
-            <height>720</height>
+            <width>${depth_width}</width>
+            <height>${depth_height}</height>
             <format>L_INT8</format>
           </image>
@@ -64,5 +65,5 @@
         </camera>
         <always_on>1</always_on>
-        <update_rate>90</update_rate>
+        <update_rate>${depth_fps}</update_rate>
         <visualize>0</visualize>
       </sensor>
@@ -71,6 +72,6 @@
           <horizontal_fov>${85.2*deg_to_rad}</horizontal_fov>
           <image>
-            <width>1280</width>
-            <height>720</height>
+            <width>${depth_width}</width>
+            <height>${depth_height}</height>
             <format>L_INT8</format>
           </image>
@@ -86,5 +87,5 @@
         </camera>
         <always_on>1</always_on>
-        <update_rate>90</update_rate>
+        <update_rate>${depth_fps}</update_rate>
         <visualize>0</visualize>
       </sensor>
@@ -93,6 +94,6 @@
           <horizontal_fov>${85.2*deg_to_rad}</horizontal_fov>
           <image>
-            <width>1280</width>
-            <height>720</height>
+            <width>${depth_width}</width>
+            <height>${depth_height}</height>
           </image>
           <clip>
@@ -107,6 +108,6 @@
         </camera>
         <always_on>1</always_on>
-        <update_rate>90</update_rate>
-        <visualize>0</visualize>
+        <update_rate>${depth_fps}</update_rate>
+        <visualize>1</visualize>
       </sensor>
     </gazebo>
@@ -114,11 +115,11 @@
       <plugin name="${topics_ns}" filename="librealsense_gazebo_plugin.so">
         <prefix>${camera_name}</prefix>
-      	<depthUpdateRate>60.0</depthUpdateRate>
-      	<colorUpdateRate>60.0</colorUpdateRate>
-      	<infraredUpdateRate>60.0</infraredUpdateRate>
+        <depthUpdateRate>${depth_fps}</depthUpdateRate>
+        <colorUpdateRate>${color_fps}</colorUpdateRate>
+        <infraredUpdateRate>${depth_fps}</infraredUpdateRate>
       	<depthTopicName>depth/image_raw</depthTopicName>
       	<depthCameraInfoTopicName>depth/camera_info</depthCameraInfoTopicName>
-      	<colorTopicName>color/image_raw</colorTopicName>
-      	<colorCameraInfoTopicName>color/camera_info</colorCameraInfoTopicName>
+        <colorTopicName>rgb/image_raw</colorTopicName>
+        <colorCameraInfoTopicName>rgb/camera_info</colorCameraInfoTopicName>
       	<infrared1TopicName>infra1/image_raw</infrared1TopicName>
       	<infrared1CameraInfoTopicName>infra1/camera_info</infrared1CameraInfoTopicName>
@@ -131,5 +132,5 @@
       	<rangeMinDepth>0.2</rangeMinDepth>
       	<rangeMaxDepth>10.0</rangeMaxDepth>
-      	<pointCloud>false</pointCloud>
+        <pointCloud>true</pointCloud>
       	<pointCloudTopicName>depth/points</pointCloudTopicName>
       	<pointCloudCutoff>0.5</pointCloudCutoff>
