Commit message: use only one realsense plugin

File: cob_description/urdf/sensors/realsense_d435.gazebo.xacro (robot description, xacro)
@@ -1,53 +1,139 @@
 <?xml version="1.0"?>
-<robot xmlns:xacro="http://www.ros.org/wiki/xacro">
-  <!-- use default values of mojin_bringup/d400_rgbd and d435 specs-->
-  <xacro:macro name="realsense_d435_gazebo" params="name
-                                               depth_fps:=15.0 depth_height:=720 depth_width:=1280
-                                               color_fps:=15.0 color_height:=720 color_width:=1280" >
-    <gazebo reference="${name}_link">
-      <sensor type="depth" name="${name}_depth_frame">
-        <always_on>true</always_on>
-        <update_rate>${color_fps}</update_rate>
-        <camera>
-          <horizontal_fov>${85.2*M_PI/180.0}</horizontal_fov>
+<!--
+License: Apache 2.0. See LICENSE file in root directory.
+Copyright(c) 2017 PAL Robotics, S.L. All Rights Reserved
+This is the Gazebo URDF model for the Intel RealSense D435 camera
+-->
+<robot xmlns:xacro="http://ros.org/wiki/xacro">
+  <xacro:macro name="gazebo_d435" params="camera_name reference_link topics_ns depth_optical_frame color_optical_frame infrared1_optical_frame infrared2_optical_frame depth_fps:=15.0 depth_height:=720 depth_width:=1280
+    color_fps:=15.0 color_height:=720 color_width:=1280">
+    <!-- Load parameters to model's main link-->
+    <xacro:property name="deg_to_rad" value="0.01745329251994329577" />
+    <gazebo reference="${reference_link}">
+      <self_collide>0</self_collide>
+      <enable_wind>0</enable_wind>
+      <kinematic>0</kinematic>
+      <gravity>1</gravity>
+      <!--<mu>1</mu>-->
+      <mu2>1</mu2>
+      <fdir1>0 0 0</fdir1>
+      <!--<slip1>0</slip1>
+      <slip2>0</slip2>-->
+      <kp>1e+13</kp>
+      <kd>1</kd>
+      <!--<max_vel>0.01</max_vel>
+      <min_depth>0</min_depth>-->
+      <sensor name="${camera_name}color" type="camera">
+        <camera name="${camera_name}">
+          <horizontal_fov>${69.4*deg_to_rad}</horizontal_fov>
           <image>
-            <format>B8G8R8</format>
             <width>${color_width}</width>
             <height>${color_height}</height>
+            <format>RGB_INT8</format>
           </image>
           <clip>
-            <near>0.2</near>
-            <far>10.0</far>
+            <near>0.1</near>
+            <far>100</far>
           </clip>
           <noise>
             <type>gaussian</type>
             <mean>0.0</mean>
-            <stddev>0.0</stddev>
+            <stddev>0.007</stddev>
           </noise>
         </camera>
-        <plugin name="${name}_frame_controller" filename="libgazebo_ros_depth_camera.so">
-          <updateRate>${color_fps}</updateRate>
-          <cameraName>${name}</cameraName>
-          <frameName>${name}_color_optical_frame</frameName>
-          <imageTopicName>rgb/image_raw</imageTopicName>
-          <cameraInfoTopicName>rgb/camera_info</cameraInfoTopicName>
-          <pointCloudTopicName>depth/points</pointCloudTopicName>
-          <depthImageTopicName>depth/image_raw</depthImageTopicName>
-          <depthImageCameraInfoTopicName>depth/camera_info</depthImageCameraInfoTopicName>
-          <pointCloudCutoff>0.2</pointCloudCutoff>
-          <pointCloudCutoffMax>5.0</pointCloudCutoffMax>
-          <distortionK1>0.0</distortionK1>
-          <distortionK2>0.0</distortionK2>
-          <distortionK3>0.0</distortionK3>
-          <distortionT1>0.0</distortionT1>
-          <distortionT2>0.0</distortionT2>
-          <CxPrime>0.0</CxPrime>
-          <Cx>0.0</Cx>
-          <Cy>0.0</Cy>
-          <focalLength>0.0</focalLength>
-        </plugin>
+        <always_on>1</always_on>
+        <update_rate>${color_fps}</update_rate>
+        <visualize>1</visualize>
       </sensor>
-      <!-- ToDo: add plugins for IMU, Fisheye, IR -->
-      <material>IPA/LightGrey</material>
+      <sensor name="${camera_name}ired1" type="camera">
+        <camera name="${camera_name}">
+          <horizontal_fov>${85.2*deg_to_rad}</horizontal_fov>
+          <image>
+            <width>${depth_width}</width>
+            <height>${depth_height}</height>
+            <format>L_INT8</format>
+          </image>
+          <clip>
+            <near>0.1</near>
+            <far>100</far>
+          </clip>
+          <noise>
+            <type>gaussian</type>
+            <mean>0.0</mean>
+            <stddev>0.05</stddev>
+          </noise>
+        </camera>
+        <always_on>1</always_on>
+        <update_rate>${depth_fps}</update_rate>
+        <visualize>0</visualize>
+      </sensor>
+      <sensor name="${camera_name}ired2" type="camera">
+        <camera name="${camera_name}">
+          <horizontal_fov>${85.2*deg_to_rad}</horizontal_fov>
+          <image>
+            <width>${depth_width}</width>
+            <height>${depth_height}</height>
+            <format>L_INT8</format>
+          </image>
+          <clip>
+            <near>0.1</near>
+            <far>100</far>
+          </clip>
+          <noise>
+            <type>gaussian</type>
+            <mean>0.0</mean>
+            <stddev>0.05</stddev>
+          </noise>
+        </camera>
+        <always_on>1</always_on>
+        <update_rate>${depth_fps}</update_rate>
+        <visualize>0</visualize>
+      </sensor>
+      <sensor name="${camera_name}depth" type="depth">
+        <camera name="${camera_name}">
+          <horizontal_fov>${85.2*deg_to_rad}</horizontal_fov>
+          <image>
+            <width>${depth_width}</width>
+            <height>${depth_height}</height>
+          </image>
+          <clip>
+            <near>0.1</near>
+            <far>100</far>
+          </clip>
+          <noise>
+            <type>gaussian</type>
+            <mean>0.0</mean>
+            <stddev>0.100</stddev>
+          </noise>
+        </camera>
+        <always_on>1</always_on>
+        <update_rate>${depth_fps}</update_rate>
+        <visualize>1</visualize>
+      </sensor>
+    </gazebo>
+    <gazebo>
+      <plugin name="${topics_ns}" filename="librealsense_gazebo_plugin.so">
+        <prefix>${camera_name}</prefix>
+        <depthUpdateRate>${depth_fps}</depthUpdateRate>
+        <colorUpdateRate>${color_fps}</colorUpdateRate>
+        <infraredUpdateRate>${depth_fps}</infraredUpdateRate>
+      	<depthTopicName>depth/image_raw</depthTopicName>
+      	<depthCameraInfoTopicName>depth/camera_info</depthCameraInfoTopicName>
+        <colorTopicName>rgb/image_raw</colorTopicName>
+        <colorCameraInfoTopicName>rgb/camera_info</colorCameraInfoTopicName>
+      	<infrared1TopicName>infra1/image_raw</infrared1TopicName>
+      	<infrared1CameraInfoTopicName>infra1/camera_info</infrared1CameraInfoTopicName>
+      	<infrared2TopicName>infra2/image_raw</infrared2TopicName>
+      	<infrared2CameraInfoTopicName>infra2/camera_info</infrared2CameraInfoTopicName>
+      	<colorOpticalframeName>${color_optical_frame}</colorOpticalframeName>
+      	<depthOpticalframeName>${depth_optical_frame}</depthOpticalframeName>
+      	<infrared1OpticalframeName>${infrared1_optical_frame}</infrared1OpticalframeName>
+      	<infrared2OpticalframeName>${infrared2_optical_frame}</infrared2OpticalframeName>
+      	<rangeMinDepth>0.2</rangeMinDepth>
+      	<rangeMaxDepth>10.0</rangeMaxDepth>
+        <pointCloud>true</pointCloud>
+      	<pointCloudTopicName>depth/points</pointCloudTopicName>
+      	<pointCloudCutoff>0.5</pointCloudCutoff>
+      </plugin>
     </gazebo>
   </xacro:macro>

File: cob_description/urdf/sensors/realsense_d435.urdf.xacro (robot description, xacro)
@@ -2,6 +2,5 @@
 <robot xmlns:xacro="http://www.ros.org/wiki/xacro">
   <xacro:include filename="$(find cob_description)/urdf/common.xacro" />
-  <!--xacro:include filename="$(find cob_description)/urdf/sensors/realsense_d435.gazebo.xacro" /-->
-  <xacro:include filename="$(find cob_description)/urdf/sensors/realsense_d435_pal.gazebo.xacro" />
+  <xacro:include filename="$(find cob_description)/urdf/sensors/realsense_d435.gazebo.xacro" />
   <xacro:macro name="realsense_d435" params="name parent *origin">
     <joint name="${name}_mount_joint" type="fixed">
