Commit message: additional links on tray

File: cob_description/urdf/tray/tray.urdf.xacro (robot description, xacro)
@@ -37,4 +37,23 @@
 			</collision>
 		</link>
+		<!-- additional links at the corners of the tray -->
+		<joint name="${name}_base_joint" type="fixed" >
+			<origin xyz="0 0 0" rpy="-2.3561 0 0"/>
+			<parent link="${name}_link" />
+			<child link="${name}_base_link" />
+		</joint>
+		<link name="${name}_base_link"/>
+		<joint name="${name}_right_joint" type="fixed" >
+			<origin xyz="0.4 -0.3 0.1" rpy="0 0 0"/>
+			<parent link="${name}_base_link" />
+			<child link="${name}_right_link" />
+		</joint>
+		<link name="${name}_right_link"/>
+		<joint name="${name}_left_joint" type="fixed" >
+			<origin xyz="0.4 0.05 0.1" rpy="0 0 0"/>
+			<parent link="${name}_base_link" />
+			<child link="${name}_left_link" />
+		</joint>
+		<link name="${name}_left_link"/>
 		<!-- extensions -->
 		<xacro:cob_tray_gazebo name="${name}" />

Commit message: add simulated phidgets sensors to tray

File: cob_description/urdf/tray/tray.urdf.xacro (robot description, xacro)
@@ -6,4 +6,5 @@
 	<include filename="$(find cob_description)/urdf/tray/tray.gazebo.xacro" />
 	<include filename="$(find cob_description)/urdf/tray/tray.transmission.xacro" />
+	<include filename="$(find cob_description)/urdf/sensors/phidgets_distance.urdf.xacro" />
 	<xacro:macro name="cob_tray" params="name parent *origin">
 		<!-- joint between base_link and tray_link -->
@@ -43,5 +44,24 @@
 			<child link="${name}_base_link" />
 		</joint>
-		<link name="${name}_base_link"/>
+		<link name="${name}_base_link">
+			<inertial>
+				<mass value="0.001" />
+				<origin xyz="0 0 0" rpy="0 0 0" />
+				<inertia ixx="0.0001" ixy="0" ixz="0" iyy="0.000001" iyz="0" izz="0.0001" />
+			</inertial>
+			<visual>
+				<origin xyz="0 0 0" rpy="0 0 0" />
+				<geometry>
+					<box size="0.001 0.001 0.001" />
+				</geometry>
+				<material name="Red" />
+			</visual>
+			<collision>
+				<origin xyz="0 0 0" rpy="0 0 0" />
+				<geometry>
+					<box size=".001 .001 .001" />
+				</geometry>
+			</collision>
+		</link>
 		<joint name="${name}_right_joint" type="fixed" >
 			<origin xyz="0.4 -0.3 0.1" rpy="0 0 0"/>
@@ -49,5 +69,24 @@
 			<child link="${name}_right_link" />
 		</joint>
-		<link name="${name}_right_link"/>
+		<link name="${name}_right_link">
+			<inertial>
+				<mass value="0.001" />
+				<origin xyz="0 0 0" rpy="0 0 0" />
+				<inertia ixx="0.0001" ixy="0" ixz="0" iyy="0.000001" iyz="0" izz="0.0001" />
+			</inertial>
+			<visual>
+				<origin xyz="0 0 0" rpy="0 0 0" />
+				<geometry>
+					<box size="0.001 0.001 0.001" />
+				</geometry>
+				<material name="Red" />
+			</visual>
+			<collision>
+				<origin xyz="0 0 0" rpy="0 0 0" />
+				<geometry>
+					<box size=".001 .001 .001" />
+				</geometry>
+			</collision>
+		</link>
 		<joint name="${name}_left_joint" type="fixed" >
 			<origin xyz="0.4 0.05 0.1" rpy="0 0 0"/>
@@ -55,5 +94,37 @@
 			<child link="${name}_left_link" />
 		</joint>
-		<link name="${name}_left_link"/>
+		<link name="${name}_left_link">
+			<inertial>
+				<mass value="0.001" />
+				<origin xyz="0 0 0" rpy="0 0 0" />
+				<inertia ixx="0.0001" ixy="0" ixz="0" iyy="0.000001" iyz="0" izz="0.0001" />
+			</inertial>
+			<visual>
+				<origin xyz="0 0 0" rpy="0 0 0" />
+				<geometry>
+					<box size="0.001 0.001 0.001" />
+				</geometry>
+				<material name="Red" />
+			</visual>
+			<collision>
+				<origin xyz="0 0 0" rpy="0 0 0" />
+				<geometry>
+					<box size=".001 .001 .001" />
+				</geometry>
+			</collision>
+		</link>
+		<!-- phidgets distance sensors -->
+		<xacro:phidgets_distance_v0 name="${name}_phidgets_1" ros_topic="/tray_sensors/range_1_sim" update_rate="10" parent="${name}_left">
+			<origin xyz="-0.275 0 0.02" rpy="0 0 ${-M_PI/2}" />
+		</xacro:phidgets_distance_v0>
+		<xacro:phidgets_distance_v0 name="${name}_phidgets_2" ros_topic="/tray_sensors/range_2_sim" update_rate="10" parent="${name}_left">
+			<origin xyz="-0.2 0 0.02" rpy="0 0 ${-M_PI/2}" />
+		</xacro:phidgets_distance_v0>
+		<xacro:phidgets_distance_v0 name="${name}_phidgets_3" ros_topic="/tray_sensors/range_3_sim" update_rate="10" parent="${name}_left">
+			<origin xyz="-0.125 0 0.02" rpy="0 0 ${-M_PI/2}" />
+		</xacro:phidgets_distance_v0>
+		<xacro:phidgets_distance_v0 name="${name}_phidgets_4" ros_topic="/tray_sensors/range_4_sim" update_rate="10" parent="${name}_left">
+			<origin xyz="-0.05 0 0.02" rpy="0 0 ${-M_PI/2}" />
+		</xacro:phidgets_distance_v0>
 		<!-- extensions -->
 		<xacro:cob_tray_gazebo name="${name}" />
