Commit message: update urdf

File: cob_description/urdf/head_v2/head.urdf.xacro (robot description, xacro)
@@ -8,5 +8,4 @@
 	<include filename="$(find cob_description)/urdf/sensors/prosilica.urdf.xacro" />
 	<include filename="$(find cob_description)/urdf/sensors/kinect.urdf.xacro" />
-	<!--include filename="$(find cob_description)/urdf/sensors/hokuyo_SR400_laser.urdf.xacro" /-->
 	<xacro:macro name="cob_head_v2" params="name parent *origin">
 		<!-- joint between torso_upper_neck_tilt_link and head_axis_link -->
@@ -18,5 +17,5 @@
 			<dynamics damping="0.1" />
 			<calibration rising="${head_axis_ref}"/>
-			<limit effort="100" lower="-3.2" upper="0.1" velocity="0.5"/>
+			<limit effort="100" lower="-3.2" upper="0.1" velocity="1.4"/>
 		</joint>
 		<link name="${name}_axis_link">
@@ -42,13 +41,13 @@
 		<!-- left camera -->
 		<xacro:cob_prosilica_v0 name="${name}_color_camera_l" ros_topic="stereo/left" parent="${name}_axis_link">
-			<origin xyz="${cam_l_x} ${cam_l_y} ${cam_l_z-0.06}" rpy="${cam_l_roll} ${cam_l_pitch+M_PI/2} ${cam_l_yaw+M_PI}" />
+			<origin xyz="${cam_l_x} ${cam_l_y} ${cam_l_z}" rpy="${cam_l_roll} ${cam_l_pitch} ${cam_l_yaw}" />
 		</xacro:cob_prosilica_v0>
 		<!-- right camera -->
 		<xacro:cob_prosilica_v0 name="${name}_color_camera_r" ros_topic="stereo/right" parent="${name}_color_camera_l_link">
-			<origin xyz="${cam_r_x-0.12} ${cam_r_y} ${cam_r_z}" rpy="${cam_r_roll} ${cam_r_pitch} ${cam_r_yaw}" />
+			<origin xyz="${cam_r_x} ${cam_r_y} ${cam_r_z}" rpy="${cam_r_roll} ${cam_r_pitch} ${cam_r_yaw}" />
 		</xacro:cob_prosilica_v0>
 		<!-- cam3d -->
-		<xacro:cob_kinect_v0 name="${name}_cam3d" ros_topic="cam3d/depth/points1" parent="${name}_color_camera_l_link">
-			<origin xyz="${cam3d_x-0.06} ${cam3d_y} ${cam3d_z}" rpy="${cam3d_roll} ${cam3d_pitch} ${cam3d_yaw+M_PI}" />
+		<xacro:cob_kinect_v0 name="${name}_cam3d" ros_topic="cam3d" parent="${name}_axis_link">
+			<origin xyz="${cam3d_x} ${cam3d_y} ${cam3d_z}" rpy="${cam3d_roll} ${cam3d_pitch} ${cam3d_yaw}" />
 		</xacro:cob_kinect_v0>
 		<!-- extensions -->
