Commit message: changed torso back to working version from robot, renamed joints

File: raw_description/urdf/torso/torso.gazebo.xacro (robot description, xacro)
@@ -4,15 +4,23 @@
        xmlns:interface="http://playerstage.sourceforge.net/gazebo/xmlschema/#interface"
        xmlns:xacro="http://ros.org/wiki/xacro">
-	<xacro:macro name="raw_torso_gazebo" params="name">
-		<gazebo reference="${name}_0_link">
+	<xacro:macro name="cob_torso_gazebo_v1" params="name">
+		<gazebo reference="${name}_tray_link">
+			<material>Gazebo/Green</material>
+			<turnGravityOff>false</turnGravityOff>
+		</gazebo>
+		<gazebo reference="${name}_lower_neck_tilt_link">
+			<material>Gazebo/Red</material>
+			<turnGravityOff>false</turnGravityOff>
+		</gazebo>
+		<gazebo reference="${name}_pan_link">
+			<material>Gazebo/Blue</material>
+			<turnGravityOff>false</turnGravityOff>
+		</gazebo>
+		<gazebo reference="${name}_upper_neck_tilt_link">
 			<material>Gazebo/Grey</material>
 			<turnGravityOff>false</turnGravityOff>
 		</gazebo>
-		<gazebo reference="${name}_tilt_link">
-			<material>Gazebo/Grey</material>
-			<turnGravityOff>false</turnGravityOff>
-		</gazebo>
-		<gazebo reference="head_axis_link">
-			<material>Gazebo/Grey</material>
+		<gazebo reference="head_cover_link">
+			<material>Gazebo/Blue</material>
 			<turnGravityOff>false</turnGravityOff>
 		</gazebo>

File: raw_description/urdf/torso/torso.transmission.xacro (robot description, xacro)
@@ -4,13 +4,23 @@
        xmlns:interface="http://playerstage.sourceforge.net/gazebo/xmlschema/#interface"
        xmlns:xacro="http://ros.org/wiki/xacro">
-	<xacro:macro name="raw_torso_transmission" params="name">
-		<transmission name="${name}_tilt_trans" type="pr2_mechanism_model/SimpleTransmission">
-			<actuator name="${name}_tilt_motor"/>
-			<joint name="${name}_tilt_joint"/>
+	<xacro:macro name="cob_torso_transmission_v1" params="name">
+		<transmission name="${name}_tray_trans" type="pr2_mechanism_model/SimpleTransmission">
+			<actuator name="${name}_tray_motor"/>
+			<joint name="${name}_tray_joint"/>
 			<mechanicalReduction>1</mechanicalReduction>
 		</transmission>
-		<transmission name="head_axis_trans" type="pr2_mechanism_model/SimpleTransmission">
-			<actuator name="head_axis_motor"/>
-			<joint name="head_axis_joint"/>
+		<transmission name="${name}_lower_neck_tilt_trans" type="pr2_mechanism_model/SimpleTransmission">
+			<actuator name="${name}_lower_neck_tilt_motor"/>
+			<joint name="${name}_lower_neck_tilt_joint"/>
+			<mechanicalReduction>1</mechanicalReduction>
+		</transmission>
+		<transmission name="${name}_pan_trans" type="pr2_mechanism_model/SimpleTransmission">
+			<actuator name="${name}_pan_motor"/>
+			<joint name="${name}_pan_joint"/>
+			<mechanicalReduction>1</mechanicalReduction>
+		</transmission>
+		<transmission name="${name}_upper_neck_tilt_trans" type="pr2_mechanism_model/SimpleTransmission">
+			<actuator name="${name}_upper_neck_tilt_motor"/>
+			<joint name="${name}_upper_neck_tilt_joint"/>
 			<mechanicalReduction>1</mechanicalReduction>
 		</transmission>

File: raw_description/urdf/torso/torso.urdf.xacro (robot description, xacro)
@@ -8,5 +8,5 @@
 	<include filename="$(find cob_description)/urdf/sensors/prosilica.urdf.xacro" />
 	<include filename="$(find cob_description)/urdf/sensors/kinect.urdf.xacro" />
-	<xacro:macro name="raw_torso" params="name parent *origin">
+	<xacro:macro name="cob_torso_v1" params="name parent *origin">
 		<!-- joint between base_link and torso_tilt_link -->
 		<joint name="${name}_0_joint" type="fixed" >
@@ -22,5 +22,5 @@
 			</inertial>
 			<visual>
-				<origin xyz="0 0 -0.26" rpy="0 0 0" />
+				<origin xyz="0 0 0" rpy="0 0 0" />
 				<geometry>
 					<cylinder length="0.521" radius="0.04"/>
@@ -29,5 +29,5 @@
 			</visual>
 			<collision>
-				<origin xyz="0 0 -0.26" rpy="0 0 0" />
+				<origin xyz="0 0 0" rpy="0 0 0" />
 				<geometry>
 					<cylinder length="0.521" radius="0.04"/>
@@ -36,8 +36,8 @@
 		</link>
 		<!-- joint between base_link and torso_lower_neck_tilt_link -->
-		<joint name="${name}_tilt_joint" type="revolute">
+		<joint name="${name}_pan_joint" type="revolute">
 			<origin xyz="0.0 0.0 0.3074" rpy="0.0 0.0 -0.48" />
 			<parent link="${name}_0_link"/>
-			<child link="${name}_tilt_link"/>
+			<child link="${name}_1_link"/>
 			<axis xyz="0 0 -1.0" />
 			<dynamics damping="25.0" friction="10.0"/>
@@ -45,5 +45,5 @@
 			<limit effort="41.4" lower="-6.2831" upper="6.2831" velocity="0.5"/>
 		</joint>
-		<link name="${name}_tilt_link">
+		<link name="${name}_1_link">
 			<inertial>
 				<origin xyz="0 0 0" rpy="0 0 0"/>
@@ -66,8 +66,8 @@
 		</link>
 		<!-- joint between torso_upper_neck_tilt_link and head_axis_link -->
-		<joint name="head_axis_joint" type="revolute">
+		<joint name="torso_tilt_joint" type="revolute">
 			<origin xyz="0.0 0.0 0.047" rpy="0.0 0.0 0.0" />
-   			<parent link="${name}_tilt_link"/>
-			<child link="head_axis_link"/>
+   			<parent link="${name}_1_link"/>
+			<child link="torso_2_link"/>
 			<axis xyz="0 0 -1.0" />
 			<dynamics damping="0.1" />
@@ -75,5 +75,5 @@
 			<limit effort="100" lower="-3.2" upper="0.1" velocity="1.4"/>
 		</joint>
-		<link name="head_axis_link">
+		<link name="torso_2_link">
 			<inertial>
 				<origin xyz="0 0 0" rpy="0 0 0"/>
@@ -96,18 +96,18 @@
 		</link>
 		<!-- left camera -->
-		<xacro:cob_prosilica_v0 name="head_color_camera_l" ros_topic="stereo/left" parent="head_axis_link">
+		<xacro:cob_prosilica_v0 name="head_color_camera_l" ros_topic="stereo/left" parent="torso_2_link">
 			<origin xyz="${cam_l_x} ${cam_l_y} ${cam_l_z}" rpy="${cam_l_roll} ${cam_l_pitch} ${cam_l_yaw}" />
 		</xacro:cob_prosilica_v0>
 		<!-- right camera -->
-		<xacro:cob_prosilica_v0 name="head_color_camera_r" ros_topic="stereo/right" parent="head_axis_link">
+		<xacro:cob_prosilica_v0 name="head_color_camera_r" ros_topic="stereo/right" parent="torso_2_link">
 			<origin xyz="${cam_r_x} ${cam_r_y} ${cam_r_z}" rpy="${cam_r_roll} ${cam_r_pitch} ${cam_r_yaw}" />
 		</xacro:cob_prosilica_v0>
 		<!-- cam3d -->
-		<xacro:cob_kinect_v0 name="head_cam3d" ros_topic="cam3d" parent="head_axis_link">
+		<xacro:cob_kinect_v0 name="head_cam3d" ros_topic="cam3d" parent="torso_2_link">
 			<origin xyz="${cam3d_x} ${cam3d_y} ${cam3d_z}" rpy="${cam3d_roll} ${cam3d_pitch} ${cam3d_yaw}" />
 		</xacro:cob_kinect_v0>
 		<!-- extensions -->
-		<xacro:raw_torso_gazebo name="${name}" />
-		<xacro:raw_torso_transmission name="${name}" />
+		<xacro:cob_torso_gazebo_v1 name="${name}" />
+		<xacro:cob_torso_transmission_v1 name="${name}" />
 	</xacro:macro>
 </robot>

Commit message: changed names from cob to raw and adapted gazebo and transmission files

File: raw_description/urdf/torso/torso.gazebo.xacro (robot description, xacro)
@@ -4,23 +4,11 @@
        xmlns:interface="http://playerstage.sourceforge.net/gazebo/xmlschema/#interface"
        xmlns:xacro="http://ros.org/wiki/xacro">
-	<xacro:macro name="cob_torso_gazebo_v1" params="name">
-		<gazebo reference="${name}_tray_link">
-			<material>Gazebo/Green</material>
-			<turnGravityOff>false</turnGravityOff>
-		</gazebo>
-		<gazebo reference="${name}_lower_neck_tilt_link">
-			<material>Gazebo/Red</material>
-			<turnGravityOff>false</turnGravityOff>
-		</gazebo>
+	<xacro:macro name="raw_torso_gazebo" params="name">
 		<gazebo reference="${name}_pan_link">
 			<material>Gazebo/Blue</material>
 			<turnGravityOff>false</turnGravityOff>
 		</gazebo>
-		<gazebo reference="${name}_upper_neck_tilt_link">
+		<gazebo reference="${name}_tilt_link">
 			<material>Gazebo/Grey</material>
-			<turnGravityOff>false</turnGravityOff>
-		</gazebo>
-		<gazebo reference="head_cover_link">
-			<material>Gazebo/Blue</material>
 			<turnGravityOff>false</turnGravityOff>
 		</gazebo>

File: raw_description/urdf/torso/torso.transmission.xacro (robot description, xacro)
@@ -4,15 +4,5 @@
        xmlns:interface="http://playerstage.sourceforge.net/gazebo/xmlschema/#interface"
        xmlns:xacro="http://ros.org/wiki/xacro">
-	<xacro:macro name="cob_torso_transmission_v1" params="name">
-		<transmission name="${name}_tray_trans" type="pr2_mechanism_model/SimpleTransmission">
-			<actuator name="${name}_tray_motor"/>
-			<joint name="${name}_tray_joint"/>
-			<mechanicalReduction>1</mechanicalReduction>
-		</transmission>
-		<transmission name="${name}_lower_neck_tilt_trans" type="pr2_mechanism_model/SimpleTransmission">
-			<actuator name="${name}_lower_neck_tilt_motor"/>
-			<joint name="${name}_lower_neck_tilt_joint"/>
-			<mechanicalReduction>1</mechanicalReduction>
-		</transmission>
+	<xacro:macro name="raw_torso_transmission" params="name">
 		<transmission name="${name}_pan_trans" type="pr2_mechanism_model/SimpleTransmission">
 			<actuator name="${name}_pan_motor"/>
@@ -20,7 +10,7 @@
 			<mechanicalReduction>1</mechanicalReduction>
 		</transmission>
-		<transmission name="${name}_upper_neck_tilt_trans" type="pr2_mechanism_model/SimpleTransmission">
-			<actuator name="${name}_upper_neck_tilt_motor"/>
-			<joint name="${name}_upper_neck_tilt_joint"/>
+		<transmission name="${name}__tilt_trans" type="pr2_mechanism_model/SimpleTransmission">
+			<actuator name="${name}__tilt_motor"/>
+			<joint name="${name}_tilt_joint"/>
 			<mechanicalReduction>1</mechanicalReduction>
 		</transmission>

File: raw_description/urdf/torso/torso.urdf.xacro (robot description, xacro)
@@ -8,5 +8,5 @@
 	<include filename="$(find cob_description)/urdf/sensors/prosilica.urdf.xacro" />
 	<include filename="$(find cob_description)/urdf/sensors/kinect.urdf.xacro" />
-	<xacro:macro name="cob_torso_v1" params="name parent *origin">
+	<xacro:macro name="raw_torso" params="name parent *origin">
 		<!-- joint between base_link and torso_tilt_link -->
 		<joint name="${name}_0_joint" type="fixed" >
@@ -108,6 +108,6 @@
 		</xacro:cob_kinect_v0>
 		<!-- extensions -->
-		<xacro:cob_torso_gazebo_v1 name="${name}" />
-		<xacro:cob_torso_transmission_v1 name="${name}" />
+		<xacro:raw_torso_gazebo name="${name}" />
+		<xacro:raw_torso_transmission name="${name}" />
 	</xacro:macro>
 </robot>
