Commit message: changes for raw

File: raw_description/urdf/torso/torso.urdf.xacro (robot description, xacro)
@@ -6,16 +6,44 @@
 	<include filename="$(find raw_description)/urdf/torso/torso.gazebo.xacro" />
 	<include filename="$(find raw_description)/urdf/torso/torso.transmission.xacro" />
+	<include filename="$(find cob_description)/urdf/sensors/prosilica.urdf.xacro" />
+	<include filename="$(find cob_description)/urdf/sensors/kinect.urdf.xacro" />
 	<xacro:macro name="cob_torso_v1" params="name parent *origin">
+		<!-- joint between base_link and torso_tilt_link -->
+		<joint name="${name}_0_joint" type="fixed" >
+			<insert_block name="origin" />
+			<parent link="${parent}" />
+			<child link="${name}_0_link" />
+		</joint>
+		<link name="${name}_0_link">
+			<inertial>
+				<origin xyz="0 0 0" rpy="0 0 0"/>
+				<mass value="0.57307"/>
+				<inertia ixx="1.415" ixy="0" ixz="0" iyy="0.819" iyz="0" izz="0.819" />
+			</inertial>
+			<visual>
+				<origin xyz="0 0 0" rpy="0 0 0" />
+				<geometry>
+					<cylinder length="0.521" radius="0.04"/>
+				</geometry>
+				<material name="Grey" />
+			</visual>
+			<collision>
+				<origin xyz="0 0 0" rpy="0 0 0" />
+				<geometry>
+					<cylinder length="0.521" radius="0.04"/>
+				</geometry>
+			</collision>
+		</link>
 		<!-- joint between base_link and torso_lower_neck_tilt_link -->
-		<joint name="${name}_lower_neck_tilt_joint" type="revolute">
-			<insert_block name="origin" />
-			<parent link="${parent}"/>
-			<child link="${name}_lower_neck_tilt_link"/>
+		<joint name="${name}_tilt_joint" type="revolute">
+			<origin xyz="0.0 0.0 0.3074" rpy="0.0 0.0 0.0" />
+			<parent link="${name}_0_link"/>
+			<child link="${name}_tilt_link"/>
 			<axis xyz="0 0 1" />
 			<dynamics damping="25.0" friction="10.0"/>
-			<calibration rising="${torso_lower_neck_tilt_ref}"/>
+			<calibration rising="0.0"/>
 			<limit effort="41.4" lower="-6.2831" upper="6.2831" velocity="0.5"/>
 		</joint>
-		<link name="${name}_lower_neck_tilt_link">
+		<link name="${name}_tilt_link">
 			<inertial>
 				<origin xyz="0 0 0" rpy="0 0 0"/>
@@ -26,5 +54,5 @@
 				<origin xyz="0 0 0" rpy="3.14 0 0" />
 				<geometry>
-					<mesh filename="package://cob_description/meshes/torso_v0/lower_neck.stl" />
+					<cylinder length="0.1" radius="0.1"/>
 				</geometry>
 				<material name="Red" />
@@ -33,38 +61,50 @@
 				<origin xyz="0 0 0" rpy="3.14 0 0" />
 				<geometry>
-					<mesh filename="package://cob_description/meshes/torso_v0/lower_neck_collision.stlb" />
+					<cylinder length="0.1" radius="0.1"/>
 				</geometry>
 			</collision>
 		</link>
-		<!-- joint between torso_lower_neck_tilt_link and torso_pan_link -->
-		<joint name="${name}_pan_joint" type="revolute">
-			<origin xyz="0 0 0" rpy="1.5708 0 0" />
-			<parent link="${name}_lower_neck_tilt_link"/>
-			<child link="${name}_pan_link"/>
+		<!-- joint between torso_upper_neck_tilt_link and head_axis_link -->
+		<joint name="head_axis_joint" type="revolute">
+			<origin xyz="0.0 0.0 0.0" rpy="0.0 0.0 0.0" />
+   			<parent link="${name}_tilt_link"/>
+			<child link="head_axis_link"/>
 			<axis xyz="0 0 1" />
-			<dynamics damping="25.0" friction="10.0"/>
-			<calibration rising="${torso_pan_ref}"/>
-			<limit effort="41.4" lower="-6.2831" upper="6.2831" velocity="0.5"/>
+			<dynamics damping="0.1" />
+			<calibration rising="0.0"/>
+			<limit effort="100" lower="-3.2" upper="0.1" velocity="1.4"/>
 		</joint>
-		<link name="${name}_pan_link">
+		<link name="head_axis_link">
 			<inertial>
 				<origin xyz="0 0 0" rpy="0 0 0"/>
-				<mass value="1.0"/>
-				<inertia ixx="0.200549" ixy="0.001322" ixz="-0.000000" iyy="0.123664" iyz="-0.000000" izz="0.104101" />
+				<mass value="0.1"/>
+				<inertia ixx="0.0001" ixy="0" ixz="0" iyy="0.0001" iyz="0" izz="0.0001" />
 			</inertial>
 			<visual>
-				<origin xyz="0 0 0.005" rpy="0 0 0" />
+				<origin xyz="0 0 0" rpy="0 0 0" />
 				<geometry>
 					<box size="0.01 0.01 0.01"/>
 				</geometry>
-				<material name="Blue" />
+				<material name="Green" />
 			</visual>
 			<collision>
-				<origin xyz="0 0 0.0005" rpy="0 0 0" />
+				<origin xyz="0 0 0" rpy="0 0 0" />
 				<geometry>
-					<box size="0.001 0.001 0.001"/>
+					<box size="0.01 0.01 0.01"/>
 				</geometry>
 			</collision>
 		</link>
+		<!-- left camera -->
+		<xacro:cob_prosilica_v0 name="${name}_color_camera_l" ros_topic="stereo/left" parent="head_axis_link">
+			<origin xyz="${cam_l_x} ${cam_l_y} ${cam_l_z}" rpy="${cam_l_roll} ${cam_l_pitch} ${cam_l_yaw}" />
+		</xacro:cob_prosilica_v0>
+		<!-- right camera -->
+		<xacro:cob_prosilica_v0 name="${name}_color_camera_r" ros_topic="stereo/right" parent="${name}_color_camera_l_link">
+			<origin xyz="${cam_r_x} ${cam_r_y} ${cam_r_z}" rpy="${cam_r_roll} ${cam_r_pitch} ${cam_r_yaw}" />
+		</xacro:cob_prosilica_v0>
+		<!-- cam3d -->
+		<xacro:cob_kinect_v0 name="${name}_cam3d" ros_topic="cam3d" parent="head_axis_link">
+			<origin xyz="${cam3d_x} ${cam3d_y} ${cam3d_z}" rpy="${cam3d_roll} ${cam3d_pitch} ${cam3d_yaw}" />
+		</xacro:cob_kinect_v0>
 		<!-- extensions -->
 		<xacro:cob_torso_gazebo_v1 name="${name}" />

Commit message: small urdf bugfix

File: raw_description/urdf/torso/torso.urdf.xacro (robot description, xacro)
@@ -37,8 +37,8 @@
 		<!-- joint between base_link and torso_lower_neck_tilt_link -->
 		<joint name="${name}_tilt_joint" type="revolute">
-			<origin xyz="0.0 0.0 0.3074" rpy="0.0 0.0 0.0" />
+			<origin xyz="0.0 0.0 0.3074" rpy="0.0 0.0 -0.48" />
 			<parent link="${name}_0_link"/>
 			<child link="${name}_tilt_link"/>
-			<axis xyz="0 0 1" />
+			<axis xyz="0 0 -1.0" />
 			<dynamics damping="25.0" friction="10.0"/>
 			<calibration rising="0.0"/>
@@ -67,8 +67,8 @@
 		<!-- joint between torso_upper_neck_tilt_link and head_axis_link -->
 		<joint name="head_axis_joint" type="revolute">
-			<origin xyz="0.0 0.0 0.0" rpy="0.0 0.0 0.0" />
+			<origin xyz="0.0 0.0 0.047" rpy="0.0 0.0 0.0" />
    			<parent link="${name}_tilt_link"/>
 			<child link="head_axis_link"/>
-			<axis xyz="0 0 1" />
+			<axis xyz="0 0 -1.0" />
 			<dynamics damping="0.1" />
 			<calibration rising="0.0"/>
@@ -96,13 +96,13 @@
 		</link>
 		<!-- left camera -->
-		<xacro:cob_prosilica_v0 name="${name}_color_camera_l" ros_topic="stereo/left" parent="head_axis_link">
+		<xacro:cob_prosilica_v0 name="head_color_camera_l" ros_topic="stereo/left" parent="head_axis_link">
 			<origin xyz="${cam_l_x} ${cam_l_y} ${cam_l_z}" rpy="${cam_l_roll} ${cam_l_pitch} ${cam_l_yaw}" />
 		</xacro:cob_prosilica_v0>
 		<!-- right camera -->
-		<xacro:cob_prosilica_v0 name="${name}_color_camera_r" ros_topic="stereo/right" parent="${name}_color_camera_l_link">
+		<xacro:cob_prosilica_v0 name="head_color_camera_r" ros_topic="stereo/right" parent="head_axis_link">
 			<origin xyz="${cam_r_x} ${cam_r_y} ${cam_r_z}" rpy="${cam_r_roll} ${cam_r_pitch} ${cam_r_yaw}" />
 		</xacro:cob_prosilica_v0>
 		<!-- cam3d -->
-		<xacro:cob_kinect_v0 name="${name}_cam3d" ros_topic="cam3d" parent="head_axis_link">
+		<xacro:cob_kinect_v0 name="head_cam3d" ros_topic="cam3d" parent="head_axis_link">
 			<origin xyz="${cam3d_x} ${cam3d_y} ${cam3d_z}" rpy="${cam3d_roll} ${cam3d_pitch} ${cam3d_yaw}" />
 		</xacro:cob_kinect_v0>

Commit message: changed limit of torso tilt

File: raw_description/urdf/torso/torso.urdf.xacro (robot description, xacro)
@@ -73,5 +73,5 @@
 			<dynamics damping="0.1" />
 			<calibration rising="0.0"/>
-			<limit effort="100" lower="-3.2" upper="0.1" velocity="1.4"/>
+			<limit effort="100" lower="-3.2" upper="1.57" velocity="1.4"/>
 		</joint>
 		<link name="torso_2_link">

Commit message: raw torso calibration

File: raw_description/urdf/torso/torso.urdf.xacro (robot description, xacro)
@@ -37,10 +37,10 @@
 		<!-- joint between base_link and torso_lower_neck_tilt_link -->
 		<joint name="${name}_pan_joint" type="revolute">
-			<origin xyz="0.0 0.0 0.3074" rpy="0.0 0.0 -0.48" />
+			<origin xyz="0.0 0.0 0.3074" rpy="0.0 0.0 0.0" />
 			<parent link="${name}_0_link"/>
 			<child link="${name}_1_link"/>
 			<axis xyz="0 0 -1.0" />
 			<dynamics damping="25.0" friction="10.0"/>
-			<calibration rising="0.0"/>
+			<calibration rising="${torso_pan_ref}"/>
 			<limit effort="41.4" lower="-6.2831" upper="6.2831" velocity="0.5"/>
 		</joint>
@@ -72,5 +72,5 @@
 			<axis xyz="0 1.0 0" />
 			<dynamics damping="0.1" />
-			<calibration rising="0.0"/>
+			<calibration rising="${torso_tilt_ref}"/>
 			<limit effort="100" lower="-3.2" upper="1.57" velocity="1.4"/>
 		</joint>

Commit message: harmonize with cob structure

File: raw_description/urdf/torso/torso.urdf.xacro (robot description, xacro)
@@ -6,6 +6,4 @@
 	<include filename="$(find raw_description)/urdf/torso/torso.gazebo.xacro" />
 	<include filename="$(find raw_description)/urdf/torso/torso.transmission.xacro" />
-	<include filename="$(find cob_description)/urdf/sensors/prosilica.urdf.xacro" />
-	<!--include filename="$(find cob_description)/urdf/sensors/kinect.urdf.xacro" /-->
 	<xacro:macro name="raw_torso" params="name parent *origin">
 		<!-- joint between base_link and torso_tilt_link -->
@@ -26,5 +24,5 @@
 					<cylinder length="0.521" radius="0.04"/>
 				</geometry>
-        		<material name="IPA/LightGrey" />
+				<material name="IPA/LightGrey" />
 			</visual>
 			<collision>
@@ -56,5 +54,5 @@
 					<cylinder length="0.3" radius="0.15"/>
 				</geometry>
-                <material name="IPA/LightGrey" />
+				<material name="IPA/LightGrey" />
 			</visual>
 			<collision>
@@ -95,16 +93,4 @@
 			</collision>
 		</link>
-		<!-- left camera -->
-		<!--xacro:cob_prosilica_v0 name="head_color_camera_l" ros_topic="stereo/left" parent="torso_2_link">
-			<origin xyz="${cam_l_x} ${cam_l_y} ${cam_l_z}" rpy="${cam_l_roll} ${cam_l_pitch} ${cam_l_yaw}" />
-		</xacro:cob_prosilica_v0-->
-		<!-- right camera -->
-		<xacro:cob_prosilica_v0 name="head_color_camera_r" ros_topic="stereo/right" parent="torso_2_link">
-			<origin xyz="${cam_r_x} ${cam_r_y} ${cam_r_z}" rpy="${cam_r_roll} ${cam_r_pitch} ${cam_r_yaw}" />
-		</xacro:cob_prosilica_v0>
-		<!-- cam3d -->
-		<xacro:cob_kinect_v0 name="head_cam3d" ros_topic="cam3d" parent="torso_2_link">
-			<origin xyz="${cam3d_x} ${cam3d_y} ${cam3d_z}" rpy="${cam3d_roll} ${cam3d_pitch} ${cam3d_yaw}" />
-		</xacro:cob_kinect_v0>
 		<!-- extensions -->
 		<xacro:raw_torso_gazebo name="${name}" />

Commit message: torso and gripper updates

File: raw_description/urdf/torso/torso.urdf.xacro (robot description, xacro)
@@ -64,5 +64,5 @@
          <parent link="${name}_1_link"/>
       <child link="torso_2_link"/>
-      <axis xyz="0 1.0 0" />
+      <axis xyz="-1.0 0 0" />
       <dynamics damping="0.1" />
       <limit effort="100" lower="-3.2" upper="1.57" velocity="1.4"/>

Commit message: torso and gripper updates

File: raw_description/urdf/torso/torso.urdf.xacro (robot description, xacro)
@@ -64,5 +64,5 @@
          <parent link="${name}_1_link"/>
       <child link="torso_2_link"/>
-      <axis xyz="0 1.0 0" />
+      <axis xyz="-1.0 0 0" />
       <dynamics damping="0.1" />
       <limit effort="100" lower="-3.2" upper="1.57" velocity="1.4"/>

File: raw_description/urdf/vacuum_gripper/gripper.urdf.xacro (robot description, xacro)
@@ -2,8 +2,8 @@
 <robot xmlns:xacro="http://www.ros.org/wiki/xacro">
   <xacro:include filename="$(find raw_description)/urdf/vacuum_gripper/gripper.gazebo.xacro" />
-  <xacro:property name="gripper_length" value="0.044"/>
-  <xacro:property name="gripper_width" value="0.088"/>
-  <xacro:property name="gripper_height" value="0.0946"/>
-  <xacro:property name="gripper_body_height" value="0.16"/>
+  <xacro:property name="gripper_length" value="0.14"/>
+  <xacro:property name="gripper_width" value="0.2"/>
+  <xacro:property name="gripper_height" value="0.14"/>
+  <xacro:property name="gripper_body_height" value="0.14"/>
   <xacro:macro name="vacuum_gripper_definition" params="name parent *origin prefix">
     <!-- joint between arm_ee_link and raw_boxgripper_link -->
@@ -34,7 +34,7 @@
 			</visual>
 			<collision>
-				<!--<origin xyz="0 0 0.03"/>-->
+				<origin xyz="0 0.03 -0.05"/>
 				<geometry>
-					<box size="${gripper_length} ${gripper_width} ${gripper_body_height}"/>
+					<box size="0.13 0.17 0.11"/>
 				</geometry>
 				<material name="another_blue2">
