Commit message: corrected torso definition

File: raw_description/urdf/torso/torso_v2.urdf.xacro (robot description, xacro)
@@ -11,24 +11,24 @@
     <link name="${name}_0_link">
       <inertial>
-        <origin xyz="0 0 0" rpy="0 0 0"/>
+        <origin xyz="0 0 0.254" rpy="0 0 0"/>
         <mass value="0.57307"/>
         <inertia ixx="1.415" ixy="0" ixz="0" iyy="0.819" iyz="0" izz="0.819" />
       </inertial>
       <visual>
-        <origin xyz="0 0 0" rpy="0 0 0" />
+        <origin xyz="0 0 0.254" rpy="0 0 0" />
         <geometry>
-          <cylinder length="0.521" radius="0.04"/>
+          <cylinder length="0.508" radius="0.04"/>
         </geometry>
         <material name="IPA/LightGrey" />
       </visual>
       <collision>
-        <origin xyz="0 0 0" rpy="0 0 0" />
+        <origin xyz="0 0 0.254" rpy="0 0 0" />
         <geometry>
-          <cylinder length="0.521" radius="0.04"/>
+          <cylinder length="0.508" radius="0.04"/>
         </geometry>
       </collision>
     </link>
     <xacro:powerball_ERB115 name="torso" parent="${name}_0_link">
-      <origin xyz="0.0 0.0 0.3074" rpy="0.0 0.0 0.0" />
+      <origin xyz="0.0 0.0 0.582" rpy="0.0 0.0 0.0" />
     </xacro:powerball_ERB115>
     <!-- ros_control plugin -->

Commit message: Using inertia macro

File: raw_description/urdf/torso/torso_v2.urdf.xacro (robot description, xacro)
@@ -10,9 +10,7 @@
     </joint>
     <link name="${name}_0_link">
-      <inertial>
-        <origin xyz="0 0 0.254" rpy="0 0 0"/>
-        <mass value="0.57307"/>
-        <inertia ixx="1.415" ixy="0" ixz="0" iyy="0.819" iyz="0" izz="0.819" />
-      </inertial>
+      <xacro:cylinder_inertial radius="0.04" length="0.508" mass="1.0">
+        <origin xyz="0 0 0.254" rpy="0 0 0" />
+      </xacro:cylinder_inertial>
       <visual>
         <origin xyz="0 0 0.254" rpy="0 0 0" />

Commit message: Use geometry macro

File: raw_description/urdf/torso/torso_v2.urdf.xacro (robot description, xacro)
@@ -15,14 +15,10 @@
       <visual>
         <origin xyz="0 0 0.254" rpy="0 0 0" />
-        <geometry>
-          <cylinder length="0.508" radius="0.04"/>
-        </geometry>
+        <xacro:cylinder_geometry radius="0.04" length="0.508">
         <material name="IPA/LightGrey" />
       </visual>
       <collision>
         <origin xyz="0 0 0.254" rpy="0 0 0" />
-        <geometry>
-          <cylinder length="0.508" radius="0.04"/>
-        </geometry>
+        <xacro:cylinder_geometry radius="0.04" length="0.508">
       </collision>
     </link>

Commit message: fix torso urdf for raw3-1 (#241)
* updated raw3-1 configuration

* Changed back to collision box

* Using inertia macro

* Use geometry macro

File: raw_description/urdf/torso/torso_v2.urdf.xacro (robot description, xacro)
@@ -10,21 +10,15 @@
     </joint>
     <link name="${name}_0_link">
-      <inertial>
-        <origin xyz="0 0 0.254" rpy="0 0 0"/>
-        <mass value="0.57307"/>
-        <inertia ixx="1.415" ixy="0" ixz="0" iyy="0.819" iyz="0" izz="0.819" />
-      </inertial>
+      <xacro:cylinder_inertial radius="0.04" length="0.508" mass="1.0">
+        <origin xyz="0 0 0.254" rpy="0 0 0" />
+      </xacro:cylinder_inertial>
       <visual>
         <origin xyz="0 0 0.254" rpy="0 0 0" />
-        <geometry>
-          <cylinder length="0.508" radius="0.04"/>
-        </geometry>
+        <xacro:cylinder_geometry radius="0.04" length="0.508">
         <material name="IPA/LightGrey" />
       </visual>
       <collision>
         <origin xyz="0 0 0.254" rpy="0 0 0" />
-        <geometry>
-          <cylinder length="0.508" radius="0.04"/>
-        </geometry>
+        <xacro:cylinder_geometry radius="0.04" length="0.508">
       </collision>
     </link>
