Commit message: Orange color for LBR

File: cob_description/urdf/lbr/lbr.gazebo.xacro (robot description, xacro)
@@ -6,33 +6,33 @@
 	<xacro:macro name="cob_lbr_gazebo" params="name">
 		<gazebo reference="${name}_0_link">
-			<material value="Gazebo/Red" />
+			<material value="IPA/Orange" />
 			<turnGravityOff>false</turnGravityOff>
 		</gazebo>
 		<gazebo reference="${name}_1_link">
-			<material value="Gazebo/Blue" />
+			<material value="IPA/Orange" />
 			<turnGravityOff>false</turnGravityOff>
 		</gazebo>
 		<gazebo reference="${name}_2_link">
-			<material value="Gazebo/Red" />
+			<material value="IPA/Orange" />
 			<turnGravityOff>false</turnGravityOff>
 		</gazebo>
 		<gazebo reference="${name}_3_link">
-			<material value="Gazebo/Blue" />
+			<material value="IPA/Orange" />
 			<turnGravityOff>false</turnGravityOff>
 		</gazebo>
 		<gazebo reference="${name}_4_link">
-			<material value="Gazebo/Red" />
+			<material value="IPA/Orange" />
 			<turnGravityOff>false</turnGravityOff>
 		</gazebo>
 		<gazebo reference="${name}_5_link">
-			<material value="Gazebo/Blue" />
+			<material value="IPA/Orange" />
 			<turnGravityOff>false</turnGravityOff>
 		</gazebo>
 		<gazebo reference="${name}_6_link">
-			<material value="Gazebo/Red" />
+			<material value="IPA/Orange" />
 			<turnGravityOff>false</turnGravityOff>
 		</gazebo>
 		<gazebo reference="${name}_7_link">
-			<material value="Gazebo/Blue" />
+			<material value="IPA/Orange" />
 			<turnGravityOff>false</turnGravityOff>
 		</gazebo>

File: cob_description/urdf/lbr/lbr.urdf.xacro (robot description, xacro)
@@ -24,5 +24,5 @@
 					<cylinder radius="0.060" length="0.14"/>
 				</geometry>
-				<material name="Red" />
+				<material name="Orange" />
 			</visual>
 			<collision>
@@ -55,5 +55,5 @@
 					<mesh filename="package://cob_description/meshes/lbr/joint_1.stl" />
 				</geometry>
-				<material name="Blue" />
+				<material name="Orange" />
 			</visual>
 			<collision>
@@ -86,5 +86,5 @@
 					<mesh filename="package://cob_description/meshes/lbr/joint_2.stl" />
 				</geometry>
-				<material name="Red" />
+				<material name="Orange" />
 			</visual>
 			<collision>
@@ -117,5 +117,5 @@
 					<mesh filename="package://cob_description/meshes/lbr/joint_3.stl" />
 				</geometry>
-				<material name="Blue" />
+				<material name="Orange" />
 			</visual>
 			<collision>
@@ -149,5 +149,5 @@
 					<mesh filename="package://cob_description/meshes/lbr/joint_4.stl" />
 				</geometry>
-				<material name="Red" />
+				<material name="Orange" />
 			</visual>
 			<collision>
@@ -179,5 +179,5 @@
 					<mesh filename="package://cob_description/meshes/lbr/joint_5.stl" />
 				</geometry>
-				<material name="Blue" />
+				<material name="Orange" />
 			</visual>
 			<collision>
@@ -210,5 +210,5 @@
 					<mesh filename="package://cob_description/meshes/lbr/joint_6.stl" />
 				</geometry>
-				<material name="Red" />
+				<material name="Orange" />
 			</visual>
 			<collision>
@@ -241,5 +241,5 @@
 					<mesh filename="package://cob_description/meshes/lbr/joint_7.stl" />
 				</geometry>
-				<material name="Blue" />
+				<material name="Orange" />
 			</visual>
 			<collision>

File: cob_description/urdf/materials.urdf.xacro (robot description, xacro)
@@ -22,10 +22,7 @@
 		<color rgba="0.0 0.0 0.0 1.0"/>
 	</material>
-        <material name="Transparent">
-                <color rgba="0.81 0.81 0.81 0.0"/>
-        </material>
-        <material name="LightBlue">
-                <color rgba="0.624 0.698 0.858 1"/>
-        </material>
+	<material name="Orange">
+		<color rgba="1.0 0.5 0.0 1.0"/>
+	</material>
 	<material name="Caster">
 		<texture filename="package://pr2_ogre/Media/materials/textures/pr2_caster_texture.png" />
