Commit message: offset for lbr set to 0

File: cob_description/urdf/lbr/lbr.urdf.xacro (robot description, xacro)
@@ -35,5 +35,5 @@
 		<!-- joint between arm_0_link and arm_1_link -->
 		<joint name="${name}_1_joint" type="revolute">
-		<origin xyz="0 0 0.0" rpy="0 0 -2.8407"/>
+		<origin xyz="0 0 0.0" rpy="0 0 0"/>
 			<parent link="${name}_0_link"/>
 			<child link="${name}_1_link"/>

Commit message: offset back in lbr.urdf.xacro else wrong calibration

File: cob_description/urdf/lbr/lbr.urdf.xacro (robot description, xacro)
@@ -35,5 +35,5 @@
 		<!-- joint between arm_0_link and arm_1_link -->
 		<joint name="${name}_1_joint" type="revolute">
-		<origin xyz="0 0 0.0" rpy="0 0 0"/>
+		<origin xyz="0 0 0.0" rpy="0 0 -2.8407"/>
 			<parent link="${name}_0_link"/>
 			<child link="${name}_1_link"/>
