Commit message: Fuerte migration cob_descriptionurdf/base/base.gazebo.xacro

File: cob_description/urdf/head_v3/head.gazebo.xacro (robot description, xacro)
@@ -6,5 +6,5 @@
 	<xacro:macro name="cob_head_gazebo_v3" params="name">
 		<gazebo reference="${name}_axis_link">
-			<material>Gazebo/Green</material>
+			<material>Green</material>
 			<turnGravityOff>false</turnGravityOff>
 		</gazebo>

File: cob_description/urdf/lbr/lbr.gazebo.xacro (robot description, xacro)
@@ -6,33 +6,33 @@
 	<xacro:macro name="cob_lbr_gazebo" params="name">
 		<gazebo reference="${name}_0_link">
-			<material value="PR2/Red" />
+			<material value="Gazebo/Red" />
 			<turnGravityOff>false</turnGravityOff>
 		</gazebo>
 		<gazebo reference="${name}_1_link">
-			<material value="PR2/Blue" />
+			<material value="Gazebo/Blue" />
 			<turnGravityOff>false</turnGravityOff>
 		</gazebo>
 		<gazebo reference="${name}_2_link">
-			<material value="PR2/Red" />
+			<material value="Gazebo/Red" />
 			<turnGravityOff>false</turnGravityOff>
 		</gazebo>
 		<gazebo reference="${name}_3_link">
-			<material value="PR2/Blue" />
+			<material value="Gazebo/Blue" />
 			<turnGravityOff>false</turnGravityOff>
 		</gazebo>
 		<gazebo reference="${name}_4_link">
-			<material value="PR2/Red" />
+			<material value="Gazebo/Red" />
 			<turnGravityOff>false</turnGravityOff>
 		</gazebo>
 		<gazebo reference="${name}_5_link">
-			<material value="PR2/Blue" />
+			<material value="Gazebo/Blue" />
 			<turnGravityOff>false</turnGravityOff>
 		</gazebo>
 		<gazebo reference="${name}_6_link">
-			<material value="PR2/Red" />
+			<material value="Gazebo/Red" />
 			<turnGravityOff>false</turnGravityOff>
 		</gazebo>
 		<gazebo reference="${name}_7_link">
-			<material value="PR2/Blue" />
+			<material value="Gazebo/Blue" />
 			<turnGravityOff>false</turnGravityOff>
 		</gazebo>

File: cob_description/urdf/materials.urdf.xacro (robot description, xacro)
@@ -11,5 +11,5 @@
 	</material>
 	<material name="Grey2">
-		<color rgba="0.9 0.9 0.9 1.0"/>
+		<color rgba="0.81 0.81 0.81 1.0"/>
 	</material>
 	<material name="Red">

File: cob_description/urdf/sensors/sick_s300_laser.gazebo.xacro (robot description, xacro)
@@ -27,5 +27,5 @@
         </controller:gazebo_ros_laser>
       </sensor:ray>
-      <material value="PR2/Yellow" />
+      <material value="Gazebo/Yellow" />
     </gazebo>
   </xacro:macro>

File: cob_description/urdf/torso_v1/torso.gazebo.xacro (robot description, xacro)
@@ -14,5 +14,5 @@
 		</gazebo>
 		<gazebo reference="${name}_upper_neck_tilt_link">
-			<material>Gazebo/Grey</material>
+			<material>IPA/Grey1</material>
 			<turnGravityOff>false</turnGravityOff>
 		</gazebo>

Commit message: Redefined Care-O-bot colors for Gazebo and Rviz

File: cob_description/urdf/head_v3/head.gazebo.xacro (robot description, xacro)
@@ -6,5 +6,5 @@
 	<xacro:macro name="cob_head_gazebo_v3" params="name">
 		<gazebo reference="${name}_axis_link">
-			<material>Green</material>
+			<material>Gazebo/Black</material>
 			<turnGravityOff>false</turnGravityOff>
 		</gazebo>

File: cob_description/urdf/head_v3/head.urdf.xacro (robot description, xacro)
@@ -30,5 +30,5 @@
 					<box size="0.01 0.01 0.01"/>
 				</geometry>
-				<material name="Green" />
+				<material name="Black" />
 			</visual>
 			<collision>

File: cob_description/urdf/materials.urdf.xacro (robot description, xacro)
@@ -25,4 +25,7 @@
 		<color rgba="1.0 0.5 0.0 1.0"/>
 	</material>
+	<material name="DarkGolden">
+		<color rgba="0.72 0.5255 0.043 1.0"/>
+	</material>
 	<material name="Caster">
 		<texture filename="package://pr2_ogre/Media/materials/textures/pr2_caster_texture.png" />

File: cob_description/urdf/sensors/hokuyo_SR400_laser.urdf.xacro (robot description, xacro)
@@ -23,5 +23,5 @@
           <box size="0.001 0.001 0.001" />
         </geometry>
-        <material name="Red" />
+        <material name="Grey" />
       </visual>
       <collision>

File: cob_description/urdf/sensors/kinect.urdf.xacro (robot description, xacro)
@@ -22,5 +22,5 @@
           <box size="0.02 0.02 0.075"/>
         </geometry>
-        <material name="Red" />
+        <material name="Grey" />
       </visual>
       <collision>
@@ -47,5 +47,5 @@
           <box size="0.01 0.01 0.01"/>
         </geometry>
-        <material name="Red" />
+        <material name="Grey" />
       </visual>
       <collision>

File: cob_description/urdf/sensors/prosilica.urdf.xacro (robot description, xacro)
@@ -23,5 +23,5 @@
 					<cylinder radius="0.01" length="0.075"/>
 				</geometry>
-				<material name="Red" />
+				<material name="Black" />
 			</visual>
 			<collision>
@@ -48,5 +48,5 @@
 					<box size="0.01 0.01 0.01"/>
 				</geometry>
-				<material name="Red" />
+				<material name="Black" />
 			</visual>
 			<collision>

File: cob_description/urdf/sensors/sick_s300_laser.gazebo.xacro (robot description, xacro)
@@ -27,5 +27,5 @@
         </controller:gazebo_ros_laser>
       </sensor:ray>
-      <material value="Gazebo/Yellow" />
+      <material value="Gazebo/Grey" />
     </gazebo>
   </xacro:macro>

File: cob_description/urdf/sensors/sick_s300_laser.urdf.xacro (robot description, xacro)
@@ -26,5 +26,5 @@
           <!--box size="0.001 0.001 0.001" /-->
         </geometry>
-        <material name="Red" />
+        <material name="Grey" />
       </visual>
       <collision>

File: cob_description/urdf/torso_v1/torso.gazebo.xacro (robot description, xacro)
@@ -6,17 +6,17 @@
 	<xacro:macro name="cob_torso_gazebo_v1" params="name">
 		<gazebo reference="${name}_lower_neck_tilt_link">
-			<material>Gazebo/Red</material>
+			<material>Gazebo/Grey</material>
 			<turnGravityOff>false</turnGravityOff>
 		</gazebo>
 		<gazebo reference="${name}_pan_link">
-			<material>Gazebo/Blue</material>
+			<material>Gazebo/Grey</material>
 			<turnGravityOff>false</turnGravityOff>
 		</gazebo>
 		<gazebo reference="${name}_upper_neck_tilt_link">
-			<material>IPA/Grey1</material>
+			<material>Gazebo/Grey</material>
 			<turnGravityOff>false</turnGravityOff>
 		</gazebo>
 		<gazebo reference="head_cover_link">
-			<material>Gazebo/Blue</material>
+			<material>Gazebo/Black</material>
 			<turnGravityOff>false</turnGravityOff>
 		</gazebo>

File: cob_description/urdf/torso_v1/torso.urdf.xacro (robot description, xacro)
@@ -28,5 +28,5 @@
 					<mesh filename="package://cob_description/meshes/torso/lower_neck.stl" />
 				</geometry>
-				<material name="Red" />
+				<material name="Grey" />
 			</visual>
 			<collision>
@@ -58,5 +58,5 @@
 					<box size="0.01 0.01 0.01"/>
 				</geometry>
-				<material name="Blue" />
+				<material name="Black" />
 			</visual>
 			<collision>
@@ -114,5 +114,5 @@
 					<mesh filename="package://cob_description/meshes/torso/head_cover.stl" />
 				</geometry>
-				<material name="Blue" />
+				<material name="Black" />
 			</visual>
 			<collision>

File: cob_description/urdf/tray/tray.gazebo.xacro (robot description, xacro)
@@ -6,5 +6,5 @@
 	<xacro:macro name="cob_tray_gazebo" params="name">
 		<gazebo reference="${name}_link">
-			<material>Gazebo/Green</material>
+			<material>IPA/Grey2</material>
 			<turnGravityOff>false</turnGravityOff>
 		</gazebo>

File: cob_description/urdf/tray/tray.urdf.xacro (robot description, xacro)
@@ -29,5 +29,5 @@
 					<mesh filename="package://cob_description/meshes/tray/tray.stl" />
 				</geometry>
-				<material name="Green" />
+				<material name="Grey" />
 			</visual>
 			<collision>

File: cob_description/urdf/tray_powerball/tray.gazebo.xacro (robot description, xacro)
@@ -6,13 +6,13 @@
 	<xacro:macro name="cob_tray_gazebo" params="name">
 		<gazebo reference="${name}_1_link">
-			<material>Gazebo/Blue</material>
+			<material>IPA/Grey</material>
 			<turnGravityOff>false</turnGravityOff>
 		</gazebo>
 		<gazebo reference="${name}_2_link">
-			<material>Gazebo/Red</material>
+			<material>IPA/Grey1</material>
 			<turnGravityOff>false</turnGravityOff>
 		</gazebo>
 		<gazebo reference="${name}_3_link">
-			<material>Gazebo/Blue</material>
+			<material>IPA/Grey</material>
 			<turnGravityOff>false</turnGravityOff>
 		</gazebo>
