Commit message: cameras have zero pos/rot offsets in head_v3

File: cob_description/urdf/head_v3/head.urdf.xacro (robot description, xacro)
@@ -41,13 +41,13 @@
 		<!-- left camera -->
 		<xacro:cob_prosilica_v0 name="${name}_color_camera_l" ros_topic="stereo/left" parent="${name}_axis_link">
-			<origin xyz="${cam_l_x} ${cam_l_y} ${cam_l_z-0.06}" rpy="${cam_l_roll} ${cam_l_pitch-1.5708} ${cam_l_yaw}" />
+			<origin xyz="${cam_l_x} ${cam_l_y} ${cam_l_z}" rpy="${cam_l_roll} ${cam_l_pitch} ${cam_l_yaw}" />
 		</xacro:cob_prosilica_v0>
 		<!-- right camera -->
 		<xacro:cob_prosilica_v0 name="${name}_color_camera_r" ros_topic="stereo/right" parent="${name}_color_camera_l_link">
-			<origin xyz="${cam_r_x+0.12} ${cam_r_y} ${cam_r_z}" rpy="${cam_r_roll} ${cam_r_pitch} ${cam_r_yaw}" />
+			<origin xyz="${cam_r_x} ${cam_r_y} ${cam_r_z}" rpy="${cam_r_roll} ${cam_r_pitch} ${cam_r_yaw}" />
 		</xacro:cob_prosilica_v0>
 		<!-- cam3d -->
 		<xacro:cob_kinect_v0 name="${name}_cam3d" ros_topic="cam3d" parent="${name}_axis_link">
-			<origin xyz="${cam3d_x+0.06} ${cam3d_y} ${cam3d_z}" rpy="${cam3d_roll} ${cam3d_pitch} ${cam3d_yaw}" />
+			<origin xyz="${cam3d_x} ${cam3d_y} ${cam3d_z}" rpy="${cam3d_roll} ${cam3d_pitch} ${cam3d_yaw}" />
 		</xacro:cob_kinect_v0>
 		<!-- extensions -->

Commit message: Renamed the colors

File: cob_description/urdf/head_v3/head.urdf.xacro (robot description, xacro)
@@ -30,5 +30,5 @@
 					<box size="0.01 0.01 0.01"/>
 				</geometry>
-				<material name="Black" />
+				<material name="IPA/Black" />
 			</visual>
 			<collision>

File: cob_description/urdf/lbr/lbr.urdf.xacro (robot description, xacro)
@@ -24,5 +24,5 @@
 					<cylinder radius="0.060" length="0.14"/>
 				</geometry>
-				<material name="Orange" />
+				<material name="IPA/Orange" />
 			</visual>
 			<collision>
@@ -55,5 +55,5 @@
 					<mesh filename="package://cob_description/meshes/lbr/joint_1.stl" />
 				</geometry>
-				<material name="Orange" />
+				<material name="IPA/Orange" />
 			</visual>
 			<collision>
@@ -86,5 +86,5 @@
 					<mesh filename="package://cob_description/meshes/lbr/joint_2.stl" />
 				</geometry>
-				<material name="Orange" />
+				<material name="IPA/Orange" />
 			</visual>
 			<collision>
@@ -117,5 +117,5 @@
 					<mesh filename="package://cob_description/meshes/lbr/joint_3.stl" />
 				</geometry>
-				<material name="Orange" />
+				<material name="IPA/Orange" />
 			</visual>
 			<collision>
@@ -149,5 +149,5 @@
 					<mesh filename="package://cob_description/meshes/lbr/joint_4.stl" />
 				</geometry>
-				<material name="Orange" />
+				<material name="IPA/Orange" />
 			</visual>
 			<collision>
@@ -179,5 +179,5 @@
 					<mesh filename="package://cob_description/meshes/lbr/joint_5.stl" />
 				</geometry>
-				<material name="Orange" />
+				<material name="IPA/Orange" />
 			</visual>
 			<collision>
@@ -210,5 +210,5 @@
 					<mesh filename="package://cob_description/meshes/lbr/joint_6.stl" />
 				</geometry>
-				<material name="Orange" />
+				<material name="IPA/Orange" />
 			</visual>
 			<collision>
@@ -241,5 +241,5 @@
 					<mesh filename="package://cob_description/meshes/lbr/joint_7.stl" />
 				</geometry>
-				<material name="Orange" />
+				<material name="IPA/Orange" />
 			</visual>
 			<collision>

File: cob_description/urdf/materials.urdf.xacro (robot description, xacro)
@@ -7,8 +7,8 @@
 		<color rgba="0.0 0.8 0.0 1.0"/>
 	</material>
-	<material name="Grey">
+	<material name="IPA/DarkGrey">
 		<color rgba="0.7 0.7 0.7 1.0"/>
 	</material>
-	<material name="Grey2">
+	<material name="IPA/LightGrey">
 		<color rgba="0.81 0.81 0.81 1.0"/>
 	</material>
@@ -19,11 +19,11 @@
 		<color rgba="1.0 1.0 1.0 1.0"/>
 	</material>
-	<material name="Black">
+	<material name="IPA/Black">
 		<color rgba="0.0 0.0 0.0 1.0"/>
 	</material>
-	<material name="Orange">
+	<material name="IPA/Orange">
 		<color rgba="1.0 0.5 0.0 1.0"/>
 	</material>
-	<material name="DarkGolden">
+	<material name="Schunk/DarkGolden">
 		<color rgba="0.72 0.5255 0.043 1.0"/>
 	</material>

File: cob_description/urdf/sensors/hokuyo_SR400_laser.urdf.xacro (robot description, xacro)
@@ -23,5 +23,5 @@
           <box size="0.001 0.001 0.001" />
         </geometry>
-        <material name="Grey" />
+        <material name="IPA/DarkGrey" />
       </visual>
       <collision>

File: cob_description/urdf/sensors/kinect.urdf.xacro (robot description, xacro)
@@ -22,5 +22,5 @@
           <box size="0.02 0.02 0.075"/>
         </geometry>
-        <material name="Grey" />
+        <material name="IPA/DarkGrey" />
       </visual>
       <collision>
@@ -47,5 +47,5 @@
           <box size="0.01 0.01 0.01"/>
         </geometry>
-        <material name="Grey" />
+        <material name="IPA/DarkGrey" />
       </visual>
       <collision>

File: cob_description/urdf/sensors/prosilica.urdf.xacro (robot description, xacro)
@@ -23,5 +23,5 @@
 					<cylinder radius="0.01" length="0.075"/>
 				</geometry>
-				<material name="Black" />
+				<material name="IPA/Black" />
 			</visual>
 			<collision>
@@ -48,5 +48,5 @@
 					<box size="0.01 0.01 0.01"/>
 				</geometry>
-				<material name="Black" />
+				<material name="IPA/Black" />
 			</visual>
 			<collision>

File: cob_description/urdf/sensors/sick_s300_laser.urdf.xacro (robot description, xacro)
@@ -26,5 +26,5 @@
           <!--box size="0.001 0.001 0.001" /-->
         </geometry>
-        <material name="Grey" />
+        <material name="IPA/DarkGrey" />
       </visual>
       <collision>

File: cob_description/urdf/torso_v0/torso.urdf.xacro (robot description, xacro)
@@ -118,5 +118,5 @@
 					<mesh filename="package://cob_description/meshes/torso/upper_neck.stl" />
 				</geometry>
-				<material name="Grey" />
+				<material name="IPA/DarkGrey" />
 			</visual>
 			<collision>

File: cob_description/urdf/torso_v1/torso.urdf.xacro (robot description, xacro)
@@ -28,5 +28,5 @@
 					<mesh filename="package://cob_description/meshes/torso/lower_neck.stl" />
 				</geometry>
-				<material name="Grey" />
+				<material name="IPA/DarkGrey" />
 			</visual>
 			<collision>
@@ -58,5 +58,5 @@
 					<box size="0.01 0.01 0.01"/>
 				</geometry>
-				<material name="Black" />
+				<material name="IPA/Black" />
 			</visual>
 			<collision>
@@ -88,5 +88,5 @@
 					<mesh filename="package://cob_description/meshes/torso/upper_neck.stl" />
 				</geometry>
-				<material name="Grey" />
+				<material name="IPA/DarkGrey" />
 			</visual>
 			<collision>
@@ -114,5 +114,5 @@
 					<mesh filename="package://cob_description/meshes/torso/head_cover.stl" />
 				</geometry>
-				<material name="Black" />
+				<material name="IPA/Black" />
 			</visual>
 			<collision>

File: cob_description/urdf/tray/tray.gazebo.xacro (robot description, xacro)
@@ -6,5 +6,5 @@
 	<xacro:macro name="cob_tray_gazebo" params="name">
 		<gazebo reference="${name}_link">
-			<material>IPA/Grey2</material>
+			<material>IPA/DarkGrey</material>
 			<turnGravityOff>false</turnGravityOff>
 		</gazebo>

File: cob_description/urdf/tray/tray.urdf.xacro (robot description, xacro)
@@ -29,5 +29,5 @@
 					<mesh filename="package://cob_description/meshes/tray/tray.stl" />
 				</geometry>
-				<material name="Grey" />
+				<material name="IPA/DarkGrey" />
 			</visual>
 			<collision>

File: cob_description/urdf/tray_powerball/tray.gazebo.xacro (robot description, xacro)
@@ -6,13 +6,13 @@
 	<xacro:macro name="cob_tray_gazebo" params="name">
 		<gazebo reference="${name}_1_link">
-			<material>IPA/Grey</material>
+			<material>IPA/LightGrey</material>
 			<turnGravityOff>false</turnGravityOff>
 		</gazebo>
 		<gazebo reference="${name}_2_link">
-			<material>IPA/Grey1</material>
+			<material>IPA/DarkGrey</material>
 			<turnGravityOff>false</turnGravityOff>
 		</gazebo>
 		<gazebo reference="${name}_3_link">
-			<material>IPA/Grey</material>
+			<material>IPA/LightGrey</material>
 			<turnGravityOff>false</turnGravityOff>
 		</gazebo>

Commit message: added fixed links for calibration

File: cob_description/urdf/head_v3/head.urdf.xacro (robot description, xacro)
@@ -9,8 +9,34 @@
 	<include filename="$(find cob_description)/urdf/sensors/kinect.urdf.xacro" />
 	<xacro:macro name="cob_head_v3" params="name parent *origin">
-		<!-- joint between torso_upper_neck_tilt_link and head_axis_link -->
-		<joint name="${name}_axis_joint" type="revolute">
+		<!-- joint between torso_upper_neck_tilt_link and head_base_link -->
+		<joint name="head_base_joint" type="fixed">
 			<insert_block name="origin" />
 			<parent link="${parent}"/>
+			<child link="head_base_link"/>
+		</joint>
+		<link name="head_base_link">
+			<inertial>
+				<origin xyz="0 0 0" rpy="0 0 0"/>
+				<mass value="0.5"/>
+				<inertia ixx="0.01" ixy="0" ixz="0" iyy="0.01" iyz="0" izz="0.01" />
+			</inertial>
+			<visual>
+				<origin xyz="0 0 0" rpy="0 0 0" />
+				<geometry>
+					<box size="0.01 0.01 0.01"/>
+				</geometry>
+				<material name="IPA/Black" />
+			</visual>
+			<collision>
+				<origin xyz="0 0 0" rpy="0 0 0" />
+				<geometry>
+					<box size="0.01 0.01 0.01"/>
+				</geometry>
+			</collision>
+		</link>
+		<!-- joint between head_base_link and head_axis_link -->
+		<joint name="${name}_axis_joint" type="revolute">
+			<parent link="head_base_link"/>
+			<origin xyz="0 0 0" rpy="0 0 0" />
 			<child link="${name}_axis_link"/>
 			<axis xyz="0 0 1" />
@@ -39,14 +65,40 @@
 			</collision>
 		</link>
+		<!-- joint between torso_upper_neck_tilt_link and head_base_link -->
+		<joint name="cam_reference_joint" type="fixed">
+			<origin xyz="${cam_l_x} ${cam_l_y} ${cam_l_z}" rpy="${cam_l_roll} ${cam_l_pitch} ${cam_l_yaw}" />
+			<parent link="head_axis_link"/>
+			<child link="cam_reference_link"/>
+		</joint>
+		<link name="cam_reference_link">
+			<inertial>
+				<origin xyz="0 0 0" rpy="0 0 0"/>
+				<mass value="0.5"/>
+				<inertia ixx="0.01" ixy="0" ixz="0" iyy="0.01" iyz="0" izz="0.01" />
+			</inertial>
+			<visual>
+				<origin xyz="0 0 0" rpy="0 0 0" />
+				<geometry>
+					<box size="0.01 0.01 0.01"/>
+				</geometry>
+				<material name="IPA/Black" />
+			</visual>
+			<collision>
+				<origin xyz="0 0 0" rpy="0 0 0" />
+				<geometry>
+					<box size="0.01 0.01 0.01"/>
+				</geometry>
+			</collision>
+		</link>
 		<!-- left camera -->
-		<xacro:cob_prosilica_v0 name="${name}_color_camera_l" ros_topic="stereo/left" parent="${name}_axis_link">
-			<origin xyz="${cam_l_x} ${cam_l_y} ${cam_l_z}" rpy="${cam_l_roll} ${cam_l_pitch} ${cam_l_yaw}" />
+		<xacro:cob_prosilica_v0 name="${name}_color_camera_l" ros_topic="stereo/left" parent="cam_reference_link">
+			<origin xyz="0 0 0" rpy="0 0 0" />
 		</xacro:cob_prosilica_v0>
 		<!-- right camera -->
-		<xacro:cob_prosilica_v0 name="${name}_color_camera_r" ros_topic="stereo/right" parent="${name}_color_camera_l_link">
+		<xacro:cob_prosilica_v0 name="${name}_color_camera_r" ros_topic="stereo/right" parent="cam_reference_link">
 			<origin xyz="${cam_r_x} ${cam_r_y} ${cam_r_z}" rpy="${cam_r_roll} ${cam_r_pitch} ${cam_r_yaw}" />
 		</xacro:cob_prosilica_v0>
-		<!-- cam3d -->
-		<xacro:cob_kinect_v0 name="${name}_cam3d" ros_topic="cam3d" parent="${name}_axis_link">
+		<!-- cam3d -->l
+		<xacro:cob_kinect_v0 name="${name}_cam3d" ros_topic="cam3d" parent="cam_reference_link">
 			<origin xyz="${cam3d_x} ${cam3d_y} ${cam3d_z}" rpy="${cam3d_roll} ${cam3d_pitch} ${cam3d_yaw}" />
 		</xacro:cob_kinect_v0>

File: cob_description/urdf/torso_v1/torso.urdf.xacro (robot description, xacro)
@@ -7,8 +7,34 @@
 	<include filename="$(find cob_description)/urdf/torso_v1/torso.transmission.xacro" />
 	<xacro:macro name="cob_torso_v1" params="name parent *origin">
+		<!-- joint between base_link and torso_base_link -->
+		<joint name="${name}_base_joint" type="fixed" >
+			<insert_block name="origin" />
+			<parent link="${parent}" />
+			<child link="${name}_base_link" />
+		</joint>
+		<link name="${name}_base_link">
+			<inertial>
+				<origin xyz="0 0 0" rpy="0 0 0"/>
+				<mass value="0.01"/>
+				<inertia ixx="1" ixy="0" ixz="0" iyy="1" iyz="0" izz="1" />
+			</inertial>
+			<visual>
+				<origin xyz="0 0 -0.00" rpy="0 0 0" />
+				<geometry>
+					<cylinder radius="0" length="0"/>
+				</geometry>
+                <material name="IPA/DarkGrey" />
+			</visual>
+			<collision>
+				<origin xyz="0 0 0" rpy="0 0 0" />
+				<geometry>
+					<box size="0 0 0"/>
+				</geometry>
+			</collision>
+		</link>
 		<!-- joint between base_link and torso_lower_neck_tilt_link -->
 		<joint name="${name}_lower_neck_tilt_joint" type="revolute">
-			<insert_block name="origin" />
-			<parent link="${parent}"/>
+			<origin xyz="0 0 0" rpy="0 0 0" />
+			<parent link="${name}_base_link"/>
 			<child link="${name}_lower_neck_tilt_link"/>
 			<axis xyz="0 0 1" />

Commit message: fixed typo

File: cob_description/urdf/head_v3/head.urdf.xacro (robot description, xacro)
@@ -99,5 +99,5 @@
 			<origin xyz="${cam_r_x} ${cam_r_y} ${cam_r_z}" rpy="${cam_r_roll} ${cam_r_pitch} ${cam_r_yaw}" />
 		</xacro:cob_prosilica_v0>
-		<!-- cam3d -->l
+		<!-- cam3d -->
 		<xacro:cob_kinect_v0 name="${name}_cam3d" ros_topic="cam3d" parent="cam_reference_link">
 			<origin xyz="${cam3d_x} ${cam3d_y} ${cam3d_z}" rpy="${cam3d_roll} ${cam3d_pitch} ${cam3d_yaw}" />

File: cob_description/urdf/sensors/kinect.urdf.xacro (robot description, xacro)
@@ -29,5 +29,5 @@
            <box size="0.02 0.02 0.075"/>
         </geometry>
-      </collision >
+      </collision>
     </link>
     <joint name="${name}_frame_joint" type="fixed">
