Commit message: fix colors and powerball tray

File: cob_description/urdf/tray_powerball/tray.gazebo.xacro (robot description, xacro)
@@ -4,5 +4,5 @@
        xmlns:interface="http://playerstage.sourceforge.net/gazebo/xmlschema/#interface"
        xmlns:xacro="http://ros.org/wiki/xacro">
-	<xacro:macro name="cob_tray_gazebo" params="name">
+	<xacro:macro name="cob_tray_powerball_gazebo" params="name">
 		<gazebo reference="${name}_1_link">
 			<material>IPA/LightGrey</material>

File: cob_description/urdf/tray_powerball/tray.transmission.xacro (robot description, xacro)
@@ -4,5 +4,5 @@
        xmlns:interface="http://playerstage.sourceforge.net/gazebo/xmlschema/#interface"
        xmlns:xacro="http://ros.org/wiki/xacro">
-	<xacro:macro name="cob_tray_transmission" params="name">
+	<xacro:macro name="cob_tray_powerball_transmission" params="name">
 		<transmission name="${name}_1_trans" type="pr2_mechanism_model/SimpleTransmission">
 			<actuator name="${name}_1_motor"/>

File: cob_description/urdf/tray_powerball/tray.urdf.xacro (robot description, xacro)
@@ -160,6 +160,6 @@
 		</xacro:phidgets_distance_v0>
 		<!-- extensions -->
-		<xacro:cob_tray_gazebo name="${name}" />
-		<xacro:cob_tray_transmission name="${name}" />
+		<xacro:cob_tray_powerball_gazebo name="${name}" />
+		<xacro:cob_tray_powerball_transmission name="${name}" />
 	</xacro:macro>
 </robot>
