Commit message: Minor changes in tray_powerball description

File: cob_description/urdf/tray_powerball/tray.urdf.xacro (robot description, xacro)
@@ -13,8 +13,8 @@
 			<parent link="${parent}"/>
 			<child link="${name}_1_link"/>
-			<axis xyz="0 1 0" />
+			<axis xyz="1 0 0" />
 			<calibration rising="${tray_1_ref}"/>
 			<dynamics damping="5.0" friction="0.5"/>
-			<limit effort="100" lower="-3.31612" upper="0.2" velocity="5"/>
+			<limit effort="100" lower="-3.31612" upper="3.31612" velocity="5"/>
 		</joint>
 		<link name="${name}_1_link">
@@ -45,5 +45,5 @@
 			<calibration rising="${tray_2_ref}"/>
 			<dynamics damping="5.0" friction="0.5"/>
-			<limit effort="100" lower="-3.31612" upper="0.2" velocity="5"/>
+			<limit effort="100" lower="-3.31612" upper="3.31612" velocity="5"/>
 		</joint>
 		<link name="${name}_2_link">
@@ -74,5 +74,5 @@
 			<calibration rising="${tray_3_ref}"/>
 			<dynamics damping="5.0" friction="0.5"/>
-			<limit effort="100" lower="-3.31612" upper="0.2" velocity="5"/>
+			<limit effort="100" lower="-3.31612" upper="3.31612" velocity="5"/>
 		</joint>
 		<link name="${name}_3_link">

Commit message: Removed stlb as collision mesh files, fuerte does not support this format

File: cob_description/urdf/tray_powerball/tray.urdf.xacro (robot description, xacro)
@@ -34,5 +34,5 @@
 				<origin xyz="0 0 0" rpy="0 0 0" />
 				<geometry>
-					<mesh filename="package://cob_description/meshes/tray_powerball/tray_link_1.stlb" />
+					<mesh filename="package://cob_description/meshes/tray_powerball/tray_link_1.stl" />
 				</geometry>
 			</collision>
@@ -63,5 +63,5 @@
 				<origin xyz="0 0 0" rpy="0 0 0" />
 				<geometry>
-					<mesh filename="package://cob_description/meshes/tray_powerball/tray_link_2.stlb" />
+					<mesh filename="package://cob_description/meshes/tray_powerball/tray_link_2.stl" />
 				</geometry>
 			</collision>
@@ -92,5 +92,5 @@
 				<origin xyz="0 0 0" rpy="0 0 0" />
 				<geometry>
-					<mesh filename="package://cob_description/meshes/tray_powerball/tray_link_3.stlb" />
+					<mesh filename="package://cob_description/meshes/tray_powerball/tray_link_3.stl" />
 				</geometry>
 			</collision>

Commit message: Updated joints axis

File: cob_description/urdf/tray_powerball/tray.urdf.xacro (robot description, xacro)
@@ -13,5 +13,5 @@
 			<parent link="${parent}"/>
 			<child link="${name}_1_link"/>
-			<axis xyz="1 0 0" />
+			<axis xyz="0 0 1" />
 			<calibration rising="${tray_1_ref}"/>
 			<dynamics damping="5.0" friction="0.5"/>
@@ -25,5 +25,5 @@
 			</inertial>
 			<visual>
-				<origin xyz="0 0 0" rpy="0 0 0" />
+				<origin xyz="0 0 0" rpy="0 1.570796 0" />
 				<geometry>
 					<mesh filename="package://cob_description/meshes/tray_powerball/tray_link_1.stl" />
@@ -32,5 +32,5 @@
 			</visual>
 			<collision>
-				<origin xyz="0 0 0" rpy="0 0 0" />
+				<origin xyz="0 0 0" rpy="0 1.570796 0" />
 				<geometry>
 					<mesh filename="package://cob_description/meshes/tray_powerball/tray_link_1.stl" />
@@ -39,8 +39,8 @@
 		</link>
 		<joint name="${name}_2_joint" type="revolute">
-			<origin xyz="0.16 0.14 0.22" rpy="0 1.570796 0"/>
+			<origin xyz="0.22 0.14 -0.16" rpy="0 1.570796 0"/>
 			<parent link="${name}_1_link"/>
 			<child link="${name}_2_link"/>
-			<axis xyz="-1 0 0" />
+			<axis xyz="0 0 1" />
 			<calibration rising="${tray_2_ref}"/>
 			<dynamics damping="5.0" friction="0.5"/>
@@ -54,5 +54,5 @@
 			</inertial>
 			<visual>
-				<origin xyz="0 0 0" rpy="0 0 0" />
+				<origin xyz="0 0 0" rpy="0 1.570796 0" />
 				<geometry>
 					<mesh filename="package://cob_description/meshes/tray_powerball/tray_link_2.stl" />
@@ -61,5 +61,5 @@
 			</visual>
 			<collision>
-				<origin xyz="0 0 0" rpy="0 0 0" />
+				<origin xyz="0 0 0" rpy="0 1.570796 0" />
 				<geometry>
 					<mesh filename="package://cob_description/meshes/tray_powerball/tray_link_2.stl" />
@@ -68,8 +68,8 @@
 		</link>
 		<joint name="${name}_3_joint" type="revolute">
-			<origin xyz="-0.067 0.07 0" rpy="-1.570796327 0 1.570796327"/>
+			<origin xyz="0 0.067 0.07" rpy="1.570796 0 0"/>
 			<parent link="${name}_2_link"/>
 			<child link="${name}_3_link"/>
-			<axis xyz="1 0 0" />
+			<axis xyz="0 0 1" />
 			<calibration rising="${tray_3_ref}"/>
 			<dynamics damping="5.0" friction="0.5"/>
@@ -83,5 +83,5 @@
 			</inertial>
 			<visual>
-				<origin xyz="0 0 0" rpy="0 0 0" />
+				<origin xyz="0 0 0" rpy="0 1.570796 0" />
 				<geometry>
 					<mesh filename="package://cob_description/meshes/tray_powerball/tray_link_3.stl" />
@@ -90,5 +90,5 @@
 			</visual>
 			<collision>
-				<origin xyz="0 0 0" rpy="0 0 0" />
+				<origin xyz="0 0 0" rpy="0 1.570796 0" />
 				<geometry>
 					<mesh filename="package://cob_description/meshes/tray_powerball/tray_link_3.stl" />

Commit message: Updated phiget sensors position

File: cob_description/urdf/tray_powerball/tray.urdf.xacro (robot description, xacro)
@@ -97,5 +97,5 @@
 		</link>
 		<joint name="${name}_right_joint" type="fixed" >
-			<origin xyz="0.3741570 0 -0.1146" rpy="0 0 0"/>
+			<origin xyz="-0.1146 0 -0.3741570" rpy="0 0 0"/>
 			<parent link="${name}_3_link" />
 			<child link="${name}_right_link" />
@@ -122,5 +122,5 @@
 		</link>
 		<joint name="${name}_left_joint" type="fixed" >
-			<origin xyz="0.06591570 0 -0.1146" rpy="0 0 0"/>
+			<origin xyz="-0.1146 0 -0.06591570" rpy="0 0 0"/>
 			<parent link="${name}_3_link" />
 			<child link="${name}_left_link" />
@@ -148,14 +148,14 @@
 		<!-- phidgets distance sensors -->
 		<xacro:phidgets_distance_v0 name="${name}_phidgets_1" ros_topic="/tray_sensors/range_1_sim" update_rate="10" parent="${name}_left">
-			<origin xyz="0.07 -0.02424 0.04" rpy="${M_PI/2} 0 0" />
+			<origin xyz="0.04 -0.02424 -0.07  " rpy="0 0 ${M_PI/2}" />
 		</xacro:phidgets_distance_v0>
 		<xacro:phidgets_distance_v0 name="${name}_phidgets_2" ros_topic="/tray_sensors/range_2_sim" update_rate="10" parent="${name}_left">
-			<origin xyz="0.07 -0.02424 0.09" rpy="${M_PI/2} 0 0" />
+			<origin xyz="0.09 -0.02424 -0.07" rpy="0 0 ${M_PI/2}" />
 		</xacro:phidgets_distance_v0>
 		<xacro:phidgets_distance_v0 name="${name}_phidgets_3" ros_topic="/tray_sensors/range_3_sim" update_rate="10" parent="${name}_left">
-			<origin xyz="0.07 -0.02424 0.14" rpy="${M_PI/2} 0 0" />
+			<origin xyz="0.14 -0.02424 -0.07" rpy="0 0 ${M_PI/2}" />
 		</xacro:phidgets_distance_v0>
 		<xacro:phidgets_distance_v0 name="${name}_phidgets_4" ros_topic="/tray_sensors/range_4_sim" update_rate="10" parent="${name}_left">
-			<origin xyz="0.07 -0.02424 0.19" rpy="${M_PI/2} 0 0" />
+			<origin xyz="0.19 -0.02424 -0.07" rpy="0 0 ${M_PI/2}" />
 		</xacro:phidgets_distance_v0>
 		<!-- extensions -->

Commit message: fix meshes and transformation for tray_powerball

File: cob_description/urdf/tray_powerball/tray.urdf.xacro (robot description, xacro)
@@ -25,5 +25,5 @@
 			</inertial>
 			<visual>
-				<origin xyz="0 0 0" rpy="0 1.570796 0" />
+				<origin xyz="0 0 0" rpy="0 0 0" />
 				<geometry>
 					<mesh filename="package://cob_description/meshes/tray_powerball/tray_link_1.stl" />
@@ -32,5 +32,5 @@
 			</visual>
 			<collision>
-				<origin xyz="0 0 0" rpy="0 1.570796 0" />
+				<origin xyz="0 0 0" rpy="0 0 0" />
 				<geometry>
 					<mesh filename="package://cob_description/meshes/tray_powerball/tray_link_1.stl" />
@@ -39,5 +39,5 @@
 		</link>
 		<joint name="${name}_2_joint" type="revolute">
-			<origin xyz="0.22 0.14 -0.16" rpy="0 1.570796 0"/>
+			<origin xyz="0.178 -0.169 0.159" rpy="0 1.570796 0"/>
 			<parent link="${name}_1_link"/>
 			<child link="${name}_2_link"/>
@@ -54,5 +54,5 @@
 			</inertial>
 			<visual>
-				<origin xyz="0 0 0" rpy="0 1.570796 0" />
+				<origin xyz="0 0 0" rpy="0 0 0" />
 				<geometry>
 					<mesh filename="package://cob_description/meshes/tray_powerball/tray_link_2.stl" />
@@ -61,5 +61,5 @@
 			</visual>
 			<collision>
-				<origin xyz="0 0 0" rpy="0 1.570796 0" />
+				<origin xyz="0 0 0" rpy="0 0 0" />
 				<geometry>
 					<mesh filename="package://cob_description/meshes/tray_powerball/tray_link_2.stl" />
@@ -68,5 +68,5 @@
 		</link>
 		<joint name="${name}_3_joint" type="revolute">
-			<origin xyz="0 0.067 0.07" rpy="1.570796 0 0"/>
+			<origin xyz="0.0671 0.0 0.0671" rpy="0 1.570796 0"/>
 			<parent link="${name}_2_link"/>
 			<child link="${name}_3_link"/>
@@ -83,5 +83,5 @@
 			</inertial>
 			<visual>
-				<origin xyz="0 0 0" rpy="0 1.570796 0" />
+				<origin xyz="0 0 0" rpy="0 0 0" />
 				<geometry>
 					<mesh filename="package://cob_description/meshes/tray_powerball/tray_link_3.stl" />
@@ -90,5 +90,5 @@
 			</visual>
 			<collision>
-				<origin xyz="0 0 0" rpy="0 1.570796 0" />
+				<origin xyz="0 0 0" rpy="0 0 0" />
 				<geometry>
 					<mesh filename="package://cob_description/meshes/tray_powerball/tray_link_3.stl" />
@@ -97,5 +97,5 @@
 		</link>
 		<joint name="${name}_right_joint" type="fixed" >
-			<origin xyz="-0.1146 0 -0.3741570" rpy="0 0 0"/>
+			<origin xyz="-0.1146 0 0.3741570" rpy="0 0 0"/>
 			<parent link="${name}_3_link" />
 			<child link="${name}_right_link" />
@@ -122,5 +122,5 @@
 		</link>
 		<joint name="${name}_left_joint" type="fixed" >
-			<origin xyz="-0.1146 0 -0.06591570" rpy="0 0 0"/>
+			<origin xyz="-0.1146 0 0.06591570" rpy="0 0 0"/>
 			<parent link="${name}_3_link" />
 			<child link="${name}_left_link" />
@@ -148,14 +148,14 @@
 		<!-- phidgets distance sensors -->
 		<xacro:phidgets_distance_v0 name="${name}_phidgets_1" ros_topic="/tray_sensors/range_1_sim" update_rate="10" parent="${name}_left">
-			<origin xyz="0.04 -0.02424 -0.07  " rpy="0 0 ${M_PI/2}" />
+			<origin xyz="0.04 -0.02424 0.07  " rpy="0 0 ${M_PI/2}" />
 		</xacro:phidgets_distance_v0>
 		<xacro:phidgets_distance_v0 name="${name}_phidgets_2" ros_topic="/tray_sensors/range_2_sim" update_rate="10" parent="${name}_left">
-			<origin xyz="0.09 -0.02424 -0.07" rpy="0 0 ${M_PI/2}" />
+			<origin xyz="0.09 -0.02424 0.07" rpy="0 0 ${M_PI/2}" />
 		</xacro:phidgets_distance_v0>
 		<xacro:phidgets_distance_v0 name="${name}_phidgets_3" ros_topic="/tray_sensors/range_3_sim" update_rate="10" parent="${name}_left">
-			<origin xyz="0.14 -0.02424 -0.07" rpy="0 0 ${M_PI/2}" />
+			<origin xyz="0.14 -0.02424 0.07" rpy="0 0 ${M_PI/2}" />
 		</xacro:phidgets_distance_v0>
 		<xacro:phidgets_distance_v0 name="${name}_phidgets_4" ros_topic="/tray_sensors/range_4_sim" update_rate="10" parent="${name}_left">
-			<origin xyz="0.19 -0.02424 -0.07" rpy="0 0 ${M_PI/2}" />
+			<origin xyz="0.19 -0.02424 0.07" rpy="0 0 ${M_PI/2}" />
 		</xacro:phidgets_distance_v0>
 		<!-- extensions -->

Commit message: Fixed tray powerball

File: cob_description/urdf/tray_powerball/tray.urdf.xacro (robot description, xacro)
@@ -68,5 +68,5 @@
 		</link>
 		<joint name="${name}_3_joint" type="revolute">
-			<origin xyz="0.0671 0.0 0.0671" rpy="0 1.5708 0"/>
+			<origin xyz="0.0 -0.0671 0.0671" rpy="1.570796 0 0"/>
 			<parent link="${name}_2_link"/>
 			<child link="${name}_3_link"/>

Commit message: Adapt tray position

File: cob_description/urdf/tray_powerball/tray.urdf.xacro (robot description, xacro)
@@ -16,5 +16,5 @@
 			<calibration rising="${tray_1_ref}"/>
 			<dynamics damping="5.0" friction="0.5"/>
-			<limit effort="100" lower="-1.37" upper="0.02" velocity="5"/>
+			<limit effort="100" lower="1.37" upper="-0.02" velocity="5"/>
 		</joint>
 		<link name="${name}_1_link">
