Commit message: renamed components

File: cob_description/urdf/base/base.gazebo.xacro (robot description, xacro)
@@ -4,5 +4,5 @@
        xmlns:interface="http://playerstage.sourceforge.net/gazebo/xmlschema/#interface"
        xmlns:xacro="http://ros.org/wiki/xacro">
-  <xacro:macro name="cob_wheel_gazebo_v0" params="suffix parent">
+  <xacro:macro name="cob_wheel_gazebo" params="suffix parent">
     <gazebo reference="${parent}_${suffix}_wheel_link">
       <mu1 value="100.0" />
@@ -13,10 +13,10 @@
     </gazebo>
   </xacro:macro>
-  <xacro:macro name="cob_caster_gazebo_v0" params="suffix">
+  <xacro:macro name="cob_caster_gazebo" params="suffix">
     <gazebo reference="${suffix}_caster_rotation_link">
       <material value="PR2/caster_texture" />
     </gazebo>
   </xacro:macro>
-  <xacro:macro name="cob_base_gazebo_v0" params="name">
+  <xacro:macro name="cob_base_gazebo" params="name">
     <gazebo reference="${name}_link">
       <selfCollide>true</selfCollide>

File: cob_description/urdf/base/base.transmission.xacro (robot description, xacro)
@@ -5,5 +5,5 @@
        xmlns:xacro="http://ros.org/wiki/xacro">
   <!--  Caster wheel transmission   -->
-  <xacro:macro name="cob_wheel_transmission_v0" params="suffix parent reflect">
+  <xacro:macro name="cob_wheel_transmission" params="suffix parent reflect">
     <transmission type="pr2_mechanism_model/SimpleTransmission" name="${parent}_${suffix}_wheel_trans">
       <actuator name="${parent}_${suffix}_wheel_motor" />
@@ -13,5 +13,5 @@
   </xacro:macro>
   <!-- Hub transmission only -->
-  <xacro:macro name="cob_caster_transmission_v0" params="suffix">
+  <xacro:macro name="cob_caster_transmission" params="suffix">
     <transmission type="pr2_mechanism_model/SimpleTransmission" name="${suffix}_rotation_trans">
       <actuator name="${suffix}_rotation_motor" />

File: cob_description/urdf/base/base.urdf.xacro (robot description, xacro)
@@ -4,9 +4,9 @@
        xmlns:interface="http://playerstage.sourceforge.net/gazebo/xmlschema/#interface"
        xmlns:xacro="http://ros.org/wiki/xacro">
-  <include filename="$(find cob_description)/ros/urdf/base_v0/base.gazebo.xacro" />
-  <include filename="$(find cob_description)/ros/urdf/base_v0/base.transmission.xacro" />
-  <!-- modify here for test -->
-  <include filename="$(find cob_description)/ros/urdf/sensors/sick_s300_laser.urdf.xacro"/>
-  <include filename="$(find cob_description)/ros/urdf/sensors/hokuyo_lx30_laser.urdf.xacro"/>
+  <include filename="$(find cob_description)/urdf/base/base.gazebo.xacro" />
+  <include filename="$(find cob_description)/urdf/base/base.transmission.xacro" />
+  <!-- sensors -->
+  <include filename="$(find cob_description)/urdf/sensors/sick_s300_laser.urdf.xacro"/>
+  <include filename="$(find cob_description)/urdf/sensors/hokuyo_lx30_laser.urdf.xacro"/>
   <!-- DATA SOURCES -->
   <!-- all link offsets, CG, limits are obtained from Function Engineering spreadsheet 090224_link_data.xls unless stated otherwise -->
@@ -60,5 +60,4 @@
         <origin xyz="0 0 0" rpy="${M_PI/2} 0 0" />
         <geometry>
-          <!--mesh filename="package://cob_description/ros/meshes/base_v0/pr2_wheel.stl" /-->
           <cylinder radius="${wheel_radius}" length="${wheel_length}" />
         </geometry>
@@ -99,5 +98,5 @@
 		<origin xyz="0 0 0.002" rpy="0.0 0.0 0.0" />
         <geometry>
-          <!--mesh filename="package://cob_description/ros/meshes/base_v0/caster.stl" /-->  <!--modified by jie-->
+          <!--mesh filename="package://cob_description/meshes/base/caster.stl" /-->  <!--modified by jie-->
           <!--box size="0.192 0.164 0.013" /-->
 		  <box size="0.001 0.001 0.001" />
@@ -127,5 +126,5 @@
   </xacro:macro>
   <!-- The xacro macro xacro:cob_base contains: base, casters and wheels -->
-  <xacro:macro name="cob_base_v1" params="name">
+  <xacro:macro name="cob_base" params="name">
   <link name="${name}_link">
       <inertial>
@@ -138,5 +137,5 @@
         <origin xyz="0 0 0" rpy="0 0 0" />
         <geometry>
-          <mesh filename="package://cob_description/ros/meshes/base_v0/base.stl"/>
+          <mesh filename="package://cob_description/meshes/base/base.stl"/>
           <!--box size="${base_size_x} ${base_size_y} ${base_collision_size_z}" /-->
         </geometry>
@@ -147,5 +146,5 @@
         <geometry>
 		  <!--box size="0.001 0.001 0.001" /-->
-	      <mesh filename="package://cob_description/ros/meshes/base_v0/base_collision.stlb"/>
+	      <mesh filename="package://cob_description/meshes/base/base_collision.stlb"/>
           <!--box size="${base_size_x} ${base_size_y} ${base_collision_size_z}" /-->
         </geometry>
@@ -169,7 +168,5 @@
       </visual>
       <collision>
-        <!-- represent base collision with a simple rectangular model, positioned by base_size_z s.t. top
-             surface of the collision box matches the top surface of the PR2 base -->
-        <origin xyz="0 0 ${0.051+base_collision_size_z/2}" rpy="0 0 0" />
+        <origin xyz="0 0 0" rpy="0 0 0" />
         <geometry>
           <box size="0.001 0.001 0.001" />
@@ -209,5 +206,5 @@
     </xacro:cob_caster_v0>
     <!-- gazebo extensions -->
-    <xacro:cob_base_gazebo_v0 name="${name}" />
+    <xacro:cob_base_gazebo name="${name}" />
   </xacro:macro>
 </robot>

File: cob_description/urdf/head_v3/head.urdf.xacro (robot description, xacro)
@@ -4,9 +4,8 @@
        xmlns:interface="http://playerstage.sourceforge.net/gazebo/xmlschema/#interface"
        xmlns:xacro="http://ros.org/wiki/xacro">
-	<include filename="$(find cob_description)/ros/urdf/head_v3/head.gazebo.xacro" />
-	<include filename="$(find cob_description)/ros/urdf/head_v3/head.transmission.xacro" />
-	<include filename="$(find cob_description)/ros/urdf/sensors/prosilica.urdf.xacro" />
-	<include filename="$(find cob_description)/ros/urdf/sensors/kinect.urdf.xacro" />
-	<!--include filename="$(find cob_description)/ros/urdf/sensors/hokuyo_SR400_laser.urdf.xacro" /-->
+	<include filename="$(find cob_description)/urdf/head_v3/head.gazebo.xacro" />
+	<include filename="$(find cob_description)/urdf/head_v3/head.transmission.xacro" />
+	<include filename="$(find cob_description)/urdf/sensors/prosilica.urdf.xacro" />
+	<include filename="$(find cob_description)/urdf/sensors/kinect.urdf.xacro" />
 	<xacro:macro name="cob_head_v3" params="name parent *origin">
 		<!-- joint between torso_upper_neck_tilt_link and head_axis_link -->
@@ -42,5 +41,5 @@
 		<!-- left camera -->
 		<xacro:cob_prosilica_v0 name="${name}_color_camera_l" ros_topic="stereo/left" parent="${name}_axis_link">
-			<origin xyz="${cam_l_x} ${cam_l_y} ${cam_l_z}-0.06" rpy="${cam_l_roll} ${cam_l_pitch}-1.5708 ${cam_l_yaw}" />
+			<origin xyz="${cam_l_x} ${cam_l_y} ${cam_l_z-0.06}" rpy="${cam_l_roll} ${cam_l_pitch-1.5708} ${cam_l_yaw}" />
 		</xacro:cob_prosilica_v0>
 		<!-- right camera -->

File: cob_description/urdf/lbr/lbr.gazebo.xacro (robot description, xacro)
@@ -4,5 +4,5 @@
        xmlns:interface="http://playerstage.sourceforge.net/gazebo/xmlschema/#interface"
        xmlns:xacro="http://ros.org/wiki/xacro">
-	<xacro:macro name="cob_lbr_gazebo_v0" params="name">
+	<xacro:macro name="cob_lbr_gazebo" params="name">
 		<gazebo reference="${name}_0_link">
 			<material value="PR2/Red" />

File: cob_description/urdf/lbr/lbr.transmission.xacro (robot description, xacro)
@@ -4,5 +4,5 @@
        xmlns:interface="http://playerstage.sourceforge.net/gazebo/xmlschema/#interface"
        xmlns:xacro="http://ros.org/wiki/xacro">
-	<xacro:macro name="cob_lbr_transmission_v0" params="name">
+	<xacro:macro name="cob_lbr_transmission" params="name">
 		<transmission name="${name}_1_trans" type="pr2_mechanism_model/SimpleTransmission">
 			<actuator name="${name}_1_motor"/>

File: cob_description/urdf/lbr/lbr.urdf.xacro (robot description, xacro)
@@ -4,7 +4,7 @@
        xmlns:interface="http://playerstage.sourceforge.net/gazebo/xmlschema/#interface"
        xmlns:xacro="http://ros.org/wiki/xacro">
-	<include filename="$(find cob_description)/ros/urdf/lbr_v0/lbr.gazebo.xacro" />
-	<include filename="$(find cob_description)/ros/urdf/lbr_v0/lbr.transmission.xacro" />
-	<xacro:macro name="cob_lbr_v0" params="parent name *origin">
+	<include filename="$(find cob_description)/urdf/lbr/lbr.gazebo.xacro" />
+	<include filename="$(find cob_description)/urdf/lbr/lbr.transmission.xacro" />
+	<xacro:macro name="cob_lbr" params="parent name *origin">
 		<!-- joint between base_link and arm_0_link -->
 		<joint name="${name}_0_joint" type="fixed" >
@@ -55,12 +55,12 @@
 				<origin xyz="0 0 0" rpy="0 0 0" />
 				<geometry>
-					<mesh filename="package://cob_description/ros/meshes/lbr_v0/joint_1.stl" />
-				</geometry>
-				<material name="Blue" />
-			</visual>
-			<collision>
-				<origin xyz="0 0 0" rpy="0 0 0" />
-				<geometry>
-					<mesh filename="package://cob_description/ros/meshes/lbr_v0/joint_1_collision.stlb" />
+					<mesh filename="package://cob_description/meshes/lbr/joint_1.stl" />
+				</geometry>
+				<material name="Blue" />
+			</visual>
+			<collision>
+				<origin xyz="0 0 0" rpy="0 0 0" />
+				<geometry>
+					<mesh filename="package://cob_description/meshes/lbr/joint_1_collision.stlb" />
 				</geometry>
 			</collision>
@@ -87,12 +87,12 @@
 				<origin xyz="0 0 0" rpy="0 0 0" />
 				<geometry>
-					<mesh filename="package://cob_description/ros/meshes/lbr_v0/joint_2.stl" />
-				</geometry>
-				<material name="Red" />
-			</visual>
-			<collision>
-				<origin xyz="0 0 0" rpy="0 0 0" />
-				<geometry>
-					<mesh filename="package://cob_description/ros/meshes/lbr_v0/joint_2_collision.stlb"/>
+					<mesh filename="package://cob_description/meshes/lbr/joint_2.stl" />
+				</geometry>
+				<material name="Red" />
+			</visual>
+			<collision>
+				<origin xyz="0 0 0" rpy="0 0 0" />
+				<geometry>
+					<mesh filename="package://cob_description/meshes/lbr/joint_2_collision.stlb"/>
 				</geometry>
 			</collision>
@@ -120,12 +120,12 @@
 				<origin xyz="0 0 0" rpy="0 0 0" />
 				<geometry>
-					<mesh filename="package://cob_description/ros/meshes/lbr_v0/joint_3.stl" />
-				</geometry>
-				<material name="Blue" />
-			</visual>
-			<collision>
-				<origin xyz="0 0 0" rpy="0 0 0" />
-				<geometry>
-					<mesh filename="package://cob_description/ros/meshes/lbr_v0/joint_3_collision.stlb"/>
+					<mesh filename="package://cob_description/meshes/lbr/joint_3.stl" />
+				</geometry>
+				<material name="Blue" />
+			</visual>
+			<collision>
+				<origin xyz="0 0 0" rpy="0 0 0" />
+				<geometry>
+					<mesh filename="package://cob_description/meshes/lbr/joint_3_collision.stlb"/>
 				</geometry>
 			</collision>
@@ -153,12 +153,12 @@
 				<origin xyz="0 0 0" rpy="0 0 0" />
 				<geometry>
-					<mesh filename="package://cob_description/ros/meshes/lbr_v0/joint_4.stl" />
-				</geometry>
-				<material name="Red" />
-			</visual>
-			<collision>
-				<origin xyz="0 0 0" rpy="0 0 0" />
-				<geometry>
-					<mesh filename="package://cob_description/ros/meshes/lbr_v0/joint_4_collision.stlb"/>
+					<mesh filename="package://cob_description/meshes/lbr/joint_4.stl" />
+				</geometry>
+				<material name="Red" />
+			</visual>
+			<collision>
+				<origin xyz="0 0 0" rpy="0 0 0" />
+				<geometry>
+					<mesh filename="package://cob_description/meshes/lbr/joint_4_collision.stlb"/>
 				</geometry>
 			</collision>
@@ -185,12 +185,12 @@
 				<origin xyz="0 0 0" rpy="0 0 0" />
 				<geometry>
-					<mesh filename="package://cob_description/ros/meshes/lbr_v0/joint_5.stl" />
-				</geometry>
-				<material name="Blue" />
-			</visual>
-			<collision>
-				<origin xyz="0 0 0" rpy="0 0 0" />
-				<geometry>
-					<mesh filename="package://cob_description/ros/meshes/lbr_v0/joint_5_collision.stlb"/>
+					<mesh filename="package://cob_description/meshes/lbr/joint_5.stl" />
+				</geometry>
+				<material name="Blue" />
+			</visual>
+			<collision>
+				<origin xyz="0 0 0" rpy="0 0 0" />
+				<geometry>
+					<mesh filename="package://cob_description/meshes/lbr/joint_5_collision.stlb"/>
 				</geometry>
 			</collision>
@@ -217,12 +217,12 @@
 				<origin xyz="0 0 0" rpy="0 0 0" />
 				<geometry>
-					<mesh filename="package://cob_description/ros/meshes/lbr_v0/joint_6.stl" />
-				</geometry>
-				<material name="Red" />
-			</visual>
-			<collision>
-				<origin xyz="0 0 0" rpy="0 0 0" />
-				<geometry>
-					<mesh filename="package://cob_description/ros/meshes/lbr_v0/joint_6_collision.stlb"/>
+					<mesh filename="package://cob_description/meshes/lbr/joint_6.stl" />
+				</geometry>
+				<material name="Red" />
+			</visual>
+			<collision>
+				<origin xyz="0 0 0" rpy="0 0 0" />
+				<geometry>
+					<mesh filename="package://cob_description/meshes/lbr/joint_6_collision.stlb"/>
 				</geometry>
 			</collision>
@@ -249,18 +249,18 @@
 				<origin xyz="0 0 0" rpy="0 0 0" />
 				<geometry>
-					<mesh filename="package://cob_description/ros/meshes/lbr_v0/joint_7.stl" />
-				</geometry>
-				<material name="Blue" />
-			</visual>
-			<collision>
-				<origin xyz="0 0 0" rpy="0 0 0" />
-				<geometry>
-					<mesh filename="package://cob_description/ros/meshes/lbr_v0/joint_7_collision.stlb"/>
+					<mesh filename="package://cob_description/meshes/lbr/joint_7.stl" />
+				</geometry>
+				<material name="Blue" />
+			</visual>
+			<collision>
+				<origin xyz="0 0 0" rpy="0 0 0" />
+				<geometry>
+					<mesh filename="package://cob_description/meshes/lbr/joint_7_collision.stlb"/>
 				</geometry>
 			</collision>
 		</link>
 		<!-- extensions -->
-		<xacro:cob_lbr_gazebo_v0 name="${name}" />
-		<xacro:cob_lbr_transmission_v0 name="${name}" />
+		<xacro:cob_lbr_gazebo name="${name}" />
+		<xacro:cob_lbr_transmission name="${name}" />
 	</xacro:macro>
 </robot>

File: cob_description/urdf/sensors/hokuyo_lx30_laser.urdf.xacro (robot description, xacro)
@@ -4,5 +4,5 @@
        xmlns:interface="http://playerstage.sourceforge.net/gazebo/xmlschema/#interface"
        xmlns:xacro="http://ros.org/wiki/xacro">
-  <include filename="$(find cob_description)/ros/urdf/sensors/hokuyo_lx30_laser.gazebo.xacro" />
+  <include filename="$(find cob_description)/urdf/sensors/hokuyo_lx30_laser.gazebo.xacro" />
   <xacro:macro name="hokuyo_lx30_laser_v0" params="name parent *origin ros_topic update_rate min_angle max_angle">
     <joint name="${name}_joint" type="fixed">

File: cob_description/urdf/sensors/kinect.urdf.xacro (robot description, xacro)
@@ -4,5 +4,5 @@
       xmlns:interface="http://playerstage.sourceforge.net/gazebo/xmlschema/#interface"
       xmlns:xacro="http://ros.org/wiki/xacro">
-  <include filename="$(find cob_description)/ros/urdf/sensors/kinect.gazebo.xacro" />
+  <include filename="$(find cob_description)/urdf/sensors/kinect.gazebo.xacro" />
   <xacro:macro name="cob_kinect_v0" params="name parent *origin ros_topic">
     <joint name="${name}_joint" type="fixed">

File: cob_description/urdf/sensors/prosilica.urdf.xacro (robot description, xacro)
@@ -5,5 +5,5 @@
        xmlns:xacro="http://playerstage.sourceforge.net/gazebo/xmlschema/#interface"
        name="LaserBlock">
-	<include filename="$(find cob_description)/ros/urdf/sensors/prosilica.gazebo.xacro" />
+	<include filename="$(find cob_description)/urdf/sensors/prosilica.gazebo.xacro" />
 	<xacro:macro name="cob_prosilica_v0" params="name parent *origin ros_topic">
 		<joint name="${name}_joint" type="fixed">

File: cob_description/urdf/sensors/sick_s300_laser.urdf.xacro (robot description, xacro)
@@ -4,5 +4,5 @@
        xmlns:interface="http://playerstage.sourceforge.net/gazebo/xmlschema/#interface"
        xmlns:xacro="http://ros.org/wiki/xacro">
-  <include filename="$(find cob_description)/ros/urdf/sensors/sick_s300_laser.gazebo.xacro" />
+  <include filename="$(find cob_description)/urdf/sensors/sick_s300_laser.gazebo.xacro" />
   <xacro:macro name="sick_s300_laser_v0" params="name parent *origin ros_topic update_rate min_angle max_angle">
     <joint name="${name}_joint" type="fixed">

File: cob_description/urdf/torso_v0/torso.urdf.xacro (robot description, xacro)
@@ -26,5 +26,5 @@
 				<origin xyz="0 0 0" rpy="0 0 0" />
 				<geometry>
-					<mesh filename="package://cob_description/ros/meshes/torso_v0/tray.stl" />
+					<mesh filename="package://cob_description/meshes/torso_v0/tray.stl" />
 				</geometry>
 				<material name="Green" />
@@ -33,5 +33,5 @@
 				<origin xyz="0 0 0" rpy="0 0 0" />
 				<geometry>
-					<mesh filename="package://cob_description/ros/meshes/torso_v0/tray_collision.stlb" />
+					<mesh filename="package://cob_description/meshes/torso_v0/tray_collision.stlb" />
 				</geometry>
 			</collision>
@@ -86,5 +86,5 @@
 				<origin xyz="0 0 0" rpy="0 0 0" />
 				<geometry>
-					<mesh filename="package://cob_description/ros/meshes/torso_v0/lower_neck.stl" />
+					<mesh filename="package://cob_description/meshes/torso_v0/lower_neck.stl" />
 				</geometry>
 				<material name="Red" />
@@ -93,5 +93,5 @@
 				<origin xyz="0 0 0" rpy="0 0 0" />
 				<geometry>
-					<mesh filename="package://cob_description/ros/meshes/torso_v0/lower_neck_collision.stlb" />
+					<mesh filename="package://cob_description/meshes/torso_v0/lower_neck_collision.stlb" />
 				</geometry>
 			</collision>
@@ -146,5 +146,5 @@
 				<origin xyz="0 0 0" rpy="0 0 0" />
 				<geometry>
-					<mesh filename="package://cob_description/ros/meshes/torso_v0/upper_neck.stl" />
+					<mesh filename="package://cob_description/meshes/torso_v0/upper_neck.stl" />
 				</geometry>
 				<material name="Grey" />
@@ -153,5 +153,5 @@
 				<origin xyz="0 0 0" rpy="0 0 0" />
 				<geometry>
-					<mesh filename="package://cob_description/ros/meshes/torso_v0/upper_neck_collision.stlb" />
+					<mesh filename="package://cob_description/meshes/torso_v0/upper_neck_collision.stlb" />
 				</geometry>
 			</collision>
@@ -172,5 +172,5 @@
 				<origin xyz="0 0 0" rpy="0 0 0" />
 				<geometry>
-					<mesh filename="package://cob_description/ros/meshes/torso_v0/head_cover.stl" />
+					<mesh filename="package://cob_description/meshes/torso_v0/head_cover.stl" />
 				</geometry>
 				<material name="Blue" />
@@ -179,5 +179,5 @@
 				<origin xyz="0 0 0" rpy="0 0 0" />
 				<geometry>
-					<mesh filename="package://cob_description/ros/meshes/torso_v0/head_cover_collision.stlb" />
+					<mesh filename="package://cob_description/meshes/torso_v0/head_cover_collision.stlb" />
 				</geometry>
 			</collision>

File: cob_description/urdf/torso_v1/torso.urdf.xacro (robot description, xacro)
@@ -4,6 +4,6 @@
        xmlns:interface="http://playerstage.sourceforge.net/gazebo/xmlschema/#interface"
        xmlns:xacro="http://ros.org/wiki/xacro">
-	<include filename="$(find cob_description)/ros/urdf/torso_v1/torso.gazebo.xacro" />
-	<include filename="$(find cob_description)/ros/urdf/torso_v1/torso.transmission.xacro" />
+	<include filename="$(find cob_description)/urdf/torso_v1/torso.gazebo.xacro" />
+	<include filename="$(find cob_description)/urdf/torso_v1/torso.transmission.xacro" />
 	<xacro:macro name="cob_torso_v1" params="name parent *origin">
 		<!-- joint between base_link and torso_tray_link -->
@@ -26,5 +26,5 @@
 				<origin xyz="0 0 0" rpy="0 0 0" />
 				<geometry>
-					<mesh filename="package://cob_description/ros/meshes/torso_v0/tray.stl" />
+					<mesh filename="package://cob_description/meshes/torso_v0/tray.stl" />
 				</geometry>
 				<material name="Green" />
@@ -33,5 +33,5 @@
 				<origin xyz="0 0 0" rpy="0 0 0" />
 				<geometry>
-					<mesh filename="package://cob_description/ros/meshes/torso_v0/tray_collision.stlb" />
+					<mesh filename="package://cob_description/meshes/torso_v0/tray_collision.stlb" />
 				</geometry>
 			</collision>
@@ -56,5 +56,5 @@
 				<origin xyz="0 0 0" rpy="3.14 0 0" />
 				<geometry>
-					<mesh filename="package://cob_description/ros/meshes/torso_v0/lower_neck.stl" />
+					<mesh filename="package://cob_description/meshes/torso_v0/lower_neck.stl" />
 				</geometry>
 				<material name="Red" />
@@ -63,5 +63,5 @@
 				<origin xyz="0 0 0" rpy="3.14 0 0" />
 				<geometry>
-					<mesh filename="package://cob_description/ros/meshes/torso_v0/lower_neck_collision.stlb" />
+					<mesh filename="package://cob_description/meshes/torso_v0/lower_neck_collision.stlb" />
 				</geometry>
 			</collision>
@@ -116,5 +116,5 @@
 				<origin xyz="0 0 0" rpy="3.1415926 0 0" />
 				<geometry>
-					<mesh filename="package://cob_description/ros/meshes/torso_v0/upper_neck.stl" />
+					<mesh filename="package://cob_description/meshes/torso_v0/upper_neck.stl" />
 				</geometry>
 				<material name="Grey" />
@@ -123,5 +123,5 @@
 				<origin xyz="0 0 0" rpy="3.1415926 0 0" />
 				<geometry>
-					<mesh filename="package://cob_description/ros/meshes/torso_v0/upper_neck_collision.stlb" />
+					<mesh filename="package://cob_description/meshes/torso_v0/upper_neck_collision.stlb" />
 				</geometry>
 			</collision>
@@ -142,5 +142,5 @@
 				<origin xyz="0 0 0" rpy="0 0 0" />
 				<geometry>
-					<mesh filename="package://cob_description/ros/meshes/torso_v0/head_cover.stl" />
+					<mesh filename="package://cob_description/meshes/torso_v0/head_cover.stl" />
 				</geometry>
 				<material name="Blue" />
@@ -149,5 +149,5 @@
 				<origin xyz="0 0 0" rpy="0 0 0" />
 				<geometry>
-					<mesh filename="package://cob_description/ros/meshes/torso_v0/head_cover_collision.stlb" />
+					<mesh filename="package://cob_description/meshes/torso_v0/head_cover_collision.stlb" />
 				</geometry>
 			</collision>
