Commit message: finished raw3-1 model --- V1

File: cob_description/urdf/base/base.gazebo.xacro (robot description, xacro)
@@ -18,4 +18,9 @@
     </gazebo>
   </xacro:macro>
+  <xacro:macro name="cob_batteries_gazebo" params="name">   <!-- added for raw model - fxmlc -->
+    <gazebo reference="${name}_battery">
+      <material value="PR2/Plug" />
+    </gazebo>
+  </xacro:macro>
   <xacro:macro name="cob_base_gazebo" params="name">
     <gazebo reference="${name}_link">
@@ -31,5 +36,11 @@
         </controller:gazebo_ros_bumper>
       </sensor:contact>
-      <material>Gazebo/Grey</material>
+      <!--material>Gazebo/Grey</material-->
+      <material value="PR2/Grey2" />
+    </gazebo>
+    <gazebo reference="${name}_tower">		<!-- added for raw model - fxmlc -->
+      <selfCollide>true</selfCollide>
+      <!--material>Gazebo/Grey</material-->
+      <material value="PR2/Grey" />
     </gazebo>
     <gazebo>

File: cob_description/urdf/sensors/sick_s300_laser.gazebo.xacro (robot description, xacro)
@@ -27,4 +27,5 @@
         </controller:gazebo_ros_laser>
       </sensor:ray>
+      <material value="PR2/Yellow" />
     </gazebo>
   </xacro:macro>

File: cob_description/urdf/sensors/sick_s300_laser.urdf.xacro (robot description, xacro)
@@ -29,5 +29,5 @@
       </visual>
       <collision>
-        <origin xyz="0 0 0" rpy="${M_PI/2} 0 0" />
+        <origin xyz="0 -0.03 0" rpy="${M_PI/2} 0 0" />
         <geometry>
    	  <!--mesh filename="package://cob_description/meshes/sensors/sick_s300_laser.stlb"/-->

File: raw_description/urdf/base/base.urdf.xacro (robot description, xacro)
@@ -15,13 +15,20 @@
   <property name="M_PI" value="3.1415926535897931" />
   <property name="caster_offset_x" value="0.368" />  <!--modify here-->
-  <property name="caster_offset_y1" value="0.126" />
-  <property name="caster_offset_y2" value="0.178" />
-  <property name="caster_offset_z" value="0.075" />
-  <property name="caster_wheel_offset_y" value="0.000" />
+  <property name="caster_offset_y_fl" value="0.170" />
+  <property name="caster_offset_y_fr" value="0.150" />
+  <property name="caster_offset_y_bl" value="0.120" />
+  <property name="caster_offset_y_br" value="0.200" />
+  <property name="caster_offset_z" value="0.09" />
+  <property name="battery_offset_x_f" value="0.141" />
+  <property name="battery_offset_x_r" value="0.139" />
+  <property name="battery_offset_y_f" value="0.021" />
+  <property name="battery_offset_y_r" value="0.036" />
+  <property name="battery_offset_z" value="0.065" />
+  <property name="caster_wheel_offset_y" value="-0.017" />
   <property name="wheel_length" value="0.034" />
   <property name="wheel_radius" value="0.074792" />   <!-- This is the 'effective' wheel radius. Wheel radius for uncompressed wheel is 0.079.  mp 20080801 -->
-  <property name="base_cg_x" value="0" />
+  <!--property name="base_cg_x" value="0" />
   <property name="base_cg_y" value="0.0" />
-  <property name="base_cg_z" value="0" />
+  <property name="base_cg_z" value="0" /!-->
   <property name="base_mass" value="116.0" />
   <!-- simplified box collision geometry for battery -->
@@ -29,14 +36,8 @@
   <property name="battery_size_y" value="0.48" />
   <property name="battery_size_z" value="0.148" />
-  <!--property name="base_collision_size_z" value="0.04" /-->
-  <!-- simplified box collision geometry for hokuyo laser -->
   <property name="base_laser_x" value="0.465" />
   <property name="base_laser_y_back" value="0.259" />
   <property name="base_laser_y_front" value="0.203" />
   <property name="base_laser_z" value="0.178" />
-  <property name="base_laser_size_x" value="0.06" />
-  <property name="base_laser_size_y" value="0.06" />
-  <property name="base_laser_size_z" value="0.03" />
-  <property name="base_laser_collision_offset_z" value="0.023" />
   <!--                                                      -->
   <!--           wheel                                      -->
@@ -99,13 +100,10 @@
       </inertial>
       <visual>
-        <!--origin xyz="0 0 0.085" rpy="0 0 0" /-->  <!--modified by jie-->
-		<origin xyz="0 0 0.002" rpy="${M_PI/2} 0.0 ${-M_PI/2}" />
-        <geometry>
-          <!--mesh filename="package://cob_description/meshes/base/caster.stl" /-->  <!--modified by jie-->
-          <!--box size="0.192 0.164 0.013" /-->
+        <origin xyz="0 0 0.002" rpy="${M_PI/2} 0.0 ${-M_PI/2}" />
+        <geometry>
 	  <mesh filename="package://raw_description/meshes/base/raw_caster.stlb"/>
 		  <!--box size="0.001 0.001 0.001" /-->
         </geometry>
-        <material name="Grey2" />
+        <material name="Grey" />
       </visual>
       <collision>
@@ -130,4 +128,30 @@
     <xacro:cob_caster_gazebo suffix="${suffix}" />
   </xacro:macro>
+  <!-- battery macros-->
+  <xacro:macro name="cob_batteries" params="name parent *origin ">
+    <joint name="${name}_battery_joint" type="fixed">
+      <insert_block name="origin" />
+      <parent link="${parent}"/>
+      <child link="${name}_battery" />
+    </joint>
+    <link name="${name}_battery">
+       <visual>
+	  <origin xyz="0 0 0" rpy="0 0 0"/>
+	  <geometry>
+            <mesh filename="package://raw_description/meshes/base/raw_battery.stl"/>
+          </geometry>
+          <material name="Red"/>
+        </visual>
+       <collision>
+        <origin xyz="0 0.075 0" rpy="${M_PI/2} ${-M_PI/2} 0"/>
+        <geometry>
+	      <box size="${battery_size_x} ${battery_size_y} ${battery_size_z}" />
+	      <!--mesh filename="package://raw_description/meshes/base/raw_battery.stlb"/-->
+        </geometry>
+        </collision>
+    </link>
+    <!-- extensions -->
+    <xacro:cob_batteries_gazebo name="${name}" />
+  </xacro:macro>
   <!-- The xacro macro xacro:cob_base contains: base, casters and wheels -->
   <xacro:macro name="raw_base" params="name">
@@ -143,14 +167,11 @@
         <geometry>
           <mesh filename="package://raw_description/meshes/base/raw_base.stl"/>
-          <!--box size="${base_size_x} ${base_size_y} ${base_collision_size_z}" /-->
-        </geometry>
-        <material name="Grey2"/>
+        </geometry>
+        <material name="Grey"/>
       </visual>
       <collision>
         <origin xyz="0 0.029 0.219" rpy="${M_PI/2} 0 ${M_PI/2}" />  <!--TODO: fix this in stl orientation not in urdf -->
         <geometry>
-	      <!--box size="0.001 0.001 0.001" /-->
-	      <mesh filename="package://raw_description/meshes/base/raw_base.stlb"/>
-          <!--box size="${base_size_x} ${base_size_y} ${base_collision_size_z}" /-->
+	   <mesh filename="package://raw_description/meshes/base/raw_base.stlb"/>
         </geometry>
       </collision>
@@ -160,47 +181,12 @@
 	  <origin xyz="0 0 0" rpy="${M_PI/2} 0 ${-M_PI/2}"/>
 	  <geometry>
-          <mesh filename="package://raw_description/meshes/base/raw_tower.stl"/>
-          <!--box size="${base_size_x} ${base_size_y} ${base_collision_size_z}" /-->
+            <mesh filename="package://raw_description/meshes/base/raw_tower.stl"/>
           </geometry>
-          <material name="Green"/>
+          <material name="Grey2"/>
         </visual>
        <collision>
         <origin xyz="0 0 0" rpy="${M_PI/2} 0 ${-M_PI/2}"/> <!--TODO: fix this in stl orientation not in urdf -->
         <geometry>
-		  <!--box size="0.001 0.001 0.001" /-->
-	      <mesh filename="package://raw_description/meshes/base/raw_tower_collision.stlb"/>
-          <!--box size="${base_size_x} ${base_size_y} ${base_collision_size_z}" /-->
-        </geometry>
-        </collision>
-    </link>
-    <link name="${name}_battery_front">
-	<visual>
-	  <origin xyz="0 0 0" rpy="${M_PI/2} 0 ${-M_PI/2}"/>
-	  <geometry>
-           <mesh filename="package://raw_description/meshes/base/raw_battery_front.stl"/>
-          </geometry>
-          <material name="Red"/>
-        </visual>
-       <collision>
-        <origin xyz="0 0 0.075" rpy="0 0 0"/>
-        <geometry>
-	      <box size="${battery_size_x} ${battery_size_y} ${battery_size_z}" />
-	      <!--mesh filename="package://raw_description/meshes/base/raw_battery_front.stlb"/-->
-        </geometry>
-        </collision>
-    </link>
-    <link name="${name}_battery_back">
-	<visual>
-	  <origin xyz="0 0 0" rpy="${M_PI/2} 0 ${-M_PI/2}"/>
-	  <geometry>
-            <mesh filename="package://raw_description/meshes/base/raw_battery_back.stl"/>
-          </geometry>
-          <material name="Red"/>
-        </visual>
-       <collision>
-        <origin xyz="0 0 0.075" rpy="0 0 0"/>
-        <geometry>
-	      <box size="${battery_size_x} ${battery_size_y} ${battery_size_z}" />
-	      <!--mesh filename="package://raw_description/meshes/base/raw_battery_back.stlb"/-->
+	   <mesh filename="package://raw_description/meshes/base/raw_tower_collision.stlb"/>
         </geometry>
         </collision>
@@ -237,14 +223,4 @@
       <origin xyz=" -0.36 0 0.48" rpy="0 0 0" /> <!-- with the right offset !-->
       <child link="${name}_tower" />
-      <parent link="${name}_link"/>
-    </joint>
-    <joint name="${name}_battery_front_joint" type="fixed">
-      <origin xyz=" -0.141 0.021 0.065" rpy="0 0 0" />
-      <child link="${name}_battery_front" />
-      <parent link="${name}_link"/>
-    </joint>
-    <joint name="${name}_battery_back_joint" type="fixed">
-      <origin xyz=" 0.139 0.036 0.065" rpy="0 0 0" />
-      <child link="${name}_battery_back" />
       <parent link="${name}_link"/>
     </joint>
@@ -258,16 +234,24 @@
       <origin xyz="${-base_laser_x} ${base_laser_y_back} ${base_laser_z}" rpy="${-M_PI/2} 0 ${-3*M_PI/4}" />
     </xacro:sick_s300_laser_v0>
+    <!-- battery front-->
+    <xacro:cob_batteries name="${name}_battery_front" parent="${name}_link">
+      <origin xyz="${-battery_offset_x_f} ${battery_offset_y_f} ${battery_offset_z}" rpy="${M_PI/2} 0 ${-M_PI/2}" />
+    </xacro:cob_batteries>
+    <!-- battery rear-->
+    <xacro:cob_batteries name="${name}_battery_rear" parent="${name}_link">
+      <origin xyz="${battery_offset_x_r} ${battery_offset_y_r} ${battery_offset_z}" rpy="${M_PI/2} 0 ${-M_PI/2}" />
+    </xacro:cob_batteries>
     <!-- all four caster macros -->
     <xacro:cob_caster suffix="fl" parent="${name}_link" ref_position="${cal_caster_fl - M_PI/4}" >
-      <origin xyz="${-caster_offset_x} ${-caster_offset_y1} ${caster_offset_z}" rpy="0 0 0" />
+      <origin xyz="${-caster_offset_x} ${-caster_offset_y_fl} ${caster_offset_z}" rpy="0 0 0" />
     </xacro:cob_caster>
     <xacro:cob_caster suffix="fr" parent="${name}_link" ref_position="${cal_caster_fr - M_PI/4}" >
-      <origin xyz="${-caster_offset_x} ${caster_offset_y2} ${caster_offset_z}" rpy="0 0 0" />
+      <origin xyz="${-caster_offset_x} ${caster_offset_y_fr} ${caster_offset_z}" rpy="0 0 0" />
     </xacro:cob_caster>
     <xacro:cob_caster suffix="bl" parent="${name}_link" ref_position="${cal_caster_bl - M_PI / 4 + M_PI}" >
-      <origin xyz="${caster_offset_x} ${-caster_offset_y1} ${caster_offset_z}" rpy="0 0 0" />
+      <origin xyz="${caster_offset_x} ${-caster_offset_y_bl} ${caster_offset_z}" rpy="0 0 0" />
     </xacro:cob_caster>
     <xacro:cob_caster suffix="br" parent="${name}_link" ref_position="${cal_caster_br - M_PI / 4 + M_PI}"  >
-      <origin xyz="${caster_offset_x} ${caster_offset_y2} ${caster_offset_z}" rpy="0 0 0" />
+      <origin xyz="${caster_offset_x} ${caster_offset_y_br} ${caster_offset_z}" rpy="0 0 0" />
     </xacro:cob_caster>
     <!-- gazebo extensions -->

File: raw_description/urdf/torso/torso.urdf.xacro (robot description, xacro)
@@ -22,5 +22,5 @@
 			</inertial>
 			<visual>
-				<origin xyz="0 0 0" rpy="0 0 0" />
+				<origin xyz="0 0 -0.26" rpy="0 0 0" />
 				<geometry>
 					<cylinder length="0.521" radius="0.04"/>
@@ -29,5 +29,5 @@
 			</visual>
 			<collision>
-				<origin xyz="0 0 0" rpy="0 0 0" />
+				<origin xyz="0 0 -0.26" rpy="0 0 0" />
 				<geometry>
 					<cylinder length="0.521" radius="0.04"/>

Commit message: undo previous changes in cob_description/urdf/base/base.gazebo.xacro

File: cob_description/urdf/base/base.gazebo.xacro (robot description, xacro)
@@ -18,9 +18,4 @@
     </gazebo>
   </xacro:macro>
-  <xacro:macro name="cob_batteries_gazebo" params="name">   <!-- added for raw model - fxmlc -->
-    <gazebo reference="${name}_battery">
-      <material value="PR2/Plug" />
-    </gazebo>
-  </xacro:macro>
   <xacro:macro name="cob_base_gazebo" params="name">
     <gazebo reference="${name}_link">
@@ -36,11 +31,5 @@
         </controller:gazebo_ros_bumper>
       </sensor:contact>
-      <!--material>Gazebo/Grey</material-->
-      <material value="PR2/Grey2" />
-    </gazebo>
-    <gazebo reference="${name}_tower">		<!-- added for raw model - fxmlc -->
-      <selfCollide>true</selfCollide>
-      <!--material>Gazebo/Grey</material-->
-      <material value="PR2/Grey" />
+      <material>Gazebo/Grey</material>
     </gazebo>
     <gazebo>

Commit message: Renamed colors

File: cob_description/urdf/base/base.gazebo.xacro (robot description, xacro)
@@ -31,5 +31,5 @@
         </controller:gazebo_ros_bumper>
       </sensor:contact>
-      <material>Gazebo/Grey</material>
+      <material>IPA/LightGrey</material>
     </gazebo>
     <gazebo>

File: cob_description/urdf/base/base.urdf.xacro (robot description, xacro)
@@ -53,5 +53,5 @@
           <cylinder radius="${wheel_radius}" length="${wheel_length}" />
         </geometry>
-        <material name="Wheel_${suffix}" />
+        <material name="IPA/Wheel_${suffix}" />
       </visual>
       <collision>
@@ -93,5 +93,5 @@
 		  <box size="0.001 0.001 0.001" />
         </geometry>
-        <material name="Green" />
+        <material name="IPA/LightGrey" />
       </visual>
       <collision>
@@ -156,5 +156,5 @@
           <box size="0.01 0.01 0.01" />
         </geometry>
-        <material name="Red" />
+        <material name="IPA/LightGrey" />
       </visual>
       <collision>

File: cob_description/urdf/head_v2/head.urdf.xacro (robot description, xacro)
@@ -30,5 +30,5 @@
 					<box size="0.01 0.01 0.12"/>
 				</geometry>
-				<material name="Green" />
+				<material name="IPA/LightGrey" />
 			</visual>
 			<collision>

File: cob_description/urdf/materials.urdf.xacro (robot description, xacro)
@@ -1,10 +1,4 @@
 <?xml version="1.0"?>
 <robot>
-	<material name="Blue">
-		<color rgba="0.0 0.0 0.8 1.0"/>
-	</material>
-	<material name="Green">
-		<color rgba="0.0 0.8 0.0 1.0"/>
-	</material>
 	<material name="IPA/DarkGrey">
 		<color rgba="0.7 0.7 0.7 1.0"/>
@@ -12,10 +6,4 @@
 	<material name="IPA/LightGrey">
 		<color rgba="0.81 0.81 0.81 1.0"/>
-	</material>
-	<material name="Red">
-		<color rgba="0.8 0.0 0.0 1.0"/>
-	</material>
-	<material name="White">
-		<color rgba="1.0 1.0 1.0 1.0"/>
 	</material>
 	<material name="IPA/Black">
@@ -25,17 +13,14 @@
 		<color rgba="1.0 0.5 0.0 1.0"/>
 	</material>
-	<material name="Schunk/DarkGolden">
-		<color rgba="0.72 0.5255 0.043 1.0"/>
-	</material>
-	<material name="Caster">
+	<material name="IPA/Caster">
 		<texture filename="package://pr2_ogre/Media/materials/textures/pr2_caster_texture.png" />
 	</material>
-	<material name="Wheel_l">
+	<material name="IPA/Wheel_l">
 		<texture filename="package://pr2_ogre/Media/materials/textures/pr2_wheel_left.png" />
 	</material>
-	<material name="Wheel_r">
+	<material name="IPA/Wheel_r">
 		<texture filename="package://pr2_ogre/Media/materials/textures/pr2_wheel_right.png" />
 	</material>
-	<material name="RollLinks">
+	<material name="IPA/RollLinks">
 		<texture filename="package://pr2_ogre/Media/materials/textures/pr2_wheel_left.png" />
 	</material>

File: cob_description/urdf/sensors/prosilica.gazebo.xacro (robot description, xacro)
@@ -34,5 +34,5 @@
 				</controller:gazebo_ros_prosilica>
 			</sensor:camera>
-			<material value="Gazebo/Black" />
+			<material value="IPA/Black" />
 			<turnGravityOff>true</turnGravityOff>
 		</gazebo>

File: cob_description/urdf/torso_v0/torso.urdf.xacro (robot description, xacro)
@@ -28,5 +28,5 @@
 					<box size="0.01 0.01 0.01"/>
 				</geometry>
-				<material name="Blue" />
+				<material name="IPA/DarkGrey" />
 			</visual>
 			<collision>
@@ -58,5 +58,5 @@
 					<mesh filename="package://cob_description/meshes/torso/lower_neck.stl" />
 				</geometry>
-				<material name="Red" />
+				<material name="IPA/Black" />
 			</visual>
 			<collision>
@@ -88,5 +88,5 @@
 					<box size="0.01 0.01 0.01"/>
 				</geometry>
-				<material name="Blue" />
+				<material name="IPA/DarkGrey" />
 			</visual>
 			<collision>
@@ -144,5 +144,5 @@
 					<mesh filename="package://cob_description/meshes/torso/head_cover.stl" />
 				</geometry>
-				<material name="Blue" />
+				<material name="IPA/Black" />
 			</visual>
 			<collision>

File: cob_description/urdf/tray_powerball/tray.gazebo.xacro (robot description, xacro)
@@ -10,5 +10,5 @@
 		</gazebo>
 		<gazebo reference="${name}_2_link">
-			<material>IPA/DarkGrey</material>
+			<material>IPA/LightGrey</material>
 			<turnGravityOff>false</turnGravityOff>
 		</gazebo>

File: cob_description/urdf/tray_powerball/tray.urdf.xacro (robot description, xacro)
@@ -29,5 +29,5 @@
 					<mesh filename="package://cob_description/meshes/tray_powerball/tray_link_1.stl" />
 				</geometry>
-				<material name="Blue" />
+				<material name="IPA/DarkGrey" />
 			</visual>
 			<collision>
@@ -58,5 +58,5 @@
 					<mesh filename="package://cob_description/meshes/tray_powerball/tray_link_2.stl" />
 				</geometry>
-				<material name="Red" />
+				<material name="IPA/DarkGrey" />
 			</visual>
 			<collision>
@@ -87,5 +87,5 @@
 					<mesh filename="package://cob_description/meshes/tray_powerball/tray_link_3.stl" />
 				</geometry>
-				<material name="Blue" />
+				<material name="IPA/DarkGrey" />
 			</visual>
 			<collision>
@@ -112,5 +112,5 @@
 					<box size="0.001 0.001 0.001" />
 				</geometry>
-				<material name="Red" />
+				<material name="IPA/DarkGrey" />
 			</visual>
 			<collision>
@@ -137,5 +137,5 @@
 					<box size="0.001 0.001 0.001" />
 				</geometry>
-				<material name="Red" />
+				<material name="IPA/DarkGrey" />
 			</visual>
 			<collision>

File: desire_description/urdf/base_desire/base.urdf.xacro (robot description, xacro)
@@ -61,5 +61,5 @@
           <mesh filename="package://cob_description/meshes/base/pr2_wheel.stl" />
         </geometry>
-        <material name="Wheel_${suffix}" />
+        <material name="IPA/Wheel_${suffix}" />
       </visual>
       <collision>
@@ -98,5 +98,5 @@
           <mesh filename="$(find cob_description)/meshes/base/caster.stl" />
         </geometry>
-        <material name="Green" />
+        <material name="IPA/DarkGrey" />
       </visual>
       <collision>
@@ -137,5 +137,5 @@
           <mesh filename="package://desire_description/meshes/base_desire/base.stl"/>
         </geometry>
-        <material name="Green"/>
+        <material name="IPA/DarkGrey" />
       </visual>
       <collision>
@@ -162,5 +162,5 @@
           <box size="0.01 0.01 0.01" />
         </geometry>
-        <material name="Red" />
+        <material name="IPA/DarkGrey" />
       </visual>
       <collision>

File: raw_description/urdf/base/base.gazebo.xacro (robot description, xacro)
@@ -10,15 +10,15 @@
       <kp  value="1000000.0" />
       <kd  value="1.0" />
-      <material value="PR2/wheel_${suffix}" />
+      <material value="IPA/wheel_${suffix}" />
     </gazebo>
   </xacro:macro>
   <xacro:macro name="cob_caster_gazebo" params="suffix">
     <gazebo reference="${suffix}_caster_rotation_link">
-      <material value="PR2/caster_texture" />
+      <material value="IPA/caster_texture" />
     </gazebo>
   </xacro:macro>
   <xacro:macro name="cob_batteries_gazebo" params="name">   <!-- added for raw model - fxmlc -->
     <gazebo reference="${name}_battery">
-      <material value="PR2/Plug" />
+      <material value="IPA/Plug" />
     </gazebo>
   </xacro:macro>
@@ -37,10 +37,10 @@
       </sensor:contact>
       <!--material>Gazebo/Grey</material-->
-      <material value="PR2/Grey2" />
+      <material value="IPA/LightGrey" />
     </gazebo>
     <gazebo reference="${name}_tower">		<!-- added for raw model - fxmlc -->
       <selfCollide>true</selfCollide>
       <!--material>Gazebo/Grey</material-->
-      <material value="PR2/Grey" />
+      <material value="IPA/LightGrey" />
     </gazebo>
     <gazebo>

File: raw_description/urdf/base/base.urdf.xacro (robot description, xacro)
@@ -69,5 +69,5 @@
 	  <mesh filename="package://raw_description/meshes/base/raw_wheel.stl"/>
         </geometry>
-        <material name="Wheel_${suffix}" />
+        <material name="IPA/Wheel_${suffix}" />
       </visual>
       <collision>
@@ -108,5 +108,5 @@
 		  <!--box size="0.001 0.001 0.001" /-->
         </geometry>
-        <material name="Grey" />
+        <material name="IPA/LightGrey" />
       </visual>
       <collision>
@@ -150,5 +150,5 @@
             <mesh filename="package://raw_description/meshes/base/raw_battery.stl"/>
           </geometry>
-          <material name="Red"/>
+        <material name="IPA/LightGrey" />
        </visual>
       <collision>
@@ -177,5 +177,5 @@
           <mesh filename="package://raw_description/meshes/base/raw_base.stl"/>
         </geometry>
-        <material name="Grey"/>
+        <material name="IPA/LightGrey" />
       </visual>
       <collision>
@@ -198,5 +198,5 @@
             <mesh filename="package://raw_description/meshes/base/raw_tower.stl"/>
           </geometry>
-          <material name="Grey2"/>
+        <material name="IPA/LightGrey" />
        </visual>
        <collision>
@@ -226,5 +226,5 @@
           <box size="0.01 0.01 0.01" />
         </geometry>
-        <material name="Red" />
+        <material name="IPA/LightGrey" />
       </visual>
       <collision>

File: raw_description/urdf/torso/torso.urdf.xacro (robot description, xacro)
@@ -26,5 +26,5 @@
 					<cylinder length="0.521" radius="0.04"/>
 				</geometry>
-				<material name="Grey" />
+        		<material name="IPA/LightGrey" />
 			</visual>
 			<collision>
@@ -56,5 +56,5 @@
 					<cylinder length="0.1" radius="0.1"/>
 				</geometry>
-				<material name="Red" />
+                <material name="IPA/LightGrey" />
 			</visual>
 			<collision>
@@ -86,5 +86,5 @@
 					<box size="0.01 0.01 0.01"/>
 				</geometry>
-				<material name="Green" />
+				<material name="IPA/LightGrey" />
 			</visual>
 			<collision>
