Commit message: Deleted texture colors

File: cob_description/urdf/base/base.gazebo.xacro (robot description, xacro)
@@ -10,5 +10,5 @@
       <kp  value="1000000.0" />
       <kd  value="1.0" />
-      <material value="PR2/wheel_${suffix}" />
+      <material>IPA/LightGrey</material>
     </gazebo>
   </xacro:macro>

File: cob_description/urdf/base/base.urdf.xacro (robot description, xacro)
@@ -53,5 +53,5 @@
           <cylinder radius="${wheel_radius}" length="${wheel_length}" />
         </geometry>
-        <material name="IPA/Wheel_${suffix}" />
+        <material name="IPA/LightGrey" />
       </visual>
       <collision>

File: cob_description/urdf/materials.urdf.xacro (robot description, xacro)
@@ -1,27 +1,15 @@
 <?xml version="1.0"?>
 <robot>
+	<material name="IPA/LightGrey">
+		<color rgba="0.81 0.81 0.81 1.0"/>
+	</material>
 	<material name="IPA/DarkGrey">
 		<color rgba="0.7 0.7 0.7 1.0"/>
 	</material>
-	<material name="IPA/LightGrey">
-		<color rgba="0.81 0.81 0.81 1.0"/>
+	<material name="IPA/Orange">
+		<color rgba="1.0 0.5 0.0 1.0"/>
 	</material>
 	<material name="IPA/Black">
 		<color rgba="0.0 0.0 0.0 1.0"/>
 	</material>
-	<material name="IPA/Orange">
-		<color rgba="1.0 0.5 0.0 1.0"/>
-	</material>
-	<material name="IPA/Caster">
-		<texture filename="package://pr2_ogre/Media/materials/textures/pr2_caster_texture.png" />
-	</material>
-	<material name="IPA/Wheel_l">
-		<texture filename="package://pr2_ogre/Media/materials/textures/pr2_wheel_left.png" />
-	</material>
-	<material name="IPA/Wheel_r">
-		<texture filename="package://pr2_ogre/Media/materials/textures/pr2_wheel_right.png" />
-	</material>
-	<material name="IPA/RollLinks">
-		<texture filename="package://pr2_ogre/Media/materials/textures/pr2_wheel_left.png" />
-	</material>
 </robot>

File: raw_description/urdf/base/base.gazebo.xacro (robot description, xacro)
@@ -10,15 +10,15 @@
       <kp  value="1000000.0" />
       <kd  value="1.0" />
-      <material value="IPA/wheel_${suffix}" />
+      <material value="IPA/LightGrey" />
     </gazebo>
   </xacro:macro>
   <xacro:macro name="cob_caster_gazebo" params="suffix">
     <gazebo reference="${suffix}_caster_rotation_link">
-      <material value="IPA/caster_texture" />
+      <material value="IPA/LightGrey" />
     </gazebo>
   </xacro:macro>
   <xacro:macro name="cob_batteries_gazebo" params="name">   <!-- added for raw model - fxmlc -->
     <gazebo reference="${name}_battery">
-      <material value="IPA/Plug" />
+      <material value="IPA/LightGrey" />
     </gazebo>
   </xacro:macro>

File: raw_description/urdf/base/base.urdf.xacro (robot description, xacro)
@@ -69,5 +69,5 @@
 	  <mesh filename="package://raw_description/meshes/base/raw_wheel.stl"/>
         </geometry>
-        <material name="IPA/Wheel_${suffix}" />
+        <material name="IPA/LightGrey" />
       </visual>
       <collision>
