Commit message: fix names in base urdf

File: cob_description/urdf/base/base.urdf.xacro (robot description, xacro)
@@ -40,5 +40,5 @@
   <!--           wheel                                      -->
   <!--                                                      -->
-  <xacro:macro name="cob_wheel_v0" params="suffix parent reflect">
+  <xacro:macro name="cob_wheel" params="suffix parent reflect">
     <joint name="${parent}_${suffix}_wheel_joint" type="continuous">
       <axis xyz="0 1 0" />
@@ -72,9 +72,9 @@
     </link>
     <!-- extensions -->
-    <xacro:cob_wheel_gazebo_v0 parent="${parent}" suffix="${suffix}" />
-    <xacro:cob_wheel_transmission_v0 parent="${parent}" suffix="${suffix}" reflect="${reflect}" />
+    <xacro:cob_wheel_gazebo parent="${parent}" suffix="${suffix}" />
+    <xacro:cob_wheel_transmission parent="${parent}" suffix="${suffix}" reflect="${reflect}" />
   </xacro:macro>
   <!-- Macro for Caster hub only -->
-  <xacro:macro name="cob_caster_hub_v0" params="suffix parent *origin ref_position" >
+  <xacro:macro name="cob_caster_hub" params="suffix parent *origin ref_position" >
     <joint name="${suffix}_rotation_joint" type="continuous">
       <axis xyz="0 0 1" />
@@ -112,16 +112,16 @@
     </link>
     <!-- extensions -->
-    <xacro:cob_caster_transmission_v0 suffix="${suffix}" />
-  </xacro:macro>
-  <xacro:macro name="cob_caster_v0" params="suffix parent *origin ref_position">
-    <xacro:cob_caster_hub_v0 parent="${parent}" suffix="${suffix}_caster"
+    <xacro:cob_caster_transmission suffix="${suffix}" />
+  </xacro:macro>
+  <xacro:macro name="cob_caster" params="suffix parent *origin ref_position">
+    <xacro:cob_caster_hub parent="${parent}" suffix="${suffix}_caster"
                              ref_position="${ref_position}" >
       <insert_block name="origin" />
-    </xacro:cob_caster_hub_v0>
+    </xacro:cob_caster_hub>
     <!-- wheel macros -->
-    <!--xacro:cob_wheel_v0 parent="${suffix}_caster" suffix="l" reflect="1" /--> <!--### modified by jie ###-->
-    <xacro:cob_wheel_v0 parent="${suffix}_caster" suffix="r" reflect="-1" />
+    <!--xacro:cob_wheel parent="${suffix}_caster" suffix="l" reflect="1" /--> <!--### modified by jie ###-->
+    <xacro:cob_wheel parent="${suffix}_caster" suffix="r" reflect="-1" />
     <!-- extensions -->
-    <xacro:cob_caster_gazebo_v0 suffix="${suffix}" />
+    <xacro:cob_caster_gazebo suffix="${suffix}" />
   </xacro:macro>
   <!-- The xacro macro xacro:cob_base contains: base, casters and wheels -->
@@ -193,16 +193,16 @@
     </xacro:hokuyo_lx30_laser_v0>
     <!-- all four caster macros -->
-    <xacro:cob_caster_v0 suffix="fl" parent="${name}_link" ref_position="${cal_caster_fl - M_PI/4}" >
+    <xacro:cob_caster suffix="fl" parent="${name}_link" ref_position="${cal_caster_fl - M_PI/4}" >
       <origin xyz="${caster_offset_x} ${caster_offset_y} ${caster_offset_z}" rpy="0 0 0" />
-    </xacro:cob_caster_v0>
-    <xacro:cob_caster_v0 suffix="fr" parent="${name}_link" ref_position="${cal_caster_fr - M_PI/4}" >
+    </xacro:cob_caster>
+    <xacro:cob_caster suffix="fr" parent="${name}_link" ref_position="${cal_caster_fr - M_PI/4}" >
       <origin xyz="${caster_offset_x} ${-caster_offset_y} ${caster_offset_z}" rpy="0 0 0" />
-    </xacro:cob_caster_v0>
-    <xacro:cob_caster_v0 suffix="bl" parent="${name}_link" ref_position="${cal_caster_bl - M_PI / 4 + M_PI}" >
+    </xacro:cob_caster>
+    <xacro:cob_caster suffix="bl" parent="${name}_link" ref_position="${cal_caster_bl - M_PI / 4 + M_PI}" >
       <origin xyz="${-caster_offset_x} ${caster_offset_y} ${caster_offset_z}" rpy="0 0 0" />
-    </xacro:cob_caster_v0>
-    <xacro:cob_caster_v0 suffix="br" parent="${name}_link" ref_position="${cal_caster_br - M_PI / 4 + M_PI}"  >
+    </xacro:cob_caster>
+    <xacro:cob_caster suffix="br" parent="${name}_link" ref_position="${cal_caster_br - M_PI / 4 + M_PI}"  >
       <origin xyz="${-caster_offset_x} ${-caster_offset_y} ${caster_offset_z}" rpy="0 0 0" />
-    </xacro:cob_caster_v0>
+    </xacro:cob_caster>
     <!-- gazebo extensions -->
     <xacro:cob_base_gazebo name="${name}" />

Commit message: using calibration for laser scanners

File: cob_description/urdf/base/base.urdf.xacro (robot description, xacro)
@@ -29,12 +29,4 @@
   <property name="base_size_z" value="0.23" />
   <property name="base_collision_size_z" value="0.04" />
-  <!-- simplified box collision geometry for hokuyo laser -->
-  <property name="base_laser_x" value="0.325" />
-  <property name="base_laser_y" value="0.0" />
-  <property name="base_laser_z" value="0.135" />
-  <property name="base_laser_size_x" value="0.06" />
-  <property name="base_laser_size_y" value="0.06" />
-  <property name="base_laser_size_z" value="0.03" />
-  <property name="base_laser_collision_offset_z" value="0.023" />
   <!--                                                      -->
   <!--           wheel                                      -->
@@ -182,13 +174,13 @@
     <!-- base laser front -->
     <xacro:sick_s300_laser_v0 name="${name}_laser_front" parent="${name}" ros_topic="scan_front_raw" update_rate="10" min_angle="-2.3562" max_angle="2.3562" >
-      <origin xyz="${base_laser_x} ${base_laser_y} ${base_laser_z}" rpy="0 0 0" />
+      <origin xyz="${laser_front_x} ${laser_front_y} ${laser_front_z}" rpy="${laser_front_roll} ${laser_front_pitch} ${laser_front_yaw}" />
     </xacro:sick_s300_laser_v0>
     <!-- base laser rear -->
     <xacro:sick_s300_laser_v0 name="${name}_laser_rear" parent="${name}" ros_topic="scan_rear_raw" update_rate="10" min_angle="-2.3562" max_angle="2.3562" >
-      <origin xyz="${-base_laser_x} ${base_laser_y} ${base_laser_z}" rpy="0 0 ${M_PI}" />
+      <origin xyz="${laser_rear_x} ${laser_rear_y} ${laser_rear_z}" rpy="${laser_rear_roll} ${laser_rear_pitch} ${laser_rear_yaw}" />
     </xacro:sick_s300_laser_v0>
     <!-- base laser top -->
     <xacro:hokuyo_lx30_laser_v0 name="${name}_laser_top" parent="${name}" ros_topic="scan_top" update_rate="10" min_angle="-2.3562" max_angle="2.3562" >
-      <origin xyz="-0.252 0 0.42" rpy="0 0 0" />
+      <origin xyz="${laser_top_x} ${laser_top_y} ${laser_top_z}" rpy="${laser_top_roll} ${laser_top_pitch} ${laser_top_yaw}" />
     </xacro:hokuyo_lx30_laser_v0>
     <!-- all four caster macros -->

Commit message: changed kinect configuration for fuerte, changed stlb links to stl

File: cob_description/urdf/base/base.urdf.xacro (robot description, xacro)
@@ -137,5 +137,5 @@
         <geometry>
 		  <!--box size="0.001 0.001 0.001" /-->
-	      <mesh filename="package://cob_description/meshes/base/base_collision.stlb"/>
+	      <mesh filename="package://cob_description/meshes/base/base_collision.stl"/>
           <!--box size="${base_size_x} ${base_size_y} ${base_collision_size_z}" /-->
         </geometry>

File: cob_description/urdf/lbr/lbr.urdf.xacro (robot description, xacro)
@@ -61,5 +61,5 @@
 				<origin xyz="0 0 0" rpy="0 0 0" />
 				<geometry>
-					<mesh filename="package://cob_description/meshes/lbr/joint_1_collision.stlb" />
+					<mesh filename="package://cob_description/meshes/lbr/joint_1_collision.stl" />
 				</geometry>
 			</collision>
@@ -93,5 +93,5 @@
 				<origin xyz="0 0 0" rpy="0 0 0" />
 				<geometry>
-					<mesh filename="package://cob_description/meshes/lbr/joint_2_collision.stlb"/>
+					<mesh filename="package://cob_description/meshes/lbr/joint_2_collision.stl"/>
 				</geometry>
 			</collision>
@@ -125,5 +125,5 @@
 				<origin xyz="0 0 0" rpy="0 0 0" />
 				<geometry>
-					<mesh filename="package://cob_description/meshes/lbr/joint_3_collision.stlb"/>
+					<mesh filename="package://cob_description/meshes/lbr/joint_3_collision.stl"/>
 				</geometry>
 			</collision>
@@ -158,5 +158,5 @@
 				<origin xyz="0 0 0" rpy="0 0 0" />
 				<geometry>
-					<mesh filename="package://cob_description/meshes/lbr/joint_4_collision.stlb"/>
+					<mesh filename="package://cob_description/meshes/lbr/joint_4_collision.stl"/>
 				</geometry>
 			</collision>
@@ -189,5 +189,5 @@
 				<origin xyz="0 0 0" rpy="0 0 0" />
 				<geometry>
-					<mesh filename="package://cob_description/meshes/lbr/joint_5_collision.stlb"/>
+					<mesh filename="package://cob_description/meshes/lbr/joint_5_collision.stl"/>
 				</geometry>
 			</collision>
@@ -221,5 +221,5 @@
 				<origin xyz="0 0 0" rpy="0 0 0" />
 				<geometry>
-					<mesh filename="package://cob_description/meshes/lbr/joint_6_collision.stlb"/>
+					<mesh filename="package://cob_description/meshes/lbr/joint_6_collision.stl"/>
 				</geometry>
 			</collision>
@@ -253,5 +253,5 @@
 				<origin xyz="0 0 0" rpy="0 0 0" />
 				<geometry>
-					<mesh filename="package://cob_description/meshes/lbr/joint_7_collision.stlb"/>
+					<mesh filename="package://cob_description/meshes/lbr/joint_7_collision.stl"/>
 				</geometry>
 			</collision>

File: cob_description/urdf/sensors/kinect.gazebo.xacro (robot description, xacro)
@@ -10,22 +10,24 @@
       <imageSize>640 480</imageSize>
       <hfov>57</hfov>
-      <nearClip>0.1</nearClip>
+      <nearClip>0.01</nearClip>
       <farClip>5</farClip>
       <updateRate>20.0</updateRate>
       <baseline>0.2</baseline>
-      <controller:gazebo_ros_camera name="${name}_frame_controller" plugin="libgazebo_ros_camera.so">
+      <controller:gazebo_ros_openni_kinect name="${name}_frame_controller" plugin="libgazebo_ros_openni_kinect.so">
         <alwaysOn>true</alwaysOn>
         <updateRate>20.0</updateRate>
         <imageTopicName>${ros_topic}/rgb/image_raw</imageTopicName>
-        <pointCloudTopicName>${ros_topic}/depth/points</pointCloudTopicName>
         <cameraInfoTopicName>${ros_topic}/camera_info</cameraInfoTopicName>
-        <frameName>/${name}_link</frameName>
+		<depthImageTopicName>${ros_topic}/depth/image_raw</depthImageTopicName>
+        <depthImageInfoTopicName>${ros_topic}/depth/camera_info</depthImageInfoTopicName>
+		<pointCloudTopicName>${ros_topic}/depth/points</pointCloudTopicName>
+		<frameName>/${name}_link</frameName>
         <pointCloudCutoff>0.5</pointCloudCutoff>
-        <distortion_k1>0.00000001</distortion_k1>
-        <distortion_k2>0.00000001</distortion_k2>
-        <distortion_k3>0.00000001</distortion_k3>
-        <distortion_t1>0.00000001</distortion_t1>
-        <distortion_t2>0.00000001</distortion_t2>
-      </controller:gazebo_ros_camera>
+    	<distortionK1>0.00000001</distortionK1>
+        <distortionK2>0.00000001</distortionK2>
+        <distortionK3>0.00000001</distortionK3>
+        <distortionT1>0.00000001</distortionT1>
+        <distortionT2>0.00000001</distortionT2>
+      </controller:gazebo_ros_openni_kinect>
     </sensor:camera>
   </gazebo>

File: cob_description/urdf/torso_v0/torso.urdf.xacro (robot description, xacro)
@@ -63,5 +63,5 @@
 				<origin xyz="0 0 0" rpy="0 0 0" />
 				<geometry>
-					<mesh filename="package://cob_description/meshes/torso/lower_neck_collision.stlb" />
+					<mesh filename="package://cob_description/meshes/torso/lower_neck_collision.stl" />
 				</geometry>
 			</collision>
@@ -123,5 +123,5 @@
 				<origin xyz="0 0 0" rpy="0 0 0" />
 				<geometry>
-					<mesh filename="package://cob_description/meshes/torso/upper_neck_collision.stlb" />
+					<mesh filename="package://cob_description/meshes/torso/upper_neck_collision.stl" />
 				</geometry>
 			</collision>
@@ -149,5 +149,5 @@
 				<origin xyz="0 0 0" rpy="0 0 0" />
 				<geometry>
-					<mesh filename="package://cob_description/meshes/torso/head_cover_collision.stlb" />
+					<mesh filename="package://cob_description/meshes/torso/head_cover_collision.stl" />
 				</geometry>
 			</collision>

File: cob_description/urdf/torso_v1/torso.urdf.xacro (robot description, xacro)
@@ -33,5 +33,5 @@
 				<origin xyz="0 0 0" rpy="${M_PI} 0 0" />
 				<geometry>
-					<mesh filename="package://cob_description/meshes/torso/lower_neck_collision.stlb" />
+					<mesh filename="package://cob_description/meshes/torso/lower_neck_collision.stl" />
 				</geometry>
 			</collision>
@@ -93,5 +93,5 @@
 				<origin xyz="0 0 0" rpy="${M_PI} 0 0" />
 				<geometry>
-					<mesh filename="package://cob_description/meshes/torso/upper_neck_collision.stlb" />
+					<mesh filename="package://cob_description/meshes/torso/upper_neck_collision.stl" />
 				</geometry>
 			</collision>
@@ -119,5 +119,5 @@
 				<origin xyz="0 0 0" rpy="0 0 0" />
 				<geometry>
-					<mesh filename="package://cob_description/meshes/torso/head_cover_collision.stlb" />
+					<mesh filename="package://cob_description/meshes/torso/head_cover_collision.stl" />
 				</geometry>
 			</collision>

File: cob_description/urdf/tray/tray.urdf.xacro (robot description, xacro)
@@ -33,5 +33,5 @@
 				<origin xyz="0 0 0" rpy="0 0 0" />
 				<geometry>
-					<mesh filename="package://cob_description/meshes/tray/tray_collision.stlb" />
+					<mesh filename="package://cob_description/meshes/tray/tray_collision.stl" />
 				</geometry>
 			</collision>

File: raw_description/urdf/base/base.urdf.xacro (robot description, xacro)
@@ -146,5 +146,5 @@
         <geometry>
 		  <!--box size="0.001 0.001 0.001" /-->
-	      <mesh filename="package://raw_description/meshes/base/base.stlb"/>
+	      <mesh filename="package://raw_description/meshes/base/base.stl"/>
           <!--box size="${base_size_x} ${base_size_y} ${base_collision_size_z}" /-->
         </geometry>

Commit message: adjust color settings

File: cob_description/urdf/base/base.urdf.xacro (robot description, xacro)
@@ -131,5 +131,5 @@
           <!--box size="${base_size_x} ${base_size_y} ${base_collision_size_z}" /-->
         </geometry>
-        <material name="IPA/DarkGrey"/>
+        <material name="IPA/LightGrey"/>
       </visual>
       <collision>

File: cob_description/urdf/torso_v1/torso.urdf.xacro (robot description, xacro)
@@ -28,5 +28,5 @@
 					<mesh filename="package://cob_description/meshes/torso/lower_neck.stl" />
 				</geometry>
-				<material name="IPA/DarkGrey" />
+				<material name="IPA/LightGrey" />
 			</visual>
 			<collision>
@@ -58,5 +58,5 @@
 					<box size="0.01 0.01 0.01"/>
 				</geometry>
-				<material name="IPA/Black" />
+				<material name="IPA/LightGrey" />
 			</visual>
 			<collision>
@@ -88,5 +88,5 @@
 					<mesh filename="package://cob_description/meshes/torso/upper_neck.stl" />
 				</geometry>
-				<material name="IPA/DarkGrey" />
+				<material name="IPA/LightGrey" />
 			</visual>
 			<collision>

Commit message: Redefined collisions in urdf files

File: cob_description/urdf/base/base.urdf.xacro (robot description, xacro)
@@ -19,8 +19,10 @@
   <property name="wheel_length" value="0.034" />
   <property name="wheel_radius" value="0.074792" />   <!-- This is the 'effective' wheel radius. Wheel radius for uncompressed wheel is 0.079.  mp 20080801 -->
+  <property name="caster_wheel_offset_y" value="0 " />
   <property name="base_cg_x" value="-0.061" />
   <property name="base_cg_y" value="0.0" />
   <property name="base_cg_z" value="0.293" />
   <property name="base_mass" value="116.0" />
+ <property name="caster_mass" value="5.9" />
   <!-- simplified box collision geometry for base -->
   <property name="base_size_x" value="0.8" />
@@ -80,21 +82,19 @@
     <link name="${suffix}_rotation_link">
       <inertial>
-        <mass value="3.473082"/>
-        <origin xyz="0 0 0.07" />
-        <inertia  ixx="0.012411765597" ixy="-0.000711733678" ixz="0.00050272983"
-                  iyy="0.015218160428" iyz="-0.000004273467" izz="0.011763977943" />
+        <mass value="${caster_mass}"/>
+        <origin xyz="0 0 0" />
+        <inertia  ixx="0.04" ixy="-0.0007" ixz="0.0"
+                  iyy="0.02" iyz="-0.000004" izz="0.05" />
       </inertial>
       <visual>
-        <!--origin xyz="0 0 0.085" rpy="0 0 0" /-->  <!--modified by jie-->
-		<origin xyz="0 0 0.002" rpy="0.0 0.0 0.0" />
+        <origin xyz="0 0 0" rpy="0 0 0" />
         <geometry>
-          <!--mesh filename="package://cob_description/meshes/base/caster.stl" /-->  <!--modified by jie-->
-          <!--box size="0.192 0.164 0.013" /-->
-		  <box size="0.001 0.001 0.001" />
+	  <mesh filename="package://raw_description/meshes/base/raw_caster.stl"/>
+		  <!--box size="0.001 0.001 0.001" /-->
         </geometry>
         <material name="IPA/LightGrey" />
       </visual>
       <collision>
-        <origin xyz="0 0 0.002" rpy="0.0 0.0 0.0" />
+        <origin xyz="0 0 0" rpy="0 0 0" />
         <geometry>
           <box size="0.001 0.001 0.001" />
@@ -136,7 +136,7 @@
         <origin xyz="0 0 0" rpy="0 0 0" />
         <geometry>
-		  <!--box size="0.001 0.001 0.001" /-->
-	      <mesh filename="package://cob_description/meshes/base/base_collision.stl"/>
+	      <!--mesh filename="package://cob_description/meshes/base/base_collision.stl"/-->
           <!--box size="${base_size_x} ${base_size_y} ${base_collision_size_z}" /-->
+          <box size="0 0 0" />
         </geometry>
       </collision>
@@ -144,25 +144,5 @@
     <!-- base_footprint is a fictitious link(frame) that is on the ground right below base_link origin,
          navigation stack dedpends on this frame -->
-    <link name="${name}_footprint">
-      <inertial>
-        <mass value="1.0" />
-        <origin xyz="0 0 0" />
-        <inertia ixx="0.01" ixy="0.0" ixz="0.0"
-                 iyy="0.01" iyz="0.0" izz="0.01" />
-      </inertial>
-      <visual>
-        <origin xyz="0 0 0" rpy="0 0 0" />
-        <geometry>
-          <box size="0.01 0.01 0.01" />
-        </geometry>
-        <material name="IPA/LightGrey" />
-      </visual>
-      <collision>
-        <origin xyz="0 0 0.1" rpy="0 0 0" />
-        <geometry>
-          <box size="0.001 0.001 0.001" />
-        </geometry>
-      </collision>
-    </link>
+    <link name="${name}_footprint"/>
     <joint name="${name}_footprint_joint" type="fixed">
       <origin xyz="0 0 0" rpy="0 0 0" />

Commit message: use collision mesh again

File: cob_description/urdf/base/base.urdf.xacro (robot description, xacro)
@@ -136,7 +136,6 @@
         <origin xyz="0 0 0" rpy="0 0 0" />
         <geometry>
-	      <!--mesh filename="package://cob_description/meshes/base/base_collision.stl"/-->
+	      <mesh filename="package://cob_description/meshes/base/base_collision.stl"/>
           <!--box size="${base_size_x} ${base_size_y} ${base_collision_size_z}" /-->
-          <box size="0 0 0" />
         </geometry>
       </collision>
