Commit message: renamed icob to raw and merged and cleaned up lots of things

File: raw_description/urdf/base/base.urdf.xacro (robot description, xacro)
@@ -138,5 +138,5 @@
         <origin xyz="0 0 0.045" rpy="${M_PI/2} 0 0" />  <!--TODO: fix this in stl orientation not in urdf -->
         <geometry>
-          <mesh filename="package://icob_description/meshes/base/base.stl"/>
+          <mesh filename="package://raw_description/meshes/base/base.stl"/>
           <!--box size="${base_size_x} ${base_size_y} ${base_collision_size_z}" /-->
         </geometry>
@@ -147,5 +147,5 @@
         <geometry>
 		  <!--box size="0.001 0.001 0.001" /-->
-	      <mesh filename="package://icob_description/meshes/base/base.stlb"/>
+	      <mesh filename="package://raw_description/meshes/base/base.stlb"/>
           <!--box size="${base_size_x} ${base_size_y} ${base_collision_size_z}" /-->
         </geometry>

Commit message: changed rotation of laser scanner to work on real robot

File: raw_description/urdf/base/base.urdf.xacro (robot description, xacro)
@@ -183,9 +183,9 @@
     <!-- base laser front -->
     <xacro:sick_s300_laser_v0 name="${name}_laser_front" parent="${name}" ros_topic="scan_front_raw" update_rate="10" min_angle="-2.3562" max_angle="2.3562" >
-      <origin xyz="${base_laser_x} ${-base_laser_y} ${base_laser_z}" rpy="0 0 ${-M_PI/2}" />
+      <origin xyz="${base_laser_x} ${-base_laser_y} ${base_laser_z}" rpy="0 0 ${-M_PI/4}" />
     </xacro:sick_s300_laser_v0>
     <!-- base laser rear -->
     <xacro:sick_s300_laser_v0 name="${name}_laser_rear" parent="${name}" ros_topic="scan_rear_raw" update_rate="10" min_angle="-2.3562" max_angle="2.3562" >
-      <origin xyz="${-base_laser_x} ${base_laser_y} ${base_laser_z}" rpy="0 0 ${M_PI/2}" />
+      <origin xyz="${-base_laser_x} ${base_laser_y} ${base_laser_z}" rpy="0 0 ${3*M_PI/4}" />
     </xacro:sick_s300_laser_v0>
     <!-- all four caster macros -->

Commit message: changed direction of urdf model to new convention

File: raw_description/urdf/base/base.urdf.xacro (robot description, xacro)
@@ -136,5 +136,5 @@
       </inertial>
       <visual>
-        <origin xyz="0 0 0.045" rpy="${M_PI/2} 0 0" />  <!--TODO: fix this in stl orientation not in urdf -->
+        <origin xyz="0 0 0.045" rpy="${M_PI/2} 0 3.14" />  <!--TODO: fix this in stl orientation not in urdf -->
         <geometry>
           <mesh filename="package://raw_description/meshes/base/base.stl"/>

Commit message: added stls and adopted model due to CAD data for raw3-1

File: raw_description/urdf/base/base.urdf.xacro (robot description, xacro)
@@ -25,13 +25,14 @@
   <property name="base_cg_z" value="0" />
   <property name="base_mass" value="116.0" />
-  <!-- simplified box collision geometry for base -->
-  <property name="base_size_x" value="0.94" />
-  <property name="base_size_y" value="0.47" />
-  <property name="base_size_z" value="0.23" />
-  <property name="base_collision_size_z" value="0.04" />
+  <!-- simplified box collision geometry for battery -->
+  <property name="battery_size_x" value="0.24" />
+  <property name="battery_size_y" value="0.48" />
+  <property name="battery_size_z" value="0.148" />
+  <!--property name="base_collision_size_z" value="0.04" /-->
   <!-- simplified box collision geometry for hokuyo laser -->
   <property name="base_laser_x" value="0.465" />
-  <property name="base_laser_y" value="0.232" />
-  <property name="base_laser_z" value="0.15607" />
+  <property name="base_laser_y_back" value="0.259" />
+  <property name="base_laser_y_front" value="0.203" />
+  <property name="base_laser_z" value="0.178" />
   <property name="base_laser_size_x" value="0.06" />
   <property name="base_laser_size_y" value="0.06" />
@@ -59,14 +60,16 @@
       </inertial>
       <visual>
-        <origin xyz="0 0 0" rpy="${M_PI/2} 0 0" />
-        <geometry>
-          <cylinder radius="${wheel_radius}" length="${wheel_length}" />
+        <origin xyz="0 0 0" rpy="0 0 0" />
+        <geometry>
+          <!--cylinder radius="${wheel_radius}" length="${wheel_length}" /-->
+	  <mesh filename="package://raw_description/meshes/base/raw_base_wheel.stlb"/>
         </geometry>
         <material name="Wheel_${suffix}" />
       </visual>
       <collision>
-        <origin xyz="0 0 0" rpy="${M_PI/2} 0 0" /> <!-- rotation because cyl. geom primitive has symmetry axis in +x direction -->
-        <geometry>
-          <cylinder radius="${wheel_radius}" length="${wheel_length}" />
+        <origin xyz="0 0 0" rpy="0 0 0" /> <!-- rotation because cyl. geom primitive has symmetry axis in +x direction -->
+        <geometry>
+          <!--cylinder radius="${wheel_radius}" length="${wheel_length}" /-->
+	  <mesh filename="package://raw_description/meshes/base/raw_base_wheel.stlb"/>
         </geometry>
       </collision>
@@ -97,11 +100,12 @@
       <visual>
         <!--origin xyz="0 0 0.085" rpy="0 0 0" /-->  <!--modified by jie-->
-		<origin xyz="0 0 0.002" rpy="0.0 0.0 0.0" />
+		<origin xyz="0 0 0.002" rpy="${M_PI/2} 0.0 ${-M_PI/2}" />
         <geometry>
           <!--mesh filename="package://cob_description/meshes/base/caster.stl" /-->  <!--modified by jie-->
           <!--box size="0.192 0.164 0.013" /-->
-		  <box size="0.001 0.001 0.001" />
-        </geometry>
-        <material name="Green" />
+	  <mesh filename="package://raw_description/meshes/base/raw_base_caster.stlb"/>
+		  <!--box size="0.001 0.001 0.001" /-->
+        </geometry>
+        <material name="Grey2" />
       </visual>
       <collision>
@@ -127,5 +131,5 @@
   </xacro:macro>
   <!-- The xacro macro xacro:cob_base contains: base, casters and wheels -->
-  <xacro:macro name="icob_base" params="name">
+  <xacro:macro name="raw_base" params="name">
   <link name="${name}_link">
       <inertial>
@@ -136,19 +140,69 @@
       </inertial>
       <visual>
-        <origin xyz="0 0 0.045" rpy="${M_PI/2} 0 0" />  <!--TODO: fix this in stl orientation not in urdf -->
-        <geometry>
-          <mesh filename="package://raw_description/meshes/base/base.stl"/>
-          <!--box size="${base_size_x} ${base_size_y} ${base_collision_size_z}" /-->
-        </geometry>
-        <material name="Green"/>
-      </visual>
-      <collision>
-        <origin xyz="0 0 0.045" rpy="${M_PI/2} 0 0" />  <!--TODO: fix this in stl orientation not in urdf -->
+        <origin xyz="0 0.029 0.219" rpy="${M_PI/2} 0 ${M_PI/2}" />  <!--TODO: fix this in stl orientation not in urdf -->
+        <geometry>
+          <mesh filename="package://raw_description/meshes/base/raw_base_frame.stl"/>
+          <!--box size="${base_size_x} ${base_size_y} ${base_collision_size_z}" /-->
+        </geometry>
+        <material name="Grey2"/>
+      </visual>
+      <collision>
+        <origin xyz="0 0.029 0.219" rpy="${M_PI/2} 0 ${M_PI/2}" />  <!--TODO: fix this in stl orientation not in urdf -->
+        <geometry>
+	      <!--box size="0.001 0.001 0.001" /-->
+	      <mesh filename="package://raw_description/meshes/base/raw_base_frame.stlb"/>
+          <!--box size="${base_size_x} ${base_size_y} ${base_collision_size_z}" /-->
+        </geometry>
+      </collision>
+    </link>
+    <link name="${name}_tower">
+	<visual>
+	  <origin xyz="0 0 0" rpy="${M_PI/2} 0 ${-M_PI/2}"/>
+	  <geometry>
+          <mesh filename="package://raw_description/meshes/base/raw_base_tower.stl"/>
+          <!--box size="${base_size_x} ${base_size_y} ${base_collision_size_z}" /-->
+          </geometry>
+          <material name="Green"/>
+        </visual>
+       <collision>
+        <origin xyz="0 0 0" rpy="${M_PI/2} 0 ${-M_PI/2}"/> <!--TODO: fix this in stl orientation not in urdf -->
         <geometry>
 		  <!--box size="0.001 0.001 0.001" /-->
-	      <mesh filename="package://raw_description/meshes/base/base.stlb"/>
-          <!--box size="${base_size_x} ${base_size_y} ${base_collision_size_z}" /-->
-        </geometry>
-      </collision>
+	      <mesh filename="package://raw_description/meshes/base/raw_base_tower_collision.stlb"/>
+          <!--box size="${base_size_x} ${base_size_y} ${base_collision_size_z}" /-->
+        </geometry>
+        </collision>
+    </link>
+    <link name="${name}_battery_front">
+	<visual>
+	  <origin xyz="0 0 0" rpy="${M_PI/2} 0 ${-M_PI/2}"/>
+	  <geometry>
+           <mesh filename="package://raw_description/meshes/base/raw_base_battery_front.stl"/>
+          </geometry>
+          <material name="Red"/>
+        </visual>
+       <collision>
+        <origin xyz="0 0 0.075" rpy="0 0 0"/>
+        <geometry>
+	      <box size="${battery_size_x} ${battery_size_y} ${battery_size_z}" />
+	      <!--mesh filename="package://raw_description/meshes/base/raw_base_battery_front.stlb"/-->
+        </geometry>
+        </collision>
+    </link>
+    <link name="${name}_battery_back">
+	<visual>
+	  <origin xyz="0 0 0" rpy="${M_PI/2} 0 ${-M_PI/2}"/>
+	  <geometry>
+            <mesh filename="package://raw_description/meshes/base/raw_base_battery_back.stl"/>
+          </geometry>
+          <material name="Red"/>
+        </visual>
+       <collision>
+        <origin xyz="0 0 0.075" rpy="0 0 0"/>
+        <geometry>
+	      <box size="${battery_size_x} ${battery_size_y} ${battery_size_z}" />
+	      <!--mesh filename="package://raw_description/meshes/base/raw_base_battery_back.stlb"/-->
+        </geometry>
+        </collision>
     </link>
     <!-- base_footprint is a fictitious link(frame) that is on the ground right below base_link origin,
@@ -180,30 +234,41 @@
       <parent link="${name}_footprint"/>
     </joint>
+    <joint name="${name}_frame_joint" type="fixed">
+      <origin xyz=" -0.36 0 0.48" rpy="0 0 0" /> <!-- with the right offset !-->
+      <child link="${name}_tower" />
+      <parent link="${name}_link"/>
+    </joint>
+    <joint name="${name}_battery_front_joint" type="fixed">
+      <origin xyz=" -0.141 0.021 0.065" rpy="0 0 0" />
+      <child link="${name}_battery_front" />
+      <parent link="${name}_link"/>
+    </joint>
+    <joint name="${name}_battery_back_joint" type="fixed">
+      <origin xyz=" 0.139 0.036 0.065" rpy="0 0 0" />
+      <child link="${name}_battery_back" />
+      <parent link="${name}_link"/>
+    </joint>
     <!--modify here for test: front,base and top lasers -->
     <!-- base laser front -->
     <xacro:sick_s300_laser_v0 name="${name}_laser_front" parent="${name}" ros_topic="scan_front_raw" update_rate="10" min_angle="-2.3562" max_angle="2.3562" >
-      <origin xyz="${base_laser_x} ${-base_laser_y} ${base_laser_z}" rpy="0 0 ${-M_PI/2}" />
+      <origin xyz="${base_laser_x} ${-base_laser_y_front} ${base_laser_z}" rpy="${-M_PI/2} 0 ${M_PI/4}" />
     </xacro:sick_s300_laser_v0>
     <!-- base laser rear -->
     <xacro:sick_s300_laser_v0 name="${name}_laser_rear" parent="${name}" ros_topic="scan_rear_raw" update_rate="10" min_angle="-2.3562" max_angle="2.3562" >
-      <origin xyz="${-base_laser_x} ${base_laser_y} ${base_laser_z}" rpy="0 0 ${M_PI/2}" />
+      <origin xyz="${-base_laser_x} ${base_laser_y_back} ${base_laser_z}" rpy="${-M_PI/2} 0 ${-3*M_PI/4}" />
     </xacro:sick_s300_laser_v0>
     <!-- all four caster macros -->
     <xacro:cob_caster suffix="fl" parent="${name}_link" ref_position="${cal_caster_fl - M_PI/4}" >
+      <origin xyz="${-caster_offset_x} ${-caster_offset_y1} ${caster_offset_z}" rpy="0 0 0" />
+    </xacro:cob_caster>
+    <xacro:cob_caster suffix="fr" parent="${name}_link" ref_position="${cal_caster_fr - M_PI/4}" >
+      <origin xyz="${-caster_offset_x} ${caster_offset_y2} ${caster_offset_z}" rpy="0 0 0" />
+    </xacro:cob_caster>
+    <xacro:cob_caster suffix="bl" parent="${name}_link" ref_position="${cal_caster_bl - M_PI / 4 + M_PI}" >
+      <origin xyz="${caster_offset_x} ${-caster_offset_y1} ${caster_offset_z}" rpy="0 0 0" />
+    </xacro:cob_caster>
+    <xacro:cob_caster suffix="br" parent="${name}_link" ref_position="${cal_caster_br - M_PI / 4 + M_PI}"  >
       <origin xyz="${caster_offset_x} ${caster_offset_y2} ${caster_offset_z}" rpy="0 0 0" />
     </xacro:cob_caster>
-    <xacro:cob_caster suffix="fr" parent="${name}_link" ref_position="${cal_caster_fr - M_PI/4}" >
-      <origin xyz="${caster_offset_x} ${-caster_offset_y1} ${caster_offset_z}" rpy="0 0 0" />
-    </xacro:cob_caster>
-    <xacro:cob_caster suffix="bl" parent="${name}_link" ref_position="${cal_caster_bl - M_PI / 4 + M_PI}" >
-      <origin xyz="${-caster_offset_x} ${caster_offset_y1} ${caster_offset_z}" rpy="0 0 0" />
-    </xacro:cob_caster>
-    <xacro:cob_caster suffix="br" parent="${name}_link" ref_position="${cal_caster_br - M_PI / 4 + M_PI}"  >
-      <origin xyz="${-caster_offset_x} ${-caster_offset_y2} ${caster_offset_z}" rpy="0 0 0" />
-    </xacro:cob_caster>
-   <!-- cam3d -->
-   <xacro:cob_kinect_v0 name="${name}_cam3d" ros_topic="cam3d" parent="${name}_link">
-      <origin xyz="0.51 0.12 0.27" rpy="-1.57 0 -1.57" />
-   </xacro:cob_kinect_v0>
     <!-- gazebo extensions -->
     <xacro:cob_base_gazebo name="${name}" />

Commit message: added new stls for raw base

File: raw_description/urdf/base/base.urdf.xacro (robot description, xacro)
@@ -63,5 +63,5 @@
         <geometry>
           <!--cylinder radius="${wheel_radius}" length="${wheel_length}" /-->
-	  <mesh filename="package://raw_description/meshes/base/raw_base_wheel.stlb"/>
+	  <mesh filename="package://raw_description/meshes/base/raw_wheel.stlb"/>
         </geometry>
         <material name="Wheel_${suffix}" />
@@ -71,5 +71,5 @@
         <geometry>
           <!--cylinder radius="${wheel_radius}" length="${wheel_length}" /-->
-	  <mesh filename="package://raw_description/meshes/base/raw_base_wheel.stlb"/>
+	  <mesh filename="package://raw_description/meshes/base/raw_wheel.stlb"/>
         </geometry>
       </collision>
@@ -104,5 +104,5 @@
           <!--mesh filename="package://cob_description/meshes/base/caster.stl" /-->  <!--modified by jie-->
           <!--box size="0.192 0.164 0.013" /-->
-	  <mesh filename="package://raw_description/meshes/base/raw_base_caster.stlb"/>
+	  <mesh filename="package://raw_description/meshes/base/raw_caster.stlb"/>
 		  <!--box size="0.001 0.001 0.001" /-->
         </geometry>
@@ -142,5 +142,5 @@
         <origin xyz="0 0.029 0.219" rpy="${M_PI/2} 0 ${M_PI/2}" />  <!--TODO: fix this in stl orientation not in urdf -->
         <geometry>
-          <mesh filename="package://raw_description/meshes/base/raw_base_frame.stl"/>
+          <mesh filename="package://raw_description/meshes/base/raw_base.stl"/>
           <!--box size="${base_size_x} ${base_size_y} ${base_collision_size_z}" /-->
         </geometry>
@@ -151,5 +151,5 @@
         <geometry>
 	      <!--box size="0.001 0.001 0.001" /-->
-	      <mesh filename="package://raw_description/meshes/base/raw_base_frame.stlb"/>
+	      <mesh filename="package://raw_description/meshes/base/raw_base.stlb"/>
           <!--box size="${base_size_x} ${base_size_y} ${base_collision_size_z}" /-->
         </geometry>
@@ -160,5 +160,5 @@
 	  <origin xyz="0 0 0" rpy="${M_PI/2} 0 ${-M_PI/2}"/>
 	  <geometry>
-          <mesh filename="package://raw_description/meshes/base/raw_base_tower.stl"/>
+          <mesh filename="package://raw_description/meshes/base/raw_tower.stl"/>
           <!--box size="${base_size_x} ${base_size_y} ${base_collision_size_z}" /-->
           </geometry>
@@ -169,5 +169,5 @@
         <geometry>
 		  <!--box size="0.001 0.001 0.001" /-->
-	      <mesh filename="package://raw_description/meshes/base/raw_base_tower_collision.stlb"/>
+	      <mesh filename="package://raw_description/meshes/base/raw_tower_collision.stlb"/>
           <!--box size="${base_size_x} ${base_size_y} ${base_collision_size_z}" /-->
         </geometry>
@@ -178,5 +178,5 @@
 	  <origin xyz="0 0 0" rpy="${M_PI/2} 0 ${-M_PI/2}"/>
 	  <geometry>
-           <mesh filename="package://raw_description/meshes/base/raw_base_battery_front.stl"/>
+           <mesh filename="package://raw_description/meshes/base/raw_battery_front.stl"/>
           </geometry>
           <material name="Red"/>
@@ -186,5 +186,5 @@
         <geometry>
 	      <box size="${battery_size_x} ${battery_size_y} ${battery_size_z}" />
-	      <!--mesh filename="package://raw_description/meshes/base/raw_base_battery_front.stlb"/-->
+	      <!--mesh filename="package://raw_description/meshes/base/raw_battery_front.stlb"/-->
         </geometry>
         </collision>
@@ -194,5 +194,5 @@
 	  <origin xyz="0 0 0" rpy="${M_PI/2} 0 ${-M_PI/2}"/>
 	  <geometry>
-            <mesh filename="package://raw_description/meshes/base/raw_base_battery_back.stl"/>
+            <mesh filename="package://raw_description/meshes/base/raw_battery_back.stl"/>
           </geometry>
           <material name="Red"/>
@@ -202,5 +202,5 @@
         <geometry>
 	      <box size="${battery_size_x} ${battery_size_y} ${battery_size_z}" />
-	      <!--mesh filename="package://raw_description/meshes/base/raw_base_battery_back.stlb"/-->
+	      <!--mesh filename="package://raw_description/meshes/base/raw_battery_back.stlb"/-->
         </geometry>
         </collision>

Commit message: final raw-model

File: raw_description/urdf/base/base.urdf.xacro (robot description, xacro)
@@ -15,8 +15,8 @@
   <property name="M_PI" value="3.1415926535897931" />
   <property name="caster_offset_x" value="0.368" />  <!--modify here-->
-  <property name="caster_offset_y_fl" value="0.170" />
-  <property name="caster_offset_y_fr" value="0.150" />
-  <property name="caster_offset_y_bl" value="0.120" />
-  <property name="caster_offset_y_br" value="0.200" />
+  <property name="caster_offset_y_fl" value="0.155" />
+  <property name="caster_offset_y_fr" value="0.165" />
+  <property name="caster_offset_y_bl" value="0.105" />
+  <property name="caster_offset_y_br" value="0.215" />
   <property name="caster_offset_z" value="0.09" />
   <property name="battery_offset_x_f" value="0.141" />
@@ -25,5 +25,5 @@
   <property name="battery_offset_y_r" value="0.036" />
   <property name="battery_offset_z" value="0.065" />
-  <property name="caster_wheel_offset_y" value="-0.017" />
+  <property name="caster_wheel_offset_y" value="0 " />
   <property name="wheel_length" value="0.034" />
   <property name="wheel_radius" value="0.074792" />   <!-- This is the 'effective' wheel radius. Wheel radius for uncompressed wheel is 0.079.  mp 20080801 -->
@@ -31,5 +31,8 @@
   <property name="base_cg_y" value="0.0" />
   <property name="base_cg_z" value="0" /!-->
-  <property name="base_mass" value="116.0" />
+  <property name="base_mass" value="83.1" />
+  <property name="battery_mass" value="83.1" />  <!--to be checked out-->
+ <property name="caster_mass" value="5.9" />
+  <property name="tower_mass" value="6.49" />
   <!-- simplified box collision geometry for battery -->
   <property name="battery_size_x" value="0.24" />
@@ -94,8 +97,8 @@
     <link name="${suffix}_rotation_link">
       <inertial>
-        <mass value="3.473082"/>
-        <origin xyz="0 0 0.07" />
-        <inertia  ixx="0.012411765597" ixy="-0.000711733678" ixz="0.00050272983"
-                  iyy="0.015218160428" iyz="-0.000004273467" izz="0.011763977943" />
+        <mass value="${caster_mass}"/>
+        <origin xyz="0 0 0" />
+        <inertia  ixx="0.04" ixy="-0.0007" ixz="0.0"
+                  iyy="0.02" iyz="-0.000004" izz="0.05" />
       </inertial>
       <visual>
@@ -136,5 +139,11 @@
     </joint>
     <link name="${name}_battery">
-       <visual>
+      <inertial>
+        <mass value="1.0" />
+        <origin xyz="0 0 0" />
+        <inertia ixx="0.01" ixy="0.0" ixz="0.0"
+                 iyy="0.01" iyz="0.0" izz="0.01" />
+      </inertial>
+      <visual>
 	  <origin xyz="0 0 0" rpy="0 0 0"/>
 	  <geometry>
@@ -142,6 +151,6 @@
           </geometry>
           <material name="Red"/>
-        </visual>
-       <collision>
+       </visual>
+      <collision>
         <origin xyz="0 0.075 0" rpy="${M_PI/2} ${-M_PI/2} 0"/>
         <geometry>
@@ -149,5 +158,5 @@
 	      <!--mesh filename="package://raw_description/meshes/base/raw_battery.stlb"/-->
         </geometry>
-        </collision>
+       </collision>
     </link>
     <!-- extensions -->
@@ -160,6 +169,6 @@
         <mass value="${base_mass}" />
         <origin xyz="0 0 0" />
-        <inertia ixx="5.652232699207" ixy="-0.009719934438" ixz="1.293988226423"
-                 iyy="5.669473158652" iyz="-0.007379583694" izz="3.683196351726" />
+        <inertia ixx="9.64" ixy="-0.02" ixz="0.44"
+                 iyy="11.33" iyz="-0.007" izz="3.07" />
       </inertial>
       <visual>
@@ -178,5 +187,11 @@
     </link>
     <link name="${name}_tower">
-	<visual>
+      <inertial>
+        <mass value="${tower_mass}" />
+        <origin xyz="0 0 0" />
+        <inertia ixx="0.1" ixy="0.002" ixz="0.01"
+                 iyy="0.26" iyz="0.0" izz="0.24" />
+      </inertial>
+      <visual>
 	  <origin xyz="0 0 0" rpy="${M_PI/2} 0 ${-M_PI/2}"/>
 	  <geometry>
@@ -184,5 +199,5 @@
           </geometry>
           <material name="Grey2"/>
-        </visual>
+       </visual>
        <collision>
         <origin xyz="0 0 0" rpy="${M_PI/2} 0 ${-M_PI/2}"/> <!--TODO: fix this in stl orientation not in urdf -->
