Commit message: use stl

File: raw_description/urdf/base/base.urdf.xacro (robot description, xacro)
@@ -67,5 +67,5 @@
         <geometry>
           <!--cylinder radius="${wheel_radius}" length="${wheel_length}" /-->
-	  <mesh filename="package://raw_description/meshes/base/raw_wheel.stlb"/>
+	  <mesh filename="package://raw_description/meshes/base/raw_wheel.stl"/>
         </geometry>
         <material name="Wheel_${suffix}" />
@@ -75,5 +75,5 @@
         <geometry>
           <!--cylinder radius="${wheel_radius}" length="${wheel_length}" /-->
-	  <mesh filename="package://raw_description/meshes/base/raw_wheel.stlb"/>
+	  <mesh filename="package://raw_description/meshes/base/raw_wheel.stl"/>
         </geometry>
       </collision>
@@ -105,5 +105,5 @@
         <origin xyz="0 0 0.002" rpy="${M_PI/2} 0.0 ${-M_PI/2}" />
         <geometry>
-	  <mesh filename="package://raw_description/meshes/base/raw_caster.stlb"/>
+	  <mesh filename="package://raw_description/meshes/base/raw_caster.stl"/>
 		  <!--box size="0.001 0.001 0.001" /-->
         </geometry>
@@ -156,5 +156,5 @@
         <geometry>
 	      <box size="${battery_size_x} ${battery_size_y} ${battery_size_z}" />
-	      <!--mesh filename="package://raw_description/meshes/base/raw_battery.stlb"/-->
+	      <!--mesh filename="package://raw_description/meshes/base/raw_battery.stl"/-->
         </geometry>
        </collision>
@@ -182,5 +182,5 @@
         <origin xyz="0 0.029 0.219" rpy="${M_PI/2} 0 ${M_PI/2}" />  <!--TODO: fix this in stl orientation not in urdf -->
         <geometry>
-	   <mesh filename="package://raw_description/meshes/base/raw_base.stlb"/>
+	   <mesh filename="package://raw_description/meshes/base/raw_base.stl"/>
         </geometry>
       </collision>
@@ -203,5 +203,5 @@
         <origin xyz="0 0 0" rpy="${M_PI/2} 0 ${-M_PI/2}"/> <!--TODO: fix this in stl orientation not in urdf -->
         <geometry>
-	   <mesh filename="package://raw_description/meshes/base/raw_tower_collision.stlb"/>
+	   <mesh filename="package://raw_description/meshes/base/raw_tower_collision.stl"/>
         </geometry>
         </collision>

Commit message: adapted raw_torso files

File: raw_description/urdf/base/base.urdf.xacro (robot description, xacro)
@@ -271,7 +271,7 @@
     </xacro:cob_caster>
    <!-- cam3d -->
-   <xacro:cob_kinect_v0 name="${name}_cam3d" ros_topic="cam3d" parent="${name}_link">
+   <!--xacro:cob_kinect_v0 name="${name}_cam3d" ros_topic="cam3d" parent="${name}_link">
       <origin xyz="0.51 0.12 0.27" rpy="-${M_PI/2} 0 -${M_PI/2}" />
-   </xacro:cob_kinect_v0>
+   </xacro:cob_kinect_v0-->
     <!-- gazebo extensions -->
     <xacro:cob_base_gazebo name="${name}" />

File: raw_description/urdf/torso/torso.gazebo.xacro (robot description, xacro)
@@ -4,23 +4,15 @@
        xmlns:interface="http://playerstage.sourceforge.net/gazebo/xmlschema/#interface"
        xmlns:xacro="http://ros.org/wiki/xacro">
-	<xacro:macro name="cob_torso_gazebo_v1" params="name">
-		<gazebo reference="${name}_tray_link">
-			<material>Gazebo/Green</material>
-			<turnGravityOff>false</turnGravityOff>
-		</gazebo>
-		<gazebo reference="${name}_lower_neck_tilt_link">
-			<material>Gazebo/Red</material>
-			<turnGravityOff>false</turnGravityOff>
-		</gazebo>
-		<gazebo reference="${name}_pan_link">
-			<material>Gazebo/Blue</material>
-			<turnGravityOff>false</turnGravityOff>
-		</gazebo>
-		<gazebo reference="${name}_upper_neck_tilt_link">
+	<xacro:macro name="raw_torso_gazebo" params="name">
+		<gazebo reference="${name}_0_link">
 			<material>Gazebo/Grey</material>
 			<turnGravityOff>false</turnGravityOff>
 		</gazebo>
-		<gazebo reference="head_cover_link">
-			<material>Gazebo/Blue</material>
+		<gazebo reference="${name}_tilt_link">
+			<material>Gazebo/Grey</material>
+			<turnGravityOff>false</turnGravityOff>
+		</gazebo>
+		<gazebo reference="head_axis_link">
+			<material>Gazebo/Grey</material>
 			<turnGravityOff>false</turnGravityOff>
 		</gazebo>

File: raw_description/urdf/torso/torso.transmission.xacro (robot description, xacro)
@@ -4,23 +4,13 @@
        xmlns:interface="http://playerstage.sourceforge.net/gazebo/xmlschema/#interface"
        xmlns:xacro="http://ros.org/wiki/xacro">
-	<xacro:macro name="cob_torso_transmission_v1" params="name">
-		<transmission name="${name}_tray_trans" type="pr2_mechanism_model/SimpleTransmission">
-			<actuator name="${name}_tray_motor"/>
-			<joint name="${name}_tray_joint"/>
+	<xacro:macro name="raw_torso_transmission" params="name">
+		<transmission name="${name}_tilt_trans" type="pr2_mechanism_model/SimpleTransmission">
+			<actuator name="${name}_tilt_motor"/>
+			<joint name="${name}_tilt_joint"/>
 			<mechanicalReduction>1</mechanicalReduction>
 		</transmission>
-		<transmission name="${name}_lower_neck_tilt_trans" type="pr2_mechanism_model/SimpleTransmission">
-			<actuator name="${name}_lower_neck_tilt_motor"/>
-			<joint name="${name}_lower_neck_tilt_joint"/>
-			<mechanicalReduction>1</mechanicalReduction>
-		</transmission>
-		<transmission name="${name}_pan_trans" type="pr2_mechanism_model/SimpleTransmission">
-			<actuator name="${name}_pan_motor"/>
-			<joint name="${name}_pan_joint"/>
-			<mechanicalReduction>1</mechanicalReduction>
-		</transmission>
-		<transmission name="${name}_upper_neck_tilt_trans" type="pr2_mechanism_model/SimpleTransmission">
-			<actuator name="${name}_upper_neck_tilt_motor"/>
-			<joint name="${name}_upper_neck_tilt_joint"/>
+		<transmission name="head_axis_trans" type="pr2_mechanism_model/SimpleTransmission">
+			<actuator name="head_axis_motor"/>
+			<joint name="head_axis_joint"/>
 			<mechanicalReduction>1</mechanicalReduction>
 		</transmission>

File: raw_description/urdf/torso/torso.urdf.xacro (robot description, xacro)
@@ -8,5 +8,5 @@
 	<include filename="$(find cob_description)/urdf/sensors/prosilica.urdf.xacro" />
 	<include filename="$(find cob_description)/urdf/sensors/kinect.urdf.xacro" />
-	<xacro:macro name="cob_torso_v1" params="name parent *origin">
+	<xacro:macro name="raw_torso" params="name parent *origin">
 		<!-- joint between base_link and torso_tilt_link -->
 		<joint name="${name}_0_joint" type="fixed" >
@@ -108,6 +108,6 @@
 		</xacro:cob_kinect_v0>
 		<!-- extensions -->
-		<xacro:cob_torso_gazebo_v1 name="${name}" />
-		<xacro:cob_torso_transmission_v1 name="${name}" />
+		<xacro:raw_torso_gazebo name="${name}" />
+		<xacro:raw_torso_transmission name="${name}" />
 	</xacro:macro>
 </robot>

Commit message: flipped front to back like on real robot

File: raw_description/urdf/base/base.urdf.xacro (robot description, xacro)
@@ -208,5 +208,5 @@
     </link>
     <joint name="${name}_frame_joint" type="fixed">
-      <origin xyz=" -0.36 0.029 0.48" rpy="0 0 0" />
+      <origin xyz=" 0.36 -0.029 0.48" rpy="0 0 3.14159265" />
       <child link="${name}_tower" />
       <parent link="${name}_link"/>

Commit message: simpler collision geometries

File: raw_description/urdf/base/base.urdf.xacro (robot description, xacro)
@@ -74,6 +74,6 @@
         <origin xyz="0 0 0" rpy="0 0 0" /> <!-- rotation because cyl. geom primitive has symmetry axis in +x direction -->
         <geometry>
-          <!--cylinder radius="${wheel_radius}" length="${wheel_length}" /-->
-	  <mesh filename="package://raw_description/meshes/base/raw_wheel.stl"/>
+          <sphere radius="${wheel_radius}"/>
+	  <!--mesh filename="package://raw_description/meshes/base/raw_wheel.stl"/-->
         </geometry>
       </collision>
@@ -180,7 +180,8 @@
       </visual>
       <collision>
-        <origin xyz="0 0 0" rpy="0 0 0" />
-        <geometry>
-	   <mesh filename="package://raw_description/meshes/base/raw_base.stl"/>
+        <origin xyz="0 0 0.17" rpy="0 0 0" />
+        <geometry>
+	   <!--mesh filename="package://raw_description/meshes/base/raw_base.stl"/-->
+	   <box size="1.04 0.58 0.31" />
         </geometry>
       </collision>
@@ -201,7 +202,8 @@
        </visual>
        <collision>
-        <origin xyz="0 0 0" rpy="0 0 0"/>
-        <geometry>
-	   <mesh filename="package://raw_description/meshes/base/raw_tower_collision.stl"/>
+        <origin xyz="0 -0.03 -0.1" rpy="0 0 0"/>
+        <geometry>
+	   <!--mesh filename="package://raw_description/meshes/base/raw_tower_collision.stl"/-->
+	   <box size="0.32 0.58 0.24" />
         </geometry>
         </collision>

File: raw_description/urdf/torso/torso.urdf.xacro (robot description, xacro)
@@ -54,5 +54,5 @@
 				<origin xyz="0 0 0" rpy="3.14 0 0" />
 				<geometry>
-					<cylinder length="0.1" radius="0.1"/>
+					<cylinder length="0.3" radius="0.15"/>
 				</geometry>
                 <material name="IPA/LightGrey" />
@@ -61,5 +61,5 @@
 				<origin xyz="0 0 0" rpy="3.14 0 0" />
 				<geometry>
-					<cylinder length="0.1" radius="0.1"/>
+					<cylinder length="0.3" radius="0.15"/>
 				</geometry>
 			</collision>

Commit message: go back to using mesh for collision instead of big box - box makes robot not movable within gazebo

File: raw_description/urdf/base/base.urdf.xacro (robot description, xacro)
@@ -180,9 +180,12 @@
       </visual>
       <collision>
-        <origin xyz="0 0 0.17" rpy="0 0 0" />
-        <geometry>
-	   <!--mesh filename="package://raw_description/meshes/base/raw_base.stl"/-->
-	   <box size="1.04 0.58 0.31" />
-        </geometry>
+		<origin xyz="0 0 0.0" rpy="0 0 0" />
+        <geometry>
+			<mesh filename="package://raw_description/meshes/base/raw_base.stl"/>
+        </geometry>
+        <!--origin xyz="0 0 0.17" rpy="0 0 0" />
+        <geometry>
+			<box size="1.04 0.58 0.31" />
+        </geometry-->
       </collision>
     </link>

Commit message: mainly beautifying

File: raw_description/urdf/base/base.urdf.xacro (robot description, xacro)
@@ -33,5 +33,5 @@
   <property name="base_mass" value="83.1" />
   <property name="battery_mass" value="83.1" />  <!--to be checked out-->
- <property name="caster_mass" value="5.9" />
+  <property name="caster_mass" value="5.9" />
   <property name="tower_mass" value="6.49" />
   <!-- simplified box collision geometry for battery -->
@@ -47,5 +47,5 @@
   <!--                                                      -->
   <xacro:macro name="cob_wheel" params="suffix parent reflect">
-    <joint name="${parent}_${suffix}_wheel_joint" type="continuous">
+	<joint name="${parent}_${suffix}_wheel_joint" type="continuous">
       <axis xyz="0 1 0" />
       <limit effort="100" velocity="100"/> <!-- alpha tested effort and velocity limits -->
@@ -55,6 +55,6 @@
       <parent link="${parent}_rotation_link"/>
       <child link="${parent}_${suffix}_wheel_link"/>
-    </joint>
-    <link name="${parent}_${suffix}_wheel_link">
+	</joint>
+	<link name="${parent}_${suffix}_wheel_link">
       <inertial>
         <mass value="0.44036" />
@@ -63,17 +63,17 @@
                   iyy="0.015218160428" iyz="-0.000004273467" izz="0.011763977943" />
       </inertial>
-      <visual>
+	  <visual>
         <origin xyz="0 0 0" rpy="0 0 0" />
         <geometry>
           <!--cylinder radius="${wheel_radius}" length="${wheel_length}" /-->
-	  <mesh filename="package://raw_description/meshes/base/raw_wheel.stl"/>
-        </geometry>
-        <material name="IPA/LightGrey" />
-      </visual>
+		  <mesh filename="package://raw_description/meshes/base/raw_wheel.stl"/>
+        </geometry>
+        <material name="IPA/LightGrey" />
+	  </visual>
       <collision>
         <origin xyz="0 0 0" rpy="0 0 0" /> <!-- rotation because cyl. geom primitive has symmetry axis in +x direction -->
         <geometry>
           <sphere radius="${wheel_radius}"/>
-	  <!--mesh filename="package://raw_description/meshes/base/raw_wheel.stl"/-->
+		  <!--mesh filename="package://raw_description/meshes/base/raw_wheel.stl"/-->
         </geometry>
       </collision>
@@ -105,6 +105,6 @@
         <origin xyz="0 0 0" rpy="0 0 0" />
         <geometry>
-	  <mesh filename="package://raw_description/meshes/base/raw_caster.stl"/>
-		  <!--box size="0.001 0.001 0.001" /-->
+			<mesh filename="package://raw_description/meshes/base/raw_caster.stl"/>
+			<!--box size="0.001 0.001 0.001" /-->
         </geometry>
         <material name="IPA/LightGrey" />
@@ -121,6 +121,5 @@
   </xacro:macro>
   <xacro:macro name="cob_caster" params="suffix parent *origin ref_position">
-    <xacro:cob_caster_hub parent="${parent}" suffix="${suffix}_caster"
-                             ref_position="${ref_position}" >
+    <xacro:cob_caster_hub parent="${parent}" suffix="${suffix}_caster" ref_position="${ref_position}" >
       <insert_block name="origin" />
     </xacro:cob_caster_hub>
@@ -146,10 +145,10 @@
       </inertial>
       <visual>
-	  <origin xyz="0 0 0" rpy="0 0 0"/>
-	  <geometry>
+		<origin xyz="0 0 0" rpy="0 0 0"/>
+		<geometry>
             <mesh filename="package://raw_description/meshes/base/raw_battery.stl"/>
-          </geometry>
-        <material name="IPA/LightGrey" />
-       </visual>
+        </geometry>
+        <material name="IPA/LightGrey" />
+      </visual>
       <collision>
         <origin xyz="0 0.075 0" rpy="0 0 0"/> <!-- TODO: Change the origin of the stl, so that collision model doesn't need to be translated  -->
@@ -158,5 +157,5 @@
 	      <!--mesh filename="package://raw_description/meshes/base/raw_battery.stl"/-->
         </geometry>
-       </collision>
+      </collision>
     </link>
     <!-- extensions -->
@@ -205,10 +204,10 @@
        </visual>
        <collision>
-        <origin xyz="0 -0.03 -0.1" rpy="0 0 0"/>
-        <geometry>
-	   <!--mesh filename="package://raw_description/meshes/base/raw_tower_collision.stl"/-->
-	   <box size="0.32 0.58 0.24" />
-        </geometry>
-        </collision>
+         <origin xyz="0 -0.03 -0.1" rpy="0 0 0"/>
+         <geometry>
+			<!--mesh filename="package://raw_description/meshes/base/raw_tower_collision.stl"/-->
+			<box size="0.32 0.58 0.24" />
+         </geometry>
+       </collision>
     </link>
     <joint name="${name}_frame_joint" type="fixed">

Commit message: changed path to tower meshes

File: raw_description/urdf/base/base.urdf.xacro (robot description, xacro)
@@ -33,5 +33,5 @@
   <property name="base_mass" value="83.1" />
   <property name="battery_mass" value="83.1" />  <!--to be checked out-->
- <property name="caster_mass" value="5.9" />
+  <property name="caster_mass" value="5.9" />
   <property name="tower_mass" value="6.49" />
   <!-- simplified box collision geometry for battery -->
@@ -105,6 +105,6 @@
         <origin xyz="0 0 0" rpy="0 0 0" />
         <geometry>
-	  <mesh filename="package://raw_description/meshes/base/raw_caster.stl"/>
-		  <!--box size="0.001 0.001 0.001" /-->
+        <mesh filename="package://raw_description/meshes/base/raw_caster.stl"/>
+		    <!--box size="0.001 0.001 0.001" /-->
         </geometry>
         <material name="IPA/LightGrey" />
@@ -182,6 +182,6 @@
         <origin xyz="0 0 0.17" rpy="0 0 0" />
         <geometry>
-	   <!--mesh filename="package://raw_description/meshes/base/raw_base.stl"/-->
-	   <box size="1.04 0.58 0.31" />
+        <!--mesh filename="package://raw_description/meshes/base/raw_base.stl"/-->
+          <box size="1.04 0.58 0.31" />
         </geometry>
       </collision>
@@ -197,5 +197,5 @@
 	  <origin xyz="0 0 0" rpy="0 0 0"/>
 	  <geometry>
-            <mesh filename="package://raw_description/meshes/base/raw_tower.stl"/>
+            <mesh filename="package://raw_description/meshes/tower/raw_tower.stl"/>
           </geometry>
         <material name="IPA/LightGrey" />
@@ -204,6 +204,6 @@
         <origin xyz="0 -0.03 -0.1" rpy="0 0 0"/>
         <geometry>
-	   <!--mesh filename="package://raw_description/meshes/base/raw_tower_collision.stl"/-->
-	   <box size="0.32 0.58 0.24" />
+          <mesh filename="package://raw_description/meshes/tower/raw_tower_collision.stl"/>
+          <!--box size="0.32 0.58 0.24" /-->
         </geometry>
         </collision>
