Commit message: moved all hardcoded offsets to cob_calibration_data

File: desire_description/urdf/head_desire/head.urdf.xacro (robot description, xacro)
@@ -70,14 +70,13 @@
 		<!-- right camera -->
 		<xacro:cob_prosilica_v0 name="${name}_color_camera_r" ros_topic="stereo/right"  parent="${name}_tilt_link">
-			<!--origin xyz="${cam_r_x} ${cam_r_y} ${cam_r_z-0.06}" rpy="${cam_r_roll} ${cam_r_pitch+1.5708} ${cam_r_yaw+3.14159}"{cam_r_roll-3.14159} /-->
-<origin xyz="${cam_r_x} ${cam_r_y} ${cam_r_z-0.06}" rpy="${cam_r_roll} ${cam_r_pitch+1.5708} ${cam_r_yaw}" />
+			<origin xyz="${cam_r_x} ${cam_r_y} ${cam_r_z}" rpy="${cam_r_roll} ${cam_r_pitch} ${cam_r_yaw}" />
 		</xacro:cob_prosilica_v0>
 		<!-- left camera -->
 		<xacro:cob_prosilica_v0 name="${name}_color_camera_l" ros_topic="stereo/left" parent="${name}_color_camera_r_link">
-			<origin xyz="${cam_l_x-0.12} ${cam_l_y} ${cam_l_z}" rpy="${cam_l_roll} ${cam_l_pitch} ${cam_l_yaw}" />
+			<origin xyz="${cam_l_x} ${cam_l_y} ${cam_l_z}" rpy="${cam_l_roll} ${cam_l_pitch} ${cam_l_yaw}" />
 		</xacro:cob_prosilica_v0>
 		<!-- tof -->
 		<xacro:cob_tof_v0 name="${name}_tof" parent="${name}_color_camera_r_link">
-			<origin xyz="${tof_x-0.06} ${tof_y} ${tof_z}" rpy="${tof_roll} ${tof_pitch} ${tof_yaw}" />
+			<origin xyz="${tof_x} ${tof_y} ${tof_z}" rpy="${tof_roll} ${tof_pitch} ${tof_yaw}" />
 		</xacro:cob_tof_v0>
 		<!-- extensions -->
