Commit message: major adaptions in gazebo.urdf.xacros according to new gazebo format for controllers

File: cob_description/gazebo/gazebo.urdf.xacro (robot description, xacro)
@@ -4,4 +4,9 @@
        xmlns:interface="http://playerstage.sourceforge.net/gazebo/xmlschema/#interface">
   <gazebo>
+	<plugin name="gazebo_ros_controller_manager" filename="libgazebo_ros_controller_manager.so">
+      <alwaysOn>true</alwaysOn>
+      <updateRate>1000.0</updateRate>
+    </plugin>
+<!--
     <controller:gazebo_ros_controller_manager name="gazebo_ros_controller_manager" plugin="libgazebo_ros_controller_manager.so">
       <alwaysOn>true</alwaysOn>
@@ -9,4 +14,18 @@
       <interface:audio name="gazebo_ros_controller_manager_dummy_iface" />
     </controller:gazebo_ros_controller_manager>
+-->
+    <plugin name="gazebo_ros_power_monitor_controller" filename="libgazebo_ros_power_monitor.so">
+      <alwaysOn>true</alwaysOn>
+      <updateRate>1.0</updateRate>
+      <timeout>5</timeout>
+      <powerStateTopic>power_state</powerStateTopic>
+      <powerStateRate>10.0</powerStateRate>
+      <fullChargeCapacity>87.78</fullChargeCapacity>
+      <dischargeRate>-474</dischargeRate>
+      <chargeRate>525</chargeRate>
+      <dischargeVoltage>15.52</dischargeVoltage>
+      <chargeVoltage>16.41</chargeVoltage>
+    </plugin>
+<!--
     <controller:gazebo_ros_power_monitor name="gazebo_ros_power_monitor_controller" plugin="libgazebo_ros_power_monitor.so">
       <alwaysOn>true</alwaysOn>
@@ -22,4 +41,5 @@
       <chargeVoltage>16.41</chargeVoltage>
     </controller:gazebo_ros_power_monitor>
+-->
   </gazebo>
 </robot>

File: cob_description/urdf/base/base.gazebo.xacro (robot description, xacro)
@@ -21,4 +21,15 @@
     <gazebo reference="${name}_link">
       <selfCollide>true</selfCollide>
+      <sensor name='${name}_contact_sensor' type='contact'>
+	    <contact>
+	      <collision>${name}_link_geom</collision>
+	    </contact>
+	    <plugin name="${name}_gazebo_ros_bumper_controller" filename="libgazebo_ros_bumper.so">
+          <alwaysOn>true</alwaysOn>
+          <updateRate>100.0</updateRate>
+          <bumperTopicName>${name}_bumper</bumperTopicName>
+        </plugin>
+	  </sensor>
+<!--
       <sensor:contact name="${name}_contact_sensor">
         <geom>${name}_link_geom</geom>
@@ -31,7 +42,19 @@
         </controller:gazebo_ros_bumper>
       </sensor:contact>
+-->
       <material>IPA/LightGrey</material>
     </gazebo>
     <gazebo>
+		<plugin name="p3d_base_controller" filename="libgazebo_ros_p3d.so">
+			<alwaysOn>true</alwaysOn>
+			<updateRate>100.0</updateRate>
+			<bodyName>${name}_link</bodyName>
+			<topicName>${name}_pose_ground_truth</topicName>
+			<gaussianNoise>0.01</gaussianNoise>
+			<frameName>map</frameName>
+			<xyzOffsets>25.7 25.7 0</xyzOffsets>
+			<rpyOffsets>0 0 0</rpyOffsets>
+      </plugin>
+<!--
       <controller:gazebo_ros_p3d name="p3d_base_controller" plugin="libgazebo_ros_p3d.so">
         <alwaysOn>true</alwaysOn>
@@ -41,8 +64,9 @@
         <gaussianNoise>0.01</gaussianNoise>
         <frameName>map</frameName>
-        <xyzOffsets>25.7 25.7 0</xyzOffsets> <!-- initialize odometry for fake localization-->
+        <xyzOffsets>25.7 25.7 0</xyzOffsets>
         <rpyOffsets>0 0 0</rpyOffsets>
         <interface:position name="p3d_base_position"/>
       </controller:gazebo_ros_p3d>
+-->
       <canonicalBody>${name}_footprint</canonicalBody>
     </gazebo>

File: desire_description/urdf/base_desire/base.gazebo.xacro (robot description, xacro)
@@ -21,4 +21,15 @@
     <gazebo reference="${name}_link">
       <selfCollide>true</selfCollide>
+       <sensor name='${name}_contact_sensor' type='contact'>
+	    <contact>
+	      <collision>${name}_link_geom</collision>
+	    </contact>
+	    <plugin name="${name}_gazebo_ros_bumper_controller" filename="libgazebo_ros_bumper.so">
+          <alwaysOn>true</alwaysOn>
+          <updateRate>100.0</updateRate>
+          <bumperTopicName>${name}_bumper</bumperTopicName>
+        </plugin>
+	  </sensor>
+<!--
       <sensor:contact name="${name}_contact_sensor">
         <geom>${name}_link_geom</geom>
@@ -31,7 +42,19 @@
         </controller:gazebo_ros_bumper>
       </sensor:contact>
+-->
       <material>Gazebo/Grey</material>
     </gazebo>
     <gazebo>
+		<plugin name="p3d_base_controller" filename="libgazebo_ros_p3d.so">
+          <alwaysOn>true</alwaysOn>
+          <updateRate>100.0</updateRate>
+          <bodyName>${name}_link</bodyName>
+          <topicName>${name}_pose_ground_truth</topicName>
+          <gaussianNoise>0.01</gaussianNoise>
+          <frameName>map</frameName>
+          <xyzOffsets>25.7 25.7 0</xyzOffsets>
+          <rpyOffsets>0 0 0</rpyOffsets>
+       </plugin>
+<!--
       <controller:gazebo_ros_p3d name="p3d_base_controller" plugin="libgazebo_ros_p3d.so">
         <alwaysOn>true</alwaysOn>
@@ -41,8 +64,9 @@
         <gaussianNoise>0.01</gaussianNoise>
         <frameName>map</frameName>
-        <xyzOffsets>25.7 25.7 0</xyzOffsets> <!-- initialize odometry for fake localization-->
+        <xyzOffsets>25.7 25.7 0</xyzOffsets>
         <rpyOffsets>0 0 0</rpyOffsets>
         <interface:position name="p3d_base_position"/>
       </controller:gazebo_ros_p3d>
+-->
       <canonicalBody>${name}_footprint</canonicalBody>
     </gazebo>

File: raw_description/urdf/base/base.gazebo.xacro (robot description, xacro)
@@ -26,4 +26,15 @@
     <gazebo reference="${name}_link">
       <selfCollide>true</selfCollide>
+      <sensor name='${name}_contact_sensor' type='contact'>
+	    <contact>
+	      <collision>${name}_link_geom</collision>
+	    </contact>
+	    <plugin name="${name}_gazebo_ros_bumper_controller" filename="libgazebo_ros_bumper.so">
+          <alwaysOn>true</alwaysOn>
+          <updateRate>100.0</updateRate>
+          <bumperTopicName>${name}_bumper</bumperTopicName>
+        </plugin>
+	  </sensor>
+<!--
       <sensor:contact name="${name}_contact_sensor">
         <geom>${name}_link_geom</geom>
@@ -36,4 +47,5 @@
         </controller:gazebo_ros_bumper>
       </sensor:contact>
+-->
       <!--material>Gazebo/Grey</material-->
       <material value="IPA/LightGrey" />
@@ -41,9 +53,19 @@
     <gazebo reference="${name}_tower">		<!-- added for raw model - fxmlc -->
       <selfCollide>true</selfCollide>
-      <!--material>Gazebo/Grey</material-->
       <material value="IPA/LightGrey" />
     </gazebo>
     <gazebo>
-      <controller:gazebo_ros_p3d name="p3d_base_controller" plugin="libgazebo_ros_p3d.so">
+		<plugin name="p3d_base_controller" filename="libgazebo_ros_p3d.so">
+			<alwaysOn>true</alwaysOn>
+			<updateRate>100.0</updateRate>
+			<bodyName>${name}_link</bodyName>
+			<topicName>${name}_pose_ground_truth</topicName>
+			<gaussianNoise>0.01</gaussianNoise>
+			<frameName>map</frameName>
+			<xyzOffsets>25.7 25.7 0</xyzOffsets>
+			<rpyOffsets>0 0 0</rpyOffsets>
+      </plugin>
+<!--
+	<controller:gazebo_ros_p3d name="p3d_base_controller" plugin="libgazebo_ros_p3d.so">
         <alwaysOn>true</alwaysOn>
         <updateRate>100.0</updateRate>
@@ -52,8 +74,9 @@
         <gaussianNoise>0.01</gaussianNoise>
         <frameName>map</frameName>
-        <xyzOffsets>25.7 25.7 0</xyzOffsets> <!-- initialize odometry for fake localization-->
+        <xyzOffsets>25.7 25.7 0</xyzOffsets>
         <rpyOffsets>0 0 0</rpyOffsets>
         <interface:position name="p3d_base_position"/>
       </controller:gazebo_ros_p3d>
+-->
       <canonicalBody>${name}_footprint</canonicalBody>
     </gazebo>
