Commit message: clean up gazebo files

File: cob_description/gazebo/gazebo.urdf.xacro (robot description, xacro)
@@ -8,11 +8,4 @@
       <updateRate>1000.0</updateRate>
     </plugin>
-<!--
-    <controller:gazebo_ros_controller_manager name="gazebo_ros_controller_manager" plugin="libgazebo_ros_controller_manager.so">
-      <alwaysOn>true</alwaysOn>
-      <updateRate>1000.0</updateRate>
-      <interface:audio name="gazebo_ros_controller_manager_dummy_iface" />
-    </controller:gazebo_ros_controller_manager>
--->
     <plugin name="gazebo_ros_power_monitor_controller" filename="libgazebo_ros_power_monitor.so">
       <alwaysOn>true</alwaysOn>
@@ -27,19 +20,4 @@
       <chargeVoltage>16.41</chargeVoltage>
     </plugin>
-<!--
-    <controller:gazebo_ros_power_monitor name="gazebo_ros_power_monitor_controller" plugin="libgazebo_ros_power_monitor.so">
-      <alwaysOn>true</alwaysOn>
-      <updateRate>1.0</updateRate>
-      <timeout>5</timeout>
-      <interface:audio name="power_monitor_dummy_interface" />
-      <powerStateTopic>power_state</powerStateTopic>
-      <powerStateRate>10.0</powerStateRate>
-      <fullChargeCapacity>87.78</fullChargeCapacity>
-      <dischargeRate>-474</dischargeRate>
-      <chargeRate>525</chargeRate>
-      <dischargeVoltage>15.52</dischargeVoltage>
-      <chargeVoltage>16.41</chargeVoltage>
-    </controller:gazebo_ros_power_monitor>
--->
   </gazebo>
 </robot>

File: cob_description/urdf/base/base.gazebo.xacro (robot description, xacro)
@@ -19,30 +19,18 @@
   </xacro:macro>
   <xacro:macro name="cob_base_gazebo" params="name">
-    <gazebo reference="${name}_link">
-      <selfCollide>true</selfCollide>
-      <sensor name='${name}_contact_sensor' type='contact'>
-	    <contact>
-	      <collision>${name}_link_geom</collision>
-	    </contact>
-	    <plugin name="${name}_gazebo_ros_bumper_controller" filename="libgazebo_ros_bumper.so">
-          <alwaysOn>true</alwaysOn>
-          <updateRate>100.0</updateRate>
-          <bumperTopicName>${name}_bumper</bumperTopicName>
-        </plugin>
-	  </sensor>
-<!--
-      <sensor:contact name="${name}_contact_sensor">
-        <geom>${name}_link_geom</geom>
-        <updateRate>100.0</updateRate>
-        <controller:gazebo_ros_bumper name="${name}_gazebo_ros_bumper_controller" plugin="libgazebo_ros_bumper.so">
-          <alwaysOn>true</alwaysOn>
-          <updateRate>100.0</updateRate>
-          <bumperTopicName>${name}_bumper</bumperTopicName>
-          <interface:bumper name="${name}_bumper_iface" />
-        </controller:gazebo_ros_bumper>
-      </sensor:contact>
--->
-      <material>IPA/LightGrey</material>
-    </gazebo>
+	<gazebo reference="${name}_link">
+		<selfCollide>true</selfCollide>
+		<sensor name='${name}_contact_sensor' type='contact'>
+			<contact>
+				<collision>${name}_link_geom</collision>
+			</contact>
+			<plugin name="${name}_gazebo_ros_bumper_controller" filename="libgazebo_ros_bumper.so">
+				<alwaysOn>true</alwaysOn>
+				<updateRate>100.0</updateRate>
+				<bumperTopicName>${name}_bumper</bumperTopicName>
+			</plugin>
+		</sensor>
+		<material>IPA/LightGrey</material>
+	</gazebo>
     <gazebo>
 		<plugin name="p3d_base_controller" filename="libgazebo_ros_p3d.so">
@@ -53,21 +41,8 @@
 			<gaussianNoise>0.01</gaussianNoise>
 			<frameName>map</frameName>
-			<xyzOffsets>25.7 25.7 0</xyzOffsets>
+			<xyzOffsets>25.7 25.7 0</xyzOffsets> <!-- initialize odometry for fake localization-->
 			<rpyOffsets>0 0 0</rpyOffsets>
-      </plugin>
-<!--
-      <controller:gazebo_ros_p3d name="p3d_base_controller" plugin="libgazebo_ros_p3d.so">
-        <alwaysOn>true</alwaysOn>
-        <updateRate>100.0</updateRate>
-        <bodyName>${name}_link</bodyName>
-        <topicName>${name}_pose_ground_truth</topicName>
-        <gaussianNoise>0.01</gaussianNoise>
-        <frameName>map</frameName>
-        <xyzOffsets>25.7 25.7 0</xyzOffsets>
-        <rpyOffsets>0 0 0</rpyOffsets>
-        <interface:position name="p3d_base_position"/>
-      </controller:gazebo_ros_p3d>
--->
-      <canonicalBody>${name}_footprint</canonicalBody>
+		</plugin>
+		<canonicalBody>${name}_footprint</canonicalBody>
     </gazebo>
   </xacro:macro>

File: cob_description/urdf/sensors/hokuyo_SR400_laser.gazebo.xacro (robot description, xacro)
@@ -34,27 +34,4 @@
 		</plugin>
       </sensor>
-<!--
-      <sensor:ray name="${name}">
-        <rayCount>150</rayCount>
-        <rangeCount>150</rangeCount>
-        <laserCount>1</laserCount>
-        <origin>0.0 0.0 0.0</origin>
-        <displayRays>false</displayRays>
-        <minAngle>${min_angle*180.0/M_PI}</minAngle>
-        <maxAngle>${max_angle*180.0/M_PI}</maxAngle>
-        <minRange>0.30</minRange>
-        <maxRange>5.0</maxRange>
-        <resRange>0.01</resRange>
-        <updateRate>${update_rate}</updateRate>
-        <controller:gazebo_ros_laser name="gazebo_ros_${name}_controller" plugin="libgazebo_ros_laser.so">
-          <gaussianNoise>0.005</gaussianNoise>
-          <alwaysOn>true</alwaysOn>
-          <updateRate>${update_rate}</updateRate>
-          <topicName>${ros_topic}</topicName>
-          <frameName>${name}_link</frameName>
-          <interface:laser name="gazebo_ros_${name}_iface" />
-        </controller:gazebo_ros_laser>
-      </sensor:ray>
--->
       <material>IPA/LightGrey</material>
     </gazebo>

File: cob_description/urdf/sensors/hokuyo_lx30_laser.gazebo.xacro (robot description, xacro)
@@ -34,27 +34,4 @@
 		</plugin>
       </sensor>
-<!--
-      <sensor:ray name="${name}">
-        <rayCount>640</rayCount>
-        <rangeCount>640</rangeCount>
-        <laserCount>1</laserCount>
-        <origin>0.0 0.0 0.0</origin>
-        <displayRays>false</displayRays>
-        <minAngle>${min_angle*180.0/M_PI}</minAngle>
-        <maxAngle>${max_angle*180.0/M_PI}</maxAngle>
-        <minRange>0.05</minRange>
-        <maxRange>10.0</maxRange>
-        <resRange>0.01</resRange>
-        <updateRate>${update_rate}</updateRate>
-        <controller:gazebo_ros_laser name="gazebo_ros_${name}_controller" plugin="libgazebo_ros_laser.so">
-          <gaussianNoise>0.005</gaussianNoise>
-          <alwaysOn>true</alwaysOn>
-          <updateRate>${update_rate}</updateRate>
-          <topicName>${ros_topic}</topicName>
-          <frameName>/${name}_link</frameName>
-          <interface:laser name="gazebo_ros_${name}_iface" />
-        </controller:gazebo_ros_laser>
-      </sensor:ray>
--->
       <material>IPA/LightGrey</material>
     </gazebo>

File: cob_description/urdf/sensors/kinect.gazebo.xacro (robot description, xacro)
@@ -7,115 +7,64 @@
   <gazebo reference="${name}_frame">
 	<sensor type="depth" name="${name}_frame_sensor">
-      <always_on>true</always_on>
-      <update_rate>20.0</update_rate>
-      <camera>
-        <horizontal_fov>${57.0*M_PI/180.0}</horizontal_fov>
-        <image>
-          <format>R8G8B8</format>
-          <width>640</width>
-          <height>480</height>
-        </image>
-        <clip>
-          <near>0.1</near>
-          <far>100</far>
-        </clip>
-      </camera>
-      <plugin name="${name}_depth_frame_controller" filename="libgazebo_ros_openni_kinect.so">
-        <alwaysOn>true</alwaysOn>
-        <updateRate>20.0</updateRate>
-        <imageTopicName>${ros_topic}/ir/image_raw</imageTopicName>
-        <cameraInfoTopicName>${ros_topic}/ir/camera_info</cameraInfoTopicName>
-        <depthImageTopicName>${ros_topic}/depth/image_raw</depthImageTopicName>
-        <depthImageInfoTopicName>${ros_topic}/depth/camera_info</depthImageInfoTopicName>
-        <pointCloudTopicName>${ros_topic}/depth/points</pointCloudTopicName>
-        <frameName>${name}_link</frameName>
-        <pointCloudCutoff>0.5</pointCloudCutoff>
-        <distortionK1>0.00000001</distortionK1>
-        <distortionK2>0.00000001</distortionK2>
-        <distortionK3>0.00000001</distortionK3>
-        <distortionT1>0.00000001</distortionT1>
-        <distortionT2>0.00000001</distortionT2>
-      </plugin>
-    </sensor>
-<!--
-    <sensor:camera name="${name}_frame_sensor">
-      <imageFormat>R8G8B8</imageFormat>
-      <imageSize>640 480</imageSize>
-      <hfov>57</hfov>
-      <nearClip>0.1</nearClip>
-      <farClip>100</farClip>
-      <updateRate>20.0</updateRate>
-      <baseline>0.2</baseline>
-      <controller:gazebo_ros_openni_kinect name="${name}_depth_frame_controller" plugin="libgazebo_ros_openni_kinect.so">
-        <alwaysOn>true</alwaysOn>
-        <updateRate>20.0</updateRate>
-        <imageTopicName>${ros_topic}/ir/image_raw</imageTopicName>
-        <cameraInfoTopicName>${ros_topic}/ir/camera_info</cameraInfoTopicName>
-        <depthImageTopicName>${ros_topic}/depth/image_raw</depthImageTopicName>
-        <depthImageInfoTopicName>${ros_topic}/depth/camera_info</depthImageInfoTopicName>
-        <pointCloudTopicName>${ros_topic}/depth/points</pointCloudTopicName>
-        <frameName>${name}_link</frameName>
-        <pointCloudCutoff>0.5</pointCloudCutoff>
-        <distortionK1>0.00000001</distortionK1>
-        <distortionK2>0.00000001</distortionK2>
-        <distortionK3>0.00000001</distortionK3>
-        <distortionT1>0.00000001</distortionT1>
-        <distortionT2>0.00000001</distortionT2>
-      </controller:gazebo_ros_openni_kinect>
-    </sensor:camera>
--->
-   <sensor type="depth" name="${name}_frame_sensor">
-      <always_on>true</always_on>
-      <update_rate>20.0</update_rate>
-      <camera>
-        <horizontal_fov>${57.0*M_PI/180.0}</horizontal_fov>
-        <image>
-          <format>R8G8B8</format>
-          <width>640</width>
-          <height>480</height>
-        </image>
-        <clip>
-          <near>0.1</near>
-          <far>100</far>
-        </clip>
-      </camera>
-      <plugin name="${name}_rgb_frame_controller" filename="libgazebo_ros_openni_kinect.so">
-        <alwaysOn>true</alwaysOn>
-        <updateRate>20.0</updateRate>
-        <imageTopicName>${ros_topic}/rgb/image_raw</imageTopicName>
-        <cameraInfoTopicName>${ros_topic}/rgb/camera_info</cameraInfoTopicName>
-        <frameName>${name}_link</frameName>
-        <pointCloudCutoff>0.5</pointCloudCutoff>
-        <distortionK1>0.00000001</distortionK1>
-        <distortionK2>0.00000001</distortionK2>
-        <distortionK3>0.00000001</distortionK3>
-        <distortionT1>0.00000001</distortionT1>
-        <distortionT2>0.00000001</distortionT2>
-      </plugin>
-    </sensor>
-<!--
-    <sensor:camera name="${name}_frame_sensor">
-      <imageFormat>R8G8B8</imageFormat>
-      <imageSize>640 480</imageSize>
-      <hfov>57</hfov>
-      <nearClip>0.1</nearClip>
-      <farClip>100</farClip>
-      <updateRate>20.0</updateRate>
-      <baseline>0.2</baseline>
-      <controller:gazebo_ros_openni_kinect name="${name}_rgb_frame_controller" plugin="libgazebo_ros_openni_kinect.so">
-        <alwaysOn>true</alwaysOn>
-        <updateRate>20.0</updateRate>
-        <imageTopicName>${ros_topic}/rgb/image_raw</imageTopicName>
-        <cameraInfoTopicName>${ros_topic}/rgb/camera_info</cameraInfoTopicName>
-        <frameName>${name}_link</frameName>
-        <pointCloudCutoff>0.5</pointCloudCutoff>
-        <distortionK1>0.00000001</distortionK1>
-        <distortionK2>0.00000001</distortionK2>
-        <distortionK3>0.00000001</distortionK3>
-        <distortionT1>0.00000001</distortionT1>
-        <distortionT2>0.00000001</distortionT2>
-      </controller:gazebo_ros_openni_kinect>
-    </sensor:camera>
--->
+		<always_on>true</always_on>
+		<update_rate>20.0</update_rate>
+		<camera>
+			<horizontal_fov>${57.0*M_PI/180.0}</horizontal_fov>
+			<image>
+				<format>R8G8B8</format>
+				<width>640</width>
+				<height>480</height>
+			</image>
+			<clip>
+				<near>0.1</near>
+				<far>100</far>
+			</clip>
+		</camera>
+		<plugin name="${name}_depth_frame_controller" filename="libgazebo_ros_openni_kinect.so">
+			<alwaysOn>true</alwaysOn>
+			<updateRate>20.0</updateRate>
+			<imageTopicName>${ros_topic}/ir/image_raw</imageTopicName>
+			<cameraInfoTopicName>${ros_topic}/ir/camera_info</cameraInfoTopicName>
+			<depthImageTopicName>${ros_topic}/depth/image_raw</depthImageTopicName>
+			<depthImageInfoTopicName>${ros_topic}/depth/camera_info</depthImageInfoTopicName>
+			<pointCloudTopicName>${ros_topic}/depth/points</pointCloudTopicName>
+			<frameName>${name}_link</frameName>
+			<pointCloudCutoff>0.5</pointCloudCutoff>
+			<distortionK1>0.00000001</distortionK1>
+			<distortionK2>0.00000001</distortionK2>
+			<distortionK3>0.00000001</distortionK3>
+			<distortionT1>0.00000001</distortionT1>
+			<distortionT2>0.00000001</distortionT2>
+		</plugin>
+	</sensor>
+	<sensor type="depth" name="${name}_frame_sensor">
+		<always_on>true</always_on>
+		<update_rate>20.0</update_rate>
+		<camera>
+			<horizontal_fov>${57.0*M_PI/180.0}</horizontal_fov>
+			<image>
+				<format>R8G8B8</format>
+				<width>640</width>
+				<height>480</height>
+			</image>
+			<clip>
+				<near>0.1</near>
+				<far>100</far>
+			</clip>
+		</camera>
+		<plugin name="${name}_rgb_frame_controller" filename="libgazebo_ros_openni_kinect.so">
+			<alwaysOn>true</alwaysOn>
+			<updateRate>20.0</updateRate>
+			<imageTopicName>${ros_topic}/rgb/image_raw</imageTopicName>
+			<cameraInfoTopicName>${ros_topic}/rgb/camera_info</cameraInfoTopicName>
+			<frameName>${name}_link</frameName>
+			<pointCloudCutoff>0.5</pointCloudCutoff>
+			<distortionK1>0.00000001</distortionK1>
+			<distortionK2>0.00000001</distortionK2>
+			<distortionK3>0.00000001</distortionK3>
+			<distortionT1>0.00000001</distortionT1>
+			<distortionT2>0.00000001</distortionT2>
+		</plugin>
+	</sensor>
     <material>IPA/LightGrey</material>
   </gazebo>

File: cob_description/urdf/sensors/phidgets_distance.gazebo.xacro (robot description, xacro)
@@ -5,58 +5,35 @@
        xmlns:xacro="http://ros.org/wiki/xacro">
   <xacro:macro name="phidgets_distance_gazebo_v0" params="name ros_topic update_rate">
-    <gazebo reference="${name}_link">
-	  <sensor name="${name}" type="ray">
-		<always_on>true</always_on>
-		<update_rate>${update_rate}</update_rate>
-		<pose>0 0 0 0 0 0</pose>
-		<visualize>false</visualize>
-		<ray>
-			<scan>
-				<horizontal>
-					<samples>10</samples>
-					<resolution>1.0</resolution>
-					<min_angle>-0.2</min_angle>
-					<max_angle>0.2</max_angle>
-				</horizontal>
-			</scan>
-			<range>
-				<min>0.01</min>
-				<max>0.4</max>
-				<resolution>0.005</resolution>
-			</range>
-		</ray>
-		<plugin name="gazebo_ros_${name}_controller" filename="libgazebo_ros_laser.so">
-          <gaussianNoise>0.005</gaussianNoise>
-          <alwaysOn>true</alwaysOn>
-          <updateRate>${update_rate}</updateRate>
-          <topicName>${ros_topic}</topicName>
-          <frameName>/${name}_link</frameName>
-		</plugin>
-      </sensor>
-<!--
-      <sensor:ray name="${name}">
-        <rayCount>10</rayCount>
-        <rangeCount>10</rangeCount>
-        <laserCount>1</laserCount>
-        <origin>0.0 0.0 0.0</origin>
-        <displayRays>false</displayRays>
-        <minAngle>${-0.2*180.0/M_PI}</minAngle>
-        <maxAngle>${0.2*180.0/M_PI}</maxAngle>
-        <minRange>0.01</minRange>
-        <maxRange>0.4</maxRange>
-        <resRange>0.005</resRange>
-        <updateRate>${update_rate}</updateRate>
-        <controller:gazebo_ros_laser name="gazebo_ros_${name}_controller" plugin="libgazebo_ros_laser.so">
-          <gaussianNoise>0.005</gaussianNoise>
-          <alwaysOn>true</alwaysOn>
-          <updateRate>${update_rate}</updateRate>
-          <topicName>${ros_topic}</topicName>
-          <frameName>/${name}_link</frameName>
-          <interface:laser name="gazebo_ros_${name}_iface" />
-        </controller:gazebo_ros_laser>
-      </sensor:ray>
--->
-      <material>IPA/LightGrey</material>
-    </gazebo>
+	<gazebo reference="${name}_link">
+		<sensor name="${name}" type="ray">
+			<always_on>true</always_on>
+			<update_rate>${update_rate}</update_rate>
+			<pose>0 0 0 0 0 0</pose>
+			<visualize>false</visualize>
+			<ray>
+				<scan>
+					<horizontal>
+						<samples>10</samples>
+						<resolution>1.0</resolution>
+						<min_angle>-0.2</min_angle>
+						<max_angle>0.2</max_angle>
+					</horizontal>
+				</scan>
+				<range>
+					<min>0.01</min>		<!-- real value from sensor datasheet is 0.04m -->
+					<max>0.4</max>		<!-- real value from sensor datasheet is 0.30m -->
+					<resolution>0.005</resolution>
+				</range>
+			</ray>
+			<plugin name="gazebo_ros_${name}_controller" filename="libgazebo_ros_laser.so">
+				<gaussianNoise>0.005</gaussianNoise>
+				<alwaysOn>true</alwaysOn>
+				<updateRate>${update_rate}</updateRate>
+				<topicName>${ros_topic}</topicName>
+				<frameName>/${name}_link</frameName>
+			</plugin>
+		</sensor>
+		<material>IPA/LightGrey</material>
+	</gazebo>
   </xacro:macro>
 </robot>

File: cob_description/urdf/sensors/prosilica.gazebo.xacro (robot description, xacro)
@@ -7,19 +7,19 @@
 		<gazebo reference="${name}_frame">
 			<sensor type="depth" name="${name}_sensor">
-			  <always_on>true</always_on>
-			  <update_rate>10.0</update_rate>
-			  <camera>
-				<horizontal_fov>0.58</horizontal_fov>
-				<image>
-				  <format>R8G8B8</format>
-				  <width>1360</width>
-				  <height>1024</height>
-				</image>
-				<clip>
-				  <near>0.1</near>
-				  <far>100</far>
-				</clip>
-			  </camera>
-			  <plugin name="${name}_controller" filename="libgazebo_ros_prosilica.so">
+				<always_on>true</always_on>
+				<update_rate>10.0</update_rate>
+				<camera>
+					<horizontal_fov>0.58</horizontal_fov>	<!--opening angle of Fujinon HF9HA-1B-->
+					<image>
+						<format>R8G8B8</format>
+						<width>1360</width>
+						<height>1024</height>
+					</image>
+					<clip>
+						<near>0.1</near>
+						<far>100</far>
+					</clip>
+				</camera>
+				<plugin name="${name}_controller" filename="libgazebo_ros_prosilica.so">
 					<alwaysOn>true</alwaysOn>
 					<updateRate>10.0</updateRate>
@@ -32,5 +32,5 @@
 					<Cx>697.69</Cx>
 					<Cy>530.51</Cy>
-					<focal_length>1450</focal_length>
+					<focal_length>1450</focal_length>	<!-- image_width / (2*tan(hfov_radian /2)) -->
 					<distortion_k1>0.00000001</distortion_k1>
 					<distortion_k2>0.00000001</distortion_k2>
@@ -38,35 +38,6 @@
 					<distortion_t1>0.00000001</distortion_t1>
 					<distortion_t2>0.00000001</distortion_t2>
-			  </plugin>
+				</plugin>
 			</sensor>
-<!--
-			<sensor:camera name="${name}_sensor">
-				<imageFormat>R8G8B8</imageFormat>
-				<imageSize>1360 1024</imageSize>
-				<hfov>33</hfov>
-				<nearClip>0.1</nearClip>
-				<farClip>100</farClip>
-				<updateRate>10.0</updateRate>
-				<controller:gazebo_ros_prosilica name="${name}_controller" plugin="libgazebo_ros_prosilica.so">
-					<alwaysOn>true</alwaysOn>
-					<updateRate>10.0</updateRate>
-					<topicName>${ros_topic}_image_data</topicName>
-					<imageTopicName>/${ros_topic}/image_raw</imageTopicName>
-					<cameraInfoTopicName>/${ros_topic}/camera_info</cameraInfoTopicName>
-					<pollServiceName>/${name}/request_image</pollServiceName>
-					<frameName>/${name}_link</frameName>
-					<CxPrime>697.69</CxPrime>
-					<Cx>697.69</Cx>
-					<Cy>530.51</Cy>
-					<focal_length>1450</focal_length>
-					<distortion_k1>0.00000001</distortion_k1>
-					<distortion_k2>0.00000001</distortion_k2>
-					<distortion_k3>0.00000001</distortion_k3>
-					<distortion_t1>0.00000001</distortion_t1>
-					<distortion_t2>0.00000001</distortion_t2>
-					<interface:camera name="${name}_iface" />
-				</controller:gazebo_ros_prosilica>
-			</sensor:camera>
--->
 			<material value="IPA/LightGrey" />
 			<turnGravityOff>true</turnGravityOff>

File: cob_description/urdf/sensors/sick_s300_laser.gazebo.xacro (robot description, xacro)
@@ -5,58 +5,35 @@
        xmlns:xacro="http://ros.org/wiki/xacro">
   <xacro:macro name="sick_s300_laser_gazebo_v0" params="name ros_topic update_rate min_angle max_angle">
-    <gazebo reference="${name}_link">
-      <sensor name="${name}" type="ray">
-		<always_on>true</always_on>
-		<update_rate>${update_rate}</update_rate>
-		<pose>0 0 0 0 0 0</pose>
-		<visualize>false</visualize>
-		<ray>
-			<scan>
-				<horizontal>
-					<samples>541</samples>
-					<resolution>1.0</resolution>
-					<min_angle>${min_angle}</min_angle>
-					<max_angle>${max_angle}</max_angle>
-				</horizontal>
-			</scan>
-			<range>
-				<min>0.05</min>
-				<max>30.0</max>
-				<resolution>0.03</resolution>
-			</range>
-		</ray>
-		<plugin name="gazebo_ros_${name}_controller" filename="libgazebo_ros_laser.so">
-			<gaussianNoise>0.005</gaussianNoise>
-			<alwaysOn>true</alwaysOn>
-			<updateRate>${update_rate}</updateRate>
-			<topicName>${ros_topic}</topicName>
-			<frameName>${name}_link</frameName>
-		</plugin>
-      </sensor>
-<!--
-      <sensor:ray name="${name}">
-        <rayCount>541</rayCount>
-        <rangeCount>541</rangeCount>
-        <laserCount>1</laserCount>
-        <origin>0.0 0.0 0.0</origin>
-        <displayRays>false</displayRays>
-        <minAngle>${min_angle*180.0/M_PI}</minAngle>
-        <maxAngle>${max_angle*180.0/M_PI}</maxAngle>
-        <minRange>0.05</minRange>
-        <maxRange>30.0</maxRange>
-        <resRange>0.03</resRange>
-        <updateRate>${update_rate}</updateRate>
-        <controller:gazebo_ros_laser name="gazebo_ros_${name}_controller" plugin="libgazebo_ros_laser.so">
-          <gaussianNoise>0.005</gaussianNoise>
-          <alwaysOn>true</alwaysOn>
-          <updateRate>${update_rate}</updateRate>
-          <topicName>${ros_topic}</topicName>
-          <frameName>/${name}_link</frameName>
-          <interface:laser name="gazebo_ros_${name}_iface" />
-        </controller:gazebo_ros_laser>
-      </sensor:ray>
--->
-      <material value="IPA/LightGrey" />
-    </gazebo>
+	<gazebo reference="${name}_link">
+		<sensor name="${name}" type="ray">
+			<always_on>true</always_on>
+			<update_rate>${update_rate}</update_rate>
+			<pose>0 0 0 0 0 0</pose>
+			<visualize>false</visualize>
+			<ray>
+				<scan>
+					<horizontal>
+						<samples>541</samples>
+						<resolution>1.0</resolution>
+						<min_angle>${min_angle}</min_angle>
+						<max_angle>${max_angle}</max_angle>
+					</horizontal>
+				</scan>
+				<range>
+					<min>0.05</min>
+					<max>30.0</max>
+					<resolution>0.03</resolution>
+				</range>
+			</ray>
+			<plugin name="gazebo_ros_${name}_controller" filename="libgazebo_ros_laser.so">
+				<gaussianNoise>0.005</gaussianNoise>
+				<alwaysOn>true</alwaysOn>
+				<updateRate>${update_rate}</updateRate>
+				<topicName>${ros_topic}</topicName>
+				<frameName>${name}_link</frameName>
+			</plugin>
+		</sensor>
+		<material value="IPA/LightGrey" />
+	</gazebo>
   </xacro:macro>
 </robot>
