Commit message: clean up gazebo files

File: cob_description/urdf/sensors/tof.gazebo.xacro (robot description, xacro)
@@ -7,7 +7,7 @@
 <xacro:macro name="cob_tof_gazebo_v0" params="name ros_topic">
   <gazebo reference="${name}_frame">
-	  <sensor name="${name}_sensor" type="ray">
+	<sensor name="${name}_sensor" type="ray">
 		<always_on>true</always_on>
-		<update_rate>10</update_rate>
+		<update_rate>10</update_rate>	<!--max50Hz-->
 		<pose>0 0 0.05 0 0 0</pose>
 		<visualize>false</visualize>
@@ -15,5 +15,5 @@
 			<scan>
 				<horizontal>
-					<samples>176</samples>
+					<samples>176</samples>		<!--true value 176-->
 					<resolution>1.0</resolution>
 					<min_angle>-0.38</min_angle>
@@ -21,5 +21,5 @@
 				</horizontal>
 				<vertical>
-					<samples>144</samples>
+					<samples>144</samples>		<!--true value 144 -->
 					<resolution>1.0</resolution>
 					<min_angle>-0.3</min_angle>
@@ -28,44 +28,17 @@
 			</scan>
 			<range>
-				<min>0.80</min>
-				<max>5.0</max>
+				<min>0.80</min>		<!--0.8m min calibrated range-->
+				<max>5.0</max>		<!--5.0m max calibrated range-->
 				<resolution>0.010</resolution>
 			</range>
 		</ray>
 		<plugin name="tof_controller" filename="libgazebo_ros_block_laser.so">
-            <gaussianNoise>0.005</gaussianNoise>
-            <alwaysOn>true</alwaysOn>
-            <updateRate>30</updateRate>
-            <topicName>${ros_topic}</topicName>
-            <frameName>/${name}_frame</frameName>
+			<gaussianNoise>0.005</gaussianNoise>
+			<alwaysOn>true</alwaysOn>
+			<updateRate>30</updateRate> 	<!--max 50Hz, cob3 30Hz -->
+			<topicName>${ros_topic}</topicName>
+			<frameName>/${name}_frame</frameName>
 		</plugin>
-      </sensor>
-<!--
-    <sensor:ray name="${name}_sensor">
-          <rayCount>176</rayCount>
-          <rangeCount>176</rangeCount>
-          <laserCount>1</laserCount>
-          <origin>0.0 0.0 0.05</origin>
-          <displayRays>false</displayRays>
-          <minAngle>-21.8</minAngle>
-          <maxAngle>21.8</maxAngle>
-          <minRange>0.80</minRange>
-          <maxRange>5.0</maxRange>
-          <resRange>0.010</resRange>
-          <updateRate>10</updateRate>
-          <verticalRayCount>144</verticalRayCount>
-          <verticalRangeCount>144</verticalRangeCount>
-          <verticalMinAngle>-17.3</verticalMinAngle>
-          <verticalMaxAngle>17.3</verticalMaxAngle>
-          <controller:gazebo_ros_block_laser name="tof_controller" plugin="libgazebo_ros_block_laser.so">
-            <gaussianNoise>0.005</gaussianNoise>
-            <alwaysOn>true</alwaysOn>
-            <updateRate>30</updateRate>
-            <topicName>${ros_topic}</topicName>
-            <frameName>/${name}_frame</frameName>
-            <interface:laser name="${name}_ray_block_iface" />
-          </controller:gazebo_ros_block_laser>
-        </sensor:ray>
--->
+	</sensor>
     <material value="IPA/LightGrey" />
     <turnGravityOff>true</turnGravityOff>

File: desire_description/urdf/base_desire/base.gazebo.xacro (robot description, xacro)
@@ -19,56 +19,31 @@
   </xacro:macro>
   <xacro:macro name="desire_base_gazebo_v0" params="name">
-    <gazebo reference="${name}_link">
-      <selfCollide>true</selfCollide>
-       <sensor name='${name}_contact_sensor' type='contact'>
-	    <contact>
-	      <collision>${name}_link_geom</collision>
-	    </contact>
-	    <plugin name="${name}_gazebo_ros_bumper_controller" filename="libgazebo_ros_bumper.so">
-          <alwaysOn>true</alwaysOn>
-          <updateRate>100.0</updateRate>
-          <bumperTopicName>${name}_bumper</bumperTopicName>
-        </plugin>
-	  </sensor>
-<!--
-      <sensor:contact name="${name}_contact_sensor">
-        <geom>${name}_link_geom</geom>
-        <updateRate>100.0</updateRate>
-        <controller:gazebo_ros_bumper name="${name}_gazebo_ros_bumper_controller" plugin="libgazebo_ros_bumper.so">
-          <alwaysOn>true</alwaysOn>
-          <updateRate>100.0</updateRate>
-          <bumperTopicName>${name}_bumper</bumperTopicName>
-          <interface:bumper name="${name}_bumper_iface" />
-        </controller:gazebo_ros_bumper>
-      </sensor:contact>
--->
-      <material>Gazebo/Grey</material>
-    </gazebo>
+	<gazebo reference="${name}_link">
+		<selfCollide>true</selfCollide>
+		<sensor name='${name}_contact_sensor' type='contact'>
+			<contact>
+			<collision>${name}_link_geom</collision>
+			</contact>
+			<plugin name="${name}_gazebo_ros_bumper_controller" filename="libgazebo_ros_bumper.so">
+				<alwaysOn>true</alwaysOn>
+				<updateRate>100.0</updateRate>
+				<bumperTopicName>${name}_bumper</bumperTopicName>
+			</plugin>
+		</sensor>
+		<material>Gazebo/Grey</material>
+	</gazebo>
     <gazebo>
 		<plugin name="p3d_base_controller" filename="libgazebo_ros_p3d.so">
-          <alwaysOn>true</alwaysOn>
-          <updateRate>100.0</updateRate>
-          <bodyName>${name}_link</bodyName>
-          <topicName>${name}_pose_ground_truth</topicName>
-          <gaussianNoise>0.01</gaussianNoise>
-          <frameName>map</frameName>
-          <xyzOffsets>25.7 25.7 0</xyzOffsets>
-          <rpyOffsets>0 0 0</rpyOffsets>
-       </plugin>
-<!--
-      <controller:gazebo_ros_p3d name="p3d_base_controller" plugin="libgazebo_ros_p3d.so">
-        <alwaysOn>true</alwaysOn>
-        <updateRate>100.0</updateRate>
-        <bodyName>${name}_link</bodyName>
-        <topicName>${name}_pose_ground_truth</topicName>
-        <gaussianNoise>0.01</gaussianNoise>
-        <frameName>map</frameName>
-        <xyzOffsets>25.7 25.7 0</xyzOffsets>
-        <rpyOffsets>0 0 0</rpyOffsets>
-        <interface:position name="p3d_base_position"/>
-      </controller:gazebo_ros_p3d>
--->
-      <canonicalBody>${name}_footprint</canonicalBody>
-    </gazebo>
+			<alwaysOn>true</alwaysOn>
+			<updateRate>100.0</updateRate>
+			<bodyName>${name}_link</bodyName>
+			<topicName>${name}_pose_ground_truth</topicName>
+			<gaussianNoise>0.01</gaussianNoise>
+			<frameName>map</frameName>
+			<xyzOffsets>25.7 25.7 0</xyzOffsets>	<!-- initialize odometry for fake localization-->
+			<rpyOffsets>0 0 0</rpyOffsets>
+		</plugin>
+		<canonicalBody>${name}_footprint</canonicalBody>
+	</gazebo>
   </xacro:macro>
 </robot>

File: raw_description/urdf/base/base.gazebo.xacro (robot description, xacro)
@@ -24,35 +24,23 @@
   </xacro:macro>
   <xacro:macro name="cob_base_gazebo" params="name">
-    <gazebo reference="${name}_link">
-      <selfCollide>true</selfCollide>
-      <sensor name='${name}_contact_sensor' type='contact'>
-	    <contact>
-	      <collision>${name}_link_geom</collision>
-	    </contact>
-	    <plugin name="${name}_gazebo_ros_bumper_controller" filename="libgazebo_ros_bumper.so">
-          <alwaysOn>true</alwaysOn>
-          <updateRate>100.0</updateRate>
-          <bumperTopicName>${name}_bumper</bumperTopicName>
-        </plugin>
-	  </sensor>
-<!--
-      <sensor:contact name="${name}_contact_sensor">
-        <geom>${name}_link_geom</geom>
-        <updateRate>100.0</updateRate>
-        <controller:gazebo_ros_bumper name="${name}_gazebo_ros_bumper_controller" plugin="libgazebo_ros_bumper.so">
-          <alwaysOn>true</alwaysOn>
-          <updateRate>100.0</updateRate>
-          <bumperTopicName>${name}_bumper</bumperTopicName>
-          <interface:bumper name="${name}_bumper_iface" />
-        </controller:gazebo_ros_bumper>
-      </sensor:contact>
--->
-      <!--material>Gazebo/Grey</material-->
-      <material value="IPA/LightGrey" />
-    </gazebo>
+	<gazebo reference="${name}_link">
+		<selfCollide>true</selfCollide>
+		<sensor name='${name}_contact_sensor' type='contact'>
+			<contact>
+				<collision>${name}_link_geom</collision>
+			</contact>
+			<plugin name="${name}_gazebo_ros_bumper_controller" filename="libgazebo_ros_bumper.so">
+				<alwaysOn>true</alwaysOn>
+				<updateRate>100.0</updateRate>
+				<bumperTopicName>${name}_bumper</bumperTopicName>
+			</plugin>
+		</sensor>
+		<!--material>Gazebo/Grey</material-->
+		<material value="IPA/LightGrey" />
+	</gazebo>
     <gazebo reference="${name}_tower">		<!-- added for raw model - fxmlc -->
-      <selfCollide>true</selfCollide>
-      <material value="IPA/LightGrey" />
-    </gazebo>
+		<selfCollide>true</selfCollide>
+		<material value="IPA/LightGrey" />
+	</gazebo>
     <gazebo>
 		<plugin name="p3d_base_controller" filename="libgazebo_ros_p3d.so">
@@ -63,22 +51,9 @@
 			<gaussianNoise>0.01</gaussianNoise>
 			<frameName>map</frameName>
-			<xyzOffsets>25.7 25.7 0</xyzOffsets>
+			<xyzOffsets>25.7 25.7 0</xyzOffsets>	<!-- initialize odometry for fake localization-->
 			<rpyOffsets>0 0 0</rpyOffsets>
-      </plugin>
-<!--
-	<controller:gazebo_ros_p3d name="p3d_base_controller" plugin="libgazebo_ros_p3d.so">
-        <alwaysOn>true</alwaysOn>
-        <updateRate>100.0</updateRate>
-        <bodyName>${name}_link</bodyName>
-        <topicName>${name}_pose_ground_truth</topicName>
-        <gaussianNoise>0.01</gaussianNoise>
-        <frameName>map</frameName>
-        <xyzOffsets>25.7 25.7 0</xyzOffsets>
-        <rpyOffsets>0 0 0</rpyOffsets>
-        <interface:position name="p3d_base_position"/>
-      </controller:gazebo_ros_p3d>
--->
-      <canonicalBody>${name}_footprint</canonicalBody>
-    </gazebo>
+		</plugin>
+		<canonicalBody>${name}_footprint</canonicalBody>
+	</gazebo>
   </xacro:macro>
 </robot>

Commit message: changes for hydro gazebo, still not fully working

File: cob_description/gazebo/gazebo.urdf.xacro (robot description, xacro)
@@ -4,20 +4,7 @@
        xmlns:interface="http://playerstage.sourceforge.net/gazebo/xmlschema/#interface">
   <gazebo>
-	<plugin name="gazebo_ros_controller_manager" filename="libgazebo_ros_controller_manager.so">
-      <alwaysOn>true</alwaysOn>
-      <updateRate>1000.0</updateRate>
-    </plugin>
-    <plugin name="gazebo_ros_power_monitor_controller" filename="libgazebo_ros_power_monitor.so">
-      <alwaysOn>true</alwaysOn>
-      <updateRate>1.0</updateRate>
-      <timeout>5</timeout>
-      <powerStateTopic>power_state</powerStateTopic>
-      <powerStateRate>10.0</powerStateRate>
-      <fullChargeCapacity>87.78</fullChargeCapacity>
-      <dischargeRate>-474</dischargeRate>
-      <chargeRate>525</chargeRate>
-      <dischargeVoltage>15.52</dischargeVoltage>
-      <chargeVoltage>16.41</chargeVoltage>
-    </plugin>
+    <plugin name="ros_control" filename="libgazebo_ros_control.so">
+      <robotSimType>gazebo_ros_control/DefaultRobotHWSim</robotSimType>
+  </plugin>
   </gazebo>
 </robot>

File: cob_description/urdf/base/base.transmission.xacro (robot description, xacro)
@@ -6,16 +6,22 @@
   <!--  Caster wheel transmission   -->
   <xacro:macro name="cob_wheel_transmission" params="suffix parent reflect">
-    <transmission type="pr2_mechanism_model/SimpleTransmission" name="${parent}_${suffix}_wheel_trans">
-      <actuator name="${parent}_${suffix}_wheel_motor" />
+    <transmission name="${parent}_${suffix}_wheel_trans">
+      <type>transmission_interface/SimpleTransmission</type>
       <joint name="${parent}_${suffix}_wheel_joint" />
-      <mechanicalReduction>${reflect * 624/35 * 80/18}</mechanicalReduction>
+      <actuator name="${parent}_${suffix}_wheel_motor">
+        <hardwareInterface>EffortJointInterface</hardwareInterface>
+        <mechanicalReduction>${reflect * 624/35 * 80/18}</mechanicalReduction>
+      </actuator>
     </transmission>
   </xacro:macro>
   <!-- Hub transmission only -->
   <xacro:macro name="cob_caster_transmission" params="suffix">
-    <transmission type="pr2_mechanism_model/SimpleTransmission" name="${suffix}_rotation_trans">
-      <actuator name="${suffix}_rotation_motor" />
+    <transmission name="${suffix}_rotation_trans">
+      <type>transmission_interface/SimpleTransmission</type>
       <joint name="${suffix}_rotation_joint" />
-      <mechanicalReduction>${-1 * 624/35 * 80/18}</mechanicalReduction>
+      <actuator name="${suffix}_rotation_motor" >
+       <hardwareInterface>EffortJointInterface</hardwareInterface>
+        <mechanicalReduction>${-1 * 624/35 * 80/18}</mechanicalReduction>
+      </actuator>
     </transmission>
   </xacro:macro>

File: cob_description/urdf/lbr/lbr.gazebo.xacro (robot description, xacro)
@@ -6,34 +6,34 @@
 	<xacro:macro name="cob_lbr_gazebo" params="name">
 		<gazebo reference="${name}_0_link">
-			<material value="IPA/Orange" />
-			<turnGravityOff>false</turnGravityOff>
+			<material>IPA/Orange</material>
+			<turnGravityOff>true</turnGravityOff>
 		</gazebo>
 		<gazebo reference="${name}_1_link">
-			<material value="IPA/Orange" />
-			<turnGravityOff>false</turnGravityOff>
+			<material>IPA/Orange</material>
+			<turnGravityOff>true</turnGravityOff>
 		</gazebo>
 		<gazebo reference="${name}_2_link">
-			<material value="IPA/Orange" />
-			<turnGravityOff>false</turnGravityOff>
+			<material>IPA/Orange</material>
+			<turnGravityOff>true</turnGravityOff>
 		</gazebo>
 		<gazebo reference="${name}_3_link">
-			<material value="IPA/Orange" />
-			<turnGravityOff>false</turnGravityOff>
+			<material>IPA/Orange</material>
+			<turnGravityOff>true</turnGravityOff>
 		</gazebo>
 		<gazebo reference="${name}_4_link">
-			<material value="IPA/Orange" />
-			<turnGravityOff>false</turnGravityOff>
+			<material>IPA/Orange</material>
+			<turnGravityOff>true</turnGravityOff>
 		</gazebo>
 		<gazebo reference="${name}_5_link">
-			<material value="IPA/Orange" />
-			<turnGravityOff>false</turnGravityOff>
+			<material>IPA/Orange</material>
+			<turnGravityOff>true</turnGravityOff>
 		</gazebo>
 		<gazebo reference="${name}_6_link">
-			<material value="IPA/Orange" />
-			<turnGravityOff>false</turnGravityOff>
+			<material>IPA/Orange</material>
+			<turnGravityOff>true</turnGravityOff>
 		</gazebo>
 		<gazebo reference="${name}_7_link">
-			<material value="IPA/Orange" />
-			<turnGravityOff>false</turnGravityOff>
+			<material>IPA/Orange</material>
+			<turnGravityOff>true</turnGravityOff>
 		</gazebo>
 	</xacro:macro>

File: cob_description/urdf/lbr/lbr.transmission.xacro (robot description, xacro)
@@ -5,38 +5,59 @@
        xmlns:xacro="http://ros.org/wiki/xacro">
 	<xacro:macro name="cob_lbr_transmission" params="name">
-		<transmission name="${name}_1_trans" type="pr2_mechanism_model/SimpleTransmission">
-			<actuator name="${name}_1_motor"/>
+		<transmission name="${name}_1_trans">
+		  	<type>transmission_interface/SimpleTransmission</type>
+	      	<actuator name="${name}_1_motor">
+	        	<hardwareInterface>EffortJointInterface</hardwareInterface>
+	        	<mechanicalReduction>1</mechanicalReduction>
+	      	</actuator>
 			<joint name="${name}_1_joint"/>
-			<mechanicalReduction>1</mechanicalReduction>
 		</transmission>
-		<transmission name="${name}_2_trans" type="pr2_mechanism_model/SimpleTransmission">
-			<actuator name="${name}_2_motor"/>
+		<transmission name="${name}_2_trans">
+			<type>transmission_interface/SimpleTransmission</type>
+			<actuator name="${name}_2_motor">
+        		<hardwareInterface>EffortJointInterface</hardwareInterface>
+        		<mechanicalReduction>1</mechanicalReduction>
+      		</actuator>
 			<joint name="${name}_2_joint"/>
-			<mechanicalReduction>1</mechanicalReduction>
 		</transmission>
-		<transmission name="${name}_3_trans" type="pr2_mechanism_model/SimpleTransmission">
-			<actuator name="${name}_3_motor"/>
+		<transmission name="${name}_3_trans">
+			<type>transmission_interface/SimpleTransmission</type>
+			<actuator name="${name}_3_motor">
+        		<hardwareInterface>EffortJointInterface</hardwareInterface>
+        		<mechanicalReduction>1</mechanicalReduction>
+      		</actuator>
 			<joint name="${name}_3_joint"/>
-			<mechanicalReduction>1</mechanicalReduction>
 		</transmission>
-		<transmission name="${name}_4_trans" type="pr2_mechanism_model/SimpleTransmission">
-			<actuator name="${name}_4_motor"/>
+		<transmission name="${name}_4_trans">
+			<type>transmission_interface/SimpleTransmission</type>
+			<actuator name="${name}_4_motor">
+        		<hardwareInterface>EffortJointInterface</hardwareInterface>
+        		<mechanicalReduction>1</mechanicalReduction>
+      		</actuator>
 			<joint name="${name}_4_joint"/>
-			<mechanicalReduction>1</mechanicalReduction>
 		</transmission>
-		<transmission name="${name}_5_trans" type="pr2_mechanism_model/SimpleTransmission">
-			<actuator name="${name}_5_motor"/>
+		<transmission name="${name}_5_trans">
+			<type>transmission_interface/SimpleTransmission</type>
+			<actuator name="${name}_5_motor">
+        		<hardwareInterface>EffortJointInterface</hardwareInterface>
+        		<mechanicalReduction>1</mechanicalReduction>
+      		</actuator>
 			<joint name="${name}_5_joint"/>
-			<mechanicalReduction>1</mechanicalReduction>
 		</transmission>
-		<transmission name="${name}_6_trans" type="pr2_mechanism_model/SimpleTransmission">
-			<actuator name="${name}_6_motor"/>
+		<transmission name="${name}_6_trans">
+			<type>transmission_interface/SimpleTransmission</type>
+			<actuator name="${name}_6_motor">
+        		<hardwareInterface>EffortJointInterface</hardwareInterface>
+        		<mechanicalReduction>1</mechanicalReduction>
+      		</actuator>
 			<joint name="${name}_6_joint"/>
-			<mechanicalReduction>1</mechanicalReduction>
 		</transmission>
-		<transmission name="${name}_7_trans" type="pr2_mechanism_model/SimpleTransmission">
-			<actuator name="${name}_7_motor"/>
+		<transmission name="${name}_7_trans">
+			<type>transmission_interface/SimpleTransmission</type>
+			<actuator name="${name}_7_motor">
+        		<hardwareInterface>EffortJointInterface</hardwareInterface>
+        		<mechanicalReduction>1</mechanicalReduction>
+      		</actuator>
 			<joint name="${name}_7_joint"/>
-			<mechanicalReduction>1</mechanicalReduction>
 		</transmission>
 	</xacro:macro>

File: cob_description/urdf/sensors/prosilica.gazebo.xacro (robot description, xacro)
@@ -21,5 +21,5 @@
 					</clip>
 				</camera>
-				<plugin name="${name}_controller" filename="libgazebo_ros_prosilica.so">
+				<!--plugin name="${name}_controller" filename="libgazebo_ros_prosilica.so">
 					<alwaysOn>true</alwaysOn>
 					<updateRate>10.0</updateRate>
@@ -38,5 +38,5 @@
 					<distortion_t1>0.00000001</distortion_t1>
 					<distortion_t2>0.00000001</distortion_t2>
-				</plugin>
+				</plugin-->
 			</sensor>
 			<material value="IPA/LightGrey" />

File: cob_description/urdf/torso_v1/torso.transmission.xacro (robot description, xacro)
@@ -5,18 +5,27 @@
        xmlns:xacro="http://ros.org/wiki/xacro">
 	<xacro:macro name="cob_torso_transmission_v1" params="name">
-		<transmission name="${name}_lower_neck_tilt_trans" type="pr2_mechanism_model/SimpleTransmission">
-			<actuator name="${name}_lower_neck_tilt_motor"/>
+		<transmission name="${name}_lower_neck_tilt_trans">
+			<type>transmission_interface/SimpleTransmission</type>
+			<actuator name="${name}_lower_neck_tilt_motor">
+				<hardwareInterface>EffortJointInterface</hardwareInterface>
+	        	<mechanicalReduction>1</mechanicalReduction>
+	      	</actuator>
 			<joint name="${name}_lower_neck_tilt_joint"/>
-			<mechanicalReduction>1</mechanicalReduction>
 		</transmission>
-		<transmission name="${name}_pan_trans" type="pr2_mechanism_model/SimpleTransmission">
-			<actuator name="${name}_pan_motor"/>
+		<transmission name="${name}_pan_trans">
+			<type>transmission_interface/SimpleTransmission</type>
+			<actuator name="${name}_pan_motor">
+				<hardwareInterface>EffortJointInterface</hardwareInterface>
+	        	<mechanicalReduction>1</mechanicalReduction>
+	      	</actuator>
 			<joint name="${name}_pan_joint"/>
-			<mechanicalReduction>1</mechanicalReduction>
 		</transmission>
-		<transmission name="${name}_upper_neck_tilt_trans" type="pr2_mechanism_model/SimpleTransmission">
-			<actuator name="${name}_upper_neck_tilt_motor"/>
+		<transmission name="${name}_upper_neck_tilt_trans">
+			<type>transmission_interface/SimpleTransmission</type>
+			<actuator name="${name}_upper_neck_tilt_motor">
+				<hardwareInterface>EffortJointInterface</hardwareInterface>
+	        	<mechanicalReduction>1</mechanicalReduction>
+	      	</actuator>
 			<joint name="${name}_upper_neck_tilt_joint"/>
-			<mechanicalReduction>1</mechanicalReduction>
 		</transmission>
 	</xacro:macro>

File: cob_description/urdf/tray/tray.transmission.xacro (robot description, xacro)
@@ -5,8 +5,11 @@
        xmlns:xacro="http://ros.org/wiki/xacro">
 	<xacro:macro name="cob_tray_transmission" params="name">
-		<transmission name="${name}_trans" type="pr2_mechanism_model/SimpleTransmission">
-			<actuator name="${name}_motor"/>
+		<transmission name="${name}_trans">
+			<type>transmission_interface/SimpleTransmission</type>
+			<actuator name="${name}_motor">
+				<hardwareInterface>EffortJointInterface</hardwareInterface>
+	        	<mechanicalReduction>1</mechanicalReduction>
+	      	</actuator>
 			<joint name="${name}_joint"/>
-			<mechanicalReduction>1</mechanicalReduction>
 		</transmission>
 	</xacro:macro>
