Commit message: Renamed ur_connector

File: cob_description/urdf/ur_connector/ur_connector.gazebo.xacro (robot description, xacro)
@@ -4,10 +4,13 @@
        xmlns:interface="http://playerstage.sourceforge.net/gazebo/xmlschema/#interface"
        xmlns:xacro="http://ros.org/wiki/xacro">
-	<xacro:macro name="cob_ur_conector_transmission" params="name">
-		<transmission name="${name}_trans" type="pr2_mechanism_model/SimpleTransmission">
-			<actuator name="${name}_motor"/>
-			<joint name="${name}_joint"/>
-			<mechanicalReduction>1</mechanicalReduction>
-		</transmission>
+	<xacro:macro name="cob_ur_connector_gazebo" params="name">
+		<gazebo reference="${name}_fixed_link">
+			<material>IPA/DarkGrey</material>
+			<turnGravityOff>false</turnGravityOff>
+		</gazebo>
+		<gazebo reference="${name}_link">
+			<material>IPA/DarkGrey</material>
+			<turnGravityOff>false</turnGravityOff>
+		</gazebo>
 	</xacro:macro>
 </robot>

File: cob_description/urdf/ur_connector/ur_connector.transmission.xacro (robot description, xacro)
@@ -4,13 +4,10 @@
        xmlns:interface="http://playerstage.sourceforge.net/gazebo/xmlschema/#interface"
        xmlns:xacro="http://ros.org/wiki/xacro">
-	<xacro:macro name="cob_ur_conector_gazebo" params="name">
-		<gazebo reference="${name}_fixed_link">
-			<material>IPA/DarkGrey</material>
-			<turnGravityOff>false</turnGravityOff>
-		</gazebo>
-		<gazebo reference="${name}_link">
-			<material>IPA/DarkGrey</material>
-			<turnGravityOff>false</turnGravityOff>
-		</gazebo>
+	<xacro:macro name="cob_ur_connector_transmission" params="name">
+		<transmission name="${name}_trans" type="pr2_mechanism_model/SimpleTransmission">
+			<actuator name="${name}_motor"/>
+			<joint name="${name}_joint"/>
+			<mechanicalReduction>1</mechanicalReduction>
+		</transmission>
 	</xacro:macro>
 </robot>

File: cob_description/urdf/ur_connector/ur_connector.urdf.xacro (robot description, xacro)
@@ -4,8 +4,8 @@
        xmlns:interface="http://playerstage.sourceforge.net/gazebo/xmlschema/#interface"
        xmlns:xacro="http://ros.org/wiki/xacro">
-	<include filename="$(find cob_description)/urdf/ur_conector/ur_conector.gazebo.xacro" />
-	<include filename="$(find cob_description)/urdf/ur_conector/ur_conector.transmission.xacro" />
-	<xacro:macro name="cob_ur_conector" params="name parent *origin">
-		<!-- joint between base_link and ur_conector_link -->
+	<include filename="$(find cob_description)/urdf/ur_connector/ur_connector.gazebo.xacro" />
+	<include filename="$(find cob_description)/urdf/ur_connector/ur_connector.transmission.xacro" />
+	<xacro:macro name="cob_ur_connector" params="name parent *origin">
+		<!-- joint between base_link and ur_connector_link -->
 		<joint name="${name}_fixed_joint" type="fixed">
 			<insert_block name="origin" />
@@ -22,5 +22,5 @@
 				<origin xyz="0 0 0" rpy="0 0 0" />
 				<geometry>
-					<mesh filename="package://cob_description/meshes/ur_conector/ur_conector1.stl" />
+					<mesh filename="package://cob_description/meshes/ur_connector/ur_connector1.stl" />
 				</geometry>
 				<material name="IPA/DarkGrey" />
@@ -29,9 +29,9 @@
 				<origin xyz="0 0 0" rpy="0 0 0" />
 				<geometry>
-					<mesh filename="package://cob_description/meshes/ur_conector/ur_conector1.stl" />
+					<mesh filename="package://cob_description/meshes/ur_connector/ur_connector1.stl" />
 				</geometry>
 			</collision>
 		</link>
-		<!-- joint between base_link and ur_conector_link -->
+		<!-- joint between base_link and ur_connector_link -->
 		<joint name="${name}_joint" type="revolute">
 			<origin xyz="-0.0201 -0.1736 0.136" rpy="0 0 0"/>
@@ -52,5 +52,5 @@
 				<origin xyz="0 0 0" rpy="0 0 0" />
 				<geometry>
-					<mesh filename="package://cob_description/meshes/ur_conector/ur_conector2.stl" />
+					<mesh filename="package://cob_description/meshes/ur_connector/ur_connector2.stl" />
 				</geometry>
 				<material name="IPA/DarkGrey" />
@@ -59,11 +59,11 @@
 				<origin xyz="0 0 0" rpy="0 0 0" />
 				<geometry>
-					<mesh filename="package://cob_description/meshes/ur_conector/ur_conector2.stl" />
+					<mesh filename="package://cob_description/meshes/ur_connector/ur_connector2.stl" />
 				</geometry>
 			</collision>
 		</link>
 		<!-- extensions -->
-		<xacro:cob_ur_conector_gazebo name="${name}" />
-		<xacro:cob_ur_conector_transmission name="${name}" />
+		<xacro:cob_ur_connector_gazebo name="${name}" />
+		<xacro:cob_ur_connector_transmission name="${name}" />
 	</xacro:macro>
 </robot>
