Commit message: Removed safety controller urdf/ur_connector/ur_connector.urdf.xacro

File: cob_description/urdf/ur_connector/ur_connector.urdf.xacro (robot description, xacro)
@@ -39,7 +39,6 @@
 			<child link="${name}_link"/>
 			<axis xyz="0 0 1"/>
-			<dynamics damping="10"/>
-			<limit effort="200" velocity="1.9634" lower="-2.9670" upper="2.9670"/>
-            <safety_controller k_position="20" k_velocity="50" soft_lower_limit="${-2.9670 + 0.01}" soft_upper_limit="${2.9670 - 0.01}" />
+			<dynamics damping="5.0" friction="0.5"/>
+			<limit effort="100" lower="-3.31612" upper="3.31612" velocity="5"/>
 		</joint>
 		<link name="${name}_link">

Commit message: adjust limits for ur_connector

File: cob_description/urdf/ur_connector/ur_connector.urdf.xacro (robot description, xacro)
@@ -40,6 +40,6 @@
 			<axis xyz="0 0 1"/>
 			<dynamics damping="10"/>
-			<limit effort="200" velocity="1.9634" lower="-2.9670" upper="2.9670"/>
-            <safety_controller k_position="20" k_velocity="50" soft_lower_limit="${-2.9670 + 0.01}" soft_upper_limit="${2.9670 - 0.01}" />
+			<limit effort="200" velocity="1.9634" lower="1.0" upper="4.6"/>
+            <safety_controller k_position="20" k_velocity="50" soft_lower_limit="${1.0 - 0.01}" soft_upper_limit="${4.6 - 0.01}" />
 		</joint>
 		<link name="${name}_link">
