Commit message: Deleted old files and copies

File: cob_description/urdf/head_v1/head.urdf.xacro (robot description, xacro)
@@ -8,5 +8,5 @@
 	<include filename="$(find cob_description)/urdf/sensors/prosilica.urdf.xacro" />
 	<include filename="$(find cob_description)/urdf/sensors/kinect.urdf.xacro" />
-	<!--include filename="$(find cob_description)/urdf/sensors/hokuyo_SR400_laser.urdf.xacro" /-->
+	<!--include filename="$(find cob_description)/ros/urdf/sensors/hokuyo_SR400_laser.urdf.xacro" /-->
 	<xacro:macro name="cob_head_v1" params="name parent *origin">
 		<!-- joint between torso_upper_neck_tilt_link and head_axis_link -->
@@ -50,5 +50,5 @@
 		<!-- cam3d -->
 		<xacro:cob_kinect_v0 name="${name}_cam3d" ros_topic="cam3d/depth/points1" parent="${name}_color_camera_l_link">
-			<origin xyz="${cam3d_x-0.06} ${cam3d_y} ${cam3d_z}" rpy="${cam3d_roll} ${cam3d_pitch} ${cam3d_yaw+3.14}" />
+			<origin xyz="${cam3d_x-0.06} ${cam3d_y} ${cam3d_z}" rpy="${cam3d_roll} ${cam3d_pitch} ${cam3d_yaw}" />
 		</xacro:cob_kinect_v0>
 		<!-- extensions -->

Commit message: increased upper joint limit and velocity for head_v1

File: cob_description/urdf/head_v1/head.urdf.xacro (robot description, xacro)
@@ -18,5 +18,5 @@
 			<dynamics damping="0.1" />
 			<calibration rising="${head_axis_ref}"/>
-			<limit effort="100" lower="-3.2" upper="0.1" velocity="0.5"/>
+			<limit effort="100" lower="-3.2" upper="0.25" velocity="1.4"/>
 		</joint>
 		<link name="${name}_axis_link">

Commit message: moved all hardcoded offsets to calibration_data

File: cob_description/urdf/head_v1/head.urdf.xacro (robot description, xacro)
@@ -42,13 +42,13 @@
 		<!-- left camera -->
 		<xacro:cob_prosilica_v0 name="${name}_color_camera_l" ros_topic="stereo/left" parent="${name}_axis_link">
-			<origin xyz="${cam_l_x} ${cam_l_y} ${cam_l_z-0.06}" rpy="${cam_l_roll} ${cam_l_pitch+M_PI/2} ${cam_l_yaw+M_PI}" />
+			<origin xyz="${cam_l_x} ${cam_l_y} ${cam_l_z}" rpy="${cam_l_roll} ${cam_l_pitch} ${cam_l_yaw}" />
 		</xacro:cob_prosilica_v0>
 		<!-- right camera -->
 		<xacro:cob_prosilica_v0 name="${name}_color_camera_r" ros_topic="stereo/right" parent="${name}_color_camera_l_link">
-			<origin xyz="${cam_r_x-0.12} ${cam_r_y} ${cam_r_z}" rpy="${cam_r_roll} ${cam_r_pitch} ${cam_r_yaw}" />
+			<origin xyz="${cam_r_x} ${cam_r_y} ${cam_r_z}" rpy="${cam_r_roll} ${cam_r_pitch} ${cam_r_yaw}" />
 		</xacro:cob_prosilica_v0>
 		<!-- cam3d -->
 		<xacro:cob_kinect_v0 name="${name}_cam3d" ros_topic="cam3d" parent="${name}_color_camera_l_link">
-			<origin xyz="${cam3d_x-0.06} ${cam3d_y} ${cam3d_z}" rpy="${cam3d_roll} ${cam3d_pitch} ${cam3d_yaw}" />
+			<origin xyz="${cam3d_x} ${cam3d_y} ${cam3d_z}" rpy="${cam3d_roll} ${cam3d_pitch} ${cam3d_yaw}" />
 		</xacro:cob_kinect_v0>
 		<!-- extensions -->

Commit message: unified head frames

File: cob_description/urdf/head_v1/head.urdf.xacro (robot description, xacro)
@@ -10,8 +10,21 @@
 	<!--include filename="$(find cob_description)/ros/urdf/sensors/hokuyo_SR400_laser.urdf.xacro" /-->
 	<xacro:macro name="cob_head_v1" params="name parent *origin">
+		<!-- joint between torso_upper_neck_tilt_link and head_base_link -->
+        <joint name="${name}_base_joint" type="fixed">
+			<insert_block name="origin" />
+			<parent link="${parent}"/>
+            <child link="${name}_base_link"/>
+		</joint>
+        <link name="${name}_base_link">
+            <inertial>
+                <origin xyz="0 0 0" rpy="0 0 0"/>
+                <mass value="0.5"/>
+                <inertia ixx="0.01" ixy="0" ixz="0" iyy="0.01" iyz="0" izz="0.01" />
+            </inertial>
+		</link>
 		<!-- joint between torso_upper_neck_tilt_link and head_axis_link -->
 		<joint name="${name}_axis_joint" type="revolute">
-			<insert_block name="origin" />
-			<parent link="${parent}"/>
+			<origin xyz="0 0 0" rpy="0 0 0" />
+            <parent link="${name}_base_link"/>
 			<child link="${name}_axis_link"/>
 			<axis xyz="0 0 1" />
@@ -40,14 +53,27 @@
 			</collision>
 		</link>
+        <!--camera reference link-->
+        <joint name="${name}_cam_reference_joint" type="fixed">
+			<origin xyz="${cam_reference_x} ${cam_reference_y} ${cam_reference_z}" rpy="${cam_reference_roll} ${cam_reference_pitch} ${cam_reference_yaw}" />
+            <parent link="${name}_axis_link"/>
+            <child link="${name}_cam_reference_link"/>
+		</joint>
+        <link name="${name}_cam_reference_link">
+			<inertial>
+				<origin xyz="0 0 0" rpy="0 0 0"/>
+				<mass value="0.5"/>
+				<inertia ixx="0.01" ixy="0" ixz="0" iyy="0.01" iyz="0" izz="0.01" />
+			</inertial>
+		</link>
 		<!-- left camera -->
-		<xacro:cob_prosilica_v0 name="${name}_color_camera_l" ros_topic="stereo/left" parent="${name}_axis_link">
+        <xacro:cob_prosilica_v0 name="${name}_color_camera_l" ros_topic="stereo/left" parent="${name}_cam_reference_link">
 			<origin xyz="${cam_l_x} ${cam_l_y} ${cam_l_z}" rpy="${cam_l_roll} ${cam_l_pitch} ${cam_l_yaw}" />
 		</xacro:cob_prosilica_v0>
 		<!-- right camera -->
-		<xacro:cob_prosilica_v0 name="${name}_color_camera_r" ros_topic="stereo/right" parent="${name}_color_camera_l_link">
+        <xacro:cob_prosilica_v0 name="${name}_color_camera_r" ros_topic="stereo/right" parent="${name}_cam_reference_link">
 			<origin xyz="${cam_r_x} ${cam_r_y} ${cam_r_z}" rpy="${cam_r_roll} ${cam_r_pitch} ${cam_r_yaw}" />
 		</xacro:cob_prosilica_v0>
 		<!-- cam3d -->
-		<xacro:cob_kinect_v0 name="${name}_cam3d" ros_topic="cam3d" parent="${name}_color_camera_l_link">
+        <xacro:cob_kinect_v0 name="${name}_cam3d" ros_topic="cam3d" parent="${name}_cam_reference_link">
 			<origin xyz="${cam3d_x} ${cam3d_y} ${cam3d_z}" rpy="${cam3d_roll} ${cam3d_pitch} ${cam3d_yaw}" />
 		</xacro:cob_kinect_v0>

File: cob_description/urdf/head_v2/head.urdf.xacro (robot description, xacro)
@@ -9,8 +9,21 @@
 	<include filename="$(find cob_description)/urdf/sensors/kinect.urdf.xacro" />
 	<xacro:macro name="cob_head_v2" params="name parent *origin">
+		<!-- joint between torso_upper_neck_tilt_link and head_base_link -->
+        <joint name="${name}_base_joint" type="fixed">
+			<insert_block name="origin" />
+			<parent link="${parent}"/>
+            <child link="${name}_base_link"/>
+		</joint>
+        <link name="${name}_base_link">
+            <inertial>
+                <origin xyz="0 0 0" rpy="0 0 0"/>
+                <mass value="0.5"/>
+                <inertia ixx="0.01" ixy="0" ixz="0" iyy="0.01" iyz="0" izz="0.01" />
+            </inertial>
+		</link>
 		<!-- joint between torso_upper_neck_tilt_link and head_axis_link -->
 		<joint name="${name}_axis_joint" type="revolute">
-			<insert_block name="origin" />
-			<parent link="${parent}"/>
+			<origin xyz="0 0 0" rpy="0 0 0" />
+			<parent link="${name}_base_link"/>
 			<child link="${name}_axis_link"/>
 			<axis xyz="0 0 1" />
@@ -39,17 +52,30 @@
 			</collision>
 		</link>
+        <!--reference joint for cameras-->
+        <joint name="${name}_cam_reference_joint" type="fixed">
+			<origin xyz="${cam_reference_x} ${cam_reference_y} ${cam_reference_z}" rpy="${cam_reference_roll} ${cam_reference_pitch} ${cam_reference_yaw}" />
+            <parent link="${name}_axis_link"/>
+            <child link="${name}_cam_reference_link"/>
+		</joint>
+        <link name="${name}_cam_reference_link">
+			<inertial>
+				<origin xyz="0 0 0" rpy="0 0 0"/>
+				<mass value="0.5"/>
+				<inertia ixx="0.01" ixy="0" ixz="0" iyy="0.01" iyz="0" izz="0.01" />
+			</inertial>
+		</link>
 		<!-- left camera -->
-		<xacro:cob_prosilica_v0 name="${name}_color_camera_l" ros_topic="stereo/left" parent="${name}_axis_link">
+        <xacro:cob_prosilica_v0 name="${name}_color_camera_l" ros_topic="stereo/left" parent="${name}_cam_reference_link">
 			<origin xyz="${cam_l_x} ${cam_l_y} ${cam_l_z}" rpy="${cam_l_roll} ${cam_l_pitch} ${cam_l_yaw}" />
 		</xacro:cob_prosilica_v0>
 		<!-- right camera -->
-		<xacro:cob_prosilica_v0 name="${name}_color_camera_r" ros_topic="stereo/right" parent="${name}_color_camera_l_link">
+        <xacro:cob_prosilica_v0 name="${name}_color_camera_r" ros_topic="stereo/right" parent="${name}_cam_reference_link">
 			<origin xyz="${cam_r_x} ${cam_r_y} ${cam_r_z}" rpy="${cam_r_roll} ${cam_r_pitch} ${cam_r_yaw}" />
 		</xacro:cob_prosilica_v0>
 		<!-- cam3d -->
-		<xacro:cob_kinect_v0 name="${name}_cam3d" ros_topic="cam3d" parent="${name}_axis_link">
+        <xacro:cob_kinect_v0 name="${name}_cam3d" ros_topic="cam3d" parent="${name}_cam_reference_link">
 			<origin xyz="${cam3d_x} ${cam3d_y} ${cam3d_z}" rpy="${cam3d_roll} ${cam3d_pitch} ${cam3d_yaw}" />
 		</xacro:cob_kinect_v0>
-		<!-- extensions -->
+        <!-- extensions -->
 		<xacro:cob_head_gazebo_v2 name="${name}" />
 		<xacro:cob_head_transmission_v2 name="${name}" />

File: cob_description/urdf/head_v3/head.urdf.xacro (robot description, xacro)
@@ -10,32 +10,19 @@
 	<xacro:macro name="cob_head_v3" params="name parent *origin">
 		<!-- joint between torso_upper_neck_tilt_link and head_base_link -->
-		<joint name="head_base_joint" type="fixed">
+        <joint name="${name}_base_joint" type="fixed">
 			<insert_block name="origin" />
 			<parent link="${parent}"/>
-			<child link="head_base_link"/>
+            <child link="${name}_base_link"/>
 		</joint>
-		<link name="head_base_link">
-			<inertial>
-				<origin xyz="0 0 0" rpy="0 0 0"/>
-				<mass value="0.5"/>
-				<inertia ixx="0.01" ixy="0" ixz="0" iyy="0.01" iyz="0" izz="0.01" />
-			</inertial>
-			<visual>
-				<origin xyz="0 0 0" rpy="0 0 0" />
-				<geometry>
-					<box size="0.01 0.01 0.01"/>
-				</geometry>
-				<material name="IPA/Black" />
-			</visual>
-			<collision>
-				<origin xyz="0 0 0" rpy="0 0 0" />
-				<geometry>
-					<box size="0.01 0.01 0.01"/>
-				</geometry>
-			</collision>
+        <link name="${name}_base_link">
+            <inertial>
+                <origin xyz="0 0 0" rpy="0 0 0"/>
+                <mass value="0.5"/>
+                <inertia ixx="0.01" ixy="0" ixz="0" iyy="0.01" iyz="0" izz="0.01" />
+            </inertial>
 		</link>
 		<!-- joint between head_base_link and head_axis_link -->
 		<joint name="${name}_axis_joint" type="revolute">
-			<parent link="head_base_link"/>
+            <parent link="${name}_base_link"/>
 			<origin xyz="0 0 0" rpy="0 0 0" />
 			<child link="${name}_axis_link"/>
@@ -65,11 +52,11 @@
 			</collision>
 		</link>
-		<!-- joint between torso_upper_neck_tilt_link and head_base_link -->
-		<joint name="cam_reference_joint" type="fixed">
-			<origin xyz="${cam_l_x} ${cam_l_y} ${cam_l_z}" rpy="${cam_l_roll} ${cam_l_pitch} ${cam_l_yaw}" />
-			<parent link="head_axis_link"/>
-			<child link="cam_reference_link"/>
+        <!--camera reference link-->
+        <joint name="${name}_cam_reference_joint" type="fixed">
+			<origin xyz="${cam_reference_x} ${cam_reference_y} ${cam_reference_z}" rpy="${cam_reference_roll} ${cam_reference_pitch} ${cam_reference_yaw}" />
+            <parent link="${name}_axis_link"/>
+            <child link="${name}_cam_reference_link"/>
 		</joint>
-		<link name="cam_reference_link">
+        <link name="${name}_cam_reference_link">
 			<inertial>
 				<origin xyz="0 0 0" rpy="0 0 0"/>
@@ -77,28 +64,15 @@
 				<inertia ixx="0.01" ixy="0" ixz="0" iyy="0.01" iyz="0" izz="0.01" />
 			</inertial>
-			<visual>
-				<origin xyz="0 0 0" rpy="0 0 0" />
-				<geometry>
-					<box size="0.01 0.01 0.01"/>
-				</geometry>
-				<material name="IPA/Black" />
-			</visual>
-			<collision>
-				<origin xyz="0 0 0" rpy="0 0 0" />
-				<geometry>
-					<box size="0.01 0.01 0.01"/>
-				</geometry>
-			</collision>
 		</link>
 		<!-- left camera -->
-		<xacro:cob_prosilica_v0 name="${name}_color_camera_l" ros_topic="stereo/left" parent="cam_reference_link">
-			<origin xyz="0 0 0" rpy="0 0 0" />
+        <xacro:cob_prosilica_v0 name="${name}_color_camera_l" ros_topic="stereo/left" parent="${name}_cam_reference_link">
+			<origin xyz="${cam_l_x} ${cam_l_y} ${cam_l_z}" rpy="${cam_l_roll} ${cam_l_pitch} ${cam_l_yaw}" />
 		</xacro:cob_prosilica_v0>
 		<!-- right camera -->
-		<xacro:cob_prosilica_v0 name="${name}_color_camera_r" ros_topic="stereo/right" parent="cam_reference_link">
+        <xacro:cob_prosilica_v0 name="${name}_color_camera_r" ros_topic="stereo/right" parent="${name}_cam_reference_link">
 			<origin xyz="${cam_r_x} ${cam_r_y} ${cam_r_z}" rpy="${cam_r_roll} ${cam_r_pitch} ${cam_r_yaw}" />
 		</xacro:cob_prosilica_v0>
 		<!-- cam3d -->
-		<xacro:cob_kinect_v0 name="${name}_cam3d" ros_topic="cam3d" parent="cam_reference_link">
+        <xacro:cob_kinect_v0 name="${name}_cam3d" ros_topic="cam3d" parent="${name}_cam_reference_link">
 			<origin xyz="${cam3d_x} ${cam3d_y} ${cam3d_z}" rpy="${cam3d_roll} ${cam3d_pitch} ${cam3d_yaw}" />
 		</xacro:cob_kinect_v0>
