Commit message: update transmission for all components

File: cob_description/urdf/head_v1/head.transmission.xacro (robot description, xacro)
@@ -2,8 +2,11 @@
 <robot xmlns:xacro="http://www.ros.org/wiki/xacro">
   <xacro:macro name="cob_head_transmission_v1" params="name">
-    <transmission name="${name}_axis_trans" type="pr2_mechanism_model/SimpleTransmission">
-      <actuator name="${name}_axis_motor"/>
+    <transmission name="${name}_axis_trans">
+      <type>transmission_interface/SimpleTransmission</type>
       <joint name="${name}_axis_joint"/>
-      <mechanicalReduction>1</mechanicalReduction>
+      <actuator name="${name}_axis_motor">
+        <hardwareInterface>EffortJointInterface</hardwareInterface>
+        <mechanicalReduction>1</mechanicalReduction>
+      </actuator>
     </transmission>
   </xacro:macro>

File: cob_description/urdf/head_v2/head.transmission.xacro (robot description, xacro)
@@ -2,8 +2,11 @@
 <robot xmlns:xacro="http://www.ros.org/wiki/xacro">
   <xacro:macro name="cob_head_transmission_v2" params="name">
-    <transmission name="${name}_axis_trans" type="pr2_mechanism_model/SimpleTransmission">
-      <actuator name="${name}_axis_motor"/>
+    <transmission name="${name}_axis_trans">
+      <type>transmission_interface/SimpleTransmission</type>
       <joint name="${name}_axis_joint"/>
-      <mechanicalReduction>1</mechanicalReduction>
+      <actuator name="${name}_axis_motor">
+        <hardwareInterface>EffortJointInterface</hardwareInterface>
+        <mechanicalReduction>1</mechanicalReduction>
+      </actuator>
     </transmission>
   </xacro:macro>

File: cob_description/urdf/lbr/lbr.transmission.xacro (robot description, xacro)
@@ -3,58 +3,58 @@
   <xacro:macro name="cob_lbr_transmission" params="name">
     <transmission name="${name}_1_trans">
-        <type>transmission_interface/SimpleTransmission</type>
-          <actuator name="${name}_1_motor">
-            <hardwareInterface>EffortJointInterface</hardwareInterface>
-            <mechanicalReduction>1</mechanicalReduction>
-          </actuator>
+      <type>transmission_interface/SimpleTransmission</type>
       <joint name="${name}_1_joint"/>
+      <actuator name="${name}_1_motor">
+        <hardwareInterface>EffortJointInterface</hardwareInterface>
+        <mechanicalReduction>1</mechanicalReduction>
+      </actuator>
     </transmission>
     <transmission name="${name}_2_trans">
       <type>transmission_interface/SimpleTransmission</type>
+      <joint name="${name}_2_joint"/>
       <actuator name="${name}_2_motor">
-            <hardwareInterface>EffortJointInterface</hardwareInterface>
-            <mechanicalReduction>1</mechanicalReduction>
-          </actuator>
-      <joint name="${name}_2_joint"/>
+        <hardwareInterface>EffortJointInterface</hardwareInterface>
+        <mechanicalReduction>1</mechanicalReduction>
+      </actuator>
     </transmission>
     <transmission name="${name}_3_trans">
       <type>transmission_interface/SimpleTransmission</type>
+      <joint name="${name}_3_joint"/>
       <actuator name="${name}_3_motor">
-            <hardwareInterface>EffortJointInterface</hardwareInterface>
-            <mechanicalReduction>1</mechanicalReduction>
-          </actuator>
-      <joint name="${name}_3_joint"/>
+        <hardwareInterface>EffortJointInterface</hardwareInterface>
+        <mechanicalReduction>1</mechanicalReduction>
+      </actuator>
     </transmission>
     <transmission name="${name}_4_trans">
       <type>transmission_interface/SimpleTransmission</type>
+      <joint name="${name}_4_joint"/>
       <actuator name="${name}_4_motor">
-            <hardwareInterface>EffortJointInterface</hardwareInterface>
-            <mechanicalReduction>1</mechanicalReduction>
-          </actuator>
-      <joint name="${name}_4_joint"/>
+        <hardwareInterface>EffortJointInterface</hardwareInterface>
+        <mechanicalReduction>1</mechanicalReduction>
+      </actuator>
     </transmission>
     <transmission name="${name}_5_trans">
       <type>transmission_interface/SimpleTransmission</type>
+      <joint name="${name}_5_joint"/>
       <actuator name="${name}_5_motor">
-            <hardwareInterface>EffortJointInterface</hardwareInterface>
-            <mechanicalReduction>1</mechanicalReduction>
-          </actuator>
-      <joint name="${name}_5_joint"/>
+        <hardwareInterface>EffortJointInterface</hardwareInterface>
+        <mechanicalReduction>1</mechanicalReduction>
+      </actuator>
     </transmission>
     <transmission name="${name}_6_trans">
       <type>transmission_interface/SimpleTransmission</type>
+      <joint name="${name}_6_joint"/>
       <actuator name="${name}_6_motor">
-            <hardwareInterface>EffortJointInterface</hardwareInterface>
-            <mechanicalReduction>1</mechanicalReduction>
-          </actuator>
-      <joint name="${name}_6_joint"/>
+        <hardwareInterface>EffortJointInterface</hardwareInterface>
+        <mechanicalReduction>1</mechanicalReduction>
+      </actuator>
     </transmission>
     <transmission name="${name}_7_trans">
       <type>transmission_interface/SimpleTransmission</type>
+      <joint name="${name}_7_joint"/>
       <actuator name="${name}_7_motor">
-            <hardwareInterface>EffortJointInterface</hardwareInterface>
-            <mechanicalReduction>1</mechanicalReduction>
-          </actuator>
-      <joint name="${name}_7_joint"/>
+        <hardwareInterface>EffortJointInterface</hardwareInterface>
+        <mechanicalReduction>1</mechanicalReduction>
+      </actuator>
     </transmission>
   </xacro:macro>

File: cob_description/urdf/torso_v0/torso.transmission.xacro (robot description, xacro)
@@ -2,23 +2,35 @@
 <robot xmlns:xacro="http://www.ros.org/wiki/xacro">
   <xacro:macro name="cob_torso_transmission_v0" params="name">
-    <transmission name="${name}_lower_neck_pan_trans" type="pr2_mechanism_model/SimpleTransmission">
-      <actuator name="${name}_lower_neck_pan_motor"/>
+    <transmission name="${name}_lower_neck_pan_trans">
+      <type>transmission_interface/SimpleTransmission</type>
       <joint name="${name}_lower_neck_pan_joint"/>
-      <mechanicalReduction>1</mechanicalReduction>
+      <actuator name="${name}_lower_neck_pan_motor">
+        <hardwareInterface>EffortJointInterface</hardwareInterface>
+        <mechanicalReduction>1</mechanicalReduction>
+      </actuator>
     </transmission>
-    <transmission name="${name}_lower_neck_tilt_trans" type="pr2_mechanism_model/SimpleTransmission">
-      <actuator name="${name}_lower_neck_tilt_motor"/>
+    <transmission name="${name}_lower_neck_tilt_trans">
+      <type>transmission_interface/SimpleTransmission</type>
       <joint name="${name}_lower_neck_tilt_joint"/>
-      <mechanicalReduction>1</mechanicalReduction>
+      <actuator name="${name}_lower_neck_tilt_motor">
+        <hardwareInterface>EffortJointInterface</hardwareInterface>
+        <mechanicalReduction>1</mechanicalReduction>
+      </actuator>
     </transmission>
-    <transmission name="${name}_upper_neck_pan_trans" type="pr2_mechanism_model/SimpleTransmission">
-      <actuator name="${name}_upper_neck_pan_motor"/>
+    <transmission name="${name}_upper_neck_pan_trans">
+      <type>transmission_interface/SimpleTransmission</type>
       <joint name="${name}_upper_neck_pan_joint"/>
-      <mechanicalReduction>1</mechanicalReduction>
+      <actuator name="${name}_upper_neck_pan_motor">
+        <hardwareInterface>EffortJointInterface</hardwareInterface>
+        <mechanicalReduction>1</mechanicalReduction>
+      </actuator>
     </transmission>
-    <transmission name="${name}_upper_neck_tilt_trans" type="pr2_mechanism_model/SimpleTransmission">
-      <actuator name="${name}_upper_neck_tilt_motor"/>
+    <transmission name="${name}_upper_neck_tilt_trans">
+      <type>transmission_interface/SimpleTransmission</type>
       <joint name="${name}_upper_neck_tilt_joint"/>
-      <mechanicalReduction>1</mechanicalReduction>
+      <actuator name="${name}_upper_neck_tilt_motor">
+        <hardwareInterface>EffortJointInterface</hardwareInterface>
+        <mechanicalReduction>1</mechanicalReduction>
+      </actuator>
     </transmission>
   </xacro:macro>

File: cob_description/urdf/torso_v1/torso.transmission.xacro (robot description, xacro)
@@ -4,25 +4,25 @@
     <transmission name="${name}_lower_neck_tilt_trans">
       <type>transmission_interface/SimpleTransmission</type>
+      <joint name="${name}_lower_neck_tilt_joint"/>
       <actuator name="${name}_lower_neck_tilt_motor">
         <hardwareInterface>EffortJointInterface</hardwareInterface>
-            <mechanicalReduction>1</mechanicalReduction>
-          </actuator>
-      <joint name="${name}_lower_neck_tilt_joint"/>
+        <mechanicalReduction>1</mechanicalReduction>
+      </actuator>
     </transmission>
     <transmission name="${name}_pan_trans">
       <type>transmission_interface/SimpleTransmission</type>
+      <joint name="${name}_pan_joint"/>
       <actuator name="${name}_pan_motor">
         <hardwareInterface>EffortJointInterface</hardwareInterface>
-            <mechanicalReduction>1</mechanicalReduction>
-          </actuator>
-      <joint name="${name}_pan_joint"/>
+        <mechanicalReduction>1</mechanicalReduction>
+      </actuator>
     </transmission>
     <transmission name="${name}_upper_neck_tilt_trans">
       <type>transmission_interface/SimpleTransmission</type>
+      <joint name="${name}_upper_neck_tilt_joint"/>
       <actuator name="${name}_upper_neck_tilt_motor">
         <hardwareInterface>EffortJointInterface</hardwareInterface>
-            <mechanicalReduction>1</mechanicalReduction>
-          </actuator>
-      <joint name="${name}_upper_neck_tilt_joint"/>
+        <mechanicalReduction>1</mechanicalReduction>
+      </actuator>
     </transmission>
   </xacro:macro>

File: cob_description/urdf/tray/tray.transmission.xacro (robot description, xacro)
@@ -4,9 +4,9 @@
     <transmission name="${name}_trans">
       <type>transmission_interface/SimpleTransmission</type>
+      <joint name="${name}_joint"/>
       <actuator name="${name}_motor">
         <hardwareInterface>EffortJointInterface</hardwareInterface>
-            <mechanicalReduction>1</mechanicalReduction>
-          </actuator>
-      <joint name="${name}_joint"/>
+        <mechanicalReduction>1</mechanicalReduction>
+      </actuator>
     </transmission>
   </xacro:macro>

File: cob_description/urdf/tray_powerball/tray.transmission.xacro (robot description, xacro)
@@ -2,18 +2,27 @@
 <robot xmlns:xacro="http://www.ros.org/wiki/xacro">
   <xacro:macro name="cob_tray_powerball_transmission" params="name">
-    <transmission name="${name}_1_trans" type="pr2_mechanism_model/SimpleTransmission">
-      <actuator name="${name}_1_motor"/>
+    <transmission name="${name}_1_trans">
+      <type>transmission_interface/SimpleTransmission</type>
       <joint name="${name}_1_joint"/>
-      <mechanicalReduction>1</mechanicalReduction>
+      <actuator name="${name}_1_motor">
+        <hardwareInterface>EffortJointInterface</hardwareInterface>
+        <mechanicalReduction>1</mechanicalReduction>
+      </actuator>
     </transmission>
-    <transmission name="${name}_2_trans" type="pr2_mechanism_model/SimpleTransmission">
-      <actuator name="${name}_2_motor"/>
+    <transmission name="${name}_2_trans">
+      <type>transmission_interface/SimpleTransmission</type>
       <joint name="${name}_2_joint"/>
-      <mechanicalReduction>1</mechanicalReduction>
+      <actuator name="${name}_2_motor">
+        <hardwareInterface>EffortJointInterface</hardwareInterface>
+        <mechanicalReduction>1</mechanicalReduction>
+      </actuator>
     </transmission>
-    <transmission name="${name}_3_trans" type="pr2_mechanism_model/SimpleTransmission">
-      <actuator name="${name}_3_motor"/>
+    <transmission name="${name}_3_trans">
+      <type>transmission_interface/SimpleTransmission</type>
       <joint name="${name}_3_joint"/>
-      <mechanicalReduction>1</mechanicalReduction>
+      <actuator name="${name}_3_motor">
+        <hardwareInterface>EffortJointInterface</hardwareInterface>
+        <mechanicalReduction>1</mechanicalReduction>
+      </actuator>
     </transmission>
   </xacro:macro>

File: cob_description/urdf/ur_connector/ur_connector.transmission.xacro (robot description, xacro)
@@ -2,8 +2,11 @@
 <robot xmlns:xacro="http://www.ros.org/wiki/xacro">
   <xacro:macro name="cob_ur_connector_transmission" params="name">
-    <transmission name="${name}_trans" type="pr2_mechanism_model/SimpleTransmission">
-      <actuator name="${name}_motor"/>
+    <transmission name="${name}_trans">
+      <type>transmission_interface/SimpleTransmission</type>
       <joint name="${name}_joint"/>
-      <mechanicalReduction>1</mechanicalReduction>
+      <actuator name="${name}_motor">
+        <hardwareInterface>EffortJointInterface</hardwareInterface>
+        <mechanicalReduction>1</mechanicalReduction>
+      </actuator>
     </transmission>
   </xacro:macro>

File: desire_description/urdf/base_desire/base.transmission.xacro (robot description, xacro)
@@ -3,16 +3,22 @@
   <!--  Caster wheel transmission   -->
   <xacro:macro name="desire_wheel_transmission_v0" params="suffix parent reflect">
-    <transmission type="pr2_mechanism_model/SimpleTransmission" name="${parent}_${suffix}_wheel_trans">
-      <actuator name="${parent}_${suffix}_wheel_motor" />
-      <joint name="${parent}_${suffix}_wheel_joint" />
-      <mechanicalReduction>${reflect * 624/35 * 80/18}</mechanicalReduction>
+    <transmission name="desire_wheel_transmission_v0">
+      <type>transmission_interface/SimpleTransmission</type>
+      <joint name="${parent}_${suffix}_wheel_joint"/>
+      <actuator name="${parent}_${suffix}_wheel_motor">
+        <hardwareInterface>EffortJointInterface</hardwareInterface>
+        <mechanicalReduction>${reflect * 624/35 * 80/18}</mechanicalReduction>
+      </actuator>
     </transmission>
   </xacro:macro>
   <!-- Hub transmission only -->
   <xacro:macro name="desire_caster_transmission_v0" params="suffix">
-    <transmission type="pr2_mechanism_model/SimpleTransmission" name="${suffix}_rotation_trans">
-      <actuator name="${suffix}_rotation_motor" />
-      <joint name="${suffix}_rotation_joint" />
-      <mechanicalReduction>${-1 * 624/35 * 80/18}</mechanicalReduction>
+    <transmission name="desire_caster_transmission_v0">
+      <type>transmission_interface/SimpleTransmission</type>
+      <joint name="${suffix}_rotation_joint"/>
+      <actuator name="${suffix}_rotation_motor">
+        <hardwareInterface>EffortJointInterface</hardwareInterface>
+        <mechanicalReduction>${-1 * 624/35 * 80/18}</mechanicalReduction>
+      </actuator>
     </transmission>
   </xacro:macro>

File: desire_description/urdf/head_desire/head.transmission.xacro (robot description, xacro)
@@ -2,13 +2,19 @@
 <robot xmlns:xacro="http://www.ros.org/wiki/xacro">
   <xacro:macro name="head_desire_transmission_v0" params="name">
-    <transmission name="${name}_pan_trans" type="pr2_mechanism_model/SimpleTransmission">
-      <actuator name="${name}_pan_motor"/>
+    <transmission name="${name}_pan_trans">
+      <type>transmission_interface/SimpleTransmission</type>
       <joint name="${name}_pan_joint"/>
-      <mechanicalReduction>1</mechanicalReduction>
+      <actuator name="${name}_pan_motor">
+        <hardwareInterface>EffortJointInterface</hardwareInterface>
+        <mechanicalReduction>1</mechanicalReduction>
+      </actuator>
     </transmission>
-    <transmission name="${name}_tilt_trans" type="pr2_mechanism_model/SimpleTransmission">
-      <actuator name="${name}_tilt_motor"/>
+    <transmission name="${name}_tilt_trans">
+      <type>transmission_interface/SimpleTransmission</type>
       <joint name="${name}_tilt_joint"/>
-      <mechanicalReduction>1</mechanicalReduction>
+      <actuator name="${name}_tilt_motor">
+        <hardwareInterface>EffortJointInterface</hardwareInterface>
+        <mechanicalReduction>1</mechanicalReduction>
+      </actuator>
     </transmission>
   </xacro:macro>

File: raw_description/urdf/base_long/base.transmission.xacro (robot description, xacro)
@@ -3,16 +3,22 @@
   <!--  Caster wheel transmission   -->
   <xacro:macro name="cob_wheel_transmission" params="suffix parent reflect">
-    <transmission type="pr2_mechanism_model/SimpleTransmission" name="${parent}_${suffix}_wheel_trans">
-      <actuator name="${parent}_${suffix}_wheel_motor" />
-      <joint name="${parent}_${suffix}_wheel_joint" />
-      <mechanicalReduction>${reflect * 624/35 * 80/18}</mechanicalReduction>
+    <transmission name="cob_wheel_transmission">
+      <type>transmission_interface/SimpleTransmission</type>
+      <joint name="${parent}_${suffix}_wheel_joint"/>
+      <actuator name="${parent}_${suffix}_wheel_motor">
+        <hardwareInterface>EffortJointInterface</hardwareInterface>
+        <mechanicalReduction>${reflect * 624/35 * 80/18}</mechanicalReduction>
+      </actuator>
     </transmission>
   </xacro:macro>
   <!-- Hub transmission only -->
   <xacro:macro name="cob_caster_transmission" params="suffix">
-    <transmission type="pr2_mechanism_model/SimpleTransmission" name="${suffix}_rotation_trans">
-      <actuator name="${suffix}_rotation_motor" />
-      <joint name="${suffix}_rotation_joint" />
-      <mechanicalReduction>${-1 * 624/35 * 80/18}</mechanicalReduction>
+    <transmission name="cob_caster_transmission">
+      <type>transmission_interface/SimpleTransmission</type>
+      <joint name="${suffix}_rotation_joint"/>
+      <actuator name="${suffix}_rotation_motor">
+        <hardwareInterface>EffortJointInterface</hardwareInterface>
+        <mechanicalReduction>${-1 * 624/35 * 80/18}</mechanicalReduction>
+      </actuator>
     </transmission>
   </xacro:macro>

File: raw_description/urdf/torso/torso.transmission.xacro (robot description, xacro)
@@ -2,13 +2,19 @@
 <robot xmlns:xacro="http://www.ros.org/wiki/xacro">
   <xacro:macro name="raw_torso_transmission" params="name">
-    <transmission name="${name}_pan_trans" type="pr2_mechanism_model/SimpleTransmission">
-      <actuator name="${name}_pan_motor"/>
+    <transmission name="${name}_pan_trans">
+      <type>transmission_interface/SimpleTransmission</type>
       <joint name="${name}_pan_joint"/>
-      <mechanicalReduction>1</mechanicalReduction>
+      <actuator name="${name}_pan_motor">
+        <hardwareInterface>EffortJointInterface</hardwareInterface>
+        <mechanicalReduction>1</mechanicalReduction>
+      </actuator>
     </transmission>
-    <transmission name="${name}_tilt_trans" type="pr2_mechanism_model/SimpleTransmission">
-      <actuator name="${name}_tilt_motor"/>
+    <transmission name="${name}_tilt_trans">
+      <type>transmission_interface/SimpleTransmission</type>
       <joint name="${name}_tilt_joint"/>
-      <mechanicalReduction>1</mechanicalReduction>
+      <actuator name="${name}_tilt_motor">
+        <hardwareInterface>EffortJointInterface</hardwareInterface>
+        <mechanicalReduction>1</mechanicalReduction>
+      </actuator>
     </transmission>
   </xacro:macro>
