Commit message: Adjust limits for tray and torso

File: cob_description/urdf/torso_v1/torso.urdf.xacro (robot description, xacro)
@@ -28,5 +28,5 @@
 			<dynamics damping="25.0" friction="10.0"/>
 			<calibration rising="${torso_lower_neck_tilt_ref}"/>
-			<limit effort="41.4" lower="-0.25" upper="0.25" velocity="0.5"/>
+			<limit effort="41.4" lower="-0.22" upper="0.22" velocity="0.5"/>
 		</joint>
 		<link name="${name}_lower_neck_tilt_link">
@@ -58,5 +58,5 @@
 			<dynamics damping="25.0" friction="10.0"/>
 			<calibration rising="${torso_pan_ref}"/>
-			<limit effort="41.4" lower="-0.2" upper="0.2" velocity="0.5"/>
+			<limit effort="41.4" lower="-0.12" upper="0.12" velocity="0.5"/>
 		</joint>
 		<link name="${name}_pan_link">
@@ -75,5 +75,5 @@
 			<dynamics damping="25.0" friction="10.0"/>
 			<calibration rising="${torso_upper_neck_tilt_ref}"/>
-			<limit effort="41.4" lower="-0.4" upper="0.4" velocity="0.5"/>
+			<limit effort="41.4" lower="-0.37" upper="0.37" velocity="0.5"/>
 		</joint>
 		<link name="${name}_upper_neck_tilt_link">

File: cob_description/urdf/tray_powerball/tray.urdf.xacro (robot description, xacro)
@@ -16,5 +16,5 @@
 			<calibration rising="${tray_1_ref}"/>
 			<dynamics damping="5.0" friction="0.5"/>
-			<limit effort="100" lower="-3.31612" upper="3.31612" velocity="5"/>
+			<limit effort="100" lower="-1.37" upper="0.02" velocity="5"/>
 		</joint>
 		<link name="${name}_1_link">
@@ -45,5 +45,5 @@
 			<calibration rising="${tray_2_ref}"/>
 			<dynamics damping="5.0" friction="0.5"/>
-			<limit effort="100" lower="-3.31612" upper="3.31612" velocity="5"/>
+			<limit effort="100" lower="-3.34" upper="3.34" velocity="5"/>
 		</joint>
 		<link name="${name}_2_link">
@@ -68,5 +68,5 @@
 		</link>
 		<joint name="${name}_3_joint" type="revolute">
-			<origin xyz="0.0671 0.0 0.0671" rpy="0 1.570796 0"/>
+			<origin xyz="0.0671 0.0 0.0671" rpy="0 1.5708 0"/>
 			<parent link="${name}_2_link"/>
 			<child link="${name}_3_link"/>
@@ -74,5 +74,5 @@
 			<calibration rising="${tray_3_ref}"/>
 			<dynamics damping="5.0" friction="0.5"/>
-			<limit effort="100" lower="-3.31612" upper="3.31612" velocity="5"/>
+			<limit effort="100" lower="-3.34" upper="3.34" velocity="5"/>
 		</joint>
 		<link name="${name}_3_link">
