Commit message: tested on robot

File: cob_description/urdf/base_cob4/base.urdf.xacro (robot description, xacro)
@@ -75,12 +75,12 @@
 		</link>
 		<!--modify here for test: front,base and top lasers -->
-		<xacro:sick_s300_laser_v0 name="${name}_laser_1" parent="${name}" ros_topic="scan_1_raw" update_rate="12" min_angle="-2.094" max_angle="2.094" >
-			<origin xyz="${laser_1_x} ${laser_1_y} ${laser_1_z}" rpy="${laser_1_roll} ${laser_1_pitch} ${laser_1_yaw}" />
+		<xacro:sick_s300_laser_v0 name="${name}_laser_front" parent="${name}" ros_topic="scan_front_raw" update_rate="12" min_angle="-2.094" max_angle="2.094" >
+			<origin xyz="${laser_front_x} ${laser_front_y} ${laser_front_z}" rpy="${laser_front_roll} ${laser_front_pitch} ${laser_front_yaw}" />
 		</xacro:sick_s300_laser_v0>
-		<xacro:sick_s300_laser_v0 name="${name}_laser_2" parent="${name}" ros_topic="scan_2_raw" update_rate="12" min_angle="-2.094" max_angle="2.094" >
-			<origin xyz="${laser_2_x} ${laser_2_y} ${laser_2_z}" rpy="${laser_2_roll} ${laser_2_pitch} ${laser_2_yaw}" />
+		<xacro:sick_s300_laser_v0 name="${name}_laser_left" parent="${name}" ros_topic="scan_left_raw" update_rate="12" min_angle="-2.094" max_angle="2.094" >
+			<origin xyz="${laser_left_x} ${laser_left_y} ${laser_left_z}" rpy="${laser_left_roll} ${laser_left_pitch} ${laser_left_yaw}" />
 		</xacro:sick_s300_laser_v0>
-		<xacro:sick_s300_laser_v0 name="${name}_laser_3" parent="${name}" ros_topic="scan_3_raw" update_rate="12" min_angle="-2.094" max_angle="2.094" >
-			<origin xyz="${laser_3_x} ${laser_3_y} ${laser_3_z}" rpy="${laser_3_roll} ${laser_3_pitch} ${laser_3_yaw}" />
+		<xacro:sick_s300_laser_v0 name="${name}_laser_right" parent="${name}" ros_topic="scan_right_raw" update_rate="12" min_angle="-2.094" max_angle="2.094" >
+			<origin xyz="${laser_right_x} ${laser_right_y} ${laser_right_z}" rpy="${laser_right_roll} ${laser_right_pitch} ${laser_right_yaw}" />
 		</xacro:sick_s300_laser_v0>
 		<xacro:cob_caster suffix="fl" parent="${name}_link" ref_position="0" >
