Commit message: New struture for cob repositories

File: cob_description/urdf/base_cob3/base.gazebo.xacro (robot description, xacro)
@@ -18,5 +18,5 @@
     </gazebo>
   </xacro:macro>
-  <xacro:macro name="cob4_base_gazebo" params="name">
+  <xacro:macro name="cob3_base_gazebo" params="name">
 	<gazebo reference="${name}_link">
 		<selfCollide>true</selfCollide>
@@ -31,5 +31,5 @@
 			</plugin>
 		</sensor>
-		<material>IPA/DarkGrey</material>
+		<material>IPA/LightGrey</material>
 	</gazebo>
     <gazebo>

File: cob_description/urdf/base_cob4/base.urdf.xacro (robot description, xacro)
@@ -24,5 +24,5 @@
 	<property name="base_size_z" value="0.23" />
 	<property name="base_collision_size_z" value="0.04" />
-	<xacro:macro name="cob_base" params="name">
+	<xacro:macro name="cob4_base" params="name">
 		<link name="base_footprint">
 			<inertial>
@@ -93,5 +93,5 @@
 			<origin xyz="${caster_offset_x/2} ${-caster_offset_y} ${caster_offset_z}" rpy="0 0 0" />
 		</xacro:cob_caster>
-	<xacro:cob_base_gazebo name="${name}" />
+	<xacro:cob4_base_gazebo name="${name}" />
 	</xacro:macro>
 	<!--                                                      -->

File: cob_description/urdf/head_cob4/head.transmission.xacro (robot description, xacro)
@@ -4,5 +4,5 @@
        xmlns:interface="http://playerstage.sourceforge.net/gazebo/xmlschema/#interface"
        xmlns:xacro="http://ros.org/wiki/xacro">
-	<xacro:macro name="cob_head_gazebo" params="name">
+	<xacro:macro name="cob4_head_gazebo" params="name">
 		<gazebo reference="${name}_base_link">
 			<material>IPA/LightGrey</material>

File: cob_description/urdf/head_cob4/head.urdf.xacro (robot description, xacro)
@@ -6,5 +6,5 @@
 	<include filename="$(find cob_description)/urdf/head_cob4/head.gazebo.xacro" />
 	<include filename="$(find cob_description)/urdf/head_cob4/head.transmission.xacro" />
-	<xacro:macro name="cob_head" params="parent name *origin">
+	<xacro:macro name="cob4_head" params="parent name *origin">
 		<joint name="head_base_joint" type="fixed">
 		  <insert_block name="origin" />
@@ -52,5 +52,5 @@
 			<origin xyz="0 0 0" rpy="0 0 0" />
 			<geometry>
-				<mesh filename="package://cob4_description/meshes/head/head_link.stl"/>
+				<mesh filename="package://cob_description/meshes/head_cob4/head_link.stl"/>
 			</geometry>
 			<material name="IPA/LightGrey"/>
@@ -64,6 +64,6 @@
 		</link>
 	<!-- extensions -->
-	<xacro:cob_head_gazebo name="${name}" />
-	<xacro:cob_head_transmission name="${name}" />
+	<xacro:cob4_head_gazebo name="${name}" />
+	<xacro:cob4_head_transmission name="${name}" />
 	</xacro:macro>
 </robot>

File: cob_description/urdf/torso_cob3_v1/torso.gazebo.xacro (robot description, xacro)
@@ -4,19 +4,23 @@
        xmlns:interface="http://playerstage.sourceforge.net/gazebo/xmlschema/#interface"
        xmlns:xacro="http://ros.org/wiki/xacro">
-	<xacro:macro name="cob4_torso_gazebo" params="name">
-		<gazebo reference="${name}_base_link">
-            <material>IPA/LightGrey</material>
-			<turnGravityOff>false</turnGravityOff>
-		</gazebo>
-		<gazebo reference="${name}_1_link">
+	<xacro:macro name="cob3_torso_gazebo_v1" params="name">
+		<gazebo reference="${name}_lower_neck_pan_link">
 			<material>IPA/LightGrey</material>
 			<turnGravityOff>false</turnGravityOff>
 		</gazebo>
-		<gazebo reference="${name}_2_link">
+		<gazebo reference="${name}_lower_neck_tilt_link">
 			<material>IPA/LightGrey</material>
 			<turnGravityOff>false</turnGravityOff>
 		</gazebo>
-		<gazebo reference="${name}_3_link">
+		<gazebo reference="${name}_upper_neck_pan_link">
 			<material>IPA/LightGrey</material>
+			<turnGravityOff>false</turnGravityOff>
+		</gazebo>
+		<gazebo reference="${name}_upper_neck_tilt_link">
+			<material>IPA/LightGrey</material>
+			<turnGravityOff>false</turnGravityOff>
+		</gazebo>
+		<gazebo reference="head_cover_link">
+			<material>IPA/Black</material>
 			<turnGravityOff>false</turnGravityOff>
 		</gazebo>

File: cob_description/urdf/torso_cob3_v2/torso.gazebo.xacro (robot description, xacro)
@@ -4,19 +4,19 @@
        xmlns:interface="http://playerstage.sourceforge.net/gazebo/xmlschema/#interface"
        xmlns:xacro="http://ros.org/wiki/xacro">
-	<xacro:macro name="cob4_torso_gazebo" params="name">
-		<gazebo reference="${name}_base_link">
-            <material>IPA/LightGrey</material>
-			<turnGravityOff>false</turnGravityOff>
-		</gazebo>
-		<gazebo reference="${name}_1_link">
+	<xacro:macro name="cob3_torso_gazebo_v2" params="name">
+		<gazebo reference="${name}_lower_neck_tilt_link">
 			<material>IPA/LightGrey</material>
 			<turnGravityOff>false</turnGravityOff>
 		</gazebo>
-		<gazebo reference="${name}_2_link">
+		<gazebo reference="${name}_pan_link">
 			<material>IPA/LightGrey</material>
 			<turnGravityOff>false</turnGravityOff>
 		</gazebo>
-		<gazebo reference="${name}_3_link">
+		<gazebo reference="${name}_upper_neck_tilt_link">
 			<material>IPA/LightGrey</material>
+			<turnGravityOff>false</turnGravityOff>
+		</gazebo>
+		<gazebo reference="head_cover_link">
+			<material>IPA/Black</material>
 			<turnGravityOff>false</turnGravityOff>
 		</gazebo>

File: cob_description/urdf/torso_cob4/torso.gazebo.xacro (robot description, xacro)
@@ -4,5 +4,5 @@
        xmlns:interface="http://playerstage.sourceforge.net/gazebo/xmlschema/#interface"
        xmlns:xacro="http://ros.org/wiki/xacro">
-	<xacro:macro name="cob_torso_transmission" params="name">
+	<xacro:macro name="cob4_torso_transmission" params="name">
 		<transmission name="${name}_1_trans" type="pr2_mechanism_model/SimpleTransmission">
 			<actuator name="${name}_1_motor"/>

File: cob_description/urdf/torso_cob4/torso.urdf.xacro (robot description, xacro)
@@ -6,5 +6,5 @@
 	<include filename="$(find cob_description)/urdf/torso_cob4/torso.gazebo.xacro" />
 	<include filename="$(find cob_description)/urdf/torso_cob4/torso.transmission.xacro" />
-	<xacro:macro name="cob_torso" params="parent name *origin">
+	<xacro:macro name="cob4_torso" params="parent name *origin">
 		<joint name="torso_base_joint" type="fixed">
 		  <insert_block name="origin" />
@@ -64,6 +64,6 @@
 		</link>
 	<!-- extensions -->
-	<xacro:cob_torso_gazebo name="${name}" />
-	<xacro:cob_torso_transmission name="${name}" />
+	<xacro:cob4_torso_gazebo name="${name}" />
+	<xacro:cob4_torso_transmission name="${name}" />
 	</xacro:macro>
 </robot>

File: cob_description/urdf/tray_cob3_3DOF/tray.gazebo.xacro (robot description, xacro)
@@ -4,19 +4,15 @@
        xmlns:interface="http://playerstage.sourceforge.net/gazebo/xmlschema/#interface"
        xmlns:xacro="http://ros.org/wiki/xacro">
-	<xacro:macro name="cob4_torso_gazebo" params="name">
-		<gazebo reference="${name}_base_link">
-            <material>IPA/LightGrey</material>
-			<turnGravityOff>false</turnGravityOff>
-		</gazebo>
+	<xacro:macro name="cob3_tray_3DOF_gazebo" params="name">
 		<gazebo reference="${name}_1_link">
-			<material>IPA/LightGrey</material>
+			<material>IPA/DarkGrey</material>
 			<turnGravityOff>false</turnGravityOff>
 		</gazebo>
 		<gazebo reference="${name}_2_link">
-			<material>IPA/LightGrey</material>
+			<material>IPA/DarkGrey</material>
 			<turnGravityOff>false</turnGravityOff>
 		</gazebo>
 		<gazebo reference="${name}_3_link">
-			<material>IPA/LightGrey</material>
+			<material>IPA/DarkGrey</material>
 			<turnGravityOff>false</turnGravityOff>
 		</gazebo>

File: cob_description/urdf/tray_cob3_3DOF/tray.transmission.xacro (robot description, xacro)
@@ -4,5 +4,5 @@
        xmlns:interface="http://playerstage.sourceforge.net/gazebo/xmlschema/#interface"
        xmlns:xacro="http://ros.org/wiki/xacro">
-	<xacro:macro name="cob4_head_transmission" params="name">
+	<xacro:macro name="cob3_tray_3DOF_transmission" params="name">
 		<transmission name="${name}_1_trans" type="pr2_mechanism_model/SimpleTransmission">
 			<actuator name="${name}_1_motor"/>
