Commit message: renamed files

File: cob_description/urdf/torso_cob4/torso.gazebo.xacro (robot description, xacro)
@@ -4,20 +4,21 @@
        xmlns:interface="http://playerstage.sourceforge.net/gazebo/xmlschema/#interface"
        xmlns:xacro="http://ros.org/wiki/xacro">
-	<xacro:macro name="cob4_torso_transmission" params="name">
-		<transmission name="${name}_1_trans" type="pr2_mechanism_model/SimpleTransmission">
-			<actuator name="${name}_1_motor"/>
-			<joint name="${name}_1_joint"/>
-			<mechanicalReduction>1</mechanicalReduction>
-		</transmission>
-		<transmission name="${name}_2_trans" type="pr2_mechanism_model/SimpleTransmission">
-			<actuator name="${name}_2_motor"/>
-			<joint name="${name}_2_joint"/>
-			<mechanicalReduction>1</mechanicalReduction>
-		</transmission>
-		<transmission name="${name}_3_trans" type="pr2_mechanism_model/SimpleTransmission">
-			<actuator name="${name}_3_motor"/>
-			<joint name="${name}_3_joint"/>
-			<mechanicalReduction>1</mechanicalReduction>
-		</transmission>
+	<xacro:macro name="cob4_torso_gazebo" params="name">
+		<gazebo reference="${name}_base_link">
+            <material>IPA/LightGrey</material>
+			<turnGravityOff>false</turnGravityOff>
+		</gazebo>
+		<gazebo reference="${name}_1_link">
+			<material>IPA/LightGrey</material>
+			<turnGravityOff>false</turnGravityOff>
+		</gazebo>
+		<gazebo reference="${name}_2_link">
+			<material>IPA/LightGrey</material>
+			<turnGravityOff>false</turnGravityOff>
+		</gazebo>
+		<gazebo reference="${name}_3_link">
+			<material>IPA/LightGrey</material>
+			<turnGravityOff>false</turnGravityOff>
+		</gazebo>
 	</xacro:macro>
 </robot>

File: cob_description/urdf/torso_cob4/torso.transmission.xacro (robot description, xacro)
@@ -4,21 +4,20 @@
        xmlns:interface="http://playerstage.sourceforge.net/gazebo/xmlschema/#interface"
        xmlns:xacro="http://ros.org/wiki/xacro">
-	<xacro:macro name="cob4_torso_gazebo" params="name">
-		<gazebo reference="${name}_base_link">
-            <material>IPA/LightGrey</material>
-			<turnGravityOff>false</turnGravityOff>
-		</gazebo>
-		<gazebo reference="${name}_1_link">
-			<material>IPA/LightGrey</material>
-			<turnGravityOff>false</turnGravityOff>
-		</gazebo>
-		<gazebo reference="${name}_2_link">
-			<material>IPA/LightGrey</material>
-			<turnGravityOff>false</turnGravityOff>
-		</gazebo>
-		<gazebo reference="${name}_3_link">
-			<material>IPA/LightGrey</material>
-			<turnGravityOff>false</turnGravityOff>
-		</gazebo>
+	<xacro:macro name="cob4_torso_transmission" params="name">
+		<transmission name="${name}_1_trans" type="pr2_mechanism_model/SimpleTransmission">
+			<actuator name="${name}_1_motor"/>
+			<joint name="${name}_1_joint"/>
+			<mechanicalReduction>1</mechanicalReduction>
+		</transmission>
+		<transmission name="${name}_2_trans" type="pr2_mechanism_model/SimpleTransmission">
+			<actuator name="${name}_2_motor"/>
+			<joint name="${name}_2_joint"/>
+			<mechanicalReduction>1</mechanicalReduction>
+		</transmission>
+		<transmission name="${name}_3_trans" type="pr2_mechanism_model/SimpleTransmission">
+			<actuator name="${name}_3_motor"/>
+			<joint name="${name}_3_joint"/>
+			<mechanicalReduction>1</mechanicalReduction>
+		</transmission>
 	</xacro:macro>
 </robot>

File: cob_description/urdf/torso_cob4/torso.urdf.xacro (robot description, xacro)
@@ -52,5 +52,6 @@
 				<origin xyz="0 0 0" rpy="0 0 0" />
 				<geometry>
-					<mesh filename="package://cob_description/meshes/torso_cob4/torso_link.stl"/>
+					<!--mesh filename="package://cob_description/meshes/torso_cob4/torso_link.stl"/-->
+					<box size="0.001 0.001 0.001" />
 				</geometry>
 				<material name="IPA/LightGrey"/>
@@ -64,6 +65,6 @@
 		</link>
 	<!-- extensions -->
-	<xacro:cob4_torso_gazebo name="${name}" />
-	<xacro:cob4_torso_transmission name="${name}" />
+	<xacro:cob4_torso_gazebo name="torso" />
+	<xacro:cob4_torso_transmission name="torso" />
 	</xacro:macro>
 </robot>
