Commit message: cob4 integration

File: cob_description/urdf/head_cob4/head.urdf.xacro (robot description, xacro)
@@ -52,5 +52,5 @@
 			<origin xyz="0 0 0" rpy="0 0 0" />
 			<geometry>
-				<mesh filename="package://cob_description/meshes/head_cob4/head_link.stl"/>
+				<mesh filename="package://cob4_description/meshes/head/head_link.stl"/>
 			</geometry>
 			<material name="IPA/LightGrey"/>

Commit message: update cob4 description

File: cob_description/urdf/head_cob4/head.urdf.xacro (robot description, xacro)
@@ -12,5 +12,11 @@
 		  <parent link="${parent}"/>
 		</joint>
-		<link name="head_base_link"/>
+		<link name="head_base_link">
+			<inertial>
+				<origin xyz="0 0 0" rpy="0 0 0"/>
+				<mass value="0.1"/>
+				<inertia ixx="0.01" ixy="0" ixz="0" iyy="0.01" iyz="0" izz="0.01" />
+			</inertial>
+		</link>
 		<joint name="head_1_joint" type="revolute">
 		  <origin xyz="0 0 0.0305" rpy="0 0 0"/>
@@ -22,5 +28,11 @@
 		  <limit effort="100" lower="-6.2831" upper="6.2831" velocity="1.4"/>
 		</joint>
-		<link name="head_1_link"/>
+		<link name="head_1_link">
+			<inertial>
+				<origin xyz="0 0 0" rpy="0 0 0"/>
+				<mass value="0.1"/>
+				<inertia ixx="0.01" ixy="0" ixz="0" iyy="0.01" iyz="0" izz="0.01" />
+			</inertial>
+		</link>
 		<joint name="head_2_joint" type="revolute">
 		  <origin xyz="0 -0.07725 -0.00439" rpy="-0.349 0 0" />
@@ -32,5 +44,11 @@
 		  <limit effort="100" lower="-6.2831" upper="6.2831" velocity="1.4"/>
 		</joint>
-		<link name="head_2_link"/>
+		<link name="head_2_link">
+			<inertial>
+				<origin xyz="0 0 0" rpy="0 0 0"/>
+				<mass value="0.1"/>
+				<inertia ixx="0.01" ixy="0" ixz="0" iyy="0.01" iyz="0" izz="0.01" />
+			</inertial>
+		</link>
 		<joint name="head_3_joint" type="revolute">
 		  <origin xyz="0 0.08001 0.06809" rpy="0.349 0 0" />

File: cob_description/urdf/sensorring/sensorring.urdf.xacro (robot description, xacro)
@@ -4,15 +4,26 @@
        xmlns:interface="http://playerstage.sourceforge.net/gazebo/xmlschema/#interface"
        xmlns:xacro="http://ros.org/wiki/xacro">
+	<include filename="$(find cob_description)/urdf/sensorring/sensorring.gazebo.xacro" />
+	<include filename="$(find cob_description)/urdf/sensorring/sensorring.transmission.xacro" />
 	<xacro:macro name="cob_sensorring" params="parent name *origin">
-		<joint name="sensorring_joint" type="revolute">
-			  <insert_block name="origin" />
-			  <child link="sensorring_link" />
-			  <parent link="${parent}"/>
-			  <calibration rising="${head_sensor_ref}"/>
-			  <axis xyz="0 0 1" />
-			  <dynamics damping="0.1" />
-			  <limit effort="100" lower="-6.2831" upper="6.2831" velocity="1.4"/>
+		<joint name="${name}_joint" type="revolute">
+			<insert_block name="origin" />
+			<parent link="${parent}"/>
+			<child link="${name}_link" />
+			<calibration rising="${sensorring_ref}"/>
+			<axis xyz="0 0 1" />
+			<dynamics damping="5.0" friction="0.5"/>
+			<limit effort="100" lower="-6.2831" upper="6.2831" velocity="1.4"/>
 		</joint>
-		<link name="sensorring_link"/>
+		<link name="${name}_link">
+			<inertial>
+				<origin xyz="0 0 0" rpy="0 0 0"/>
+				<mass value="0.1"/>
+				<inertia ixx="0.01" ixy="0" ixz="0" iyy="0.01" iyz="0" izz="0.01" />
+			</inertial>
+		</link>
+		<!-- extensions -->
+		<xacro:sensorring_gazebo name="${name}" />
+		<xacro:sensorring_transmission name="${name}" />
 	</xacro:macro>
 </robot>

File: cob_description/urdf/torso_cob4/torso.urdf.xacro (robot description, xacro)
@@ -12,5 +12,11 @@
 		  <parent link="${parent}"/>
 		</joint>
-		<link name="torso_base_link"/>
+		<link name="torso_base_link">
+			<inertial>
+				<origin xyz="0 0 0" rpy="0 0 0"/>
+				<mass value="0.1"/>
+				<inertia ixx="0.01" ixy="0" ixz="0" iyy="0.01" iyz="0" izz="0.01" />
+			</inertial>
+		</link>
 		<joint name="torso_1_joint" type="revolute">
 		  <origin xyz="0 0 0.04642" rpy="0 0 0"/>
@@ -22,5 +28,11 @@
 		  <limit effort="100" lower="-6.2831" upper="6.2831" velocity="1.4"/>
 		</joint>
-		<link name="torso_1_link"/>
+		<link name="torso_1_link">
+			<inertial>
+				<origin xyz="0 0 0" rpy="0 0 0"/>
+				<mass value="2"/>
+				<inertia ixx="0.01" ixy="0" ixz="0" iyy="0.01" iyz="0" izz="0.01" />
+			</inertial>
+		</link>
 		<joint name="torso_2_joint" type="revolute">
 		  <origin xyz="0 -0.14734 0.07547" rpy="-0.5236 0 0" />
@@ -32,5 +44,11 @@
 		  <limit effort="100" lower="-6.2831" upper="6.2831" velocity="1.4"/>
 		</joint>
-		<link name="torso_2_link"/>
+		<link name="torso_2_link">
+			<inertial>
+				<origin xyz="0 0 0" rpy="0 0 0"/>
+				<mass value="2"/>
+				<inertia ixx="0.01" ixy="0" ixz="0" iyy="0.01" iyz="0" izz="0.01" />
+			</inertial>
+		</link>
 		<joint name="torso_3_joint" type="revolute">
 		  <origin xyz="0 0.06223 0.15206" rpy="0.5236 0 0" />
@@ -52,6 +70,5 @@
 				<origin xyz="0 0 0" rpy="0 0 0" />
 				<geometry>
-					<!--mesh filename="package://cob_description/meshes/torso_cob4/torso_link.stl"/-->
-					<box size="0.001 0.001 0.001" />
+					<mesh filename="package://cob_description/meshes/torso_cob4/torso_link.stl"/>
 				</geometry>
 				<material name="IPA/LightGrey"/>
