Commit message: cob_description structuration

File: cob_description/urdf/cob3_head/head_v1.gazebo.xacro (robot description, xacro)
@@ -4,10 +4,9 @@
        xmlns:interface="http://playerstage.sourceforge.net/gazebo/xmlschema/#interface"
        xmlns:xacro="http://ros.org/wiki/xacro">
-	<xacro:macro name="ur_connector_transmission" params="name">
-		<transmission name="${name}_trans" type="pr2_mechanism_model/SimpleTransmission">
-			<actuator name="${name}_motor"/>
-			<joint name="${name}_joint"/>
-			<mechanicalReduction>1</mechanicalReduction>
-		</transmission>
+	<xacro:macro name="head_gazebo" params="name">
+		<gazebo reference="${name}_axis_link">
+			<material>IPA/LightGrey</material>
+			<turnGravityOff>false</turnGravityOff>
+		</gazebo>
 	</xacro:macro>
 </robot>

File: cob_description/urdf/cob3_head/head_v1.transmission.xacro (robot description, xacro)
@@ -4,8 +4,8 @@
        xmlns:interface="http://playerstage.sourceforge.net/gazebo/xmlschema/#interface"
        xmlns:xacro="http://ros.org/wiki/xacro">
-	<xacro:macro name="ur_connector_transmission" params="name">
-		<transmission name="${name}_trans" type="pr2_mechanism_model/SimpleTransmission">
-			<actuator name="${name}_motor"/>
-			<joint name="${name}_joint"/>
+	<xacro:macro name="head_transmission" params="name">
+		<transmission name="${name}_axis_trans" type="pr2_mechanism_model/SimpleTransmission">
+			<actuator name="${name}_axis_motor"/>
+			<joint name="${name}_axis_joint"/>
 			<mechanicalReduction>1</mechanicalReduction>
 		</transmission>

File: cob_description/urdf/cob3_head/head_v3.gazebo.xacro (robot description, xacro)
@@ -4,10 +4,9 @@
        xmlns:interface="http://playerstage.sourceforge.net/gazebo/xmlschema/#interface"
        xmlns:xacro="http://ros.org/wiki/xacro">
-	<xacro:macro name="ur_connector_transmission" params="name">
-		<transmission name="${name}_trans" type="pr2_mechanism_model/SimpleTransmission">
-			<actuator name="${name}_motor"/>
-			<joint name="${name}_joint"/>
-			<mechanicalReduction>1</mechanicalReduction>
-		</transmission>
+	<xacro:macro name="head_gazebo" params="name">
+		<gazebo reference="${name}_axis_link">
+			<material>IPA/Black</material>
+			<turnGravityOff>false</turnGravityOff>
+		</gazebo>
 	</xacro:macro>
 </robot>

File: cob_description/urdf/cob3_tray/tray.gazebo.xacro (robot description, xacro)
@@ -4,10 +4,9 @@
        xmlns:interface="http://playerstage.sourceforge.net/gazebo/xmlschema/#interface"
        xmlns:xacro="http://ros.org/wiki/xacro">
-	<xacro:macro name="ur_connector_transmission" params="name">
-		<transmission name="${name}_trans" type="pr2_mechanism_model/SimpleTransmission">
-			<actuator name="${name}_motor"/>
-			<joint name="${name}_joint"/>
-			<mechanicalReduction>1</mechanicalReduction>
-		</transmission>
+	<xacro:macro name="tray_gazebo" params="name">
+		<gazebo reference="${name}_link">
+			<material>IPA/DarkGrey</material>
+			<turnGravityOff>false</turnGravityOff>
+		</gazebo>
 	</xacro:macro>
 </robot>

File: cob_description/urdf/cob3_tray/tray.transmission.xacro (robot description, xacro)
@@ -4,5 +4,5 @@
        xmlns:interface="http://playerstage.sourceforge.net/gazebo/xmlschema/#interface"
        xmlns:xacro="http://ros.org/wiki/xacro">
-	<xacro:macro name="ur_connector_transmission" params="name">
+	<xacro:macro name="tray_transmission" params="name">
 		<transmission name="${name}_trans" type="pr2_mechanism_model/SimpleTransmission">
 			<actuator name="${name}_motor"/>

File: cob_description/urdf/cob3_tray/tray_3DOF.gazebo.xacro (robot description, xacro)
@@ -4,10 +4,14 @@
        xmlns:interface="http://playerstage.sourceforge.net/gazebo/xmlschema/#interface"
        xmlns:xacro="http://ros.org/wiki/xacro">
-	<xacro:macro name="ur_connector_gazebo" params="name">
-		<gazebo reference="${name}_fixed_link">
+	<xacro:macro name="tray_gazebo" params="name">
+		<gazebo reference="${name}_1_link">
 			<material>IPA/DarkGrey</material>
 			<turnGravityOff>false</turnGravityOff>
 		</gazebo>
-		<gazebo reference="${name}_link">
+		<gazebo reference="${name}_2_link">
+			<material>IPA/DarkGrey</material>
+			<turnGravityOff>false</turnGravityOff>
+		</gazebo>
+		<gazebo reference="${name}_3_link">
 			<material>IPA/DarkGrey</material>
 			<turnGravityOff>false</turnGravityOff>

File: cob_description/urdf/cob3_tray/tray_3DOF.transmission.xacro (robot description, xacro)
@@ -4,5 +4,5 @@
        xmlns:interface="http://playerstage.sourceforge.net/gazebo/xmlschema/#interface"
        xmlns:xacro="http://ros.org/wiki/xacro">
-	<xacro:macro name="lbr_transmission" params="name">
+	<xacro:macro name="tray_transmission" params="name">
 		<transmission name="${name}_1_trans" type="pr2_mechanism_model/SimpleTransmission">
 			<actuator name="${name}_1_motor"/>
@@ -20,24 +20,4 @@
 			<mechanicalReduction>1</mechanicalReduction>
 		</transmission>
-		<transmission name="${name}_4_trans" type="pr2_mechanism_model/SimpleTransmission">
-			<actuator name="${name}_4_motor"/>
-			<joint name="${name}_4_joint"/>
-			<mechanicalReduction>1</mechanicalReduction>
-		</transmission>
-		<transmission name="${name}_5_trans" type="pr2_mechanism_model/SimpleTransmission">
-			<actuator name="${name}_5_motor"/>
-			<joint name="${name}_5_joint"/>
-			<mechanicalReduction>1</mechanicalReduction>
-		</transmission>
-		<transmission name="${name}_6_trans" type="pr2_mechanism_model/SimpleTransmission">
-			<actuator name="${name}_6_motor"/>
-			<joint name="${name}_6_joint"/>
-			<mechanicalReduction>1</mechanicalReduction>
-		</transmission>
-		<transmission name="${name}_7_trans" type="pr2_mechanism_model/SimpleTransmission">
-			<actuator name="${name}_7_motor"/>
-			<joint name="${name}_7_joint"/>
-			<mechanicalReduction>1</mechanicalReduction>
-		</transmission>
 	</xacro:macro>
 </robot>

File: cob_description/urdf/cob4_head/head.transmission.xacro (robot description, xacro)
@@ -4,5 +4,5 @@
        xmlns:interface="http://playerstage.sourceforge.net/gazebo/xmlschema/#interface"
        xmlns:xacro="http://ros.org/wiki/xacro">
-	<xacro:macro name="lbr_transmission" params="name">
+	<xacro:macro name="head_transmission" params="name">
 		<transmission name="${name}_1_trans" type="pr2_mechanism_model/SimpleTransmission">
 			<actuator name="${name}_1_motor"/>
@@ -20,24 +20,4 @@
 			<mechanicalReduction>1</mechanicalReduction>
 		</transmission>
-		<transmission name="${name}_4_trans" type="pr2_mechanism_model/SimpleTransmission">
-			<actuator name="${name}_4_motor"/>
-			<joint name="${name}_4_joint"/>
-			<mechanicalReduction>1</mechanicalReduction>
-		</transmission>
-		<transmission name="${name}_5_trans" type="pr2_mechanism_model/SimpleTransmission">
-			<actuator name="${name}_5_motor"/>
-			<joint name="${name}_5_joint"/>
-			<mechanicalReduction>1</mechanicalReduction>
-		</transmission>
-		<transmission name="${name}_6_trans" type="pr2_mechanism_model/SimpleTransmission">
-			<actuator name="${name}_6_motor"/>
-			<joint name="${name}_6_joint"/>
-			<mechanicalReduction>1</mechanicalReduction>
-		</transmission>
-		<transmission name="${name}_7_trans" type="pr2_mechanism_model/SimpleTransmission">
-			<actuator name="${name}_7_motor"/>
-			<joint name="${name}_7_joint"/>
-			<mechanicalReduction>1</mechanicalReduction>
-		</transmission>
 	</xacro:macro>
 </robot>

File: cob_description/urdf/cob4_torso/torso.transmission.xacro (robot description, xacro)
@@ -4,5 +4,5 @@
        xmlns:interface="http://playerstage.sourceforge.net/gazebo/xmlschema/#interface"
        xmlns:xacro="http://ros.org/wiki/xacro">
-	<xacro:macro name="lbr_transmission" params="name">
+	<xacro:macro name="torso_transmission" params="name">
 		<transmission name="${name}_1_trans" type="pr2_mechanism_model/SimpleTransmission">
 			<actuator name="${name}_1_motor"/>
@@ -20,24 +20,4 @@
 			<mechanicalReduction>1</mechanicalReduction>
 		</transmission>
-		<transmission name="${name}_4_trans" type="pr2_mechanism_model/SimpleTransmission">
-			<actuator name="${name}_4_motor"/>
-			<joint name="${name}_4_joint"/>
-			<mechanicalReduction>1</mechanicalReduction>
-		</transmission>
-		<transmission name="${name}_5_trans" type="pr2_mechanism_model/SimpleTransmission">
-			<actuator name="${name}_5_motor"/>
-			<joint name="${name}_5_joint"/>
-			<mechanicalReduction>1</mechanicalReduction>
-		</transmission>
-		<transmission name="${name}_6_trans" type="pr2_mechanism_model/SimpleTransmission">
-			<actuator name="${name}_6_motor"/>
-			<joint name="${name}_6_joint"/>
-			<mechanicalReduction>1</mechanicalReduction>
-		</transmission>
-		<transmission name="${name}_7_trans" type="pr2_mechanism_model/SimpleTransmission">
-			<actuator name="${name}_7_motor"/>
-			<joint name="${name}_7_joint"/>
-			<mechanicalReduction>1</mechanicalReduction>
-		</transmission>
 	</xacro:macro>
 </robot>

File: cob_description/urdf/lbr/lbr.gazebo.xacro (robot description, xacro)
@@ -4,5 +4,5 @@
        xmlns:interface="http://playerstage.sourceforge.net/gazebo/xmlschema/#interface"
        xmlns:xacro="http://ros.org/wiki/xacro">
-	<xacro:macro name="cob_lbr_gazebo" params="name">
+	<xacro:macro name="lbr_gazebo" params="name">
 		<gazebo reference="${name}_0_link">
 			<material value="IPA/Orange" />

File: cob_description/urdf/lbr/lbr.urdf.xacro (robot description, xacro)
@@ -6,5 +6,5 @@
 	<include filename="$(find cob_description)/urdf/lbr/lbr.gazebo.xacro" />
 	<include filename="$(find cob_description)/urdf/lbr/lbr.transmission.xacro" />
-	<xacro:macro name="cob_lbr" params="parent name *origin">
+	<xacro:macro name="lbr" params="parent name *origin">
 		<!-- joint between base_link and arm_0_link -->
 		<joint name="${name}_0_joint" type="fixed" >
@@ -251,6 +251,6 @@
 		</link>
 		<!-- extensions -->
-		<xacro:cob_lbr_gazebo name="${name}" />
-		<xacro:cob_lbr_transmission name="${name}" />
+		<xacro:lbr_gazebo name="${name}" />
+		<xacro:lbr_transmission name="${name}" />
 	</xacro:macro>
 </robot>

File: cob_description/urdf/ur_arm/ur5_arm.urdf.xacro (robot description, xacro)
@@ -5,5 +5,5 @@
        xmlns:xacro="http://ros.org/wiki/xacro">
 	<include filename="$(find ur_description)/urdf/ur5.urdf.xacro" />
-	<xacro:macro name="cob_ur5" params="parent name *origin">
+	<xacro:macro name="ur5" params="parent name *origin">
 		<!-- mount the arm to the robot -->
 		<joint name="${name}_base_joint" type="fixed" >

File: cob_description/urdf/ur_connector/ur_connector.urdf.xacro (robot description, xacro)
@@ -6,5 +6,5 @@
 	<include filename="$(find cob_description)/urdf/ur_connector/ur_connector.gazebo.xacro" />
 	<include filename="$(find cob_description)/urdf/ur_connector/ur_connector.transmission.xacro" />
-	<xacro:macro name="cob_ur_connector" params="name parent *origin">
+	<xacro:macro name="ur_connector" params="name parent *origin">
 		<!-- joint between base_link and ur_connector_link -->
 		<joint name="${name}_fixed_joint" type="fixed">
@@ -64,6 +64,6 @@
 		</link>
 		<!-- extensions -->
-		<xacro:cob_ur_connector_gazebo name="${name}" />
-		<xacro:cob_ur_connector_transmission name="${name}" />
+		<xacro:ur_connector_gazebo name="${name}" />
+		<xacro:ur_connector_transmission name="${name}" />
 	</xacro:macro>
 </robot>
