Commit message: New head model for cob3-8

File: cob_description/urdf/cob3_head/head_v1.urdf.xacro (robot description, xacro)
@@ -8,20 +8,20 @@
   <xacro:macro name="head" params="name parent *origin">
     <!-- joint between torso_upper_neck_tilt_link and head_base_link -->
-        <joint name="${name}_base_joint" type="fixed">
-      <insert_block name="origin" />
-      <parent link="${parent}"/>
-            <child link="${name}_base_link"/>
+    <joint name="${name}_base_joint" type="fixed">
+        <insert_block name="origin" />
+        <parent link="${parent}"/>
+        <child link="${name}_base_link"/>
     </joint>
-        <link name="${name}_base_link">
-            <inertial>
-                <origin xyz="0 0 0" rpy="0 0 0"/>
-                <mass value="0.5"/>
-                <inertia ixx="0.01" ixy="0" ixz="0" iyy="0.01" iyz="0" izz="0.01" />
-            </inertial>
+    <link name="${name}_base_link">
+      <inertial>
+        <origin xyz="0 0 0" rpy="0 0 0"/>
+        <mass value="0.5"/>
+        <inertia ixx="0.01" ixy="0" ixz="0" iyy="0.01" iyz="0" izz="0.01" />
+      </inertial>
     </link>
     <!-- joint between torso_upper_neck_tilt_link and head_axis_link -->
     <joint name="${name}_axis_joint" type="revolute">
       <origin xyz="0 0 0" rpy="0 0 0" />
-            <parent link="${name}_base_link"/>
+      <parent link="${name}_base_link"/>
       <child link="${name}_axis_link"/>
       <axis xyz="0 0 1" />
@@ -50,11 +50,11 @@
       </collision>
     </link>
-        <!--camera reference link-->
-        <joint name="${name}_cam_reference_joint" type="fixed">
-      <origin xyz="${cam_reference_x} ${cam_reference_y} ${cam_reference_z}" rpy="${cam_reference_roll} ${cam_reference_pitch} ${cam_reference_yaw}" />
-            <parent link="${name}_axis_link"/>
-            <child link="${name}_cam_reference_link"/>
+    <!--camera reference link-->
+    <joint name="${name}_cam_reference_joint" type="fixed">
+        <origin xyz="${cam_reference_x} ${cam_reference_y} ${cam_reference_z}" rpy="${cam_reference_roll} ${cam_reference_pitch} ${cam_reference_yaw}" />
+        <parent link="${name}_axis_link"/>
+        <child link="${name}_cam_reference_link"/>
     </joint>
-        <link name="${name}_cam_reference_link">
+    <link name="${name}_cam_reference_link">
       <inertial>
         <origin xyz="0 0 0" rpy="0 0 0"/>
@@ -64,13 +64,13 @@
     </link>
     <!-- left camera -->
-        <xacro:cob_prosilica_v0 name="${name}_color_camera_l" ros_topic="stereo/left" parent="${name}_cam_reference_link">
+    <xacro:cob_prosilica_v0 name="${name}_color_camera_l" ros_topic="stereo/left" parent="${name}_cam_reference_link">
       <origin xyz="${cam_l_x} ${cam_l_y} ${cam_l_z}" rpy="${cam_l_roll} ${cam_l_pitch} ${cam_l_yaw}" />
     </xacro:cob_prosilica_v0>
     <!-- right camera -->
-        <xacro:cob_prosilica_v0 name="${name}_color_camera_r" ros_topic="stereo/right" parent="${name}_cam_reference_link">
+    <xacro:cob_prosilica_v0 name="${name}_color_camera_r" ros_topic="stereo/right" parent="${name}_cam_reference_link">
       <origin xyz="${cam_r_x} ${cam_r_y} ${cam_r_z}" rpy="${cam_r_roll} ${cam_r_pitch} ${cam_r_yaw}" />
     </xacro:cob_prosilica_v0>
     <!-- cam3d -->
-        <xacro:cob_kinect_v0 name="${name}_cam3d" ros_topic="cam3d" parent="${name}_cam_reference_link">
+    <xacro:cob_kinect_v0 name="${name}_cam3d" ros_topic="cam3d" parent="${name}_cam_reference_link">
       <origin xyz="${cam3d_x} ${cam3d_y} ${cam3d_z}" rpy="${cam3d_roll} ${cam3d_pitch} ${cam3d_yaw}" />
     </xacro:cob_kinect_v0>

File: cob_description/urdf/cob3_head/head_v2.urdf.xacro (robot description, xacro)
@@ -7,15 +7,15 @@
   <xacro:macro name="head" params="name parent *origin">
     <!-- joint between torso_upper_neck_tilt_link and head_base_link -->
-        <joint name="${name}_base_joint" type="fixed">
+    <joint name="${name}_base_joint" type="fixed">
       <insert_block name="origin" />
       <parent link="${parent}"/>
-            <child link="${name}_base_link"/>
+      <child link="${name}_base_link"/>
     </joint>
-        <link name="${name}_base_link">
-            <inertial>
-                <origin xyz="0 0 0" rpy="0 0 0"/>
-                <mass value="0.5"/>
-                <inertia ixx="0.01" ixy="0" ixz="0" iyy="0.01" iyz="0" izz="0.01" />
-            </inertial>
+    <link name="${name}_base_link">
+      <inertial>
+        <origin xyz="0 0 0" rpy="0 0 0"/>
+        <mass value="0.5"/>
+        <inertia ixx="0.01" ixy="0" ixz="0" iyy="0.01" iyz="0" izz="0.01" />
+      </inertial>
     </link>
     <!-- joint between torso_upper_neck_tilt_link and head_axis_link -->
@@ -49,11 +49,11 @@
       </collision>
     </link>
-        <!--reference joint for cameras-->
-        <joint name="${name}_cam_reference_joint" type="fixed">
-      <origin xyz="${cam_reference_x} ${cam_reference_y} ${cam_reference_z}" rpy="${cam_reference_roll} ${cam_reference_pitch} ${cam_reference_yaw}" />
-            <parent link="${name}_axis_link"/>
-            <child link="${name}_cam_reference_link"/>
+    <!--reference joint for cameras-->
+    <joint name="${name}_cam_reference_joint" type="fixed">
+        <origin xyz="${cam_reference_x} ${cam_reference_y} ${cam_reference_z}" rpy="${cam_reference_roll} ${cam_reference_pitch} ${cam_reference_yaw}" />
+        <parent link="${name}_axis_link"/>
+        <child link="${name}_cam_reference_link"/>
     </joint>
-        <link name="${name}_cam_reference_link">
+    <link name="${name}_cam_reference_link">
       <inertial>
         <origin xyz="0 0 0" rpy="0 0 0"/>
@@ -63,16 +63,16 @@
     </link>
     <!-- left camera -->
-        <xacro:cob_prosilica_v0 name="${name}_color_camera_l" ros_topic="stereo/left" parent="${name}_cam_reference_link">
+    <xacro:cob_prosilica_v0 name="${name}_color_camera_l" ros_topic="stereo/left" parent="${name}_cam_reference_link">
       <origin xyz="${cam_l_x} ${cam_l_y} ${cam_l_z}" rpy="${cam_l_roll} ${cam_l_pitch} ${cam_l_yaw}" />
     </xacro:cob_prosilica_v0>
     <!-- right camera -->
-        <xacro:cob_prosilica_v0 name="${name}_color_camera_r" ros_topic="stereo/right" parent="${name}_cam_reference_link">
+    <xacro:cob_prosilica_v0 name="${name}_color_camera_r" ros_topic="stereo/right" parent="${name}_cam_reference_link">
       <origin xyz="${cam_r_x} ${cam_r_y} ${cam_r_z}" rpy="${cam_r_roll} ${cam_r_pitch} ${cam_r_yaw}" />
     </xacro:cob_prosilica_v0>
     <!-- cam3d -->
-        <xacro:cob_kinect_v0 name="${name}_cam3d" ros_topic="cam3d" parent="${name}_cam_reference_link">
+    <xacro:cob_kinect_v0 name="${name}_cam3d" ros_topic="cam3d" parent="${name}_cam_reference_link">
       <origin xyz="${cam3d_x} ${cam3d_y} ${cam3d_z}" rpy="${cam3d_roll} ${cam3d_pitch} ${cam3d_yaw}" />
     </xacro:cob_kinect_v0>
-        <!-- extensions -->
+    <!-- extensions -->
     <xacro:head_gazebo name="${name}" />
     <xacro:head_transmission name="${name}" />

File: cob_description/urdf/cob3_head/head_v4.urdf.xacro (robot description, xacro)
@@ -1,7 +1,6 @@
 <?xml version="1.0"?>
 <robot xmlns:xacro="http://www.ros.org/wiki/xacro">
-  <xacro:include filename="$(find cob_description)/urdf/cob3_head/head_v3.gazebo.xacro" />
-  <xacro:include filename="$(find cob_description)/urdf/cob3_head/head_v3.transmission.xacro" />
-  <xacro:include filename="$(find cob_description)/urdf/sensors/prosilica.urdf.xacro" />
+  <xacro:include filename="$(find cob_description)/urdf/cob3_head/head_v4.gazebo.xacro" />
+  <xacro:include filename="$(find cob_description)/urdf/cob3_head/head_v4.transmission.xacro" />
   <xacro:include filename="$(find cob_description)/urdf/sensors/kinect.urdf.xacro" />
   <xacro:macro name="head" params="name parent *origin">
@@ -62,12 +61,4 @@
       </inertial>
     </link>
-    <!-- left camera -->
-    <xacro:cob_prosilica_v0 name="${name}_color_camera_l" ros_topic="stereo/left" parent="${name}_cam_reference_link">
-      <origin xyz="${cam_l_x} ${cam_l_y} ${cam_l_z}" rpy="${cam_l_roll} ${cam_l_pitch} ${cam_l_yaw}" />
-    </xacro:cob_prosilica_v0>
-    <!-- right camera -->
-    <xacro:cob_prosilica_v0 name="${name}_color_camera_r" ros_topic="stereo/right" parent="${name}_cam_reference_link">
-      <origin xyz="${cam_r_x} ${cam_r_y} ${cam_r_z}" rpy="${cam_r_roll} ${cam_r_pitch} ${cam_r_yaw}" />
-    </xacro:cob_prosilica_v0>
     <!-- cam3d -->
     <xacro:cob_kinect_v0 name="${name}_cam3d" ros_topic="cam3d" parent="${name}_cam_reference_link">
