Commit message: consitency changes due to new transmission format

File: cob_description/urdf/cob3_head/head.transmission.xacro (robot description, xacro)
@@ -8,5 +8,4 @@
       </joint>
       <actuator name="${name}_axis_motor">
-        <hardwareInterface>EffortJointInterface</hardwareInterface>
         <mechanicalReduction>1</mechanicalReduction>
       </actuator>

File: cob_description/urdf/cob3_torso/torso_v1.transmission.xacro (robot description, xacro)
@@ -8,5 +8,4 @@
       </joint>
       <actuator name="${name}_lower_neck_pan_motor">
-        <hardwareInterface>EffortJointInterface</hardwareInterface>
         <mechanicalReduction>1</mechanicalReduction>
       </actuator>
@@ -18,5 +17,4 @@
       </joint>
       <actuator name="${name}_lower_neck_tilt_motor">
-        <hardwareInterface>EffortJointInterface</hardwareInterface>
         <mechanicalReduction>1</mechanicalReduction>
       </actuator>
@@ -28,5 +26,4 @@
       </joint>
       <actuator name="${name}_upper_neck_pan_motor">
-        <hardwareInterface>EffortJointInterface</hardwareInterface>
         <mechanicalReduction>1</mechanicalReduction>
       </actuator>
@@ -38,5 +35,4 @@
       </joint>
       <actuator name="${name}_upper_neck_tilt_motor">
-        <hardwareInterface>EffortJointInterface</hardwareInterface>
         <mechanicalReduction>1</mechanicalReduction>
       </actuator>

File: cob_description/urdf/cob3_torso/torso_v2.transmission.xacro (robot description, xacro)
@@ -8,5 +8,4 @@
       </joint>
       <actuator name="${name}_lower_neck_tilt_motor">
-        <hardwareInterface>EffortJointInterface</hardwareInterface>
         <mechanicalReduction>1</mechanicalReduction>
       </actuator>
@@ -18,5 +17,4 @@
       </joint>
       <actuator name="${name}_pan_motor">
-        <hardwareInterface>EffortJointInterface</hardwareInterface>
         <mechanicalReduction>1</mechanicalReduction>
       </actuator>
@@ -28,5 +26,4 @@
       </joint>
       <actuator name="${name}_upper_neck_tilt_motor">
-        <hardwareInterface>EffortJointInterface</hardwareInterface>
         <mechanicalReduction>1</mechanicalReduction>
       </actuator>

File: cob_description/urdf/cob3_tray/tray.transmission.xacro (robot description, xacro)
@@ -8,5 +8,4 @@
       </joint>
       <actuator name="${name}_motor">
-        <hardwareInterface>EffortJointInterface</hardwareInterface>
         <mechanicalReduction>1</mechanicalReduction>
       </actuator>

File: cob_description/urdf/cob3_tray/tray_3DOF.transmission.xacro (robot description, xacro)
@@ -8,5 +8,4 @@
       </joint>
       <actuator name="${name}_1_motor">
-        <hardwareInterface>EffortJointInterface</hardwareInterface>
         <mechanicalReduction>1</mechanicalReduction>
       </actuator>
@@ -18,5 +17,4 @@
       </joint>
       <actuator name="${name}_2_motor">
-        <hardwareInterface>EffortJointInterface</hardwareInterface>
         <mechanicalReduction>1</mechanicalReduction>
       </actuator>
@@ -28,5 +26,4 @@
       </joint>
       <actuator name="${name}_3_motor">
-        <hardwareInterface>EffortJointInterface</hardwareInterface>
         <mechanicalReduction>1</mechanicalReduction>
       </actuator>

File: cob_description/urdf/cob4_base/base.transmission.xacro (robot description, xacro)
@@ -5,7 +5,8 @@
     <transmission name="${parent}_${suffix}_wheel_trans">
       <type>transmission_interface/SimpleTransmission</type>
-      <joint name="${parent}_${suffix}_wheel_joint" />
+      <joint name="${parent}_${suffix}_wheel_joint" >
+        <hardwareInterface>EffortJointInterface</hardwareInterface>
+      </joint>
       <actuator name="${parent}_${suffix}_wheel_motor">
-        <hardwareInterface>EffortJointInterface</hardwareInterface>
         <mechanicalReduction>${reflect * 624/35 * 80/18}</mechanicalReduction>
       </actuator>
@@ -16,7 +17,8 @@
     <transmission name="${suffix}_rotation_trans">
       <type>transmission_interface/SimpleTransmission</type>
-      <joint name="${suffix}_rotation_joint" />
+      <joint name="${suffix}_rotation_joint" >
+        <hardwareInterface>EffortJointInterface</hardwareInterface>
+      </joint>
       <actuator name="${suffix}_rotation_motor" >
-       <hardwareInterface>EffortJointInterface</hardwareInterface>
         <mechanicalReduction>${-1 * 624/35 * 80/18}</mechanicalReduction>
       </actuator>

File: cob_description/urdf/cob4_head/head.transmission.xacro (robot description, xacro)
@@ -8,5 +8,4 @@
       </joint>
       <actuator name="${name}_1_motor">
-        <hardwareInterface>EffortJointInterface</hardwareInterface>
         <mechanicalReduction>1</mechanicalReduction>
       </actuator>
@@ -18,5 +17,4 @@
       </joint>
       <actuator name="${name}_2_motor">
-        <hardwareInterface>EffortJointInterface</hardwareInterface>
         <mechanicalReduction>1</mechanicalReduction>
       </actuator>
@@ -28,5 +26,4 @@
       </joint>
       <actuator name="${name}_3_motor">
-        <hardwareInterface>EffortJointInterface</hardwareInterface>
         <mechanicalReduction>1</mechanicalReduction>
       </actuator>

File: cob_description/urdf/cob4_sensorring/sensorring.transmission.xacro (robot description, xacro)
@@ -8,5 +8,4 @@
       </joint>
       <actuator name="${name}_motor">
-        <hardwareInterface>EffortJointInterface</hardwareInterface>
         <mechanicalReduction>1</mechanicalReduction>
       </actuator>

File: cob_description/urdf/cob4_torso/torso.transmission.xacro (robot description, xacro)
@@ -8,5 +8,4 @@
       </joint>
       <actuator name="${name}_1_motor">
-        <hardwareInterface>EffortJointInterface</hardwareInterface>
         <mechanicalReduction>1</mechanicalReduction>
       </actuator>
@@ -18,5 +17,4 @@
       </joint>
       <actuator name="${name}_2_motor">
-        <hardwareInterface>EffortJointInterface</hardwareInterface>
         <mechanicalReduction>1</mechanicalReduction>
       </actuator>
@@ -28,5 +26,4 @@
       </joint>
       <actuator name="${name}_3_motor">
-        <hardwareInterface>EffortJointInterface</hardwareInterface>
         <mechanicalReduction>1</mechanicalReduction>
       </actuator>

File: cob_description/urdf/lbr/lbr.transmission.xacro (robot description, xacro)
@@ -8,5 +8,4 @@
       </joint>
       <actuator name="${name}_1_motor">
-        <hardwareInterface>EffortJointInterface</hardwareInterface>
         <mechanicalReduction>1</mechanicalReduction>
       </actuator>
@@ -18,5 +17,4 @@
       </joint>
       <actuator name="${name}_2_motor">
-        <hardwareInterface>EffortJointInterface</hardwareInterface>
         <mechanicalReduction>1</mechanicalReduction>
       </actuator>
@@ -28,5 +26,4 @@
       </joint>
       <actuator name="${name}_3_motor">
-        <hardwareInterface>EffortJointInterface</hardwareInterface>
         <mechanicalReduction>1</mechanicalReduction>
       </actuator>
@@ -38,5 +35,4 @@
       </joint>
       <actuator name="${name}_4_motor">
-        <hardwareInterface>EffortJointInterface</hardwareInterface>
         <mechanicalReduction>1</mechanicalReduction>
       </actuator>
@@ -48,5 +44,4 @@
       </joint>
       <actuator name="${name}_5_motor">
-        <hardwareInterface>EffortJointInterface</hardwareInterface>
         <mechanicalReduction>1</mechanicalReduction>
       </actuator>
@@ -58,5 +53,4 @@
       </joint>
       <actuator name="${name}_6_motor">
-        <hardwareInterface>EffortJointInterface</hardwareInterface>
         <mechanicalReduction>1</mechanicalReduction>
       </actuator>
@@ -68,5 +62,4 @@
       </joint>
       <actuator name="${name}_7_motor">
-        <hardwareInterface>EffortJointInterface</hardwareInterface>
         <mechanicalReduction>1</mechanicalReduction>
       </actuator>

File: cob_description/urdf/ur_connector/ur_connector.transmission.xacro (robot description, xacro)
@@ -8,5 +8,4 @@
       </joint>
       <actuator name="${name}_motor">
-        <hardwareInterface>EffortJointInterface</hardwareInterface>
         <mechanicalReduction>1</mechanicalReduction>
       </actuator>

File: desire_description/urdf/base_desire/base.transmission.xacro (robot description, xacro)
@@ -9,5 +9,4 @@
       </joint>
       <actuator name="${parent}_${suffix}_wheel_motor">
-        <hardwareInterface>EffortJointInterface</hardwareInterface>
         <mechanicalReduction>${reflect * 624/35 * 80/18}</mechanicalReduction>
       </actuator>
@@ -22,5 +21,4 @@
       </joint>
       <actuator name="${suffix}_rotation_motor">
-        <hardwareInterface>EffortJointInterface</hardwareInterface>
         <mechanicalReduction>${-1 * 624/35 * 80/18}</mechanicalReduction>
       </actuator>

File: desire_description/urdf/head_desire/head.transmission.xacro (robot description, xacro)
@@ -8,5 +8,4 @@
       </joint>
       <actuator name="${name}_pan_motor">
-        <hardwareInterface>EffortJointInterface</hardwareInterface>
         <mechanicalReduction>1</mechanicalReduction>
       </actuator>
@@ -18,5 +17,4 @@
       </joint>
       <actuator name="${name}_tilt_motor">
-        <hardwareInterface>EffortJointInterface</hardwareInterface>
         <mechanicalReduction>1</mechanicalReduction>
       </actuator>

File: raw_description/urdf/base_long/base.transmission.xacro (robot description, xacro)
@@ -9,5 +9,4 @@
       </joint>
       <actuator name="${parent}_${suffix}_wheel_motor">
-        <hardwareInterface>EffortJointInterface</hardwareInterface>
         <mechanicalReduction>${reflect * 624/35 * 80/18}</mechanicalReduction>
       </actuator>
@@ -22,5 +21,4 @@
       </joint>
       <actuator name="${suffix}_rotation_motor">
-        <hardwareInterface>EffortJointInterface</hardwareInterface>
         <mechanicalReduction>${-1 * 624/35 * 80/18}</mechanicalReduction>
       </actuator>

File: raw_description/urdf/base_short/base.transmission.xacro (robot description, xacro)
@@ -9,5 +9,4 @@
       </joint>
       <actuator name="${parent}_${suffix}_wheel_motor">
-        <hardwareInterface>EffortJointInterface</hardwareInterface>
         <mechanicalReduction>${reflect * 624/35 * 80/18}</mechanicalReduction>
       </actuator>
@@ -22,5 +21,4 @@
       </joint>
       <actuator name="${suffix}_rotation_motor" >
-       <hardwareInterface>EffortJointInterface</hardwareInterface>
         <mechanicalReduction>${-1 * 624/35 * 80/18}</mechanicalReduction>
       </actuator>

File: raw_description/urdf/torso/torso.transmission.xacro (robot description, xacro)
@@ -8,5 +8,4 @@
       </joint>
       <actuator name="${name}_pan_motor">
-        <hardwareInterface>EffortJointInterface</hardwareInterface>
         <mechanicalReduction>1</mechanicalReduction>
       </actuator>
@@ -18,5 +17,4 @@
       </joint>
       <actuator name="${name}_tilt_motor">
-        <hardwareInterface>EffortJointInterface</hardwareInterface>
         <mechanicalReduction>1</mechanicalReduction>
       </actuator>
