Commit message: allow cob3 components to be used with PositionJointInterface

File: cob_description/urdf/cob3_head/head_kinect.urdf.xacro (robot description, xacro)
@@ -12,14 +12,22 @@
     </joint>
     <link name="${name}_base_link">
-      <inertial>
-        <origin xyz="0 0 0" rpy="0 0 0"/>
-        <mass value="0.5"/>
-        <inertia ixx="0.01" ixy="0" ixz="0" iyy="0.01" iyz="0" izz="0.01" />
-      </inertial>
+      <xacro:default_inertial/>
+      <visual>
+        <origin xyz="0 0 0" rpy="0 0 0" />
+        <geometry>
+          <box size="0.001 0.001 0.001" />
+        </geometry>
+      </visual>
+      <collision>
+        <origin xyz="0 0 0" rpy="0 0 0" />
+        <geometry>
+          <box size="0.001 0.001 0.001" />
+        </geometry>
+      </collision>
     </link>
     <!-- joint between head_base_link and head_axis_link -->
     <joint name="${name}_axis_joint" type="revolute">
+      <origin xyz="0 0 0" rpy="0 0 0" />
       <parent link="${name}_base_link"/>
-      <origin xyz="0 0 0" rpy="0 0 0" />
       <child link="${name}_axis_link"/>
       <axis xyz="0 0 1" />
@@ -29,20 +37,15 @@
     </joint>
     <link name="${name}_axis_link">
-      <inertial>
-        <origin xyz="0 0 0" rpy="0 0 0"/>
-        <mass value="0.1"/>
-        <inertia ixx="0.0001" ixy="0" ixz="0" iyy="0.0001" iyz="0" izz="0.0001" />
-      </inertial>
+      <xacro:default_inertial/>
       <visual>
         <origin xyz="0 0 0" rpy="0 0 0" />
         <geometry>
-          <box size="0.01 0.01 0.01"/>
+          <box size="0.001 0.001 0.001" />
         </geometry>
-        <material name="IPA/Black" />
       </visual>
       <collision>
         <origin xyz="0 0 0" rpy="0 0 0" />
         <geometry>
-          <box size="0.01 0.01 0.01"/>
+          <box size="0.001 0.001 0.001" />
         </geometry>
       </collision>
@@ -55,9 +58,17 @@
     </joint>
     <link name="${name}_cam_reference_link">
-      <inertial>
-        <origin xyz="0 0 0" rpy="0 0 0"/>
-        <mass value="0.5"/>
-        <inertia ixx="0.01" ixy="0" ixz="0" iyy="0.01" iyz="0" izz="0.01" />
-      </inertial>
+      <xacro:default_inertial/>
+      <visual>
+        <origin xyz="0 0 0" rpy="0 0 0" />
+        <geometry>
+          <box size="0.001 0.001 0.001" />
+        </geometry>
+      </visual>
+      <collision>
+        <origin xyz="0 0 0" rpy="0 0 0" />
+        <geometry>
+          <box size="0.001 0.001 0.001" />
+        </geometry>
+      </collision>
     </link>
     <!-- cam3d -->

File: cob_description/urdf/cob3_head/head_prosilicas_kinect.urdf.xacro (robot description, xacro)
@@ -13,9 +13,17 @@
     </joint>
     <link name="${name}_base_link">
-      <inertial>
-        <origin xyz="0 0 0" rpy="0 0 0"/>
-        <mass value="0.5"/>
-        <inertia ixx="0.01" ixy="0" ixz="0" iyy="0.01" iyz="0" izz="0.01" />
-      </inertial>
+      <xacro:default_inertial/>
+      <visual>
+        <origin xyz="0 0 0" rpy="0 0 0" />
+        <geometry>
+          <box size="0.001 0.001 0.001" />
+        </geometry>
+      </visual>
+      <collision>
+        <origin xyz="0 0 0" rpy="0 0 0" />
+        <geometry>
+          <box size="0.001 0.001 0.001" />
+        </geometry>
+      </collision>
     </link>
     <!-- joint between torso_upper_neck_tilt_link and head_axis_link -->
@@ -30,20 +38,15 @@
     </joint>
     <link name="${name}_axis_link">
-      <inertial>
-        <origin xyz="0 0 0" rpy="0 0 0"/>
-        <mass value="0.1"/>
-        <inertia ixx="0.0001" ixy="0" ixz="0" iyy="0.0001" iyz="0" izz="0.0001" />
-      </inertial>
+      <xacro:default_inertial/>
       <visual>
         <origin xyz="0 0 0" rpy="0 0 0" />
         <geometry>
-          <box size="0.01 0.01 0.01"/>
+          <box size="0.001 0.001 0.001" />
         </geometry>
-        <material name="IPA/LightGrey" />
       </visual>
       <collision>
         <origin xyz="0 0 0" rpy="0 0 0" />
         <geometry>
-          <box size="0.01 0.01 0.01"/>
+          <box size="0.001 0.001 0.001" />
         </geometry>
       </collision>
@@ -56,9 +59,17 @@
     </joint>
     <link name="${name}_cam_reference_link">
-      <inertial>
-        <origin xyz="0 0 0" rpy="0 0 0"/>
-        <mass value="0.5"/>
-        <inertia ixx="0.01" ixy="0" ixz="0" iyy="0.01" iyz="0" izz="0.01" />
-      </inertial>
+      <xacro:default_inertial/>
+      <visual>
+        <origin xyz="0 0 0" rpy="0 0 0" />
+        <geometry>
+          <box size="0.001 0.001 0.001" />
+        </geometry>
+      </visual>
+      <collision>
+        <origin xyz="0 0 0" rpy="0 0 0" />
+        <geometry>
+          <box size="0.001 0.001 0.001" />
+        </geometry>
+      </collision>
     </link>
     <!-- left camera -->

File: cob_description/urdf/cob3_torso/torso_v1.urdf.xacro (robot description, xacro)
@@ -11,9 +11,17 @@
     </joint>
     <link name="${name}_base_link">
-      <inertial>
-        <origin xyz="0 0 0" rpy="0 0 0"/>
-        <mass value="0.01"/>
-        <inertia ixx="1" ixy="0" ixz="0" iyy="1" iyz="0" izz="1" />
-      </inertial>
+      <xacro:default_inertial/>
+      <visual>
+        <origin xyz="0 0 0" rpy="0 0 0" />
+        <geometry>
+          <box size="0.001 0.001 0.001" />
+        </geometry>
+      </visual>
+      <collision>
+        <origin xyz="0 0 0" rpy="0 0 0" />
+        <geometry>
+          <box size="0.001 0.001 0.001" />
+        </geometry>
+      </collision>
     </link>
     <!-- joint between base_link and torso_lower_neck_pan_link -->
@@ -28,20 +36,20 @@
     </joint>
     <link name="${name}_lower_neck_pan_link">
-      <inertial>
+      <xacro:default_inertial/>
+      <!--inertial>
         <origin xyz="0 0 0" rpy="0 0 0"/>
         <mass value="1.0"/>
         <inertia ixx="0.200549" ixy="0.001322" ixz="-0.000000" iyy="0.123664" iyz="-0.000000" izz="0.104101" />
-      </inertial>
+      </inertial-->
       <visual>
-        <origin xyz="0 0 0.005" rpy="0 0 0" />
+        <origin xyz="0 0 0" rpy="0 0 0" />
         <geometry>
-          <box size="0.01 0.01 0.01"/>
+          <box size="0.001 0.001 0.001" />
         </geometry>
-        <material name="IPA/LightGrey" />
       </visual>
       <collision>
-        <origin xyz="0 0 0.0005" rpy="0 0 0" />
+        <origin xyz="0 0 0" rpy="0 0 0" />
         <geometry>
-          <box size="0.001 0.001 0.001"/>
+          <box size="0.001 0.001 0.001" />
         </geometry>
       </collision>
@@ -58,9 +66,10 @@
     </joint>
     <link name="${name}_lower_neck_tilt_link">
-      <inertial>
+      <xacro:default_inertial/>
+      <!--inertial>
         <origin xyz="0 0 0" rpy="0 0 0"/>
         <mass value="6.209720"/>
         <inertia ixx="0.171118" ixy="0.002544" ixz="-0.000000" iyy="0.083077" iyz="0.000000" izz="0.120948" />
-      </inertial>
+      </inertial-->
       <visual>
         <origin xyz="0 0 0" rpy="0 0 0" />
@@ -88,20 +97,20 @@
     </joint>
     <link name="${name}_upper_neck_pan_link">
-      <inertial>
+      <xacro:default_inertial/>
+      <!--inertial>
         <origin xyz="0 0 0" rpy="0 0 0"/>
         <mass value="1.0"/>
         <inertia ixx="0.01" ixy="0" ixz="0" iyy="0.01" iyz="0" izz="0.01" />
-      </inertial>
+      </inertial-->
       <visual>
-        <origin xyz="0 0 0.005" rpy="0 0 0" />
+        <origin xyz="0 0 0" rpy="0 0 0" />
         <geometry>
-          <box size="0.01 0.01 0.01"/>
+          <box size="0.001 0.001 0.001" />
         </geometry>
-        <material name="IPA/LightGrey" />
       </visual>
       <collision>
-        <origin xyz="0 0 0.0005" rpy="0 0 0" />
+        <origin xyz="0 0 0" rpy="0 0 0" />
         <geometry>
-          <box size="0.001 0.001 0.001"/>
+          <box size="0.001 0.001 0.001" />
         </geometry>
       </collision>
@@ -118,9 +127,10 @@
     </joint>
     <link name="${name}_upper_neck_tilt_link">
-      <inertial>
+      <xacro:default_inertial/>
+      <!--inertial>
         <origin xyz="0 0 0" rpy="0 0 0"/>
         <mass value="6.744238"/>
         <inertia ixx="0.01" ixy="0" ixz="0" iyy="0.01" iyz="0" izz="0.01" />
-      </inertial>
+      </inertial-->
       <visual>
         <origin xyz="0 0 0" rpy="0 0 0" />
@@ -144,9 +154,5 @@
     </joint>
     <link name="head_cover_link">
-      <inertial>
-        <origin xyz="0 0 0" rpy="0 0 0"/>
-        <mass value="0.5"/>
-        <inertia ixx="0.01" ixy="0" ixz="0" iyy="0.01" iyz="0" izz="0.01" />
-      </inertial>
+      <xacro:default_inertial/>
       <visual>
         <origin xyz="0 0 0" rpy="0 0 0" />

File: cob_description/urdf/cob3_torso/torso_v2.urdf.xacro (robot description, xacro)
@@ -11,9 +11,17 @@
     </joint>
     <link name="${name}_base_link">
-      <inertial>
-        <origin xyz="0 0 0" rpy="0 0 0"/>
-        <mass value="0.01"/>
-        <inertia ixx="1" ixy="0" ixz="0" iyy="1" iyz="0" izz="1" />
-      </inertial>
+      <xacro:default_inertial/>
+      <visual>
+        <origin xyz="0 0 0" rpy="0 0 0" />
+        <geometry>
+          <box size="0.001 0.001 0.001" />
+        </geometry>
+      </visual>
+      <collision>
+        <origin xyz="0 0 0" rpy="0 0 0" />
+        <geometry>
+          <box size="0.001 0.001 0.001" />
+        </geometry>
+      </collision>
     </link>
     <!-- joint between base_link and torso_lower_neck_tilt_link -->
@@ -29,9 +37,10 @@
     </joint>
     <link name="${name}_lower_neck_tilt_link">
-      <inertial>
+      <xacro:default_inertial/>
+      <!--inertial>
         <origin xyz="0 0 0" rpy="0 0 0"/>
         <mass value="6.209720"/>
         <inertia ixx="0.171118" ixy="0.002544" ixz="-0.000000" iyy="0.083077" iyz="0.000000" izz="0.120948" />
-      </inertial>
+      </inertial-->
       <visual>
         <origin xyz="0 0 0" rpy="${M_PI} 0 0" />
@@ -60,9 +69,17 @@
     </joint>
     <link name="${name}_pan_link">
-      <inertial>
-        <origin xyz="0 0 0" rpy="0 0 0"/>
-        <mass value="1.0"/>
-        <inertia ixx="0.200549" ixy="0.001322" ixz="-0.000000" iyy="0.123664" iyz="-0.000000" izz="0.104101" />
-      </inertial>
+      <xacro:default_inertial/>
+      <visual>
+        <origin xyz="0 0 0" rpy="0 0 0" />
+        <geometry>
+          <box size="0.001 0.001 0.001" />
+        </geometry>
+      </visual>
+      <collision>
+        <origin xyz="0 0 0" rpy="0 0 0" />
+        <geometry>
+          <box size="0.001 0.001 0.001" />
+        </geometry>
+      </collision>
     </link>
     <!-- joint between torso_pan_link and torso_upper_neck_tilt_link -->
@@ -78,9 +95,5 @@
     </joint>
     <link name="${name}_upper_neck_tilt_link">
-      <inertial>
-        <origin xyz="0 0 0" rpy="0 0 0"/>
-        <mass value="6.744238"/>
-        <inertia ixx="0.01" ixy="0" ixz="0" iyy="0.01" iyz="0" izz="0.01" />
-      </inertial>
+      <xacro:default_inertial/>
       <visual>
         <origin xyz="0 0 0" rpy="${M_PI} 0 0" />
@@ -105,9 +118,5 @@
     </joint>
     <link name="head_cover_link">
-      <inertial>
-        <origin xyz="0 0 0" rpy="0 0 0"/>
-        <mass value="0.5"/>
-        <inertia ixx="0.01" ixy="0" ixz="0" iyy="0.01" iyz="0" izz="0.01" />
-      </inertial>
+      <xacro:default_inertial/>
       <visual>
         <origin xyz="0 0 0" rpy="0 0 0" />

File: cob_description/urdf/cob3_tray/tray.urdf.xacro (robot description, xacro)
@@ -16,9 +16,5 @@
     </joint>
     <link name="${name}_link">
-      <inertial>
-        <origin xyz="0 0 0" rpy="0 0 0"/>
-        <mass value="0.1"/>
-        <inertia ixx="0.01" ixy="0" ixz="0" iyy="0.01" iyz="0" izz="0.01" />
-      </inertial>
+      <xacro:default_inertial/>
       <visual>
         <origin xyz="0 0 0" rpy="0 0 0" />
@@ -41,5 +37,19 @@
       <child link="${name}_base_link" />
     </joint>
-    <link name="${name}_base_link"/>
+    <link name="${name}_base_link">
+      <xacro:default_inertial/>
+      <visual>
+        <origin xyz="0 0 0" rpy="0 0 0" />
+        <geometry>
+          <box size="0.001 0.001 0.001" />
+        </geometry>
+      </visual>
+      <collision>
+        <origin xyz="0 0 0" rpy="0 0 0" />
+        <geometry>
+          <box size="0.001 0.001 0.001" />
+        </geometry>
+      </collision>
+    </link>
     <joint name="${name}_right_joint" type="fixed" >
       <origin xyz="0.4 -0.3 0.1" rpy="0 0 0"/>
@@ -47,5 +57,19 @@
       <child link="${name}_right_link" />
     </joint>
-    <link name="${name}_right_link"/>
+    <link name="${name}_right_link">
+      <xacro:default_inertial/>
+      <visual>
+        <origin xyz="0 0 0" rpy="0 0 0" />
+        <geometry>
+          <box size="0.001 0.001 0.001" />
+        </geometry>
+      </visual>
+      <collision>
+        <origin xyz="0 0 0" rpy="0 0 0" />
+        <geometry>
+          <box size="0.001 0.001 0.001" />
+        </geometry>
+      </collision>
+    </link>
     <joint name="${name}_left_joint" type="fixed" >
       <origin xyz="0.4 0.05 0.1" rpy="0 0 0"/>

File: cob_description/urdf/cob3_tray/tray_3DOF.urdf.xacro (robot description, xacro)
@@ -16,9 +16,5 @@
     </joint>
     <link name="${name}_1_link">
-      <inertial>
-        <origin xyz="0 0 0" rpy="0 0 0"/>
-        <mass value="1.6"/>
-        <inertia ixx="0.01" ixy="0" ixz="0" iyy="0.01" iyz="0" izz="0.01" />
-      </inertial>
+      <xacro:default_inertial/>
       <visual>
         <origin xyz="0 0 0" rpy="0 0 0" />
@@ -45,9 +41,5 @@
     </joint>
     <link name="${name}_2_link">
-      <inertial>
-        <origin xyz="0 0 0" rpy="0 0 0"/>
-        <mass value="1"/>
-        <inertia ixx="0.01" ixy="0" ixz="0" iyy="0.01" iyz="0" izz="0.01" />
-      </inertial>
+      <xacro:default_inertial/>
       <visual>
         <origin xyz="0 0 0" rpy="0 0 0" />
@@ -74,9 +66,5 @@
     </joint>
     <link name="${name}_3_link">
-      <inertial>
-        <origin xyz="0 0 0" rpy="0 0 0"/>
-        <mass value="1"/>
-        <inertia ixx="0.01" ixy="0" ixz="0" iyy="0.01" iyz="0" izz="0.01" />
-      </inertial>
+      <xacro:default_inertial/>
       <visual>
         <origin xyz="0 0 0" rpy="0 0 0" />
@@ -99,9 +87,5 @@
     </joint>
     <link name="${name}_right_link">
-      <inertial>
-        <mass value="0.001" />
-        <origin xyz="0 0 0" rpy="0 0 0" />
-        <inertia ixx="0.0001" ixy="0" ixz="0" iyy="0.000001" iyz="0" izz="0.0001" />
-      </inertial>
+      <xacro:default_inertial/>
       <visual>
         <origin xyz="0 0 0" rpy="0 0 0" />
@@ -124,9 +108,5 @@
     </joint>
     <link name="${name}_left_link">
-      <inertial>
-        <mass value="0.001" />
-        <origin xyz="0 0 0" rpy="0 0 0" />
-        <inertia ixx="0.0001" ixy="0" ixz="0" iyy="0.000001" iyz="0" izz="0.0001" />
-      </inertial>
+      <xacro:default_inertial/>
       <visual>
         <origin xyz="0 0 0" rpy="0 0 0" />
