Commit message: prosilica: ros_topic -> topic_prefix

File: cob_description/urdf/cob3_head/head_prosilicas_kinect.urdf.xacro (robot description, xacro)
@@ -73,9 +73,9 @@
     </link>
     <!-- left camera -->
-    <xacro:cob_prosilica_v0 name="${name}_color_camera_l" ros_topic="stereo/left" parent="${name}_cam_reference_link">
+    <xacro:cob_prosilica_v0 name="${name}_color_camera_l" topic_prefix="stereo/left/" parent="${name}_cam_reference_link">
       <origin xyz="${cam_l_x} ${cam_l_y} ${cam_l_z}" rpy="${cam_l_roll} ${cam_l_pitch} ${cam_l_yaw}" />
     </xacro:cob_prosilica_v0>
     <!-- right camera -->
-    <xacro:cob_prosilica_v0 name="${name}_color_camera_r" ros_topic="stereo/right" parent="${name}_cam_reference_link">
+    <xacro:cob_prosilica_v0 name="${name}_color_camera_r" topic_prefix="stereo/right/" parent="${name}_cam_reference_link">
       <origin xyz="${cam_r_x} ${cam_r_y} ${cam_r_z}" rpy="${cam_r_roll} ${cam_r_pitch} ${cam_r_yaw}" />
     </xacro:cob_prosilica_v0>

File: cob_description/urdf/sensors/prosilica.gazebo.xacro (robot description, xacro)
@@ -1,5 +1,5 @@
 <?xml version="1.0"?>
 <root xmlns:xacro="http://www.ros.org/wiki/xacro">
-  <xacro:macro name="cob_prosilica_gazebo_v0" params="name ros_topic">
+  <xacro:macro name="cob_prosilica_gazebo_v0" params="name topic_prefix">
     <gazebo reference="${name}_frame">
       <sensor type="camera" name="${name}_sensor">
@@ -27,7 +27,7 @@
           <cameraName>${name}</cameraName>
           <frameName>${name}_link</frameName>
-          <topicName>${ros_topic}_image_data</topicName>
-          <imageTopicName>${ros_topic}_image_raw</imageTopicName>
-          <cameraInfoTopicName>${ros_topic}_camera_info</cameraInfoTopicName>
+          <topicName>${topic_prefix}image_data</topicName>
+          <imageTopicName>${topic_prefix}image_raw</imageTopicName>
+          <cameraInfoTopicName>${topic_prefix}camera_info</cameraInfoTopicName>
           <pollServiceName>request_image</pollServiceName>
           <CxPrime>697.69</CxPrime>

File: cob_description/urdf/sensors/prosilica.urdf.xacro (robot description, xacro)
@@ -3,5 +3,5 @@
        name="LaserBlock">
   <xacro:include filename="$(find cob_description)/urdf/sensors/prosilica.gazebo.xacro" />
-  <xacro:macro name="cob_prosilica_v0" params="name parent *origin ros_topic">
+  <xacro:macro name="cob_prosilica_v0" params="name parent *origin topic_prefix">
     <joint name="${name}_joint" type="fixed">
       <insert_block name="origin" />
@@ -35,5 +35,5 @@
     </joint>
     <link name="${name}_frame"/>
-    <xacro:cob_prosilica_gazebo_v0 name="${name}" ros_topic="${ros_topic}"/>
+    <xacro:cob_prosilica_gazebo_v0 name="${name}" topic_prefix="${topic_prefix}"/>
   </xacro:macro>
 </robot>

File: raw_description/urdf/head/head.urdf.xacro (robot description, xacro)
@@ -26,9 +26,9 @@
     <link name="${name}_cam_reference_link"/>
     <!-- left camera -->
-    <xacro:cob_prosilica_v0 name="${name}_color_camera_left" ros_topic="stereo" parent="${name}_cam_reference_link">
+    <xacro:cob_prosilica_v0 name="${name}_color_camera_left" topic_prefix="stereo" parent="${name}_cam_reference_link">
       <origin xyz="${cam_l_x} ${cam_l_y} ${cam_l_z}" rpy="${cam_l_roll} ${cam_l_pitch} ${cam_l_yaw}" />
     </xacro:cob_prosilica_v0>
     <!-- right camera -->
-    <xacro:cob_prosilica_v0 name="${name}_color_camera_right" ros_topic="stereo" parent="${name}_cam_reference_link">
+    <xacro:cob_prosilica_v0 name="${name}_color_camera_right" topic_prefix="stereo" parent="${name}_cam_reference_link">
       <origin xyz="${cam_r_x} ${cam_r_y} ${cam_r_z}" rpy="${cam_r_roll} ${cam_r_pitch} ${cam_r_yaw}" />
     </xacro:cob_prosilica_v0>
