Commit message: Tested on simulation

File: cob_description/urdf/cob3_torso/torso_v2.urdf.xacro (robot description, xacro)
@@ -4,6 +4,6 @@
        xmlns:interface="http://playerstage.sourceforge.net/gazebo/xmlschema/#interface"
        xmlns:xacro="http://ros.org/wiki/xacro">
-	<include filename="$(find cob_description)/urdf/cob3_torso/torso.gazebo.xacro" />
-	<include filename="$(find cob_description)/urdf/cob3_torso/torso.transmission.xacro" />
+	<include filename="$(find cob_description)/urdf/cob3_torso/torso_v2.gazebo.xacro" />
+	<include filename="$(find cob_description)/urdf/cob3_torso/torso_v2.transmission.xacro" />
 	<xacro:macro name="torso" params="name parent *origin">
 		<!-- joint between base_link and torso_base_link -->

File: cob_description/urdf/cob3_tray/tray_3DOF.urdf.xacro (robot description, xacro)
@@ -160,6 +160,6 @@
 		</xacro:phidgets_distance_v0>
 		<!-- extensions -->
-		<xacro:cob3_tray_3DOF_gazebo name="${name}" />
-		<xacro:cob3_tray_3DOF_transmission name="${name}" />
+		<xacro:tray_gazebo name="${name}" />
+		<xacro:tray_transmission name="${name}" />
 	</xacro:macro>
 </robot>

File: cob_description/urdf/lookat/lookat.urdf.xacro (robot description, xacro)
@@ -4,5 +4,5 @@
 	   xmlns:interface="http://playerstage.sourceforge.net/gazebo/xmlschema/#interface"
 	   xmlns:xacro="http://ros.org/wiki/xacro">
-	<xacro:macro name="cob_lookat" params="name parent *origin *axis lower upper">
+	<xacro:macro name="lookat" params="name parent *origin *axis lower upper">
 		<!-- joint between torso_upper_neck_tilt_link and lookat_base_link -->
 		<joint name="${name}_base_joint" type="fixed">
