Commit message: fixes while testing in simulation

File: cob_description/urdf/cob3_torso/torso_v1.urdf.xacro (robot description, xacro)
@@ -3,5 +3,5 @@
   <xacro:include filename="$(find cob_description)/urdf/cob3_torso/torso_v1.gazebo.xacro" />
   <xacro:include filename="$(find cob_description)/urdf/cob3_torso/torso_v1.transmission.xacro" />
-  <xacro:macro name="cob_torso_v0" params="name parent *origin">
+  <xacro:macro name="torso" params="name parent *origin">
     <!-- joint between base_link and torso_base_link -->
     <joint name="${name}_base_joint" type="fixed" >

File: cob_description/urdf/cob3_tray/tray_3DOF.urdf.xacro (robot description, xacro)
@@ -13,5 +13,5 @@
       <calibration rising="${tray_1_ref}"/>
       <dynamics damping="5.0" friction="0.5"/>
-      <limit effort="100" lower="1.37" upper="-0.02" velocity="5"/>
+      <limit effort="100" lower="-0.02" upper="1.37" velocity="5"/>
     </joint>
     <link name="${name}_1_link">

File: cob_description/urdf/cob4_base/base.urdf.xacro (robot description, xacro)
@@ -152,5 +152,6 @@
         <origin xyz="0 0 0" rpy="0 0 0" />
         <geometry>
-          <mesh filename="package://cob_description/meshes/cob4_base/caster.stl"/>
+          <!--mesh filename="package://cob_description/meshes/cob4_base/caster.stl"/-->
+          <box size="0.01 0.01 0.01" />
         </geometry>
         <material name="IPA/LightGrey" />

File: desire_description/urdf/base_desire/base.urdf.xacro (robot description, xacro)
@@ -57,5 +57,5 @@
         <origin xyz="0 0 0" rpy="0 0 0" />
         <geometry>
-          <mesh filename="package://cob_description/meshes/base/pr2_wheel.stl" />
+          <mesh filename="package://desire_description/meshes/base_desire/cob_wheel.stl" />
         </geometry>
         <material name="IPA/LightGrey" />
@@ -94,5 +94,5 @@
         <origin xyz="0 0 0" rpy="0 0 0" />
         <geometry>
-          <mesh filename="$(find cob_description)/meshes/base/caster.stl" />
+          <mesh filename="$(find desire_description)/meshes/base_desire/caster.stl" />
         </geometry>
         <material name="IPA/DarkGrey" />
