Commit message: added velocity and position controllers

File: cob_description/urdf/cob3_torso/torso_v2.transmission.xacro (robot description, xacro)
@@ -6,4 +6,6 @@
       <joint name="${name}_lower_neck_tilt_joint">
         <hardwareInterface>EffortJointInterface</hardwareInterface>
+        <hardwareInterface>PositionJointInterface</hardwareInterface>
+        <hardwareInterface>VelocityJointInterface</hardwareInterface>
       </joint>
       <actuator name="${name}_lower_neck_tilt_motor">
@@ -15,4 +17,6 @@
       <joint name="${name}_pan_joint">
         <hardwareInterface>EffortJointInterface</hardwareInterface>
+        <hardwareInterface>PositionJointInterface</hardwareInterface>
+        <hardwareInterface>VelocityJointInterface</hardwareInterface>
       </joint>
       <actuator name="${name}_pan_motor">
@@ -24,4 +28,6 @@
       <joint name="${name}_upper_neck_tilt_joint">
         <hardwareInterface>EffortJointInterface</hardwareInterface>
+        <hardwareInterface>PositionJointInterface</hardwareInterface>
+        <hardwareInterface>VelocityJointInterface</hardwareInterface>
       </joint>
       <actuator name="${name}_upper_neck_tilt_motor">

File: cob_description/urdf/cob3_tray/tray.transmission.xacro (robot description, xacro)
@@ -6,4 +6,6 @@
       <joint name="${name}_joint">
         <hardwareInterface>EffortJointInterface</hardwareInterface>
+        <hardwareInterface>PositionJointInterface</hardwareInterface>
+        <hardwareInterface>VelocityJointInterface</hardwareInterface>
       </joint>
       <actuator name="${name}_motor">

File: cob_description/urdf/cob3_tray/tray_3DOF.transmission.xacro (robot description, xacro)
@@ -6,4 +6,6 @@
       <joint name="${name}_1_joint">
         <hardwareInterface>EffortJointInterface</hardwareInterface>
+        <hardwareInterface>PositionJointInterface</hardwareInterface>
+        <hardwareInterface>VelocityJointInterface</hardwareInterface>
       </joint>
       <actuator name="${name}_1_motor">
@@ -15,4 +17,6 @@
       <joint name="${name}_2_joint">
         <hardwareInterface>EffortJointInterface</hardwareInterface>
+        <hardwareInterface>PositionJointInterface</hardwareInterface>
+        <hardwareInterface>VelocityJointInterface</hardwareInterface>
       </joint>
       <actuator name="${name}_2_motor">
@@ -22,6 +26,7 @@
     <transmission name="${name}_3_trans">
       <type>transmission_interface/SimpleTransmission</type>
-      <joint name="${name}_3_joint">
         <hardwareInterface>EffortJointInterface</hardwareInterface>
+        <hardwareInterface>PositionJointInterface</hardwareInterface>
+        <hardwareInterface>VelocityJointInterface</hardwareInterface>
       </joint>
       <actuator name="${name}_3_motor">
