Commit message: renamed tray 3DOF

File: cob_description/urdf/cob3_tray/tray_3DOF.urdf.xacro (robot description, xacro)
@@ -27,5 +27,5 @@
 				<origin xyz="0 0 0" rpy="0 0 0" />
 				<geometry>
-					<mesh filename="package://cob_description/meshes/cob3_3DOF_tray/tray_link_1.stl" />
+					<mesh filename="package://cob_description/meshes/cob3_tray_3DOF/tray_link_1.stl" />
 				</geometry>
 				<material name="IPA/DarkGrey" />
@@ -34,5 +34,5 @@
 				<origin xyz="0 0 0" rpy="0 0 0" />
 				<geometry>
-					<mesh filename="package://cob_description/meshes/cob3_3DOF_tray/tray_link_1.stl" />
+					<mesh filename="package://cob_description/meshes/cob3_tray_3DOF/tray_link_1.stl" />
 				</geometry>
 			</collision>
@@ -56,5 +56,5 @@
 				<origin xyz="0 0 0" rpy="0 0 0" />
 				<geometry>
-					<mesh filename="package://cob_description/meshes/cob3_3DOF_tray/tray_link_2.stl" />
+					<mesh filename="package://cob_description/meshes/cob3_tray_3DOF/tray_link_2.stl" />
 				</geometry>
 				<material name="IPA/DarkGrey" />
@@ -63,5 +63,5 @@
 				<origin xyz="0 0 0" rpy="0 0 0" />
 				<geometry>
-					<mesh filename="package://cob_description/meshes/cob3_3DOF_tray/tray_link_2.stl" />
+					<mesh filename="package://cob_description/meshes/cob3_tray_3DOF/tray_link_2.stl" />
 				</geometry>
 			</collision>
@@ -85,5 +85,5 @@
 				<origin xyz="0 0 0" rpy="0 0 0" />
 				<geometry>
-					<mesh filename="package://cob_description/meshes/cob3_3DOF_tray/tray_link_3.stl" />
+					<mesh filename="package://cob_description/meshes/cob3_tray_3DOF/tray_link_3.stl" />
 				</geometry>
 				<material name="IPA/DarkGrey" />
@@ -92,5 +92,5 @@
 				<origin xyz="0 0 0" rpy="0 0 0" />
 				<geometry>
-					<mesh filename="package://cob_description/meshes/cob3_3DOF_tray/tray_link_3.stl" />
+					<mesh filename="package://cob_description/meshes/cob3_tray_3DOF/tray_link_3.stl" />
 				</geometry>
 			</collision>
