Commit message: fixed path to file

File: cob_description/urdf/cob3_tray/tray.urdf.xacro (robot description, xacro)
@@ -34,5 +34,5 @@
 				<origin xyz="0 0 0" rpy="0 0 0" />
 				<geometry>
-					<mesh filename="package://cob_description/meshes/tray_cob3/tray_collision.stl" />
+					<mesh filename="package://cob_description/meshes/cob3_tray/tray_collision.stl" />
 				</geometry>
 			</collision>
