Commit message: fix syntax

File: cob_description/urdf/cob3_tray/tray_3DOF.transmission.xacro (robot description, xacro)
@@ -26,4 +26,5 @@
     <transmission name="${name}_3_trans">
       <type>transmission_interface/SimpleTransmission</type>
+      <joint name="${name}_3_joint">
         <hardwareInterface>EffortJointInterface</hardwareInterface>
         <hardwareInterface>PositionJointInterface</hardwareInterface>
