Commit message: Improvements cob4 simulation, the inertia values are still not correct

File: cob_description/urdf/cob4_head/head.gazebo.xacro (robot description, xacro)
@@ -7,17 +7,17 @@
 		<gazebo reference="${name}_base_link">
 			<material>IPA/LightGrey</material>
-			<turnGravityOff>false</turnGravityOff>
+			<gravity>true</gravity>
 		</gazebo>
 		<gazebo reference="${name}_1_link">
             <material>IPA/LightGrey</material>
-			<turnGravityOff>false</turnGravityOff>
+			<gravity>true</gravity>
 		</gazebo>
 		<gazebo reference="${name}_2_link">
 			<material>IPA/LightGrey</material>
-			<turnGravityOff>false</turnGravityOff>
+			<gravity>true</gravity>
 		</gazebo>
 		<gazebo reference="${name}_3_link">
 			<material>IPA/LightGrey</material>
-			<turnGravityOff>false</turnGravityOff>
+			<gravity>true</gravity>
 		</gazebo>
 	</xacro:macro>

File: cob_description/urdf/cob4_head/head.urdf.xacro (robot description, xacro)
@@ -15,5 +15,5 @@
 			<inertial>
 				<origin xyz="0 0 0" rpy="0 0 0"/>
-				<mass value="1"/>
+				<mass value="0.1"/>
 				<inertia ixx="0.01" ixy="0" ixz="0" iyy="0.01" iyz="0" izz="0.01" />
 			</inertial>
@@ -31,5 +31,5 @@
 			<inertial>
 				<origin xyz="0 0 0" rpy="0 0 0"/>
-				<mass value="1"/>
+				<mass value="0.2"/>
 				<inertia ixx="0.01" ixy="0" ixz="0" iyy="0.01" iyz="0" izz="0.01" />
 			</inertial>
@@ -47,5 +47,5 @@
 			<inertial>
 				<origin xyz="0 0 0" rpy="0 0 0"/>
-				<mass value="1"/>
+				<mass value="0.1"/>
 				<inertia ixx="0.01" ixy="0" ixz="0" iyy="0.01" iyz="0" izz="0.01" />
 			</inertial>
@@ -64,6 +64,5 @@
 			<mass value="1" />
 			<origin xyz="0 0 0" />
-			<inertia ixx="5.652232699207" ixy="-0.009719934438" ixz="1.293988226423"
-					 iyy="5.669473158652" iyz="-0.007379583694" izz="3.683196351726" />
+				<inertia ixx="0.01" ixy="0" ixz="0" iyy="0.01" iyz="0" izz="0.01" />
 		  </inertial>
 		  <visual>

File: cob_description/urdf/cob4_sensorring/sensorring.gazebo.xacro (robot description, xacro)
@@ -7,5 +7,5 @@
 		<gazebo reference="${name}_link">
 			<material>IPA/DarkGrey</material>
-			<turnGravityOff>false</turnGravityOff>
+			<gravity>true</gravity>
 		</gazebo>
 	</xacro:macro>

File: cob_description/urdf/cob4_torso/torso.gazebo.xacro (robot description, xacro)
@@ -7,17 +7,17 @@
 		<gazebo reference="${name}_base_link">
             <material>IPA/LightGrey</material>
-			<turnGravityOff>false</turnGravityOff>
+			<gravity>true</gravity>
 		</gazebo>
 		<gazebo reference="${name}_1_link">
 			<material>IPA/LightGrey</material>
-			<turnGravityOff>false</turnGravityOff>
+			<gravity>true</gravity>
 		</gazebo>
 		<gazebo reference="${name}_2_link">
 			<material>IPA/LightGrey</material>
-			<turnGravityOff>false</turnGravityOff>
+			<gravity>true</gravity>
 		</gazebo>
 		<gazebo reference="${name}_3_link">
 			<material>IPA/LightGrey</material>
-			<turnGravityOff>false</turnGravityOff>
+			<gravity>true</gravity>
 		</gazebo>
 	</xacro:macro>

File: cob_description/urdf/cob4_torso/torso.urdf.xacro (robot description, xacro)
@@ -27,5 +27,5 @@
 		  <calibration rising="${torso_1_ref}"/>
 		  <axis xyz="0 0 1" />
-		  <dynamics damping="0.1" />
+		  <dynamics damping="2.0" friction="0.0"/>
 		  <limit effort="100" lower="-6.2831" upper="6.2831" velocity="1.4"/>
 		</joint>
@@ -33,5 +33,5 @@
 			<inertial>
 				<origin xyz="0 0 0" rpy="0 0 0"/>
-				<mass value="5"/>
+				<mass value="50"/>
 				<inertia ixx="0.01" ixy="0" ixz="0" iyy="0.01" iyz="0" izz="0.01" />
 			</inertial>
@@ -43,5 +43,5 @@
 		  <calibration rising="${torso_2_ref}"/>
 		  <axis xyz="0 0 1" />
-		  <dynamics damping="0.1" />
+		  <dynamics damping="2.0" friction="0.0"/>
 		  <limit effort="100" lower="-6.2831" upper="6.2831" velocity="1.4"/>
 		</joint>
@@ -59,13 +59,12 @@
 		  <calibration rising="${torso_3_ref}"/>
 		  <axis xyz="0 0 1" />
-		  <dynamics damping="0.1" />
+		  <dynamics damping="2.0" friction="0.0"/>
 		  <limit effort="100" lower="-6.2831" upper="6.2831" velocity="1.4"/>
 		</joint>
 		<link name="torso_3_link">
 			<inertial>
-				<origin xyz="0 0 0" rpy="0 0 0"/>
+				<origin xyz="0 0 0.3" rpy="0 0 0"/>
 				<mass value="20" />
-			<inertia ixx="0.1" ixy="0" ixz="0"
-						 iyy="0.01" iyz="0" izz="0.01" />
+			<inertia ixx="0.1" ixy="0" ixz="0" iyy="0.01" iyz="0" izz="0.01" />
 			</inertial>
 			<visual>

File: cob_description/urdf/sensors/kinect.urdf.xacro (robot description, xacro)
@@ -20,5 +20,5 @@
         <origin xyz="0 0 0.015" rpy="0 0 0" />
         <geometry>
-          <box size="0.02 0.02 0.075"/>
+          <box size="0.002 0.002 0.002"/>
         </geometry>
         <material name="IPA/LightGrey" />
@@ -27,5 +27,5 @@
         <origin xyz="0 0 0.015" rpy="0 0 0" />
         <geometry>
-           <box size="0.02 0.02 0.075"/>
+           <box size="0.002 0.002 0.002"/>
         </geometry>
       </collision>

File: cob_description/urdf/sensors/softkinetic.gazebo.xacro (robot description, xacro)
@@ -1,7 +1,4 @@
 <?xml version="1.0"?>
-<root xmlns:sensor="http://playerstage.sourceforge.net/gazebo/xmlschema/#sensor"
-      xmlns:controller="http://playerstage.sourceforge.net/gazebo/xmlschema/#controller"
-      xmlns:interface="http://playerstage.sourceforge.net/gazebo/xmlschema/#interface"
-      xmlns:xacro="http://ros.org/wiki/xacro">
+<root xmlns:xacro="http://ros.org/wiki/xacro">
 <xacro:macro name="softkinetic_gazebo" params="name ros_topic">
   <gazebo reference="${name}_frame">
@@ -21,9 +18,8 @@
         </clip>
       </camera>
-      <plugin name="${name}_controller" filename="libgazebo_ros_openni_kinect.so">
+      <plugin name="${name}_frame_controller" filename="libgazebo_ros_openni_kinect.so">
         <alwaysOn>true</alwaysOn>
         <updateRate>25.0</updateRate>
         <cameraName>${ros_topic}</cameraName>
-        <frameName>${name}_link</frameName>
         <imageTopicName>rgb/image_raw</imageTopicName>
         <depthImageTopicName>depth/image_raw</depthImageTopicName>
@@ -31,6 +27,6 @@
         <cameraInfoTopicName>rgb/camera_info</cameraInfoTopicName>
         <depthImageCameraInfoTopicName>depth_registered/camera_info</depthImageCameraInfoTopicName>
+        <frameName>${name}_optical_frame</frameName>
         <pointCloudCutoff>0.5</pointCloudCutoff>
-        <hackBaseline>0.0</hackBaseline>
         <distortionK1>0.0</distortionK1>
         <distortionK2>0.0</distortionK2>

File: cob_description/urdf/sensors/softkinetic.urdf.xacro (robot description, xacro)
@@ -5,5 +5,5 @@
       xmlns:xacro="http://ros.org/wiki/xacro">
   <include filename="$(find cob_description)/urdf/sensors/softkinetic.gazebo.xacro" />
-  <xacro:macro name="softkinetic" params="name parent *origin ros_topic">
+  <xacro:macro name="softkinetic" params="name parent ros_topic *origin">
     <joint name="${name}_joint" type="fixed">
       <insert_block name="origin" />
@@ -11,30 +11,37 @@
       <child link="${name}_link"/>
     </joint>
-    <link name="${name}_link">
+    <link name="${name}_link"/>
+    <joint name="${name}_frame_joint" type="fixed">
+      <origin xyz="0 0 0" rpy="${-M_PI/2} ${-M_PI/2} 0" />
+      <parent link="${name}_link"/>
+      <child link="${name}_frame"/>
+    </joint>
+    <link name="${name}_frame">
       <inertial>
-        <mass value="0.01" />
+        <mass value="0.1" />
         <origin xyz="0 0 0" rpy="0 0 0"/>
-        <inertia ixx="0.0001" ixy="0" ixz="0" iyy="0.0001" iyz="0" izz="0.0001" />
+        <inertia ixx="0.01"  ixy="0.0"  ixz="0.0"
+                 iyy="0.01"  iyz="0.0"
+                 izz="0.01" />
       </inertial>
       <visual>
-        <origin xyz="0 0 0.015" rpy="0 0 0" />
+        <origin xyz="0.0 0.0 0" rpy="0 0 0"/>
         <geometry>
-          <box size="0.02 0.02 0.075"/>
+          <box size="0.002 0.002 0.002"/>
         </geometry>
-        <material name="IPA/LightGrey" />
       </visual>
       <collision>
-        <origin xyz="0 0 0.015" rpy="0 0 0" />
+        <origin xyz="0.0 0.0 0" rpy="0 0 0"/>
         <geometry>
-           <box size="0.02 0.02 0.075"/>
+          <box size="0.002 0.002 0.002"/>>
         </geometry>
       </collision>
     </link>
-    <joint name="${name}_frame_joint" type="fixed">
-      <origin xyz="0 0 0" rpy="${M_PI/2} -${M_PI/2} 0" />
-      <parent link="${name}_link"/>
-      <child link="${name}_frame"/>
+    <joint name="${name}_optical_joint" type="fixed">
+      <origin xyz="0 0 0" rpy="${-M_PI/2} 0.0 ${-M_PI/2}" />
+      <parent link="${name}_frame"/>
+      <child link="${name}_optical_frame"/>
     </joint>
-    <link name="${name}_frame"/>
+    <link name="${name}_optical_frame"/>
     <!-- extensions -->
     <xacro:softkinetic_gazebo name="${name}" ros_topic="${ros_topic}" />
