Commit message: prepare cob4 component descriptions for new structure

File: cob_description/urdf/cob4_head/head.transmission.xacro (robot description, xacro)
@@ -5,5 +5,6 @@
       <type>transmission_interface/SimpleTransmission</type>
       <joint name="${name}_1_joint">
-        <hardwareInterface>EffortJointInterface</hardwareInterface>
+        <hardwareInterface>PositionJointInterface</hardwareInterface>
+        <hardwareInterface>VelocityJointInterface</hardwareInterface>
       </joint>
       <actuator name="${name}_1_motor">
@@ -14,5 +15,6 @@
       <type>transmission_interface/SimpleTransmission</type>
       <joint name="${name}_2_joint">
-        <hardwareInterface>EffortJointInterface</hardwareInterface>
+        <hardwareInterface>PositionJointInterface</hardwareInterface>
+        <hardwareInterface>VelocityJointInterface</hardwareInterface>
       </joint>
       <actuator name="${name}_2_motor">
@@ -23,5 +25,6 @@
       <type>transmission_interface/SimpleTransmission</type>
       <joint name="${name}_3_joint">
-        <hardwareInterface>EffortJointInterface</hardwareInterface>
+        <hardwareInterface>PositionJointInterface</hardwareInterface>
+        <hardwareInterface>VelocityJointInterface</hardwareInterface>
       </joint>
       <actuator name="${name}_3_motor">

File: cob_description/urdf/cob4_head/head.urdf.xacro (robot description, xacro)
@@ -10,57 +10,38 @@
     </joint>
     <link name="${name}_base_link">
-      <inertial>
-        <origin xyz="0 0 0" rpy="0 0 0"/>
-        <mass value="0.1"/>
-        <inertia ixx="0.01" ixy="0" ixz="0" iyy="0.01" iyz="0" izz="0.01" />
-      </inertial>
+      <xacro:default_inertial/>
     </link>
     <joint name="${name}_1_joint" type="revolute">
       <origin xyz="0 0 0.0305" rpy="0 0 0"/>
+      <parent link="${name}_base_link"/>
       <child link="${name}_1_link" />
-      <parent link="${name}_base_link"/>
+      <axis xyz="0 0 1" />
       <calibration rising="${head_1_ref}"/>
-      <axis xyz="0 0 1" />
-      <dynamics damping="0.1" />
       <limit effort="100" lower="-6.2831" upper="6.2831" velocity="1.4"/>
     </joint>
     <link name="${name}_1_link">
-      <inertial>
-        <origin xyz="0 0 0" rpy="0 0 0"/>
-        <mass value="0.1"/>
-        <inertia ixx="0.01" ixy="0" ixz="0" iyy="0.01" iyz="0" izz="0.01" />
-      </inertial>
+      <xacro:default_inertial/>
     </link>
     <joint name="${name}_2_joint" type="revolute">
       <origin xyz="0 -0.07725 -0.00439" rpy="-0.349 0 0" />
+      <parent link="${name}_1_link"/>
       <child link="${name}_2_link" />
-      <parent link="${name}_1_link"/>
+      <axis xyz="0 0 1" />
       <calibration rising="${head_2_ref}"/>
-      <axis xyz="0 0 1" />
-      <dynamics damping="0.1" />
       <limit effort="100" lower="-6.2831" upper="6.2831" velocity="1.4"/>
     </joint>
     <link name="${name}_2_link">
-      <inertial>
-        <origin xyz="0 0 0" rpy="0 0 0"/>
-        <mass value="0.1"/>
-        <inertia ixx="0.01" ixy="0" ixz="0" iyy="0.01" iyz="0" izz="0.01" />
-      </inertial>
+      <xacro:default_inertial/>
     </link>
     <joint name="${name}_3_joint" type="revolute">
       <origin xyz="0 0.04668 0.0976" rpy="0.349 0 0" />
+      <parent link="${name}_2_link"/>
       <child link="${name}_3_link" />
-      <parent link="${name}_2_link"/>
+      <axis xyz="0 0 1" />
       <calibration rising="${head_3_ref}"/>
-      <axis xyz="0 0 1" />
-      <dynamics damping="0.1" />
       <limit effort="100" lower="-6.2831" upper="6.2831" velocity="1.4"/>
     </joint>
     <link name="${name}_3_link">
-      <inertial>
-        <mass value="1" />
-        <origin xyz="0 0 0" />
-        <inertia ixx="0.01" ixy="0" ixz="0" iyy="0.01" iyz="0" izz="0.01" />
-      </inertial>
+      <xacro:default_inertial/>
       <visual>
         <origin xyz="0 0 0" rpy="0 0 0" />
@@ -72,5 +53,5 @@
         <origin xyz="0 0 0" rpy="0 0 0" />
         <geometry>
-          <mesh filename="package://cob_description/meshes/cob4_head/head_link.dae"/>
+          <mesh filename="package://cob_description/meshes/cob4_head/head_link_collision.stl"/>
         </geometry>
       </collision>
@@ -78,6 +59,6 @@
     <joint name="${name}_center_joint" type="fixed">
       <origin xyz="0.0 0.0 -0.28247" rpy="0 0 0" />
+      <parent link="${name}_3_link"/>
       <child link="${name}_center_link" />
-      <parent link="${name}_3_link"/>
     </joint>
     <link name="${name}_center_link"/>

File: cob_description/urdf/cob4_sensorring/sensorring.transmission.xacro (robot description, xacro)
@@ -5,5 +5,6 @@
       <type>transmission_interface/SimpleTransmission</type>
       <joint name="${name}_joint">
-        <hardwareInterface>EffortJointInterface</hardwareInterface>
+        <hardwareInterface>PositionJointInterface</hardwareInterface>
+        <hardwareInterface>VelocityJointInterface</hardwareInterface>
       </joint>
       <actuator name="${name}_motor">

File: cob_description/urdf/cob4_sensorring/sensorring.urdf.xacro (robot description, xacro)
@@ -10,9 +10,5 @@
     </joint>
     <link name="${name}_base_link">
-      <inertial>
-        <origin xyz="0 0 0" rpy="0 0 0"/>
-        <mass value="0.1"/>
-        <inertia ixx="0.01" ixy="0" ixz="0" iyy="0.01" iyz="0" izz="0.01" />
-      </inertial>
+      <xacro:default_inertial/>
     </link>
     <joint name="${name}_joint" type="revolute">
@@ -20,13 +16,15 @@
       <parent link="${name}_base_link"/>
       <child link="${name}_link" />
+      <axis xyz="0 0 1" />
       <calibration rising="${sensorring_ref}"/>
-      <axis xyz="0 0 1" />
-      <dynamics damping="5.0" friction="0.5"/>
       <limit effort="100" lower="-6.2831" upper="6.2831" velocity="1.4"/>
     </joint>
     <link name="${name}_link">
+      <xacro:default_inertial/>
+<!--
       <xacro:cylinder_inertial radius="0.250" length="0.1" mass="1.0">
         <origin xyz="0 0 0" rpy="0 0 0" />
       </xacro:cylinder_inertial>
+-->
     </link>
     <!-- extensions -->

File: cob_description/urdf/cob4_torso/torso.transmission.xacro (robot description, xacro)
@@ -5,4 +5,5 @@
       <type>transmission_interface/SimpleTransmission</type>
       <joint name="${name}_1_joint">
+        <hardwareInterface>PositionJointInterface</hardwareInterface>
         <hardwareInterface>VelocityJointInterface</hardwareInterface>
       </joint>
@@ -14,4 +15,5 @@
       <type>transmission_interface/SimpleTransmission</type>
       <joint name="${name}_2_joint">
+        <hardwareInterface>PositionJointInterface</hardwareInterface>
         <hardwareInterface>VelocityJointInterface</hardwareInterface>
       </joint>
@@ -23,4 +25,5 @@
       <type>transmission_interface/SimpleTransmission</type>
       <joint name="${name}_3_joint">
+        <hardwareInterface>PositionJointInterface</hardwareInterface>
         <hardwareInterface>VelocityJointInterface</hardwareInterface>
       </joint>

File: cob_description/urdf/cob4_torso/torso.urdf.xacro (robot description, xacro)
@@ -12,50 +12,58 @@
     </joint>
     <link name="${name}_base_link">
+      <xacro:default_inertial/>
+<!--
        <xacro:cylinder_inertial radius="0.300" length="0.046" mass="5.0">
         <origin xyz="0.03 0.08 0.01" rpy="0 0 0" />
       </xacro:cylinder_inertial>
+-->
     </link>
     <joint name="${name}_1_joint" type="revolute">
       <origin xyz="0 0 0.04642" rpy="0 0 0"/>
+      <parent link="${name}_base_link"/>
       <child link="${name}_1_link" />
-      <parent link="${name}_base_link"/>
+      <axis xyz="0 0 1" />
       <calibration rising="${torso_1_ref}"/>
-      <axis xyz="0 0 1" />
-      <dynamics damping="0.0" friction="0.0"/>
       <limit effort="100" lower="-6.2831" upper="6.2831" velocity="1.4"/>
     </joint>
     <link name="${name}_1_link">
+      <xacro:default_inertial/>
+<!--
       <xacro:hollow_spherical_cap_inertial r="0.295" h="0.075" t="0.010" mass="6">
-          <!--origin xyz="0.006 0.010 0.110" rpy="0 0 0"/-->
-          <origin xyz="0 0 ${0.075/2}" rpy="0 0 0"/>
+        <origin xyz="0 0 ${0.075/2}" rpy="0 0 0"/>
       </xacro:hollow_spherical_cap_inertial>
+-->
     </link>
     <joint name="${name}_2_joint" type="revolute">
       <origin xyz="0 -0.14734 0.07547" rpy="-0.5236 0 0" />
+      <parent link="${name}_1_link"/>
       <child link="${name}_2_link" />
-      <parent link="${name}_1_link"/>
+      <axis xyz="0 0 1" />
       <calibration rising="${torso_2_ref}"/>
-      <axis xyz="0 0 1" />
-      <dynamics damping="0.0" friction="0.0"/>
       <limit effort="100" lower="-6.2831" upper="6.2831" velocity="1.4"/>
     </joint>
     <link name="${name}_2_link">
-        <xacro:spherical_cap_inertial r="0.295" h="0.075" mass="19.5">
-            <origin xyz="0.034 0.102 0.092" rpy="0.5236 0 0"/>
-        </xacro:spherical_cap_inertial>
+      <xacro:default_inertial/>
+<!--
+      <xacro:spherical_cap_inertial r="0.295" h="0.075" mass="19.5">
+        <origin xyz="0.034 0.102 0.092" rpy="0.5236 0 0"/>
+      </xacro:spherical_cap_inertial>
+-->
     </link>
     <joint name="${name}_3_joint" type="revolute">
       <origin xyz="0 0.09228 0.13477" rpy="0.5236 0 0" />
+      <parent link="${name}_2_link"/>
       <child link="${name}_3_link" />
-      <parent link="${name}_2_link"/>
+      <axis xyz="0 0 1" />
       <calibration rising="${torso_3_ref}"/>
-      <axis xyz="0 0 1" />
-      <dynamics damping="0.0" friction="0.0"/>
       <limit effort="100" lower="-6.2831" upper="6.2831" velocity="1.4"/>
     </joint>
     <link name="${name}_3_link">
-       <xacro:cylinder_inertial radius="0.250" length="0.610" mass="23.8">
+      <xacro:default_inertial/>
+<!--
+      <xacro:cylinder_inertial radius="0.250" length="0.610" mass="23.8">
         <origin xyz="-0.028 0.005 0.233" rpy="0 0 0" />
       </xacro:cylinder_inertial>
+-->
       <visual>
         <origin xyz="0 0 0" rpy="0 0 0" />
@@ -67,6 +75,5 @@
         <origin xyz="0 0 0" rpy="0 0 0" />
         <geometry>
-          <mesh filename="package://cob_description/meshes/cob4_torso/torso_link.dae"/>
-          <!--box size="0.001 0.001 0.001" /-->
+          <mesh filename="package://cob_description/meshes/cob4_torso/torso_link_collision.stl"/>
         </geometry>
       </collision>
@@ -74,6 +81,6 @@
     <joint name="${name}_center_joint" type="fixed">
       <origin xyz="0.0 0.0 0.18566" rpy="0 0 0" />
+      <parent link="${name}_3_link"/>
       <child link="${name}_center_link" />
-      <parent link="${name}_3_link"/>
     </joint>
     <link name="${name}_center_link"/>

Commit message: unify head xacros

File: cob_description/urdf/cob4_head/head.transmission.xacro (robot description, xacro)
@@ -1,35 +1,15 @@
 <?xml version="1.0"?>
 <robot xmlns:xacro="http://www.ros.org/wiki/xacro">
-  <xacro:macro name="head_transmission" params="name">
-    <transmission name="${name}_1_trans">
-      <type>transmission_interface/SimpleTransmission</type>
-      <joint name="${name}_1_joint">
-        <hardwareInterface>PositionJointInterface</hardwareInterface>
-        <hardwareInterface>VelocityJointInterface</hardwareInterface>
-      </joint>
-      <actuator name="${name}_1_motor">
-        <mechanicalReduction>1</mechanicalReduction>
-      </actuator>
-    </transmission>
-    <transmission name="${name}_2_trans">
-      <type>transmission_interface/SimpleTransmission</type>
-      <joint name="${name}_2_joint">
-        <hardwareInterface>PositionJointInterface</hardwareInterface>
-        <hardwareInterface>VelocityJointInterface</hardwareInterface>
-      </joint>
-      <actuator name="${name}_2_motor">
-        <mechanicalReduction>1</mechanicalReduction>
-      </actuator>
-    </transmission>
-    <transmission name="${name}_3_trans">
-      <type>transmission_interface/SimpleTransmission</type>
-      <joint name="${name}_3_joint">
-        <hardwareInterface>PositionJointInterface</hardwareInterface>
-        <hardwareInterface>VelocityJointInterface</hardwareInterface>
-      </joint>
-      <actuator name="${name}_3_motor">
-        <mechanicalReduction>1</mechanicalReduction>
-      </actuator>
-    </transmission>
+  <xacro:include filename="$(find schunk_description)/urdf/common.xacro" />
+  <xacro:macro name="head_transmission" params="name dof1 dof2 dof3">
+    <xacro:if value="${dof1}">
+      <xacro:default_transmission jname="${name}_1"></xacro:default_transmission>
+    </xacro:if>
+    <xacro:if value="${dof2}">
+      <xacro:default_transmission jname="${name}_2"></xacro:default_transmission>
+    </xacro:if>
+    <xacro:if value="${dof3}">
+      <xacro:default_transmission jname="${name}_3"></xacro:default_transmission>
+    </xacro:if>
   </xacro:macro>
 </robot>

File: cob_description/urdf/cob4_head/head.urdf.xacro (robot description, xacro)
@@ -3,5 +3,5 @@
   <xacro:include filename="$(find cob_description)/urdf/cob4_head/head.gazebo.xacro" />
   <xacro:include filename="$(find cob_description)/urdf/cob4_head/head.transmission.xacro" />
-  <xacro:macro name="head" params="parent name *origin">
+  <xacro:macro name="head" params="parent name *origin dof1:=false dof2:=false dof3:=false">
     <joint name="${name}_base_joint" type="fixed">
       <insert_block name="origin" />
@@ -24,11 +24,20 @@
       </collision>
     </link>
-    <joint name="${name}_1_joint" type="revolute">
-      <origin xyz="0 0 0.0305" rpy="0 0 0"/>
-      <parent link="${name}_base_link"/>
-      <child link="${name}_1_link" />
-      <axis xyz="0 0 1" />
-      <limit effort="100" lower="-6.2831" upper="6.2831" velocity="1.4"/>
-    </joint>
+    <xacro:unless value="${dof1}">
+      <joint name="${name}_1_joint" type="fixed">
+        <origin xyz="0 0 0.0305" rpy="0 0 0"/>
+        <parent link="${name}_base_link"/>
+        <child link="${name}_1_link" />
+      </joint>
+    </xacro:unless>
+    <xacro:if value="${dof1}">
+      <joint name="${name}_1_joint" type="revolute">
+        <origin xyz="0 0 0.0305" rpy="0 0 0"/>
+        <parent link="${name}_base_link"/>
+        <child link="${name}_1_link" />
+        <axis xyz="0 0 1" />
+        <limit effort="100" lower="-6.2831" upper="6.2831" velocity="1.4"/>
+      </joint>
+    </xacro:if>
     <link name="${name}_1_link">
       <xacro:default_inertial/>
@@ -46,11 +55,20 @@
       </collision>
     </link>
-    <joint name="${name}_2_joint" type="revolute">
-      <origin xyz="0 -0.07725 0.00439" rpy="0.349 0 0" />
-      <parent link="${name}_1_link"/>
-      <child link="${name}_2_link" />
-      <axis xyz="0 0 1" />
-      <limit effort="100" lower="-6.2831" upper="6.2831" velocity="1.4"/>
-    </joint>
+    <xacro:unless value="${dof2}">
+      <joint name="${name}_2_joint" type="fixed">
+        <origin xyz="0 -0.07725 0.00439" rpy="0.349 0 0" />
+        <parent link="${name}_1_link"/>
+        <child link="${name}_2_link" />
+      </joint>
+    </xacro:unless>
+    <xacro:if value="${dof2}">
+      <joint name="${name}_2_joint" type="revolute">
+        <origin xyz="0 -0.07725 0.00439" rpy="0.349 0 0" />
+        <parent link="${name}_1_link"/>
+        <child link="${name}_2_link" />
+        <axis xyz="0 0 1" />
+        <limit effort="100" lower="-6.2831" upper="6.2831" velocity="1.4"/>
+      </joint>
+    </xacro:if>
     <link name="${name}_2_link">
       <xacro:default_inertial/>
@@ -68,11 +86,20 @@
       </collision>
     </link>
-    <joint name="${name}_3_joint" type="revolute">
-      <origin xyz="0 0.09849 0.04476" rpy="-0.349 0 0" />
-      <parent link="${name}_2_link"/>
-      <child link="${name}_3_link" />
-      <axis xyz="0 0 1" />
-      <limit effort="100" lower="-6.2831" upper="6.2831" velocity="1.4"/>
-    </joint>
+    <xacro:unless value="${dof3}">
+      <joint name="${name}_3_joint" type="fixed">
+        <origin xyz="0 0.09849 0.04476" rpy="-0.349 0 0" />
+        <parent link="${name}_2_link"/>
+        <child link="${name}_3_link" />
+      </joint>
+    </xacro:unless>
+    <xacro:if value="${dof3}">
+      <joint name="${name}_3_joint" type="revolute">
+        <origin xyz="0 0.09849 0.04476" rpy="-0.349 0 0" />
+        <parent link="${name}_2_link"/>
+        <child link="${name}_3_link" />
+        <axis xyz="0 0 1" />
+        <limit effort="100" lower="-6.2831" upper="6.2831" velocity="1.4"/>
+      </joint>
+    </xacro:if>
     <link name="${name}_3_link">
       <xacro:default_inertial/>
@@ -98,5 +125,5 @@
   <!-- extensions -->
   <xacro:head_gazebo name="${name}" />
-  <xacro:head_transmission name="${name}" />
+  <xacro:head_transmission name="${name}" dof1="${dof1}" dof2="${dof2}" dof3="${dof3}" />
   </xacro:macro>
 </robot>

Commit message: unify torso xacros, use default transmission macro

File: cob_description/urdf/cob4_head/head.transmission.xacro (robot description, xacro)
@@ -1,14 +1,14 @@
 <?xml version="1.0"?>
 <robot xmlns:xacro="http://www.ros.org/wiki/xacro">
-  <xacro:include filename="$(find schunk_description)/urdf/common.xacro" />
+  <xacro:include filename="$(find cob_description)/urdf/common.xacro" />
   <xacro:macro name="head_transmission" params="name dof1 dof2 dof3">
     <xacro:if value="${dof1}">
-      <xacro:default_transmission jname="${name}_1"></xacro:default_transmission>
+      <xacro:default_transmission jname="${name}_1"/>
     </xacro:if>
     <xacro:if value="${dof2}">
-      <xacro:default_transmission jname="${name}_2"></xacro:default_transmission>
+      <xacro:default_transmission jname="${name}_2"/>
     </xacro:if>
     <xacro:if value="${dof3}">
-      <xacro:default_transmission jname="${name}_3"></xacro:default_transmission>
+      <xacro:default_transmission jname="${name}_3"/>
     </xacro:if>
   </xacro:macro>

File: cob_description/urdf/cob4_torso/torso.urdf.xacro (robot description, xacro)
@@ -3,5 +3,5 @@
   <xacro:include filename="$(find cob_description)/urdf/cob4_torso/torso.gazebo.xacro" />
   <xacro:include filename="$(find cob_description)/urdf/cob4_torso/torso.transmission.xacro" />
-  <xacro:macro name="torso" params="parent name *origin">
+  <xacro:macro name="torso" params="parent name *origin" dof1:=false dof2:=false dof3:=false">
     <joint name="${name}_base_joint" type="fixed">
       <insert_block name="origin" />
@@ -29,9 +29,20 @@
       </collision>
     </link>
-    <joint name="${name}_1_joint" type="fixed">
-      <origin xyz="0 0 0.04642" rpy="0 0 0"/>
-      <parent link="${name}_base_link"/>
-      <child link="${name}_1_link" />
-    </joint>
+    <xacro:unless value="${dof1}">
+      <joint name="${name}_1_joint" type="fixed">
+        <origin xyz="0 0 0.04642" rpy="0 0 0"/>
+        <parent link="${name}_base_link"/>
+        <child link="${name}_1_link" />
+      </joint>
+    </xacro:unless>
+    <xacro:if value="${dof1}">
+      <joint name="${name}_1_joint" type="revolute">
+        <origin xyz="0 0 0.04642" rpy="0 0 0"/>
+        <parent link="${name}_base_link"/>
+        <child link="${name}_1_link" />
+        <axis xyz="0 0 1" />
+        <limit effort="100" lower="-6.2831" upper="6.2831" velocity="1.4"/>
+      </joint>
+    </xacro:if>
     <link name="${name}_1_link">
       <xacro:default_inertial/>
@@ -54,11 +65,20 @@
       </collision>
     </link>
-    <joint name="${name}_2_joint" type="revolute">
-      <origin xyz="0 0.14734 0.07547" rpy="0.5236 0 0" />
-      <parent link="${name}_1_link"/>
-      <child link="${name}_2_link" />
-      <axis xyz="0 0 1" />
-      <limit effort="100" lower="-6.2831" upper="6.2831" velocity="1.4"/>
-    </joint>
+    <xacro:unless value="${dof2}">
+      <joint name="${name}_2_joint" type="fixed">
+        <origin xyz="0 0.14734 0.07547" rpy="0.5236 0 0" />
+        <parent link="${name}_1_link"/>
+        <child link="${name}_2_link" />
+      </joint>
+    </xacro:unless>
+    <xacro:if value="${dof2}">
+      <joint name="${name}_2_joint" type="revolute">
+        <origin xyz="0 0.14734 0.07547" rpy="0.5236 0 0" />
+        <parent link="${name}_1_link"/>
+        <child link="${name}_2_link" />
+        <axis xyz="0 0 1" />
+        <limit effort="100" lower="-6.2831" upper="6.2831" velocity="1.4"/>
+      </joint>
+    </xacro:if>
     <link name="${name}_2_link">
       <xacro:default_inertial/>
@@ -81,11 +101,20 @@
       </collision>
     </link>
-    <joint name="${name}_3_joint" type="revolute">
-      <origin xyz="0 -0.09228 0.13477" rpy="-0.5236 0 0" />
-      <parent link="${name}_2_link"/>
-      <child link="${name}_3_link" />
-      <axis xyz="0 0 1" />
-      <limit effort="100" lower="-6.2831" upper="6.2831" velocity="1.4"/>
-    </joint>
+    <xacro:unless value="${dof3}">
+      <joint name="${name}_3_joint" type="fixed">
+        <origin xyz="0 -0.09228 0.13477" rpy="-0.5236 0 0" />
+        <parent link="${name}_2_link"/>
+        <child link="${name}_3_link" />
+      </joint>
+    </xacro:unless>
+    <xacro:if value="${dof3}">
+      <joint name="${name}_3_joint" type="revolute">
+        <origin xyz="0 -0.09228 0.13477" rpy="-0.5236 0 0" />
+        <parent link="${name}_2_link"/>
+        <child link="${name}_3_link" />
+        <axis xyz="0 0 1" />
+        <limit effort="100" lower="-6.2831" upper="6.2831" velocity="1.4"/>
+      </joint>
+    </xacro:if>
     <link name="${name}_3_link">
       <xacro:default_inertial/>
@@ -130,5 +159,5 @@
     <!-- extensions -->
     <xacro:torso_gazebo name="torso" />
-    <xacro:torso_transmission name="torso" />
+    <xacro:torso_transmission name="torso" dof1="${dof1}" dof2="${dof2}" dof3="${dof3}" />
   </xacro:macro>
 </robot>
