Commit message: Fixed kinematic error

File: cob_description/urdf/cob4_head/head.urdf.xacro (robot description, xacro)
@@ -52,5 +52,5 @@
 		</link>
 		<joint name="head_3_joint" type="revolute">
-		  <origin xyz="0 0.08001 0.06809" rpy="0.349 0 0" />
+		  <origin xyz="0 0.04668 0.0976" rpy="0.349 0 0" />
 		  <child link="head_3_link" />
 		  <parent link="head_2_link"/>

File: cob_description/urdf/cob4_torso/torso.urdf.xacro (robot description, xacro)
@@ -52,5 +52,5 @@
 		</link>
 		<joint name="torso_3_joint" type="revolute">
-		  <origin xyz="0 0.06223 0.15206" rpy="0.5236 0 0" />
+		  <origin xyz="0 0.09228 0.13477" rpy="0.5236 0 0" />
 		  <child link="torso_3_link" />
 		  <parent link="torso_2_link"/>

Commit message: New head_center_link

File: cob_description/urdf/cob4_head/head.urdf.xacro (robot description, xacro)
@@ -77,4 +77,16 @@
       </collision>
     </link>
+    <joint name="head_center_joint" type="fixed">
+      <origin xyz="0.0 0.0 -0.28247" rpy="0 0 0" />
+      <child link="head_center_link" />
+      <parent link="head_3_link"/>
+    </joint>
+    <link name="head_center_link">
+      <inertial>
+        <origin xyz="0 0 0" rpy="0 0 0"/>
+        <mass value="0.1"/>
+        <inertia ixx="0.01" ixy="0" ixz="0" iyy="0.01" iyz="0" izz="0.01" />
+      </inertial>
+    </link>
   <!-- extensions -->
   <xacro:head_gazebo name="${name}" />

Commit message: use correct mesh for collision geometry

File: cob_description/urdf/cob4_head/head.urdf.xacro (robot description, xacro)
@@ -59,20 +59,21 @@
     <link name="head_3_link">
       <inertial>
-      <mass value="1" />
-      <origin xyz="0 0 0" />
-      <inertia ixx="0.01" ixy="0" ixz="0" iyy="0.01" iyz="0" izz="0.01" />
+        <mass value="1" />
+        <origin xyz="0 0 0" />
+        <inertia ixx="0.01" ixy="0" ixz="0" iyy="0.01" iyz="0" izz="0.01" />
       </inertial>
       <visual>
-      <origin xyz="0 0 0" rpy="0 0 0" />
-      <geometry>
-        <mesh filename="package://cob_description/meshes/cob4_head/head_link.stl"/>
-      </geometry>
-      <material name="IPA/LightGrey"/>
+        <origin xyz="0 0 0" rpy="0 0 0" />
+        <geometry>
+          <mesh filename="package://cob_description/meshes/cob4_head/head_link.stl"/>
+        </geometry>
+        <material name="IPA/LightGrey"/>
       </visual>
       <collision>
-      <origin xyz="0 0 0" rpy="0 0 0" />
-      <geometry>
-        <box size="0.001 0.001 0.001" />
-      </geometry>
+        <origin xyz="0 0 0" rpy="0 0 0" />
+        <geometry>
+          <mesh filename="package://cob_description/meshes/cob4_head/head_link.stl"/>
+          <!--box size="0.001 0.001 0.001" /-->
+        </geometry>
       </collision>
     </link>
@@ -82,11 +83,5 @@
       <parent link="head_3_link"/>
     </joint>
-    <link name="head_center_link">
-      <inertial>
-        <origin xyz="0 0 0" rpy="0 0 0"/>
-        <mass value="0.1"/>
-        <inertia ixx="0.01" ixy="0" ixz="0" iyy="0.01" iyz="0" izz="0.01" />
-      </inertial>
-    </link>
+    <link name="head_center_link"/>
   <!-- extensions -->
   <xacro:head_gazebo name="${name}" />

File: cob_description/urdf/cob4_torso/torso.urdf.xacro (robot description, xacro)
@@ -68,5 +68,6 @@
         <origin xyz="0 0 0" rpy="0 0 0" />
         <geometry>
-          <box size="0.001 0.001 0.001" />
+          <mesh filename="package://cob_description/meshes/cob4_torso/torso_link.stl"/>
+          <!--box size="0.001 0.001 0.001" /-->
         </geometry>
       </collision>

Commit message: recalculated head joint positions

File: cob_description/urdf/cob4_head/head.urdf.xacro (robot description, xacro)
@@ -48,5 +48,5 @@
     </link>
     <joint name="${name}_2_joint" type="revolute">
-      <origin xyz="0 -0.07725 -0.00439" rpy="-0.349 0 0" />
+      <origin xyz="0 -0.07725 -0.00439" rpy="0.349 0 0" />
       <parent link="${name}_1_link"/>
       <child link="${name}_2_link" />
@@ -71,5 +71,5 @@
     </link>
     <joint name="${name}_3_joint" type="revolute">
-      <origin xyz="0 0.04668 0.0976" rpy="0.349 0 0" />
+      <origin xyz="0 0.09849 0.04476" rpy="-0.349 0 0" />
       <parent link="${name}_2_link"/>
       <child link="${name}_3_link" />

Commit message: check head urdf model

File: cob_description/urdf/cob4_head/head.urdf.xacro (robot description, xacro)
@@ -47,5 +47,5 @@
     </link>
     <joint name="${name}_2_joint" type="revolute">
-      <origin xyz="0 -0.07725 -0.00439" rpy="0.349 0 0" />
+      <origin xyz="0 0.07725 -0.00439" rpy="-0.349 0 0" />
       <parent link="${name}_1_link"/>
       <child link="${name}_2_link" />
@@ -69,5 +69,5 @@
     </link>
     <joint name="${name}_3_joint" type="revolute">
-      <origin xyz="0 0.09849 0.04476" rpy="-0.349 0 0" />
+      <origin xyz="0 -0.09849 0.04476" rpy="0.349 0 0" />
       <parent link="${name}_2_link"/>
       <child link="${name}_3_link" />

Commit message: adapt head urdf to hardware kinematics

File: cob_description/urdf/cob4_head/head.urdf.xacro (robot description, xacro)
@@ -47,5 +47,5 @@
     </link>
     <joint name="${name}_2_joint" type="revolute">
-      <origin xyz="0 0.07725 -0.00439" rpy="-0.349 0 0" />
+      <origin xyz="0 -0.07725 0.00439" rpy="0.349 0 0" />
       <parent link="${name}_1_link"/>
       <child link="${name}_2_link" />
@@ -69,5 +69,5 @@
     </link>
     <joint name="${name}_3_joint" type="revolute">
-      <origin xyz="0 -0.09849 0.04476" rpy="0.349 0 0" />
+      <origin xyz="0 0.09849 0.04476" rpy="-0.349 0 0" />
       <parent link="${name}_2_link"/>
       <child link="${name}_3_link" />

Commit message: added head_cam frame to urdf

File: cob_description/urdf/cob4_head/head.urdf.xacro (robot description, xacro)
@@ -3,4 +3,5 @@
   <xacro:include filename="$(find cob_description)/urdf/cob4_head/head.gazebo.xacro" />
   <xacro:include filename="$(find cob_description)/urdf/cob4_head/head.transmission.xacro" />
+  <xacro:include filename="$(find cob_description)/urdf/sensors/head_cam.urdf.xacro" />
   <xacro:macro name="head" params="parent name *origin">
     <joint name="${name}_base_joint" type="fixed">
@@ -96,4 +97,7 @@
     </joint>
     <link name="${name}_center_link"/>
+    <xacro:head_cam name="${name}_cam" parent="${name}_3_link" ros_topic="${name}_cam">
+      <origin xyz="${head_cam_x} ${head_cam_y} ${head_cam_z}" rpy="${head_cam_roll} ${head_cam_pitch} ${head_cam_yaw}" />
+    </xacro:head_cam>
   <!-- extensions -->
   <xacro:head_gazebo name="${name}" />

File: cob_description/urdf/cob4_head/head_static.urdf.xacro (robot description, xacro)
@@ -3,4 +3,5 @@
   <xacro:include filename="$(find cob_description)/urdf/cob4_head/head.gazebo.xacro" />
   <xacro:include filename="$(find cob_description)/urdf/cob4_head/head.transmission.xacro" />
+  <xacro:include filename="$(find cob_description)/urdf/sensors/head_cam.urdf.xacro" />
   <xacro:macro name="head" params="parent name *origin">
     <joint name="${name}_base_joint" type="fixed">
@@ -90,4 +91,7 @@
     </joint>
     <link name="${name}_center_link"/>
+    <xacro:head_cam name="${name}_cam" parent="${name}_3_link" ros_topic="${name}_cam">
+      <origin xyz="${head_cam_x} ${head_cam_y} ${head_cam_z}" rpy="${head_cam_roll} ${head_cam_pitch} ${head_cam_yaw}" />
+    </xacro:head_cam>
   <!-- extensions -->
   <xacro:head_gazebo name="${name}" />

Commit message: renamed xacro and files(head_cam -> usb_cam)

File: cob_description/urdf/cob4_head/head.urdf.xacro (robot description, xacro)
@@ -3,5 +3,5 @@
   <xacro:include filename="$(find cob_description)/urdf/cob4_head/head.gazebo.xacro" />
   <xacro:include filename="$(find cob_description)/urdf/cob4_head/head.transmission.xacro" />
-  <xacro:include filename="$(find cob_description)/urdf/sensors/head_cam.urdf.xacro" />
+  <xacro:include filename="$(find cob_description)/urdf/sensors/usb_cam.urdf.xacro" />
   <xacro:macro name="head" params="parent name *origin">
     <joint name="${name}_base_joint" type="fixed">
@@ -97,7 +97,7 @@
     </joint>
     <link name="${name}_center_link"/>
-    <xacro:head_cam name="${name}_cam" parent="${name}_3_link" ros_topic="${name}_cam">
+    <xacro:usb_cam name="${name}_cam" parent="${name}_3_link" ros_topic="${name}_cam">
       <origin xyz="${head_cam_x} ${head_cam_y} ${head_cam_z}" rpy="${head_cam_roll} ${head_cam_pitch} ${head_cam_yaw}" />
-    </xacro:head_cam>
+    </xacro:usb_cam>
   <!-- extensions -->
   <xacro:head_gazebo name="${name}" />

File: cob_description/urdf/cob4_head/head_static.urdf.xacro (robot description, xacro)
@@ -3,5 +3,5 @@
   <xacro:include filename="$(find cob_description)/urdf/cob4_head/head.gazebo.xacro" />
   <xacro:include filename="$(find cob_description)/urdf/cob4_head/head.transmission.xacro" />
-  <xacro:include filename="$(find cob_description)/urdf/sensors/head_cam.urdf.xacro" />
+  <xacro:include filename="$(find cob_description)/urdf/sensors/usb_cam.urdf.xacro" />
   <xacro:macro name="head" params="parent name *origin">
     <joint name="${name}_base_joint" type="fixed">
@@ -91,7 +91,7 @@
     </joint>
     <link name="${name}_center_link"/>
-    <xacro:head_cam name="${name}_cam" parent="${name}_3_link" ros_topic="${name}_cam">
+    <xacro:usb_cam name="${name}_cam" parent="${name}_3_link" ros_topic="${name}_cam">
       <origin xyz="${head_cam_x} ${head_cam_y} ${head_cam_z}" rpy="${head_cam_roll} ${head_cam_pitch} ${head_cam_yaw}" />
-    </xacro:head_cam>
+    </xacro:usb_cam>
   <!-- extensions -->
   <xacro:head_gazebo name="${name}" />

File: cob_description/urdf/sensors/usb_cam.gazebo.xacro (robot description, xacro)
@@ -1,5 +1,5 @@
 <?xml version="1.0"?>
 <robot xmlns:xacro="http://www.ros.org/wiki/xacro">
-  <xacro:macro name="head_cam_gazebo" params="name ros_topic">
+  <xacro:macro name="usb_cam_gazebo" params="name ros_topic">
     <gazebo reference="${name}_frame">
     <sensor type="camera" name="${name}">

File: cob_description/urdf/sensors/usb_cam.urdf.xacro (robot description, xacro)
@@ -1,6 +1,6 @@
 <?xml version="1.0"?>
 <robot xmlns:xacro="http://www.ros.org/wiki/xacro">
-  <xacro:include filename="$(find cob_description)/urdf/sensors/head_cam.gazebo.xacro" />
-  <xacro:macro name="head_cam" params="name parent ros_topic *origin">
+  <xacro:include filename="$(find cob_description)/urdf/sensors/usb_cam.gazebo.xacro" />
+  <xacro:macro name="usb_cam" params="name parent ros_topic *origin">
     <joint name="${name}_joint" type="fixed">
       <insert_block name="origin" />
@@ -34,5 +34,5 @@
     <link name="${name}_frame"/>
     <!-- extensions -->
-    <xacro:head_cam_gazebo name="${name}" ros_topic="${ros_topic}" />
+    <xacro:usb_cam_gazebo name="${name}" ros_topic="${ros_topic}" />
   </xacro:macro>
 </robot>

Commit message: move sensors from head xacro to robot xacro

File: cob_description/urdf/cob4_head/head.urdf.xacro (robot description, xacro)
@@ -3,5 +3,4 @@
   <xacro:include filename="$(find cob_description)/urdf/cob4_head/head.gazebo.xacro" />
   <xacro:include filename="$(find cob_description)/urdf/cob4_head/head.transmission.xacro" />
-  <xacro:include filename="$(find cob_description)/urdf/sensors/usb_cam.urdf.xacro" />
   <xacro:macro name="head" params="parent name *origin">
     <joint name="${name}_base_joint" type="fixed">
@@ -97,7 +96,4 @@
     </joint>
     <link name="${name}_center_link"/>
-    <xacro:usb_cam name="${name}_cam" parent="${name}_3_link" ros_topic="${name}_cam">
-      <origin xyz="${head_cam_x} ${head_cam_y} ${head_cam_z}" rpy="${head_cam_roll} ${head_cam_pitch} ${head_cam_yaw}" />
-    </xacro:usb_cam>
   <!-- extensions -->
   <xacro:head_gazebo name="${name}" />

File: cob_description/urdf/cob4_head/head_static.urdf.xacro (robot description, xacro)
@@ -3,5 +3,4 @@
   <xacro:include filename="$(find cob_description)/urdf/cob4_head/head.gazebo.xacro" />
   <xacro:include filename="$(find cob_description)/urdf/cob4_head/head.transmission.xacro" />
-  <xacro:include filename="$(find cob_description)/urdf/sensors/usb_cam.urdf.xacro" />
   <xacro:macro name="head" params="parent name *origin">
     <joint name="${name}_base_joint" type="fixed">
@@ -91,7 +90,4 @@
     </joint>
     <link name="${name}_center_link"/>
-    <xacro:usb_cam name="${name}_cam" parent="${name}_3_link" ros_topic="${name}_cam">
-      <origin xyz="${head_cam_x} ${head_cam_y} ${head_cam_z}" rpy="${head_cam_roll} ${head_cam_pitch} ${head_cam_yaw}" />
-    </xacro:usb_cam>
   <!-- extensions -->
   <xacro:head_gazebo name="${name}" />

Commit message: use latest xacro syntax

File: cob_description/urdf/cob4_head/head.urdf.xacro (robot description, xacro)
@@ -5,5 +5,5 @@
   <xacro:macro name="head" params="parent name *origin dof1:=false dof2:=false dof3:=false">
     <joint name="${name}_base_joint" type="fixed">
-      <insert_block name="origin" />
+      <xacro:insert_block name="origin" />
       <child link="${name}_base_link" />
       <parent link="${parent}"/>

File: cob_description/urdf/cob4_sensorring/sensorring.urdf.xacro (robot description, xacro)
@@ -5,5 +5,5 @@
   <xacro:macro name="sensorring" params="parent name *origin">
     <joint name="${name}_base_joint" type="fixed">
-      <insert_block name="origin" />
+      <xacro:insert_block name="origin" />
       <parent link="${parent}"/>
       <child link="${name}_base_link" />

File: cob_description/urdf/cob4_torso/torso.urdf.xacro (robot description, xacro)
@@ -5,5 +5,5 @@
   <xacro:macro name="torso" params="parent name *origin" dof1:=false dof2:=false dof3:=false">
     <joint name="${name}_base_joint" type="fixed">
-      <insert_block name="origin" />
+      <xacro:insert_block name="origin" />
       <parent link="${parent}"/>
       <child link="${name}_base_link" />

File: cob_description/urdf/common.xacro (robot description, xacro)
@@ -1,5 +1,5 @@
 <?xml version="1.0"?>
 <robot xmlns:xacro="http://www.ros.org/wiki/xacro">
-  <property name="M_PI" value="3.1415926535897931" />
+  <xacro:property name="M_PI" value="3.1415926535897931" />
   <!-- geometry macros for modeling geometric primitives with according meshes -->
   <xacro:macro name="sphere_geometry" params="radius">
@@ -22,5 +22,5 @@
     <inertial>
       <mass value="${mass}" />
-      <insert_block name="origin" />
+      <xacro:insert_block name="origin" />
       <inertia ixx="${0.4 * mass * radius * radius}" ixy="0.0" ixz="0.0"
         iyy="${0.4 * mass * radius * radius}" iyz="0.0"
@@ -31,5 +31,5 @@
     <inertial>
       <mass value="${mass}" />
-      <insert_block name="origin" />
+      <xacro:insert_block name="origin" />
       <inertia ixx="${0.0833333 * mass * (3 * radius * radius + length * length)}" ixy="0.0" ixz="0.0"
         iyy="${0.0833333 * mass * (3 * radius * radius + length * length)}" iyz="0.0"
@@ -40,5 +40,5 @@
     <inertial>
       <mass value="${mass}" />
-      <insert_block name="origin" />
+      <xacro:insert_block name="origin" />
       <inertia ixx="${0.0833333 * mass * (y*y + z*z)}" ixy="0.0" ixz="0.0"
         iyy="${0.0833333 * mass * (x*x + z*z)}" iyz="0.0"
@@ -49,5 +49,5 @@
     <inertial>
       <mass value="${mass}" />
-      <insert_block name="origin" />
+      <xacro:insert_block name="origin" />
       <inertia ixx="${(-3*h*h*h/20+3*h*h*r/4-4*h*r*r/3+r*r*r)*3*mass/(3*r-h)+(3/4*(h-2*r)*(h-2*r)/(3*r-h))*(3/4*(h-2*r)*(h-2*r)/(3*r-h))}" ixy="0.0" ixz="0.0"
         iyy="${(-3*h*h*h/20+3*h*h*r/4-4*h*r*r/3+r*r*r)*3*mass/(3*r-h)+(3/4*(h-2*r)*(h-2*r)/(3*r-h))*(3/4*(h-2*r)*(h-2*r)/(3*r-h))}" iyz="0.0"
@@ -59,5 +59,5 @@
     <inertial>
       <mass value="${mass}" />
-      <insert_block name="origin" />
+      <xacro:insert_block name="origin" />
       <inertia ixx="${mass/20*(20*h*h*h*r-10*h*h*h*t-60*h*h*r*r+30*h*h*r*t+120*h*r*r*r-120*h*r*r*t+60*h*r*t*t-15*h*t*t*t-60*r*r*r*t+100*r*r*t*t-65*r*t*t*t+16*t*t*t*t)/(2*t*t*-3*r*t-3*h*t+6*h*r)+(3/4*(t-2*r)*(2*r*r-4*r*r+2*r*t-t*t)/(6*r*r-3*r*t-3*r*t+2*t*t))*(3/4*(t-2*r)*(2*r*r-4*r*r+2*r*t-t*t)/(6*r*r-3*r*t-3*r*t+2*t*t))}" ixy="0.0" ixz="0.0"
         iyy="${mass/20*(20*h*h*h*r-10*h*h*h*t-60*h*h*r*r+30*h*h*r*t+120*h*r*r*r-120*h*r*r*t+60*h*r*t*t-15*h*t*t*t-60*r*r*r*t+100*r*r*t*t-65*r*t*t*t+16*t*t*t*t)/(2*t*t*-3*r*t-3*h*t+6*h*r)+(3/4*(t-2*r)*(2*r*r-4*r*r+2*r*t-t*t)/(6*r*r-3*r*t-3*r*t+2*t*t))*(3/4*(t-2*r)*(2*r*r-4*r*r+2*r*t-t*t)/(6*r*r-3*r*t-3*r*t+2*t*t))}" iyz="0.0"

File: raw_description/urdf/torso/torso.urdf.xacro (robot description, xacro)
@@ -6,5 +6,5 @@
     <!-- joint between base_link and torso_tilt_link -->
     <joint name="${name}_0_joint" type="fixed" >
-      <insert_block name="origin" />
+      <xacro:insert_block name="origin" />
       <parent link="${parent}" />
       <child link="${name}_0_link" />
