Commit message: fixed urdf

File: raw_description/urdf/base_short/base.urdf.xacro (robot description, xacro)
@@ -15,8 +15,8 @@
   <!-- all simplified collision geometry are hand approximated from CAD model, sometimes from respective bounding boxes -->
   <property name="caster_offset_x" value="0.228" />  <!--modify here-->
-  <property name="caster_offset_y_bl" value="0.134" />
-  <property name="caster_offset_y_br" value="0.186" />
-  <property name="caster_offset_y_fl" value="0.186" />
-  <property name="caster_offset_y_fr" value="0.134" />
+  <property name="caster_offset_y_bl" value="0.186" />
+  <property name="caster_offset_y_br" value="0.134" />
+  <property name="caster_offset_y_fl" value="0.134" />
+  <property name="caster_offset_y_fr" value="0.186" />
   <property name="caster_offset_z" value="0.09" />
   <property name="battery_offset_x_f" value="0.0" />
@@ -223,14 +223,14 @@
     <!-- all four caster macros -->
     <xacro:cob_caster suffix="fl" parent="${name}_link" ref_position="${cal_caster_fl - M_PI/4}" >
-      <origin xyz="${-caster_offset_x} ${-caster_offset_y_bl} ${caster_offset_z}" rpy="0 0 0" />
+      <origin xyz="${caster_offset_x} ${caster_offset_y_bl} ${caster_offset_z}" rpy="0 0 0" />
     </xacro:cob_caster>
     <xacro:cob_caster suffix="fr" parent="${name}_link" ref_position="${cal_caster_fr - M_PI/4}" >
-      <origin xyz="${-caster_offset_x} ${caster_offset_y_br} ${caster_offset_z}" rpy="0 0 0" />
+      <origin xyz="${caster_offset_x} ${-caster_offset_y_br} ${caster_offset_z}" rpy="0 0 0" />
     </xacro:cob_caster>
     <xacro:cob_caster suffix="bl" parent="${name}_link" ref_position="${cal_caster_bl - M_PI / 4 + M_PI}" >
-      <origin xyz="${caster_offset_x} ${-caster_offset_y_fl} ${caster_offset_z}" rpy=" 0 0 0" />
+      <origin xyz="${-caster_offset_x} ${caster_offset_y_fl} ${caster_offset_z}" rpy=" 0 0 0" />
     </xacro:cob_caster>
     <xacro:cob_caster suffix="br" parent="${name}_link" ref_position="${cal_caster_br - M_PI / 4 + M_PI}"  >
-      <origin xyz="${caster_offset_x} ${caster_offset_y_fr} ${caster_offset_z}" rpy="0 0 0" />
+      <origin xyz="${-caster_offset_x} ${-caster_offset_y_fr} ${caster_offset_z}" rpy="0 0 0" />
     </xacro:cob_caster>
    <!-- cam3d -->

Commit message: urdf fix

File: raw_description/urdf/base_short/base.urdf.xacro (robot description, xacro)
@@ -223,14 +223,14 @@
     <!-- all four caster macros -->
     <xacro:cob_caster suffix="fl" parent="${name}_link" ref_position="${cal_caster_fl - M_PI/4}" >
-      <origin xyz="${-caster_offset_x} ${-caster_offset_y_bl} ${caster_offset_z}" rpy="0 0 0" />
+      <origin xyz="${caster_offset_x} ${caster_offset_y_bl} ${caster_offset_z}" rpy="0 0 0" />
     </xacro:cob_caster>
     <xacro:cob_caster suffix="fr" parent="${name}_link" ref_position="${cal_caster_fr - M_PI/4}" >
-      <origin xyz="${-caster_offset_x} ${caster_offset_y_br} ${caster_offset_z}" rpy="0 0 0" />
+      <origin xyz="${caster_offset_x} ${-caster_offset_y_br} ${caster_offset_z}" rpy="0 0 0" />
     </xacro:cob_caster>
     <xacro:cob_caster suffix="bl" parent="${name}_link" ref_position="${cal_caster_bl - M_PI / 4 + M_PI}" >
-      <origin xyz="${caster_offset_x} ${-caster_offset_y_fl} ${caster_offset_z}" rpy=" 0 0 0" />
+      <origin xyz="${-caster_offset_x} ${caster_offset_y_fl} ${caster_offset_z}" rpy=" 0 0 0" />
     </xacro:cob_caster>
     <xacro:cob_caster suffix="br" parent="${name}_link" ref_position="${cal_caster_br - M_PI / 4 + M_PI}"  >
-      <origin xyz="${caster_offset_x} ${caster_offset_y_fr} ${caster_offset_z}" rpy="0 0 0" />
+      <origin xyz="${-caster_offset_x} ${-caster_offset_y_fr} ${caster_offset_z}" rpy="0 0 0" />
     </xacro:cob_caster>
    <!-- cam3d -->

Commit message: raw_description: added laser calibration data for base_short

File: raw_description/urdf/base_short/base.urdf.xacro (robot description, xacro)
@@ -4,4 +4,5 @@
   <xacro:include filename="$(find raw_description)/urdf/base_short/base.gazebo.xacro" />
   <xacro:include filename="$(find raw_description)/urdf/base_short/base.transmission.xacro" />
+  <xacro:include filename="$(find cob_hardware_config)/raw3-3/urdf/properties.urdf.xacro" />
   <!-- sensors -->
   <xacro:include filename="$(find cob_description)/urdf/sensors/kinect.urdf.xacro" />
@@ -192,9 +193,9 @@
     <!-- base laser front -->
     <xacro:sick_s300_laser_v0 name="${name}_laser_front" parent="${name}" ros_topic="scan_front_raw" update_rate="10" min_angle="-2.3562" max_angle="2.3562" >
-      <origin xyz="${base_laser_x} ${-base_laser_y_front} ${base_laser_z}" rpy="${M_PI} 0 ${-M_PI/4}" />
+      <origin xyz="${laser_front_x} ${laser_front_y} ${base_laser_z}" rpy="${M_PI} 0 ${laser_front_yaw}" />
     </xacro:sick_s300_laser_v0>
     <!-- base laser rear -->
     <xacro:sick_s300_laser_v0 name="${name}_laser_rear" parent="${name}" ros_topic="scan_rear_raw" update_rate="10" min_angle="-2.3562" max_angle="2.3562" >
-      <origin xyz="${-base_laser_x} ${base_laser_y_back} ${base_laser_z}" rpy="${M_PI} 0 ${-5*M_PI/4}" />
+      <origin xyz="${laser_rear_x} ${laser_rear_y} ${base_laser_z}" rpy="${M_PI} 0 ${laser_rear_yaw}" />
     </xacro:sick_s300_laser_v0>
     <!-- battery-->

Commit message: fixed copy paste error for base_short laser mounting position

File: raw_description/urdf/base_short/base.urdf.xacro (robot description, xacro)
@@ -102,5 +102,5 @@
     <!-- base laser rear -->
     <xacro:sick_s300_laser_v0 name="${name}_laser_rear" parent="${name}" ros_topic="scan_rear_raw" update_rate="10" min_angle="-2.3562" max_angle="2.3562" >
-      <origin xyz="${laser_front_x} ${laser_front_y} ${laser_front_z}" rpy="${laser_front_roll} ${laser_front_pitch} ${laser_front_yaw}" />
+      <origin xyz="${laser_rear_x} ${laser_rear_y} ${laser_rear_z}" rpy="${laser_rear_roll} ${laser_rear_pitch} ${laser_rear_yaw}" />
     </xacro:sick_s300_laser_v0>
     <!-- cam3d -->

Commit message: Changed raw model to box.

File: raw_description/urdf/base_short/base.urdf.xacro (robot description, xacro)
@@ -70,5 +70,6 @@
         <origin xyz="0 0 0.209" rpy="0 0 0" />
         <geometry>
-          <mesh filename="package://raw_description/meshes/base/raw_base_short.dae"/>
+          <!-- <mesh filename="package://raw_description/meshes/base/raw_base_short.dae"/> -->
+          <box size="0.688 0.503 0.096"/>
         </geometry>
       </visual>
@@ -76,6 +77,6 @@
         <origin xyz="0 0 0.209" rpy="0 0 0" />
         <geometry>
-          <mesh filename="package://raw_description/meshes/base/raw_base_short.stl"/>
-          <!--box size="0.758 0.573 0.096"/-->
+          <!-- <mesh filename="package://raw_description/meshes/base/raw_base_short.stl"/> -->
+          <box size="0.678 0.493 0.096"/>
         </geometry>
       </collision>
