Commit message: Added sensors to cob4 description

File: cob_description/urdf/cob4_base/base.gazebo.xacro (robot description, xacro)
@@ -32,5 +32,5 @@
 			</plugin>
 		</sensor>
-		<material>IPA/DarkGrey</material>
+		<material>IPA/LightGrey</material>
 	</gazebo>
     <gazebo>

File: cob_description/urdf/cob4_base/base.urdf.xacro (robot description, xacro)
@@ -53,5 +53,5 @@
 		<link name="base_link">
 			<inertial>
-				<mass value="50" />
+				<mass value="100" />
 				<origin xyz="0 0 0" />
 				<inertia ixx="5.652232699207" ixy="-0.009719934438" ixz="1.293988226423"
@@ -69,6 +69,6 @@
 				<origin xyz="0 0 0.05" rpy="0 0 3.14159" />
 				<geometry>
-					<mesh filename="package://cob_description/meshes/cob4_base/base_link.stl"/>
-					<!--box size="0.01 0.01 0.01" /-->
+					<!--mesh filename="package://cob_description/meshes/cob4_base/base_link.stl"/-->
+					<box size="0.01 0.01 0.01" />
 				</geometry>
 			</collision>

File: cob_description/urdf/cob4_head/head.urdf.xacro (robot description, xacro)
@@ -15,5 +15,5 @@
 			<inertial>
 				<origin xyz="0 0 0" rpy="0 0 0"/>
-				<mass value="0.1"/>
+				<mass value="1"/>
 				<inertia ixx="0.01" ixy="0" ixz="0" iyy="0.01" iyz="0" izz="0.01" />
 			</inertial>
@@ -31,5 +31,5 @@
 			<inertial>
 				<origin xyz="0 0 0" rpy="0 0 0"/>
-				<mass value="0.1"/>
+				<mass value="1"/>
 				<inertia ixx="0.01" ixy="0" ixz="0" iyy="0.01" iyz="0" izz="0.01" />
 			</inertial>
@@ -47,5 +47,5 @@
 			<inertial>
 				<origin xyz="0 0 0" rpy="0 0 0"/>
-				<mass value="0.1"/>
+				<mass value="1"/>
 				<inertia ixx="0.01" ixy="0" ixz="0" iyy="0.01" iyz="0" izz="0.01" />
 			</inertial>
@@ -62,5 +62,5 @@
 		<link name="head_3_link">
 		  <inertial>
-			<mass value="10" />
+			<mass value="1" />
 			<origin xyz="0 0 0" />
 			<inertia ixx="5.652232699207" ixy="-0.009719934438" ixz="1.293988226423"

File: cob_description/urdf/cob4_torso/torso.urdf.xacro (robot description, xacro)
@@ -6,4 +6,6 @@
 	<include filename="$(find cob_description)/urdf/cob4_torso/torso.gazebo.xacro" />
 	<include filename="$(find cob_description)/urdf/cob4_torso/torso.transmission.xacro" />
+	<include filename="$(find cob_description)/urdf/sensors/kinect.urdf.xacro" />
+	<include filename="$(find cob_description)/urdf/sensors/softkinetic.urdf.xacro" />
 	<xacro:macro name="torso" params="parent name *origin">
 		<joint name="torso_base_joint" type="fixed">
@@ -15,6 +17,6 @@
 			<inertial>
 				<origin xyz="0 0 0" rpy="0 0 0"/>
-				<mass value="0.1"/>
-				<inertia ixx="0.01" ixy="0" ixz="0" iyy="0.01" iyz="0" izz="0.01" />
+				<mass value="1"/>
+				<inertia ixx="0.01" ixy="0" ixz="0" iyy="0" iyz="0" izz="0" />
 			</inertial>
 		</link>
@@ -31,5 +33,5 @@
 			<inertial>
 				<origin xyz="0 0 0" rpy="0 0 0"/>
-				<mass value="2"/>
+				<mass value="5"/>
 				<inertia ixx="0.01" ixy="0" ixz="0" iyy="0.01" iyz="0" izz="0.01" />
 			</inertial>
@@ -47,5 +49,5 @@
 			<inertial>
 				<origin xyz="0 0 0" rpy="0 0 0"/>
-				<mass value="2"/>
+				<mass value="5"/>
 				<inertia ixx="0.01" ixy="0" ixz="0" iyy="0.01" iyz="0" izz="0.01" />
 			</inertial>
@@ -62,8 +64,8 @@
 		<link name="torso_3_link">
 			<inertial>
-				<mass value="10" />
-				<origin xyz="0 0 0" />
-			<inertia ixx="5.652232699207" ixy="-0.009719934438" ixz="1.293988226423"
-						 iyy="5.669473158652" iyz="-0.007379583694" izz="3.683196351726" />
+				<origin xyz="0 0 0" rpy="0 0 0"/>
+				<mass value="20" />
+			<inertia ixx="0.1" ixy="0" ixz="0"
+						 iyy="0.01" iyz="0" izz="0.01" />
 			</inertial>
 			<visual>
@@ -81,4 +83,16 @@
 			</collision>
 		</link>
+		<!-- left camera -->
+        <xacro:cob_kinect_v0 name="${name}_cam3d_left" ros_topic="cam3d_left" parent="${name}_3_link">
+			<origin xyz="${torso_cam3d_left_x} ${torso_cam3d_left_y} ${torso_cam3d_left_z}" rpy="${torso_cam3d_left_roll} ${torso_cam3d_left_pitch} ${torso_cam3d_left_yaw}" />
+		</xacro:cob_kinect_v0>
+		<!-- right camera -->
+        <xacro:cob_kinect_v0 name="${name}_cam3d_right" ros_topic="cam3d_right" parent="${name}_3_link">
+			<origin xyz="${torso_cam3d_right_x} ${torso_cam3d_right_y} ${torso_cam3d_right_z}" rpy="${torso_cam3d_right_roll} ${torso_cam3d_right_pitch} ${torso_cam3d_right_yaw}" />
+		</xacro:cob_kinect_v0>
+		<!-- down camera -->
+        <xacro:softkinetic name="${name}_cam3d_down" ros_topic="cam3d_down" parent="${name}_3_link">
+			<origin xyz="${torso_cam3d_down_x} ${torso_cam3d_down_y} ${torso_cam3d_down_z}" rpy="${torso_cam3d_down_roll} ${torso_cam3d_down_pitch} ${torso_cam3d_down_yaw}" />
+		</xacro:softkinetic>
 	<!-- extensions -->
 	<xacro:torso_gazebo name="torso" />

File: cob_description/urdf/sensors/softkinetic.gazebo.xacro (robot description, xacro)
@@ -12,5 +12,5 @@
         <horizontal_fov>${74.0*M_PI/180.0}</horizontal_fov>
         <image>
-          <format>QVGA</format>
+          <format>R8G8B8</format>
           <width>320</width>
           <height>240</height>
@@ -18,5 +18,5 @@
         <clip>
           <near>0.15</near>
-          <far>1</far>
+          <far>10</far>
         </clip>
       </camera>

Commit message: merge cob4

File: cob_description/urdf/cob4_base/base.gazebo.xacro (robot description, xacro)
@@ -29,5 +29,5 @@
       </plugin>
     </sensor>
-    <material>IPA/DarkGrey</material>
+    <material>IPA/LightGrey</material>
   </gazebo>
     <gazebo>

File: cob_description/urdf/cob4_base/base.urdf.xacro (robot description, xacro)
@@ -152,6 +152,5 @@
         <origin xyz="0 0 0" rpy="0 0 0" />
         <geometry>
-          <!--mesh filename="package://cob_description/meshes/cob4_base/caster.stl"/-->
-          <box size="0.01 0.01 0.01" />
+          <mesh filename="package://cob_description/meshes/cob4_base/caster.stl"/>
         </geometry>
         <material name="IPA/LightGrey" />

File: cob_description/urdf/cob4_head/head.urdf.xacro (robot description, xacro)
@@ -49,5 +49,5 @@
     </link>
     <joint name="head_3_joint" type="revolute">
-      <origin xyz="0 0.08001 0.06809" rpy="0.349 0 0" />
+      <origin xyz="0 0.04668 0.0976" rpy="0.349 0 0" />
       <child link="head_3_link" />
       <parent link="head_2_link"/>
@@ -59,8 +59,7 @@
     <link name="head_3_link">
       <inertial>
-      <mass value="10" />
+      <mass value="1" />
       <origin xyz="0 0 0" />
-      <inertia ixx="5.652232699207" ixy="-0.009719934438" ixz="1.293988226423"
-           iyy="5.669473158652" iyz="-0.007379583694" izz="3.683196351726" />
+      <inertia ixx="0.01" ixy="0" ixz="0" iyy="0.01" iyz="0" izz="0.01" />
       </inertial>
       <visual>

File: cob_description/urdf/cob4_torso/torso.urdf.xacro (robot description, xacro)
@@ -3,4 +3,6 @@
   <xacro:include filename="$(find cob_description)/urdf/cob4_torso/torso.gazebo.xacro" />
   <xacro:include filename="$(find cob_description)/urdf/cob4_torso/torso.transmission.xacro" />
+  <xacro:include filename="$(find cob_description)/urdf/sensors/softkinetic.urdf.xacro" />
+  <xacro:include filename="$(find cob_description)/urdf/sensors/kinect.urdf.xacro" />
   <xacro:macro name="torso" params="parent name *origin">
     <joint name="torso_base_joint" type="fixed">
@@ -22,5 +24,5 @@
       <calibration rising="${torso_1_ref}"/>
       <axis xyz="0 0 1" />
-      <dynamics damping="0.1" />
+      <dynamics damping="2.0" friction="0.0"/>
       <limit effort="100" lower="-6.2831" upper="6.2831" velocity="1.4"/>
     </joint>
@@ -28,5 +30,5 @@
       <inertial>
         <origin xyz="0 0 0" rpy="0 0 0"/>
-        <mass value="2"/>
+        <mass value="50"/>
         <inertia ixx="0.01" ixy="0" ixz="0" iyy="0.01" iyz="0" izz="0.01" />
       </inertial>
@@ -38,5 +40,5 @@
       <calibration rising="${torso_2_ref}"/>
       <axis xyz="0 0 1" />
-      <dynamics damping="0.1" />
+      <dynamics damping="2.0" friction="0.0"/>
       <limit effort="100" lower="-6.2831" upper="6.2831" velocity="1.4"/>
     </joint>
@@ -44,23 +46,22 @@
       <inertial>
         <origin xyz="0 0 0" rpy="0 0 0"/>
-        <mass value="2"/>
+        <mass value="5"/>
         <inertia ixx="0.01" ixy="0" ixz="0" iyy="0.01" iyz="0" izz="0.01" />
       </inertial>
     </link>
     <joint name="torso_3_joint" type="revolute">
-      <origin xyz="0 0.06223 0.15206" rpy="0.5236 0 0" />
+      <origin xyz="0 0.09228 0.13477" rpy="0.5236 0 0" />
       <child link="torso_3_link" />
       <parent link="torso_2_link"/>
       <calibration rising="${torso_3_ref}"/>
       <axis xyz="0 0 1" />
-      <dynamics damping="0.1" />
+      <dynamics damping="2.0" friction="0.0"/>
       <limit effort="100" lower="-6.2831" upper="6.2831" velocity="1.4"/>
     </joint>
     <link name="torso_3_link">
       <inertial>
-        <mass value="10" />
-        <origin xyz="0 0 0" />
-      <inertia ixx="5.652232699207" ixy="-0.009719934438" ixz="1.293988226423"
-             iyy="5.669473158652" iyz="-0.007379583694" izz="3.683196351726" />
+        <mass value="20" />
+        <origin xyz="0 0 0.3" rpy="0 0 0"/>
+      <inertia ixx="0.1" ixy="0" ixz="0" iyy="0.01" iyz="0" izz="0.01" />
       </inertial>
       <visual>
@@ -78,7 +79,19 @@
       </collision>
     </link>
-  <!-- extensions -->
-  <xacro:torso_gazebo name="torso" />
-  <xacro:torso_transmission name="torso" />
-  </xacro:macro>
+    <!-- left camera -->
+    <xacro:cob_kinect_v0 name="${name}_cam3d_left" ros_topic="cam3d_left" parent="${name}_3_link">
+        <origin xyz="${torso_cam3d_left_x} ${torso_cam3d_left_y} ${torso_cam3d_left_z}" rpy="${torso_cam3d_left_roll} ${torso_cam3d_left_pitch} ${torso_cam3d_left_yaw}" />
+    </xacro:cob_kinect_v0>
+    <!-- right camera -->
+    <xacro:cob_kinect_v0 name="${name}_cam3d_right" ros_topic="cam3d_right" parent="${name}_3_link">
+        <origin xyz="${torso_cam3d_right_x} ${torso_cam3d_right_y} ${torso_cam3d_right_z}" rpy="${torso_cam3d_right_roll} ${torso_cam3d_right_pitch} ${torso_cam3d_right_yaw}" />
+    </xacro:cob_kinect_v0>
+    <!-- down camera -->
+    <xacro:softkinetic name="${name}_cam3d_down" ros_topic="cam3d_down" parent="${name}_3_link">
+        <origin xyz="${torso_cam3d_down_x} ${torso_cam3d_down_y} ${torso_cam3d_down_z}" rpy="${torso_cam3d_down_roll} ${torso_cam3d_down_pitch} ${torso_cam3d_down_yaw}" />
+    </xacro:softkinetic>
+	<!-- extensions -->
+	<xacro:torso_gazebo name="torso" />
+	<xacro:torso_transmission name="torso" />
+	</xacro:macro>
 </robot>

File: cob_description/urdf/sensors/kinect.gazebo.xacro (robot description, xacro)
@@ -23,9 +23,9 @@
       <cameraName>${ros_topic}</cameraName>
       <frameName>${name}_link</frameName>
-      <imageTopicName>${ros_topic}/rgb/image_raw</imageTopicName>
-      <depthImageTopicName>${ros_topic}/depth/image_raw</depthImageTopicName>
-      <pointCloudTopicName>${ros_topic}/depth/points</pointCloudTopicName>
-      <cameraInfoTopicName>${ros_topic}/rgb/camera_info</cameraInfoTopicName>
-      <depthImageCameraInfoTopicName>${ros_topic}/depth/camera_info</depthImageCameraInfoTopicName>
+      <imageTopicName>rgb/image_raw</imageTopicName>
+      <depthImageTopicName>depth/image_raw</depthImageTopicName>
+      <pointCloudTopicName>depth_registered/points</pointCloudTopicName>
+      <cameraInfoTopicName>rgb/camera_info</cameraInfoTopicName>
+      <depthImageCameraInfoTopicName>depth_registered/camera_info</depthImageCameraInfoTopicName>
       <pointCloudCutoff>0.5</pointCloudCutoff>
       <baseline>0.2</baseline>

File: cob_description/urdf/sensors/kinect.urdf.xacro (robot description, xacro)
@@ -17,5 +17,5 @@
         <origin xyz="0 0 -0.03" rpy="0 0 0" />
         <geometry>
-          <box size="0.06 0.02 0.02"/>
+          <box size="0.02 0.02 0.02"/>
         </geometry>
         <material name="IPA/LightGrey" />
@@ -24,5 +24,5 @@
         <origin xyz="0 0 -0.03" rpy="0 0 0" />
         <geometry>
-           <box size="0.06 0.02 0.02"/>
+           <box size="0.02 0.02 0.02"/>
         </geometry>
       </collision>

Commit message: beautify mesh files

File: cob_description/urdf/cob4_base/base.gazebo.xacro (robot description, xacro)
@@ -29,5 +29,4 @@
       </plugin>
     </sensor>
-    <material>IPA/LightGrey</material>
   </gazebo>
     <gazebo>

File: cob_description/urdf/cob4_base/base.urdf.xacro (robot description, xacro)
@@ -58,13 +58,12 @@
         <origin xyz="0 0 0.0" rpy="0 0 0" />
         <geometry>
-          <mesh filename="package://cob_description/meshes/cob4_base/base_link.stl"/>
+          <mesh filename="package://cob_description/meshes/cob4_base/base.dae"/>
           <!--box size="0.01 0.01 0.01" /-->
         </geometry>
-        <material name="IPA/LightGrey"/>
       </visual>
       <collision>
         <origin xyz="0 0 0.0" rpy="0 0 0" />
         <geometry>
-          <mesh filename="package://cob_description/meshes/cob4_base/base_link.stl"/>
+          <mesh filename="package://cob_description/meshes/cob4_base/base.dae"/>
           <!--box size="0.01 0.01 0.01" /-->
         </geometry>
