Commit message: deleted offset

File: cob_description/urdf/cob4_base/base.urdf.xacro (robot description, xacro)
@@ -56,5 +56,5 @@
       </inertial>
       <visual>
-        <origin xyz="0 0 0.05" rpy="0 0 3.14159" />
+        <origin xyz="0 0 0.0" rpy="0 0 0" />
         <geometry>
           <mesh filename="package://cob_description/meshes/cob4_base/base_link.stl"/>
@@ -64,5 +64,5 @@
       </visual>
       <collision>
-        <origin xyz="0 0 0.05" rpy="0 0 3.14159" />
+        <origin xyz="0 0 0.0" rpy="0 0 0" />
         <geometry>
           <mesh filename="package://cob_description/meshes/cob4_base/base_link.stl"/>

Commit message: no inertia in base_footprint

File: cob_description/urdf/cob4_base/base.urdf.xacro (robot description, xacro)
@@ -22,25 +22,5 @@
   <property name="base_collision_size_z" value="0.04" />
   <xacro:macro name="base" params="name">
-    <link name="base_footprint">
-      <inertial>
-        <mass value="1.0" />
-        <origin xyz="0 0 0" />
-        <inertia ixx="0.01" ixy="0.0" ixz="0.0"
-             iyy="0.01" iyz="0.0" izz="0.01" />
-        </inertial>
-        <visual>
-        <origin xyz="0 0 0" rpy="0 0 0" />
-        <geometry>
-          <box size="0.01 0.01 0.01" />
-        </geometry>
-        <material name="IPA/LightGrey" />
-        </visual>
-        <collision>
-        <origin xyz="0 0 0.1" rpy="0 0 0" />
-        <geometry>
-          <box size="0.001 0.001 0.001" />
-        </geometry>
-        </collision>
-    </link>
+    <link name="base_footprint"/>
     <joint name="base_footprint_joint" type="fixed">
       <origin xyz="0 0 0" rpy="0 0 0" />

File: desire_description/urdf/base_desire/base.urdf.xacro (robot description, xacro)
@@ -148,27 +148,5 @@
     <!-- base_footprint is a fictitious link(frame) that is on the ground right below base_link origin,
          navigation stack dedpends on this frame -->
-    <link name="${name}_footprint">
-      <inertial>
-        <mass value="1.0" />
-        <origin xyz="0 0 0" />
-        <inertia ixx="0.01" ixy="0.0" ixz="0.0"
-                 iyy="0.01" iyz="0.0" izz="0.01" />
-      </inertial>
-      <visual>
-        <origin xyz="0 0 0" rpy="0 0 0" />
-        <geometry>
-          <box size="0.01 0.01 0.01" />
-        </geometry>
-        <material name="IPA/DarkGrey" />
-      </visual>
-      <collision>
-        <!-- represent base collision with a simple rectangular model, positioned by base_size_z s.t. top
-             surface of the collision box matches the top surface of the PR2 base -->
-        <origin xyz="0 0 ${0.051+base_collision_size_z/2}" rpy="0 0 0" />
-        <geometry>
-          <box size="0.001 0.001 0.001" />
-        </geometry>
-      </collision>
-    </link>
+    <link name="${name}_footprint"/>
     <joint name="${name}_footprint_joint" type="fixed">
       <origin xyz="0 0 0" rpy="0 0 0" />

File: raw_description/urdf/base_long/base.urdf.xacro (robot description, xacro)
@@ -186,25 +186,5 @@
     <!-- base_footprint is a fictitious link(frame) that is on the ground right below base_link origin,
          navigation stack dedpends on this frame -->
-    <link name="${name}_footprint">
-      <inertial>
-        <mass value="1.0" />
-        <origin xyz="0 0 0" />
-        <inertia ixx="0.01" ixy="0.0" ixz="0.0"
-                 iyy="0.01" iyz="0.0" izz="0.01" />
-      </inertial>
-      <visual>
-        <origin xyz="0 0 0" rpy="0 0 0" />
-        <geometry>
-          <box size="0.01 0.01 0.01" />
-        </geometry>
-        <material name="IPA/LightGrey" />
-      </visual>
-      <collision>
-        <origin xyz="0 0 0.1" rpy="0 0 0" />
-        <geometry>
-          <box size="0.001 0.001 0.001" />
-        </geometry>
-      </collision>
-    </link>
+    <link name="${name}_footprint"/>
     <joint name="${name}_footprint_joint" type="fixed">
       <origin xyz="0 0 0" rpy="0 0 0" />

File: raw_description/urdf/base_short/base.urdf.xacro (robot description, xacro)
@@ -185,25 +185,5 @@
     <!-- base_footprint is a fictitious link(frame) that is on the ground right below base_link origin,
          navigation stack dedpends on this frame -->
-    <link name="${name}_footprint">
-      <inertial>
-        <mass value="1.0" />
-        <origin xyz="0 0 0" />
-        <inertia ixx="0.01" ixy="0.0" ixz="0.0"
-                 iyy="0.01" iyz="0.0" izz="0.01" />
-      </inertial>
-      <visual>
-        <origin xyz="0 0 0" rpy="0 0 0" />
-        <geometry>
-          <box size="0.01 0.01 0.01" />
-        </geometry>
-        <material name="IPA/LightGrey" />
-      </visual>
-      <collision>
-        <origin xyz="0 0 0.1" rpy="0 0 0" />
-        <geometry>
-          <box size="0.001 0.001 0.001" />
-        </geometry>
-      </collision>
-    </link>
+    <link name="${name}_footprint"/>
     <joint name="${name}_footprint_joint" type="fixed">
       <origin xyz="0 0 0" rpy="0 0 0" />

Commit message: use base mesh with less vertices for collision checking

File: cob_description/urdf/cob4_base/base.urdf.xacro (robot description, xacro)
@@ -45,5 +45,5 @@
         <origin xyz="0 0 0.0" rpy="0 0 0" />
         <geometry>
-          <mesh filename="package://cob_description/meshes/cob4_base/base.dae"/>
+          <mesh filename="package://cob_description/meshes/cob4_base/base_reduced.stl"/>
           <!--box size="0.01 0.01 0.01" /-->
         </geometry>

Commit message: new collision mesh

File: cob_description/urdf/cob4_base/base.urdf.xacro (robot description, xacro)
@@ -45,5 +45,5 @@
         <origin xyz="0 0 0.0" rpy="0 0 0" />
         <geometry>
-          <mesh filename="package://cob_description/meshes/cob4_base/base_reduced.stl"/>
+          <mesh filename="package://cob_description/meshes/cob4_base/base_collision.stl"/>
           <!--box size="0.01 0.01 0.01" /-->
         </geometry>

Commit message: Limits now come from the yaml files

File: cob_description/urdf/cob4_base/base.urdf.xacro (robot description, xacro)
@@ -77,6 +77,6 @@
     <joint name="${parent}_${suffix}_wheel_joint" type="continuous">
       <axis xyz="0 1 0" />
-      <limit effort="100" velocity="100"/> <!-- alpha tested effort and velocity limits -->
-      <safety_controller  k_velocity="10" />
+      <!--limit effort="100" velocity="100"/--> <!-- alpha tested effort and velocity limits -->
+      <!--safety_controller  k_velocity="10" /-->
       <dynamics damping="0.0" friction="0.0" />
       <origin xyz="0 ${reflect*caster_wheel_offset_y} 0" rpy="0 0 0" />
@@ -113,6 +113,6 @@
     <joint name="${suffix}_rotation_joint" type="continuous">
       <axis xyz="0 0 1" />
-      <limit effort="100" velocity="100"/> <!-- alpha tested velocity and effort limits -->
-      <safety_controller  k_velocity="10" />
+      <!--limit effort="100" velocity="100"/--> <!-- alpha tested velocity and effort limits -->
+      <!--safety_controller  k_velocity="10" /-->
       <calibration rising="${ref_position}"/>
       <dynamics damping="0.0" friction="0.0" />

Commit message: add temporary fix urdf argument for cob4_base joint_names

File: cob_description/urdf/cob4_base/base.urdf.xacro (robot description, xacro)
@@ -21,5 +21,5 @@
   <property name="base_size_z" value="0.23" />
   <property name="base_collision_size_z" value="0.04" />
-  <xacro:macro name="base" params="name">
+  <xacro:macro name="base" params="name use_old_joint_names">
     <link name="base_footprint"/>
     <joint name="base_footprint_joint" type="fixed">
@@ -60,13 +60,26 @@
       <origin xyz="${laser_right_x} ${laser_right_y} ${laser_right_z}" rpy="${laser_right_roll} ${laser_right_pitch} ${laser_right_yaw}" />
     </xacro:sick_s300_laser_v0>
-    <xacro:cob_caster suffix="fl" parent="${name}_link" ref_position="0" >
-      <origin xyz="${caster_offset_x/2} ${caster_offset_y} ${caster_offset_z}" rpy="0 0 0" />
-    </xacro:cob_caster>
-    <xacro:cob_caster suffix="b" parent="${name}_link" ref_position="0" >
-      <origin xyz="${-caster_offset_x} 0 ${caster_offset_z}" rpy="0 0 0" />
-    </xacro:cob_caster>
-    <xacro:cob_caster suffix="fr" parent="${name}_link" ref_position="0" >
-      <origin xyz="${caster_offset_x/2} ${-caster_offset_y} ${caster_offset_z}" rpy="0 0 0" />
-    </xacro:cob_caster>
+    <xacro:if value="${use_old_joint_names}">
+      <xacro:cob_caster suffix="fl" parent="${name}_link" ref_position="0" >
+        <origin xyz="${caster_offset_x/2} ${caster_offset_y} ${caster_offset_z}" rpy="0 0 0" />
+      </xacro:cob_caster>
+      <xacro:cob_caster suffix="bl" parent="${name}_link" ref_position="0" >
+        <origin xyz="${-caster_offset_x} 0 ${caster_offset_z}" rpy="0 0 0" />
+      </xacro:cob_caster>
+      <xacro:cob_caster suffix="br" parent="${name}_link" ref_position="0" >
+        <origin xyz="${caster_offset_x/2} ${-caster_offset_y} ${caster_offset_z}" rpy="0 0 0" />
+      </xacro:cob_caster>
+    </xacro:if>
+    <xacro:unless value="${use_old_joint_names}">
+      <xacro:cob_caster suffix="fl" parent="${name}_link" ref_position="0" >
+        <origin xyz="${caster_offset_x/2} ${caster_offset_y} ${caster_offset_z}" rpy="0 0 0" />
+      </xacro:cob_caster>
+      <xacro:cob_caster suffix="b" parent="${name}_link" ref_position="0" >
+        <origin xyz="${-caster_offset_x} 0 ${caster_offset_z}" rpy="0 0 0" />
+      </xacro:cob_caster>
+      <xacro:cob_caster suffix="fr" parent="${name}_link" ref_position="0" >
+        <origin xyz="${caster_offset_x/2} ${-caster_offset_y} ${caster_offset_z}" rpy="0 0 0" />
+      </xacro:cob_caster>
+    </xacro:unless>
   <xacro:base_gazebo name="${name}" />
   </xacro:macro>

Commit message: set proper velocity limits for cob4 drive_wheel

File: cob_description/urdf/cob4_base/base.urdf.xacro (robot description, xacro)
@@ -12,4 +12,6 @@
   <xacro:property name="base_mass" value="50" />
   <xacro:macro name="base" params="name use_old_joint_names">
+    <xacro:property name="drive_vel" value="19.95" />
+    <xacro:property name="steer_vel" value="117.81" />
     <link name="${name}_footprint"/>
     <joint name="${name}_footprint_joint" type="fixed">

File: cob_description/urdf/drive_wheel/drive_wheel.urdf.xacro (robot description, xacro)
@@ -6,5 +6,5 @@
   <xacro:property name="caster_mass" value="5.9" />
   <xacro:property name="wheel_mass" value="0.44036" />
-  <xacro:macro name="cob_wheel" params="parent suffix reflect">
+  <xacro:macro name="cob_wheel" params="parent suffix reflect drive_vel:=^">
     <joint name="${parent}_${suffix}_wheel_joint" type="continuous">
       <origin xyz="0 ${reflect*caster_wheel_offset_y} 0" rpy="0 0 0" />
@@ -12,6 +12,6 @@
       <child link="${parent}_${suffix}_wheel_link"/>
       <axis xyz="0 1 0" />
-      <limit effort="100" velocity="100"/> <!-- alpha tested effort and velocity limits -->
       <safety_controller  k_velocity="10" />
+      <limit effort="0" velocity="${drive_vel}"/>
       <dynamics damping="0.0" friction="0.0" />
     </joint>
@@ -39,5 +39,5 @@
   </xacro:macro>
   <!-- Macro for Caster hub only -->
-  <xacro:macro name="cob_caster_hub" params="*origin parent suffix" >
+  <xacro:macro name="cob_caster_hub" params="*origin parent suffix steer_vel:=^" >
     <joint name="${suffix}_rotation_joint" type="continuous">
       <xacro:insert_block name="origin" />
@@ -45,6 +45,6 @@
       <child link="${suffix}_rotation_link" />
       <axis xyz="0 0 1" />
-      <limit effort="100" velocity="100"/> <!-- alpha tested velocity and effort limits -->
       <safety_controller  k_velocity="10" />
+      <limit effort="0" velocity="${steer_vel}"/>
       <dynamics damping="0.0" friction="0.0" />
     </joint>
@@ -71,5 +71,5 @@
     <xacro:cob_caster_transmission suffix="${suffix}" />
   </xacro:macro>
-  <xacro:macro name="drive_wheel" params="*origin parent suffix">
+  <xacro:macro name="drive_wheel" params="*origin parent suffix drive_vel:=^|100 steer_vel:=^|100">
     <xacro:cob_caster_hub parent="${parent}" suffix="${suffix}_caster" >
       <xacro:insert_block name="origin" />

Commit message: separate laser scanner from base

File: cob_description/urdf/cob4_base/base.urdf.xacro (robot description, xacro)
@@ -4,6 +4,4 @@
   <!-- drive_wheel module -->
   <xacro:include filename="$(find cob_description)/urdf/drive_wheel/drive_wheel.urdf.xacro" />
-  <!-- sensors -->
-  <xacro:include filename="$(find cob_description)/urdf/sensors/sick_s300_laser.urdf.xacro"/>
   <!-- properties -->
   <xacro:property name="caster_offset_x" value="0.24844" />  <!--modify here-->
@@ -65,14 +63,4 @@
       </xacro:drive_wheel>
     </xacro:unless>
-    <!-- sensors -->
-    <xacro:sick_s300_laser_v0 name="${name}_laser_front" parent="${name}">
-      <origin xyz="${laser_front_x} ${laser_front_y} ${laser_front_z}" rpy="${laser_front_roll} ${laser_front_pitch} ${laser_front_yaw}" />
-    </xacro:sick_s300_laser_v0>
-    <xacro:sick_s300_laser_v0 name="${name}_laser_left" parent="${name}">
-      <origin xyz="${laser_left_x} ${laser_left_y} ${laser_left_z}" rpy="${laser_left_roll} ${laser_left_pitch} ${laser_left_yaw}" />
-    </xacro:sick_s300_laser_v0>
-    <xacro:sick_s300_laser_v0 name="${name}_laser_right" parent="${name}">
-      <origin xyz="${laser_right_x} ${laser_right_y} ${laser_right_z}" rpy="${laser_right_roll} ${laser_right_pitch} ${laser_right_yaw}" />
-    </xacro:sick_s300_laser_v0>
     <!-- gazebo extensions -->
     <xacro:base_gazebo name="${name}" />

File: raw_description/urdf/base_long/base.urdf.xacro (robot description, xacro)
@@ -5,7 +5,4 @@
   <!-- drive_wheel module -->
   <xacro:include filename="$(find cob_description)/urdf/drive_wheel/drive_wheel.urdf.xacro" />
-  <!-- sensors -->
-  <xacro:include filename="$(find cob_description)/urdf/sensors/sick_s300_laser.urdf.xacro"/>
-  <xacro:include filename="$(find cob_description)/urdf/sensors/kinect.urdf.xacro"/>
   <!-- properties -->
   <xacro:property name="caster_offset_x" value="0.368" />  <!--modify here-->
@@ -92,16 +89,4 @@
       <origin xyz="${-caster_offset_x} ${caster_offset_y_br} ${caster_offset_z}" rpy="0 0 0" />
     </xacro:drive_wheel>
-    <!-- base laser front -->
-    <xacro:sick_s300_laser_v0 name="${name}_laser_front" parent="${name}">
-      <origin xyz="${laser_front_x} ${laser_front_y} ${laser_front_z}" rpy="${laser_front_roll} ${laser_front_pitch} ${laser_front_yaw}" />
-    </xacro:sick_s300_laser_v0>
-    <!-- base laser rear -->
-    <xacro:sick_s300_laser_v0 name="${name}_laser_rear" parent="${name}">
-      <origin xyz="${laser_rear_x} ${laser_rear_y} ${laser_rear_z}" rpy="${laser_rear_roll} ${laser_rear_pitch} ${laser_rear_yaw}" />
-    </xacro:sick_s300_laser_v0>
-    <!-- cam3d -->
-    <!--xacro:cob_kinect_v0 name="${name}_cam3d" ros_topic="cam3d" parent="${name}_link">
-      <origin xyz="0.51 0.12 0.27" rpy="-${M_PI/2} 0 -${M_PI/2}" />
-    </xacro:cob_kinect_v0-->
     <!-- battery front-->
     <xacro:cob_batteries name="${name}_battery_front" parent="${name}_link">

File: raw_description/urdf/base_short/base.urdf.xacro (robot description, xacro)
@@ -5,7 +5,4 @@
   <!-- drive_wheel module -->
   <xacro:include filename="$(find cob_description)/urdf/drive_wheel/drive_wheel.urdf.xacro" />
-  <!-- sensors -->
-  <xacro:include filename="$(find cob_description)/urdf/sensors/sick_s300_laser.urdf.xacro"/>
-  <xacro:include filename="$(find cob_description)/urdf/sensors/kinect.urdf.xacro"/>
   <!-- properties -->
   <xacro:property name="caster_offset_x" value="0.228" />  <!--modify here-->
@@ -96,16 +93,4 @@
       <origin xyz="${-caster_offset_x} ${caster_offset_y_br} ${caster_offset_z}" rpy="0 0 0" />
     </xacro:drive_wheel>
-    <!-- base laser front -->
-    <xacro:sick_s300_laser_v0 name="${name}_laser_front" parent="${name}">
-      <origin xyz="${laser_front_x} ${laser_front_y} ${laser_front_z}" rpy="${laser_front_roll} ${laser_front_pitch} ${laser_front_yaw}" />
-    </xacro:sick_s300_laser_v0>
-    <!-- base laser rear -->
-    <xacro:sick_s300_laser_v0 name="${name}_laser_rear" parent="${name}">
-      <origin xyz="${laser_rear_x} ${laser_rear_y} ${laser_rear_z}" rpy="${laser_rear_roll} ${laser_rear_pitch} ${laser_rear_yaw}" />
-    </xacro:sick_s300_laser_v0>
-    <!-- cam3d -->
-    <!--xacro:cob_kinect_v0 name="${name}_cam3d" ros_topic="cam3d" parent="${name}_link">
-      <origin xyz="0.51 0.12 0.27" rpy="-${M_PI/2} 0 -${M_PI/2}" />
-    </xacro:cob_kinect_v0-->
     <!-- battery-->
     <xacro:cob_batteries name="${name}_battery" parent="${name}_link">

Commit message: tweak inertia

File: cob_description/urdf/cob4_base/base.urdf.xacro (robot description, xacro)
@@ -8,5 +8,5 @@
   <xacro:property name="caster_offset_y" value="0.21515" />
   <xacro:property name="caster_offset_z" value="0.08" />
-  <xacro:property name="base_mass" value="50" />
+  <xacro:property name="base_mass" value="100" />
   <xacro:macro name="base" params="name use_old_joint_names">
     <xacro:property name="drive_vel" value="19.95" />

File: cob_description/urdf/sensors/kinect.urdf.xacro (robot description, xacro)
@@ -9,7 +9,5 @@
     </joint>
     <link name="${name}_link">
-      <xacro:box_inertial x="0.18" y="0.035" z="0.05" mass="0.3">
-        <origin xyz="0 0 0" rpy="0 0 0" />
-      </xacro:box_inertial>
+      <xacro:default_inertial/>
       <visual>
         <origin xyz="0 0 -0.03" rpy="0 0 0" />

File: cob_description/urdf/sensors/realsense.urdf.xacro (robot description, xacro)
@@ -9,9 +9,5 @@
     </joint>
     <link name="${name}_link">
-      <inertial>
-        <mass value="0.564" />
-        <origin xyz="0 0 0" />
-        <inertia ixx="0.003881243" ixy="0.0" ixz="0.0" iyy="0.000498940" iyz="0.0" izz="0.003879257" />
-      </inertial>
+      <xacro:default_inertial/>
       <visual>
        <origin xyz="0 0 0" rpy="0 0 0"/>

File: cob_description/urdf/sensors/realsense_zr300.urdf.xacro (robot description, xacro)
@@ -9,9 +9,5 @@
     </joint>
     <link name="${name}_link">
-      <inertial>
-        <mass value="0.564" />
-        <origin xyz="0 0 0" />
-        <inertia ixx="0.003881243" ixy="0.0" ixz="0.0" iyy="0.000498940" iyz="0.0" izz="0.003879257" />
-      </inertial>
+      <xacro:default_inertial/>
       <visual>
        <origin xyz="0 0 0" rpy="0 0 0"/>

File: cob_description/urdf/sensors/usb_cam.urdf.xacro (robot description, xacro)
@@ -9,9 +9,5 @@
     </joint>
     <link name="${name}_link">
-      <inertial>
-        <mass value="0.1" />
-        <origin xyz="0 0 0" />
-        <inertia ixx="0.003881243" ixy="0.0" ixz="0.0" iyy="0.000498940" iyz="0.0" izz="0.003879257" />
-      </inertial>
+      <xacro:default_inertial/>
       <visual>
        <origin xyz="0 0 0" rpy="0 0 0"/>

Commit message: remove obsolete argument use_old_joint_names

File: cob_description/urdf/cob4_base/base.urdf.xacro (robot description, xacro)
@@ -9,5 +9,5 @@
   <xacro:property name="caster_offset_z" value="0.08" />
   <xacro:property name="base_mass" value="100" />
-  <xacro:macro name="base" params="name use_old_joint_names">
+  <xacro:macro name="base" params="name">
     <xacro:property name="drive_vel" value="19.95" />
     <xacro:property name="steer_vel" value="117.81" />
@@ -41,26 +41,13 @@
     </link>
     <!-- arrangement of the three drive_wheel modules -->
-    <xacro:if value="${use_old_joint_names}">
-      <xacro:drive_wheel parent="${name}_link" suffix="fl" >
-        <origin xyz="${caster_offset_x/2} ${caster_offset_y} ${caster_offset_z}" rpy="0 0 0" />
-      </xacro:drive_wheel>
-      <xacro:drive_wheel parent="${name}_link" suffix="bl" >
-        <origin xyz="${-caster_offset_x} 0.0 ${caster_offset_z}" rpy="0 0 0" />
-      </xacro:drive_wheel>
-      <xacro:drive_wheel parent="${name}_link" suffix="br" >
-        <origin xyz="${caster_offset_x/2} ${-caster_offset_y} ${caster_offset_z}" rpy="0 0 0" />
-      </xacro:drive_wheel>
-    </xacro:if>
-    <xacro:unless value="${use_old_joint_names}">
-      <xacro:drive_wheel parent="${name}_link" suffix="fl" >
-        <origin xyz="${caster_offset_x/2} ${caster_offset_y} ${caster_offset_z}" rpy="0 0 0" />
-      </xacro:drive_wheel>
-      <xacro:drive_wheel parent="${name}_link" suffix="b" >
-        <origin xyz="${-caster_offset_x} 0.0 ${caster_offset_z}" rpy="0 0 0" />
-      </xacro:drive_wheel>
-      <xacro:drive_wheel parent="${name}_link" suffix="fr" >
-        <origin xyz="${caster_offset_x/2} ${-caster_offset_y} ${caster_offset_z}" rpy="0 0 0" />
-      </xacro:drive_wheel>
-    </xacro:unless>
+    <xacro:drive_wheel parent="${name}_link" suffix="fl" >
+      <origin xyz="${caster_offset_x/2} ${caster_offset_y} ${caster_offset_z}" rpy="0 0 0" />
+    </xacro:drive_wheel>
+    <xacro:drive_wheel parent="${name}_link" suffix="b" >
+      <origin xyz="${-caster_offset_x} 0.0 ${caster_offset_z}" rpy="0 0 0" />
+    </xacro:drive_wheel>
+    <xacro:drive_wheel parent="${name}_link" suffix="fr" >
+      <origin xyz="${caster_offset_x/2} ${-caster_offset_y} ${caster_offset_z}" rpy="0 0 0" />
+    </xacro:drive_wheel>
     <!-- gazebo extensions -->
     <xacro:base_gazebo name="${name}" />
