Commit message: allow tricycle_mode

File: cob_description/urdf/cob4_base/base.urdf.xacro (robot description, xacro)
@@ -9,5 +9,5 @@
   <xacro:property name="caster_offset_z" value="0.08" />
   <xacro:property name="base_mass" value="100" />
-  <xacro:macro name="base" params="name">
+  <xacro:macro name="base" params="name tricycle_mode:=false">
     <xacro:property name="drive_vel" value="19.95" />
     <xacro:property name="steer_vel" value="117.81" />
@@ -41,13 +41,26 @@
     </link>
     <!-- arrangement of the three drive_wheel modules -->
-    <xacro:drive_wheel parent="${name}_link" suffix="fl" >
-      <origin xyz="${caster_offset_x/2} ${caster_offset_y} ${caster_offset_z}" rpy="0 0 0" />
-    </xacro:drive_wheel>
-    <xacro:drive_wheel parent="${name}_link" suffix="b" >
-      <origin xyz="${-caster_offset_x} 0.0 ${caster_offset_z}" rpy="0 0 0" />
-    </xacro:drive_wheel>
-    <xacro:drive_wheel parent="${name}_link" suffix="fr" >
-      <origin xyz="${caster_offset_x/2} ${-caster_offset_y} ${caster_offset_z}" rpy="0 0 0" />
-    </xacro:drive_wheel>
+    <xacro:if value="${tricycle_mode}">
+      <xacro:drive_wheel parent="${name}_link" suffix="fl" passive="true" >
+        <origin xyz="${caster_offset_x/2} ${caster_offset_y} ${caster_offset_z}" rpy="0 0 0" />
+      </xacro:drive_wheel>
+      <xacro:drive_wheel parent="${name}_link" suffix="b" >
+        <origin xyz="${-caster_offset_x} 0.0 ${caster_offset_z}" rpy="0 0 0" />
+      </xacro:drive_wheel>
+      <xacro:drive_wheel parent="${name}_link" suffix="fr" passive="true">
+        <origin xyz="${caster_offset_x/2} ${-caster_offset_y} ${caster_offset_z}" rpy="0 0 0" />
+      </xacro:drive_wheel>
+    </xacro:if>
+    <xacro:unless value="${tricycle_mode}">
+      <xacro:drive_wheel parent="${name}_link" suffix="fl" >
+        <origin xyz="${caster_offset_x/2} ${caster_offset_y} ${caster_offset_z}" rpy="0 0 0" />
+      </xacro:drive_wheel>
+      <xacro:drive_wheel parent="${name}_link" suffix="b" >
+        <origin xyz="${-caster_offset_x} 0.0 ${caster_offset_z}" rpy="0 0 0" />
+      </xacro:drive_wheel>
+      <xacro:drive_wheel parent="${name}_link" suffix="fr" >
+        <origin xyz="${caster_offset_x/2} ${-caster_offset_y} ${caster_offset_z}" rpy="0 0 0" />
+      </xacro:drive_wheel>
+    </xacro:unless>
     <!-- gazebo extensions -->
     <xacro:base_gazebo name="${name}" />

Commit message: rotate base link (close to working), docking missing

File: cob_description/urdf/cob4_base/base.urdf.xacro (robot description, xacro)
@@ -18,5 +18,11 @@
       <child link="${name}_link" />
     </joint>
-    <link name="${name}_link">
+    <link name="${name}_link"/>
+    <joint name="${name}_rotated_joint" type="fixed">
+      <origin xyz="0 0 0" rpy="0 0 3.14159" />
+      <parent link="${name}_link"/>
+      <child link="${name}_rotated_link" />
+    </joint>
+    <link name="${name}_rotated_link">
       <inertial>
         <origin xyz="0 0 0" />
@@ -42,22 +48,22 @@
     <!-- arrangement of the three drive_wheel modules -->
     <xacro:if value="${tricycle_mode}">
-      <xacro:drive_wheel parent="${name}_link" suffix="fl" passive="true" >
+      <xacro:drive_wheel parent="${name}_rotated_link" suffix="fl" passive="true" >
         <origin xyz="${caster_offset_x/2} ${caster_offset_y} ${caster_offset_z}" rpy="0 0 0" />
       </xacro:drive_wheel>
-      <xacro:drive_wheel parent="${name}_link" suffix="b" >
+      <xacro:drive_wheel parent="${name}_rotated_link" suffix="b" >
         <origin xyz="${-caster_offset_x} 0.0 ${caster_offset_z}" rpy="0 0 0" />
       </xacro:drive_wheel>
-      <xacro:drive_wheel parent="${name}_link" suffix="fr" passive="true">
+      <xacro:drive_wheel parent="${name}_rotated_link" suffix="fr" passive="true">
         <origin xyz="${caster_offset_x/2} ${-caster_offset_y} ${caster_offset_z}" rpy="0 0 0" />
       </xacro:drive_wheel>
     </xacro:if>
     <xacro:unless value="${tricycle_mode}">
-      <xacro:drive_wheel parent="${name}_link" suffix="fl" >
+      <xacro:drive_wheel parent="${name}_rotated_link" suffix="fl" >
         <origin xyz="${caster_offset_x/2} ${caster_offset_y} ${caster_offset_z}" rpy="0 0 0" />
       </xacro:drive_wheel>
-      <xacro:drive_wheel parent="${name}_link" suffix="b" >
+      <xacro:drive_wheel parent="${name}_rotated_link" suffix="b" >
         <origin xyz="${-caster_offset_x} 0.0 ${caster_offset_z}" rpy="0 0 0" />
       </xacro:drive_wheel>
-      <xacro:drive_wheel parent="${name}_link" suffix="fr" >
+      <xacro:drive_wheel parent="${name}_rotated_link" suffix="fr" >
         <origin xyz="${caster_offset_x/2} ${-caster_offset_y} ${caster_offset_z}" rpy="0 0 0" />
       </xacro:drive_wheel>

File: cob_description/urdf/drive_wheel/drive_wheel.urdf.xacro (robot description, xacro)
@@ -98,6 +98,12 @@
   </xacro:macro>
   <xacro:macro name="drive_wheel" params="*origin parent suffix drive_vel:=^|100 steer_vel:=^|100 passive:=false">
-    <xacro:cob_caster_hub parent="${parent}" suffix="${suffix}_caster" passive="${passive}" >
-      <xacro:insert_block name="origin" />
+    <link name="${suffix}_link"/>
+    <joint name="${suffix}_joint" type="fixed">
+        <xacro:insert_block name="origin" />
+        <parent link="${parent}"/>
+        <child link="${suffix}_link" />
+    </joint>
+    <xacro:cob_caster_hub parent="${suffix}_link" suffix="${suffix}_caster" passive="${passive}" >
+      <origin xyz="0 0 0" rpy="0 0 0" />
     </xacro:cob_caster_hub>
     <xacro:cob_wheel parent="${suffix}_caster" suffix="r" reflect="-1"  passive="${passive}" />

Commit message: added parameter for drive direction

File: cob_description/urdf/cob4_base/base.urdf.xacro (robot description, xacro)
@@ -9,5 +9,5 @@
   <xacro:property name="caster_offset_z" value="0.08" />
   <xacro:property name="base_mass" value="100" />
-  <xacro:macro name="base" params="name tricycle_mode:=false">
+  <xacro:macro name="base" params="name tricycle_mode:=false drive_dir_angle:=0">
     <xacro:property name="drive_vel" value="19.95" />
     <xacro:property name="steer_vel" value="117.81" />
@@ -20,5 +20,5 @@
     <link name="${name}_link"/>
     <joint name="${name}_rotated_joint" type="fixed">
-      <origin xyz="0 0 0" rpy="0 0 3.14159" />
+      <origin xyz="0 0 0" rpy="0 0 ${drive_dir_angle}" />
       <parent link="${name}_link"/>
       <child link="${name}_rotated_link" />

Commit message: fixed wheel radius

File: cob_description/urdf/cob4_base/base.urdf.xacro (robot description, xacro)
@@ -7,5 +7,5 @@
   <xacro:property name="caster_offset_x" value="0.24844" />  <!--modify here-->
   <xacro:property name="caster_offset_y" value="0.21515" />
-  <xacro:property name="caster_offset_z" value="0.08" />
+  <xacro:property name="caster_offset_z" value="0.0782" />
   <xacro:property name="base_mass" value="100" />
   <xacro:macro name="base" params="name tricycle_mode:=false">

Commit message: cleanup and rename links

File: cob_description/urdf/cob4_base/base.urdf.xacro (robot description, xacro)
@@ -19,10 +19,10 @@
     </joint>
     <link name="${name}_link"/>
-    <joint name="${name}_rotated_joint" type="fixed">
+    <joint name="${name}_chassis_joint" type="fixed">
       <origin xyz="0 0 0" rpy="0 0 ${drive_dir_angle}" />
       <parent link="${name}_link"/>
-      <child link="${name}_rotated_link" />
+      <child link="${name}_chassis_link" />
     </joint>
-    <link name="${name}_rotated_link">
+    <link name="${name}_chassis_link">
       <inertial>
         <origin xyz="0 0 0" />
@@ -48,22 +48,22 @@
     <!-- arrangement of the three drive_wheel modules -->
     <xacro:if value="${tricycle_mode}">
-      <xacro:drive_wheel parent="${name}_rotated_link" suffix="fl" passive="true" >
+      <xacro:drive_wheel parent="${name}_chassis_link" suffix="fl" passive="true" >
         <origin xyz="${caster_offset_x/2} ${caster_offset_y} ${caster_offset_z}" rpy="0 0 0" />
       </xacro:drive_wheel>
-      <xacro:drive_wheel parent="${name}_rotated_link" suffix="b" >
+      <xacro:drive_wheel parent="${name}_chassis_link" suffix="b" >
         <origin xyz="${-caster_offset_x} 0.0 ${caster_offset_z}" rpy="0 0 0" />
       </xacro:drive_wheel>
-      <xacro:drive_wheel parent="${name}_rotated_link" suffix="fr" passive="true">
+      <xacro:drive_wheel parent="${name}_chassis_link" suffix="fr" passive="true">
         <origin xyz="${caster_offset_x/2} ${-caster_offset_y} ${caster_offset_z}" rpy="0 0 0" />
       </xacro:drive_wheel>
     </xacro:if>
     <xacro:unless value="${tricycle_mode}">
-      <xacro:drive_wheel parent="${name}_rotated_link" suffix="fl" >
+      <xacro:drive_wheel parent="${name}_chassis_link" suffix="fl" >
         <origin xyz="${caster_offset_x/2} ${caster_offset_y} ${caster_offset_z}" rpy="0 0 0" />
       </xacro:drive_wheel>
-      <xacro:drive_wheel parent="${name}_rotated_link" suffix="b" >
+      <xacro:drive_wheel parent="${name}_chassis_link" suffix="b" >
         <origin xyz="${-caster_offset_x} 0.0 ${caster_offset_z}" rpy="0 0 0" />
       </xacro:drive_wheel>
-      <xacro:drive_wheel parent="${name}_rotated_link" suffix="fr" >
+      <xacro:drive_wheel parent="${name}_chassis_link" suffix="fr" >
         <origin xyz="${caster_offset_x/2} ${-caster_offset_y} ${caster_offset_z}" rpy="0 0 0" />
       </xacro:drive_wheel>

File: cob_description/urdf/drive_wheel/drive_wheel.urdf.xacro (robot description, xacro)
@@ -98,12 +98,6 @@
   </xacro:macro>
   <xacro:macro name="drive_wheel" params="*origin parent suffix drive_vel:=^|100 steer_vel:=^|100 passive:=false">
-    <link name="${suffix}_link"/>
-    <joint name="${suffix}_joint" type="fixed">
-        <xacro:insert_block name="origin" />
-        <parent link="${parent}"/>
-        <child link="${suffix}_link" />
-    </joint>
-    <xacro:cob_caster_hub parent="${suffix}_link" suffix="${suffix}_caster" passive="${passive}" >
-      <origin xyz="0 0 0" rpy="0 0 0" />
+    <xacro:cob_caster_hub parent="${parent}" suffix="${suffix}_caster" passive="${passive}" >
+      <xacro:insert_block name="origin" />
     </xacro:cob_caster_hub>
     <xacro:cob_wheel parent="${suffix}_caster" suffix="r" reflect="-1"  passive="${passive}" />

Commit message: add base_charger_link

File: cob_description/urdf/cob4_base/base.urdf.xacro (robot description, xacro)
@@ -46,4 +46,10 @@
       </collision>
     </link>
+    <joint name="${name}_charger_joint" type="fixed">
+      <origin xyz="0.2992 0.0 0.09089" rpy="0 0 0" />
+      <parent link="${name}_chassis_link"/>
+      <child link="${name}_charger_link" />
+    </joint>
+    <link name="${name}_charger_link"/>
     <!-- arrangement of the three drive_wheel modules -->
     <xacro:if value="${tricycle_mode}">

Commit message: add base_pivot_link for tricycle mode

File: cob_description/urdf/cob4_base/base.urdf.xacro (robot description, xacro)
@@ -54,4 +54,10 @@
     <!-- arrangement of the three drive_wheel modules -->
     <xacro:if value="${tricycle_mode}">
+      <joint name="${name}_pivot_joint" type="fixed">
+        <origin xyz="${caster_offset_x/2} 0.0 0.0" rpy="0 0 0" />
+        <parent link="${name}_chassis_link"/>
+        <child link="${name}_pivot_link" />
+      </joint>
+      <link name="${name}_pivot_link"/>
       <xacro:drive_wheel parent="${name}_chassis_link" suffix="fl" passive="true" >
         <origin xyz="${caster_offset_x/2} ${caster_offset_y} ${caster_offset_z}" rpy="0 0 0" />

Commit message: proper tf hierarchy for base_pivot_link

File: cob_description/urdf/cob4_base/base.urdf.xacro (robot description, xacro)
@@ -12,4 +12,12 @@
     <xacro:property name="drive_vel" value="19.95" />
     <xacro:property name="steer_vel" value="117.81" />
+    <xacro:if value="${tricycle_mode}">
+      <link name="${name}_pivot_link"/>
+      <joint name="${name}_pivot_joint" type="fixed">
+        <origin xyz="${-caster_offset_x/2} 0.0 0.0" rpy="0 0 0" />
+        <parent link="${name}_pivot_link"/>
+        <child link="${name}_footprint" />
+      </joint>
+    </xacro:if>
     <link name="${name}_footprint"/>
     <joint name="${name}_footprint_joint" type="fixed">
@@ -54,10 +62,4 @@
     <!-- arrangement of the three drive_wheel modules -->
     <xacro:if value="${tricycle_mode}">
-      <joint name="${name}_pivot_joint" type="fixed">
-        <origin xyz="${caster_offset_x/2} 0.0 0.0" rpy="0 0 0" />
-        <parent link="${name}_chassis_link"/>
-        <child link="${name}_pivot_link" />
-      </joint>
-      <link name="${name}_pivot_link"/>
       <xacro:drive_wheel parent="${name}_chassis_link" suffix="fl" passive="true" >
         <origin xyz="${caster_offset_x/2} ${caster_offset_y} ${caster_offset_z}" rpy="0 0 0" />

Commit message: allow drive backwards with tricycle

File: cob_description/urdf/cob4_base/base.urdf.xacro (robot description, xacro)
@@ -9,14 +9,23 @@
   <xacro:property name="caster_offset_z" value="0.0782" />
   <xacro:property name="base_mass" value="100" />
-  <xacro:macro name="base" params="name tricycle_mode:=false drive_dir_angle:=0">
+  <xacro:macro name="base" params="name tricycle_mode:=false forward:=true">
     <xacro:property name="drive_vel" value="19.95" />
     <xacro:property name="steer_vel" value="117.81" />
     <xacro:if value="${tricycle_mode}">
       <link name="${name}_pivot_link"/>
-      <joint name="${name}_pivot_joint" type="fixed">
-        <origin xyz="${-caster_offset_x/2} 0.0 0.0" rpy="0 0 0" />
-        <parent link="${name}_pivot_link"/>
-        <child link="${name}_footprint" />
-      </joint>
+      <xacro:if value="${forward}">
+        <joint name="${name}_pivot_joint" type="fixed">
+          <origin xyz="${-caster_offset_x/2} 0.0 0.0" rpy="0 0 0" />
+          <parent link="${name}_pivot_link"/>
+          <child link="${name}_footprint" />
+        </joint>
+      </xacro:if>
+      <xacro:unless value="${forward}">
+        <joint name="${name}_pivot_joint" type="fixed">
+          <origin xyz="${caster_offset_x/2} 0.0 0.0" rpy="0 0 0" />
+          <parent link="${name}_pivot_link"/>
+          <child link="${name}_footprint" />
+        </joint>
+      </xacro:unless>
     </xacro:if>
     <link name="${name}_footprint"/>
@@ -27,9 +36,18 @@
     </joint>
     <link name="${name}_link"/>
-    <joint name="${name}_chassis_joint" type="fixed">
-      <origin xyz="0 0 0" rpy="0 0 ${drive_dir_angle}" />
-      <parent link="${name}_link"/>
-      <child link="${name}_chassis_link" />
-    </joint>
+    <xacro:if value="${forward}">
+      <joint name="${name}_chassis_joint" type="fixed">
+        <origin xyz="0 0 0" rpy="0 0 0" />
+        <parent link="${name}_link"/>
+        <child link="${name}_chassis_link" />
+      </joint>
+    </xacro:if>
+    <xacro:unless value="${forward}">
+      <joint name="${name}_chassis_joint" type="fixed">
+        <origin xyz="0 0 0" rpy="0 0 ${M_PI}" />
+        <parent link="${name}_link"/>
+        <child link="${name}_chassis_link" />
+      </joint>
+    </xacro:unless>
     <link name="${name}_chassis_link">
       <inertial>

Commit message: allow simulate backwards driving

File: cob_description/urdf/cob4_base/base.urdf.xacro (robot description, xacro)
@@ -80,22 +80,22 @@
     <!-- arrangement of the three drive_wheel modules -->
     <xacro:if value="${tricycle_mode}">
-      <xacro:drive_wheel parent="${name}_chassis_link" suffix="fl" passive="true" >
+      <xacro:drive_wheel parent="${name}_chassis_link" suffix="fl" passive="true" forward="${forward}">
         <origin xyz="${caster_offset_x/2} ${caster_offset_y} ${caster_offset_z}" rpy="0 0 0" />
       </xacro:drive_wheel>
-      <xacro:drive_wheel parent="${name}_chassis_link" suffix="b" >
+      <xacro:drive_wheel parent="${name}_chassis_link" suffix="b" forward="${forward}">
         <origin xyz="${-caster_offset_x} 0.0 ${caster_offset_z}" rpy="0 0 0" />
       </xacro:drive_wheel>
-      <xacro:drive_wheel parent="${name}_chassis_link" suffix="fr" passive="true">
+      <xacro:drive_wheel parent="${name}_chassis_link" suffix="fr" passive="true" forward="${forward}">
         <origin xyz="${caster_offset_x/2} ${-caster_offset_y} ${caster_offset_z}" rpy="0 0 0" />
       </xacro:drive_wheel>
     </xacro:if>
     <xacro:unless value="${tricycle_mode}">
-      <xacro:drive_wheel parent="${name}_chassis_link" suffix="fl" >
+      <xacro:drive_wheel parent="${name}_chassis_link" suffix="fl" forward="${forward}">
         <origin xyz="${caster_offset_x/2} ${caster_offset_y} ${caster_offset_z}" rpy="0 0 0" />
       </xacro:drive_wheel>
-      <xacro:drive_wheel parent="${name}_chassis_link" suffix="b" >
+      <xacro:drive_wheel parent="${name}_chassis_link" suffix="b" forward="${forward}">
         <origin xyz="${-caster_offset_x} 0.0 ${caster_offset_z}" rpy="0 0 0" />
       </xacro:drive_wheel>
-      <xacro:drive_wheel parent="${name}_chassis_link" suffix="fr" >
+      <xacro:drive_wheel parent="${name}_chassis_link" suffix="fr" forward="${forward}">
         <origin xyz="${caster_offset_x/2} ${-caster_offset_y} ${caster_offset_z}" rpy="0 0 0" />
       </xacro:drive_wheel>

File: cob_description/urdf/drive_wheel/drive_wheel.urdf.xacro (robot description, xacro)
@@ -6,5 +6,5 @@
   <xacro:property name="caster_mass" value="5.9" />
   <xacro:property name="wheel_mass" value="0.44036" />
-  <xacro:macro name="cob_wheel" params="parent suffix reflect drive_vel:=^ passive:=false">
+  <xacro:macro name="cob_wheel" params="parent suffix reflect drive_vel:=^ passive:=false forward:=true">
     <xacro:if value="${passive}">
       <joint name="${parent}_${suffix}_wheel_joint" type="continuous">
@@ -12,5 +12,10 @@
         <parent link="${parent}_rotation_link"/>
         <child link="${parent}_${suffix}_wheel_link"/>
-        <axis xyz="0 1 0" />
+        <xacro:if value="${forward}">
+          <axis xyz="0 1 0" />
+        </xacro:if>
+        <xacro:unless value="${forward}">
+          <axis xyz="0 -1 0" />
+        </xacro:unless>
         <safety_controller  k_velocity="10" />
         <limit effort="0.0" velocity="${drive_vel}"/>
@@ -23,5 +28,10 @@
         <parent link="${parent}_rotation_link"/>
         <child link="${parent}_${suffix}_wheel_link"/>
-        <axis xyz="0 1 0" />
+        <xacro:if value="${forward}">
+          <axis xyz="0 1 0" />
+        </xacro:if>
+        <xacro:unless value="${forward}">
+          <axis xyz="0 -1 0" />
+        </xacro:unless>
         <safety_controller  k_velocity="10" />
         <limit effort="100" velocity="${drive_vel}"/>
@@ -97,9 +107,9 @@
     </xacro:unless>
   </xacro:macro>
-  <xacro:macro name="drive_wheel" params="*origin parent suffix drive_vel:=^|100 steer_vel:=^|100 passive:=false">
+  <xacro:macro name="drive_wheel" params="*origin parent suffix drive_vel:=^|100 steer_vel:=^|100 passive:=false forward:=true">
     <xacro:cob_caster_hub parent="${parent}" suffix="${suffix}_caster" passive="${passive}" >
       <xacro:insert_block name="origin" />
     </xacro:cob_caster_hub>
-    <xacro:cob_wheel parent="${suffix}_caster" suffix="r" reflect="-1"  passive="${passive}" />
+    <xacro:cob_wheel parent="${suffix}_caster" suffix="r" reflect="-1"  passive="${passive}" forward="${forward}" />
     <!-- extensions -->
     <xacro:cob_caster_gazebo suffix="${suffix}" />
