Commit message: fixed path to file

File: cob_description/urdf/ur_arm/ur10_arm.urdf.xacro (robot description, xacro)
@@ -4,6 +4,6 @@
        xmlns:interface="http://playerstage.sourceforge.net/gazebo/xmlschema/#interface"
        xmlns:xacro="http://ros.org/wiki/xacro">
-	<include filename="$(find ur_description)/urdf/ur5.urdf.xacro" />
-	<xacro:macro name="cob_ur5" params="parent name *origin">
+	<include filename="$(find ur_description)/urdf/ur10.urdf.xacro" />
+	<xacro:macro name="ur10" params="parent name *origin">
 		<!-- mount the arm to the robot -->
 		<joint name="${name}_base_joint" type="fixed" >
@@ -13,5 +13,5 @@
 		</joint>
 		<!-- include universal_robot arm -->
-		<xacro:ur5_robot prefix="arm_"/>
+		<xacro:ur10_robot prefix="arm_">  </xacro:ur10_robot>
 	</xacro:macro>
 </robot>

Commit message: added arm_ee_link

File: cob_description/urdf/ur_arm/ur10_arm.urdf.xacro (robot description, xacro)
@@ -5,4 +5,5 @@
        xmlns:xacro="http://ros.org/wiki/xacro">
 	<include filename="$(find ur_description)/urdf/ur10.urdf.xacro" />
+	<property name="wrist_3_length" value="0.0857" />
 	<xacro:macro name="ur10" params="parent name *origin">
 		<!-- mount the arm to the robot -->
@@ -14,4 +15,11 @@
 		<!-- include universal_robot arm -->
 		<xacro:ur10_robot prefix="arm_">  </xacro:ur10_robot>
+		<!-- additional ee_link -->
+		<joint name="${name}_ee_fixed_joint" type="fixed">
+			<parent link="${name}_wrist_3_link" />
+			<child link = "${name}_ee_link" />
+			<origin xyz="0.0 ${wrist_3_length} 0.0" rpy="0.0 0.0 ${pi/2.0}" />
+		</joint>
+		<link name="${name}_ee_link" />
 	</xacro:macro>
 </robot>

File: cob_description/urdf/ur_arm/ur5_arm.urdf.xacro (robot description, xacro)
@@ -5,4 +5,5 @@
        xmlns:xacro="http://ros.org/wiki/xacro">
 	<include filename="$(find ur_description)/urdf/ur5.urdf.xacro" />
+	<property name="wrist_3_length" value="0.0823" />
 	<xacro:macro name="ur5" params="parent name *origin">
 		<!-- mount the arm to the robot -->
@@ -14,4 +15,11 @@
 		<!-- include universal_robot arm -->
 		<xacro:ur5_robot prefix="arm_"/>
+		<!-- additional ee_link -->
+		<joint name="${name}_ee_fixed_joint" type="fixed">
+			<parent link="${name}_wrist_3_link" />
+			<child link = "${name}_ee_link" />
+			<origin xyz="0.0 ${wrist_3_length} 0.0" rpy="0.0 0.0 ${pi/2.0}" />
+		</joint>
+		<link name="${name}_ee_link" />
 	</xacro:macro>
 </robot>

Commit message: fixed some includes and property definitions

File: cob_description/urdf/ur_arm/ur10_arm.urdf.xacro (robot description, xacro)
@@ -4,4 +4,5 @@
        xmlns:interface="http://playerstage.sourceforge.net/gazebo/xmlschema/#interface"
        xmlns:xacro="http://ros.org/wiki/xacro">
+	<include filename="$(find cob_description)/urdf/common.xacro" />
 	<include filename="$(find ur_description)/urdf/ur10.urdf.xacro" />
 	<property name="wrist_3_length" value="0.0857" />
@@ -19,5 +20,5 @@
 			<parent link="${name}_wrist_3_link" />
 			<child link = "${name}_ee_link" />
-			<origin xyz="0.0 ${wrist_3_length} 0.0" rpy="0.0 0.0 ${pi/2.0}" />
+			<origin xyz="0.0 ${wrist_3_length} 0.0" rpy="0.0 0.0 ${M_PI/2.0}" />
 		</joint>
 		<link name="${name}_ee_link" />

File: cob_description/urdf/ur_arm/ur5_arm.urdf.xacro (robot description, xacro)
@@ -4,4 +4,5 @@
        xmlns:interface="http://playerstage.sourceforge.net/gazebo/xmlschema/#interface"
        xmlns:xacro="http://ros.org/wiki/xacro">
+	<include filename="$(find cob_description)/urdf/common.xacro" />
 	<include filename="$(find ur_description)/urdf/ur5.urdf.xacro" />
 	<property name="wrist_3_length" value="0.0823" />
@@ -19,5 +20,5 @@
 			<parent link="${name}_wrist_3_link" />
 			<child link = "${name}_ee_link" />
-			<origin xyz="0.0 ${wrist_3_length} 0.0" rpy="0.0 0.0 ${pi/2.0}" />
+			<origin xyz="0.0 ${wrist_3_length} 0.0" rpy="0.0 0.0 ${M_PI/2.0}" />
 		</joint>
 		<link name="${name}_ee_link" />

Commit message: ee_link is now back in ur_description

File: cob_description/urdf/ur_arm/ur10_arm.urdf.xacro (robot description, xacro)
@@ -13,11 +13,4 @@
     <!-- include universal_robot arm -->
     <xacro:ur10_robot prefix="arm_"/>
-    <!-- additional ee_link -->
-    <joint name="${name}_ee_fixed_joint" type="fixed">
-      <parent link="${name}_wrist_3_link" />
-      <child link = "${name}_ee_link" />
-      <origin xyz="0.0 ${wrist_3_length} 0.0" rpy="0.0 0.0 ${M_PI/2.0}" />
-    </joint>
-    <link name="${name}_ee_link" />
   </xacro:macro>
 </robot>

File: cob_description/urdf/ur_arm/ur5_arm.urdf.xacro (robot description, xacro)
@@ -13,11 +13,4 @@
     <!-- include universal_robot arm -->
     <xacro:ur5_robot prefix="arm_"/>
-    <!-- additional ee_link -->
-    <joint name="${name}_ee_fixed_joint" type="fixed">
-      <parent link="${name}_wrist_3_link" />
-      <child link = "${name}_ee_link" />
-      <origin xyz="0.0 ${wrist_3_length} 0.0" rpy="0.0 0.0 ${M_PI/2.0}" />
-    </joint>
-    <link name="${name}_ee_link" />
   </xacro:macro>
 </robot>

Commit message: un-hardcodize ur-macro

File: cob_description/urdf/ur_arm/ur10_arm.urdf.xacro (robot description, xacro)
@@ -10,8 +10,8 @@
       <insert_block name="origin" />
       <parent link="${parent}" />
-      <child link="arm_base_link" />
+      <child link="${name}_base_link" />
     </joint>
     <!-- include universal_robot arm -->
-    <xacro:ur10_robot prefix="arm_"/>
+    <xacro:ur10_robot prefix="${name}_"/>
   </xacro:macro>
 </robot>

File: cob_description/urdf/ur_arm/ur5_arm.urdf.xacro (robot description, xacro)
@@ -10,8 +10,8 @@
       <insert_block name="origin" />
       <parent link="${parent}" />
-      <child link="arm_base_link" />
+      <child link="${name}_base_link" />
     </joint>
     <!-- include universal_robot arm -->
-    <xacro:ur5_robot prefix="arm_"/>
+    <xacro:ur5_robot prefix="${name}_"/>
   </xacro:macro>
 </robot>
