Commit message: temporary commit for torso inertias

File: cob_description/urdf/cob4_torso/torso.gazebo.xacro (robot description, xacro)
@@ -3,18 +3,22 @@
   <xacro:macro name="torso_gazebo" params="name">
     <gazebo reference="${name}_base_link">
-            <material>IPA/LightGrey</material>
+      <material>IPA/LightGrey</material>
       <turnGravityOff>false</turnGravityOff>
+      <selfCollide>true</selfCollide>
     </gazebo>
     <gazebo reference="${name}_1_link">
       <material>IPA/LightGrey</material>
       <turnGravityOff>false</turnGravityOff>
+      <selfCollide>true</selfCollide>
     </gazebo>
     <gazebo reference="${name}_2_link">
       <material>IPA/LightGrey</material>
       <turnGravityOff>false</turnGravityOff>
+      <selfCollide>true</selfCollide>
     </gazebo>
     <gazebo reference="${name}_3_link">
       <material>IPA/LightGrey</material>
       <turnGravityOff>false</turnGravityOff>
+      <selfCollide>true</selfCollide>
     </gazebo>
   </xacro:macro>

File: cob_description/urdf/cob4_torso/torso.urdf.xacro (robot description, xacro)
@@ -24,5 +24,5 @@
       <calibration rising="${torso_1_ref}"/>
       <axis xyz="0 0 1" />
-      <dynamics damping="2.0" friction="0.0"/>
+      <dynamics damping="0.0" friction="0.0"/>
       <limit effort="100" lower="-6.2831" upper="6.2831" velocity="1.4"/>
     </joint>
@@ -40,5 +40,5 @@
       <calibration rising="${torso_2_ref}"/>
       <axis xyz="0 0 1" />
-      <dynamics damping="2.0" friction="0.0"/>
+      <dynamics damping="0.0" friction="0.0"/>
       <limit effort="100" lower="-6.2831" upper="6.2831" velocity="1.4"/>
     </joint>
@@ -56,5 +56,5 @@
       <calibration rising="${torso_3_ref}"/>
       <axis xyz="0 0 1" />
-      <dynamics damping="2.0" friction="0.0"/>
+      <dynamics damping="0.0" friction="0.0"/>
       <limit effort="100" lower="-6.2831" upper="6.2831" velocity="1.4"/>
     </joint>
