Commit message: fix torso joint orientation in urdf

File: cob_description/urdf/cob4_torso/torso_2dof.urdf.xacro (robot description, xacro)
@@ -33,5 +33,5 @@
     </link>
     <joint name="${name}_2_joint" type="revolute">
-      <origin xyz="0 -0.14734 0.07547" rpy="-0.5236 0 0" />
+      <origin xyz="0 -0.14734 0.07547" rpy="2.618 0 0" />
       <parent link="${name}_1_link"/>
       <child link="${name}_2_link" />
@@ -48,5 +48,5 @@
     </link>
     <joint name="${name}_3_joint" type="revolute">
-      <origin xyz="0 0.09228 0.13477" rpy="0.5236 0 0" />
+      <origin xyz="0 -0.09228 -0.13477" rpy="-2.618 0 0" />
       <parent link="${name}_2_link"/>
       <child link="${name}_3_link" />

Commit message: fix joint origins for torsos

File: cob_description/urdf/cob4_torso/torso_2dof.urdf.xacro (robot description, xacro)
@@ -8,6 +8,6 @@
     <joint name="${name}_base_joint" type="fixed">
       <insert_block name="origin" />
+      <parent link="${parent}"/>
       <child link="${name}_base_link" />
-      <parent link="${parent}"/>
     </joint>
     <link name="${name}_base_link">
@@ -18,9 +18,21 @@
       </xacro:cylinder_inertial>
 -->
+      <visual>
+        <origin xyz="0 0 0" rpy="0 0 0" />
+        <geometry>
+          <box size="0.001 0.001 0.001" />
+        </geometry>
+      </visual>
+      <collision>
+        <origin xyz="0 0 0" rpy="0 0 0" />
+        <geometry>
+          <box size="0.001 0.001 0.001" />
+        </geometry>
+      </collision>
     </link>
     <joint name="${name}_1_joint" type="fixed">
       <origin xyz="0 0 0.04642" rpy="0 0 0"/>
+      <parent link="${name}_base_link"/>
       <child link="${name}_1_link" />
-      <parent link="${name}_base_link"/>
     </joint>
     <link name="${name}_1_link">
@@ -31,7 +43,19 @@
       </xacro:hollow_spherical_cap_inertial>
 -->
+      <visual>
+        <origin xyz="0 0 0" rpy="0 0 0" />
+        <geometry>
+          <box size="0.001 0.001 0.001" />
+        </geometry>
+      </visual>
+      <collision>
+        <origin xyz="0 0 0" rpy="0 0 0" />
+        <geometry>
+          <box size="0.001 0.001 0.001" />
+        </geometry>
+      </collision>
     </link>
     <joint name="${name}_2_joint" type="revolute">
-      <origin xyz="0 -0.14734 0.07547" rpy="2.618 0 0" />
+      <origin xyz="0 0.14734 0.07547" rpy="0.5236 0 0" />
       <parent link="${name}_1_link"/>
       <child link="${name}_2_link" />
@@ -46,7 +70,19 @@
       </xacro:spherical_cap_inertial>
 -->
+      <visual>
+        <origin xyz="0 0 0" rpy="0 0 0" />
+        <geometry>
+          <box size="0.001 0.001 0.001" />
+        </geometry>
+      </visual>
+      <collision>
+        <origin xyz="0 0 0" rpy="0 0 0" />
+        <geometry>
+          <box size="0.001 0.001 0.001" />
+        </geometry>
+      </collision>
     </link>
     <joint name="${name}_3_joint" type="revolute">
-      <origin xyz="0 -0.09228 -0.13477" rpy="-2.618 0 0" />
+      <origin xyz="0 -0.09228 0.13477" rpy="-0.5236 0 0" />
       <parent link="${name}_2_link"/>
       <child link="${name}_3_link" />
@@ -79,5 +115,19 @@
       <child link="${name}_center_link" />
     </joint>
-    <link name="${name}_center_link"/>
+    <link name="${name}_center_link">
+      <xacro:default_inertial/>
+      <visual>
+        <origin xyz="0 0 0" rpy="0 0 0" />
+        <geometry>
+          <box size="0.001 0.001 0.001" />
+        </geometry>
+      </visual>
+      <collision>
+        <origin xyz="0 0 0" rpy="0 0 0" />
+        <geometry>
+          <box size="0.001 0.001 0.001" />
+        </geometry>
+      </collision>
+    </link>
     <!-- left camera -->
     <xacro:cob_kinect_v0 name="${name}_cam3d_left" ros_topic="torso_cam3d_left" parent="${name}_3_link">

Commit message: move sensors from torso xacro to robot xacro

File: cob_description/urdf/cob4_torso/torso_2dof.urdf.xacro (robot description, xacro)
@@ -3,6 +3,4 @@
   <xacro:include filename="$(find cob_description)/urdf/cob4_torso/torso.gazebo.xacro" />
   <xacro:include filename="$(find cob_description)/urdf/cob4_torso/torso.transmission.xacro" />
-  <xacro:include filename="$(find cob_description)/urdf/sensors/realsense.urdf.xacro" />
-  <xacro:include filename="$(find cob_description)/urdf/sensors/kinect.urdf.xacro" />
   <xacro:macro name="torso" params="parent name *origin">
     <joint name="${name}_base_joint" type="fixed">
@@ -130,16 +128,4 @@
       </collision>
     </link>
-    <!-- left camera -->
-    <xacro:cob_kinect_v0 name="${name}_cam3d_left" ros_topic="torso_cam3d_left" parent="${name}_3_link">
-      <origin xyz="${torso_cam3d_left_x} ${torso_cam3d_left_y} ${torso_cam3d_left_z}" rpy="${torso_cam3d_left_roll} ${torso_cam3d_left_pitch} ${torso_cam3d_left_yaw}" />
-    </xacro:cob_kinect_v0>
-    <!-- right camera -->
-    <xacro:cob_kinect_v0 name="${name}_cam3d_right" ros_topic="torso_cam3d_right" parent="${name}_3_link">
-      <origin xyz="${torso_cam3d_right_x} ${torso_cam3d_right_y} ${torso_cam3d_right_z}" rpy="${torso_cam3d_right_roll} ${torso_cam3d_right_pitch} ${torso_cam3d_right_yaw}" />
-    </xacro:cob_kinect_v0>
-    <!-- down camera -->
-    <xacro:realsense name="${name}_cam3d_down" ros_topic="torso_cam3d_down" parent="${name}_3_link">
-      <origin xyz="${torso_cam3d_down_x} ${torso_cam3d_down_y} ${torso_cam3d_down_z}" rpy="${torso_cam3d_down_roll} ${torso_cam3d_down_pitch} ${torso_cam3d_down_yaw}" />
-    </xacro:realsense>
     <!-- extensions -->
     <xacro:torso_gazebo name="torso" />

File: cob_description/urdf/cob4_torso/torso_static.urdf.xacro (robot description, xacro)
@@ -3,6 +3,4 @@
   <xacro:include filename="$(find cob_description)/urdf/cob4_torso/torso.gazebo.xacro" />
   <xacro:include filename="$(find cob_description)/urdf/cob4_torso/torso.transmission.xacro" />
-  <xacro:include filename="$(find cob_description)/urdf/sensors/realsense.urdf.xacro" />
-  <xacro:include filename="$(find cob_description)/urdf/sensors/kinect.urdf.xacro" />
   <xacro:macro name="torso" params="parent name *origin">
     <joint name="${name}_base_joint" type="fixed">
@@ -126,16 +124,4 @@
       </collision>
     </link>
-    <!-- left camera -->
-    <xacro:cob_kinect_v0 name="${name}_cam3d_left" ros_topic="torso_cam3d_left" parent="${name}_3_link">
-      <origin xyz="${torso_cam3d_left_x} ${torso_cam3d_left_y} ${torso_cam3d_left_z}" rpy="${torso_cam3d_left_roll} ${torso_cam3d_left_pitch} ${torso_cam3d_left_yaw}" />
-    </xacro:cob_kinect_v0>
-    <!-- right camera -->
-    <xacro:cob_kinect_v0 name="${name}_cam3d_right" ros_topic="torso_cam3d_right" parent="${name}_3_link">
-      <origin xyz="${torso_cam3d_right_x} ${torso_cam3d_right_y} ${torso_cam3d_right_z}" rpy="${torso_cam3d_right_roll} ${torso_cam3d_right_pitch} ${torso_cam3d_right_yaw}" />
-    </xacro:cob_kinect_v0>
-    <!-- down camera -->
-    <xacro:realsense name="${name}_cam3d_down" ros_topic="torso_cam3d_down" parent="${name}_3_link">
-      <origin xyz="${torso_cam3d_down_x} ${torso_cam3d_down_y} ${torso_cam3d_down_z}" rpy="${torso_cam3d_down_roll} ${torso_cam3d_down_pitch} ${torso_cam3d_down_yaw}" />
-    </xacro:realsense>
     <!-- extensions -->
     <xacro:torso_gazebo name="torso" />
