Commit message: New center joint on torso

File: cob_description/urdf/cob4_torso/torso.urdf.xacro (robot description, xacro)
@@ -62,5 +62,5 @@
       <inertial>
         <mass value="20" />
-        <origin xyz="0 0 0.3" rpy="0 0 0"/>
+        <origin xyz="0 0 0.18566" rpy="0 0 0"/>
       <inertia ixx="0.1" ixy="0" ixz="0" iyy="0.01" iyz="0" izz="0.01" />
       </inertial>
@@ -78,4 +78,16 @@
         </geometry>
       </collision>
+    </link>
+    <joint name="torso_3center_joint" type="fixed">
+      <origin xyz="0.0 0.0 0.18566" rpy="0 0 0" />
+      <child link="torso_center_link" />
+      <parent link="torso_3_link"/>
+    </joint>
+    <link name="torso_center_link">
+      <inertial>
+        <origin xyz="0 0 0" rpy="0 0 0"/>
+        <mass value="0.1"/>
+        <inertia ixx="0.01" ixy="0" ixz="0" iyy="0.01" iyz="0" izz="0.01" />
+      </inertial>
     </link>
     <!-- left camera -->

Commit message: New center joint on torso

File: cob_description/urdf/cob4_torso/torso.urdf.xacro (robot description, xacro)
@@ -79,5 +79,5 @@
       </collision>
     </link>
-    <joint name="torso_3center_joint" type="fixed">
+    <joint name="torso_center_joint" type="fixed">
       <origin xyz="0.0 0.0 0.18566" rpy="0 0 0" />
       <child link="torso_center_link" />

Commit message: correct inertias for cob4 torso

File: cob_description/urdf/cob4_torso/torso.urdf.xacro (robot description, xacro)
@@ -12,9 +12,7 @@
     </joint>
     <link name="torso_base_link">
-      <inertial>
-        <origin xyz="0 0 0" rpy="0 0 0"/>
-        <mass value="0.1"/>
-        <inertia ixx="0.01" ixy="0" ixz="0" iyy="0.01" iyz="0" izz="0.01" />
-      </inertial>
+       <xacro:cylinder_inertial radius="0.300" length="0.046" mass="5.0">
+        <origin xyz="0 0 0" rpy="0 0 0" />
+      </xacro:cylinder_inertial>
     </link>
     <joint name="torso_1_joint" type="revolute">
@@ -28,9 +26,7 @@
     </joint>
     <link name="torso_1_link">
-      <inertial>
-        <origin xyz="0 0 0" rpy="0 0 0"/>
-        <mass value="50"/>
-        <inertia ixx="0.01" ixy="0" ixz="0" iyy="0.01" iyz="0" izz="0.01" />
-      </inertial>
+      <xacro:hollow_spherical_cap_inertial r="0.295" h="0.075" t="0.010" mass="6">
+          <origin xyz="0.006 0.010 0.110" rpy="0 0 0"/>
+      </xacro:hollow_spherical_cap_inertial>
     </link>
     <joint name="torso_2_joint" type="revolute">
@@ -40,13 +36,11 @@
       <calibration rising="${torso_2_ref}"/>
       <axis xyz="0 0 1" />
-      <dynamics damping="0.0" friction="0.0"/>
+      <dynamics damping="1.0" friction="0.0"/>
       <limit effort="100" lower="-6.2831" upper="6.2831" velocity="1.4"/>
     </joint>
     <link name="torso_2_link">
-      <inertial>
-        <origin xyz="0 0 0" rpy="0 0 0"/>
-        <mass value="5"/>
-        <inertia ixx="0.01" ixy="0" ixz="0" iyy="0.01" iyz="0" izz="0.01" />
-      </inertial>
+        <xacro:spherical_cap_inertial r="0.295" h="0.075" mass="19.5">
+            <origin xyz="0.034 0.102 0.092" rpy="0 0 0"/>
+        </xacro:spherical_cap_inertial>
     </link>
     <joint name="torso_3_joint" type="revolute">
@@ -60,9 +54,7 @@
     </joint>
     <link name="torso_3_link">
-      <inertial>
-        <mass value="20" />
-        <origin xyz="0 0 0.18566" rpy="0 0 0"/>
-      <inertia ixx="0.1" ixy="0" ixz="0" iyy="0.01" iyz="0" izz="0.01" />
-      </inertial>
+       <xacro:cylinder_inertial radius="0.250" length="0.610" mass="23.8">
+        <origin xyz="-0.028 0.005 0.233" rpy="0 0 0" />
+      </xacro:cylinder_inertial>
       <visual>
         <origin xyz="0 0 0" rpy="0 0 0" />

File: cob_description/urdf/common.xacro (robot description, xacro)
@@ -35,8 +35,27 @@
     </inertial>
   </xacro:macro>
+  <xacro:macro name="spherical_cap_inertial" params="r h mass *origin">
+    <inertial>
+      <mass value="${mass}" />
+      <insert_block name="origin" />
+      <inertia ixx="${mass*h/(10*(3*r-h))*(3*h*h-15*h*r+20*r*r)}" ixy="0.0" ixz="0.0"
+        iyy="${(-3*h*h*h/20+3*h*h*r/4-4*h*r*r/3+r*r*r)*3*mass/(3*r-h)}" iyz="0.0"
+        izz="${(-3*h*h*h/20+3*h*h*r/4-4*h*r*r/3+r*r*r)*3*mass/(3*r-h)}" />
+      <origin></origin>
+    </inertial>
+  </xacro:macro>
+  <xacro:macro name="hollow_spherical_cap_inertial" params="r h t mass *origin">
+    <inertial>
+      <mass value="${mass}" />
+      <insert_block name="origin" />
+      <inertia ixx="${mass/(10*(2*t*t*t-3*r*t*t-3*h*t*t+6*h*t*r))*(h*h*h*(3*h*h-15*h*r+20*r*r)-(h-t)*(h-t)*(h-t)*(3*(h-t)*(h-t)*(h-t)-15*(h-t)*(r-t)+20*(r-t)*(r-t)))}" ixy="0.0" ixz="0.0"
+        iyy="${mass*t/20*(20*h*h*h*r-10*h*h*h*t-60*h*h*r*r+30*h*h*r*t+120*h*r*r*r-120*h*r*r*t+60*h*r*t*t-15*h*t*t*t-60*r*r*r*t+100*r*r*t*t-65*r*t*t*t+16*t*t*t*t)/(2*t*t*t-3*r*t*t-3*h*t*t+6*h*t*r)}" iyz="0.0"
+        izz="${mass*t/20*(20*h*h*h*r-10*h*h*h*t-60*h*h*r*r+30*h*h*r*t+120*h*r*r*r-120*h*r*r*t+60*h*r*t*t-15*h*t*t*t-60*r*r*r*t+100*r*r*t*t-65*r*t*t*t+16*t*t*t*t)/(2*t*t*t-3*r*t*t-3*h*t*t+6*h*t*r)}" />
+    </inertial>
+  </xacro:macro>
   <xacro:macro name="default_inertial">
     <inertial>
-      <mass value="0.01" />
-      <origin xyz="0 0 0" />
+      <mass value="0.01"/>
+      <origin xyz="0 0 0"/>
       <inertia ixx="0.001" ixy="0.0" ixz="0.0" iyy="0.001" iyz="0.0" izz="0.001" />
     </inertial>

Commit message: use default damping

File: cob_description/urdf/cob4_torso/torso.urdf.xacro (robot description, xacro)
@@ -36,5 +36,5 @@
       <calibration rising="${torso_2_ref}"/>
       <axis xyz="0 0 1" />
-      <dynamics damping="1.0" friction="0.0"/>
+      <dynamics damping="0.0" friction="0.0"/>
       <limit effort="100" lower="-6.2831" upper="6.2831" velocity="1.4"/>
     </joint>

Commit message: fixed center of masses

File: cob_description/urdf/cob4_torso/torso.urdf.xacro (robot description, xacro)
@@ -27,5 +27,6 @@
     <link name="torso_1_link">
       <xacro:hollow_spherical_cap_inertial r="0.295" h="0.075" t="0.010" mass="6">
-          <origin xyz="0.006 0.010 0.110" rpy="0 0 0"/>
+          <!--origin xyz="0.006 0.010 0.110" rpy="0 0 0"/-->
+          <origin xyz="0 0 0" rpy="0 0 0"/>
       </xacro:hollow_spherical_cap_inertial>
     </link>
@@ -41,5 +42,5 @@
     <link name="torso_2_link">
         <xacro:spherical_cap_inertial r="0.295" h="0.075" mass="19.5">
-            <origin xyz="0.034 0.102 0.092" rpy="0 0 0"/>
+            <origin xyz="0.034 0.102 0.092" rpy="0.5236 0 0"/>
         </xacro:spherical_cap_inertial>
     </link>
@@ -76,11 +77,5 @@
       <parent link="torso_3_link"/>
     </joint>
-    <link name="torso_center_link">
-      <inertial>
-        <origin xyz="0 0 0" rpy="0 0 0"/>
-        <mass value="0.1"/>
-        <inertia ixx="0.01" ixy="0" ixz="0" iyy="0.01" iyz="0" izz="0.01" />
-      </inertial>
-    </link>
+    <link name="torso_center_link"/>
     <!-- left camera -->
     <xacro:cob_kinect_v0 name="${name}_cam3d_left" ros_topic="torso_cam3d_left" parent="${name}_3_link">

Commit message: fixed center of gravity and inertia formulas

File: cob_description/urdf/cob4_torso/torso.urdf.xacro (robot description, xacro)
@@ -13,5 +13,5 @@
     <link name="${name}_base_link">
        <xacro:cylinder_inertial radius="0.300" length="0.046" mass="5.0">
-        <origin xyz="0 0 0" rpy="0 0 0" />
+        <origin xyz="0.03 0.08 0.01" rpy="0 0 0" />
       </xacro:cylinder_inertial>
     </link>
@@ -28,5 +28,5 @@
       <xacro:hollow_spherical_cap_inertial r="0.295" h="0.075" t="0.010" mass="6">
           <!--origin xyz="0.006 0.010 0.110" rpy="0 0 0"/-->
-          <origin xyz="0 0 0" rpy="0 0 0"/>
+          <origin xyz="0 0 ${0.075/2}" rpy="0 0 0"/>
       </xacro:hollow_spherical_cap_inertial>
     </link>

File: cob_description/urdf/common.xacro (robot description, xacro)
@@ -39,7 +39,7 @@
       <mass value="${mass}" />
       <insert_block name="origin" />
-      <inertia ixx="${mass*h/(10*(3*r-h))*(3*h*h-15*h*r+20*r*r)}" ixy="0.0" ixz="0.0"
-        iyy="${(-3*h*h*h/20+3*h*h*r/4-4*h*r*r/3+r*r*r)*3*mass/(3*r-h)}" iyz="0.0"
-        izz="${(-3*h*h*h/20+3*h*h*r/4-4*h*r*r/3+r*r*r)*3*mass/(3*r-h)}" />
+      <inertia ixx="${(-3*h*h*h/20+3*h*h*r/4-4*h*r*r/3+r*r*r)*3*mass/(3*r-h)+(3/4*(h-2*r)*(h-2*r)/(3*r-h))*(3/4*(h-2*r)*(h-2*r)/(3*r-h))}" ixy="0.0" ixz="0.0"
+        iyy="${(-3*h*h*h/20+3*h*h*r/4-4*h*r*r/3+r*r*r)*3*mass/(3*r-h)+(3/4*(h-2*r)*(h-2*r)/(3*r-h))*(3/4*(h-2*r)*(h-2*r)/(3*r-h))}" iyz="0.0"
+        izz="${mass*h/(10*(3*r-h))*(3*h*h-15*h*r+20*r*r)}" />
       <origin></origin>
     </inertial>
@@ -49,7 +49,7 @@
       <mass value="${mass}" />
       <insert_block name="origin" />
-      <inertia ixx="${mass/(10*(2*t*t*t-3*r*t*t-3*h*t*t+6*h*t*r))*(h*h*h*(3*h*h-15*h*r+20*r*r)-(h-t)*(h-t)*(h-t)*(3*(h-t)*(h-t)*(h-t)-15*(h-t)*(r-t)+20*(r-t)*(r-t)))}" ixy="0.0" ixz="0.0"
-        iyy="${mass*t/20*(20*h*h*h*r-10*h*h*h*t-60*h*h*r*r+30*h*h*r*t+120*h*r*r*r-120*h*r*r*t+60*h*r*t*t-15*h*t*t*t-60*r*r*r*t+100*r*r*t*t-65*r*t*t*t+16*t*t*t*t)/(2*t*t*t-3*r*t*t-3*h*t*t+6*h*t*r)}" iyz="0.0"
-        izz="${mass*t/20*(20*h*h*h*r-10*h*h*h*t-60*h*h*r*r+30*h*h*r*t+120*h*r*r*r-120*h*r*r*t+60*h*r*t*t-15*h*t*t*t-60*r*r*r*t+100*r*r*t*t-65*r*t*t*t+16*t*t*t*t)/(2*t*t*t-3*r*t*t-3*h*t*t+6*h*t*r)}" />
+      <inertia ixx="${mass/20*(20*h*h*h*r-10*h*h*h*t-60*h*h*r*r+30*h*h*r*t+120*h*r*r*r-120*h*r*r*t+60*h*r*t*t-15*h*t*t*t-60*r*r*r*t+100*r*r*t*t-65*r*t*t*t+16*t*t*t*t)/(2*t*t*-3*r*t-3*h*t+6*h*r)+(3/4*(t-2*r)*(2*r*r-4*r*r+2*r*t-t*t)/(6*r*r-3*r*t-3*r*t+2*t*t))*(3/4*(t-2*r)*(2*r*r-4*r*r+2*r*t-t*t)/(6*r*r-3*r*t-3*r*t+2*t*t))}" ixy="0.0" ixz="0.0"
+        iyy="${mass/20*(20*h*h*h*r-10*h*h*h*t-60*h*h*r*r+30*h*h*r*t+120*h*r*r*r-120*h*r*r*t+60*h*r*t*t-15*h*t*t*t-60*r*r*r*t+100*r*r*t*t-65*r*t*t*t+16*t*t*t*t)/(2*t*t*-3*r*t-3*h*t+6*h*r)+(3/4*(t-2*r)*(2*r*r-4*r*r+2*r*t-t*t)/(6*r*r-3*r*t-3*r*t+2*t*t))*(3/4*(t-2*r)*(2*r*r-4*r*r+2*r*t-t*t)/(6*r*r-3*r*t-3*r*t+2*t*t))}" iyz="0.0"
+        izz="${mass/(10*(2*t*t-3*r*t-3*h*t+6*h*r))*(-20*h*h*h*r+10*h*h*h*t+60*h*h*r*r-30*h*h*r*t-60*h*r*r*t+60*h*r*t*t-15*h*t*t*t+20*r*r*t*t-25*r*t*t*t+8*t*t*t*t)}" />
     </inertial>
   </xacro:macro>

Commit message: fix syntax error

File: cob_description/urdf/cob4_torso/torso.urdf.xacro (robot description, xacro)
@@ -3,5 +3,5 @@
   <xacro:include filename="$(find cob_description)/urdf/cob4_torso/torso.gazebo.xacro" />
   <xacro:include filename="$(find cob_description)/urdf/cob4_torso/torso.transmission.xacro" />
-  <xacro:macro name="torso" params="parent name *origin" dof1:=false dof2:=false dof3:=false">
+  <xacro:macro name="torso" params="parent name *origin dof1:=false dof2:=false dof3:=false">
     <joint name="${name}_base_joint" type="fixed">
       <insert_block name="origin" />
