Commit message: New desire base links and joints name

File: desire_description/urdf/base_desire/base.urdf.xacro (robot description, xacro)
@@ -59,5 +59,5 @@
         <origin xyz="0 0 0" rpy="0 0 0" />
         <geometry>
-          <mesh filename="package://cob_description/meshes/base/pr2_wheel.stl" />
+          <mesh filename="package://cob_description/meshes/base_desire/pr2_wheel.stl" />
         </geometry>
         <material name="Wheel_${suffix}" />
@@ -96,5 +96,5 @@
         <origin xyz="0 0 0" rpy="0 0 0" />
         <geometry>
-          <mesh filename="$(find cob_description)/meshes/base/caster.stl" />
+          <mesh filename="$(find cob_description)/meshes/base_desire/caster.stl" />
         </geometry>
         <material name="Green" />

Commit message: Fixed desired description

File: desire_description/urdf/base_desire/base.urdf.xacro (robot description, xacro)
@@ -59,5 +59,5 @@
         <origin xyz="0 0 0" rpy="0 0 0" />
         <geometry>
-          <mesh filename="package://cob_description/meshes/base_desire/pr2_wheel.stl" />
+          <mesh filename="package://cob_description/meshes/base/pr2_wheel.stl" />
         </geometry>
         <material name="Wheel_${suffix}" />
@@ -96,5 +96,5 @@
         <origin xyz="0 0 0" rpy="0 0 0" />
         <geometry>
-          <mesh filename="$(find cob_description)/meshes/base_desire/caster.stl" />
+          <mesh filename="$(find cob_description)/meshes/base/caster.stl" />
         </geometry>
         <material name="Green" />

Commit message: adapt color

File: desire_description/urdf/base_desire/base.urdf.xacro (robot description, xacro)
@@ -62,5 +62,5 @@
           <mesh filename="package://cob_description/meshes/base/pr2_wheel.stl" />
         </geometry>
-        <material name="IPA/Wheel_${suffix}" />
+        <material name="IPA/LightGrey" />
       </visual>
       <collision>

Commit message: fix file to mesh files

File: desire_description/urdf/base_desire/base.urdf.xacro (robot description, xacro)
@@ -60,5 +60,5 @@
         <origin xyz="0 0 0" rpy="0 0 0" />
         <geometry>
-          <mesh filename="package://cob_description/meshes/base/pr2_wheel.stl" />
+          <mesh filename="package://cob_description/meshes/cob3_base/pr2_wheel.stl" />
         </geometry>
         <material name="IPA/LightGrey" />
@@ -81,5 +81,5 @@
       <limit effort="100" velocity="100"/> <!-- alpha tested velocity and effort limits -->
       <safety_controller  k_velocity="10" />
-      <calibration rising="${ref_position}" falling="${ref_position}" />
+      <calibration rising="${ref_position}" />
       <dynamics damping="0.0" friction="0.0" />
       <insert_block name="origin" />
@@ -97,5 +97,5 @@
         <origin xyz="0 0 0" rpy="0 0 0" />
         <geometry>
-          <mesh filename="$(find cob_description)/meshes/base/caster.stl" />
+          <mesh filename="package://cob_description/meshes/cob3_base/caster.stl" />
         </geometry>
         <material name="IPA/DarkGrey" />

File: desire_description/urdf/head_desire/head.urdf.xacro (robot description, xacro)
@@ -16,5 +16,5 @@
 			<axis xyz="0 0 1" />
 			<dynamics damping="0.1" />
-			<calibration rising="${head_pan_ref}" falling="${head_pan_ref}"/>
+			<calibration rising="${head_pan_ref}"/>
 			<limit effort="100" lower="-1.4" upper="1.4" velocity="0.5"/>
 		</joint>
@@ -45,5 +45,5 @@
 			<axis xyz="0 0 1" />
 			<dynamics damping="0.1" />
-			<calibration rising="${head_tilt_ref}" falling="${head_tilt_ref}"/>
+			<calibration rising="${head_tilt_ref}"/>
 			<limit effort="100" lower="-0.25" upper="0.35" velocity="0.5"/>
 		</joint>

Commit message: switch laser scanner orientation

File: desire_description/urdf/base_desire/base.urdf.xacro (robot description, xacro)
@@ -179,9 +179,9 @@
     <!-- base laser front -->
     <xacro:sick_s300_laser_v0 name="${name}_laser_front" parent="${name}" ros_topic="scan_front_raw" update_rate="10" min_angle="-2.3562" max_angle="2.3562" >
-      <origin xyz="${base_laser_x} ${base_laser_y} ${base_laser_z}" rpy="0 0 0" />
+      <origin xyz="${base_laser_x} ${base_laser_y} ${base_laser_z}" rpy="3.1416 0 0" />
     </xacro:sick_s300_laser_v0>
     <!-- base laser rear -->
     <xacro:sick_s300_laser_v0 name="${name}_laser_rear" parent="${name}" ros_topic="scan_rear_raw" update_rate="10" min_angle="-2.3562" max_angle="2.3562" >
-      <origin xyz="${-base_laser_x} ${base_laser_y} ${base_laser_z}" rpy="0 0 ${M_PI}" />
+      <origin xyz="${-base_laser_x} ${base_laser_y} ${base_laser_z}" rpy="3.1416 0 ${M_PI}" />
     </xacro:sick_s300_laser_v0>
      <!-- cam3d -->

File: raw_description/urdf/base_long/base.urdf.xacro (robot description, xacro)
@@ -215,9 +215,9 @@
     <!-- base laser front -->
     <xacro:sick_s300_laser_v0 name="${name}_laser_front" parent="${name}" ros_topic="scan_front_raw" update_rate="10" min_angle="-2.3562" max_angle="2.3562" >
-      <origin xyz="${base_laser_x} ${-base_laser_y_front} ${base_laser_z}" rpy="0 0 ${-M_PI/4}" />
+      <origin xyz="${base_laser_x} ${-base_laser_y_front} ${base_laser_z}" rpy="3.1416 0 ${-M_PI/4}" />
     </xacro:sick_s300_laser_v0>
     <!-- base laser rear -->
     <xacro:sick_s300_laser_v0 name="${name}_laser_rear" parent="${name}" ros_topic="scan_rear_raw" update_rate="10" min_angle="-2.3562" max_angle="2.3562" >
-      <origin xyz="${-base_laser_x} ${base_laser_y_back} ${base_laser_z}" rpy="0 0 ${-5*M_PI/4}" />
+      <origin xyz="${-base_laser_x} ${base_laser_y_back} ${base_laser_z}" rpy="3.1416 0 ${-5*M_PI/4}" />
     </xacro:sick_s300_laser_v0>
     <!-- battery front-->

File: raw_description/urdf/base_short/base.urdf.xacro (robot description, xacro)
@@ -214,9 +214,9 @@
     <!-- base laser front -->
     <xacro:sick_s300_laser_v0 name="${name}_laser_front" parent="${name}" ros_topic="scan_front_raw" update_rate="10" min_angle="-2.3562" max_angle="2.3562" >
-      <origin xyz="${base_laser_x} ${-base_laser_y_front} ${base_laser_z}" rpy="0 0 ${-M_PI/4}" />
+      <origin xyz="${base_laser_x} ${-base_laser_y_front} ${base_laser_z}" rpy="3.1416 0 ${-M_PI/4}" />
     </xacro:sick_s300_laser_v0>
     <!-- base laser rear -->
     <xacro:sick_s300_laser_v0 name="${name}_laser_rear" parent="${name}" ros_topic="scan_rear_raw" update_rate="10" min_angle="-2.3562" max_angle="2.3562" >
-      <origin xyz="${-base_laser_x} ${base_laser_y_back} ${base_laser_z}" rpy="0 0 ${-5*M_PI/4}" />
+      <origin xyz="${-base_laser_x} ${base_laser_y_back} ${base_laser_z}" rpy="3.1416 0 ${-5*M_PI/4}" />
     </xacro:sick_s300_laser_v0>
     <!-- battery-->

Commit message: use the  macros instead 3.14...

File: desire_description/urdf/base_desire/base.urdf.xacro (robot description, xacro)
@@ -179,9 +179,9 @@
     <!-- base laser front -->
     <xacro:sick_s300_laser_v0 name="${name}_laser_front" parent="${name}" ros_topic="scan_front_raw" update_rate="10" min_angle="-2.3562" max_angle="2.3562" >
-      <origin xyz="${base_laser_x} ${base_laser_y} ${base_laser_z}" rpy="3.1416 0 0" />
+      <origin xyz="${base_laser_x} ${base_laser_y} ${base_laser_z}" rpy="${M_PI} 0 0" />
     </xacro:sick_s300_laser_v0>
     <!-- base laser rear -->
     <xacro:sick_s300_laser_v0 name="${name}_laser_rear" parent="${name}" ros_topic="scan_rear_raw" update_rate="10" min_angle="-2.3562" max_angle="2.3562" >
-      <origin xyz="${-base_laser_x} ${base_laser_y} ${base_laser_z}" rpy="3.1416 0 ${M_PI}" />
+      <origin xyz="${-base_laser_x} ${base_laser_y} ${base_laser_z}" rpy="${M_PI} 0 ${M_PI}" />
     </xacro:sick_s300_laser_v0>
      <!-- cam3d -->

File: raw_description/urdf/base_long/base.urdf.xacro (robot description, xacro)
@@ -215,9 +215,9 @@
     <!-- base laser front -->
     <xacro:sick_s300_laser_v0 name="${name}_laser_front" parent="${name}" ros_topic="scan_front_raw" update_rate="10" min_angle="-2.3562" max_angle="2.3562" >
-      <origin xyz="${base_laser_x} ${-base_laser_y_front} ${base_laser_z}" rpy="3.1416 0 ${-M_PI/4}" />
+      <origin xyz="${base_laser_x} ${-base_laser_y_front} ${base_laser_z}" rpy="${M_PI} 0 ${-M_PI/4}" />
     </xacro:sick_s300_laser_v0>
     <!-- base laser rear -->
     <xacro:sick_s300_laser_v0 name="${name}_laser_rear" parent="${name}" ros_topic="scan_rear_raw" update_rate="10" min_angle="-2.3562" max_angle="2.3562" >
-      <origin xyz="${-base_laser_x} ${base_laser_y_back} ${base_laser_z}" rpy="3.1416 0 ${-5*M_PI/4}" />
+      <origin xyz="${-base_laser_x} ${base_laser_y_back} ${base_laser_z}" rpy="${M_PI} 0 ${-5*M_PI/4}" />
     </xacro:sick_s300_laser_v0>
     <!-- battery front-->

File: raw_description/urdf/base_short/base.urdf.xacro (robot description, xacro)
@@ -214,9 +214,9 @@
     <!-- base laser front -->
     <xacro:sick_s300_laser_v0 name="${name}_laser_front" parent="${name}" ros_topic="scan_front_raw" update_rate="10" min_angle="-2.3562" max_angle="2.3562" >
-      <origin xyz="${base_laser_x} ${-base_laser_y_front} ${base_laser_z}" rpy="3.1416 0 ${-M_PI/4}" />
+      <origin xyz="${base_laser_x} ${-base_laser_y_front} ${base_laser_z}" rpy="${M_PI} 0 ${-M_PI/4}" />
     </xacro:sick_s300_laser_v0>
     <!-- base laser rear -->
     <xacro:sick_s300_laser_v0 name="${name}_laser_rear" parent="${name}" ros_topic="scan_rear_raw" update_rate="10" min_angle="-2.3562" max_angle="2.3562" >
-      <origin xyz="${-base_laser_x} ${base_laser_y_back} ${base_laser_z}" rpy="3.1416 0 ${-5*M_PI/4}" />
+      <origin xyz="${-base_laser_x} ${base_laser_y_back} ${base_laser_z}" rpy="${M_PI} 0 ${-5*M_PI/4}" />
     </xacro:sick_s300_laser_v0>
     <!-- battery-->
