Commit message: simplified lookat component

File: cob_description/urdf/lookat/lookat.urdf.xacro (robot description, xacro)
@@ -4,6 +4,4 @@
        xmlns:interface="http://playerstage.sourceforge.net/gazebo/xmlschema/#interface"
        xmlns:xacro="http://ros.org/wiki/xacro">
-	<include filename="$(find cob_description)/urdf/lookat/lookat.gazebo.xacro" />
-	<include filename="$(find cob_description)/urdf/lookat/lookat.transmission.xacro" />
 	<xacro:macro name="cob_lookat" params="name parent *origin *axis">
 		<joint name="${name}_axis_joint" type="fixed">
@@ -19,5 +17,5 @@
 			<insert_block name="axis" />	<!--axis xyz="-1 0 0" /-->
 			<dynamics damping="5.0" friction="0.5"/>
-			<limit effort="100" lower="0.3" upper="5.0" velocity="1"/>
+			<limit effort="100" lower="-5.0" upper="5.0" velocity="1"/>
 		</joint>
 		<link name="${name}_x_link"/>
@@ -49,4 +47,5 @@
 		</joint>
 		<link name="${name}_focus_frame">
+<!--
 			<visual>
 				<origin xyz="0 0 0" rpy="0 0 0" />
@@ -56,8 +55,6 @@
 				<material name="IPA/Black" />
 			</visual>
+-->
 		</link>
-		<!-- extensions -->
-		<xacro:cob_lookat_gazebo name="${name}" />
-		<xacro:cob_lookat_transmission name="${name}" />
 	</xacro:macro>
 </robot>

Commit message: latest changes in lookat component

File: cob_description/urdf/lookat/lookat.urdf.xacro (robot description, xacro)
@@ -1,17 +1,24 @@
 <?xml version="1.0"?>
 <robot xmlns:sensor="http://playerstage.sourceforge.net/gazebo/xmlschema/#sensor"
-       xmlns:controller="http://playerstage.sourceforge.net/gazebo/xmlschema/#controller"
-       xmlns:interface="http://playerstage.sourceforge.net/gazebo/xmlschema/#interface"
-       xmlns:xacro="http://ros.org/wiki/xacro">
+	   xmlns:controller="http://playerstage.sourceforge.net/gazebo/xmlschema/#controller"
+	   xmlns:interface="http://playerstage.sourceforge.net/gazebo/xmlschema/#interface"
+	   xmlns:xacro="http://ros.org/wiki/xacro">
 	<xacro:macro name="cob_lookat" params="name parent *origin *axis">
-		<joint name="${name}_axis_joint" type="fixed">
+		<!-- joint between torso_upper_neck_tilt_link and lookat_base_link -->
+		<joint name="${name}_base_joint" type="fixed">
 			<insert_block name="origin" />
 			<parent link="${parent}"/>
-			<child link="${name}_axis_link"/>
+			<child link="${name}_base_link"/>
 		</joint>
-		<link name="${name}_axis_link"/>
-		<joint name="${name}_back_joint" type="prismatic">
+		<link name="${name}_base_link">
+			<inertial>
+				<origin xyz="0 0 0" rpy="0 0 0"/>
+				<mass value="0.5"/>
+				<inertia ixx="0.01" ixy="0" ixz="0" iyy="0.01" iyz="0" izz="0.01" />
+			</inertial>
+		</link>
+		<joint name="${name}_lin_joint" type="prismatic">
 			<origin xyz="0 0 0" rpy="0 0 0" />
-			<parent link="${name}_axis_link"/>
+			<parent link="${name}_base_link"/>
 			<child link="${name}_x_link"/>
 			<insert_block name="axis" />	<!--axis xyz="-1 0 0" /-->

Commit message: make lookat work with raw

File: cob_description/urdf/lookat/lookat.urdf.xacro (robot description, xacro)
@@ -4,5 +4,5 @@
 	   xmlns:interface="http://playerstage.sourceforge.net/gazebo/xmlschema/#interface"
 	   xmlns:xacro="http://ros.org/wiki/xacro">
-	<xacro:macro name="cob_lookat" params="name parent *origin *axis">
+	<xacro:macro name="cob_lookat" params="name parent *origin *axis lower upper">
 		<!-- joint between torso_upper_neck_tilt_link and lookat_base_link -->
 		<joint name="${name}_base_joint" type="fixed">
@@ -24,5 +24,5 @@
 			<insert_block name="axis" />	<!--axis xyz="-1 0 0" /-->
 			<dynamics damping="5.0" friction="0.5"/>
-			<limit effort="100" lower="-5.0" upper="5.0" velocity="1"/>
+			<limit effort="100" lower="${lower}" upper="${upper}" velocity="1"/>
 		</joint>
 		<link name="${name}_x_link"/>

Commit message: make lookat arbitrarily fast

File: cob_description/urdf/lookat/lookat.urdf.xacro (robot description, xacro)
@@ -14,6 +14,6 @@
       <child link="${name}_x_link"/>
       <insert_block name="axis" />  <!--axis xyz="-1 0 0" /-->
-      <dynamics damping="5.0" friction="0.5"/>
-      <limit effort="100" lower="${lower}" upper="${upper}" velocity="1"/>
+      <dynamics damping="0.0" friction="0.0"/>
+      <limit effort="100000" lower="${lower}" upper="${upper}" velocity="100000"/>
     </joint>
     <link name="${name}_x_link"/>
@@ -23,6 +23,6 @@
       <child link="${name}_y_link"/>
       <axis xyz="1 0 0" />
-      <dynamics damping="5.0" friction="0.5"/>
-      <limit effort="100" lower="-${M_PI}" upper="${M_PI}" velocity="1"/>
+      <dynamics damping="0.0" friction="0.0"/>
+      <limit effort="100000" lower="-${M_PI}" upper="${M_PI}" velocity="100000"/>
     </joint>
     <link name="${name}_y_link"/>
@@ -32,6 +32,6 @@
       <child link="${name}_z_link"/>
       <axis xyz="0 1 0" />
-      <dynamics damping="5.0" friction="0.5"/>
-      <limit effort="100" lower="-${M_PI}" upper="${M_PI}" velocity="1"/>
+      <dynamics damping="0.0" friction="0.0"/>
+      <limit effort="100000" lower="-${M_PI}" upper="${M_PI}" velocity="100000"/>
     </joint>
     <link name="${name}_z_link"/>
@@ -41,6 +41,6 @@
       <child link="${name}_focus_frame"/>
       <axis xyz="0 0 1" />
-      <dynamics damping="5.0" friction="0.5"/>
-      <limit effort="100" lower="-${M_PI}" upper="${M_PI}" velocity="1"/>
+      <dynamics damping="0.0" friction="0.0"/>
+      <limit effort="100000" lower="-${M_PI}" upper="${M_PI}" velocity="100000"/>
     </joint>
     <link name="${name}_focus_frame">
