Commit message: modified raw3-1 urdf description

File: raw_description/urdf/boxgripper/boxgripper.urdf.xacro (robot description, xacro)
@@ -21,5 +21,5 @@
 				<origin xyz="0 0 0" rpy="0 0 0" />
 				<geometry>
-					<box size="0.005 0.2 0.04"/>
+					<box size="0.003 0.26 0.04"/>
 				</geometry>
 				<material name="Grey" />
@@ -28,5 +28,5 @@
 				<origin xyz="0 0 0" rpy="0 0 0" />
 				<geometry>
-					<box size="0.005 0.2 0.04"/>
+					<box size="0.003 0.26 0.04"/>
 				</geometry>
 			</collision>

File: raw_description/urdf/torso/torso.urdf.xacro (robot description, xacro)
@@ -70,5 +70,5 @@
    			<parent link="${name}_1_link"/>
 			<child link="torso_2_link"/>
-			<axis xyz="0 0 -1.0" />
+			<axis xyz="0 1.0 0" />
 			<dynamics damping="0.1" />
 			<calibration rising="0.0"/>

Commit message: better visual/collision model for the boxgripper

File: raw_description/urdf/boxgripper/boxgripper.urdf.xacro (robot description, xacro)
@@ -7,7 +7,57 @@
 	<xacro:macro name="raw_boxgripper" params="name parent *origin">
 		<!-- joint between arm_ee_link and raw_boxgripper_link -->
-		<joint name="${name}_joint" type="fixed" >
+		<joint name="${name}_base_joint" type="fixed" >
 			<insert_block name="origin" />
 			<parent link="${parent}" />
+			<child link="${name}_base_link" />
+		</joint>
+		<link name="${name}_base_link">
+			<visual>
+				<origin xyz="0.001 0 0" rpy="0 0 0" />
+				<geometry>
+					<box size="0.002 0.045 0.045"/>
+				</geometry>
+				<material name="IPA/DarkGrey" />
+			</visual>
+			<collision>
+				<origin xyz="0.001 0 0" rpy="0 0 0" />
+				<geometry>
+					<box size="0.002 0.045 0.045"/>
+				</geometry>
+			</collision>
+			<inertial>
+				<origin xyz="0 0 0" rpy="0 0 0"/>
+				<mass value="0.02"/>
+				<inertia ixx="1" ixy="0" ixz="0" iyy="1" iyz="0" izz="1" />
+			</inertial>
+		</link>
+		<joint name="${name}_middle_joint" type="fixed" >
+			<origin xyz="0.02 0 -0.061" rpy="0 -0.24 0" />
+			<parent link="${name}_base_link" />
+			<child link="${name}_middle_link" />
+		</joint>
+		<link name="${name}_middle_link">
+			<inertial>
+				<origin xyz="0 0 0" rpy="0 0 0"/>
+				<mass value="0.02"/>
+				<inertia ixx="1" ixy="0" ixz="0" iyy="1" iyz="0" izz="1" />
+			</inertial>
+			<visual>
+				<origin xyz="0 0 0" rpy="0 0 0" />
+				<geometry>
+					<box size="0.002 0.03 0.1433"/>
+				</geometry>
+				<material name="IPA/DarkGrey" />
+			</visual>
+			<collision>
+				<origin xyz="0 0 0" rpy="0 0 0" />
+				<geometry>
+					<box size="0.002 0.03 0.1433"/>
+				</geometry>
+			</collision>
+		</link>
+		<joint name="${name}_joint" type="fixed" >
+			<origin xyz="0.04 0 -0.122" rpy="0 0.12 0" />
+			<parent link="${name}_base_link" />
 			<child link="${name}_link" />
 		</joint>
@@ -21,5 +71,5 @@
 				<origin xyz="0 0 0" rpy="0 0 0" />
 				<geometry>
-					<box size="0.003 0.26 0.04"/>
+					<box size="0.002 0.26 0.04"/>
 				</geometry>
 				<material name="IPA/DarkGrey" />
@@ -28,5 +78,5 @@
 				<origin xyz="0 0 0" rpy="0 0 0" />
 				<geometry>
-					<box size="0.003 0.26 0.04"/>
+					<box size="0.002 0.26 0.04"/>
 				</geometry>
 			</collision>

Commit message: fixed box_gripper position

File: raw_description/urdf/boxgripper/boxgripper.urdf.xacro (robot description, xacro)
@@ -21,5 +21,5 @@
 				<origin xyz="0 0 0" rpy="0 0 0" />
 				<geometry>
-					<box size="0.003 0.26 0.04"/>
+					<box size="0.04 0.26 0.003"/>
 				</geometry>
 				<material name="IPA/DarkGrey" />
@@ -28,5 +28,5 @@
 				<origin xyz="0 0 0" rpy="0 0 0" />
 				<geometry>
-					<box size="0.003 0.26 0.04"/>
+					<box size="0.04 0.26 0.003"/>
 				</geometry>
 			</collision>

Commit message: adjusted boxgripper collision geometry

File: raw_description/urdf/boxgripper/boxgripper.urdf.xacro (robot description, xacro)
@@ -26,7 +26,7 @@
 			</visual>
 			<collision>
-				<origin xyz="0 0 0" rpy="0 0 0" />
+				<origin xyz="0.06 0 -0.02" rpy="0 0 0" />
 				<geometry>
-					<box size="0.04 0.26 0.003"/>
+					<box size="0.16 0.28 0.07"/>
 				</geometry>
 			</collision>

Commit message: modified boxgripper

File: raw_description/urdf/boxgripper/boxgripper.urdf.xacro (robot description, xacro)
@@ -7,7 +7,13 @@
 	<xacro:macro name="raw_boxgripper" params="name parent *origin">
 		<!-- joint between arm_ee_link and raw_boxgripper_link -->
-		<joint name="${name}_joint" type="fixed" >
+		<joint name="${name}_base_joint" type="fixed" >
 			<insert_block name="origin" />
 			<parent link="${parent}" />
+			<child link="${name}_base_link" />
+		</joint>
+		<link name="${name}_base_link"/>
+		<joint name="${name}_joint" type="fixed" >
+			<origin xyz="0.04 0.122 0" rpy="0 0 0.12" />
+			<parent link="${name}_base_link" />
 			<child link="${name}_link" />
 		</joint>
@@ -21,12 +27,12 @@
 				<origin xyz="0 0 0" rpy="0 0 0" />
 				<geometry>
-					<box size="0.04 0.26 0.003"/>
+					<box size="0.002 0.04 0.26"/>
 				</geometry>
 				<material name="IPA/DarkGrey" />
 			</visual>
 			<collision>
-				<origin xyz="0.06 0 -0.02" rpy="0 0 0" />
+				<origin xyz="-0.02 -0.06 0" rpy="0 0 -0.45" />
 				<geometry>
-					<box size="0.16 0.28 0.07"/>
+					<box size="0.05 0.16 0.27"/>
 				</geometry>
 			</collision>

Commit message: use boxgripper mesh in urdf

File: raw_description/urdf/boxgripper/boxgripper.urdf.xacro (robot description, xacro)
@@ -32,8 +32,12 @@
 			</visual>
 			<collision>
-				<origin xyz="-0.02 -0.06 0" rpy="0 0 -0.45" />
+				<origin xyz="0 0 0" rpy="0 0 -0.45" />
+				<geometry>
+				  <mesh filename="package://raw_description/meshes/boxgripper/boxgripper_collision.stl"/>
+				</geometry>
+				<!--origin xyz="-0.02 -0.06 0" rpy="0 0 -0.45" />
 				<geometry>
 					<box size="0.05 0.16 0.27"/>
-				</geometry>
+				</geometry-->
 			</collision>
 		</link>

Commit message: better approximation of inertias

File: raw_description/urdf/boxgripper/boxgripper.urdf.xacro (robot description, xacro)
@@ -16,9 +16,7 @@
     </joint>
     <link name="${name}_link">
-      <inertial>
-        <origin xyz="0 0 0" rpy="0 0 0"/>
-        <mass value="0.57307"/>
-        <inertia ixx="1.415" ixy="0" ixz="0" iyy="0.819" iyz="0" izz="0.819" />
-      </inertial>
+       <xacro:box_inertial x="0.002" y="0.04" z="0.26" mass="0.57307">
+        <origin xyz="0.0 0.0 0.0" rpy="0 0 0" />
+      </xacro:box_inertial>
       <visual>
         <origin xyz="0 0 0" rpy="0 0 0" />
