Commit message: Defined new colors

File: cob_description/urdf/materials.urdf.xacro (robot description, xacro)
@@ -22,4 +22,10 @@
 		<color rgba="0.0 0.0 0.0 1.0"/>
 	</material>
+        <material name="Transparent">
+                <color rgba="0.81 0.81 0.81 0.0"/>
+        </material>
+        <material name="LightBlue">
+                <color rgba="0.624 0.698 0.858 1"/>
+        </material>
 	<material name="Caster">
 		<texture filename="package://pr2_ogre/Media/materials/textures/pr2_caster_texture.png" />

Commit message: unify materials

File: cob_description/urdf/materials.urdf.xacro (robot description, xacro)
@@ -7,9 +7,15 @@
     <color rgba="0.4 0.4 0.4 1.0"/>
   </material>
+  <material name="IPA/Black">
+    <color rgba="0.0 0.0 0.0 1.0"/>
+  </material>
+  <material name="IPA/Metall">
+    <color rgba="0.7 0.7 0.7 1.0"/>
+  </material>
+  <material name="IPA/YellowRubber">
+    <color rgba="0.4 0.27 0.16 1.0"/>
+  </material>
   <material name="IPA/Orange">
     <color rgba="1.0 0.4 0.0 1.0"/>
-  </material>
-  <material name="IPA/Black">
-    <color rgba="0.0 0.0 0.0 1.0"/>
   </material>
   <material name="IPA/Blue">
