Commit message: fixed gazebo_plugins

File: cob_description/urdf/cob3_base/base.gazebo.xacro (robot description, xacro)
@@ -10,10 +10,10 @@
       <kp  value="1000000.0" />
       <kd  value="1.0" />
-      <material>IPA/LightGrey</material>
+      <material value="IPA/LightGrey"/>
     </gazebo>
   </xacro:macro>
   <xacro:macro name="cob_caster_gazebo" params="suffix">
     <gazebo reference="${suffix}_caster_rotation_link">
-      <material value="PR2/caster_texture" />
+      <material value="IPA/Metal" />
     </gazebo>
   </xacro:macro>
@@ -29,4 +29,5 @@
 				<updateRate>100.0</updateRate>
 				<bumperTopicName>${name}_bumper</bumperTopicName>
+				<frameName>world</frameName>
 			</plugin>
 		</sensor>

File: cob_description/urdf/cob4_base/base.gazebo.xacro (robot description, xacro)
@@ -10,10 +10,10 @@
       <kp  value="1000000.0" />
       <kd  value="1.0" />
-      <material>IPA/LightGrey</material>
+      <material value="IPA/LightGrey"/>
     </gazebo>
   </xacro:macro>
   <xacro:macro name="cob_caster_gazebo" params="suffix">
     <gazebo reference="${suffix}_caster_rotation_link">
-      <material value="PR2/caster_texture" />
+      <material value="IPA/Metal" />
     </gazebo>
   </xacro:macro>
@@ -28,4 +28,5 @@
 				<alwaysOn>true</alwaysOn>
 				<updateRate>100.0</updateRate>
+				<frameName>world</frameName>
 				<bumperTopicName>${name}_bumper</bumperTopicName>
 			</plugin>

File: cob_description/urdf/sensors/hokuyo_SR400_laser.gazebo.xacro (robot description, xacro)
@@ -7,30 +7,31 @@
     <gazebo reference="${name}_link">
       <sensor name="${name}" type="ray">
-		<always_on>true</always_on>
-		<update_rate>${update_rate}</update_rate>
-		<pose>0 0 0 0 0 0</pose>
-		<visualize>false</visualize>
-		<ray>
-			<scan>
-				<horizontal>
-					<samples>150</samples>
-					<resolution>1.0</resolution>
-					<min_angle>${min_angle}</min_angle>
-					<max_angle>${max_angle}</max_angle>
-				</horizontal>
-			</scan>
-			<range>
-				<min>0.30</min>
-				<max>5.0</max>
-				<resolution>0.01</resolution>
-			</range>
-		</ray>
-		<plugin name="gazebo_ros_${name}_controller" filename="libgazebo_ros_laser.so">
-			<gaussianNoise>0.005</gaussianNoise>
-			<alwaysOn>true</alwaysOn>
-			<updateRate>${update_rate}</updateRate>
-			<topicName>${ros_topic}</topicName>
-			<frameName>${name}_link</frameName>
-		</plugin>
+        <always_on>true</always_on>
+        <update_rate>${update_rate}</update_rate>
+        <pose>0 0 0 0 0 0</pose>
+        <visualize>false</visualize>
+        <ray>
+          <scan>
+            <horizontal>
+              <samples>150</samples>
+              <resolution>1.0</resolution>
+              <min_angle>${min_angle}</min_angle>
+              <max_angle>${max_angle}</max_angle>
+            </horizontal>
+          </scan>
+          <range>
+            <min>0.30</min>
+            <max>5.0</max>
+            <resolution>0.01</resolution>
+          </range>
+        </ray>
+        <plugin name="gazebo_ros_${name}_controller" filename="libgazebo_ros_laser.so">
+          <gaussianNoise>0.005</gaussianNoise>
+          <alwaysOn>true</alwaysOn>
+          <updateRate>${update_rate}</updateRate>
+          <topicName>${ros_topic}</topicName>
+          <frameName>${name}_link</frameName>
+          <hokuyoMinIntensity>101.0</hokuyoMinIntensity>
+        </plugin>
       </sensor>
       <material>IPA/LightGrey</material>

File: cob_description/urdf/sensors/hokuyo_lx30_laser.gazebo.xacro (robot description, xacro)
@@ -7,30 +7,31 @@
     <gazebo reference="${name}_link">
       <sensor name="${name}" type="ray">
-		<always_on>true</always_on>
-		<update_rate>${update_rate}</update_rate>
-		<pose>0 0 0 0 0 0</pose>
-		<visualize>false</visualize>
-		<ray>
-			<scan>
-				<horizontal>
-					<samples>640</samples>
-					<resolution>1.0</resolution>
-					<min_angle>${min_angle}</min_angle>
-					<max_angle>${max_angle}</max_angle>
-				</horizontal>
-			</scan>
-			<range>
-				<min>0.05</min>
-				<max>10.0</max>
-				<resolution>0.01</resolution>
-			</range>
-		</ray>
-		<plugin name="gazebo_ros_${name}_controller" filename="libgazebo_ros_laser.so">
-			<gaussianNoise>0.005</gaussianNoise>
-			<alwaysOn>true</alwaysOn>
-			<updateRate>${update_rate}</updateRate>
-			<topicName>${ros_topic}</topicName>
-			<frameName>${name}_link</frameName>
-		</plugin>
+        <always_on>true</always_on>
+        <update_rate>${update_rate}</update_rate>
+        <pose>0 0 0 0 0 0</pose>
+        <visualize>false</visualize>
+        <ray>
+          <scan>
+            <horizontal>
+              <samples>640</samples>
+              <resolution>1.0</resolution>
+              <min_angle>${min_angle}</min_angle>
+              <max_angle>${max_angle}</max_angle>
+            </horizontal>
+          </scan>
+          <range>
+            <min>0.05</min>
+            <max>10.0</max>
+            <resolution>0.01</resolution>
+          </range>
+        </ray>
+        <plugin name="gazebo_ros_${name}_controller" filename="libgazebo_ros_laser.so">
+          <gaussianNoise>0.005</gaussianNoise>
+          <alwaysOn>true</alwaysOn>
+          <updateRate>${update_rate}</updateRate>
+          <topicName>${ros_topic}</topicName>
+          <frameName>${name}_link</frameName>
+          <hokuyoMinIntensity>101.0</hokuyoMinIntensity>
+        </plugin>
       </sensor>
       <material>IPA/LightGrey</material>

File: cob_description/urdf/sensors/kinect.gazebo.xacro (robot description, xacro)
@@ -6,65 +6,42 @@
 <xacro:macro name="cob_kinect_gazebo_v0" params="name ros_topic">
   <gazebo reference="${name}_frame">
-	<sensor type="depth" name="${name}_frame_sensor">
-		<always_on>true</always_on>
-		<update_rate>20.0</update_rate>
-		<camera>
-			<horizontal_fov>${62.0*M_PI/180.0}</horizontal_fov>
-			<image>
-				<format>R8G8B8</format>
-				<width>640</width>
-				<height>480</height>
-			</image>
-			<clip>
-				<near>0.1</near>
-				<far>100</far>
-			</clip>
-		</camera>
-		<plugin name="${name}_depth_frame_controller" filename="libgazebo_ros_openni_kinect.so">
-			<alwaysOn>true</alwaysOn>
-			<updateRate>20.0</updateRate>
-			<imageTopicName>${ros_topic}/ir/image_raw</imageTopicName>
-			<cameraInfoTopicName>${ros_topic}/ir/camera_info</cameraInfoTopicName>
-			<depthImageTopicName>${ros_topic}/depth/image_raw</depthImageTopicName>
-			<depthImageInfoTopicName>${ros_topic}/depth/camera_info</depthImageInfoTopicName>
-			<pointCloudTopicName>${ros_topic}/depth/points</pointCloudTopicName>
-			<frameName>${name}_link</frameName>
-			<pointCloudCutoff>0.5</pointCloudCutoff>
-			<distortionK1>0.00000001</distortionK1>
-			<distortionK2>0.00000001</distortionK2>
-			<distortionK3>0.00000001</distortionK3>
-			<distortionT1>0.00000001</distortionT1>
-			<distortionT2>0.00000001</distortionT2>
-		</plugin>
-	</sensor>
-	<sensor type="depth" name="${name}_frame_sensor">
-		<always_on>true</always_on>
-		<update_rate>20.0</update_rate>
-		<camera>
-			<horizontal_fov>${62.0*M_PI/180.0}</horizontal_fov>
-			<image>
-				<format>R8G8B8</format>
-				<width>640</width>
-				<height>480</height>
-			</image>
-			<clip>
-				<near>0.1</near>
-				<far>100</far>
-			</clip>
-		</camera>
-		<plugin name="${name}_rgb_frame_controller" filename="libgazebo_ros_openni_kinect.so">
-			<alwaysOn>true</alwaysOn>
-			<updateRate>20.0</updateRate>
-			<imageTopicName>${ros_topic}/rgb/image_raw</imageTopicName>
-			<cameraInfoTopicName>${ros_topic}/rgb/camera_info</cameraInfoTopicName>
-			<frameName>${name}_link</frameName>
-			<pointCloudCutoff>0.5</pointCloudCutoff>
-			<distortionK1>0.00000001</distortionK1>
-			<distortionK2>0.00000001</distortionK2>
-			<distortionK3>0.00000001</distortionK3>
-			<distortionT1>0.00000001</distortionT1>
-			<distortionT2>0.00000001</distortionT2>
-		</plugin>
-	</sensor>
+    <sensor type="depth" name="${name}_frame_sensor">
+      <always_on>true</always_on>
+      <update_rate>20.0</update_rate>
+      <camera>
+        <horizontal_fov>${62.0*M_PI/180.0}</horizontal_fov>
+        <image>
+          <format>R8G8B8</format>
+          <width>640</width>
+          <height>480</height>
+        </image>
+        <clip>
+          <near>0.1</near>
+          <far>100</far>
+        </clip>
+      </camera>
+      <plugin name="${name}_controller" filename="libgazebo_ros_openni_kinect.so">
+        <alwaysOn>true</alwaysOn>
+        <updateRate>20.0</updateRate>
+        <cameraName>${name}</cameraName>
+        <frameName>${name}_link</frameName>
+        <imageTopicName>${ros_topic}/rgb/image_raw</imageTopicName>
+        <depthImageTopicName>${ros_topic}/depth/image_raw</depthImageTopicName>
+        <pointCloudTopicName>${ros_topic}/depth/points</pointCloudTopicName>
+        <cameraInfoTopicName>${ros_topic}/rgb/camera_info</cameraInfoTopicName>
+        <depthImageCameraInfoTopicName>${ros_topic}/depth/camera_info</depthImageCameraInfoTopicName>
+        <pointCloudCutoff>0.5</pointCloudCutoff>
+        <hackBaseline>0.0</hackBaseline>
+        <distortionK1>0.0</distortionK1>
+        <distortionK2>0.0</distortionK2>
+        <distortionK3>0.0</distortionK3>
+        <distortionT1>0.0</distortionT1>
+        <distortionT2>0.0</distortionT2>
+        <CxPrime>0.0</CxPrime>
+        <Cx>0.0</Cx>
+        <Cy>0.0</Cy>
+        <focalLength>0.0</focalLength>
+      </plugin>
+    </sensor>
     <material>IPA/LightGrey</material>
   </gazebo>

File: cob_description/urdf/sensors/phidgets_distance.gazebo.xacro (robot description, xacro)
@@ -5,35 +5,36 @@
        xmlns:xacro="http://ros.org/wiki/xacro">
   <xacro:macro name="phidgets_distance_gazebo_v0" params="name ros_topic update_rate">
-	<gazebo reference="${name}_link">
-		<sensor name="${name}" type="ray">
-			<always_on>true</always_on>
-			<update_rate>${update_rate}</update_rate>
-			<pose>0 0 0 0 0 0</pose>
-			<visualize>false</visualize>
-			<ray>
-				<scan>
-					<horizontal>
-						<samples>10</samples>
-						<resolution>1.0</resolution>
-						<min_angle>-0.2</min_angle>
-						<max_angle>0.2</max_angle>
-					</horizontal>
-				</scan>
-				<range>
-					<min>0.01</min>		<!-- real value from sensor datasheet is 0.04m -->
-					<max>0.4</max>		<!-- real value from sensor datasheet is 0.30m -->
-					<resolution>0.005</resolution>
-				</range>
-			</ray>
-			<plugin name="gazebo_ros_${name}_controller" filename="libgazebo_ros_laser.so">
-				<gaussianNoise>0.005</gaussianNoise>
-				<alwaysOn>true</alwaysOn>
-				<updateRate>${update_rate}</updateRate>
-				<topicName>${ros_topic}</topicName>
-				<frameName>/${name}_link</frameName>
-			</plugin>
-		</sensor>
-		<material>IPA/LightGrey</material>
-	</gazebo>
+  <gazebo reference="${name}_link">
+    <sensor name="${name}" type="ray">
+      <always_on>true</always_on>
+      <update_rate>${update_rate}</update_rate>
+      <pose>0 0 0 0 0 0</pose>
+      <visualize>false</visualize>
+      <ray>
+        <scan>
+          <horizontal>
+            <samples>10</samples>
+            <resolution>1.0</resolution>
+            <min_angle>-0.2</min_angle>
+            <max_angle>0.2</max_angle>
+          </horizontal>
+        </scan>
+        <range>
+          <min>0.01</min>    <!-- real value from sensor datasheet is 0.04m -->
+          <max>0.4</max>    <!-- real value from sensor datasheet is 0.30m -->
+          <resolution>0.005</resolution>
+        </range>
+      </ray>
+      <plugin name="gazebo_ros_${name}_controller" filename="libgazebo_ros_laser.so">
+        <gaussianNoise>0.005</gaussianNoise>
+        <alwaysOn>true</alwaysOn>
+        <updateRate>${update_rate}</updateRate>
+        <topicName>${ros_topic}</topicName>
+        <frameName>/${name}_link</frameName>
+        <hokuyoMinIntensity>101.0</hokuyoMinIntensity>
+      </plugin>
+    </sensor>
+    <material>IPA/LightGrey</material>
+  </gazebo>
   </xacro:macro>
 </robot>

File: cob_description/urdf/sensors/prosilica.gazebo.xacro (robot description, xacro)
@@ -24,18 +24,20 @@
 					<alwaysOn>true</alwaysOn>
 					<updateRate>10.0</updateRate>
+					<cameraName>${name}</cameraName>
+					<frameName>/${name}_link</frameName>
 					<topicName>${ros_topic}_image_data</topicName>
 					<imageTopicName>/${ros_topic}/image_raw</imageTopicName>
 					<cameraInfoTopicName>/${ros_topic}/camera_info</cameraInfoTopicName>
 					<pollServiceName>/${name}/request_image</pollServiceName>
-					<frameName>/${name}_link</frameName>
 					<CxPrime>697.69</CxPrime>
 					<Cx>697.69</Cx>
 					<Cy>530.51</Cy>
-					<focal_length>1450</focal_length>	<!-- image_width / (2*tan(hfov_radian /2)) -->
-					<distortion_k1>0.00000001</distortion_k1>
-					<distortion_k2>0.00000001</distortion_k2>
-					<distortion_k3>0.00000001</distortion_k3>
-					<distortion_t1>0.00000001</distortion_t1>
-					<distortion_t2>0.00000001</distortion_t2>
+					<focalLength>2278.722731</focalLength>	<!-- focal_length = width_ / (2.0 * tan( HFOV/2.0 )) -->
+					<hackBaseline>0.0</hackBaseline>
+					<distortionK1>0.0</distortionK1>
+					<distortionK2>0.0</distortionK2>
+					<distortionK3>0.0</distortionK3>
+					<distortionT1>0.0</distortionT1>
+					<distortionT2>0.0</distortionT2>
 				</plugin>
 			</sensor>

File: cob_description/urdf/sensors/sick_s300_laser.gazebo.xacro (robot description, xacro)
@@ -6,32 +6,33 @@
   <xacro:macro name="sick_s300_laser_gazebo_v0" params="name ros_topic update_rate min_angle max_angle">
     <gazebo reference="${name}_link">
-		<sensor name="${name}" type="ray">
-			<always_on>true</always_on>
-			<update_rate>${update_rate}</update_rate>
-			<pose>0 0 0 0 0 0</pose>
-			<visualize>false</visualize>
-			<ray>
-				<scan>
-					<horizontal>
-						<samples>541</samples>
-						<resolution>1.0</resolution>
-						<min_angle>${min_angle}</min_angle>
-						<max_angle>${max_angle}</max_angle>
-					</horizontal>
-				</scan>
-				<range>
-					<min>0.05</min>
-					<max>30.0</max>
-					<resolution>0.03</resolution>
-				</range>
-			</ray>
-			<plugin name="gazebo_ros_${name}_controller" filename="libgazebo_ros_laser.so">
+      <sensor name="${name}" type="ray">
+        <always_on>true</always_on>
+        <update_rate>${update_rate}</update_rate>
+        <pose>0 0 0 0 0 0</pose>
+        <visualize>false</visualize>
+        <ray>
+          <scan>
+            <horizontal>
+              <samples>541</samples>
+              <resolution>1.0</resolution>
+              <min_angle>${min_angle}</min_angle>
+              <max_angle>${max_angle}</max_angle>
+            </horizontal>
+          </scan>
+          <range>
+            <min>0.05</min>
+            <max>30.0</max>
+            <resolution>0.03</resolution>
+          </range>
+        </ray>
+        <plugin name="gazebo_ros_${name}_controller" filename="libgazebo_ros_laser.so">
           <gaussianNoise>0.005</gaussianNoise>
           <alwaysOn>true</alwaysOn>
           <updateRate>${update_rate}</updateRate>
           <topicName>${ros_topic}</topicName>
-				<frameName>${name}_link</frameName>
-			</plugin>
-		</sensor>
+          <frameName>${name}_link</frameName>
+          <hokuyoMinIntensity>101.0</hokuyoMinIntensity>
+        </plugin>
+      </sensor>
       <!--material value="IPA/LightGrey" /-->
     </gazebo>

File: cob_description/urdf/sensors/tof.gazebo.xacro (robot description, xacro)
@@ -7,38 +7,38 @@
 <xacro:macro name="cob_tof_gazebo_v0" params="name ros_topic">
   <gazebo reference="${name}_frame">
-	<sensor name="${name}_sensor" type="ray">
-		<always_on>true</always_on>
-		<update_rate>10</update_rate>	<!--max50Hz-->
-		<pose>0 0 0.05 0 0 0</pose>
-		<visualize>false</visualize>
-		<ray>
-			<scan>
-				<horizontal>
-					<samples>176</samples>		<!--true value 176-->
-					<resolution>1.0</resolution>
-					<min_angle>-0.38</min_angle>
-					<max_angle>0.38</max_angle>
-				</horizontal>
-				<vertical>
-					<samples>144</samples>		<!--true value 144 -->
-					<resolution>1.0</resolution>
-					<min_angle>-0.3</min_angle>
-					<max_angle>0.3</max_angle>
-				</vertical>
-			</scan>
-			<range>
-				<min>0.80</min>		<!--0.8m min calibrated range-->
-				<max>5.0</max>		<!--5.0m max calibrated range-->
-				<resolution>0.010</resolution>
-			</range>
-		</ray>
-		<plugin name="tof_controller" filename="libgazebo_ros_block_laser.so">
-			<gaussianNoise>0.005</gaussianNoise>
-			<alwaysOn>true</alwaysOn>
-			<updateRate>30</updateRate> 	<!--max 50Hz, cob3 30Hz -->
-			<topicName>${ros_topic}</topicName>
-			<frameName>/${name}_frame</frameName>
-		</plugin>
-	</sensor>
+    <sensor name="${name}_sensor" type="ray">
+      <always_on>true</always_on>
+      <update_rate>10</update_rate>  <!--max50Hz-->
+      <pose>0 0 0.05 0 0 0</pose>
+      <visualize>false</visualize>
+      <ray>
+        <scan>
+          <horizontal>
+            <samples>176</samples>    <!--true value 176-->
+            <resolution>1.0</resolution>
+            <min_angle>-0.38</min_angle>
+            <max_angle>0.38</max_angle>
+          </horizontal>
+          <vertical>
+            <samples>144</samples>    <!--true value 144 -->
+            <resolution>1.0</resolution>
+            <min_angle>-0.3</min_angle>
+            <max_angle>0.3</max_angle>
+          </vertical>
+        </scan>
+        <range>
+          <min>0.80</min>    <!--0.8m min calibrated range-->
+          <max>5.0</max>    <!--5.0m max calibrated range-->
+          <resolution>0.010</resolution>
+        </range>
+      </ray>
+      <plugin name="tof_controller" filename="libgazebo_ros_block_laser.so">
+        <gaussianNoise>0.005</gaussianNoise>
+        <alwaysOn>true</alwaysOn>
+        <updateRate>30</updateRate>   <!--max 50Hz, cob3 30Hz -->
+        <topicName>${ros_topic}</topicName>
+        <frameName>/${name}_frame</frameName>
+      </plugin>
+    </sensor>
     <material value="IPA/LightGrey" />
     <turnGravityOff>true</turnGravityOff>

File: desire_description/urdf/base_desire/base.gazebo.xacro (robot description, xacro)
@@ -10,10 +10,10 @@
       <kp  value="1000000.0" />
       <kd  value="1.0" />
-      <material value="PR2/wheel_${suffix}" />
+      <material value="IPA/LightGrey"/>
     </gazebo>
   </xacro:macro>
   <xacro:macro name="desire_caster_gazebo_v0" params="suffix">
     <gazebo reference="${suffix}_caster_rotation_link">
-      <material value="PR2/caster_texture" />
+      <material value="IPA/Metal" />
     </gazebo>
   </xacro:macro>
@@ -28,4 +28,5 @@
 				<alwaysOn>true</alwaysOn>
 				<updateRate>100.0</updateRate>
+				<frameName>world</frameName>
 				<bumperTopicName>${name}_bumper</bumperTopicName>
 			</plugin>

File: raw_description/urdf/base_long/base.gazebo.xacro (robot description, xacro)
@@ -33,4 +33,5 @@
           <alwaysOn>true</alwaysOn>
           <updateRate>100.0</updateRate>
+          <frameName>world</frameName>
           <bumperTopicName>${name}_bumper</bumperTopicName>
         </plugin>

Commit message: remove material physic properties of wheels to use default, fixes #90

File: cob_description/urdf/cob3_base/base.gazebo.xacro (robot description, xacro)
@@ -3,9 +3,5 @@
   <xacro:macro name="cob_wheel_gazebo" params="suffix parent">
     <gazebo reference="${parent}_${suffix}_wheel_link">
-      <mu1 value="100.0" />
-      <mu2 value="100.0" />
-      <kp  value="1000000.0" />
-      <kd  value="1.0" />
-      <material value="IPA/LightGrey"/>
+          <material value="IPA/LightGrey"/>
     </gazebo>
   </xacro:macro>

File: raw_description/urdf/base_long/base.gazebo.xacro (robot description, xacro)
@@ -3,9 +3,5 @@
   <xacro:macro name="cob_wheel_gazebo" params="suffix parent">
     <gazebo reference="${parent}_${suffix}_wheel_link">
-      <mu1 value="100.0" />
-      <mu2 value="100.0" />
-      <kp  value="1000000.0" />
-      <kd  value="1.0" />
-      <!--material value="IPA/YellowRubber" /-->
+      <material value="IPA/LightGrey"/>
     </gazebo>
   </xacro:macro>

File: raw_description/urdf/base_short/base.gazebo.xacro (robot description, xacro)
@@ -3,9 +3,5 @@
   <xacro:macro name="cob_wheel_gazebo" params="suffix parent">
     <gazebo reference="${parent}_${suffix}_wheel_link">
-      <mu1 value="100.0" />
-      <mu2 value="100.0" />
-      <kp  value="1000000.0" />
-      <kd  value="1.0" />
-      <!--material value="IPA/YellowRubber" /-->
+      <material value="IPA/LightGrey"/>
     </gazebo>
   </xacro:macro>
