Commit message: removed bumpers and changed transmission config to new syntax

File: cob_description/urdf/cob3_base/base.gazebo.xacro (robot description, xacro)
@@ -12,19 +12,4 @@
   </xacro:macro>
   <xacro:macro name="base_gazebo" params="name">
-  <gazebo reference="${name}_link">
-    <selfCollide>true</selfCollide>
-    <sensor name='${name}_contact_sensor' type='contact'>
-      <contact>
-        <collision>${name}_link_geom</collision>
-      </contact>
-      <plugin name="${name}_gazebo_ros_bumper_controller" filename="libgazebo_ros_bumper.so">
-        <alwaysOn>true</alwaysOn>
-        <updateRate>100.0</updateRate>
-        <bumperTopicName>${name}_bumper</bumperTopicName>
-		<frameName>world</frameName>
-		</plugin>
-    </sensor>
-    <material>IPA/LightGrey</material>
-  </gazebo>
     <gazebo>
     <plugin name="p3d_base_controller" filename="libgazebo_ros_p3d.so">

File: cob_description/urdf/cob3_base/base.transmission.xacro (robot description, xacro)
@@ -5,7 +5,8 @@
     <transmission name="${parent}_${suffix}_wheel_trans">
       <type>transmission_interface/SimpleTransmission</type>
-      <joint name="${parent}_${suffix}_wheel_joint" />
+      <joint name="${parent}_${suffix}_wheel_joint" >
+        <hardwareInterface>EffortJointInterface</hardwareInterface>
+      </joint>
       <actuator name="${parent}_${suffix}_wheel_motor">
-        <hardwareInterface>EffortJointInterface</hardwareInterface>
         <mechanicalReduction>${reflect * 624/35 * 80/18}</mechanicalReduction>
       </actuator>
@@ -16,7 +17,8 @@
     <transmission name="${suffix}_rotation_trans">
       <type>transmission_interface/SimpleTransmission</type>
-      <joint name="${suffix}_rotation_joint" />
+      <joint name="${suffix}_rotation_joint" >
+        <hardwareInterface>EffortJointInterface</hardwareInterface>
+      </joint>
       <actuator name="${suffix}_rotation_motor" >
-       <hardwareInterface>EffortJointInterface</hardwareInterface>
         <mechanicalReduction>${-1 * 624/35 * 80/18}</mechanicalReduction>
       </actuator>

File: cob_description/urdf/cob3_head/head_v1.transmission.xacro (robot description, xacro)
@@ -4,5 +4,7 @@
     <transmission name="${name}_axis_trans">
       <type>transmission_interface/SimpleTransmission</type>
-      <joint name="${name}_axis_joint"/>
+      <joint name="${name}_axis_joint">
+        <hardwareInterface>EffortJointInterface</hardwareInterface>
+      </joint>
       <actuator name="${name}_axis_motor">
         <hardwareInterface>EffortJointInterface</hardwareInterface>

File: cob_description/urdf/cob3_head/head_v2.transmission.xacro (robot description, xacro)
@@ -8,5 +8,7 @@
         <mechanicalReduction>1</mechanicalReduction>
       </actuator>
-      <joint name="${name}_axis_joint"/>
+      <joint name="${name}_axis_joint">
+        <hardwareInterface>EffortJointInterface</hardwareInterface>
+      </joint>
     </transmission>
   </xacro:macro>

File: cob_description/urdf/cob3_torso/torso_v1.transmission.xacro (robot description, xacro)
@@ -4,5 +4,7 @@
     <transmission name="${name}_lower_neck_pan_trans">
       <type>transmission_interface/SimpleTransmission</type>
-      <joint name="${name}_lower_neck_pan_joint"/>
+      <joint name="${name}_lower_neck_pan_joint">
+        <hardwareInterface>EffortJointInterface</hardwareInterface>
+      </joint>
       <actuator name="${name}_lower_neck_pan_motor">
         <hardwareInterface>EffortJointInterface</hardwareInterface>
@@ -12,5 +14,7 @@
     <transmission name="${name}_lower_neck_tilt_trans">
       <type>transmission_interface/SimpleTransmission</type>
-      <joint name="${name}_lower_neck_tilt_joint"/>
+      <joint name="${name}_lower_neck_tilt_joint">
+        <hardwareInterface>EffortJointInterface</hardwareInterface>
+      </joint>
       <actuator name="${name}_lower_neck_tilt_motor">
         <hardwareInterface>EffortJointInterface</hardwareInterface>
@@ -20,5 +24,7 @@
     <transmission name="${name}_upper_neck_pan_trans">
       <type>transmission_interface/SimpleTransmission</type>
-      <joint name="${name}_upper_neck_pan_joint"/>
+      <joint name="${name}_upper_neck_pan_joint">
+        <hardwareInterface>EffortJointInterface</hardwareInterface>
+      </joint>
       <actuator name="${name}_upper_neck_pan_motor">
         <hardwareInterface>EffortJointInterface</hardwareInterface>
@@ -28,5 +34,7 @@
     <transmission name="${name}_upper_neck_tilt_trans">
       <type>transmission_interface/SimpleTransmission</type>
-      <joint name="${name}_upper_neck_tilt_joint"/>
+      <joint name="${name}_upper_neck_tilt_joint">
+        <hardwareInterface>EffortJointInterface</hardwareInterface>
+      </joint>
       <actuator name="${name}_upper_neck_tilt_motor">
         <hardwareInterface>EffortJointInterface</hardwareInterface>

File: cob_description/urdf/cob3_torso/torso_v2.transmission.xacro (robot description, xacro)
@@ -4,5 +4,7 @@
     <transmission name="${name}_lower_neck_tilt_trans">
       <type>transmission_interface/SimpleTransmission</type>
-      <joint name="${name}_lower_neck_tilt_joint"/>
+      <joint name="${name}_lower_neck_tilt_joint">
+        <hardwareInterface>EffortJointInterface</hardwareInterface>
+      </joint>
       <actuator name="${name}_lower_neck_tilt_motor">
         <hardwareInterface>EffortJointInterface</hardwareInterface>
@@ -12,5 +14,7 @@
     <transmission name="${name}_pan_trans">
       <type>transmission_interface/SimpleTransmission</type>
-      <joint name="${name}_pan_joint"/>
+      <joint name="${name}_pan_joint">
+        <hardwareInterface>EffortJointInterface</hardwareInterface>
+      </joint>
       <actuator name="${name}_pan_motor">
         <hardwareInterface>EffortJointInterface</hardwareInterface>
@@ -20,5 +24,7 @@
     <transmission name="${name}_upper_neck_tilt_trans">
       <type>transmission_interface/SimpleTransmission</type>
-      <joint name="${name}_upper_neck_tilt_joint"/>
+      <joint name="${name}_upper_neck_tilt_joint">
+        <hardwareInterface>EffortJointInterface</hardwareInterface>
+      </joint>
       <actuator name="${name}_upper_neck_tilt_motor">
         <hardwareInterface>EffortJointInterface</hardwareInterface>

File: cob_description/urdf/cob3_tray/tray.transmission.xacro (robot description, xacro)
@@ -4,5 +4,7 @@
     <transmission name="${name}_trans">
       <type>transmission_interface/SimpleTransmission</type>
-      <joint name="${name}_joint"/>
+      <joint name="${name}_joint">
+        <hardwareInterface>EffortJointInterface</hardwareInterface>
+      </joint>
       <actuator name="${name}_motor">
         <hardwareInterface>EffortJointInterface</hardwareInterface>

File: cob_description/urdf/cob3_tray/tray_3DOF.transmission.xacro (robot description, xacro)
@@ -4,5 +4,7 @@
     <transmission name="${name}_1_trans">
       <type>transmission_interface/SimpleTransmission</type>
-      <joint name="${name}_1_joint"/>
+      <joint name="${name}_1_joint">
+        <hardwareInterface>EffortJointInterface</hardwareInterface>
+      </joint>
       <actuator name="${name}_1_motor">
         <hardwareInterface>EffortJointInterface</hardwareInterface>
@@ -12,5 +14,7 @@
     <transmission name="${name}_2_trans">
       <type>transmission_interface/SimpleTransmission</type>
-      <joint name="${name}_2_joint"/>
+      <joint name="${name}_2_joint">
+        <hardwareInterface>EffortJointInterface</hardwareInterface>
+      </joint>
       <actuator name="${name}_2_motor">
         <hardwareInterface>EffortJointInterface</hardwareInterface>
@@ -20,5 +24,7 @@
     <transmission name="${name}_3_trans">
       <type>transmission_interface/SimpleTransmission</type>
-      <joint name="${name}_3_joint"/>
+      <joint name="${name}_3_joint">
+        <hardwareInterface>EffortJointInterface</hardwareInterface>
+      </joint>
       <actuator name="${name}_3_motor">
         <hardwareInterface>EffortJointInterface</hardwareInterface>

File: cob_description/urdf/cob4_base/base.gazebo.xacro (robot description, xacro)
@@ -15,19 +15,4 @@
     </gazebo>
   </xacro:macro>
-  <xacro:macro name="base_gazebo" params="name">
-  <gazebo reference="${name}_link">
-    <selfCollide>true</selfCollide>
-    <sensor name='${name}_contact_sensor' type='contact'>
-      <contact>
-        <collision>${name}_link_geom</collision>
-      </contact>
-      <plugin name="${name}_gazebo_ros_bumper_controller" filename="libgazebo_ros_bumper.so">
-        <alwaysOn>true</alwaysOn>
-        <updateRate>100.0</updateRate>
-        <frameName>world</frameName>
-        <bumperTopicName>${name}_bumper</bumperTopicName>
-      </plugin>
-    </sensor>
-  </gazebo>
     <gazebo>
     <plugin name="p3d_base_controller" filename="libgazebo_ros_p3d.so">

File: cob_description/urdf/cob4_head/head.transmission.xacro (robot description, xacro)
@@ -4,5 +4,7 @@
     <transmission name="${name}_1_trans">
       <type>transmission_interface/SimpleTransmission</type>
-      <joint name="${name}_1_joint"/>
+      <joint name="${name}_1_joint">
+        <hardwareInterface>EffortJointInterface</hardwareInterface>
+      </joint>
       <actuator name="${name}_1_motor">
         <hardwareInterface>EffortJointInterface</hardwareInterface>
@@ -12,5 +14,7 @@
     <transmission name="${name}_2_trans">
       <type>transmission_interface/SimpleTransmission</type>
-      <joint name="${name}_2_joint"/>
+      <joint name="${name}_2_joint">
+        <hardwareInterface>EffortJointInterface</hardwareInterface>
+      </joint>
       <actuator name="${name}_2_motor">
         <hardwareInterface>EffortJointInterface</hardwareInterface>
@@ -20,5 +24,7 @@
     <transmission name="${name}_3_trans">
       <type>transmission_interface/SimpleTransmission</type>
-      <joint name="${name}_3_joint"/>
+      <joint name="${name}_3_joint">
+        <hardwareInterface>EffortJointInterface</hardwareInterface>
+      </joint>
       <actuator name="${name}_3_motor">
         <hardwareInterface>EffortJointInterface</hardwareInterface>

File: cob_description/urdf/cob4_sensorring/sensorring.transmission.xacro (robot description, xacro)
@@ -4,5 +4,7 @@
     <transmission name="${name}_trans">
       <type>transmission_interface/SimpleTransmission</type>
-      <joint name="${name}_joint"/>
+      <joint name="${name}_joint">
+        <hardwareInterface>EffortJointInterface</hardwareInterface>
+      </joint>
       <actuator name="${name}_motor">
         <hardwareInterface>EffortJointInterface</hardwareInterface>

File: cob_description/urdf/cob4_torso/torso.transmission.xacro (robot description, xacro)
@@ -4,5 +4,7 @@
     <transmission name="${name}_1_trans">
       <type>transmission_interface/SimpleTransmission</type>
-      <joint name="${name}_1_joint"/>
+      <joint name="${name}_1_joint">
+        <hardwareInterface>EffortJointInterface</hardwareInterface>
+      </joint>
       <actuator name="${name}_1_motor">
         <hardwareInterface>EffortJointInterface</hardwareInterface>
@@ -12,5 +14,7 @@
     <transmission name="${name}_2_trans">
       <type>transmission_interface/SimpleTransmission</type>
-      <joint name="${name}_2_joint"/>
+      <joint name="${name}_2_joint">
+        <hardwareInterface>EffortJointInterface</hardwareInterface>
+      </joint>
       <actuator name="${name}_2_motor">
         <hardwareInterface>EffortJointInterface</hardwareInterface>
@@ -20,5 +24,7 @@
     <transmission name="${name}_3_trans">
       <type>transmission_interface/SimpleTransmission</type>
-      <joint name="${name}_3_joint"/>
+      <joint name="${name}_3_joint">
+        <hardwareInterface>EffortJointInterface</hardwareInterface>
+      </joint>
       <actuator name="${name}_3_motor">
         <hardwareInterface>EffortJointInterface</hardwareInterface>

File: cob_description/urdf/lbr/lbr.transmission.xacro (robot description, xacro)
@@ -4,5 +4,7 @@
     <transmission name="${name}_1_trans">
       <type>transmission_interface/SimpleTransmission</type>
-      <joint name="${name}_1_joint"/>
+      <joint name="${name}_1_joint">
+        <hardwareInterface>EffortJointInterface</hardwareInterface>
+      </joint>
       <actuator name="${name}_1_motor">
         <hardwareInterface>EffortJointInterface</hardwareInterface>
@@ -12,5 +14,7 @@
     <transmission name="${name}_2_trans">
       <type>transmission_interface/SimpleTransmission</type>
-      <joint name="${name}_2_joint"/>
+      <joint name="${name}_2_joint">
+        <hardwareInterface>EffortJointInterface</hardwareInterface>
+      </joint>
       <actuator name="${name}_2_motor">
         <hardwareInterface>EffortJointInterface</hardwareInterface>
@@ -20,5 +24,7 @@
     <transmission name="${name}_3_trans">
       <type>transmission_interface/SimpleTransmission</type>
-      <joint name="${name}_3_joint"/>
+      <joint name="${name}_3_joint">
+        <hardwareInterface>EffortJointInterface</hardwareInterface>
+      </joint>
       <actuator name="${name}_3_motor">
         <hardwareInterface>EffortJointInterface</hardwareInterface>
@@ -28,5 +34,7 @@
     <transmission name="${name}_4_trans">
       <type>transmission_interface/SimpleTransmission</type>
-      <joint name="${name}_4_joint"/>
+      <joint name="${name}_4_joint">
+        <hardwareInterface>EffortJointInterface</hardwareInterface>
+      </joint>
       <actuator name="${name}_4_motor">
         <hardwareInterface>EffortJointInterface</hardwareInterface>
@@ -36,5 +44,7 @@
     <transmission name="${name}_5_trans">
       <type>transmission_interface/SimpleTransmission</type>
-      <joint name="${name}_5_joint"/>
+      <joint name="${name}_5_joint">
+        <hardwareInterface>EffortJointInterface</hardwareInterface>
+      </joint>
       <actuator name="${name}_5_motor">
         <hardwareInterface>EffortJointInterface</hardwareInterface>
@@ -44,5 +54,7 @@
     <transmission name="${name}_6_trans">
       <type>transmission_interface/SimpleTransmission</type>
-      <joint name="${name}_6_joint"/>
+      <joint name="${name}_6_joint">
+        <hardwareInterface>EffortJointInterface</hardwareInterface>
+      </joint>
       <actuator name="${name}_6_motor">
         <hardwareInterface>EffortJointInterface</hardwareInterface>
@@ -52,5 +64,7 @@
     <transmission name="${name}_7_trans">
       <type>transmission_interface/SimpleTransmission</type>
-      <joint name="${name}_7_joint"/>
+      <joint name="${name}_7_joint">
+        <hardwareInterface>EffortJointInterface</hardwareInterface>
+      </joint>
       <actuator name="${name}_7_motor">
         <hardwareInterface>EffortJointInterface</hardwareInterface>

File: cob_description/urdf/ur_connector/ur_connector.transmission.xacro (robot description, xacro)
@@ -4,5 +4,7 @@
     <transmission name="${name}_trans">
       <type>transmission_interface/SimpleTransmission</type>
-      <joint name="${name}_joint"/>
+      <joint name="${name}_joint">
+        <hardwareInterface>EffortJointInterface</hardwareInterface>
+      </joint>
       <actuator name="${name}_motor">
         <hardwareInterface>EffortJointInterface</hardwareInterface>

File: desire_description/urdf/base_desire/base.gazebo.xacro (robot description, xacro)
@@ -16,19 +16,4 @@
   </xacro:macro>
   <xacro:macro name="desire_base_gazebo_v0" params="name">
-  <gazebo reference="${name}_link">
-    <selfCollide>true</selfCollide>
-    <sensor name='${name}_contact_sensor' type='contact'>
-      <contact>
-      <collision>${name}_link_geom</collision>
-      </contact>
-      <plugin name="${name}_gazebo_ros_bumper_controller" filename="libgazebo_ros_bumper.so">
-        <alwaysOn>true</alwaysOn>
-        <updateRate>100.0</updateRate>
-        <frameName>world</frameName>
-        <bumperTopicName>${name}_bumper</bumperTopicName>
-      </plugin>
-    </sensor>
-    <material>Gazebo/Grey</material>
-  </gazebo>
     <gazebo>
     <plugin name="p3d_base_controller" filename="libgazebo_ros_p3d.so">

File: desire_description/urdf/base_desire/base.transmission.xacro (robot description, xacro)
@@ -5,5 +5,7 @@
     <transmission name="desire_wheel_transmission_v0">
       <type>transmission_interface/SimpleTransmission</type>
-      <joint name="${parent}_${suffix}_wheel_joint"/>
+      <joint name="${parent}_${suffix}_wheel_joint">
+        <hardwareInterface>EffortJointInterface</hardwareInterface>
+      </joint>
       <actuator name="${parent}_${suffix}_wheel_motor">
         <hardwareInterface>EffortJointInterface</hardwareInterface>
@@ -16,5 +18,7 @@
     <transmission name="desire_caster_transmission_v0">
       <type>transmission_interface/SimpleTransmission</type>
-      <joint name="${suffix}_rotation_joint"/>
+      <joint name="${suffix}_rotation_joint">
+        <hardwareInterface>EffortJointInterface</hardwareInterface>
+      </joint>
       <actuator name="${suffix}_rotation_motor">
         <hardwareInterface>EffortJointInterface</hardwareInterface>

File: desire_description/urdf/head_desire/head.transmission.xacro (robot description, xacro)
@@ -4,5 +4,7 @@
     <transmission name="${name}_pan_trans">
       <type>transmission_interface/SimpleTransmission</type>
-      <joint name="${name}_pan_joint"/>
+      <joint name="${name}_pan_joint">
+        <hardwareInterface>EffortJointInterface</hardwareInterface>
+      </joint>
       <actuator name="${name}_pan_motor">
         <hardwareInterface>EffortJointInterface</hardwareInterface>
@@ -12,5 +14,7 @@
     <transmission name="${name}_tilt_trans">
       <type>transmission_interface/SimpleTransmission</type>
-      <joint name="${name}_tilt_joint"/>
+      <joint name="${name}_tilt_joint">
+        <hardwareInterface>EffortJointInterface</hardwareInterface>
+      </joint>
       <actuator name="${name}_tilt_motor">
         <hardwareInterface>EffortJointInterface</hardwareInterface>

File: raw_description/urdf/base_long/base.gazebo.xacro (robot description, xacro)
@@ -17,20 +17,4 @@
   </xacro:macro>
   <xacro:macro name="cob_base_gazebo" params="name">
-    <gazebo reference="${name}_link">
-      <selfCollide>true</selfCollide>
-      <sensor name='${name}_contact_sensor' type='contact'>
-        <contact>
-          <collision>${name}_link_geom</collision>
-        </contact>
-        <plugin name="${name}_gazebo_ros_bumper_controller" filename="libgazebo_ros_bumper.so">
-          <alwaysOn>true</alwaysOn>
-          <updateRate>100.0</updateRate>
-          <frameName>world</frameName>
-          <bumperTopicName>${name}_bumper</bumperTopicName>
-        </plugin>
-      </sensor>
-      <!--material>Gazebo/Grey</material-->
-      <!--material value="IPA/Metal" /-->
-    </gazebo>
     <gazebo>
       <plugin name="p3d_base_controller" filename="libgazebo_ros_p3d.so">

File: raw_description/urdf/base_long/base.transmission.xacro (robot description, xacro)
@@ -5,5 +5,7 @@
     <transmission name="cob_wheel_transmission">
       <type>transmission_interface/SimpleTransmission</type>
-      <joint name="${parent}_${suffix}_wheel_joint"/>
+      <joint name="${parent}_${suffix}_wheel_joint">
+        <hardwareInterface>EffortJointInterface</hardwareInterface>
+      </joint>
       <actuator name="${parent}_${suffix}_wheel_motor">
         <hardwareInterface>EffortJointInterface</hardwareInterface>
@@ -16,5 +18,7 @@
     <transmission name="cob_caster_transmission">
       <type>transmission_interface/SimpleTransmission</type>
-      <joint name="${suffix}_rotation_joint"/>
+      <joint name="${suffix}_rotation_joint">
+        <hardwareInterface>EffortJointInterface</hardwareInterface>
+      </joint>
       <actuator name="${suffix}_rotation_motor">
         <hardwareInterface>EffortJointInterface</hardwareInterface>

File: raw_description/urdf/base_short/base.gazebo.xacro (robot description, xacro)
@@ -17,19 +17,4 @@
   </xacro:macro>
   <xacro:macro name="cob_base_gazebo" params="name">
-    <gazebo reference="${name}_link">
-      <selfCollide>true</selfCollide>
-      <sensor name='${name}_contact_sensor' type='contact'>
-        <contact>
-          <collision>${name}_link_geom</collision>
-        </contact>
-        <plugin name="${name}_gazebo_ros_bumper_controller" filename="libgazebo_ros_bumper.so">
-          <alwaysOn>true</alwaysOn>
-          <updateRate>100.0</updateRate>
-          <bumperTopicName>${name}_bumper</bumperTopicName>
-        </plugin>
-      </sensor>
-      <!--material>Gazebo/Grey</material-->
-      <!--material value="IPA/Metal" /-->
-    </gazebo>
     <gazebo>
       <plugin name="p3d_base_controller" filename="libgazebo_ros_p3d.so">
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