Commit message: beautify indentation

File: cob_description/urdf/cob3_base/base.gazebo.xacro (robot description, xacro)
@@ -3,5 +3,5 @@
   <xacro:macro name="cob_wheel_gazebo" params="suffix parent">
     <gazebo reference="${parent}_${suffix}_wheel_link">
-          <material value="IPA/LightGrey"/>
+      <material value="IPA/LightGrey"/>
     </gazebo>
   </xacro:macro>
@@ -12,31 +12,31 @@
   </xacro:macro>
   <xacro:macro name="base_gazebo" params="name">
-  <gazebo reference="${name}_link">
-    <selfCollide>true</selfCollide>
-    <sensor name='${name}_contact_sensor' type='contact'>
-      <contact>
-        <collision>${name}_link_geom</collision>
-      </contact>
-      <plugin name="${name}_gazebo_ros_bumper_controller" filename="libgazebo_ros_bumper.so">
+    <gazebo reference="${name}_link">
+      <selfCollide>true</selfCollide>
+      <sensor name='${name}_contact_sensor' type='contact'>
+        <contact>
+          <collision>${name}_link_geom</collision>
+        </contact>
+        <plugin name="${name}_gazebo_ros_bumper_controller" filename="libgazebo_ros_bumper.so">
+          <alwaysOn>true</alwaysOn>
+          <updateRate>100.0</updateRate>
+          <bumperTopicName>${name}_bumper</bumperTopicName>
+          <frameName>world</frameName>
+        </plugin>
+      </sensor>
+      <material>IPA/LightGrey</material>
+    </gazebo>
+    <gazebo>
+      <plugin name="p3d_base_controller" filename="libgazebo_ros_p3d.so">
         <alwaysOn>true</alwaysOn>
         <updateRate>100.0</updateRate>
-        <bumperTopicName>${name}_bumper</bumperTopicName>
-		<frameName>world</frameName>
-		</plugin>
-    </sensor>
-    <material>IPA/LightGrey</material>
-  </gazebo>
-    <gazebo>
-    <plugin name="p3d_base_controller" filename="libgazebo_ros_p3d.so">
-      <alwaysOn>true</alwaysOn>
-      <updateRate>100.0</updateRate>
-      <bodyName>${name}_link</bodyName>
-      <topicName>${name}_pose_ground_truth</topicName>
-      <gaussianNoise>0.01</gaussianNoise>
-      <frameName>map</frameName>
-      <xyzOffsets>25.7 25.7 0</xyzOffsets> <!-- initialize odometry for fake localization-->
-      <rpyOffsets>0 0 0</rpyOffsets>
-    </plugin>
-    <canonicalBody>${name}_footprint</canonicalBody>
+        <bodyName>${name}_link</bodyName>
+        <topicName>${name}_pose_ground_truth</topicName>
+        <gaussianNoise>0.01</gaussianNoise>
+        <frameName>map</frameName>
+        <xyzOffsets>25.7 25.7 0</xyzOffsets> <!-- initialize odometry for fake localization-->
+        <rpyOffsets>0 0 0</rpyOffsets>
+      </plugin>
+      <canonicalBody>${name}_footprint</canonicalBody>
     </gazebo>
   </xacro:macro>

File: cob_description/urdf/cob3_base/base.urdf.xacro (robot description, xacro)
@@ -21,5 +21,5 @@
   <property name="base_cg_z" value="0.293" />
   <property name="base_mass" value="116.0" />
- <property name="caster_mass" value="5.9" />
+  <property name="caster_mass" value="5.9" />
   <!-- simplified box collision geometry for base -->
   <property name="base_size_x" value="0.8" />
@@ -104,5 +104,5 @@
   <xacro:macro name="cob_caster" params="suffix parent *origin ref_position">
     <xacro:cob_caster_hub parent="${parent}" suffix="${suffix}_caster"
-                             ref_position="${ref_position}" >
+                          ref_position="${ref_position}" >
       <insert_block name="origin" />
     </xacro:cob_caster_hub>
@@ -115,5 +115,5 @@
   <!-- The xacro macro xacro:cob_base contains: base, casters and wheels -->
   <xacro:macro name="base" params="name">
-  <link name="${name}_link">
+    <link name="${name}_link">
       <inertial>
         <mass value="${base_mass}" />

File: cob_description/urdf/cob3_head/head_kinect.urdf.xacro (robot description, xacro)
@@ -7,24 +7,24 @@
     <!-- joint between torso_upper_neck_tilt_link and head_base_link -->
     <joint name="${name}_base_joint" type="fixed">
-        <insert_block name="origin" />
-        <parent link="${parent}"/>
-        <child link="${name}_base_link"/>
+      <insert_block name="origin" />
+      <parent link="${parent}"/>
+      <child link="${name}_base_link"/>
     </joint>
     <link name="${name}_base_link">
-        <inertial>
-            <origin xyz="0 0 0" rpy="0 0 0"/>
-            <mass value="0.5"/>
-            <inertia ixx="0.01" ixy="0" ixz="0" iyy="0.01" iyz="0" izz="0.01" />
-        </inertial>
+      <inertial>
+        <origin xyz="0 0 0" rpy="0 0 0"/>
+        <mass value="0.5"/>
+        <inertia ixx="0.01" ixy="0" ixz="0" iyy="0.01" iyz="0" izz="0.01" />
+      </inertial>
     </link>
     <!-- joint between head_base_link and head_axis_link -->
     <joint name="${name}_axis_joint" type="revolute">
-        <parent link="${name}_base_link"/>
-        <origin xyz="0 0 0" rpy="0 0 0" />
-        <child link="${name}_axis_link"/>
-        <axis xyz="0 0 1" />
-        <dynamics damping="0.1" />
-        <calibration rising="${head_axis_ref}"/>
-        <limit effort="100" lower="-3.2" upper="0.1" velocity="1.4"/>
+      <parent link="${name}_base_link"/>
+      <origin xyz="0 0 0" rpy="0 0 0" />
+      <child link="${name}_axis_link"/>
+      <axis xyz="0 0 1" />
+      <dynamics damping="0.1" />
+      <calibration rising="${head_axis_ref}"/>
+      <limit effort="100" lower="-3.2" upper="0.1" velocity="1.4"/>
     </joint>
     <link name="${name}_axis_link">
@@ -50,7 +50,7 @@
     <!--camera reference link-->
     <joint name="${name}_cam_reference_joint" type="fixed">
-        <origin xyz="${cam_reference_x} ${cam_reference_y} ${cam_reference_z}" rpy="${cam_reference_roll} ${cam_reference_pitch} ${cam_reference_yaw}" />
-        <parent link="${name}_axis_link"/>
-        <child link="${name}_cam_reference_link"/>
+      <origin xyz="${cam_reference_x} ${cam_reference_y} ${cam_reference_z}" rpy="${cam_reference_roll} ${cam_reference_pitch} ${cam_reference_yaw}" />
+      <parent link="${name}_axis_link"/>
+      <child link="${name}_cam_reference_link"/>
     </joint>
     <link name="${name}_cam_reference_link">

File: cob_description/urdf/cob3_head/head_prosilicas_kinect.urdf.xacro (robot description, xacro)
@@ -8,69 +8,69 @@
     <!-- joint between torso_upper_neck_tilt_link and head_base_link -->
     <joint name="${name}_base_joint" type="fixed">
-        <insert_block name="origin" />
-        <parent link="${parent}"/>
-        <child link="${name}_base_link"/>
+      <insert_block name="origin" />
+      <parent link="${parent}"/>
+      <child link="${name}_base_link"/>
     </joint>
     <link name="${name}_base_link">
-        <inertial>
-            <origin xyz="0 0 0" rpy="0 0 0"/>
-            <mass value="0.5"/>
-            <inertia ixx="0.01" ixy="0" ixz="0" iyy="0.01" iyz="0" izz="0.01" />
-        </inertial>
+      <inertial>
+        <origin xyz="0 0 0" rpy="0 0 0"/>
+        <mass value="0.5"/>
+        <inertia ixx="0.01" ixy="0" ixz="0" iyy="0.01" iyz="0" izz="0.01" />
+      </inertial>
     </link>
     <!-- joint between torso_upper_neck_tilt_link and head_axis_link -->
     <joint name="${name}_axis_joint" type="revolute">
-        <origin xyz="0 0 0" rpy="0 0 0" />
-        <parent link="${name}_base_link"/>
-        <child link="${name}_axis_link"/>
-        <axis xyz="0 0 1" />
-        <dynamics damping="0.1" />
-        <calibration rising="${head_axis_ref}"/>
-        <limit effort="100" lower="-3.2" upper="0.1" velocity="1.4"/>
+      <origin xyz="0 0 0" rpy="0 0 0" />
+      <parent link="${name}_base_link"/>
+      <child link="${name}_axis_link"/>
+      <axis xyz="0 0 1" />
+      <dynamics damping="0.1" />
+      <calibration rising="${head_axis_ref}"/>
+      <limit effort="100" lower="-3.2" upper="0.1" velocity="1.4"/>
     </joint>
     <link name="${name}_axis_link">
-        <inertial>
-            <origin xyz="0 0 0" rpy="0 0 0"/>
-            <mass value="0.1"/>
-            <inertia ixx="0.0001" ixy="0" ixz="0" iyy="0.0001" iyz="0" izz="0.0001" />
-        </inertial>
-        <visual>
-            <origin xyz="0 0 0" rpy="0 0 0" />
-            <geometry>
-                <box size="0.01 0.01 0.01"/>
-            </geometry>
-            <material name="IPA/LightGrey" />
-        </visual>
-        <collision>
-            <origin xyz="0 0 0" rpy="0 0 0" />
-            <geometry>
-                <box size="0.01 0.01 0.01"/>
-            </geometry>
-        </collision>
+      <inertial>
+        <origin xyz="0 0 0" rpy="0 0 0"/>
+        <mass value="0.1"/>
+        <inertia ixx="0.0001" ixy="0" ixz="0" iyy="0.0001" iyz="0" izz="0.0001" />
+      </inertial>
+      <visual>
+        <origin xyz="0 0 0" rpy="0 0 0" />
+        <geometry>
+          <box size="0.01 0.01 0.01"/>
+        </geometry>
+        <material name="IPA/LightGrey" />
+      </visual>
+      <collision>
+        <origin xyz="0 0 0" rpy="0 0 0" />
+        <geometry>
+          <box size="0.01 0.01 0.01"/>
+        </geometry>
+      </collision>
     </link>
     <!--camera reference link-->
     <joint name="${name}_cam_reference_joint" type="fixed">
-        <origin xyz="${cam_reference_x} ${cam_reference_y} ${cam_reference_z}" rpy="${cam_reference_roll} ${cam_reference_pitch} ${cam_reference_yaw}" />
-        <parent link="${name}_axis_link"/>
-        <child link="${name}_cam_reference_link"/>
+      <origin xyz="${cam_reference_x} ${cam_reference_y} ${cam_reference_z}" rpy="${cam_reference_roll} ${cam_reference_pitch} ${cam_reference_yaw}" />
+      <parent link="${name}_axis_link"/>
+      <child link="${name}_cam_reference_link"/>
     </joint>
     <link name="${name}_cam_reference_link">
-        <inertial>
-            <origin xyz="0 0 0" rpy="0 0 0"/>
-            <mass value="0.5"/>
-            <inertia ixx="0.01" ixy="0" ixz="0" iyy="0.01" iyz="0" izz="0.01" />
-        </inertial>
+      <inertial>
+        <origin xyz="0 0 0" rpy="0 0 0"/>
+        <mass value="0.5"/>
+        <inertia ixx="0.01" ixy="0" ixz="0" iyy="0.01" iyz="0" izz="0.01" />
+      </inertial>
     </link>
     <!-- left camera -->
     <xacro:cob_prosilica_v0 name="${name}_color_camera_l" ros_topic="stereo/left" parent="${name}_cam_reference_link">
-        <origin xyz="${cam_l_x} ${cam_l_y} ${cam_l_z}" rpy="${cam_l_roll} ${cam_l_pitch} ${cam_l_yaw}" />
+      <origin xyz="${cam_l_x} ${cam_l_y} ${cam_l_z}" rpy="${cam_l_roll} ${cam_l_pitch} ${cam_l_yaw}" />
     </xacro:cob_prosilica_v0>
     <!-- right camera -->
     <xacro:cob_prosilica_v0 name="${name}_color_camera_r" ros_topic="stereo/right" parent="${name}_cam_reference_link">
-        <origin xyz="${cam_r_x} ${cam_r_y} ${cam_r_z}" rpy="${cam_r_roll} ${cam_r_pitch} ${cam_r_yaw}" />
+      <origin xyz="${cam_r_x} ${cam_r_y} ${cam_r_z}" rpy="${cam_r_roll} ${cam_r_pitch} ${cam_r_yaw}" />
     </xacro:cob_prosilica_v0>
     <!-- cam3d -->
     <xacro:cob_kinect_v0 name="${name}_cam3d" ros_topic="cam3d" parent="${name}_cam_reference_link">
-        <origin xyz="${cam3d_x} ${cam3d_y} ${cam3d_z}" rpy="${cam3d_roll} ${cam3d_pitch} ${cam3d_yaw}" />
+      <origin xyz="${cam3d_x} ${cam3d_y} ${cam3d_z}" rpy="${cam3d_roll} ${cam3d_pitch} ${cam3d_yaw}" />
     </xacro:cob_kinect_v0>
     <!-- extensions -->

File: cob_description/urdf/cob4_base/base.gazebo.xacro (robot description, xacro)
@@ -16,30 +16,30 @@
   </xacro:macro>
   <xacro:macro name="base_gazebo" params="name">
-  <gazebo reference="${name}_link">
-    <selfCollide>true</selfCollide>
-    <sensor name='${name}_contact_sensor' type='contact'>
-      <contact>
-        <collision>${name}_link_geom</collision>
-      </contact>
-      <plugin name="${name}_gazebo_ros_bumper_controller" filename="libgazebo_ros_bumper.so">
+    <gazebo reference="${name}_link">
+      <selfCollide>true</selfCollide>
+      <sensor name='${name}_contact_sensor' type='contact'>
+        <contact>
+          <collision>${name}_link_geom</collision>
+        </contact>
+        <plugin name="${name}_gazebo_ros_bumper_controller" filename="libgazebo_ros_bumper.so">
+          <alwaysOn>true</alwaysOn>
+          <updateRate>100.0</updateRate>
+          <frameName>world</frameName>
+          <bumperTopicName>${name}_bumper</bumperTopicName>
+        </plugin>
+      </sensor>
+    </gazebo>
+    <gazebo>
+      <plugin name="p3d_base_controller" filename="libgazebo_ros_p3d.so">
         <alwaysOn>true</alwaysOn>
         <updateRate>100.0</updateRate>
-        <frameName>world</frameName>
-        <bumperTopicName>${name}_bumper</bumperTopicName>
+        <bodyName>${name}_link</bodyName>
+        <topicName>${name}_pose_ground_truth</topicName>
+        <gaussianNoise>0.01</gaussianNoise>
+        <frameName>map</frameName>
+        <xyzOffsets>25.7 25.7 0</xyzOffsets> <!-- initialize odometry for fake localization-->
+        <rpyOffsets>0 0 0</rpyOffsets>
       </plugin>
-    </sensor>
-  </gazebo>
-    <gazebo>
-    <plugin name="p3d_base_controller" filename="libgazebo_ros_p3d.so">
-      <alwaysOn>true</alwaysOn>
-      <updateRate>100.0</updateRate>
-      <bodyName>${name}_link</bodyName>
-      <topicName>${name}_pose_ground_truth</topicName>
-      <gaussianNoise>0.01</gaussianNoise>
-      <frameName>map</frameName>
-      <xyzOffsets>25.7 25.7 0</xyzOffsets> <!-- initialize odometry for fake localization-->
-      <rpyOffsets>0 0 0</rpyOffsets>
-    </plugin>
-    <canonicalBody>${name}_footprint</canonicalBody>
+      <canonicalBody>${name}_footprint</canonicalBody>
     </gazebo>
   </xacro:macro>

File: cob_description/urdf/cob4_head/head.urdf.xacro (robot description, xacro)
@@ -4,10 +4,10 @@
   <xacro:include filename="$(find cob_description)/urdf/cob4_head/head.transmission.xacro" />
   <xacro:macro name="head" params="parent name *origin">
-    <joint name="head_base_joint" type="fixed">
+    <joint name="${name}_base_joint" type="fixed">
       <insert_block name="origin" />
-      <child link="head_base_link" />
+      <child link="${name}_base_link" />
       <parent link="${parent}"/>
     </joint>
-    <link name="head_base_link">
+    <link name="${name}_base_link">
       <inertial>
         <origin xyz="0 0 0" rpy="0 0 0"/>
@@ -16,8 +16,8 @@
       </inertial>
     </link>
-    <joint name="head_1_joint" type="revolute">
+    <joint name="${name}_1_joint" type="revolute">
       <origin xyz="0 0 0.0305" rpy="0 0 0"/>
-      <child link="head_1_link" />
-      <parent link="head_base_link"/>
+      <child link="${name}_1_link" />
+      <parent link="${name}_base_link"/>
       <calibration rising="${head_1_ref}"/>
       <axis xyz="0 0 1" />
@@ -25,5 +25,5 @@
       <limit effort="100" lower="-6.2831" upper="6.2831" velocity="1.4"/>
     </joint>
-    <link name="head_1_link">
+    <link name="${name}_1_link">
       <inertial>
         <origin xyz="0 0 0" rpy="0 0 0"/>
@@ -32,8 +32,8 @@
       </inertial>
     </link>
-    <joint name="head_2_joint" type="revolute">
+    <joint name="${name}_2_joint" type="revolute">
       <origin xyz="0 -0.07725 -0.00439" rpy="-0.349 0 0" />
-      <child link="head_2_link" />
-      <parent link="head_1_link"/>
+      <child link="${name}_2_link" />
+      <parent link="${name}_1_link"/>
       <calibration rising="${head_2_ref}"/>
       <axis xyz="0 0 1" />
@@ -41,5 +41,5 @@
       <limit effort="100" lower="-6.2831" upper="6.2831" velocity="1.4"/>
     </joint>
-    <link name="head_2_link">
+    <link name="${name}_2_link">
       <inertial>
         <origin xyz="0 0 0" rpy="0 0 0"/>
@@ -48,8 +48,8 @@
       </inertial>
     </link>
-    <joint name="head_3_joint" type="revolute">
+    <joint name="${name}_3_joint" type="revolute">
       <origin xyz="0 0.04668 0.0976" rpy="0.349 0 0" />
-      <child link="head_3_link" />
-      <parent link="head_2_link"/>
+      <child link="${name}_3_link" />
+      <parent link="${name}_2_link"/>
       <calibration rising="${head_3_ref}"/>
       <axis xyz="0 0 1" />
@@ -57,5 +57,5 @@
       <limit effort="100" lower="-6.2831" upper="6.2831" velocity="1.4"/>
     </joint>
-    <link name="head_3_link">
+    <link name="${name}_3_link">
       <inertial>
         <mass value="1" />
@@ -76,10 +76,10 @@
       </collision>
     </link>
-    <joint name="head_center_joint" type="fixed">
+    <joint name="${name}_center_joint" type="fixed">
       <origin xyz="0.0 0.0 -0.28247" rpy="0 0 0" />
-      <child link="head_center_link" />
-      <parent link="head_3_link"/>
+      <child link="${name}_center_link" />
+      <parent link="${name}_3_link"/>
     </joint>
-    <link name="head_center_link"/>
+    <link name="${name}_center_link"/>
   <!-- extensions -->
   <xacro:head_gazebo name="${name}" />

File: cob_description/urdf/cob4_torso/torso.urdf.xacro (robot description, xacro)
@@ -6,18 +6,18 @@
   <xacro:include filename="$(find cob_description)/urdf/sensors/kinect.urdf.xacro" />
   <xacro:macro name="torso" params="parent name *origin">
-    <joint name="torso_base_joint" type="fixed">
+    <joint name="${name}_base_joint" type="fixed">
       <insert_block name="origin" />
-      <child link="torso_base_link" />
+      <child link="${name}_base_link" />
       <parent link="${parent}"/>
     </joint>
-    <link name="torso_base_link">
+    <link name="${name}_base_link">
        <xacro:cylinder_inertial radius="0.300" length="0.046" mass="5.0">
         <origin xyz="0 0 0" rpy="0 0 0" />
       </xacro:cylinder_inertial>
     </link>
-    <joint name="torso_1_joint" type="revolute">
+    <joint name="${name}_1_joint" type="revolute">
       <origin xyz="0 0 0.04642" rpy="0 0 0"/>
-      <child link="torso_1_link" />
-      <parent link="torso_base_link"/>
+      <child link="${name}_1_link" />
+      <parent link="${name}_base_link"/>
       <calibration rising="${torso_1_ref}"/>
       <axis xyz="0 0 1" />
@@ -25,5 +25,5 @@
       <limit effort="100" lower="-6.2831" upper="6.2831" velocity="1.4"/>
     </joint>
-    <link name="torso_1_link">
+    <link name="${name}_1_link">
       <xacro:hollow_spherical_cap_inertial r="0.295" h="0.075" t="0.010" mass="6">
           <!--origin xyz="0.006 0.010 0.110" rpy="0 0 0"/-->
@@ -31,8 +31,8 @@
       </xacro:hollow_spherical_cap_inertial>
     </link>
-    <joint name="torso_2_joint" type="revolute">
+    <joint name="${name}_2_joint" type="revolute">
       <origin xyz="0 -0.14734 0.07547" rpy="-0.5236 0 0" />
-      <child link="torso_2_link" />
-      <parent link="torso_1_link"/>
+      <child link="${name}_2_link" />
+      <parent link="${name}_1_link"/>
       <calibration rising="${torso_2_ref}"/>
       <axis xyz="0 0 1" />
@@ -40,13 +40,13 @@
       <limit effort="100" lower="-6.2831" upper="6.2831" velocity="1.4"/>
     </joint>
-    <link name="torso_2_link">
+    <link name="${name}_2_link">
         <xacro:spherical_cap_inertial r="0.295" h="0.075" mass="19.5">
             <origin xyz="0.034 0.102 0.092" rpy="0.5236 0 0"/>
         </xacro:spherical_cap_inertial>
     </link>
-    <joint name="torso_3_joint" type="revolute">
+    <joint name="${name}_3_joint" type="revolute">
       <origin xyz="0 0.09228 0.13477" rpy="0.5236 0 0" />
-      <child link="torso_3_link" />
-      <parent link="torso_2_link"/>
+      <child link="${name}_3_link" />
+      <parent link="${name}_2_link"/>
       <calibration rising="${torso_3_ref}"/>
       <axis xyz="0 0 1" />
@@ -54,5 +54,5 @@
       <limit effort="100" lower="-6.2831" upper="6.2831" velocity="1.4"/>
     </joint>
-    <link name="torso_3_link">
+    <link name="${name}_3_link">
        <xacro:cylinder_inertial radius="0.250" length="0.610" mass="23.8">
         <origin xyz="-0.028 0.005 0.233" rpy="0 0 0" />
@@ -72,25 +72,25 @@
       </collision>
     </link>
-    <joint name="torso_center_joint" type="fixed">
+    <joint name="${name}_center_joint" type="fixed">
       <origin xyz="0.0 0.0 0.18566" rpy="0 0 0" />
-      <child link="torso_center_link" />
-      <parent link="torso_3_link"/>
+      <child link="${name}_center_link" />
+      <parent link="${name}_3_link"/>
     </joint>
-    <link name="torso_center_link"/>
+    <link name="${name}_center_link"/>
     <!-- left camera -->
     <xacro:cob_kinect_v0 name="${name}_cam3d_left" ros_topic="torso_cam3d_left" parent="${name}_3_link">
-        <origin xyz="${torso_cam3d_left_x} ${torso_cam3d_left_y} ${torso_cam3d_left_z}" rpy="${torso_cam3d_left_roll} ${torso_cam3d_left_pitch} ${torso_cam3d_left_yaw}" />
+      <origin xyz="${torso_cam3d_left_x} ${torso_cam3d_left_y} ${torso_cam3d_left_z}" rpy="${torso_cam3d_left_roll} ${torso_cam3d_left_pitch} ${torso_cam3d_left_yaw}" />
     </xacro:cob_kinect_v0>
     <!-- right camera -->
     <xacro:cob_kinect_v0 name="${name}_cam3d_right" ros_topic="torso_cam3d_right" parent="${name}_3_link">
-        <origin xyz="${torso_cam3d_right_x} ${torso_cam3d_right_y} ${torso_cam3d_right_z}" rpy="${torso_cam3d_right_roll} ${torso_cam3d_right_pitch} ${torso_cam3d_right_yaw}" />
+      <origin xyz="${torso_cam3d_right_x} ${torso_cam3d_right_y} ${torso_cam3d_right_z}" rpy="${torso_cam3d_right_roll} ${torso_cam3d_right_pitch} ${torso_cam3d_right_yaw}" />
     </xacro:cob_kinect_v0>
     <!-- down camera -->
     <xacro:softkinetic name="${name}_cam3d_down" ros_topic="torso_cam3d_down" parent="${name}_3_link">
-        <origin xyz="${torso_cam3d_down_x} ${torso_cam3d_down_y} ${torso_cam3d_down_z}" rpy="${torso_cam3d_down_roll} ${torso_cam3d_down_pitch} ${torso_cam3d_down_yaw}" />
+      <origin xyz="${torso_cam3d_down_x} ${torso_cam3d_down_y} ${torso_cam3d_down_z}" rpy="${torso_cam3d_down_roll} ${torso_cam3d_down_pitch} ${torso_cam3d_down_yaw}" />
     </xacro:softkinetic>
-	<!-- extensions -->
-	<xacro:torso_gazebo name="torso" />
-	<xacro:torso_transmission name="torso" />
-	</xacro:macro>
+    <!-- extensions -->
+    <xacro:torso_gazebo name="torso" />
+    <xacro:torso_transmission name="torso" />
+  </xacro:macro>
 </robot>

File: cob_description/urdf/ur_arm/ur10_arm.urdf.xacro (robot description, xacro)
@@ -3,6 +3,5 @@
   <xacro:include filename="$(find cob_description)/urdf/common.xacro" />
   <xacro:include filename="$(find ur_description)/urdf/ur10.urdf.xacro" />
-  <!--xacro:include filename="$(find ur_description)/urdf/ur10_joint_limited.urdf.xacro" /-->
-  <property name="wrist_3_length" value="0.0857" />
+  <!--property name="wrist_3_length" value="0.0857" /-->
   <xacro:macro name="ur10" params="parent name *origin">
     <!-- mount the arm to the robot -->

File: cob_description/urdf/ur_arm/ur5_arm.urdf.xacro (robot description, xacro)
@@ -3,6 +3,5 @@
   <xacro:include filename="$(find cob_description)/urdf/common.xacro" />
   <xacro:include filename="$(find ur_description)/urdf/ur5.urdf.xacro" />
-  <!--xacro:include filename="$(find ur_description)/urdf/ur5_joint_limited.urdf.xacro" /-->
-  <property name="wrist_3_length" value="0.0823" />
+  <!--property name="wrist_3_length" value="0.0823" /-->
   <xacro:macro name="ur5" params="parent name *origin">
     <!-- mount the arm to the robot -->
@@ -13,5 +12,5 @@
     </joint>
     <!-- include universal_robot arm -->
-    <xacro:ur5_robot prefix="${name}_"/>
+    <xacro:ur5_robot prefix="${name}_" joint_limited="true"/>
   </xacro:macro>
 </robot>
