Commit message: beautify indentation + cleaning up

File: cob_description/urdf/cob3_base/base.gazebo.xacro (robot description, xacro)
@@ -14,16 +14,17 @@
     <gazebo reference="${name}_link">
       <selfCollide>true</selfCollide>
+      <material>IPA/LightGrey</material>
       <sensor name='${name}_contact_sensor' type='contact'>
+        <always_on>true</always_on>
+        <update_rate>100.0</update_rate>
         <contact>
           <collision>${name}_link_geom</collision>
+          <topic>${name}_bumper</topic>
         </contact>
         <plugin name="${name}_gazebo_ros_bumper_controller" filename="libgazebo_ros_bumper.so">
-          <alwaysOn>true</alwaysOn>
-          <updateRate>100.0</updateRate>
+          <frameName>world</frameName>
           <bumperTopicName>${name}_bumper</bumperTopicName>
-          <frameName>world</frameName>
         </plugin>
       </sensor>
-      <material>IPA/LightGrey</material>
     </gazebo>
     <gazebo>
@@ -33,8 +34,8 @@
         <bodyName>${name}_link</bodyName>
         <topicName>${name}_pose_ground_truth</topicName>
-        <gaussianNoise>0.01</gaussianNoise>
         <frameName>map</frameName>
         <xyzOffsets>25.7 25.7 0</xyzOffsets> <!-- initialize odometry for fake localization-->
         <rpyOffsets>0 0 0</rpyOffsets>
+        <gaussianNoise>0.01</gaussianNoise>
       </plugin>
       <canonicalBody>${name}_footprint</canonicalBody>

File: cob_description/urdf/cob4_base/base.gazebo.xacro (robot description, xacro)
@@ -19,10 +19,11 @@
       <selfCollide>true</selfCollide>
       <sensor name='${name}_contact_sensor' type='contact'>
+        <always_on>true</always_on>
+        <update_rate>100.0</update_rate>
         <contact>
           <collision>${name}_link_geom</collision>
+          <topic>${name}_bumper</topic>
         </contact>
         <plugin name="${name}_gazebo_ros_bumper_controller" filename="libgazebo_ros_bumper.so">
-          <alwaysOn>true</alwaysOn>
-          <updateRate>100.0</updateRate>
           <frameName>world</frameName>
           <bumperTopicName>${name}_bumper</bumperTopicName>
@@ -36,8 +37,8 @@
         <bodyName>${name}_link</bodyName>
         <topicName>${name}_pose_ground_truth</topicName>
-        <gaussianNoise>0.01</gaussianNoise>
         <frameName>map</frameName>
         <xyzOffsets>25.7 25.7 0</xyzOffsets> <!-- initialize odometry for fake localization-->
         <rpyOffsets>0 0 0</rpyOffsets>
+        <gaussianNoise>0.01</gaussianNoise>
       </plugin>
       <canonicalBody>${name}_footprint</canonicalBody>

File: cob_description/urdf/cob4_sensorring/sensorring.urdf.xacro (robot description, xacro)
@@ -4,7 +4,19 @@
   <xacro:include filename="$(find cob_description)/urdf/cob4_sensorring/sensorring.transmission.xacro" />
   <xacro:macro name="sensorring" params="parent name *origin">
-    <joint name="${name}_joint" type="revolute">
+    <joint name="${name}_base_joint" type="fixed">
       <insert_block name="origin" />
       <parent link="${parent}"/>
+      <child link="${name}_base_link" />
+    </joint>
+    <link name="${name}_base_link">
+      <inertial>
+        <origin xyz="0 0 0" rpy="0 0 0"/>
+        <mass value="0.1"/>
+        <inertia ixx="0.01" ixy="0" ixz="0" iyy="0.01" iyz="0" izz="0.01" />
+      </inertial>
+    </link>
+    <joint name="${name}_joint" type="revolute">
+      <origin xyz="0 0 0" rpy="0 0 0" />
+      <parent link="${name}_base_link"/>
       <child link="${name}_link" />
       <calibration rising="${sensorring_ref}"/>

File: cob_description/urdf/cob4_torso/torso.urdf.xacro (robot description, xacro)
@@ -67,5 +67,5 @@
         <origin xyz="0 0 0" rpy="0 0 0" />
         <geometry>
-          <mesh filename="package://cob_description/meshes/cob4_torso/torso_link.stl"/>
+          <mesh filename="package://cob_description/meshes/cob4_torso/torso_link.dae"/>
           <!--box size="0.001 0.001 0.001" /-->
         </geometry>

File: desire_description/urdf/base_desire/base.urdf.xacro (robot description, xacro)
@@ -122,5 +122,5 @@
   <!--xacro:macro name="desire_base_v0" params="name"-->
   <xacro:macro name="desire_base" params="name">
-  <link name="${name}_link">
+    <link name="${name}_link">
       <inertial>
         <mass value="${base_mass}" />
@@ -131,5 +131,4 @@
       <visual>
         <origin xyz="0 0 0" rpy="0 0 0" />
-        <!-- modify here for test-->
         <geometry>
           <mesh filename="package://desire_description/meshes/base_desire/base.stl"/>
@@ -165,5 +164,5 @@
      <!-- cam3d -->
      <xacro:cob_kinect_v0 name="head_cam3d" ros_topic="cam3d" parent="base_link">
-        <origin xyz="0.40 0 1.4246" rpy="0 0 0" />
+      <origin xyz="0.40 0 1.4246" rpy="0 0 0" />
      </xacro:cob_kinect_v0>
     <!-- all four caster macros -->

File: raw_description/urdf/base_long/base.urdf.xacro (robot description, xacro)
@@ -66,5 +66,4 @@
           <mesh filename="package://raw_description/meshes/base/raw_wheel.dae"/>
         </geometry>
-        <!--material name="IPA/LightGrey" /-->
       </visual>
       <collision>
@@ -72,5 +71,5 @@
         <geometry>
           <sphere radius="${wheel_radius}"/>
-    <!--mesh filename="package://raw_description/meshes/base/raw_wheel.stl"/-->
+          <!--mesh filename="package://raw_description/meshes/base/raw_wheel.stl"/-->
         </geometry>
       </collision>
@@ -102,6 +101,6 @@
         <origin xyz="0 0 0" rpy="0 0 0" />
         <geometry>
-        <mesh filename="package://raw_description/meshes/base/raw_caster.stl"/>
-        <!--box size="0.001 0.001 0.001" /-->
+          <mesh filename="package://raw_description/meshes/base/raw_caster.stl"/>
+          <!--box size="0.001 0.001 0.001" /-->
         </geometry>
         <material name="IPA/LightGrey" />
@@ -143,15 +142,15 @@
       </inertial>
       <visual>
-    <origin xyz="0 0 0" rpy="0 0 0"/>
-    <geometry>
-            <mesh filename="package://raw_description/meshes/base/raw_battery.stl"/>
-          </geometry>
+        <origin xyz="0 0 0" rpy="0 0 0"/>
+        <geometry>
+          <mesh filename="package://raw_description/meshes/base/raw_battery.stl"/>
+        </geometry>
         <material name="Gazebo/Black" />
-       </visual>
+      </visual>
       <collision>
         <origin xyz="0 0.075 0" rpy="0 0 0"/> <!-- TODO: Change the origin of the stl, so that collision model doesn't need to be translated  -->
         <geometry>
-        <box size="${battery_size_x} ${battery_size_y} ${battery_size_z}" />
-        <!--mesh filename="package://raw_description/meshes/base/raw_battery.stl"/-->
+          <box size="${battery_size_x} ${battery_size_y} ${battery_size_z}" />
+          <!--mesh filename="package://raw_description/meshes/base/raw_battery.stl"/-->
         </geometry>
        </collision>
@@ -162,5 +161,5 @@
   <!-- The xacro macro xacro:cob_base contains: base, casters and wheels -->
   <xacro:macro name="raw_base" params="name">
-  <link name="${name}_link">
+    <link name="${name}_link">
       <inertial>
         <mass value="${base_mass}" />
@@ -174,5 +173,4 @@
           <mesh filename="package://raw_description/meshes/base/raw_base_long.dae"/>
         </geometry>
-        <!--material name="IPA/LightGrey" /-->
       </visual>
       <collision>

File: raw_description/urdf/base_short/base.gazebo.xacro (robot description, xacro)
@@ -20,15 +20,15 @@
       <selfCollide>true</selfCollide>
       <sensor name='${name}_contact_sensor' type='contact'>
+        <always_on>true</always_on>
+        <update_rate>100.0</update_rate>
         <contact>
           <collision>${name}_link_geom</collision>
+          <topic>${name}_bumper</topic>
         </contact>
         <plugin name="${name}_gazebo_ros_bumper_controller" filename="libgazebo_ros_bumper.so">
-          <alwaysOn>true</alwaysOn>
-          <updateRate>100.0</updateRate>
+          <frameName>world</frameName>
           <bumperTopicName>${name}_bumper</bumperTopicName>
         </plugin>
       </sensor>
-      <!--material>Gazebo/Grey</material-->
-      <!--material value="IPA/Metal" /-->
     </gazebo>
     <gazebo>
@@ -38,8 +38,8 @@
         <bodyName>${name}_link</bodyName>
         <topicName>${name}_pose_ground_truth</topicName>
-        <gaussianNoise>0.01</gaussianNoise>
         <frameName>map</frameName>
         <xyzOffsets>25.7 25.7 0</xyzOffsets>  <!-- initialize odometry for fake localization-->
         <rpyOffsets>0 0 0</rpyOffsets>
+        <gaussianNoise>0.01</gaussianNoise>
       </plugin>
       <canonicalBody>${name}_footprint</canonicalBody>

File: raw_description/urdf/base_short/base.urdf.xacro (robot description, xacro)
@@ -64,5 +64,4 @@
           <mesh filename="package://raw_description/meshes/base/raw_wheel.dae"/>
         </geometry>
-        <!--material name="IPA/LightGrey" /-->
       </visual>
       <collision>
@@ -142,8 +141,8 @@
       </inertial>
       <visual>
-    <origin xyz="0 0 0" rpy="0 0 0"/>
-    <geometry>
-            <mesh filename="package://raw_description/meshes/base/raw_battery.stl"/>
-          </geometry>
+        <origin xyz="0 0 0" rpy="0 0 0"/>
+        <geometry>
+          <mesh filename="package://raw_description/meshes/base/raw_battery.stl"/>
+        </geometry>
         <material name="Gazebo/Black" />
        </visual>
@@ -151,6 +150,6 @@
         <origin xyz="0 0.075 0" rpy="0 0 0"/> <!-- TODO: Change the origin of the stl, so that collision model doesn't need to be translated  -->
         <geometry>
-        <box size="${battery_size_x} ${battery_size_y} ${battery_size_z}" />
-        <!--mesh filename="package://raw_description/meshes/base/raw_battery.stl"/-->
+          <box size="${battery_size_x} ${battery_size_y} ${battery_size_z}" />
+          <!--mesh filename="package://raw_description/meshes/base/raw_battery.stl"/-->
         </geometry>
        </collision>
@@ -173,5 +172,4 @@
           <mesh filename="package://raw_description/meshes/base/raw_base_short.dae"/>
         </geometry>
-        <material name="IPA/LightGrey" />
       </visual>
       <collision>

File: raw_description/urdf/boxgripper/boxgripper.urdf.xacro (robot description, xacro)
@@ -31,8 +31,4 @@
           <mesh filename="package://raw_description/meshes/boxgripper/boxgripper_collision.stl"/>
         </geometry>
-        <!--origin xyz="-0.02 -0.06 0" rpy="0 0 -0.45" />
-        <geometry>
-          <box size="0.05 0.16 0.27"/>
-        </geometry-->
       </collision>
     </link>
