Commit message: Revert "[Indigo] Velocity interface controller indigo"

File: cob_description/urdf/cob3_base/base.gazebo.xacro (robot description, xacro)
@@ -3,6 +3,4 @@
   <xacro:macro name="cob_wheel_gazebo" params="suffix parent">
     <gazebo reference="${parent}_${suffix}_wheel_link">
-      <gravity>true</gravity>
-      <self_collide>false</self_collide>
       <material value="IPA/LightGrey"/>
     </gazebo>
@@ -10,6 +8,4 @@
   <xacro:macro name="cob_caster_gazebo" params="suffix">
     <gazebo reference="${suffix}_caster_rotation_link">
-      <gravity>true</gravity>
-      <self_collide>false</self_collide>
       <material value="IPA/Metal"/>
     </gazebo>
@@ -17,9 +13,6 @@
   <xacro:macro name="base_gazebo" params="name">
     <gazebo reference="${name}_link">
-      <gravity>true</gravity>
-      <self_collide>false</self_collide>
+      <selfCollide>true</selfCollide>
       <material>IPA/LightGrey</material>
-<!-- FXM: the contact sensor currently does not work (the reason is within gazebo, NOT the bumper_plugin) -->
-<!--
       <sensor name='${name}_contact_sensor' type='contact'>
         <always_on>true</always_on>
@@ -34,5 +27,4 @@
         </plugin>
       </sensor>
--->
     </gazebo>
     <gazebo>

File: cob_description/urdf/cob3_base/base.transmission.xacro (robot description, xacro)
@@ -5,8 +5,7 @@
     <transmission name="${parent}_${suffix}_wheel_trans">
       <type>transmission_interface/SimpleTransmission</type>
-      <joint name="${parent}_${suffix}_wheel_joint" >
+      <joint name="${parent}_${suffix}_wheel_joint" />
+      <actuator name="${parent}_${suffix}_wheel_motor">
         <hardwareInterface>EffortJointInterface</hardwareInterface>
-      </joint>
-      <actuator name="${parent}_${suffix}_wheel_motor">
         <mechanicalReduction>${reflect * 624/35 * 80/18}</mechanicalReduction>
       </actuator>
@@ -17,8 +16,7 @@
     <transmission name="${suffix}_rotation_trans">
       <type>transmission_interface/SimpleTransmission</type>
-      <joint name="${suffix}_rotation_joint" >
-        <hardwareInterface>EffortJointInterface</hardwareInterface>
-      </joint>
+      <joint name="${suffix}_rotation_joint" />
       <actuator name="${suffix}_rotation_motor" >
+       <hardwareInterface>EffortJointInterface</hardwareInterface>
         <mechanicalReduction>${-1 * 624/35 * 80/18}</mechanicalReduction>
       </actuator>

File: cob_description/urdf/cob3_head/head.gazebo.xacro (robot description, xacro)
@@ -3,7 +3,6 @@
   <xacro:macro name="head_gazebo" params="name">
     <gazebo reference="${name}_axis_link">
-      <gravity>true</gravity>
-      <self_collide>false</self_collide>
       <material>IPA/LightGrey</material>
+      <turnGravityOff>false</turnGravityOff>
     </gazebo>
   </xacro:macro>

File: cob_description/urdf/cob3_head/head.transmission.xacro (robot description, xacro)
@@ -4,8 +4,7 @@
     <transmission name="${name}_axis_trans">
       <type>transmission_interface/SimpleTransmission</type>
-      <joint name="${name}_axis_joint">
+      <joint name="${name}_axis_joint"/>
+      <actuator name="${name}_axis_motor">
         <hardwareInterface>EffortJointInterface</hardwareInterface>
-      </joint>
-      <actuator name="${name}_axis_motor">
         <mechanicalReduction>1</mechanicalReduction>
       </actuator>

File: cob_description/urdf/cob3_torso/torso_v1.gazebo.xacro (robot description, xacro)
@@ -3,27 +3,22 @@
   <xacro:macro name="torso_gazebo" params="name">
     <gazebo reference="${name}_lower_neck_pan_link">
-      <gravity>true</gravity>
-      <self_collide>false</self_collide>
       <material>IPA/LightGrey</material>
+      <turnGravityOff>false</turnGravityOff>
     </gazebo>
     <gazebo reference="${name}_lower_neck_tilt_link">
-      <gravity>true</gravity>
-      <self_collide>false</self_collide>
       <material>IPA/LightGrey</material>
+      <turnGravityOff>false</turnGravityOff>
     </gazebo>
     <gazebo reference="${name}_upper_neck_pan_link">
-      <gravity>true</gravity>
-      <self_collide>false</self_collide>
       <material>IPA/LightGrey</material>
+      <turnGravityOff>false</turnGravityOff>
     </gazebo>
     <gazebo reference="${name}_upper_neck_tilt_link">
-      <gravity>true</gravity>
-      <self_collide>false</self_collide>
       <material>IPA/LightGrey</material>
+      <turnGravityOff>false</turnGravityOff>
     </gazebo>
     <gazebo reference="head_cover_link">
-      <gravity>true</gravity>
-      <self_collide>false</self_collide>
       <material>IPA/Black</material>
+      <turnGravityOff>false</turnGravityOff>
     </gazebo>
   </xacro:macro>

File: cob_description/urdf/cob3_torso/torso_v1.transmission.xacro (robot description, xacro)
@@ -4,8 +4,7 @@
     <transmission name="${name}_lower_neck_pan_trans">
       <type>transmission_interface/SimpleTransmission</type>
-      <joint name="${name}_lower_neck_pan_joint">
+      <joint name="${name}_lower_neck_pan_joint"/>
+      <actuator name="${name}_lower_neck_pan_motor">
         <hardwareInterface>EffortJointInterface</hardwareInterface>
-      </joint>
-      <actuator name="${name}_lower_neck_pan_motor">
         <mechanicalReduction>1</mechanicalReduction>
       </actuator>
@@ -13,8 +12,7 @@
     <transmission name="${name}_lower_neck_tilt_trans">
       <type>transmission_interface/SimpleTransmission</type>
-      <joint name="${name}_lower_neck_tilt_joint">
+      <joint name="${name}_lower_neck_tilt_joint"/>
+      <actuator name="${name}_lower_neck_tilt_motor">
         <hardwareInterface>EffortJointInterface</hardwareInterface>
-      </joint>
-      <actuator name="${name}_lower_neck_tilt_motor">
         <mechanicalReduction>1</mechanicalReduction>
       </actuator>
@@ -22,8 +20,7 @@
     <transmission name="${name}_upper_neck_pan_trans">
       <type>transmission_interface/SimpleTransmission</type>
-      <joint name="${name}_upper_neck_pan_joint">
+      <joint name="${name}_upper_neck_pan_joint"/>
+      <actuator name="${name}_upper_neck_pan_motor">
         <hardwareInterface>EffortJointInterface</hardwareInterface>
-      </joint>
-      <actuator name="${name}_upper_neck_pan_motor">
         <mechanicalReduction>1</mechanicalReduction>
       </actuator>
@@ -31,8 +28,7 @@
     <transmission name="${name}_upper_neck_tilt_trans">
       <type>transmission_interface/SimpleTransmission</type>
-      <joint name="${name}_upper_neck_tilt_joint">
+      <joint name="${name}_upper_neck_tilt_joint"/>
+      <actuator name="${name}_upper_neck_tilt_motor">
         <hardwareInterface>EffortJointInterface</hardwareInterface>
-      </joint>
-      <actuator name="${name}_upper_neck_tilt_motor">
         <mechanicalReduction>1</mechanicalReduction>
       </actuator>

File: cob_description/urdf/cob3_torso/torso_v2.gazebo.xacro (robot description, xacro)
@@ -3,22 +3,18 @@
   <xacro:macro name="torso_gazebo" params="name">
     <gazebo reference="${name}_lower_neck_tilt_link">
-      <gravity>true</gravity>
-      <self_collide>false</self_collide>
       <material>IPA/LightGrey</material>
+      <turnGravityOff>false</turnGravityOff>
     </gazebo>
     <gazebo reference="${name}_pan_link">
-      <gravity>true</gravity>
-      <self_collide>false</self_collide>
       <material>IPA/LightGrey</material>
+      <turnGravityOff>false</turnGravityOff>
     </gazebo>
     <gazebo reference="${name}_upper_neck_tilt_link">
-      <gravity>true</gravity>
-      <self_collide>false</self_collide>
       <material>IPA/LightGrey</material>
+      <turnGravityOff>false</turnGravityOff>
     </gazebo>
     <gazebo reference="head_cover_link">
-      <gravity>true</gravity>
-      <self_collide>false</self_collide>
       <material>IPA/Black</material>
+      <turnGravityOff>false</turnGravityOff>
     </gazebo>
   </xacro:macro>

File: cob_description/urdf/cob3_torso/torso_v2.transmission.xacro (robot description, xacro)
@@ -4,8 +4,7 @@
     <transmission name="${name}_lower_neck_tilt_trans">
       <type>transmission_interface/SimpleTransmission</type>
-      <joint name="${name}_lower_neck_tilt_joint">
+      <joint name="${name}_lower_neck_tilt_joint"/>
+      <actuator name="${name}_lower_neck_tilt_motor">
         <hardwareInterface>EffortJointInterface</hardwareInterface>
-      </joint>
-      <actuator name="${name}_lower_neck_tilt_motor">
         <mechanicalReduction>1</mechanicalReduction>
       </actuator>
@@ -13,8 +12,7 @@
     <transmission name="${name}_pan_trans">
       <type>transmission_interface/SimpleTransmission</type>
-      <joint name="${name}_pan_joint">
+      <joint name="${name}_pan_joint"/>
+      <actuator name="${name}_pan_motor">
         <hardwareInterface>EffortJointInterface</hardwareInterface>
-      </joint>
-      <actuator name="${name}_pan_motor">
         <mechanicalReduction>1</mechanicalReduction>
       </actuator>
@@ -22,8 +20,7 @@
     <transmission name="${name}_upper_neck_tilt_trans">
       <type>transmission_interface/SimpleTransmission</type>
-      <joint name="${name}_upper_neck_tilt_joint">
+      <joint name="${name}_upper_neck_tilt_joint"/>
+      <actuator name="${name}_upper_neck_tilt_motor">
         <hardwareInterface>EffortJointInterface</hardwareInterface>
-      </joint>
-      <actuator name="${name}_upper_neck_tilt_motor">
         <mechanicalReduction>1</mechanicalReduction>
       </actuator>

File: cob_description/urdf/cob3_tray/tray.gazebo.xacro (robot description, xacro)
@@ -3,7 +3,6 @@
   <xacro:macro name="tray_gazebo" params="name">
     <gazebo reference="${name}_link">
-      <gravity>true</gravity>
-      <self_collide>false</self_collide>
       <material>IPA/DarkGrey</material>
+      <turnGravityOff>false</turnGravityOff>
     </gazebo>
   </xacro:macro>

File: cob_description/urdf/cob3_tray/tray.transmission.xacro (robot description, xacro)
@@ -4,8 +4,7 @@
     <transmission name="${name}_trans">
       <type>transmission_interface/SimpleTransmission</type>
-      <joint name="${name}_joint">
+      <joint name="${name}_joint"/>
+      <actuator name="${name}_motor">
         <hardwareInterface>EffortJointInterface</hardwareInterface>
-      </joint>
-      <actuator name="${name}_motor">
         <mechanicalReduction>1</mechanicalReduction>
       </actuator>

File: cob_description/urdf/cob3_tray/tray_3DOF.gazebo.xacro (robot description, xacro)
@@ -3,17 +3,14 @@
   <xacro:macro name="tray_gazebo" params="name">
     <gazebo reference="${name}_1_link">
-      <gravity>true</gravity>
-      <self_collide>false</self_collide>
       <material>IPA/DarkGrey</material>
+      <turnGravityOff>false</turnGravityOff>
     </gazebo>
     <gazebo reference="${name}_2_link">
-      <gravity>true</gravity>
-      <self_collide>false</self_collide>
       <material>IPA/DarkGrey</material>
+      <turnGravityOff>false</turnGravityOff>
     </gazebo>
     <gazebo reference="${name}_3_link">
-      <gravity>true</gravity>
-      <self_collide>false</self_collide>
       <material>IPA/DarkGrey</material>
+      <turnGravityOff>false</turnGravityOff>
     </gazebo>
   </xacro:macro>

File: cob_description/urdf/cob3_tray/tray_3DOF.transmission.xacro (robot description, xacro)
@@ -4,8 +4,7 @@
     <transmission name="${name}_1_trans">
       <type>transmission_interface/SimpleTransmission</type>
-      <joint name="${name}_1_joint">
+      <joint name="${name}_1_joint"/>
+      <actuator name="${name}_1_motor">
         <hardwareInterface>EffortJointInterface</hardwareInterface>
-      </joint>
-      <actuator name="${name}_1_motor">
         <mechanicalReduction>1</mechanicalReduction>
       </actuator>
@@ -13,8 +12,7 @@
     <transmission name="${name}_2_trans">
       <type>transmission_interface/SimpleTransmission</type>
-      <joint name="${name}_2_joint">
+      <joint name="${name}_2_joint"/>
+      <actuator name="${name}_2_motor">
         <hardwareInterface>EffortJointInterface</hardwareInterface>
-      </joint>
-      <actuator name="${name}_2_motor">
         <mechanicalReduction>1</mechanicalReduction>
       </actuator>
@@ -22,8 +20,7 @@
     <transmission name="${name}_3_trans">
       <type>transmission_interface/SimpleTransmission</type>
-      <joint name="${name}_3_joint">
+      <joint name="${name}_3_joint"/>
+      <actuator name="${name}_3_motor">
         <hardwareInterface>EffortJointInterface</hardwareInterface>
-      </joint>
-      <actuator name="${name}_3_motor">
         <mechanicalReduction>1</mechanicalReduction>
       </actuator>

File: cob_description/urdf/cob4_base/base.gazebo.xacro (robot description, xacro)
@@ -12,6 +12,4 @@
   <xacro:macro name="cob_caster_gazebo" params="suffix">
     <gazebo reference="${suffix}_caster_rotation_link">
-      <gravity>true</gravity>
-      <self_collide>false</self_collide>
       <material value="IPA/Metal" />
     </gazebo>
@@ -19,8 +17,5 @@
   <xacro:macro name="base_gazebo" params="name">
     <gazebo reference="${name}_link">
-      <gravity>true</gravity>
-      <self_collide>false</self_collide>
-<!-- FXM: the contact sensor currently does not work (the reason is within gazebo, NOT the bumper_plugin) -->
-<!--
+      <selfCollide>true</selfCollide>
       <sensor name='${name}_contact_sensor' type='contact'>
         <always_on>true</always_on>
@@ -35,5 +30,4 @@
         </plugin>
       </sensor>
--->
     </gazebo>
     <gazebo>

File: cob_description/urdf/cob4_base/base.transmission.xacro (robot description, xacro)
@@ -5,8 +5,7 @@
     <transmission name="${parent}_${suffix}_wheel_trans">
       <type>transmission_interface/SimpleTransmission</type>
-      <joint name="${parent}_${suffix}_wheel_joint" >
+      <joint name="${parent}_${suffix}_wheel_joint" />
+      <actuator name="${parent}_${suffix}_wheel_motor">
         <hardwareInterface>EffortJointInterface</hardwareInterface>
-      </joint>
-      <actuator name="${parent}_${suffix}_wheel_motor">
         <mechanicalReduction>${reflect * 624/35 * 80/18}</mechanicalReduction>
       </actuator>
@@ -17,8 +16,7 @@
     <transmission name="${suffix}_rotation_trans">
       <type>transmission_interface/SimpleTransmission</type>
-      <joint name="${suffix}_rotation_joint" >
-        <hardwareInterface>EffortJointInterface</hardwareInterface>
-      </joint>
+      <joint name="${suffix}_rotation_joint" />
       <actuator name="${suffix}_rotation_motor" >
+       <hardwareInterface>EffortJointInterface</hardwareInterface>
         <mechanicalReduction>${-1 * 624/35 * 80/18}</mechanicalReduction>
       </actuator>

File: cob_description/urdf/cob4_head/head.gazebo.xacro (robot description, xacro)
@@ -3,18 +3,14 @@
   <xacro:macro name="head_gazebo" params="name">
     <gazebo reference="${name}_base_link">
-      <gravity>true</gravity>
-      <self_collide>false</self_collide>
+      <turnGravityOff>false</turnGravityOff>
     </gazebo>
     <gazebo reference="${name}_1_link">
-      <gravity>true</gravity>
-      <self_collide>false</self_collide>
+      <turnGravityOff>false</turnGravityOff>
     </gazebo>
     <gazebo reference="${name}_2_link">
-      <gravity>true</gravity>
-      <self_collide>false</self_collide>
+      <turnGravityOff>false</turnGravityOff>
     </gazebo>
     <gazebo reference="${name}_3_link">
-      <gravity>true</gravity>
-      <self_collide>false</self_collide>
+      <turnGravityOff>false</turnGravityOff>
     </gazebo>
   </xacro:macro>

File: cob_description/urdf/cob4_head/head.transmission.xacro (robot description, xacro)
@@ -4,8 +4,7 @@
     <transmission name="${name}_1_trans">
       <type>transmission_interface/SimpleTransmission</type>
-      <joint name="${name}_1_joint">
+      <joint name="${name}_1_joint"/>
+      <actuator name="${name}_1_motor">
         <hardwareInterface>EffortJointInterface</hardwareInterface>
-      </joint>
-      <actuator name="${name}_1_motor">
         <mechanicalReduction>1</mechanicalReduction>
       </actuator>
@@ -13,8 +12,7 @@
     <transmission name="${name}_2_trans">
       <type>transmission_interface/SimpleTransmission</type>
-      <joint name="${name}_2_joint">
+      <joint name="${name}_2_joint"/>
+      <actuator name="${name}_2_motor">
         <hardwareInterface>EffortJointInterface</hardwareInterface>
-      </joint>
-      <actuator name="${name}_2_motor">
         <mechanicalReduction>1</mechanicalReduction>
       </actuator>
@@ -22,8 +20,7 @@
     <transmission name="${name}_3_trans">
       <type>transmission_interface/SimpleTransmission</type>
-      <joint name="${name}_3_joint">
+      <joint name="${name}_3_joint"/>
+      <actuator name="${name}_3_motor">
         <hardwareInterface>EffortJointInterface</hardwareInterface>
-      </joint>
-      <actuator name="${name}_3_motor">
         <mechanicalReduction>1</mechanicalReduction>
       </actuator>

File: cob_description/urdf/cob4_sensorring/sensorring.gazebo.xacro (robot description, xacro)
@@ -3,7 +3,6 @@
   <xacro:macro name="sensorring_gazebo" params="name">
     <gazebo reference="${name}_link">
-      <gravity>true</gravity>
-      <self_collide>false</self_collide>
       <material>IPA/DarkGrey</material>
+      <turnGravityOff>false</turnGravityOff>
     </gazebo>
   </xacro:macro>

File: cob_description/urdf/cob4_sensorring/sensorring.transmission.xacro (robot description, xacro)
@@ -4,8 +4,7 @@
     <transmission name="${name}_trans">
       <type>transmission_interface/SimpleTransmission</type>
-      <joint name="${name}_joint">
+      <joint name="${name}_joint"/>
+      <actuator name="${name}_motor">
         <hardwareInterface>EffortJointInterface</hardwareInterface>
-      </joint>
-      <actuator name="${name}_motor">
         <mechanicalReduction>1</mechanicalReduction>
       </actuator>

File: cob_description/urdf/cob4_torso/torso.gazebo.xacro (robot description, xacro)
@@ -3,18 +3,14 @@
   <xacro:macro name="torso_gazebo" params="name">
     <gazebo reference="${name}_base_link">
-      <gravity>true</gravity>
-      <self_collide>false</self_collide>
+      <selfCollide>true</selfCollide>
     </gazebo>
     <gazebo reference="${name}_1_link">
-      <gravity>true</gravity>
-      <self_collide>false</self_collide>
+      <selfCollide>true</selfCollide>
     </gazebo>
     <gazebo reference="${name}_2_link">
-      <gravity>true</gravity>
-      <self_collide>false</self_collide>
+      <selfCollide>true</selfCollide>
     </gazebo>
     <gazebo reference="${name}_3_link">
-      <gravity>true</gravity>
-      <self_collide>false</self_collide>
+      <selfCollide>true</selfCollide>
     </gazebo>
   </xacro:macro>

File: cob_description/urdf/cob4_torso/torso.transmission.xacro (robot description, xacro)
@@ -4,8 +4,7 @@
     <transmission name="${name}_1_trans">
       <type>transmission_interface/SimpleTransmission</type>
-      <joint name="${name}_1_joint">
-        <hardwareInterface>VelocityJointInterface</hardwareInterface>
-      </joint>
+      <joint name="${name}_1_joint"/>
       <actuator name="${name}_1_motor">
+        <hardwareInterface>EffortJointInterface</hardwareInterface>
         <mechanicalReduction>1</mechanicalReduction>
       </actuator>
@@ -13,8 +12,7 @@
     <transmission name="${name}_2_trans">
       <type>transmission_interface/SimpleTransmission</type>
-      <joint name="${name}_2_joint">
-        <hardwareInterface>VelocityJointInterface</hardwareInterface>
-      </joint>
+      <joint name="${name}_2_joint"/>
       <actuator name="${name}_2_motor">
+        <hardwareInterface>EffortJointInterface</hardwareInterface>
         <mechanicalReduction>1</mechanicalReduction>
       </actuator>
@@ -22,8 +20,7 @@
     <transmission name="${name}_3_trans">
       <type>transmission_interface/SimpleTransmission</type>
-      <joint name="${name}_3_joint">
-        <hardwareInterface>VelocityJointInterface</hardwareInterface>
-      </joint>
+      <joint name="${name}_3_joint"/>
       <actuator name="${name}_3_motor">
+        <hardwareInterface>EffortJointInterface</hardwareInterface>
         <mechanicalReduction>1</mechanicalReduction>
       </actuator>
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