Commit message: fix bumper plugins

File: cob_description/urdf/cob3_base/base.gazebo.xacro (robot description, xacro)
@@ -20,11 +20,9 @@
       <self_collide>false</self_collide>
       <material>IPA/LightGrey</material>
-<!-- FXM: the contact sensor currently does not work (the reason is within gazebo, NOT the bumper_plugin) -->
-<!--
       <sensor name='${name}_contact_sensor' type='contact'>
         <always_on>true</always_on>
         <update_rate>100.0</update_rate>
         <contact>
-          <collision>${name}_link_geom</collision>
+          <collision>${name}_link_collision</collision>
           <topic>${name}_bumper</topic>
         </contact>
@@ -34,5 +32,4 @@
         </plugin>
       </sensor>
--->
     </gazebo>
     <gazebo>

File: cob_description/urdf/cob4_base/base.gazebo.xacro (robot description, xacro)
@@ -21,11 +21,9 @@
       <gravity>true</gravity>
       <self_collide>false</self_collide>
-<!-- FXM: the contact sensor currently does not work (the reason is within gazebo, NOT the bumper_plugin) -->
-<!--
       <sensor name='${name}_contact_sensor' type='contact'>
         <always_on>true</always_on>
         <update_rate>100.0</update_rate>
         <contact>
-          <collision>${name}_link_geom</collision>
+          <collision>${name}_link_collision</collision>
           <topic>${name}_bumper</topic>
         </contact>
@@ -35,5 +33,4 @@
         </plugin>
       </sensor>
--->
     </gazebo>
     <gazebo>

File: desire_description/urdf/base_desire/base.gazebo.xacro (robot description, xacro)
@@ -18,11 +18,9 @@
     <gazebo reference="${name}_link">
       <material>Gazebo/Grey</material>
-<!-- FXM: the contact sensor currently does not work (the reason is within gazebo, NOT the bumper_plugin) -->
-<!--
       <sensor name='${name}_contact_sensor' type='contact'>
         <always_on>true</always_on>
         <update_rate>100.0</update_rate>
         <contact>
-          <collision>${name}_link_geom</collision>
+          <collision>${name}_link_collision</collision>
           <topic>${name}_bumper</topic>
         </contact>
@@ -32,5 +30,4 @@
         </plugin>
       </sensor>
--->
     </gazebo>
     <gazebo>

File: raw_description/urdf/base_long/base.gazebo.xacro (robot description, xacro)
@@ -22,11 +22,9 @@
       <gravity>true</gravity>
       <self_collide>false</self_collide>
-<!-- FXM: the contact sensor currently does not work (the reason is within gazebo, NOT the bumper_plugin) -->
-<!--
       <sensor name='${name}_contact_sensor' type='contact'>
         <always_on>true</always_on>
         <update_rate>100.0</update_rate>
         <contact>
-          <collision>${name}_link_geom</collision>
+          <collision>${name}_link_collision</collision>
           <topic>${name}_bumper</topic>
         </contact>
@@ -36,5 +34,4 @@
         </plugin>
       </sensor>
--->
     </gazebo>
     <gazebo>

File: raw_description/urdf/base_short/base.gazebo.xacro (robot description, xacro)
@@ -22,11 +22,9 @@
       <gravity>true</gravity>
       <self_collide>false</self_collide>
-<!-- FXM: the contact sensor currently does not work (the reason is within gazebo, NOT the bumper_plugin) -->
-<!--
       <sensor name='${name}_contact_sensor' type='contact'>
-        <always_on>true</always_on>
+        <always_on>1</always_on>
         <update_rate>100.0</update_rate>
         <contact>
-          <collision>${name}_link_geom</collision>
+          <collision>${name}_link_collision</collision>
           <topic>${name}_bumper</topic>
         </contact>
@@ -36,5 +34,4 @@
         </plugin>
       </sensor>
--->
     </gazebo>
     <gazebo>
