Commit message: some missed changes

File: cob_description/urdf/cob3_base/base.urdf.xacro (robot description, xacro)
@@ -87,6 +87,6 @@
         <origin xyz="0 0 0" rpy="0 0 0" />
         <geometry>
-    <mesh filename="package://raw_description/meshes/base/raw_caster.stl"/>
-      <!--box size="0.001 0.001 0.001" /-->
+          <mesh filename="package://raw_description/meshes/cob3_base/raw_caster.stl"/>
+          <!--box size="0.001 0.001 0.001" /-->
         </geometry>
         <material name="IPA/LightGrey" />
@@ -125,5 +125,5 @@
         <origin xyz="0 0 0" rpy="0 0 0" />
         <geometry>
-          <mesh filename="package://cob_description/meshes/base/base.stl"/>
+          <mesh filename="package://cob_description/meshes/cob3_base/base.stl"/>
           <!--box size="${base_size_x} ${base_size_y} ${base_collision_size_z}" /-->
         </geometry>
@@ -133,5 +133,5 @@
         <origin xyz="0 0 0" rpy="0 0 0" />
         <geometry>
-        <mesh filename="package://cob_description/meshes/base/base_collision.stl"/>
+        <mesh filename="package://cob_description/meshes/cob3_base/base_collision.stl"/>
           <!--box size="${base_size_x} ${base_size_y} ${base_collision_size_z}" /-->
         </geometry>

File: cob_description/urdf/cob3_torso/torso_v1.urdf.xacro (robot description, xacro)
@@ -126,5 +126,5 @@
         <origin xyz="0 0 0" rpy="0 0 0" />
         <geometry>
-          <mesh filename="package://cob_description/meshes/torso/upper_neck.stl" />
+          <mesh filename="package://cob_description/meshes/cob3_torso/upper_neck.stl" />
         </geometry>
         <material name="IPA/LightGrey" />

File: cob_description/urdf/cob3_torso/torso_v2.urdf.xacro (robot description, xacro)
@@ -93,5 +93,5 @@
         <origin xyz="0 0 0" rpy="${M_PI} 0 0" />
         <geometry>
-          <!--mesh filename="package://cob_description/meshes/torso/upper_neck_collision.stl" /-->
+          <!--mesh filename="package://cob_description/meshes/cob3_torso/upper_neck_collision.stl" /-->
           <mesh filename="package://cob_description/meshes/cob3_torso/upper_neck.stl" />
         </geometry>

File: cob_description/urdf/cob4_base/base.urdf.xacro (robot description, xacro)
@@ -155,5 +155,5 @@
 				<origin xyz="0 0 0" rpy="0 0 0" />
 				<geometry>
-					<mesh filename="package://raw_description/meshes/base/raw_caster.stl"/>
+					<mesh filename="package://raw_description/meshes/cob4_base/raw_caster.stl"/>
 				</geometry>
 				<material name="IPA/LightGrey" />

Commit message: Coloured mesh files

File: cob_description/urdf/cob3_base/base.urdf.xacro (robot description, xacro)
@@ -166,8 +166,8 @@
       <origin xyz="${caster_offset_x} ${-caster_offset_y} ${caster_offset_z}" rpy="0 0 0" />
     </xacro:cob_caster>
-    <xacro:cob_caster suffix="bl" parent="${name}_link" ref_position="${cal_caster_bl - M_PI / 4 + M_PI}" >
+    <xacro:cob_caster suffix="bl" parent="${name}_link" ref_position="${cal_caster_bl - M_PI/4 + M_PI}" >
       <origin xyz="${-caster_offset_x} ${caster_offset_y} ${caster_offset_z}" rpy="0 0 0" />
     </xacro:cob_caster>
-    <xacro:cob_caster suffix="br" parent="${name}_link" ref_position="${cal_caster_br - M_PI / 4 + M_PI}"  >
+    <xacro:cob_caster suffix="br" parent="${name}_link" ref_position="${cal_caster_br - M_PI/4 + M_PI}"  >
       <origin xyz="${-caster_offset_x} ${-caster_offset_y} ${caster_offset_z}" rpy="0 0 0" />
     </xacro:cob_caster>

File: cob_description/urdf/cob4_head/head.urdf.xacro (robot description, xacro)
@@ -66,7 +66,6 @@
       <origin xyz="0 0 0" rpy="0 0 0" />
       <geometry>
-        <mesh filename="package://cob_description/meshes/cob4_head/head_link.stl"/>
+        <mesh filename="package://cob_description/meshes/cob4_head/head_link.dae"/>
       </geometry>
-      <material name="IPA/LightGrey"/>
       </visual>
       <collision>

File: cob_description/urdf/cob4_torso/torso.gazebo.xacro (robot description, xacro)
@@ -3,17 +3,13 @@
   <xacro:macro name="torso_gazebo" params="name">
     <gazebo reference="${name}_base_link">
-            <material>IPA/LightGrey</material>
       <turnGravityOff>false</turnGravityOff>
     </gazebo>
     <gazebo reference="${name}_1_link">
-      <material>IPA/LightGrey</material>
       <turnGravityOff>false</turnGravityOff>
     </gazebo>
     <gazebo reference="${name}_2_link">
-      <material>IPA/LightGrey</material>
       <turnGravityOff>false</turnGravityOff>
     </gazebo>
     <gazebo reference="${name}_3_link">
-      <material>IPA/LightGrey</material>
       <turnGravityOff>false</turnGravityOff>
     </gazebo>

File: cob_description/urdf/cob4_torso/torso.urdf.xacro (robot description, xacro)
@@ -68,7 +68,6 @@
         <origin xyz="0 0 0" rpy="0 0 0" />
         <geometry>
-          <mesh filename="package://cob_description/meshes/cob4_torso/torso_link.stl"/>
+          <mesh filename="package://cob_description/meshes/cob4_torso/torso_link.dae"/>
         </geometry>
-        <material name="IPA/LightGrey"/>
       </visual>
       <collision>

Commit message: remove unsupported calibration_rising

File: cob_description/urdf/cob3_base/base.urdf.xacro (robot description, xacro)
@@ -11,8 +11,4 @@
   <property name="caster_offset_y" value="0.185" />
   <property name="caster_offset_z" value="0.075" />
-  <property name="cal_caster_fl" value="0.0" />
-  <property name="cal_caster_fr" value="0.0" />
-  <property name="cal_caster_bl" value="0.0" />
-  <property name="cal_caster_br" value="0.0" />
   <property name="base_mass" value="116.0" />
   <xacro:macro name="base" params="name">
@@ -45,14 +41,14 @@
     </link>
     <!-- arrangement of the four drive_wheel modules -->
-    <xacro:drive_wheel parent="${name}_link" suffix="fl" ref_position="${cal_caster_fl - M_PI/4}" >
+    <xacro:drive_wheel parent="${name}_link" suffix="fl" >
       <origin xyz="${caster_offset_x} ${caster_offset_y} ${caster_offset_z}" rpy="0 0 0" />
     </xacro:drive_wheel>
-    <xacro:drive_wheel parent="${name}_link" suffix="fr" ref_position="${cal_caster_fr - M_PI/4}" >
+    <xacro:drive_wheel parent="${name}_link" suffix="fr" >
       <origin xyz="${caster_offset_x} ${-caster_offset_y} ${caster_offset_z}" rpy="0 0 0" />
     </xacro:drive_wheel>
-    <xacro:drive_wheel parent="${name}_link" suffix="bl" ref_position="${cal_caster_bl - M_PI/4 + M_PI}" >
+    <xacro:drive_wheel parent="${name}_link" suffix="bl" >
       <origin xyz="${-caster_offset_x} ${caster_offset_y} ${caster_offset_z}" rpy="0 0 0" />
     </xacro:drive_wheel>
-    <xacro:drive_wheel parent="${name}_link" suffix="br" ref_position="${cal_caster_br - M_PI/4 + M_PI}"  >
+    <xacro:drive_wheel parent="${name}_link" suffix="br"  >
       <origin xyz="${-caster_offset_x} ${-caster_offset_y} ${caster_offset_z}" rpy="0 0 0" />
     </xacro:drive_wheel>

File: cob_description/urdf/cob4_base/base.urdf.xacro (robot description, xacro)
@@ -42,22 +42,22 @@
     <!-- arrangement of the three drive_wheel modules -->
     <xacro:if value="${use_old_joint_names}">
-      <xacro:drive_wheel parent="${name}_link" suffix="fl" ref_position="0" >
+      <xacro:drive_wheel parent="${name}_link" suffix="fl" >
         <origin xyz="${caster_offset_x/2} ${caster_offset_y} ${caster_offset_z}" rpy="0 0 0" />
       </xacro:drive_wheel>
-      <xacro:drive_wheel parent="${name}_link" suffix="bl" ref_position="0" >
+      <xacro:drive_wheel parent="${name}_link" suffix="bl" >
         <origin xyz="${-caster_offset_x} 0.0 ${caster_offset_z}" rpy="0 0 0" />
       </xacro:drive_wheel>
-      <xacro:drive_wheel parent="${name}_link" suffix="br" ref_position="0" >
+      <xacro:drive_wheel parent="${name}_link" suffix="br" >
         <origin xyz="${caster_offset_x/2} ${-caster_offset_y} ${caster_offset_z}" rpy="0 0 0" />
       </xacro:drive_wheel>
     </xacro:if>
     <xacro:unless value="${use_old_joint_names}">
-      <xacro:drive_wheel parent="${name}_link" suffix="fl" ref_position="0" >
+      <xacro:drive_wheel parent="${name}_link" suffix="fl" >
         <origin xyz="${caster_offset_x/2} ${caster_offset_y} ${caster_offset_z}" rpy="0 0 0" />
       </xacro:drive_wheel>
-      <xacro:drive_wheel parent="${name}_link" suffix="b" ref_position="0" >
+      <xacro:drive_wheel parent="${name}_link" suffix="b" >
         <origin xyz="${-caster_offset_x} 0.0 ${caster_offset_z}" rpy="0 0 0" />
       </xacro:drive_wheel>
-      <xacro:drive_wheel parent="${name}_link" suffix="fr" ref_position="0" >
+      <xacro:drive_wheel parent="${name}_link" suffix="fr" >
         <origin xyz="${caster_offset_x/2} ${-caster_offset_y} ${caster_offset_z}" rpy="0 0 0" />
       </xacro:drive_wheel>

File: cob_description/urdf/drive_wheel/drive_wheel.urdf.xacro (robot description, xacro)
@@ -39,5 +39,5 @@
   </xacro:macro>
   <!-- Macro for Caster hub only -->
-  <xacro:macro name="cob_caster_hub" params="*origin parent suffix ref_position" >
+  <xacro:macro name="cob_caster_hub" params="*origin parent suffix" >
     <joint name="${suffix}_rotation_joint" type="continuous">
       <insert_block name="origin" />
@@ -45,5 +45,4 @@
       <child link="${suffix}_rotation_link" />
       <axis xyz="0 0 1" />
-      <calibration rising="${ref_position}"/>
       <limit effort="100" velocity="100"/> <!-- alpha tested velocity and effort limits -->
       <safety_controller  k_velocity="10" />
@@ -72,7 +71,6 @@
     <xacro:cob_caster_transmission suffix="${suffix}" />
   </xacro:macro>
-  <xacro:macro name="drive_wheel" params="*origin parent suffix ref_position">
-    <xacro:cob_caster_hub parent="${parent}" suffix="${suffix}_caster"
-                          ref_position="${ref_position}" >
+  <xacro:macro name="drive_wheel" params="*origin parent suffix">
+    <xacro:cob_caster_hub parent="${parent}" suffix="${suffix}_caster" >
       <insert_block name="origin" />
     </xacro:cob_caster_hub>

File: raw_description/urdf/base_long/base.urdf.xacro (robot description, xacro)
@@ -15,8 +15,4 @@
   <property name="caster_offset_y_fr" value="-0.134" />
   <property name="caster_offset_z" value="0.09" />
-  <property name="cal_caster_fl" value="0.0" />
-  <property name="cal_caster_fr" value="0.0" />
-  <property name="cal_caster_bl" value="0.0" />
-  <property name="cal_caster_br" value="0.0" />
   <property name="battery_offset_x_f" value="0.141" />
   <property name="battery_offset_x_r" value="0.139" />
@@ -94,14 +90,14 @@
     </link>
     <!-- arrangement of the four drive_wheel modules -->
-    <xacro:drive_wheel parent="${name}_link" suffix="fl" ref_position="${cal_caster_fl - M_PI/4}" >
+    <xacro:drive_wheel parent="${name}_link" suffix="fl" >
       <origin xyz="${caster_offset_x} ${caster_offset_y_fl} ${caster_offset_z}" rpy="0 0 0" />
     </xacro:drive_wheel>
-    <xacro:drive_wheel parent="${name}_link" suffix="fr" ref_position="${cal_caster_fr - M_PI/4}" >
+    <xacro:drive_wheel parent="${name}_link" suffix="fr" >
       <origin xyz="${caster_offset_x} ${caster_offset_y_fr} ${caster_offset_z}" rpy="0 0 0" />
     </xacro:drive_wheel>
-    <xacro:drive_wheel parent="${name}_link" suffix="bl" ref_position="${cal_caster_bl - M_PI / 4 + M_PI}" >
+    <xacro:drive_wheel parent="${name}_link" suffix="bl" >
       <origin xyz="${-caster_offset_x} ${caster_offset_y_bl} ${caster_offset_z}" rpy=" 0 0 0" />
     </xacro:drive_wheel>
-    <xacro:drive_wheel parent="${name}_link" suffix="br" ref_position="${cal_caster_br - M_PI / 4 + M_PI}"  >
+    <xacro:drive_wheel parent="${name}_link" suffix="br" >
       <origin xyz="${-caster_offset_x} ${caster_offset_y_br} ${caster_offset_z}" rpy="0 0 0" />
     </xacro:drive_wheel>

File: raw_description/urdf/base_short/base.urdf.xacro (robot description, xacro)
@@ -15,8 +15,4 @@
   <property name="caster_offset_y_fr" value="-0.134" />
   <property name="caster_offset_z" value="0.09" />
-  <property name="cal_caster_fl" value="0.0" />
-  <property name="cal_caster_fr" value="0.0" />
-  <property name="cal_caster_bl" value="0.0" />
-  <property name="cal_caster_br" value="0.0" />
   <property name="battery_offset_x" value="0.0" />
   <property name="battery_offset_y" value="-0.008" />
@@ -92,14 +88,14 @@
     </link>
     <!-- arrangement of the four drive_wheel modules -->
-    <xacro:drive_wheel parent="${name}_link" suffix="fl" ref_position="${cal_caster_fl - M_PI/4}" >
+    <xacro:drive_wheel parent="${name}_link" suffix="fl" >
       <origin xyz="${caster_offset_x} ${caster_offset_y_fl} ${caster_offset_z}" rpy="0 0 0" />
     </xacro:drive_wheel>
-    <xacro:drive_wheel parent="${name}_link" suffix="fr" ref_position="${cal_caster_fr - M_PI/4}" >
+    <xacro:drive_wheel parent="${name}_link" suffix="fr" >
       <origin xyz="${caster_offset_x} ${caster_offset_y_fr} ${caster_offset_z}" rpy="0 0 0" />
     </xacro:drive_wheel>
-    <xacro:drive_wheel parent="${name}_link" suffix="bl" ref_position="${cal_caster_bl - M_PI / 4 + M_PI}" >
+    <xacro:drive_wheel parent="${name}_link" suffix="bl" >
       <origin xyz="${-caster_offset_x} ${caster_offset_y_bl} ${caster_offset_z}" rpy=" 0 0 0" />
     </xacro:drive_wheel>
-    <xacro:drive_wheel parent="${name}_link" suffix="br" ref_position="${cal_caster_br - M_PI / 4 + M_PI}"  >
+    <xacro:drive_wheel parent="${name}_link" suffix="br"  >
       <origin xyz="${-caster_offset_x} ${caster_offset_y_br} ${caster_offset_z}" rpy="0 0 0" />
     </xacro:drive_wheel>
