Commit message: simplify, unify simulated sensor makros according to new convention and hardware

File: cob_description/urdf/cob3_base/base.urdf.xacro (robot description, xacro)
@@ -54,13 +54,13 @@
     </xacro:drive_wheel>
     <!-- base laser front -->
-    <xacro:sick_s300_laser_v0 name="${name}_laser_front" parent="${name}" ros_topic="laser_front/scan_raw" update_rate="10" min_angle="-2.3562" max_angle="2.3562" >
+    <xacro:sick_s300_laser_v0 name="${name}_laser_front" parent="${name}">
       <origin xyz="${laser_front_x} ${laser_front_y} ${laser_front_z}" rpy="${laser_front_roll} ${laser_front_pitch} ${laser_front_yaw}" />
     </xacro:sick_s300_laser_v0>
     <!-- base laser rear -->
-    <xacro:sick_s300_laser_v0 name="${name}_laser_rear" parent="${name}" ros_topic="laser_rear/scan_raw" update_rate="10" min_angle="-2.3562" max_angle="2.3562" >
+    <xacro:sick_s300_laser_v0 name="${name}_laser_rear" parent="${name}">
       <origin xyz="${laser_rear_x} ${laser_rear_y} ${laser_rear_z}" rpy="${laser_rear_roll} ${laser_rear_pitch} ${laser_rear_yaw}" />
     </xacro:sick_s300_laser_v0>
     <!-- base laser top -->
-    <xacro:hokuyo_lx30_laser_v0 name="${name}_laser_top" parent="${name}" ros_topic="laser_top/scan_raw" update_rate="10" min_angle="-2.3562" max_angle="2.3562" >
+    <xacro:hokuyo_lx30_laser_v0 name="${name}_laser_top" parent="${name}">
       <origin xyz="${laser_top_x} ${laser_top_y} ${laser_top_z}" rpy="${laser_top_roll} ${laser_top_pitch} ${laser_top_yaw}" />
     </xacro:hokuyo_lx30_laser_v0>

File: cob_description/urdf/cob3_head/head_kinect.urdf.xacro (robot description, xacro)
@@ -72,5 +72,5 @@
     </link>
     <!-- cam3d -->
-    <xacro:cob_kinect_v0 name="cam3d" ros_topic="cam3d" parent="${name}_cam_reference_link">
+    <xacro:cob_kinect_v0 name="cam3d" parent="${name}_cam_reference_link">
       <origin xyz="${cam3d_x} ${cam3d_y} ${cam3d_z}" rpy="${cam3d_roll} ${cam3d_pitch} ${cam3d_yaw}" />
     </xacro:cob_kinect_v0>

File: cob_description/urdf/cob3_head/head_prosilicas_kinect.urdf.xacro (robot description, xacro)
@@ -73,13 +73,13 @@
     </link>
     <!-- left camera -->
-    <xacro:cob_prosilica_v0 name="${name}_color_camera_l" topic_prefix="stereo/left/" parent="${name}_cam_reference_link">
+    <xacro:cob_prosilica_v0 name="${name}_color_camera_stereo_left" parent="${name}_cam_reference_link">
       <origin xyz="${cam_l_x} ${cam_l_y} ${cam_l_z}" rpy="${cam_l_roll} ${cam_l_pitch} ${cam_l_yaw}" />
     </xacro:cob_prosilica_v0>
     <!-- right camera -->
-    <xacro:cob_prosilica_v0 name="${name}_color_camera_r" topic_prefix="stereo/right/" parent="${name}_cam_reference_link">
+    <xacro:cob_prosilica_v0 name="${name}_color_camera_stereo_right" parent="${name}_cam_reference_link">
       <origin xyz="${cam_r_x} ${cam_r_y} ${cam_r_z}" rpy="${cam_r_roll} ${cam_r_pitch} ${cam_r_yaw}" />
     </xacro:cob_prosilica_v0>
     <!-- cam3d -->
-    <xacro:cob_kinect_v0 name="cam3d" ros_topic="cam3d" parent="${name}_cam_reference_link">
+    <xacro:cob_kinect_v0 name="cam3d" parent="${name}_cam_reference_link">
       <origin xyz="${cam3d_x} ${cam3d_y} ${cam3d_z}" rpy="${cam3d_roll} ${cam3d_pitch} ${cam3d_yaw}" />
     </xacro:cob_kinect_v0>

File: cob_description/urdf/cob3_tray/tray.urdf.xacro (robot description, xacro)
@@ -78,14 +78,14 @@
     <link name="${name}_left_link"/>
     <!-- phidgets distance sensors -->
-    <xacro:phidgets_distance_v0 name="${name}_phidgets_1" ros_topic="/tray_sensors/range_1_sim" update_rate="10" parent="${name}_left">
+    <xacro:phidgets_distance_v0 name="${name}_phidgets_1" ros_topic="/tray_sensors/range_1_sim" parent="${name}_left_link">
       <origin xyz="-0.275 0 0.02" rpy="0 0 ${-M_PI/2}" />
     </xacro:phidgets_distance_v0>
-    <xacro:phidgets_distance_v0 name="${name}_phidgets_2" ros_topic="/tray_sensors/range_2_sim" update_rate="10" parent="${name}_left">
+    <xacro:phidgets_distance_v0 name="${name}_phidgets_2" ros_topic="/tray_sensors/range_2_sim" parent="${name}_left_link">
       <origin xyz="-0.2 0 0.02" rpy="0 0 ${-M_PI/2}" />
     </xacro:phidgets_distance_v0>
-    <xacro:phidgets_distance_v0 name="${name}_phidgets_3" ros_topic="/tray_sensors/range_3_sim" update_rate="10" parent="${name}_left">
+    <xacro:phidgets_distance_v0 name="${name}_phidgets_3" ros_topic="/tray_sensors/range_3_sim" parent="${name}_left_link">
       <origin xyz="-0.125 0 0.02" rpy="0 0 ${-M_PI/2}" />
     </xacro:phidgets_distance_v0>
-    <xacro:phidgets_distance_v0 name="${name}_phidgets_4" ros_topic="/tray_sensors/range_4_sim" update_rate="10" parent="${name}_left">
+    <xacro:phidgets_distance_v0 name="${name}_phidgets_4" ros_topic="/tray_sensors/range_4_sim" parent="${name}_left_link">
       <origin xyz="-0.05 0 0.02" rpy="0 0 ${-M_PI/2}" />
     </xacro:phidgets_distance_v0>

File: cob_description/urdf/cob3_tray/tray_3dof.urdf.xacro (robot description, xacro)
@@ -121,14 +121,14 @@
     </link>
     <!-- phidgets distance sensors -->
-    <xacro:phidgets_distance_v0 name="${name}_phidgets_1" ros_topic="/tray_sensors/range_1_sim" update_rate="10" parent="${name}_left">
+    <xacro:phidgets_distance_v0 name="${name}_phidgets_1" ros_topic="/tray_sensors/range_1_sim" parent="${name}_left_link">
       <origin xyz="0.04 -0.02424 0.07  " rpy="0 0 ${M_PI/2}" />
     </xacro:phidgets_distance_v0>
-    <xacro:phidgets_distance_v0 name="${name}_phidgets_2" ros_topic="/tray_sensors/range_2_sim" update_rate="10" parent="${name}_left">
+    <xacro:phidgets_distance_v0 name="${name}_phidgets_2" ros_topic="/tray_sensors/range_2_sim" parent="${name}_left_link">
       <origin xyz="0.09 -0.02424 0.07" rpy="0 0 ${M_PI/2}" />
     </xacro:phidgets_distance_v0>
-    <xacro:phidgets_distance_v0 name="${name}_phidgets_3" ros_topic="/tray_sensors/range_3_sim" update_rate="10" parent="${name}_left">
+    <xacro:phidgets_distance_v0 name="${name}_phidgets_3" ros_topic="/tray_sensors/range_3_sim" parent="${name}_left_link">
       <origin xyz="0.14 -0.02424 0.07" rpy="0 0 ${M_PI/2}" />
     </xacro:phidgets_distance_v0>
-    <xacro:phidgets_distance_v0 name="${name}_phidgets_4" ros_topic="/tray_sensors/range_4_sim" update_rate="10" parent="${name}_left">
+    <xacro:phidgets_distance_v0 name="${name}_phidgets_4" ros_topic="/tray_sensors/range_4_sim" parent="${name}_left_link">
       <origin xyz="0.19 -0.02424 0.07" rpy="0 0 ${M_PI/2}" />
     </xacro:phidgets_distance_v0>

File: cob_description/urdf/cob4_base/base.urdf.xacro (robot description, xacro)
@@ -64,11 +64,11 @@
     </xacro:unless>
     <!-- sensors -->
-    <xacro:sick_s300_laser_v0 name="${name}_laser_front" parent="${name}" ros_topic="laser_front/scan_raw" update_rate="12" min_angle="-2.094" max_angle="2.094" >
+    <xacro:sick_s300_laser_v0 name="${name}_laser_front" parent="${name}">
       <origin xyz="${laser_front_x} ${laser_front_y} ${laser_front_z}" rpy="${laser_front_roll} ${laser_front_pitch} ${laser_front_yaw}" />
     </xacro:sick_s300_laser_v0>
-    <xacro:sick_s300_laser_v0 name="${name}_laser_left" parent="${name}" ros_topic="laser_left/scan_raw" update_rate="12" min_angle="-2.094" max_angle="2.094" >
+    <xacro:sick_s300_laser_v0 name="${name}_laser_left" parent="${name}">
       <origin xyz="${laser_left_x} ${laser_left_y} ${laser_left_z}" rpy="${laser_left_roll} ${laser_left_pitch} ${laser_left_yaw}" />
     </xacro:sick_s300_laser_v0>
-    <xacro:sick_s300_laser_v0 name="${name}_laser_right" parent="${name}" ros_topic="laser_right/scan_raw" update_rate="12" min_angle="-2.094" max_angle="2.094" >
+    <xacro:sick_s300_laser_v0 name="${name}_laser_right" parent="${name}">
       <origin xyz="${laser_right_x} ${laser_right_y} ${laser_right_z}" rpy="${laser_right_roll} ${laser_right_pitch} ${laser_right_yaw}" />
     </xacro:sick_s300_laser_v0>

File: cob_description/urdf/cob4_torso/torso_2dof.urdf.xacro (robot description, xacro)
@@ -131,13 +131,13 @@
     </link>
     <!-- left camera -->
-    <xacro:cob_kinect_v0 name="${name}_cam3d_left" ros_topic="torso_cam3d_left" parent="${name}_3_link">
+    <xacro:cob_kinect_v0 name="${name}_cam3d_left" parent="${name}_3_link">
       <origin xyz="${torso_cam3d_left_x} ${torso_cam3d_left_y} ${torso_cam3d_left_z}" rpy="${torso_cam3d_left_roll} ${torso_cam3d_left_pitch} ${torso_cam3d_left_yaw}" />
     </xacro:cob_kinect_v0>
     <!-- right camera -->
-    <xacro:cob_kinect_v0 name="${name}_cam3d_right" ros_topic="torso_cam3d_right" parent="${name}_3_link">
+    <xacro:cob_kinect_v0 name="${name}_cam3d_right" parent="${name}_3_link">
       <origin xyz="${torso_cam3d_right_x} ${torso_cam3d_right_y} ${torso_cam3d_right_z}" rpy="${torso_cam3d_right_roll} ${torso_cam3d_right_pitch} ${torso_cam3d_right_yaw}" />
     </xacro:cob_kinect_v0>
     <!-- down camera -->
-    <xacro:softkinetic name="${name}_cam3d_down" ros_topic="torso_cam3d_down" parent="${name}_3_link">
+    <xacro:softkinetic name="${name}_cam3d_down" parent="${name}_3_link">
       <origin xyz="${torso_cam3d_down_x} ${torso_cam3d_down_y} ${torso_cam3d_down_z}" rpy="${torso_cam3d_down_roll} ${torso_cam3d_down_pitch} ${torso_cam3d_down_yaw}" />
     </xacro:softkinetic>

File: cob_description/urdf/cob4_torso/torso_3dof.urdf.xacro (robot description, xacro)
@@ -133,13 +133,13 @@
     </link>
     <!-- left camera -->
-    <xacro:cob_kinect_v0 name="${name}_cam3d_left" ros_topic="torso_cam3d_left" parent="${name}_3_link">
+    <xacro:cob_kinect_v0 name="${name}_cam3d_left" parent="${name}_3_link">
       <origin xyz="${torso_cam3d_left_x} ${torso_cam3d_left_y} ${torso_cam3d_left_z}" rpy="${torso_cam3d_left_roll} ${torso_cam3d_left_pitch} ${torso_cam3d_left_yaw}" />
     </xacro:cob_kinect_v0>
     <!-- right camera -->
-    <xacro:cob_kinect_v0 name="${name}_cam3d_right" ros_topic="torso_cam3d_right" parent="${name}_3_link">
+    <xacro:cob_kinect_v0 name="${name}_cam3d_right" parent="${name}_3_link">
       <origin xyz="${torso_cam3d_right_x} ${torso_cam3d_right_y} ${torso_cam3d_right_z}" rpy="${torso_cam3d_right_roll} ${torso_cam3d_right_pitch} ${torso_cam3d_right_yaw}" />
     </xacro:cob_kinect_v0>
     <!-- down camera -->
-    <xacro:softkinetic name="${name}_cam3d_down" ros_topic="torso_cam3d_down" parent="${name}_3_link">
+    <xacro:softkinetic name="${name}_cam3d_down" parent="${name}_3_link">
       <origin xyz="${torso_cam3d_down_x} ${torso_cam3d_down_y} ${torso_cam3d_down_z}" rpy="${torso_cam3d_down_roll} ${torso_cam3d_down_pitch} ${torso_cam3d_down_yaw}" />
     </xacro:softkinetic>

File: cob_description/urdf/cob4_torso/torso_static.urdf.xacro (robot description, xacro)
@@ -127,13 +127,13 @@
     </link>
     <!-- left camera -->
-    <xacro:cob_kinect_v0 name="${name}_cam3d_left" ros_topic="torso_cam3d_left" parent="${name}_3_link">
+    <xacro:cob_kinect_v0 name="${name}_cam3d_left" parent="${name}_3_link">
       <origin xyz="${torso_cam3d_left_x} ${torso_cam3d_left_y} ${torso_cam3d_left_z}" rpy="${torso_cam3d_left_roll} ${torso_cam3d_left_pitch} ${torso_cam3d_left_yaw}" />
     </xacro:cob_kinect_v0>
     <!-- right camera -->
-    <xacro:cob_kinect_v0 name="${name}_cam3d_right" ros_topic="torso_cam3d_right" parent="${name}_3_link">
+    <xacro:cob_kinect_v0 name="${name}_cam3d_right" parent="${name}_3_link">
       <origin xyz="${torso_cam3d_right_x} ${torso_cam3d_right_y} ${torso_cam3d_right_z}" rpy="${torso_cam3d_right_roll} ${torso_cam3d_right_pitch} ${torso_cam3d_right_yaw}" />
     </xacro:cob_kinect_v0>
     <!-- down camera -->
-    <xacro:softkinetic name="${name}_cam3d_down" ros_topic="torso_cam3d_down" parent="${name}_3_link">
+    <xacro:softkinetic name="${name}_cam3d_down" parent="${name}_3_link">
       <origin xyz="${torso_cam3d_down_x} ${torso_cam3d_down_y} ${torso_cam3d_down_z}" rpy="${torso_cam3d_down_roll} ${torso_cam3d_down_pitch} ${torso_cam3d_down_yaw}" />
     </xacro:softkinetic>

File: cob_description/urdf/sensors/kinect.gazebo.xacro (robot description, xacro)
@@ -1,5 +1,5 @@
 <?xml version="1.0"?>
 <root xmlns:xacro="http://www.ros.org/wiki/xacro">
-  <xacro:macro name="cob_kinect_gazebo_v0" params="name ros_topic">
+  <xacro:macro name="cob_kinect_gazebo_v0" params="name">
     <gazebo reference="${name}_frame">
       <sensor type="depth" name="${name}_frame_sensor">
@@ -25,5 +25,5 @@
         <plugin name="${name}_controller" filename="libgazebo_ros_openni_kinect.so">
           <updateRate>20.0</updateRate>
-          <cameraName>${ros_topic}</cameraName>
+          <cameraName>${name}</cameraName>
           <frameName>${name}_link</frameName>
           <imageTopicName>rgb/image_raw</imageTopicName>

File: cob_description/urdf/sensors/kinect.urdf.xacro (robot description, xacro)
@@ -2,5 +2,5 @@
 <root xmlns:xacro="http://www.ros.org/wiki/xacro">
   <xacro:include filename="$(find cob_description)/urdf/sensors/kinect.gazebo.xacro" />
-  <xacro:macro name="cob_kinect_v0" params="name parent *origin ros_topic">
+  <xacro:macro name="cob_kinect_v0" params="name parent *origin">
     <joint name="${name}_joint" type="fixed">
       <insert_block name="origin" />
@@ -33,5 +33,5 @@
     <link name="${name}_frame"/>
     <!-- extensions -->
-    <xacro:cob_kinect_gazebo_v0 name="${name}" ros_topic="${ros_topic}" />
+    <xacro:cob_kinect_gazebo_v0 name="${name}"/>
   </xacro:macro>
 </root>

File: cob_description/urdf/sensors/phidgets_distance.gazebo.xacro (robot description, xacro)
@@ -1,9 +1,9 @@
 <?xml version="1.0"?>
 <robot xmlns:xacro="http://www.ros.org/wiki/xacro">
-  <xacro:macro name="phidgets_distance_gazebo_v0" params="name ros_topic update_rate">
+  <xacro:macro name="phidgets_distance_gazebo_v0" params="name ros_topic">
     <gazebo reference="${name}_link">
       <sensor name="${name}" type="ray">
         <always_on>true</always_on>
-        <update_rate>${update_rate}</update_rate>
+        <update_rate>10.0</update_rate>
         <pose>0 0 0 0 0 0</pose>
         <visualize>false</visualize>

File: cob_description/urdf/sensors/phidgets_distance.urdf.xacro (robot description, xacro)
@@ -2,14 +2,14 @@
 <robot xmlns:xacro="http://www.ros.org/wiki/xacro">
   <xacro:include filename="$(find cob_description)/urdf/sensors/phidgets_distance.gazebo.xacro" />
-  <xacro:macro name="phidgets_distance_v0" params="name parent *origin ros_topic update_rate">
+  <xacro:macro name="phidgets_distance_v0" params="name parent *origin ros_topic">
     <joint name="${name}_joint" type="fixed">
       <axis xyz="0 1 0" />
       <insert_block name="origin" />
-      <parent link="${parent}_link"/>
+      <parent link="${parent}"/>
       <child link="${name}_link"/>
     </joint>
     <link name="${name}_link"/>
     <!-- gazebo extensions -->
-    <xacro:phidgets_distance_gazebo_v0 name="${name}" ros_topic="${ros_topic}" update_rate="${update_rate}" />
+    <xacro:phidgets_distance_gazebo_v0 name="${name}" ros_topic="${ros_topic}" />
   </xacro:macro>
 </robot>

File: cob_description/urdf/sensors/prosilica.gazebo.xacro (robot description, xacro)
@@ -1,5 +1,5 @@
 <?xml version="1.0"?>
 <root xmlns:xacro="http://www.ros.org/wiki/xacro">
-  <xacro:macro name="cob_prosilica_gazebo_v0" params="name topic_prefix">
+  <xacro:macro name="cob_prosilica_gazebo_v0" params="name">
     <gazebo reference="${name}_frame">
       <sensor type="camera" name="${name}_sensor">
@@ -27,7 +27,7 @@
           <cameraName>${name}</cameraName>
           <frameName>${name}_link</frameName>
-          <topicName>${topic_prefix}image_data</topicName>
-          <imageTopicName>${topic_prefix}image_raw</imageTopicName>
-          <cameraInfoTopicName>${topic_prefix}camera_info</cameraInfoTopicName>
+          <topicName>image_data</topicName>
+          <imageTopicName>image_raw</imageTopicName>
+          <cameraInfoTopicName>camera_info</cameraInfoTopicName>
           <pollServiceName>request_image</pollServiceName>
           <CxPrime>697.69</CxPrime>

File: cob_description/urdf/sensors/prosilica.urdf.xacro (robot description, xacro)
@@ -3,5 +3,5 @@
        name="LaserBlock">
   <xacro:include filename="$(find cob_description)/urdf/sensors/prosilica.gazebo.xacro" />
-  <xacro:macro name="cob_prosilica_v0" params="name parent *origin topic_prefix">
+  <xacro:macro name="cob_prosilica_v0" params="name parent *origin">
     <joint name="${name}_joint" type="fixed">
       <insert_block name="origin" />
@@ -35,5 +35,5 @@
     </joint>
     <link name="${name}_frame"/>
-    <xacro:cob_prosilica_gazebo_v0 name="${name}" topic_prefix="${topic_prefix}"/>
+    <xacro:cob_prosilica_gazebo_v0 name="${name}"/>
   </xacro:macro>
 </robot>

File: cob_description/urdf/sensors/sick_s300_laser.gazebo.xacro (robot description, xacro)
@@ -1,9 +1,9 @@
 <?xml version="1.0"?>
 <robot xmlns:xacro="http://www.ros.org/wiki/xacro">
-  <xacro:macro name="sick_s300_laser_gazebo_v0" params="name ros_topic update_rate min_angle max_angle">
+  <xacro:macro name="sick_s300_laser_gazebo_v0" params="name">
     <gazebo reference="${name}_link">
       <sensor name="${name}" type="ray">
         <always_on>true</always_on>
-        <update_rate>${update_rate}</update_rate>
+        <update_rate>25.0</update_rate>
         <pose>0 0 0 0 0 0</pose>
         <visualize>false</visualize>
@@ -13,6 +13,6 @@
               <samples>541</samples>
               <resolution>1.0</resolution>
-              <min_angle>${min_angle}</min_angle>
-              <max_angle>${max_angle}</max_angle>
+              <min_angle>-2.3562</min_angle>
+              <max_angle>2.3562</max_angle>
             </horizontal>
           </scan>
@@ -29,5 +29,5 @@
         </ray>
         <plugin name="gazebo_ros_${name}_controller" filename="libgazebo_ros_laser.so">
-          <topicName>${ros_topic}</topicName>
+          <topicName>${name}/scan_raw</topicName>
           <frameName>${name}_link</frameName>
         </plugin>

File: cob_description/urdf/sensors/softkinetic.gazebo.xacro (robot description, xacro)
@@ -1,5 +1,5 @@
 <?xml version="1.0"?>
 <robot xmlns:xacro="http://www.ros.org/wiki/xacro">
-  <xacro:macro name="softkinetic_gazebo" params="name ros_topic">
+  <xacro:macro name="softkinetic_gazebo" params="name">
     <gazebo reference="${name}_frame">
       <sensor type="depth" name="${name}_frame_sensor">
@@ -25,5 +25,5 @@
         <plugin name="${name}_frame_controller" filename="libgazebo_ros_openni_kinect.so">
           <updateRate>25.0</updateRate>
-          <cameraName>${ros_topic}</cameraName>
+          <cameraName>${name}</cameraName>
           <imageTopicName>rgb/image_raw</imageTopicName>
           <depthImageTopicName>depth/image_raw</depthImageTopicName>

File: cob_description/urdf/sensors/softkinetic.urdf.xacro (robot description, xacro)
@@ -2,5 +2,5 @@
 <robot xmlns:xacro="http://www.ros.org/wiki/xacro">
   <xacro:include filename="$(find cob_description)/urdf/sensors/softkinetic.gazebo.xacro" />
-  <xacro:macro name="softkinetic" params="name parent ros_topic *origin">
+  <xacro:macro name="softkinetic" params="name parent *origin">
     <joint name="${name}_joint" type="fixed">
       <insert_block name="origin" />
@@ -38,5 +38,5 @@
     <link name="${name}_optical_frame"/>
     <!-- extensions -->
-    <xacro:softkinetic_gazebo name="${name}" ros_topic="${ros_topic}" />
+    <xacro:softkinetic_gazebo name="${name}"/>
   </xacro:macro>
 </robot>

File: raw_description/urdf/base_long/base.urdf.xacro (robot description, xacro)
@@ -99,13 +99,13 @@
     </xacro:drive_wheel>
     <!-- base laser front -->
-    <xacro:sick_s300_laser_v0 name="${name}_laser_front" parent="${name}" ros_topic="laser_front/scan_raw" update_rate="10" min_angle="-2.3562" max_angle="2.3562" >
+    <xacro:sick_s300_laser_v0 name="${name}_laser_front" parent="${name}">
       <origin xyz="${laser_front_x} ${laser_front_y} ${laser_front_z}" rpy="${laser_front_roll} ${laser_front_pitch} ${laser_front_yaw}" />
     </xacro:sick_s300_laser_v0>
     <!-- base laser rear -->
-    <xacro:sick_s300_laser_v0 name="${name}_laser_rear" parent="${name}" ros_topic="laser_rear/scan_raw" update_rate="10" min_angle="-2.3562" max_angle="2.3562" >
+    <xacro:sick_s300_laser_v0 name="${name}_laser_rear" parent="${name}">
       <origin xyz="${laser_rear_x} ${laser_rear_y} ${laser_rear_z}" rpy="${laser_rear_roll} ${laser_rear_pitch} ${laser_rear_yaw}" />
     </xacro:sick_s300_laser_v0>
     <!-- cam3d -->
-    <!--xacro:cob_kinect_v0 name="${name}_cam3d" ros_topic="cam3d" parent="${name}_link">
+    <!--xacro:cob_kinect_v0 name="${name}_cam3d" parent="${name}_link">
       <origin xyz="0.51 0.12 0.27" rpy="-${M_PI/2} 0 -${M_PI/2}" />
     </xacro:cob_kinect_v0-->

File: raw_description/urdf/base_short/base.urdf.xacro (robot description, xacro)
@@ -97,13 +97,13 @@
     </xacro:drive_wheel>
     <!-- base laser front -->
-    <xacro:sick_s300_laser_v0 name="${name}_laser_front" parent="${name}" ros_topic="laser_front/scan_raw" update_rate="10" min_angle="-2.3562" max_angle="2.3562" >
+    <xacro:sick_s300_laser_v0 name="${name}_laser_front" parent="${name}">
       <origin xyz="${laser_front_x} ${laser_front_y} ${laser_front_z}" rpy="${laser_front_roll} ${laser_front_pitch} ${laser_front_yaw}" />
     </xacro:sick_s300_laser_v0>
     <!-- base laser rear -->
-    <xacro:sick_s300_laser_v0 name="${name}_laser_rear" parent="${name}" ros_topic="laser_rear/scan_raw" update_rate="10" min_angle="-2.3562" max_angle="2.3562" >
+    <xacro:sick_s300_laser_v0 name="${name}_laser_rear" parent="${name}">
       <origin xyz="${laser_rear_x} ${laser_rear_y} ${laser_rear_z}" rpy="${laser_rear_roll} ${laser_rear_pitch} ${laser_rear_yaw}" />
     </xacro:sick_s300_laser_v0>
     <!-- cam3d -->
-    <!--xacro:cob_kinect_v0 name="${name}_cam3d" ros_topic="cam3d" parent="${name}_link">
+    <!--xacro:cob_kinect_v0 name="${name}_cam3d" parent="${name}_link">
       <origin xyz="0.51 0.12 0.27" rpy="-${M_PI/2} 0 -${M_PI/2}" />
     </xacro:cob_kinect_v0-->
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