Commit message: set default inertias

File: cob_description/urdf/cob4_gripper/gripper.urdf.xacro (robot description, xacro)
@@ -11,9 +11,22 @@
     </joint>
     <link name="${name}_base_link">
-      <inertial>
-        <origin xyz="0 0 0" rpy="0 0 0"/>
-        <mass value="0.01"/>
-        <inertia ixx="1" ixy="0" ixz="0" iyy="1" iyz="0" izz="1" />
-      </inertial>
+      <xacro:default_inertial/>
+<!--
+       <xacro:cylinder_inertial radius="0.300" length="0.046" mass="5.0">
+        <origin xyz="0.03 0.08 0.01" rpy="0 0 0" />
+      </xacro:cylinder_inertial>
+-->
+      <visual>
+        <origin xyz="0 0 0" rpy="0 0 0" />
+        <geometry>
+          <box size="0.001 0.001 0.001" />
+        </geometry>
+      </visual>
+      <collision>
+        <origin xyz="0 0 0" rpy="0 0 0" />
+        <geometry>
+          <box size="0.001 0.001 0.001" />
+        </geometry>
+      </collision>
     </link>
     <!-- joint between base_link and gripper_palm_link -->
@@ -24,9 +37,5 @@
     </joint>
     <link name="${name}_palm_link">
-      <inertial>
-        <origin xyz="0 0 0" rpy="0 0 0"/>
-        <mass value="1.0"/>
-        <inertia ixx="0.200549" ixy="0.001322" ixz="-0.000000" iyy="0.123664" iyz="-0.000000" izz="0.104101" />
-      </inertial>
+      <xacro:default_inertial/>
       <visual>
         <origin xyz="0 0 0.005" rpy="0 0 0" />
@@ -54,9 +63,5 @@
     </joint>
     <link name="${name}_finger_1_link">
-      <inertial>
-        <origin xyz="0 0 0" rpy="0 0 0"/>
-        <mass value="6.209720"/>
-        <inertia ixx="0.171118" ixy="0.002544" ixz="-0.000000" iyy="0.083077" iyz="0.000000" izz="0.120948" />
-      </inertial>
+      <xacro:default_inertial/>
       <visual>
         <origin xyz="0 0 0" rpy="0 0 0" />
@@ -84,9 +89,5 @@
     </joint>
     <link name="${name}_finger_2_link">
-      <inertial>
-        <origin xyz="0 0 0" rpy="0 0 0"/>
-        <mass value="1.0"/>
-        <inertia ixx="0.01" ixy="0" ixz="0" iyy="0.01" iyz="0" izz="0.01" />
-      </inertial>
+      <xacro:default_inertial/>
       <visual>
         <origin xyz="0 0 0" rpy="0 0 0" />

Commit message: addapted urdf to the real gripper positions

File: cob_description/urdf/cob4_gripper/gripper.urdf.xacro (robot description, xacro)
@@ -34,5 +34,5 @@
       <xacro:default_inertial/>
       <visual>
-        <!--origin xyz="0 0 0.005" rpy="0 0 0" /-->
+        <origin xyz="0 0 0" rpy="0 0 0" />
         <geometry>
           <mesh filename="package://cob_description/meshes/cob4_gripper/palm.stl" />
@@ -41,5 +41,5 @@
       </visual>
       <collision>
-        <!--origin xyz="0 0 0.0005" rpy="0 0 0" /-->
+        <origin xyz="0 0 0" rpy="0 0 0" />
         <geometry>
           <mesh filename="package://cob_description/meshes/cob4_gripper/palm.stl" />
@@ -47,10 +47,31 @@
       </collision>
     </link>
+    <!-- joint between base_link and gripper_base_link -->
+    <joint name="${name}_camera_joint" type="fixed" >
+      <origin xyz="0 0 0" rpy="0 ${M_PI/2} 0" />
+      <parent link="${name}_palm_link" />
+      <child link="${name}_camera_link" />
+    </joint>
+    <link name="${name}_camera_link">
+      <xacro:default_inertial/>
+      <visual>
+        <origin xyz="0 0 0" rpy="0 0 0" />
+        <geometry>
+          <box size="0.001 0.001 0.001" />
+        </geometry>
+      </visual>
+      <collision>
+        <origin xyz="0 0 0" rpy="0 0 0" />
+        <geometry>
+          <box size="0.001 0.001 0.001" />
+        </geometry>
+      </collision>
+    </link>
     <!-- joint between gripper_palm_link and gripper_finger_1_link -->
     <joint name="${name}_finger_1_joint" type="revolute">
-      <origin xyz="0 0.02163 0.04409" rpy="0 ${M_PI/2} 0.11" />
-      <parent link="${name}_palm_link"/>
+      <origin xyz="-0.04409 0.02163  0" rpy="0 0 -0.2" />
+      <parent link="${name}_camera_link"/>
       <child link="${name}_finger_1_link"/>
-      <axis xyz="0 0 1" />
+      <axis xyz="0 0 -1" />
       <dynamics damping="0.0" friction="0.0"/>
       <calibration rising="${finger_1_ref}"/>
@@ -75,8 +96,8 @@
     <!-- joint between gripper_finger_1_link and gripper_finger_2_link -->
     <joint name="${name}_finger_2_joint" type="revolute">
-      <origin xyz="-0.0712 0 0" rpy="0 0 0" />
+      <origin xyz="-0.0712 0 0" rpy="0 0 -0.3" />
       <parent link="${name}_finger_1_link"/>
       <child link="${name}_finger_2_link"/>
-      <axis xyz="0 0 1" />
+      <axis xyz="0 0 -1" />
       <dynamics damping="0.0" friction="0.0"/>
       <calibration rising="${finger_2_ref}"/>

Commit message: redefined meshes origin

File: cob_description/urdf/cob4_gripper/gripper.urdf.xacro (robot description, xacro)
@@ -70,8 +70,8 @@
     <!-- joint between gripper_palm_link and gripper_finger_1_link -->
     <joint name="${name}_finger_1_joint" type="revolute">
-      <origin xyz="-0.04409 0.02163  0" rpy="0 0 -0.2" />
+      <origin xyz="-0.04409 0.02163  0" rpy="${M_PI} 0 -0.2" />
       <parent link="${name}_camera_link"/>
       <child link="${name}_finger_1_link"/>
-      <axis xyz="0 0 -1" />
+      <axis xyz="0 0 1" />
       <dynamics damping="0.0" friction="0.0"/>
       <calibration rising="${finger_1_ref}"/>
@@ -96,8 +96,8 @@
     <!-- joint between gripper_finger_1_link and gripper_finger_2_link -->
     <joint name="${name}_finger_2_joint" type="revolute">
-      <origin xyz="-0.0712 0 0" rpy="0 0 -0.3" />
+      <origin xyz="-0.0712 0 0" rpy="0 0 0.3" />
       <parent link="${name}_finger_1_link"/>
       <child link="${name}_finger_2_link"/>
-      <axis xyz="0 0 -1" />
+      <axis xyz="0 0 1" />
       <dynamics damping="0.0" friction="0.0"/>
       <calibration rising="${finger_2_ref}"/>
