Commit message: collada meshes for cob4_gripper

File: cob_description/urdf/cob4_gripper/gripper.gazebo.xacro (robot description, xacro)
@@ -5,15 +5,12 @@
       <gravity>true</gravity>
       <self_collide>false</self_collide>
-      <material>IPA/LightGrey</material>
     </gazebo>
     <gazebo reference="${name}_finger_1_link">
       <gravity>true</gravity>
       <self_collide>false</self_collide>
-      <material>IPA/LightGrey</material>
     </gazebo>
     <gazebo reference="${name}_finger_2_link">
       <gravity>true</gravity>
       <self_collide>false</self_collide>
-      <material>IPA/LightGrey</material>
     </gazebo>
   </xacro:macro>

File: cob_description/urdf/cob4_gripper/gripper.urdf.xacro (robot description, xacro)
@@ -36,7 +36,6 @@
         <origin xyz="0 0 0" rpy="0 0 0" />
         <geometry>
-          <mesh filename="package://cob_description/meshes/cob4_gripper/palm.stl" />
+          <mesh filename="package://cob_description/meshes/cob4_gripper/palm.dae" />
         </geometry>
-        <material name="IPA/LightGrey" />
       </visual>
       <collision>
@@ -83,7 +82,6 @@
         <origin xyz="0 0 0" rpy="0 0 0" />
         <geometry>
-          <mesh filename="package://cob_description/meshes/cob4_gripper/finger_1.stl" />
+          <mesh filename="package://cob_description/meshes/cob4_gripper/finger_1.dae" />
         </geometry>
-        <material name="IPA/LightGrey" />
       </visual>
       <collision>
@@ -109,7 +107,6 @@
         <origin xyz="0 0 0" rpy="0 0 0" />
         <geometry>
-          <mesh filename="package://cob_description/meshes/cob4_gripper/finger_2.stl" />
+          <mesh filename="package://cob_description/meshes/cob4_gripper/finger_2.dae" />
         </geometry>
-        <material name="IPA/LightGrey" />
       </visual>
       <collision>
