Commit message: review velocity axis limit

File: cob_description/urdf/cob4_sensorring/sensorring_3dcs.urdf.xacro (robot description, xacro)
@@ -30,5 +30,5 @@
       <child link="${name}_link" />
       <axis xyz="0 0 1" />
-      <limit effort="100" lower="-6.2831" upper="6.2831" velocity="6.28"/>
+      <limit effort="100" lower="-6.2831" upper="6.2831" velocity="2.62"/>
     </joint>
     <link name="${name}_link">

File: cob_description/urdf/cob4_sensorring/sensorring_3dcs_asus.urdf.xacro (robot description, xacro)
@@ -31,5 +31,5 @@
       <child link="${name}_link" />
       <axis xyz="0 0 1" />
-      <limit effort="100" lower="-6.2831" upper="6.2831" velocity="6.28"/>
+      <limit effort="100" lower="-6.2831" upper="6.2831" velocity="2.62"/>
     </joint>
     <link name="${name}_link">
