Commit message: move sensors from sensorring xacro to robot xacro

File: cob_description/urdf/cob4_sensorring/sensorring_3dcs_asus.urdf.xacro (robot description, xacro)
@@ -3,6 +3,4 @@
   <xacro:include filename="$(find cob_description)/urdf/cob4_sensorring/sensorring.gazebo.xacro" />
   <xacro:include filename="$(find cob_description)/urdf/cob4_sensorring/sensorring.transmission.xacro" />
-  <xacro:include filename="$(find cob_description)/urdf/sensors/sick_3dcs.urdf.xacro" />
-  <xacro:include filename="$(find cob_description)/urdf/sensors/kinect.urdf.xacro" />
   <xacro:macro name="sensorring" params="parent name *origin">
     <joint name="${name}_base_joint" type="fixed">
@@ -53,11 +51,4 @@
       </collision>
     </link>
-    <!-- camera -->
-    <xacro:sick_3dcs name="${name}_cam3d_front" ros_topic="${name}_cam3d_front" parent="${name}_link">
-      <origin xyz="${sensorring_cam3d_front_x} ${sensorring_cam3d_front_y} ${sensorring_cam3d_front_z}" rpy="${sensorring_cam3d_front_roll} ${sensorring_cam3d_front_pitch} ${sensorring_cam3d_front_yaw}" />
-    </xacro:sick_3dcs>
-    <xacro:cob_kinect_v0 name="${name}_cam3d_back" ros_topic="${name}_cam3d_back" parent="${name}_link">
-      <origin xyz="${sensorring_cam3d_back_x} ${sensorring_cam3d_back_y} ${sensorring_cam3d_back_z}" rpy="${sensorring_cam3d_back_roll} ${sensorring_cam3d_back_pitch} ${sensorring_cam3d_back_yaw}" />
-    </xacro:cob_kinect_v0>
     <!-- extensions -->
     <xacro:sensorring_gazebo name="${name}" />

File: cob_description/urdf/cob4_sensorring/sensorring_asus.urdf.xacro (robot description, xacro)
@@ -3,5 +3,4 @@
   <xacro:include filename="$(find cob_description)/urdf/cob4_sensorring/sensorring.gazebo.xacro" />
   <xacro:include filename="$(find cob_description)/urdf/cob4_sensorring/sensorring.transmission.xacro" />
-  <xacro:include filename="$(find cob_description)/urdf/sensors/kinect.urdf.xacro" />
   <xacro:macro name="sensorring" params="parent name *origin">
     <joint name="${name}_base_joint" type="fixed">
@@ -52,7 +51,4 @@
       </collision>
     </link>
-    <xacro:cob_kinect_v0 name="${name}_cam3d" ros_topic="${name}_cam3d" parent="${name}_link">
-      <origin xyz="${sensorring_cam3d_x} ${sensorring_cam3d_y} ${sensorring_cam3d_z}" rpy="${sensorring_cam3d_roll} ${sensorring_cam3d_pitch} ${sensorring_cam3d_yaw}" />
-    </xacro:cob_kinect_v0>
     <!-- extensions -->
     <xacro:sensorring_gazebo name="${name}" />
