Commit message: use default transmission macro

File: cob_description/urdf/cob4_sensorring/sensorring.transmission.xacro (robot description, xacro)
@@ -1,15 +1,7 @@
 <?xml version="1.0"?>
 <robot xmlns:xacro="http://www.ros.org/wiki/xacro">
+  <xacro:include filename="$(find cob_description)/urdf/common.xacro" />
   <xacro:macro name="sensorring_transmission" params="name">
-    <transmission name="${name}_trans">
-      <type>transmission_interface/SimpleTransmission</type>
-      <joint name="${name}_joint">
-        <hardwareInterface>PositionJointInterface</hardwareInterface>
-        <hardwareInterface>VelocityJointInterface</hardwareInterface>
-      </joint>
-      <actuator name="${name}_motor">
-        <mechanicalReduction>1</mechanicalReduction>
-      </actuator>
-    </transmission>
+    <xacro:default_transmission jname="${name}"/>
   </xacro:macro>
 </robot>

Commit message: allow static sensorring

File: cob_description/urdf/cob4_sensorring/sensorring.transmission.xacro (robot description, xacro)
@@ -2,6 +2,8 @@
 <robot xmlns:xacro="http://www.ros.org/wiki/xacro">
   <xacro:include filename="$(find cob_description)/urdf/common.xacro" />
-  <xacro:macro name="sensorring_transmission" params="name">
-    <xacro:default_transmission jname="${name}"/>
+  <xacro:macro name="sensorring_transmission" params="name active">
+    <xacro:if value="${active}">
+      <xacro:default_transmission jname="${name}"/>
+    </xacro:if>
   </xacro:macro>
 </robot>

File: cob_description/urdf/cob4_sensorring/sensorring.urdf.xacro (robot description, xacro)
@@ -3,5 +3,5 @@
   <xacro:include filename="$(find cob_description)/urdf/cob4_sensorring/sensorring.gazebo.xacro" />
   <xacro:include filename="$(find cob_description)/urdf/cob4_sensorring/sensorring.transmission.xacro" />
-  <xacro:macro name="sensorring" params="parent name *origin">
+  <xacro:macro name="sensorring" params="parent name *origin active:=false">
     <joint name="${name}_base_joint" type="fixed">
       <insert_block name="origin" />
@@ -24,11 +24,20 @@
       </collision>
     </link>
-    <joint name="${name}_joint" type="revolute">
-      <origin xyz="0 0 0" rpy="0 0 0" />
-      <parent link="${name}_base_link"/>
-      <child link="${name}_link" />
-      <axis xyz="0 0 1" />
-      <limit effort="100" lower="-6.2831" upper="6.2831" velocity="2.62"/>
-    </joint>
+    <xacro:unless value="${active}">
+      <joint name="${name}_joint" type="fixed">
+        <origin xyz="0 0 0" rpy="0 0 0" />
+        <parent link="${name}_base_link"/>
+        <child link="${name}_link" />
+      </joint>
+    </xacro:unless>
+    <xacro:if value="${active}">
+      <joint name="${name}_joint" type="revolute">
+        <origin xyz="0 0 0" rpy="0 0 0" />
+        <parent link="${name}_base_link"/>
+        <child link="${name}_link" />
+        <axis xyz="0 0 1" />
+        <limit effort="100" lower="-6.2831" upper="6.2831" velocity="2.62"/>
+      </joint>
+    </xacro:if>
     <link name="${name}_link">
       <xacro:default_inertial/>
@@ -53,5 +62,5 @@
     <!-- extensions -->
     <xacro:sensorring_gazebo name="${name}" />
-    <xacro:sensorring_transmission name="${name}" />
+    <xacro:sensorring_transmission name="${name}" active="${active}" />
   </xacro:macro>
 </robot>
