Commit message: better approximation of inertias for some more cob4 components

File: cob_description/urdf/cob4_sensorring/sensorring.urdf.xacro (robot description, xacro)
@@ -14,9 +14,7 @@
     </joint>
     <link name="${name}_link">
-      <inertial>
-        <origin xyz="0 0 0" rpy="0 0 0"/>
-        <mass value="0.1"/>
-        <inertia ixx="0.01" ixy="0" ixz="0" iyy="0.01" iyz="0" izz="0.01" />
-      </inertial>
+      <xacro:cylinder_inertial radius="0.250" length="0.1" mass="1.0">
+        <origin xyz="0 0 0" rpy="0 0 0" />
+      </xacro:cylinder_inertial>
     </link>
     <!-- extensions -->

File: cob_description/urdf/sensors/sick_s300_laser.urdf.xacro (robot description, xacro)
@@ -2,6 +2,6 @@
 <robot xmlns:xacro="http://www.ros.org/wiki/xacro">
   <xacro:include filename="$(find cob_description)/urdf/sensors/sick_s300_laser.gazebo.xacro" />
-  <property name="cylinder_radius" value="0.044" />  <!--simple collision model for the laser -->
-  <property name="cylinder_length" value="0.09" />
+  <property name="cylinder_radius" value="0.05" />  <!--simple collision model for the laser -->
+  <property name="cylinder_length" value="0.15" />
   <xacro:macro name="sick_s300_laser_v0" params="name parent *origin ros_topic update_rate min_angle max_angle">
     <joint name="${name}_joint" type="fixed">
@@ -12,13 +12,11 @@
     </joint>
     <link name="${name}_link" type="laser">
-      <inertial>
-        <mass value="0.001" />
+      <xacro:cylinder_inertial radius="${cylinder_radius}" length="${cylinder_length}" mass="1.2">
         <origin xyz="0 0 0" rpy="0 0 0" />
-        <inertia ixx="0.0001" ixy="0" ixz="0" iyy="0.000001" iyz="0" izz="0.0001" />
-      </inertial>
+      </xacro:cylinder_inertial>
       <visual>
         <origin xyz="0 0 0" rpy="0 0 0" />
         <geometry>
-    <mesh filename="package://cob_description/meshes/sensors/sick_s300_laser.dae"/>
+          <mesh filename="package://cob_description/meshes/sensors/sick_s300_laser.dae"/>
           <!--box size="0.001 0.001 0.001" /-->
         </geometry>

Commit message: set limit for sensorring

File: cob_description/urdf/cob4_sensorring/sensorring.urdf.xacro (robot description, xacro)
@@ -18,5 +18,5 @@
       <axis xyz="0 0 1" />
       <calibration rising="${sensorring_ref}"/>
-      <limit effort="100" lower="-6.2831" upper="6.2831" velocity="1.4"/>
+      <limit effort="100" lower="-6.2831" upper="6.2831" velocity="6.28"/>
     </joint>
     <link name="${name}_link">

Commit message: fixed xacro:if condition for melodic

File: cob_description/urdf/cob4_sensorring/sensorring.urdf.xacro (robot description, xacro)
@@ -3,5 +3,5 @@
   <xacro:include filename="$(find cob_description)/urdf/cob4_sensorring/sensorring.gazebo.xacro" />
   <xacro:include filename="$(find cob_description)/urdf/cob4_sensorring/sensorring.transmission.xacro" />
-  <xacro:macro name="sensorring" params="parent name *origin active:=false">
+  <xacro:macro name="sensorring" params="parent name *origin active:=True">
     <joint name="${name}_base_joint" type="fixed">
       <xacro:insert_block name="origin" />

Commit message: fix default value

File: cob_description/urdf/cob4_sensorring/sensorring.urdf.xacro (robot description, xacro)
@@ -3,5 +3,5 @@
   <xacro:include filename="$(find cob_description)/urdf/cob4_sensorring/sensorring.gazebo.xacro" />
   <xacro:include filename="$(find cob_description)/urdf/cob4_sensorring/sensorring.transmission.xacro" />
-  <xacro:macro name="sensorring" params="parent name *origin active:=True">
+  <xacro:macro name="sensorring" params="parent name *origin active:=False">
     <joint name="${name}_base_joint" type="fixed">
       <xacro:insert_block name="origin" />
