Commit message: new gazebo sensor structure

File: raw_description/urdf/base_long/base.gazebo.xacro (robot description, xacro)
@@ -26,19 +26,19 @@
     <gazebo reference="${name}_link">
       <selfCollide>true</selfCollide>
-      <sensor:contact name="${name}_contact_sensor">
-        <geom>${name}_link_geom</geom>
-        <updateRate>100.0</updateRate>
-        <controller:gazebo_ros_bumper name="${name}_gazebo_ros_bumper_controller" plugin="libgazebo_ros_bumper.so">
+      <sensor name='${name}_contact_sensor' type='contact'>
+        <contact>
+          <collision>${name}_link_geom</collision>
+        </contact>
+        <plugin name="${name}_gazebo_ros_bumper_controller" filename="libgazebo_ros_bumper.so">
           <alwaysOn>true</alwaysOn>
           <updateRate>100.0</updateRate>
           <bumperTopicName>${name}_bumper</bumperTopicName>
-          <interface:bumper name="${name}_bumper_iface" />
-        </controller:gazebo_ros_bumper>
-      </sensor:contact>
+        </plugin>
+      </sensor>
       <!--material>Gazebo/Grey</material-->
       <!--material value="IPA/Metal" /-->
     </gazebo>
     <gazebo>
-      <controller:gazebo_ros_p3d name="p3d_base_controller" plugin="libgazebo_ros_p3d.so">
+      <plugin name="p3d_base_controller" filename="libgazebo_ros_p3d.so">
         <alwaysOn>true</alwaysOn>
         <updateRate>100.0</updateRate>
@@ -47,8 +47,7 @@
         <gaussianNoise>0.01</gaussianNoise>
         <frameName>map</frameName>
-        <xyzOffsets>25.7 25.7 0</xyzOffsets> <!-- initialize odometry for fake localization-->
+        <xyzOffsets>25.7 25.7 0</xyzOffsets>  <!-- initialize odometry for fake localization-->
         <rpyOffsets>0 0 0</rpyOffsets>
-        <interface:position name="p3d_base_position"/>
-      </controller:gazebo_ros_p3d>
+      </plugin>
       <canonicalBody>${name}_footprint</canonicalBody>
     </gazebo>

Commit message: joint needs to be revolute do detect collision

File: raw_description/urdf/base_long/base.gazebo.xacro (robot description, xacro)
@@ -9,4 +9,5 @@
   </xacro:macro>
   <xacro:macro name="base_gazebo" params="name">
+    <!-- -->
     <gazebo reference="${name}_link">
       <gravity>true</gravity>

File: raw_description/urdf/vacuum_gripper/gripper.gazebo.xacro (robot description, xacro)
@@ -2,30 +2,18 @@
 <robot xmlns:xacro="http://www.ros.org/wiki/xacro">
   <xacro:macro name="vacuum_gripper_gazebo" params="name">
-	<gazebo reference="${name}_body">
-      <gravity>true</gravity>
+    <gazebo reference="${name}_frame">
       <self_collide>false</self_collide>
-      <sensor name='${name}_contact_sensor' type='contact'>
+      <sensor name='${name}_frame_sensor' type='contact'>
         <always_on>true</always_on>
-        <update_rate>10.0</update_rate>
+        <update_rate>100.0</update_rate>
         <contact>
-          <collision>${name}_body</collision>
-          <topic>${name}_bumper</topic>
+          <collision>${name}_frame_collision</collision>
+          <topic>$test_bumper</topic>
         </contact>
-        <plugin name="${name}_gazebo_ros_bumper_controller" filename="libgazebo_ros_bumper.so">
-          <alwaysOn>true</alwaysOn>
-          <frameName>world</frameName>
-          <bumperTopicName>${name}_bumper</bumperTopicName>
+        <plugin name="${name}_frame_gazebo_ros_bumper_controller" filename="libgazebo_ros_bumper.so">
+          <bodyName>${name}_frame</bodyName>
+          <bumperTopicName>test_bumper</bumperTopicName>
         </plugin>
       </sensor>
-      <mu1 value="500.0" />
-      <mu2 value="500.0" />
-      <kp  value="10000000.0" />
-      <kd  value="1.0" />
-    </gazebo>
-    <gazebo reference="gripper_to_tcp">
-      <stopKd value="1.0" />
-      <stopKp value="10000000.0" />
-      <fudgeFactor value="1.0" />
-      <provideFeedback value="true"/>
     </gazebo>
   </xacro:macro>

File: raw_description/urdf/vacuum_gripper/gripper.urdf.xacro (robot description, xacro)
@@ -10,10 +10,20 @@
   <xacro:macro name="vacuum_gripper" params="name parent *origin">
     <!-- joint between arm_ee_link and vacuum_gripper_link -->
-    <joint name="${name}_base_joint" type="fixed">
+    <joint name="${name}_base_joint" type="revolute">
         <xacro:insert_block name="origin"/>
         <parent link="${parent}"/>
         <child link="${name}_frame"/>
+        <axis xyz="0 1 0" />
+        <limit lower="${-2.0 * pi}" upper="${2.0 * pi}" effort="54.0" velocity="3.2"/>
+        <dynamics damping="0.0" friction="0.0"/>
     </joint>
-    <link name="${name}_frame"/>
+    <link name="${name}_frame">
+      <collision>
+        <geometry>
+          <box size="0.01 0.01 0.01"/>
+        </geometry>
+        <origin rpy="0 0 0" xyz="-0.01 0 0"/>
+      </collision>
+    </link>
     <joint name="gripper_to_palm" type="fixed">
         <parent link="${name}_frame"/>
@@ -22,11 +32,4 @@
     </joint>
     <link name="${name}_body">
-      	<inertial>
-            <mass value="0.04419" />
-            <origin xyz="0.00423 0.00284 0.0" rpy="0 0 0" />
-            <inertia  ixx="0.00000837047" ixy="0.00000583632" ixz="0.0"
-                      iyy="0.00000987067" iyz="0.0"
-                      izz="0.00001541768" />
-      	</inertial>
         <visual>
             <origin xyz="0 0 -0.048" rpy="0 0 0"/>

Commit message: identation

File: raw_description/urdf/base_long/base.gazebo.xacro (robot description, xacro)
@@ -9,5 +9,4 @@
   </xacro:macro>
   <xacro:macro name="base_gazebo" params="name">
-    <!-- -->
     <gazebo reference="${name}_link">
       <gravity>true</gravity>

File: raw_description/urdf/vacuum_gripper/gripper.urdf.xacro (robot description, xacro)
@@ -8,5 +8,5 @@
   <xacro:property name="gripper_height" value="0.14"/>
   <xacro:property name="gripper_body_height" value="0.14"/>
-  <xacro:property name="gripper_radius" value="0.05"/>
+  <xacro:property name="gripper_radius" value="0.01"/>
   <xacro:macro name="vacuum_gripper" params="name parent *origin">
     <!-- joint between arm_ee_link and vacuum_gripper_link -->
@@ -17,13 +17,13 @@
     </joint>
     <link name="${name}_frame">
-      <collision>
-        <geometry>
-          <box size="0.01 0.01 0.01"/>
-        </geometry>
-        <origin rpy="0 0 0" xyz="-0.01 0 0"/>
-      </collision>
-      <xacro:cylinder_inertial radius="0.075" length="0.12" mass="0.01">
-        <origin xyz="0.0 0.0 0.0" rpy="0 0 0" />
-      </xacro:cylinder_inertial>
+        <collision>
+            <geometry>
+                <box size="0.01 0.01 0.01"/>
+            </geometry>
+            <origin rpy="0 0 0" xyz="-0.01 0 0"/>
+        </collision>
+        <xacro:cylinder_inertial radius="0.075" length="0.12" mass="0.01">
+            <origin xyz="0.0 0.0 0.0" rpy="0 0 0" />
+        </xacro:cylinder_inertial>
     </link>
     <joint name="gripper_to_palm" type="fixed">
@@ -48,7 +48,7 @@
             </geometry>
         </collision>
-      <xacro:cylinder_inertial radius="0.075" length="0.12" mass="0.01">
-        <origin xyz="0.0 0.0 0.0" rpy="0 0 0" />
-      </xacro:cylinder_inertial>
+        <xacro:cylinder_inertial radius="0.075" length="0.12" mass="0.01">
+            <origin xyz="0.0 0.0 0.0" rpy="0 0 0" />
+        </xacro:cylinder_inertial>
     </link>
     <joint name="gripper_to_tcp" type="prismatic">
@@ -71,6 +71,6 @@
         </collision>
         <xacro:cylinder_inertial radius="0.075" length="0.12" mass="0.1">
-          <origin xyz="0.0 0.0 0.0" rpy="0 0 0" />
-        </xacro:cylinder_inertial>
+            <origin xyz="0.0 0.0 0.0" rpy="0 0 0" />
+      </xacro:cylinder_inertial>
      </link>
     <!-- extensions -->
