Commit message: changed wheel positions to make rotation right, also changed some bugs in the asymetric tower

File: raw_description/urdf/base_long/base.urdf.xacro (robot description, xacro)
@@ -15,8 +15,8 @@
   <!-- all simplified collision geometry are hand approximated from CAD model, sometimes from respective bounding boxes -->
   <property name="caster_offset_x" value="0.368" />  <!--modify here-->
-  <property name="caster_offset_y_bl" value="0.184" />
-  <property name="caster_offset_y_br" value="0.136" />
-  <property name="caster_offset_y_fl" value="0.134" />
-  <property name="caster_offset_y_fr" value="0.186" />
+  <property name="caster_offset_y_bl" value="0.134" />
+  <property name="caster_offset_y_br" value="-0.184" />
+  <property name="caster_offset_y_fl" value="0.184" />
+  <property name="caster_offset_y_fr" value="-0.134" />
   <property name="caster_offset_z" value="0.09" />
   <property name="battery_offset_x_f" value="0.141" />
@@ -234,14 +234,14 @@
     <!-- all four caster macros -->
     <xacro:cob_caster suffix="fl" parent="${name}_link" ref_position="${cal_caster_fl - M_PI/4}" >
-      <origin xyz="${-caster_offset_x} ${-caster_offset_y_bl} ${caster_offset_z}" rpy="0 0 0" />
+      <origin xyz="${caster_offset_x} ${caster_offset_y_fl} ${caster_offset_z}" rpy="0 0 0" />
     </xacro:cob_caster>
     <xacro:cob_caster suffix="fr" parent="${name}_link" ref_position="${cal_caster_fr - M_PI/4}" >
+      <origin xyz="${caster_offset_x} ${caster_offset_y_fr} ${caster_offset_z}" rpy="0 0 0" />
+    </xacro:cob_caster>
+    <xacro:cob_caster suffix="bl" parent="${name}_link" ref_position="${cal_caster_bl - M_PI / 4 + M_PI}" >
+      <origin xyz="${-caster_offset_x} ${caster_offset_y_bl} ${caster_offset_z}" rpy=" 0 0 0" />
+    </xacro:cob_caster>
+    <xacro:cob_caster suffix="br" parent="${name}_link" ref_position="${cal_caster_br - M_PI / 4 + M_PI}"  >
       <origin xyz="${-caster_offset_x} ${caster_offset_y_br} ${caster_offset_z}" rpy="0 0 0" />
-    </xacro:cob_caster>
-    <xacro:cob_caster suffix="bl" parent="${name}_link" ref_position="${cal_caster_bl - M_PI / 4 + M_PI}" >
-      <origin xyz="${caster_offset_x} ${-caster_offset_y_fl} ${caster_offset_z}" rpy=" 0 0 0" />
-    </xacro:cob_caster>
-    <xacro:cob_caster suffix="br" parent="${name}_link" ref_position="${cal_caster_br - M_PI / 4 + M_PI}"  >
-      <origin xyz="${caster_offset_x} ${caster_offset_y_fr} ${caster_offset_z}" rpy="0 0 0" />
     </xacro:cob_caster>
    <!-- cam3d -->

File: raw_description/urdf/base_short/base.urdf.xacro (robot description, xacro)
@@ -15,8 +15,8 @@
   <!-- all simplified collision geometry are hand approximated from CAD model, sometimes from respective bounding boxes -->
   <property name="caster_offset_x" value="0.228" />  <!--modify here-->
-  <property name="caster_offset_y_bl" value="0.186" />
-  <property name="caster_offset_y_br" value="0.134" />
-  <property name="caster_offset_y_fl" value="0.134" />
-  <property name="caster_offset_y_fr" value="0.186" />
+  <property name="caster_offset_y_bl" value="0.134" />
+  <property name="caster_offset_y_br" value="-0.184" />
+  <property name="caster_offset_y_fl" value="0.184" />
+  <property name="caster_offset_y_fr" value="-0.134" />
   <property name="caster_offset_z" value="0.09" />
   <property name="battery_offset_x_f" value="0.0" />
@@ -229,14 +229,14 @@
     <!-- all four caster macros -->
     <xacro:cob_caster suffix="fl" parent="${name}_link" ref_position="${cal_caster_fl - M_PI/4}" >
-      <origin xyz="${caster_offset_x} ${caster_offset_y_bl} ${caster_offset_z}" rpy="0 0 0" />
+      <origin xyz="${caster_offset_x} ${caster_offset_y_fl} ${caster_offset_z}" rpy="0 0 0" />
     </xacro:cob_caster>
     <xacro:cob_caster suffix="fr" parent="${name}_link" ref_position="${cal_caster_fr - M_PI/4}" >
-      <origin xyz="${caster_offset_x} ${-caster_offset_y_br} ${caster_offset_z}" rpy="0 0 0" />
+      <origin xyz="${caster_offset_x} ${caster_offset_y_fr} ${caster_offset_z}" rpy="0 0 0" />
     </xacro:cob_caster>
     <xacro:cob_caster suffix="bl" parent="${name}_link" ref_position="${cal_caster_bl - M_PI / 4 + M_PI}" >
-      <origin xyz="${-caster_offset_x} ${caster_offset_y_fl} ${caster_offset_z}" rpy=" 0 0 0" />
+      <origin xyz="${-caster_offset_x} ${caster_offset_y_bl} ${caster_offset_z}" rpy=" 0 0 0" />
     </xacro:cob_caster>
     <xacro:cob_caster suffix="br" parent="${name}_link" ref_position="${cal_caster_br - M_PI / 4 + M_PI}"  >
-      <origin xyz="${-caster_offset_x} ${-caster_offset_y_fr} ${caster_offset_z}" rpy="0 0 0" />
+      <origin xyz="${-caster_offset_x} ${caster_offset_y_br} ${caster_offset_z}" rpy="0 0 0" />
     </xacro:cob_caster>
    <!-- cam3d -->

File: raw_description/urdf/tower_asymetric/tower.gazebo.xacro (robot description, xacro)
@@ -4,5 +4,5 @@
        xmlns:interface="http://playerstage.sourceforge.net/gazebo/xmlschema/#interface"
        xmlns:xacro="http://ros.org/wiki/xacro">
-	<xacro:macro name="raw_tower_symetric_gazebo" params="name">
+	<xacro:macro name="raw_tower_asymetric_gazebo" params="name">
 		<gazebo reference="${name}_base_link">
 			<selfCollide>false</selfCollide>

File: raw_description/urdf/tower_asymetric/tower.urdf.xacro (robot description, xacro)
@@ -4,8 +4,8 @@
        xmlns:interface="http://playerstage.sourceforge.net/gazebo/xmlschema/#interface"
        xmlns:xacro="http://ros.org/wiki/xacro">
-  <include filename="$(find raw_description)/urdf/tower_symetric/tower.gazebo.xacro" />
+  <include filename="$(find raw_description)/urdf/tower_asymetric/tower.gazebo.xacro" />
   <!-- Properties -->
   <property name="tower_mass" value="6.49" />
-  <xacro:macro name="tower_symetric" params="name parent *origin" >
+  <xacro:macro name="tower_asymetric" params="name parent *origin" >
     <joint name="${name}_joint" type="fixed">
       <insert_block name="origin" />
@@ -29,13 +29,13 @@
       </visual>
        <collision>
-        <origin xyz="0 -0.03 -0.1" rpy="0 0 0"/>
+        <origin xyz="0 0 0.0865" rpy="0 0 0"/>
         <geometry>
           <!--mesh filename="package://raw_description/meshes/base/raw_tower_collision.stl"/-->
-          <box size="0.32 0.58 0.24" />
+          <box size="0.316 0.573 0.173" />
         </geometry>
         </collision>
     </link>
     <!-- extensions -->
-    <xacro:raw_tower_symetric_gazebo name="${name}" />
+    <xacro:raw_tower_asymetric_gazebo name="${name}" />
   </xacro:macro>
 </robot>

Commit message: allow laser calibration

File: raw_description/urdf/base_long/base.urdf.xacro (robot description, xacro)
@@ -25,8 +25,4 @@
   <property name="battery_size_y" value="0.148" />
   <property name="battery_size_z" value="0.26" />
-  <property name="base_laser_x" value="0.465" />
-  <property name="base_laser_y_back" value="0.23" />
-  <property name="base_laser_y_front" value="0.232" />
-  <property name="base_laser_z" value="0.178" />
   <!-- battery macros-->
   <xacro:macro name="cob_batteries" params="name parent *origin ">
@@ -104,9 +100,9 @@
     <!-- base laser front -->
     <xacro:sick_s300_laser_v0 name="${name}_laser_front" parent="${name}" ros_topic="scan_front_raw" update_rate="10" min_angle="-2.3562" max_angle="2.3562" >
-      <origin xyz="${base_laser_x} ${-base_laser_y_front} ${base_laser_z}" rpy="${M_PI} 0 ${-M_PI/4}" />
+      <origin xyz="${laser_front_x} ${laser_front_y} ${laser_front_z}" rpy="${laser_front_roll} ${laser_front_pitch} ${laser_front_yaw}" />
     </xacro:sick_s300_laser_v0>
     <!-- base laser rear -->
     <xacro:sick_s300_laser_v0 name="${name}_laser_rear" parent="${name}" ros_topic="scan_rear_raw" update_rate="10" min_angle="-2.3562" max_angle="2.3562" >
-      <origin xyz="${-base_laser_x} ${base_laser_y_back} ${base_laser_z}" rpy="${M_PI} 0 ${-5*M_PI/4}" />
+      <origin xyz="${laser_rear_x} ${laser_rear_y} ${laser_rear_z}" rpy="${laser_rear_roll} ${laser_rear_pitch} ${laser_rear_yaw}" />
     </xacro:sick_s300_laser_v0>
     <!-- cam3d -->

File: raw_description/urdf/base_short/base.urdf.xacro (robot description, xacro)
@@ -23,8 +23,4 @@
   <property name="battery_size_y" value="0.148" />
   <property name="battery_size_z" value="0.26" />
-  <property name="base_laser_x" value="0.32501" />
-  <property name="base_laser_y_back" value="0.232" />
-  <property name="base_laser_y_front" value="0.232" />
-  <property name="base_laser_z" value="0.178" />
   <!-- battery macros-->
   <xacro:macro name="cob_batteries" params="name parent *origin ">
@@ -102,9 +98,9 @@
     <!-- base laser front -->
     <xacro:sick_s300_laser_v0 name="${name}_laser_front" parent="${name}" ros_topic="scan_front_raw" update_rate="10" min_angle="-2.3562" max_angle="2.3562" >
-      <origin xyz="${base_laser_x} ${-base_laser_y_front} ${base_laser_z}" rpy="${M_PI} 0 ${-M_PI/4}" />
+      <origin xyz="${laser_front_x} ${laser_front_y} ${laser_front_z}" rpy="${laser_front_roll} ${laser_front_pitch} ${laser_front_yaw}" />
     </xacro:sick_s300_laser_v0>
     <!-- base laser rear -->
     <xacro:sick_s300_laser_v0 name="${name}_laser_rear" parent="${name}" ros_topic="scan_rear_raw" update_rate="10" min_angle="-2.3562" max_angle="2.3562" >
-      <origin xyz="${-base_laser_x} ${base_laser_y_back} ${base_laser_z}" rpy="${M_PI} 0 ${-5*M_PI/4}" />
+      <origin xyz="${laser_front_x} ${laser_front_y} ${laser_front_z}" rpy="${laser_front_roll} ${laser_front_pitch} ${laser_front_yaw}" />
     </xacro:sick_s300_laser_v0>
     <!-- cam3d -->

Commit message: get a stable behavior by tweaking the base mass/inertia

File: raw_description/urdf/base_long/base.urdf.xacro (robot description, xacro)
@@ -33,7 +33,7 @@
     </joint>
     <link name="${name}_battery">
-      <xacro:box_inertial x="${battery_size_x}" y="${battery_size_y}" z="${battery_size_z}" mass="${battery_mass}">
-        <origin xyz="0 0 0" rpy="0 0 0" />
-      </xacro:box_inertial>
+      <xacro:box_inertia width="${battery_size_x}" length="${battery_size_y}" height="${battery_size_z}" mass="${battery_mass}">
+        <origin xyz="0.0 0.0 0.0" rpy="0 0 0" />
+      </xacro:box_inertia>
       <visual>
         <origin xyz="0 0 0" rpy="0 0 0"/>
@@ -54,4 +54,13 @@
     <xacro:batteries_gazebo name="${name}" />
   </xacro:macro>
+  <xacro:macro name="box_inertia" params="width length height mass *origin">
+    <inertial>
+      <mass value="${mass}" />
+      <xacro:insert_block name="origin" />
+      <inertia ixx="${0.0833333 * mass * (width * width + height * height)}" ixy="0.0" ixz="0.0"
+        iyy="${0.0833333 * mass * (height * height + length * length)}" iyz="0.0"
+        izz="${0.0833333 * mass * (width * width + length * length)}" />
+    </inertial>
+  </xacro:macro>
   <xacro:macro name="raw_base" params="name">
     <link name="${name}_footprint"/>
@@ -62,10 +71,7 @@
     </joint>
     <link name="${name}_link">
-      <inertial>
-        <origin xyz="0 0 0" />
-        <mass value="${base_mass}" />
-        <inertia ixx="9.64" ixy="-0.02" ixz="0.44"
-                 iyy="11.33" iyz="-0.007" izz="3.07" />
-      </inertial>
+      <xacro:box_inertia width="1.04" length="0.58" height="0.12" mass="${base_mass}">
+        <origin xyz="0.0 0.0 0.0" rpy="0 0 0" />
+      </xacro:box_inertia>
       <visual>
         <origin xyz="0 0 0.209" rpy="0 0 0" />

Commit message: stable behavior by tweaking the base mass/inertia achieved

File: raw_description/urdf/base_long/base.urdf.xacro (robot description, xacro)
@@ -21,5 +21,5 @@
   <xacro:property name="battery_offset_z" value="0.065" />
   <xacro:property name="base_mass" value="83.1" />
-  <xacro:property name="battery_mass" value="25.0" />
+  <xacro:property name="battery_mass" value="50.0" />
   <xacro:property name="battery_size_x" value="0.5" />
   <xacro:property name="battery_size_y" value="0.148" />

Commit message: gripper mesh simplified

File: raw_description/urdf/base_long/base.urdf.xacro (robot description, xacro)
@@ -33,7 +33,7 @@
     </joint>
     <link name="${name}_battery">
-      <xacro:box_inertia width="${battery_size_x}" length="${battery_size_y}" height="${battery_size_z}" mass="${battery_mass}">
+      <xacro:box_inertial x="${battery_size_x}" y="${battery_size_y}" z="${battery_size_z}" mass="${battery_mass}">
         <origin xyz="0.0 0.0 0.0" rpy="0 0 0" />
-      </xacro:box_inertia>
+      </xacro:box_inertial>
       <visual>
         <origin xyz="0 0 0" rpy="0 0 0"/>
@@ -54,13 +54,4 @@
     <xacro:batteries_gazebo name="${name}" />
   </xacro:macro>
-  <xacro:macro name="box_inertia" params="width length height mass *origin">
-    <inertial>
-      <mass value="${mass}" />
-      <xacro:insert_block name="origin" />
-      <inertia ixx="${0.0833333 * mass * (width * width + height * height)}" ixy="0.0" ixz="0.0"
-        iyy="${0.0833333 * mass * (height * height + length * length)}" iyz="0.0"
-        izz="${0.0833333 * mass * (width * width + length * length)}" />
-    </inertial>
-  </xacro:macro>
   <xacro:macro name="raw_base" params="name">
     <link name="${name}_footprint"/>
@@ -71,7 +62,7 @@
     </joint>
     <link name="${name}_link">
-      <xacro:box_inertia width="1.04" length="0.58" height="0.12" mass="${base_mass}">
+      <xacro:box_inertial x="1.04" y="0.58" z="0.12" mass="${base_mass}">
         <origin xyz="0.0 0.0 0.0" rpy="0 0 0" />
-      </xacro:box_inertia>
+      </xacro:box_inertial>
       <visual>
         <origin xyz="0 0 0.209" rpy="0 0 0" />

File: raw_description/urdf/vacuum_gripper/gripper.urdf.xacro (robot description, xacro)
@@ -6,5 +6,5 @@
   <xacro:property name="gripper_height" value="0.14"/>
   <xacro:property name="gripper_body_height" value="0.14"/>
-  <xacro:property name="radius" value="0.005"/>
+  <xacro:property name="gripper_radius" value="0.005"/>
   <xacro:macro name="vacuum_gripper" params="name parent *origin">
     <!-- joint between arm_ee_link and raw_boxgripper_link -->
@@ -12,21 +12,17 @@
         <insert_block name="origin" />
         <parent link="${parent}" />
-        <child link="gripper_frame" />
+        <child link="${name}_frame" />
     </joint>
-    <link name="gripper_frame"/>
+    <link name="${name}_frame"/>
     <joint name="gripper_to_palm" type="fixed">
-        <parent link="gripper_frame"/>
-        <child link="gripper_body"/>
+        <parent link="${name}_frame"/>
+        <child link="${name}_body"/>
         <origin xyz="0.08015 0.0475 0.0" rpy="1.57079632679 0 3.1415"/>
     </joint>
-    <link name="gripper_body">
+    <link name="${name}_body">
         <visual>
-            <!--origin xyz="0 0.036 -0.0473" rpy="0 0 0"/-->
-              <!--geometry>
-                <box size="${gripper_length} ${gripper_width} ${gripper_height}"/>
-              </geometry-->
             <origin xyz="0 0 -0.048" rpy="0 0 0"/>
             <geometry>
-                <mesh filename="package://raw_description/meshes/vacuum_gripper/segmentgreifer_2.stl" />
+                <mesh filename="package://raw_description/meshes/vacuum_gripper/vacuum_gripper.stl" />
             </geometry>
             <material name="silver">
@@ -37,7 +33,7 @@
             <origin xyz="0 0.03 -0.05"/>
             <geometry>
-                <box size="${gripper_length} ${gripper_width} ${gripper_height}"/>
+                <mesh filename="package://raw_description/meshes/vacuum_gripper/vacuum_gripper.stl" />
             </geometry>
-            <material name="another_blue2">
+            <material name="blue">
                 <color rgba="0.38 0.54 0.83 1"/>
             </material>
@@ -45,22 +41,20 @@
     </link>
     <joint name="gripper_to_tcp" type="fixed">
-        <parent link="gripper_frame"/>
-        <child link="gripper"/>
+        <parent link="${name}_frame"/>
+        <child link="${name}"/>
         <origin xyz=" 0.1263 0.0 0.0" rpy="0 0 0"/>
     </joint>
-    <link name="gripper">
-      <visual>
-        <geometry>
-            <sphere radius="0.005"/>
-        </geometry>
-        <material name="white">
-            <color rgba="1 1 1 0.5"/>
-        </material>
-      </visual>
-      <collision>
-        <geometry>
-            <mesh filename="package://cob_description/meshes/unit_sphere.stl" scale="${radius} ${radius} ${radius}"/>
-        </geometry>
-      </collision>
+    <link name="${name}">
+        <visual>
+            <xacro:macro name="sphere_geometry" radius="${gripper_radius}">
+            </xacro:macro>
+            <material name="white">
+                <color rgba="1 1 1 0.5"/>
+            </material>
+        </visual>
+          <collision>
+              <xacro:macro name="sphere_geometry" radius="${gripper_radius}">
+              </xacro:macro>
+          </collision>
      </link>
     <!-- extensions -->

Commit message: finalizing

File: raw_description/urdf/base_long/base.urdf.xacro (robot description, xacro)
@@ -34,5 +34,5 @@
     <link name="${name}_battery">
       <xacro:box_inertial x="${battery_size_x}" y="${battery_size_y}" z="${battery_size_z}" mass="${battery_mass}">
-        <origin xyz="0.0 0.0 0.0" rpy="0 0 0" />
+        <origin xyz="0 0 0" rpy="0 0 0"/>
       </xacro:box_inertial>
       <visual>
@@ -63,5 +63,5 @@
     <link name="${name}_link">
       <xacro:box_inertial x="1.04" y="0.58" z="0.12" mass="${base_mass}">
-        <origin xyz="0.0 0.0 0.0" rpy="0 0 0" />
+        <origin xyz="0 0 0" rpy="0 0 0"/>
       </xacro:box_inertial>
       <visual>

File: raw_description/urdf/vacuum_gripper/gripper.urdf.xacro (robot description, xacro)
@@ -1,6 +1,6 @@
 <?xml version="1.0"?>
 <robot xmlns:xacro="http://www.ros.org/wiki/xacro">
+  <xacro:include filename="$(find cob_description)/urdf/common.xacro"/>
   <xacro:include filename="$(find raw_description)/urdf/vacuum_gripper/gripper.gazebo.xacro" />
-  <xacro:include filename="$(find cob_description)/urdf/common.xacro"/>
   <xacro:property name="gripper_length" value="0.14"/>
   <xacro:property name="gripper_width" value="0.2"/>
@@ -9,9 +9,9 @@
   <xacro:property name="gripper_radius" value="0.005"/>
   <xacro:macro name="vacuum_gripper" params="name parent *origin">
-    <!-- joint between arm_ee_link and raw_boxgripper_link -->
-    <joint name="${name}_base_joint" type="fixed" >
-        <insert_block name="origin" />
-        <parent link="${parent}" />
-        <child link="${name}_frame" />
+    <!-- joint between arm_ee_link and vacuum_gripper_link -->
+    <joint name="${name}_base_joint" type="fixed">
+        <xacro:insert_block name="origin"/>
+        <parent link="${parent}"/>
+        <child link="${name}_frame"/>
     </joint>
     <link name="${name}_frame"/>
@@ -25,5 +25,5 @@
             <origin xyz="0 0 -0.048" rpy="0 0 0"/>
             <geometry>
-                <mesh filename="package://raw_description/meshes/vacuum_gripper/vacuum_gripper.stl" />
+                <mesh filename="package://raw_description/meshes/vacuum_gripper/vacuum_gripper.stl"/>
             </geometry>
             <material name="silver">
@@ -32,11 +32,8 @@
         </visual>
         <collision>
-            <origin xyz="0 0.0 -0.048"/>
+            <origin xyz="0 0 -0.048" rpy="0 0 0"/>
             <geometry>
-                <mesh filename="package://raw_description/meshes/vacuum_gripper/vacuum_gripper.stl" />
+                <mesh filename="package://raw_description/meshes/vacuum_gripper/vacuum_gripper.stl"/>
             </geometry>
-            <material name="red">
-                <color rgba="0.38 0.54 0.83 1"/>
-            </material>
         </collision>
     </link>
@@ -48,17 +45,15 @@
     <link name="${name}">
         <visual>
-            <xacro:sphere_geometry radius="${gripper_radius}">
-            </xacro:sphere_geometry>
+            <xacro:sphere_geometry radius="${gripper_radius}"/>
             <material name="white">
                 <color rgba="1 1 1 0.5"/>
             </material>
         </visual>
-          <collision>
-              <xacro:sphere_geometry radius="${gripper_radius}">
-              </xacro:sphere_geometry>
-          </collision>
+        <collision>
+            <xacro:sphere_geometry radius="${gripper_radius}"/>
+        </collision>
      </link>
     <!-- extensions -->
-    <xacro:vacuum_gripper_gazebo name="${name}" />
+    <xacro:vacuum_gripper_gazebo name="${name}"/>
   </xacro:macro>
 </robot>

Commit message: fix the wheel radius to meet with the actual hardware radii

File: raw_description/urdf/base_long/base.urdf.xacro (robot description, xacro)
@@ -11,5 +11,5 @@
   <xacro:property name="caster_offset_y_fl" value="0.184" />
   <xacro:property name="caster_offset_y_fr" value="-0.134" />
-  <xacro:property name="caster_offset_z" value="0.09" />
+  <xacro:property name="caster_offset_z" value="0.08" />
   <xacro:property name="battery_offset_x_f" value="0.141" />
   <xacro:property name="battery_offset_x_r" value="0.139" />

File: raw_description/urdf/base_short/base.urdf.xacro (robot description, xacro)
@@ -11,5 +11,5 @@
   <xacro:property name="caster_offset_y_fl" value="0.184" />
   <xacro:property name="caster_offset_y_fr" value="-0.134" />
-  <xacro:property name="caster_offset_z" value="0.09" />
+  <xacro:property name="caster_offset_z" value="0.08" />
   <xacro:property name="battery_offset_x" value="0.0" />
   <xacro:property name="battery_offset_y" value="-0.008" />

Commit message: Updated stuff for raw3-1 and ipp.

File: raw_description/urdf/base_long/base.urdf.xacro (robot description, xacro)
@@ -22,4 +22,5 @@
   <xacro:property name="battery_size_y" value="0.148" />
   <xacro:property name="battery_size_z" value="0.26" />
+  <xacro:arg name="robot_namespace" default="" />
   <!-- battery macros-->
   <xacro:macro name="cob_batteries" params="name parent *origin ">
@@ -71,6 +72,6 @@
         <origin xyz="0 0 0.209" rpy="0 0 0" />
         <geometry>
-          <mesh filename="package://raw_description/meshes/base/raw_base_long.stl"/>
-          <!--box size="1.04 0.58 0.31" /-->
+          <!--<mesh filename="package://raw_description/meshes/base/raw_base_long.stl"/>-->
+          <box size="0.93 0.49 0.31" />
         </geometry>
       </collision>
@@ -102,5 +103,5 @@
     <gazebo>
       <plugin name="ros_control" filename="libhwi_switch_gazebo_ros_control.so">
-        <robotNamespace>${name}</robotNamespace>
+        <robotNamespace>$(arg robot_namespace)/${name}</robotNamespace>
         <filterJointsParam>joint_names</filterJointsParam>
       </plugin>
