Commit message: Changed base back to stl

File: raw_description/urdf/base_long/base.urdf.xacro (robot description, xacro)
@@ -72,6 +72,6 @@
         <origin xyz="0 0 0.209" rpy="0 0 0" />
         <geometry>
-          <!--<mesh filename="package://raw_description/meshes/base/raw_base_long.stl"/>-->
-          <box size="0.93 0.49 0.31" />
+          <mesh filename="package://raw_description/meshes/base/raw_base_long.stl"/>
+          <!--<box size="0.93 0.49 0.31" />-->
         </geometry>
       </collision>

File: raw_description/urdf/base_short/base.urdf.xacro (robot description, xacro)
@@ -70,6 +70,6 @@
         <origin xyz="0 0 0.209" rpy="0 0 0" />
         <geometry>
-          <!-- <mesh filename="package://raw_description/meshes/base/raw_base_short.dae"/> -->
-          <box size="0.688 0.503 0.096"/>
+          <mesh filename="package://raw_description/meshes/base/raw_base_short.dae"/>
+          <!--<box size="0.688 0.503 0.096"/>-->
         </geometry>
       </visual>
@@ -77,6 +77,6 @@
         <origin xyz="0 0 0.209" rpy="0 0 0" />
         <geometry>
-          <!-- <mesh filename="package://raw_description/meshes/base/raw_base_short.stl"/> -->
-          <box size="0.678 0.493 0.096"/>
+          <mesh filename="package://raw_description/meshes/base/raw_base_short.stl"/>
+          <!--<box size="0.678 0.493 0.096"/>-->
         </geometry>
       </collision>
