Commit message: raise effort limit. fixes https://github.com/ipa320/cob_robots/issues/641

File: cob_description/urdf/drive_wheel/drive_wheel.urdf.xacro (robot description, xacro)
@@ -13,5 +13,5 @@
       <axis xyz="0 1 0" />
       <safety_controller  k_velocity="10" />
-      <limit effort="0" velocity="${drive_vel}"/>
+      <limit effort="100" velocity="${drive_vel}"/>
       <dynamics damping="0.0" friction="0.0" />
     </joint>
@@ -46,5 +46,5 @@
       <axis xyz="0 0 1" />
       <safety_controller  k_velocity="10" />
-      <limit effort="0" velocity="${steer_vel}"/>
+      <limit effort="100" velocity="${steer_vel}"/>
       <dynamics damping="0.0" friction="0.0" />
     </joint>

Commit message: gripper joint defined as prismatic

File: cob_description/urdf/drive_wheel/drive_wheel.urdf.xacro (robot description, xacro)
@@ -6,5 +6,5 @@
   <xacro:property name="caster_mass" value="5.9" />
   <xacro:property name="wheel_mass" value="0.44036" />
-  <xacro:macro name="cob_wheel" params="parent suffix reflect drive_vel:=^">
+  <xacro:macro name="cob_wheel" params="parent suffix reflect drive_vel:=1.0">
     <joint name="${parent}_${suffix}_wheel_joint" type="continuous">
       <origin xyz="0 ${reflect*caster_wheel_offset_y} 0" rpy="0 0 0" />
@@ -39,5 +39,5 @@
   </xacro:macro>
   <!-- Macro for Caster hub only -->
-  <xacro:macro name="cob_caster_hub" params="*origin parent suffix steer_vel:=^" >
+  <xacro:macro name="cob_caster_hub" params="*origin parent suffix steer_vel:=1.0" >
     <joint name="${suffix}_rotation_joint" type="continuous">
       <xacro:insert_block name="origin" />
@@ -71,5 +71,5 @@
     <xacro:cob_caster_transmission suffix="${suffix}" />
   </xacro:macro>
-  <xacro:macro name="drive_wheel" params="*origin parent suffix drive_vel:=^|100 steer_vel:=^|100">
+  <xacro:macro name="drive_wheel" params="*origin parent suffix drive_vel:=100.0 steer_vel:=100.0">
     <xacro:cob_caster_hub parent="${parent}" suffix="${suffix}_caster" >
       <xacro:insert_block name="origin" />

File: raw_description/urdf/vacuum_gripper/gripper.urdf.xacro (robot description, xacro)
@@ -52,11 +52,11 @@
       </xacro:cylinder_inertial>
     </link>
-    <joint name="gripper_to_tcp" type="revolute">
+    <joint name="gripper_to_tcp" type="prismatic">
         <parent link="${name}_frame"/>
         <child link="${name}"/>
         <origin xyz=" 0.1263 0.0 0.0" rpy="0 0 0"/>
         <axis xyz="0 1 0" />
-        <limit lower="${-2.0 * pi}" upper="${2.0 * pi}" effort="54.0" velocity="3.2"/>
-        <dynamics damping="0.0" friction="0.0"/>
+        <limit lower="0.001" upper="0.001" effort="54.0" velocity="0.01"/>
+        <dynamics damping="0.0" friction="10.0"/>
     </joint>
     <link name="${name}">
@@ -64,5 +64,5 @@
             <xacro:sphere_geometry radius="${gripper_radius}"/>
             <material name="white">
-                <color rgba="1 1 1 0.5"/>
+                <color rgba="1 1 1 1"/>
             </material>
         </visual>

Commit message: correct file name upload of gripper transmission

File: cob_description/urdf/drive_wheel/drive_wheel.urdf.xacro (robot description, xacro)
@@ -6,5 +6,5 @@
   <xacro:property name="caster_mass" value="5.9" />
   <xacro:property name="wheel_mass" value="0.44036" />
-  <xacro:macro name="cob_wheel" params="parent suffix reflect drive_vel:=1.0">
+  <xacro:macro name="cob_wheel" params="parent suffix reflect drive_vel:=^">
     <joint name="${parent}_${suffix}_wheel_joint" type="continuous">
       <origin xyz="0 ${reflect*caster_wheel_offset_y} 0" rpy="0 0 0" />
@@ -39,5 +39,5 @@
   </xacro:macro>
   <!-- Macro for Caster hub only -->
-  <xacro:macro name="cob_caster_hub" params="*origin parent suffix steer_vel:=1.0" >
+  <xacro:macro name="cob_caster_hub" params="*origin parent suffix steer_vel:=^" >
     <joint name="${suffix}_rotation_joint" type="continuous">
       <xacro:insert_block name="origin" />
@@ -71,5 +71,5 @@
     <xacro:cob_caster_transmission suffix="${suffix}" />
   </xacro:macro>
-  <xacro:macro name="drive_wheel" params="*origin parent suffix drive_vel:=100.0 steer_vel:=100.0">
+  <xacro:macro name="drive_wheel" params="*origin parent suffix drive_vel:=^|100 steer_vel:=^|100">
     <xacro:cob_caster_hub parent="${parent}" suffix="${suffix}_caster" >
       <xacro:insert_block name="origin" />

File: raw_description/urdf/vacuum_gripper/gripper.gazebo.xacro (robot description, xacro)
@@ -9,5 +9,5 @@
         <contact>
           <collision>${name}_collision</collision>
-          <topic>${name}_bumper</topic>
+            <topic>${name}_bumper</topic>
         </contact>
         <plugin name="${name}_gazebo_ros_bumper_controller" filename="libgazebo_ros_bumper.so">

File: raw_description/urdf/vacuum_gripper/gripper.transmission.xacro (robot description, xacro)
@@ -1,15 +1,15 @@
 <?xml version="1.0"?>
 <robot xmlns:xacro="http://ros.org/wiki/xacro">
-    <xacro:macro name="vacuum_gripper_transmission" params="name">
-        <transmission name="${name}_base_trans">
-            <type>transmission_interface/SimpleTransmission</type>
-            <joint name="${name}_base_joint">
-                <hardwareInterface>PositionJointInterface</hardwareInterface>
-                <hardwareInterface>VelocityJointInterface</hardwareInterface>
-            </joint>
-            <actuator name="${name}_base_motor">
-                <mechanicalReduction>1</mechanicalReduction>
-            </actuator>
-        </transmission>
-    </xacro:macro>
+  <xacro:macro name="vacuum_gripper_transmission" params="name">
+    <transmission name="${name}_base_trans">
+      <type>transmission_interface/SimpleTransmission</type>
+      <joint name="${name}_base_joint">
+        <hardwareInterface>PositionJointInterface</hardwareInterface>
+        <hardwareInterface>VelocityJointInterface</hardwareInterface>
+      </joint>
+      <actuator name="${name}_base_motor">
+        <mechanicalReduction>1</mechanicalReduction>
+      </actuator>
+    </transmission>
+  </xacro:macro>
 </robot>

File: raw_description/urdf/vacuum_gripper/gripper.urdf.xacro (robot description, xacro)
@@ -2,5 +2,5 @@
 <robot xmlns:xacro="http://www.ros.org/wiki/xacro">
   <xacro:include filename="$(find cob_description)/urdf/common.xacro"/>
-  <xacro:include filename="$(find raw_description)/urdf/vacuum_gripper/vacuum_gripper.transmission.xacro" />
+  <xacro:include filename="$(find raw_description)/urdf/vacuum_gripper/gripper.transmission.xacro" />
   <xacro:include filename="$(find raw_description)/urdf/vacuum_gripper/gripper.gazebo.xacro" />
   <xacro:property name="gripper_length" value="0.14"/>
@@ -10,71 +10,71 @@
   <xacro:property name="gripper_radius" value="0.01"/>
   <xacro:macro name="vacuum_gripper" params="name parent *origin">
-    <!-- joint between arm_ee_link and vacuum_gripper_link -->
-    <joint name="${name}_base_joint" type="fixed">
-        <xacro:insert_block name="origin"/>
-        <parent link="${parent}"/>
-        <child link="${name}_frame"/>
-    </joint>
-    <link name="${name}_frame">
-        <collision>
-            <geometry>
-                <box size="0.01 0.01 0.01"/>
-            </geometry>
-            <origin rpy="0 0 0" xyz="-0.01 0 0"/>
-        </collision>
-        <xacro:cylinder_inertial radius="0.075" length="0.12" mass="0.01">
-            <origin xyz="0.0 0.0 0.0" rpy="0 0 0" />
-        </xacro:cylinder_inertial>
-    </link>
-    <joint name="gripper_to_palm" type="fixed">
-        <parent link="${name}_frame"/>
-        <child link="${name}_body"/>
-        <origin xyz="0.08015 0.0475 0.0" rpy="1.57079632679 0 3.1415"/>
-    </joint>
-    <link name="${name}_body">
-        <visual>
-            <origin xyz="0 0 -0.048" rpy="0 0 0"/>
-            <geometry>
-                <mesh filename="package://raw_description/meshes/vacuum_gripper/vacuum_gripper.stl"/>
-            </geometry>
-            <material name="silver">
-                <color rgba="0.8 0.8 0.8 1"/>
-            </material>
-        </visual>
-        <collision>
-            <origin xyz="0 0 -0.048" rpy="0 0 0"/>
-            <geometry>
-                <mesh filename="package://raw_description/meshes/vacuum_gripper/vacuum_gripper.stl"/>
-            </geometry>
-        </collision>
-        <xacro:cylinder_inertial radius="0.075" length="0.12" mass="0.01">
-            <origin xyz="0.0 0.0 0.0" rpy="0 0 0" />
-        </xacro:cylinder_inertial>
-    </link>
-    <joint name="gripper_to_tcp" type="prismatic">
-        <parent link="${name}_frame"/>
-        <child link="${name}"/>
-        <origin xyz=" 0.1263 0.0 0.0" rpy="0 0 0"/>
-        <axis xyz="0 1 0" />
-        <limit lower="0.001" upper="0.001" effort="54.0" velocity="0.01"/>
-        <dynamics damping="0.0" friction="10.0"/>
-    </joint>
-    <link name="${name}">
-        <visual>
-            <xacro:sphere_geometry radius="${gripper_radius}"/>
-            <material name="white">
-                <color rgba="1 1 1 1"/>
-            </material>
-        </visual>
-        <collision>
-            <xacro:sphere_geometry radius="${gripper_radius}"/>
-        </collision>
-        <xacro:cylinder_inertial radius="0.075" length="0.12" mass="0.1">
-            <origin xyz="0.0 0.0 0.0" rpy="0 0 0" />
-      </xacro:cylinder_inertial>
-     </link>
-    <!-- extensions -->
-    <xacro:vacuum_gripper_transmission name="${name}"/>
-    <xacro:vacuum_gripper_gazebo name="${name}"/>
+  <!-- joint between arm_ee_link and vacuum_gripper_link -->
+  <joint name="${name}_base_joint" type="fixed">
+    <xacro:insert_block name="origin"/>
+    <parent link="${parent}"/>
+    <child link="${name}_frame"/>
+  </joint>
+  <link name="${name}_frame">
+    <collision>
+      <geometry>
+        <box size="0.01 0.01 0.01"/>
+      </geometry>
+      <origin rpy="0 0 0" xyz="-0.01 0 0"/>
+    </collision>
+    <xacro:cylinder_inertial radius="0.075" length="0.12" mass="0.01">
+      <origin xyz="0.0 0.0 0.0" rpy="0 0 0" />
+    </xacro:cylinder_inertial>
+  </link>
+  <joint name="gripper_to_palm" type="fixed">
+    <parent link="${name}_frame"/>
+    <child link="${name}_body"/>
+    <origin xyz="0.08015 0.0475 0.0" rpy="1.57079632679 0 3.1415"/>
+  </joint>
+  <link name="${name}_body">
+    <visual>
+      <origin xyz="0 0 -0.048" rpy="0 0 0"/>
+      <geometry>
+        <mesh filename="package://raw_description/meshes/vacuum_gripper/vacuum_gripper.stl"/>
+      </geometry>
+      <material name="silver">
+        <color rgba="0.8 0.8 0.8 1"/>
+      </material>
+    </visual>
+    <collision>
+      <origin xyz="0 0 -0.048" rpy="0 0 0"/>
+      <geometry>
+        <mesh filename="package://raw_description/meshes/vacuum_gripper/vacuum_gripper.stl"/>
+      </geometry>
+    </collision>
+    <xacro:cylinder_inertial radius="0.075" length="0.12" mass="0.01">
+      <origin xyz="0.0 0.0 0.0" rpy="0 0 0" />
+    </xacro:cylinder_inertial>
+  </link>
+  <joint name="gripper_to_tcp" type="prismatic">
+    <parent link="${name}_frame"/>
+    <child link="${name}"/>
+    <origin xyz=" 0.1263 0.0 0.0" rpy="0 0 0"/>
+    <axis xyz="0 1 0" />
+    <limit lower="0.001" upper="0.001" effort="54.0" velocity="0.01"/>
+    <dynamics damping="0.0" friction="10.0"/>
+  </joint>
+  <link name="${name}">
+    <visual>
+      <xacro:sphere_geometry radius="${gripper_radius}"/>
+      <material name="white">
+        <color rgba="1 1 1 1"/>
+      </material>
+    </visual>
+    <collision>
+      <xacro:sphere_geometry radius="${gripper_radius}"/>
+    </collision>
+    <xacro:cylinder_inertial radius="0.075" length="0.12" mass="0.1">
+      <origin xyz="0.0 0.0 0.0" rpy="0 0 0" />
+    </xacro:cylinder_inertial>
+  </link>
+  <!-- extensions -->
+  <xacro:vacuum_gripper_transmission name="${name}"/>
+  <xacro:vacuum_gripper_gazebo name="${name}"/>
   </xacro:macro>
 </robot>
