Commit message: test_bumper_contact_sensor

File: raw_description/urdf/vacuum_gripper/gripper.gazebo.xacro (robot description, xacro)
@@ -2,7 +2,19 @@
 <robot xmlns:xacro="http://www.ros.org/wiki/xacro">
   <xacro:macro name="vacuum_gripper_gazebo" params="name">
-    <gazebo reference="${name}_ee_link">
+	<gazebo reference="${name}">
       <gravity>true</gravity>
       <self_collide>false</self_collide>
+      <sensor name='${name}_contact_sensor' type='contact'>
+        <always_on>true</always_on>
+        <update_rate>100.0</update_rate>
+        <contact>
+          <collision>${name}_link_collision</collision>
+          <topic>${name}_bumper</topic>
+        </contact>
+        <plugin name="${name}_gazebo_ros_bumper_controller" filename="libgazebo_ros_bumper.so">
+          <frameName>world</frameName>
+          <bumperTopicName>${name}_bumper</bumperTopicName>
+        </plugin>
+      </sensor>
     </gazebo>
   </xacro:macro>

Commit message: update bumper sensor

File: raw_description/urdf/vacuum_gripper/gripper.gazebo.xacro (robot description, xacro)
@@ -2,19 +2,30 @@
 <robot xmlns:xacro="http://www.ros.org/wiki/xacro">
   <xacro:macro name="vacuum_gripper_gazebo" params="name">
-	<gazebo reference="${name}">
+	<gazebo reference="${name}_body">
       <gravity>true</gravity>
       <self_collide>false</self_collide>
       <sensor name='${name}_contact_sensor' type='contact'>
         <always_on>true</always_on>
-        <update_rate>100.0</update_rate>
+        <update_rate>10.0</update_rate>
         <contact>
-          <collision>${name}_link_collision</collision>
+          <collision>${name}_body</collision>
           <topic>${name}_bumper</topic>
         </contact>
         <plugin name="${name}_gazebo_ros_bumper_controller" filename="libgazebo_ros_bumper.so">
+          <alwaysOn>true</alwaysOn>
           <frameName>world</frameName>
           <bumperTopicName>${name}_bumper</bumperTopicName>
         </plugin>
       </sensor>
+      <mu1 value="500.0" />
+      <mu2 value="500.0" />
+      <kp  value="10000000.0" />
+      <kd  value="1.0" />
+    </gazebo>
+    <gazebo reference="gripper_to_tcp">
+      <stopKd value="1.0" />
+      <stopKp value="10000000.0" />
+      <fudgeFactor value="1.0" />
+      <provideFeedback value="true"/>
     </gazebo>
   </xacro:macro>

File: raw_description/urdf/vacuum_gripper/gripper.urdf.xacro (robot description, xacro)
@@ -22,4 +22,11 @@
     </joint>
     <link name="${name}_body">
+      	<inertial>
+            <mass value="0.04419" />
+            <origin xyz="0.00423 0.00284 0.0" rpy="0 0 0" />
+            <inertia  ixx="0.00000837047" ixy="0.00000583632" ixz="0.0"
+                      iyy="0.00000987067" iyz="0.0"
+                      izz="0.00001541768" />
+      	</inertial>
         <visual>
             <origin xyz="0 0 -0.048" rpy="0 0 0"/>

Commit message: gripper sensor working but the data is not good

File: raw_description/urdf/vacuum_gripper/gripper.gazebo.xacro (robot description, xacro)
@@ -2,16 +2,16 @@
 <robot xmlns:xacro="http://www.ros.org/wiki/xacro">
   <xacro:macro name="vacuum_gripper_gazebo" params="name">
-    <gazebo reference="${name}_frame">
+    <gazebo reference="${name}">
       <self_collide>false</self_collide>
-      <sensor name='${name}_frame_sensor' type='contact'>
+      <sensor name='${name}_sensor' type='contact'>
         <always_on>true</always_on>
         <update_rate>100.0</update_rate>
         <contact>
-          <collision>${name}_frame_collision</collision>
-          <topic>$test_bumper</topic>
+          <collision>${name}_collision</collision>
+          <topic>${name}_bumper</topic>
         </contact>
-        <plugin name="${name}_frame_gazebo_ros_bumper_controller" filename="libgazebo_ros_bumper.so">
-          <bodyName>${name}_frame</bodyName>
-          <bumperTopicName>test_bumper</bumperTopicName>
+        <plugin name="${name}_gazebo_ros_bumper_controller" filename="libgazebo_ros_bumper.so">
+          <frameName>${name}</frameName>
+          <bumperTopicName>${name}_bumper</bumperTopicName>
         </plugin>
       </sensor>

File: raw_description/urdf/vacuum_gripper/gripper.urdf.xacro (robot description, xacro)
@@ -2,4 +2,5 @@
 <robot xmlns:xacro="http://www.ros.org/wiki/xacro">
   <xacro:include filename="$(find cob_description)/urdf/common.xacro"/>
+  <xacro:include filename="$(find raw_description)/urdf/vacuum_gripper/vacuum_gripper.transmission.xacro" />
   <xacro:include filename="$(find raw_description)/urdf/vacuum_gripper/gripper.gazebo.xacro" />
   <xacro:property name="gripper_length" value="0.14"/>
@@ -10,11 +11,8 @@
   <xacro:macro name="vacuum_gripper" params="name parent *origin">
     <!-- joint between arm_ee_link and vacuum_gripper_link -->
-    <joint name="${name}_base_joint" type="revolute">
+    <joint name="${name}_base_joint" type="fixed">
         <xacro:insert_block name="origin"/>
         <parent link="${parent}"/>
         <child link="${name}_frame"/>
-        <axis xyz="0 1 0" />
-        <limit lower="${-2.0 * pi}" upper="${2.0 * pi}" effort="54.0" velocity="3.2"/>
-        <dynamics damping="0.0" friction="0.0"/>
     </joint>
     <link name="${name}_frame">
@@ -25,4 +23,7 @@
         <origin rpy="0 0 0" xyz="-0.01 0 0"/>
       </collision>
+      <xacro:cylinder_inertial radius="0.075" length="0.12" mass="0.01">
+        <origin xyz="0.0 0.0 0.0" rpy="0 0 0" />
+      </xacro:cylinder_inertial>
     </link>
     <joint name="gripper_to_palm" type="fixed">
@@ -47,9 +48,15 @@
             </geometry>
         </collision>
+      <xacro:cylinder_inertial radius="0.075" length="0.12" mass="0.01">
+        <origin xyz="0.0 0.0 0.0" rpy="0 0 0" />
+      </xacro:cylinder_inertial>
     </link>
-    <joint name="gripper_to_tcp" type="fixed">
+    <joint name="gripper_to_tcp" type="revolute">
         <parent link="${name}_frame"/>
         <child link="${name}"/>
         <origin xyz=" 0.1263 0.0 0.0" rpy="0 0 0"/>
+        <axis xyz="0 1 0" />
+        <limit lower="${-2.0 * pi}" upper="${2.0 * pi}" effort="54.0" velocity="3.2"/>
+        <dynamics damping="0.0" friction="0.0"/>
     </joint>
     <link name="${name}">
@@ -63,6 +70,10 @@
             <xacro:sphere_geometry radius="${gripper_radius}"/>
         </collision>
+        <xacro:cylinder_inertial radius="0.075" length="0.12" mass="0.1">
+          <origin xyz="0.0 0.0 0.0" rpy="0 0 0" />
+        </xacro:cylinder_inertial>
      </link>
     <!-- extensions -->
+    <xacro:vacuum_gripper_transmission name="${name}"/>
     <xacro:vacuum_gripper_gazebo name="${name}"/>
   </xacro:macro>

Commit message: attach bumper sensor to tool0 frame

File: raw_description/urdf/vacuum_gripper/gripper.gazebo.xacro (robot description, xacro)
@@ -2,16 +2,16 @@
 <robot xmlns:xacro="http://www.ros.org/wiki/xacro">
   <xacro:macro name="vacuum_gripper_gazebo" params="name">
-    <gazebo reference="${name}">
+    <gazebo reference="arm_tool0">
       <self_collide>false</self_collide>
-      <sensor name='${name}_sensor' type='contact'>
+      <sensor name='arm_tool0_sensor' type='contact'>
         <always_on>true</always_on>
         <update_rate>100.0</update_rate>
         <contact>
-          <collision>${name}_collision</collision>
-            <topic>${name}_bumper</topic>
+          <collision>arm_tool0_collision</collision>
+            <topic>arm_tool0_bumper</topic>
         </contact>
-        <plugin name="${name}_gazebo_ros_bumper_controller" filename="libgazebo_ros_bumper.so">
-          <frameName>${name}</frameName>
-          <bumperTopicName>${name}_bumper</bumperTopicName>
+        <plugin name="arm_tool0_gazebo_ros_bumper_controller" filename="libgazebo_ros_bumper.so">
+          <frameName>arm_tool0</frameName>
+          <bumperTopicName>arm_tool0_bumper</bumperTopicName>
         </plugin>
       </sensor>

File: raw_description/urdf/vacuum_gripper/gripper.urdf.xacro (robot description, xacro)
@@ -9,5 +9,5 @@
   <xacro:property name="gripper_body_height" value="0.14"/>
   <xacro:property name="gripper_radius" value="0.01"/>
-  <xacro:macro name="vacuum_gripper" params="name parent *origin">
+  <xacro:macro name="vacuum_gripper" params="name parent *origin sensor_frame">
   <!-- joint between arm_ee_link and vacuum_gripper_link -->
   <joint name="${name}_base_joint" type="fixed">
@@ -52,5 +52,5 @@
     </xacro:cylinder_inertial>
   </link>
-  <joint name="gripper_to_tcp" type="prismatic">
+  <joint name="gripper_to_tcp" type="fixed">
     <parent link="${name}_frame"/>
     <child link="${name}"/>
@@ -76,5 +76,5 @@
   <!-- extensions -->
   <xacro:vacuum_gripper_transmission name="${name}"/>
-  <xacro:vacuum_gripper_gazebo name="${name}"/>
+  <xacro:vacuum_gripper_gazebo name="${sensor_frame}"/>
   </xacro:macro>
 </robot>
