Commit message: New STL file for the vacuum gripper

File: raw_description/urdf/vacuum_gripper/gripper.urdf.xacro (robot description, xacro)
@@ -27,5 +27,5 @@
 				<origin xyz="0 0 -0.048" rpy="0 0 0"/>
 				<geometry>
-					<mesh filename="package://raw_description/meshes/vacuum_gripper/vacuum_gripper_single_suction_cup.STL" />
+					<mesh filename="package://raw_description/meshes/vacuum_gripper/Segmentgreifer.STL" />
 				</geometry>
 				<material name="silver">

Commit message: Vacuum Gripper file description updated

File: raw_description/urdf/vacuum_gripper/gripper.urdf.xacro (robot description, xacro)
@@ -17,5 +17,5 @@
 		<parent link="${prefix}gripper_frame"/>
 		<child link="${prefix}gripper_body"/>
-		<origin xyz="0 0 ${gripper_height * 0.5}" rpy="0 0 0"/>
+		<origin xyz="0.08015 0.0475 0.0" rpy="1.57079632679 0 3.1415"/>
 	</joint>
     <link name="${prefix}gripper_body">
@@ -27,5 +27,5 @@
 				<origin xyz="0 0 -0.048" rpy="0 0 0"/>
 				<geometry>
-					<mesh filename="package://raw_description/meshes/vacuum_gripper/Segmentgreifer.STL" />
+					<mesh filename="package://raw_description/meshes/vacuum_gripper/Segmentgreifer_2.STL" />
 				</geometry>
 				<material name="silver">

Commit message: requested changes

File: raw_description/urdf/vacuum_gripper/gripper.urdf.xacro (robot description, xacro)
@@ -9,58 +9,58 @@
     <!-- joint between arm_ee_link and raw_boxgripper_link -->
     <joint name="${name}_base_joint" type="fixed" >
-      <insert_block name="origin" />
-      <parent link="${parent}" />
-      <child link="${prefix}gripper_frame" />
+        <insert_block name="origin" />
+        <parent link="${parent}" />
+        <child link="${prefix}gripper_frame" />
     </joint>
     <link name="${prefix}gripper_frame"/>
     <joint name="${prefix}gripper_to_palm" type="fixed">
-		<parent link="${prefix}gripper_frame"/>
-		<child link="${prefix}gripper_body"/>
-		<origin xyz="0.08015 0.0475 0.0" rpy="1.57079632679 0 3.1415"/>
-	</joint>
+        <parent link="${prefix}gripper_frame"/>
+        <child link="${prefix}gripper_body"/>
+        <origin xyz="0.08015 0.0475 0.0" rpy="1.57079632679 0 3.1415"/>
+    </joint>
     <link name="${prefix}gripper_body">
-			<visual>
-				<!--origin xyz="0 0.036 -0.0473" rpy="0 0 0"/-->
-				<!--geometry>
-					<box size="${gripper_length} ${gripper_width} ${gripper_height}"/>
-				</geometry-->
-				<origin xyz="0 0 -0.048" rpy="0 0 0"/>
-				<geometry>
-					<mesh filename="package://raw_description/meshes/vacuum_gripper/Segmentgreifer_2.STL" />
-				</geometry>
-				<material name="silver">
-					<color rgba="0.8 0.8 0.8 1"/>
-				</material>
-			</visual>
-			<collision>
-				<origin xyz="0 0.03 -0.05"/>
-				<geometry>
-					<box size="0.13 0.17 0.11"/>
-				</geometry>
-				<material name="another_blue2">
-					<color rgba="0.38 0.54 0.83 1"/>
-				</material>
-			</collision>
-	</link>
-	<joint name="${prefix}gripper_to_tcp" type="fixed">
-			<parent link="${prefix}gripper_frame"/>
-			<child link="gripper"/>
-			<origin xyz=" 0.1263 0.0 0.0" rpy="0 0 0"/>
-	</joint>
-	<link name="gripper">
-		<visual>
-			<geometry>
-				<sphere radius="0.005"/>
-			</geometry>
-			<material name="white">
-				<color rgba="1 1 1 0.5"/>
-			</material>
-		</visual>
-		<collision>
-			<geometry>
-				<sphere radius="0.005"/>
-			</geometry>
-		</collision>
-	</link>
+        <visual>
+            <!--origin xyz="0 0.036 -0.0473" rpy="0 0 0"/-->
+            <!--geometry>
+                <box size="${gripper_length} ${gripper_width} ${gripper_height}"/>
+            </geometry-->
+            <origin xyz="0 0 -0.048" rpy="0 0 0"/>
+            <geometry>
+                <mesh filename="package://raw_description/meshes/vacuum_gripper/Segmentgreifer_2.STL" />
+            </geometry>
+            <material name="silver">
+                <color rgba="0.8 0.8 0.8 1"/>
+            </material>
+        </visual>
+        <collision>
+            <origin xyz="0 0.03 -0.05"/>
+            <geometry>
+                <box size="0.13 0.17 0.11"/>
+            </geometry>
+            <material name="another_blue2">
+                <color rgba="0.38 0.54 0.83 1"/>
+            </material>
+        </collision>
+    </link>
+    <joint name="${prefix}gripper_to_tcp" type="fixed">
+        <parent link="${prefix}gripper_frame"/>
+        <child link="gripper"/>
+        <origin xyz=" 0.1263 0.0 0.0" rpy="0 0 0"/>
+    </joint>
+    <link name="gripper">
+      <visual>
+        <geometry>
+            <sphere radius="0.005"/>
+        </geometry>
+        <material name="white">
+            <color rgba="1 1 1 0.5"/>
+        </material>
+      </visual>
+      <collision>
+        <geometry>
+            <sphere radius="0.005"/>
+        </geometry>
+      </collision>
+     </link>
     <!-- extensions -->
     <xacro:vacuum_gripper_gazebo name="${name}" />

Commit message: tabs vs spaces solved

File: raw_description/urdf/vacuum_gripper/gripper.urdf.xacro (robot description, xacro)
@@ -22,7 +22,7 @@
         <visual>
             <!--origin xyz="0 0.036 -0.0473" rpy="0 0 0"/-->
-            <!--geometry>
+              <!--geometry>
                 <box size="${gripper_length} ${gripper_width} ${gripper_height}"/>
-            </geometry-->
+              </geometry-->
             <origin xyz="0 0 -0.048" rpy="0 0 0"/>
             <geometry>

Commit message: gripper macro name changed and prefix removed as argument

File: raw_description/urdf/vacuum_gripper/gripper.urdf.xacro (robot description, xacro)
@@ -6,18 +6,18 @@
   <xacro:property name="gripper_height" value="0.14"/>
   <xacro:property name="gripper_body_height" value="0.14"/>
-  <xacro:macro name="vacuum_gripper_definition" params="name parent *origin prefix">
+  <xacro:macro name="vacuum_gripper" params="name parent *origin">
     <!-- joint between arm_ee_link and raw_boxgripper_link -->
     <joint name="${name}_base_joint" type="fixed" >
         <insert_block name="origin" />
         <parent link="${parent}" />
-        <child link="${prefix}gripper_frame" />
+        <child link="gripper_frame" />
     </joint>
-    <link name="${prefix}gripper_frame"/>
-    <joint name="${prefix}gripper_to_palm" type="fixed">
-        <parent link="${prefix}gripper_frame"/>
-        <child link="${prefix}gripper_body"/>
+    <link name="gripper_frame"/>
+    <joint name="gripper_to_palm" type="fixed">
+        <parent link="gripper_frame"/>
+        <child link="gripper_body"/>
         <origin xyz="0.08015 0.0475 0.0" rpy="1.57079632679 0 3.1415"/>
     </joint>
-    <link name="${prefix}gripper_body">
+    <link name="gripper_body">
         <visual>
             <!--origin xyz="0 0.036 -0.0473" rpy="0 0 0"/-->
@@ -43,6 +43,6 @@
         </collision>
     </link>
-    <joint name="${prefix}gripper_to_tcp" type="fixed">
-        <parent link="${prefix}gripper_frame"/>
+    <joint name="gripper_to_tcp" type="fixed">
+        <parent link="gripper_frame"/>
         <child link="gripper"/>
         <origin xyz=" 0.1263 0.0 0.0" rpy="0 0 0"/>

Commit message: file name and suffix all small letters.

File: raw_description/urdf/vacuum_gripper/gripper.urdf.xacro (robot description, xacro)
@@ -27,5 +27,5 @@
             <origin xyz="0 0 -0.048" rpy="0 0 0"/>
             <geometry>
-                <mesh filename="package://raw_description/meshes/vacuum_gripper/Segmentgreifer_2.STL" />
+                <mesh filename="package://raw_description/meshes/vacuum_gripper/segmentgreifer_2.stl" />
             </geometry>
             <material name="silver">

Commit message: use the properties at the top for the collision properties

File: raw_description/urdf/vacuum_gripper/gripper.urdf.xacro (robot description, xacro)
@@ -36,5 +36,5 @@
             <origin xyz="0 0.03 -0.05"/>
             <geometry>
-                <box size="0.13 0.17 0.11"/>
+                <box size="${gripper_length} ${gripper_width} ${gripper_height}"/>
             </geometry>
             <material name="another_blue2">

Commit message: use scalable primitive meshes

File: raw_description/urdf/vacuum_gripper/gripper.urdf.xacro (robot description, xacro)
@@ -6,4 +6,5 @@
   <xacro:property name="gripper_height" value="0.14"/>
   <xacro:property name="gripper_body_height" value="0.14"/>
+  <xacro:property name="radius" value="0.005"/>
   <xacro:macro name="vacuum_gripper" params="name parent *origin">
     <!-- joint between arm_ee_link and raw_boxgripper_link -->
@@ -59,5 +60,5 @@
       <collision>
         <geometry>
-            <sphere radius="0.005"/>
+            <mesh filename="package://cob_description/meshes/unit_sphere.stl" scale="${radius} ${radius} ${radius}"/>
         </geometry>
       </collision>

Commit message: origin of the colision mesh corrected

File: raw_description/urdf/vacuum_gripper/gripper.urdf.xacro (robot description, xacro)
@@ -31,5 +31,5 @@
         </visual>
         <collision>
-            <origin xyz="0 0.03 -0.05"/>
+            <origin xyz="0 0.0 0.0"/>
             <geometry>
                 <mesh filename="package://raw_description/meshes/vacuum_gripper/vacuum_gripper.stl" />

Commit message: origin of the colision mesh corrected according with visual values

File: raw_description/urdf/vacuum_gripper/gripper.urdf.xacro (robot description, xacro)
@@ -31,5 +31,5 @@
         </visual>
         <collision>
-            <origin xyz="0 0.0 0.0"/>
+            <origin xyz="0 0.0 -0.048"/>
             <geometry>
                 <mesh filename="package://raw_description/meshes/vacuum_gripper/vacuum_gripper.stl" />

Commit message: changes acoording to pull request

File: raw_description/urdf/vacuum_gripper/gripper.urdf.xacro (robot description, xacro)
@@ -2,4 +2,5 @@
 <robot xmlns:xacro="http://www.ros.org/wiki/xacro">
   <xacro:include filename="$(find raw_description)/urdf/vacuum_gripper/gripper.gazebo.xacro" />
+  <xacro:include filename="$(find cob_description)/urdf/common.xacro"/>
   <xacro:property name="gripper_length" value="0.14"/>
   <xacro:property name="gripper_width" value="0.2"/>
@@ -35,5 +36,5 @@
                 <mesh filename="package://raw_description/meshes/vacuum_gripper/vacuum_gripper.stl" />
             </geometry>
-            <material name="blue">
+            <material name="red">
                 <color rgba="0.38 0.54 0.83 1"/>
             </material>
@@ -47,6 +48,6 @@
     <link name="${name}">
         <visual>
-            <xacro:macro name="sphere_geometry" radius="${gripper_radius}">
-            </xacro:macro>
+            <xacro:sphere_geometry radius="${gripper_radius}">
+            </xacro:sphere_geometry>
             <material name="white">
                 <color rgba="1 1 1 0.5"/>
@@ -54,6 +55,6 @@
         </visual>
           <collision>
-              <xacro:macro name="sphere_geometry" radius="${gripper_radius}">
-              </xacro:macro>
+              <xacro:sphere_geometry radius="${gripper_radius}">
+              </xacro:sphere_geometry>
           </collision>
      </link>

Commit message: contact sensor in gripper fixed

File: raw_description/urdf/vacuum_gripper/gripper.urdf.xacro (robot description, xacro)
@@ -8,5 +8,5 @@
   <xacro:property name="gripper_height" value="0.14"/>
   <xacro:property name="gripper_body_height" value="0.14"/>
-  <xacro:property name="gripper_radius" value="0.005"/>
+  <xacro:property name="gripper_radius" value="0.05"/>
   <xacro:macro name="vacuum_gripper" params="name parent *origin">
     <!-- joint between arm_ee_link and vacuum_gripper_link -->

Commit message: orient_gripper

File: raw_description/urdf/vacuum_gripper/gripper.urdf.xacro (robot description, xacro)
@@ -19,5 +19,5 @@
         <parent link="${name}_frame"/>
         <child link="${name}_body"/>
-        <origin xyz="0.08015 0.0475 0.0" rpy="1.57079632679 0 3.1415"/>
+        <origin xyz="0.08015 -0.0475 0.0" rpy="-1.57079632679 0 3.1415"/>
     </joint>
     <link name="${name}_body">
@@ -41,5 +41,5 @@
         <parent link="${name}_frame"/>
         <child link="${name}"/>
-        <origin xyz=" 0.1263 0.0 0.0" rpy="0 0 0"/>
+        <origin xyz=" 0.1263 0.0 0.0" rpy="3.1415 0 0"/>
     </joint>
     <link name="${name}">

Commit message: updated raw3-1 configuration

File: raw_description/urdf/vacuum_gripper/gripper.urdf.xacro (robot description, xacro)
@@ -32,7 +32,7 @@
         </visual>
         <collision>
-            <origin xyz="0.01 0.04 -0.048" rpy="0 0 0"/>
+            <origin xyz="0 0 -0.048" rpy="0 0 0"/>
             <geometry>
-                <box size="0.13 0.14 0.071"/>
+                <mesh filename="package://raw_description/meshes/vacuum_gripper/vacuum_gripper.stl"/>
             </geometry>
         </collision>

Commit message: add temporary goemetry and collision object for schmalz

File: raw_description/urdf/vacuum_gripper/gripper.urdf.xacro (robot description, xacro)
@@ -3,9 +3,10 @@
   <xacro:include filename="$(find cob_description)/urdf/common.xacro"/>
   <xacro:include filename="$(find raw_description)/urdf/vacuum_gripper/gripper.gazebo.xacro" />
-  <xacro:property name="gripper_length" value="0.14"/>
-  <xacro:property name="gripper_width" value="0.2"/>
-  <xacro:property name="gripper_height" value="0.14"/>
+  <xacro:property name="gripper_length" value="0.0886"/>
+  <xacro:property name="gripper_width" value="0.1515"/>
+  <xacro:property name="gripper_height" value="0.1515"/>
   <xacro:property name="gripper_body_height" value="0.14"/>
   <xacro:property name="gripper_radius" value="0.005"/>
+  <xacro:property name="gripper_collision_value" value="0.003"/>
   <xacro:macro name="vacuum_gripper" params="name parent *origin">
     <!-- joint between arm_ee_link and vacuum_gripper_link -->
@@ -19,5 +20,6 @@
         <parent link="${name}_frame"/>
         <child link="${name}_body"/>
-        <origin xyz="0.08015 -0.0475 0.0" rpy="-1.57079632679 0 3.1415"/>
+        <!--origin xyz="0.08015 -0.0475 0.0" rpy="-1.57079632679 0 3.1415"/-->
+        <origin xyz="0.00 0.00 0.0" rpy="-1.57079632679 0 1.57079632679"/>
     </joint>
     <link name="${name}_body">
@@ -25,5 +27,6 @@
             <origin xyz="0 0 -0.048" rpy="0 0 0"/>
             <geometry>
-                <mesh filename="package://raw_description/meshes/vacuum_gripper/vacuum_gripper.stl"/>
+                <!--mesh filename="package://raw_description/meshes/vacuum_gripper/vacuum_gripper.stl"/-->
+                <cylinder radius="${gripper_width}" length="${gripper_length}"/>
             </geometry>
             <material name="silver">
@@ -34,9 +37,10 @@
             <origin xyz="0.01 0.04 -0.048" rpy="0 0 0"/>
             <geometry>
-                <box size="0.13 0.14 0.071"/>
+                <!--box size="0.13 0.14 0.071"/-->
+                <cylinder radius="${gripper_width + gripper_collision_value}" length="${gripper_length + gripper_collision_value}"/>
             </geometry>
         </collision>
     </link>
-    <joint name="gripper_to_tcp" type="fixed">
+    <!--joint name="gripper_to_tcp" type="fixed">
         <parent link="${name}_frame"/>
         <child link="${name}"/>
@@ -53,5 +57,5 @@
             <xacro:sphere_geometry radius="${gripper_radius}"/>
         </collision>
-     </link>
+     </link-->
     <!-- extensions -->
     <xacro:vacuum_gripper_gazebo name="${name}"/>

Commit message: uncomment gripper tcp link

File: raw_description/urdf/vacuum_gripper/gripper.urdf.xacro (robot description, xacro)
@@ -35,5 +35,6 @@
         </visual>
         <collision>
-            <origin xyz="0.01 0.04 -0.048" rpy="0 0 0"/>
+            <!--origin xyz="0.01 0.04 -0.048" rpy="0 0 0"/-->
+            <origin xyz="0.00 0.00 -0.048" rpy="0 0 0"/>
             <geometry>
                 <!--box size="0.13 0.14 0.071"/-->
@@ -42,5 +43,5 @@
         </collision>
     </link>
-    <!--joint name="gripper_to_tcp" type="fixed">
+    <joint name="gripper_to_tcp" type="fixed">
         <parent link="${name}_frame"/>
         <child link="${name}"/>
@@ -49,5 +50,5 @@
     <link name="${name}">
         <visual>
-            <xacro:sphere_geometry radius="${gripper_radius}"/>
+            <xacro:sphere_geometry radius="${gripper_collision_value}"/>
             <material name="white">
                 <color rgba="1 1 1 0.5"/>
@@ -55,7 +56,7 @@
         </visual>
         <collision>
-            <xacro:sphere_geometry radius="${gripper_radius}"/>
+            <xacro:sphere_geometry radius="${gripper_collision_value}"/>
         </collision>
-     </link-->
+     </link>
     <!-- extensions -->
     <xacro:vacuum_gripper_gazebo name="${name}"/>

Commit message: added vacume gripper but mannually set origin, also give warning It starts with the word 'solid', indicating that it's an ASCII STL file, but it does not contain the word 'endsolid' so it is either a malformed ASCII STL file or it is actually a binary STL file

File: raw_description/urdf/vacuum_gripper/gripper.urdf.xacro (robot description, xacro)
@@ -21,12 +21,18 @@
         <child link="${name}_body"/>
         <!--origin xyz="0.08015 -0.0475 0.0" rpy="-1.57079632679 0 3.1415"/-->
-        <origin xyz="0.00 0.00 0.0" rpy="-1.57079632679 0 1.57079632679"/>
+        <origin xyz="0.200 -0.0750 -0.08" rpy="0.0 0.0 1.57079632679"/>
     </joint>
     <link name="${name}_body">
+       <inertial>
+       <!--choose randomly-->
+        <origin xyz="0 0 0" rpy="0.0 0 0.0"/>
+        <mass value="1.57307"/>
+        <inertia ixx="0.819" ixy="0" ixz="0" iyy="0.819" iyz="0" izz="0.819" />
+      </inertial>
         <visual>
-            <origin xyz="0 0 -0.048" rpy="0 0 0"/>
+            <origin xyz="0.0 0 0.0" rpy="0.0 0 0"/>
             <geometry>
-                <!--mesh filename="package://raw_description/meshes/vacuum_gripper/vacuum_gripper.stl"/-->
-                <cylinder radius="${gripper_width}" length="${gripper_length}"/>
+                <mesh filename="package://raw_description/meshes/vacuum_gripper/vacuum_gripper.STL" scale="0.001 0.001 0.001"/>
+                <!--cylinder radius="${gripper_width}" length="${gripper_length}"/-->
             </geometry>
             <material name="silver">
@@ -34,14 +40,6 @@
             </material>
         </visual>
-        <collision>
-            <!--origin xyz="0.01 0.04 -0.048" rpy="0 0 0"/-->
-            <origin xyz="0.00 0.00 -0.048" rpy="0 0 0"/>
-            <geometry>
-                <!--box size="0.13 0.14 0.071"/-->
-                <cylinder radius="${gripper_width + gripper_collision_value}" length="${gripper_length + gripper_collision_value}"/>
-            </geometry>
-        </collision>
     </link>
-    <joint name="gripper_to_tcp" type="fixed">
+    <!--joint name="gripper_to_tcp" type="fixed">
         <parent link="${name}_frame"/>
         <child link="${name}"/>
@@ -58,5 +56,5 @@
             <xacro:sphere_geometry radius="${gripper_collision_value}"/>
         </collision>
-     </link>
+     </link-->
     <!-- extensions -->
     <xacro:vacuum_gripper_gazebo name="${name}"/>

Commit message: manually added collision bounding box

File: raw_description/urdf/vacuum_gripper/gripper.urdf.xacro (robot description, xacro)
@@ -3,10 +3,7 @@
   <xacro:include filename="$(find cob_description)/urdf/common.xacro"/>
   <xacro:include filename="$(find raw_description)/urdf/vacuum_gripper/gripper.gazebo.xacro" />
-  <xacro:property name="gripper_length" value="0.0886"/>
-  <xacro:property name="gripper_width" value="0.1515"/>
-  <xacro:property name="gripper_height" value="0.1515"/>
-  <xacro:property name="gripper_body_height" value="0.14"/>
-  <xacro:property name="gripper_radius" value="0.005"/>
-  <xacro:property name="gripper_collision_value" value="0.003"/>
+  <xacro:property name="gripper_length" value="0.22"/>
+  <xacro:property name="gripper_width" value="0.07"/>
+  <xacro:property name="gripper_collision_value" value="0.01"/>
   <xacro:macro name="vacuum_gripper" params="name parent *origin">
     <!-- joint between arm_ee_link and vacuum_gripper_link -->
@@ -40,9 +37,16 @@
             </material>
         </visual>
+        <collision>
+            <origin xyz="0.075 0.10 0.08" rpy="1.57079632679 0 0.0"/>
+            <geometry>
+                <cylinder radius="${gripper_width + gripper_collision_value}" length="${gripper_length + gripper_collision_value}"/>
+                <!--cylinder radius="0.11" length="0.10"/--> <!--move to center of gripper-->
+            </geometry>
+        </collision>
     </link>
-    <!--joint name="gripper_to_tcp" type="fixed">
+    <joint name="gripper_to_tcp" type="fixed">
         <parent link="${name}_frame"/>
         <child link="${name}"/>
-        <origin xyz=" 0.1263 0.0 0.0" rpy="3.1415 0 0"/>
+        <origin xyz=" 0.20 0.0 0.0" rpy="3.1415 0 0"/>
     </joint>
     <link name="${name}">
@@ -56,5 +60,5 @@
             <xacro:sphere_geometry radius="${gripper_collision_value}"/>
         </collision>
-     </link-->
+     </link>
     <!-- extensions -->
     <xacro:vacuum_gripper_gazebo name="${name}"/>

Commit message: change mass of gripper

File: raw_description/urdf/vacuum_gripper/gripper.urdf.xacro (robot description, xacro)
@@ -4,5 +4,5 @@
   <xacro:include filename="$(find raw_description)/urdf/vacuum_gripper/gripper.gazebo.xacro" />
   <xacro:property name="gripper_length" value="0.22"/>
-  <xacro:property name="gripper_width" value="0.07"/>
+  <xacro:property name="gripper_dia" value="0.07"/>
   <xacro:property name="gripper_collision_value" value="0.01"/>
   <xacro:macro name="vacuum_gripper" params="name parent *origin">
@@ -17,5 +17,4 @@
         <parent link="${name}_frame"/>
         <child link="${name}_body"/>
-        <!--origin xyz="0.08015 -0.0475 0.0" rpy="-1.57079632679 0 3.1415"/-->
         <origin xyz="0.200 -0.0750 -0.08" rpy="0.0 0.0 1.57079632679"/>
     </joint>
@@ -24,5 +23,5 @@
        <!--choose randomly-->
         <origin xyz="0 0 0" rpy="0.0 0 0.0"/>
-        <mass value="1.57307"/>
+        <mass value="0.57307"/>
         <inertia ixx="0.819" ixy="0" ixz="0" iyy="0.819" iyz="0" izz="0.819" />
       </inertial>
@@ -31,5 +30,5 @@
             <geometry>
                 <mesh filename="package://raw_description/meshes/vacuum_gripper/vacuum_gripper.STL" scale="0.001 0.001 0.001"/>
-                <!--cylinder radius="${gripper_width}" length="${gripper_length}"/-->
+                <!--cylinder radius="${gripper_dia}" length="${gripper_length}"/-->
             </geometry>
             <material name="silver">
@@ -38,8 +37,8 @@
         </visual>
         <collision>
+        	<!-- move gripper_body frame to center of gripper and rotate same as arm_ee_link -->
             <origin xyz="0.075 0.10 0.08" rpy="1.57079632679 0 0.0"/>
             <geometry>
-                <cylinder radius="${gripper_width + gripper_collision_value}" length="${gripper_length + gripper_collision_value}"/>
-                <!--cylinder radius="0.11" length="0.10"/--> <!--move to center of gripper-->
+                <cylinder radius="${gripper_dia + gripper_collision_value}" length="${gripper_length + gripper_collision_value}"/>
             </geometry>
         </collision>
