Commit message: add cemera collision but still need to work

File: raw_description/urdf/vacuum_gripper/gripper.urdf.xacro (robot description, xacro)
@@ -14,8 +14,66 @@
     </joint>
     <link name="${name}_frame"/>
+    <joint name="${name}_coupling_joint" type="fixed">
+        <parent link="${name}_frame"/>
+        <child link="${name}_coupling_link"/>
+        <origin xyz=" 0.0 0.0 0.0" rpy="0 1.57079632679 0"/>
+    </joint>
+    <link name="${name}_coupling_link">
+       <inertial>
+       <!--choose randomly-->
+        <origin xyz="0 0 0" rpy="0.0 0 0.0"/>
+        <mass value="0.0057307"/>
+        <inertia ixx="0.819" ixy="0" ixz="0" iyy="0.819" iyz="0" izz="0.819" />
+      </inertial>
+        <visual>
+            <origin xyz="0.0 0 0.0" rpy="0.0 0 0"/>
+            <geometry>
+                <cylinder radius="${gripper_dia*0.5}" length="0.030"/> <!--${gripper_length}-->
+            </geometry>
+            <material name="silver">
+                <color rgba="0.8 0.8 0.8 1"/>
+            </material>
+        </visual>
+        <collision>
+                <!-- move gripper_body frame to center of gripper and rotate same as arm_ee_link -->
+            <origin xyz="0.030 0.00 0.00" rpy="0 0 0.0"/>
+            <geometry>
+                <cylinder radius="${gripper_dia + gripper_collision_value}" length="0.04"/>
+            </geometry>
+        </collision>
+    </link>
+    <joint name="${name}_camera_coupling_joint" type="fixed">
+        <parent link="${name}_coupling_link"/>
+        <child link="${name}_camera_coupling_link"/>
+        <origin xyz=" 0.00 0.0 0.0" rpy="0 0.0 0"/>
+    </joint>
+    <link name="${name}_camera_coupling_link">
+       <inertial>
+       <!--choose randomly-->
+        <origin xyz="0 0 0" rpy="0.0 0 0.0"/>
+        <mass value="0.0057307"/>
+        <inertia ixx="0.819" ixy="0" ixz="0" iyy="0.819" iyz="0" izz="0.819" />
+      </inertial>
+        <visual>
+            <origin xyz="0.083 0 0.0" rpy="0.0 0 0"/>
+            <geometry>
+                <box size="0.126 0.170 0.043"/> <!-- hwl-->
+            </geometry>
+            <material name="silver">
+                <color rgba="0.8 0.8 0.8 1"/>
+            </material>
+        </visual>
+        <collision>
+                <!-- move gripper_body frame to center of gripper and rotate same as arm_ee_link -->
+            <origin xyz="0.083 0.00 0.00" rpy="0 0 0.0"/>
+            <geometry>
+                <box size="0.126 0.170 0.043 "/> <!-- hwl-->
+            </geometry>
+        </collision>
+    </link>
     <joint name="gripper_to_palm" type="fixed">
         <parent link="${name}_frame"/>
         <child link="${name}_body"/>
-        <origin xyz="0.200 -0.0750 -0.08" rpy="0.0 0.0 1.57079632679"/>
+        <origin xyz="0.215 -0.0750 -0.08" rpy="0.0 0.0 1.57079632679"/>
     </joint>
     <link name="${name}_body">
@@ -37,5 +95,5 @@
         </visual>
         <collision>
-        	<!-- move gripper_body frame to center of gripper and rotate same as arm_ee_link -->
+                <!-- move gripper_body frame to center of gripper and rotate same as arm_ee_link -->
             <origin xyz="0.075 0.10 0.08" rpy="1.57079632679 0 0.0"/>
             <geometry>
@@ -47,5 +105,5 @@
         <parent link="${name}_frame"/>
         <child link="${name}"/>
-        <origin xyz=" 0.20 0.0 0.0" rpy="3.1415 0 0"/>
+        <origin xyz=" 0.215 0.0 0.0" rpy="3.1415 0 0"/>
     </joint>
     <link name="${name}">

Commit message: add cemera collision

File: raw_description/urdf/vacuum_gripper/gripper.urdf.xacro (robot description, xacro)
@@ -46,5 +46,5 @@
         <parent link="${name}_coupling_link"/>
         <child link="${name}_camera_coupling_link"/>
-        <origin xyz=" 0.00 0.0 0.0" rpy="0 0.0 0"/>
+        <origin xyz=" 0.00 0.0 0.0" rpy="0 0.0 0.5"/>
     </joint>
     <link name="${name}_camera_coupling_link">
@@ -58,5 +58,5 @@
             <origin xyz="0.083 0 0.0" rpy="0.0 0 0"/>
             <geometry>
-                <box size="0.126 0.170 0.043"/> <!-- hwl-->
+                <box size="0.126 0.170 0.043 "/> <!-- hwl-->
             </geometry>
             <material name="silver">
@@ -85,5 +85,5 @@
       </inertial>
         <visual>
-            <origin xyz="0.0 0 0.0" rpy="0.0 0 0"/>
+            <origin xyz="0.0 0 0.0" rpy="0 0 0"/>
             <geometry>
                 <mesh filename="package://raw_description/meshes/vacuum_gripper/vacuum_gripper.STL" scale="0.001 0.001 0.001"/>

Commit message: change orientation of gripper frame

File: raw_description/urdf/vacuum_gripper/gripper.urdf.xacro (robot description, xacro)
@@ -105,5 +105,5 @@
         <parent link="${name}_frame"/>
         <child link="${name}"/>
-        <origin xyz=" 0.215 0.0 0.0" rpy="3.1415 0 0"/>
+        <origin xyz=" 0.215 0.0 0.0" rpy="3.1415 0 0"/> # 3.1415 => 0.0
     </joint>
     <link name="${name}">

Commit message: added new stl file with correct gripper frame

File: raw_description/urdf/vacuum_gripper/gripper.urdf.xacro (robot description, xacro)
@@ -14,4 +14,5 @@
     </joint>
     <link name="${name}_frame"/>
+    <!-- camera collision -->
     <joint name="${name}_coupling_joint" type="fixed">
         <parent link="${name}_frame"/>
@@ -43,8 +44,9 @@
         </collision>
     </link>
+    <!-- ====== Camera collision ==== -->
     <joint name="${name}_camera_coupling_joint" type="fixed">
         <parent link="${name}_coupling_link"/>
         <child link="${name}_camera_coupling_link"/>
-        <origin xyz=" 0.00 0.0 0.0" rpy="0 0.0 0.5"/>
+        <origin xyz=" 0.00 0.0 0.0" rpy="0 0.0 0.0"/>
     </joint>
     <link name="${name}_camera_coupling_link">
@@ -72,8 +74,10 @@
         </collision>
     </link>
+    <!-- ======= Gripper ========-->
+    <!-- with parent link gripper_frame, origin 0.0 1.57079632679 0.0 -->
     <joint name="gripper_to_palm" type="fixed">
-        <parent link="${name}_frame"/>
+        <parent link="${name}_coupling_link"/>
         <child link="${name}_body"/>
-        <origin xyz="0.215 -0.0750 -0.08" rpy="0.0 0.0 1.57079632679"/>
+        <origin xyz="0.0 0.0 0.00" rpy="0.0 0.0 -1.57079632679"/> #1.57079632679  0.0 1.57079632679
     </joint>
     <link name="${name}_body">
@@ -88,5 +92,4 @@
             <geometry>
                 <mesh filename="package://raw_description/meshes/vacuum_gripper/vacuum_gripper.STL" scale="0.001 0.001 0.001"/>
-                <!--cylinder radius="${gripper_dia}" length="${gripper_length}"/-->
             </geometry>
             <material name="silver">

Commit message: add comment

File: raw_description/urdf/vacuum_gripper/gripper.urdf.xacro (robot description, xacro)
@@ -79,5 +79,6 @@
         <parent link="${name}_coupling_link"/>
         <child link="${name}_body"/>
-        <origin xyz="0.0 0.0 0.00" rpy="0.0 0.0 -1.57079632679"/> #1.57079632679  0.0 1.57079632679
+        # yaw rotation used for rotate gripper or display of gripper upside or roll gripper
+        <origin xyz="0.0 0.0 0.00" rpy="0.0 0.0 -1.57079632679"/>  #1.57079632679  0.0 1.57079632679
     </joint>
     <link name="${name}_body">

Commit message: change gripper collision object urdf

File: raw_description/urdf/vacuum_gripper/gripper.urdf.xacro (robot description, xacro)
@@ -100,5 +100,5 @@
         <collision>
                 <!-- move gripper_body frame to center of gripper and rotate same as arm_ee_link -->
-            <origin xyz="0.075 0.10 0.08" rpy="1.57079632679 0 0.0"/>
+            <origin xyz="0.00 0.0 0.08" rpy="0.0 0 0.0"/>
             <geometry>
                 <cylinder radius="${gripper_dia + gripper_collision_value}" length="${gripper_length + gripper_collision_value}"/>

Commit message: change orientation of gripper

File: raw_description/urdf/vacuum_gripper/gripper.urdf.xacro (robot description, xacro)
@@ -80,5 +80,5 @@
         <child link="${name}_body"/>
         # yaw rotation used for rotate gripper or display of gripper upside or roll gripper
-        <origin xyz="0.0 0.0 0.00" rpy="0.0 0.0 -1.57079632679"/>  #1.57079632679  0.0 1.57079632679
+        <origin xyz="0.0 0.0 0.00" rpy="0.0 0.0 1.57079632679"/> #new: 0.0 0.0 -1.57079632679 #1.57079632679  0.0 1.57079632679
     </joint>
     <link name="${name}_body">

Commit message: add offset on gripper link

File: raw_description/urdf/vacuum_gripper/gripper.urdf.xacro (robot description, xacro)
@@ -109,5 +109,5 @@
         <parent link="${name}_frame"/>
         <child link="${name}"/>
-        <origin xyz=" 0.215 0.0 0.0" rpy="3.1415 0 0"/> # 3.1415 => 0.0
+        <origin xyz=" 0.215 0.0 0.03" rpy="3.1415 0 0"/> # 3.1415 => 0.0
     </joint>
     <link name="${name}">

Commit message: undo ur gripper

File: raw_description/urdf/vacuum_gripper/gripper.urdf.xacro (robot description, xacro)
@@ -3,7 +3,9 @@
   <xacro:include filename="$(find cob_description)/urdf/common.xacro"/>
   <xacro:include filename="$(find raw_description)/urdf/vacuum_gripper/gripper.gazebo.xacro" />
-  <xacro:property name="gripper_length" value="0.22"/>
-  <xacro:property name="gripper_dia" value="0.07"/>
-  <xacro:property name="gripper_collision_value" value="0.01"/>
+  <xacro:property name="gripper_length" value="0.14"/>
+  <xacro:property name="gripper_width" value="0.2"/>
+  <xacro:property name="gripper_height" value="0.14"/>
+  <xacro:property name="gripper_body_height" value="0.14"/>
+  <xacro:property name="gripper_radius" value="0.005"/>
   <xacro:macro name="vacuum_gripper" params="name parent *origin">
     <!-- joint between arm_ee_link and vacuum_gripper_link -->
@@ -14,21 +16,14 @@
     </joint>
     <link name="${name}_frame"/>
-    <!-- camera collision -->
-    <joint name="${name}_coupling_joint" type="fixed">
+    <joint name="gripper_to_palm" type="fixed">
         <parent link="${name}_frame"/>
-        <child link="${name}_coupling_link"/>
-        <origin xyz=" 0.0 0.0 0.0" rpy="0 1.57079632679 0"/>
+        <child link="${name}_body"/>
+        <origin xyz="0.08015 -0.0475 0.0" rpy="-1.57079632679 0 3.1415"/>
     </joint>
-    <link name="${name}_coupling_link">
-       <inertial>
-       <!--choose randomly-->
-        <origin xyz="0 0 0" rpy="0.0 0 0.0"/>
-        <mass value="0.0057307"/>
-        <inertia ixx="0.819" ixy="0" ixz="0" iyy="0.819" iyz="0" izz="0.819" />
-      </inertial>
+    <link name="${name}_body">
         <visual>
-            <origin xyz="0.0 0 0.0" rpy="0.0 0 0"/>
+            <origin xyz="0 0 -0.048" rpy="0 0 0"/>
             <geometry>
-                <cylinder radius="${gripper_dia*0.5}" length="0.030"/> <!--${gripper_length}-->
+                <mesh filename="package://raw_description/meshes/vacuum_gripper/vacuum_gripper.stl"/>
             </geometry>
             <material name="silver">
@@ -37,70 +32,7 @@
         </visual>
         <collision>
-                <!-- move gripper_body frame to center of gripper and rotate same as arm_ee_link -->
-            <origin xyz="0.030 0.00 0.00" rpy="0 0 0.0"/>
+            <origin xyz="0.01 0.04 -0.048" rpy="0 0 0"/>
             <geometry>
-                <cylinder radius="${gripper_dia + gripper_collision_value}" length="0.04"/>
-            </geometry>
-        </collision>
-    </link>
-    <!-- ====== Camera collision ==== -->
-    <joint name="${name}_camera_coupling_joint" type="fixed">
-        <parent link="${name}_coupling_link"/>
-        <child link="${name}_camera_coupling_link"/>
-        <origin xyz=" 0.00 0.0 0.0" rpy="0 0.0 0.0"/>
-    </joint>
-    <link name="${name}_camera_coupling_link">
-       <inertial>
-       <!--choose randomly-->
-        <origin xyz="0 0 0" rpy="0.0 0 0.0"/>
-        <mass value="0.0057307"/>
-        <inertia ixx="0.819" ixy="0" ixz="0" iyy="0.819" iyz="0" izz="0.819" />
-      </inertial>
-        <visual>
-            <origin xyz="0.083 0 0.0" rpy="0.0 0 0"/>
-            <geometry>
-                <box size="0.126 0.170 0.043 "/> <!-- hwl-->
-            </geometry>
-            <material name="silver">
-                <color rgba="0.8 0.8 0.8 1"/>
-            </material>
-        </visual>
-        <collision>
-                <!-- move gripper_body frame to center of gripper and rotate same as arm_ee_link -->
-            <origin xyz="0.083 0.00 0.00" rpy="0 0 0.0"/>
-            <geometry>
-                <box size="0.126 0.170 0.043 "/> <!-- hwl-->
-            </geometry>
-        </collision>
-    </link>
-    <!-- ======= Gripper ========-->
-    <!-- with parent link gripper_frame, origin 0.0 1.57079632679 0.0 -->
-    <joint name="gripper_to_palm" type="fixed">
-        <parent link="${name}_coupling_link"/>
-        <child link="${name}_body"/>
-        # yaw rotation used for rotate gripper or display of gripper upside or roll gripper
-        <origin xyz="0.0 0.0 0.00" rpy="0.0 0.0 1.57079632679"/> #new: 0.0 0.0 -1.57079632679 #1.57079632679  0.0 1.57079632679
-    </joint>
-    <link name="${name}_body">
-       <inertial>
-       <!--choose randomly-->
-        <origin xyz="0 0 0" rpy="0.0 0 0.0"/>
-        <mass value="0.57307"/>
-        <inertia ixx="0.819" ixy="0" ixz="0" iyy="0.819" iyz="0" izz="0.819" />
-      </inertial>
-        <visual>
-            <origin xyz="0.0 0 0.0" rpy="0 0 0"/>
-            <geometry>
-                <mesh filename="package://raw_description/meshes/vacuum_gripper/vacuum_gripper.STL" scale="0.001 0.001 0.001"/>
-            </geometry>
-            <material name="silver">
-                <color rgba="0.8 0.8 0.8 1"/>
-            </material>
-        </visual>
-        <collision>
-                <!-- move gripper_body frame to center of gripper and rotate same as arm_ee_link -->
-            <origin xyz="0.00 0.0 0.08" rpy="0.0 0 0.0"/>
-            <geometry>
-                <cylinder radius="${gripper_dia + gripper_collision_value}" length="${gripper_length + gripper_collision_value}"/>
+                <box size="0.13 0.14 0.071"/>
             </geometry>
         </collision>
@@ -109,9 +41,9 @@
         <parent link="${name}_frame"/>
         <child link="${name}"/>
-        <origin xyz=" 0.215 0.0 0.03" rpy="3.1415 0 0"/> # 3.1415 => 0.0
+        <origin xyz=" 0.1263 0.0 0.0" rpy="3.1415 0 0"/>
     </joint>
     <link name="${name}">
         <visual>
-            <xacro:sphere_geometry radius="${gripper_collision_value}"/>
+            <xacro:sphere_geometry radius="${gripper_radius}"/>
             <material name="white">
                 <color rgba="1 1 1 0.5"/>
@@ -119,5 +51,5 @@
         </visual>
         <collision>
-            <xacro:sphere_geometry radius="${gripper_collision_value}"/>
+            <xacro:sphere_geometry radius="${gripper_radius}"/>
         </collision>
      </link>
