Commit message: change corrdinate of camera frame

File: raw_description/urdf/arm_camera/arm_camera.urdf.xacro (robot description, xacro)
@@ -18,5 +18,5 @@
         <parent link="${name}_frame"/>
         <child link="${name}_link"/>
-        <origin xyz=" 0.00 0.0 0.0" rpy="0 0.0 0.0"/>
+        <origin xyz=" 0.083 0.0 0.0" rpy="0.0 -1.57 -3.1415"/>
     </joint>
     <link name="${name}_link">
@@ -28,5 +28,5 @@
       </inertial>
         <visual>
-            <origin xyz="0.083 0 0.0" rpy="0.0 0 0"/>
+            <origin xyz="0.00 0 0.0" rpy="0.0 0 0"/>
             <geometry>
                 <box size="${arm_camera_height} ${arm_camera_width} ${arm_camera_length}"/> <!-- hwl-->
@@ -38,5 +38,5 @@
         <collision>
             <!-- move gripper_body frame to center of gripper and rotate same as arm_ee_link -->
-            <origin xyz="0.083 0.00 0.00" rpy="0 0 0.0"/>
+            <origin xyz="0.00 0.00 0.00" rpy="0 0 0.0"/>
             <geometry>
                 <box size="${arm_camera_height} ${arm_camera_width} ${arm_camera_length}"/> <!-- hwl-->

Commit message: changerandom  intertia to app intertia

File: raw_description/urdf/arm_camera/arm_camera.urdf.xacro (robot description, xacro)
@@ -21,14 +21,11 @@
     </joint>
     <link name="${name}_link">
-       <inertial>
-       <!--choose randomly-->
-        <origin xyz="0 0 0" rpy="0.0 0 0.0"/>
-        <mass value="0.0057307"/>
-        <inertia ixx="0.819" ixy="0" ixz="0" iyy="0.819" iyz="0" izz="0.819" />
-      </inertial>
+		<xacro:box_inertial x="0.002" y="0.04" z="0.26" mass="0.0057307">
+        	<origin xyz="0.0 0.0 0.0" rpy="0 0 0" />
+      	</xacro:box_inertial>
         <visual>
             <origin xyz="0.00 0 0.0" rpy="0.0 0 0"/>
             <geometry>
-                <box size="${arm_camera_height} ${arm_camera_width} ${arm_camera_length}"/> <!-- hwl-->
+                <box size="${arm_camera_length} ${arm_camera_width} ${arm_camera_height}"/> <!-- hwl-->
             </geometry>
             <material name="silver">
@@ -40,5 +37,5 @@
             <origin xyz="0.00 0.00 0.00" rpy="0 0 0.0"/>
             <geometry>
-                <box size="${arm_camera_height} ${arm_camera_width} ${arm_camera_length}"/> <!-- hwl-->
+                <box size="${arm_camera_length} ${arm_camera_width} ${arm_camera_height}"/> <!-- hwl-->
             </geometry>
         </collision>

File: raw_description/urdf/schmaltz_gripper/gripper.urdf.xacro (robot description, xacro)
@@ -21,10 +21,7 @@
     </joint>
     <link name="${name}_coupling_link">
-       <inertial>
-       <!--choose randomly-->
-        <origin xyz="0 0 0" rpy="0.0 0 0.0"/>
-        <mass value="0.0057307"/>
-        <inertia ixx="0.819" ixy="0" ixz="0" iyy="0.819" iyz="0" izz="0.819" />
-      </inertial>
+		<xacro:box_inertial x="0.002" y="0.04" z="0.26" mass="0.0057307">
+        	<origin xyz="0.0 0.0 0.0" rpy="0 0 0" />
+      	</xacro:box_inertial>
         <visual>
             <origin xyz="0.0 0 0.0" rpy="0.0 0 0"/>
@@ -51,10 +48,7 @@
     </joint>
     <link name="${name}_body">
-       <inertial>
-       <!--choose randomly-->
-        <origin xyz="0 0 0" rpy="0.0 0 0.0"/>
-        <mass value="0.57307"/>
-        <inertia ixx="0.819" ixy="0" ixz="0" iyy="0.819" iyz="0" izz="0.819" />
-      </inertial>
+		<xacro:box_inertial x="0.002" y="0.04" z="0.26" mass="0.57307">
+        	<origin xyz="0.0 0.0 0.0" rpy="0 0 0" />
+      	</xacro:box_inertial>
         <visual>
             <origin xyz="0.0 0 0.0" rpy="0 0 0"/>

Commit message: change origin and collisoin origin from link to joint

File: raw_description/urdf/arm_camera/arm_camera.urdf.xacro (robot description, xacro)
@@ -21,11 +21,11 @@
     </joint>
     <link name="${name}_link">
-		<xacro:box_inertial x="0.002" y="0.04" z="0.26" mass="0.0057307">
-        	<origin xyz="0.0 0.0 0.0" rpy="0 0 0" />
-      	</xacro:box_inertial>
+        <xacro:box_inertial x="0.002" y="0.04" z="0.26" mass="0.0057307">
+            <origin xyz="0.0 0.0 0.0" rpy="0 0 0" />
+        </xacro:box_inertial>
         <visual>
-            <origin xyz="0.00 0 0.0" rpy="0.0 0 0"/>
+            <origin xyz="0.0 0.0 0.0" rpy="0.0 0.0 0.0"/>
             <geometry>
-                <box size="${arm_camera_length} ${arm_camera_width} ${arm_camera_height}"/> <!-- hwl-->
+                <box size="${arm_camera_length} ${arm_camera_width} ${arm_camera_height}"/> <!-- lwh-->
             </geometry>
             <material name="silver">
@@ -35,7 +35,7 @@
         <collision>
             <!-- move gripper_body frame to center of gripper and rotate same as arm_ee_link -->
-            <origin xyz="0.00 0.00 0.00" rpy="0 0 0.0"/>
+            <origin xyz="0.0 0.0 0.0" rpy="0.0 0.0 0.0"/>
             <geometry>
-                <box size="${arm_camera_length} ${arm_camera_width} ${arm_camera_height}"/> <!-- hwl-->
+                <box size="${arm_camera_length} ${arm_camera_width} ${arm_camera_height}"/> <!-- lwh-->
             </geometry>
         </collision>

File: raw_description/urdf/schmaltz_gripper/gripper.urdf.xacro (robot description, xacro)
@@ -21,9 +21,9 @@
     </joint>
     <link name="${name}_coupling_link">
-		<xacro:box_inertial x="0.002" y="0.04" z="0.26" mass="0.0057307">
-        	<origin xyz="0.0 0.0 0.0" rpy="0 0 0" />
-      	</xacro:box_inertial>
+        <xacro:box_inertial x="0.002" y="0.04" z="0.26" mass="0.0057307">
+            <origin xyz="0.0 0.0 0.0" rpy="0 0 0" />
+        </xacro:box_inertial>
         <visual>
-            <origin xyz="0.0 0 0.0" rpy="0.0 0 0"/>
+            <origin xyz="0.0 0.0 0.0" rpy="0.0 0.0 0.0"/>
             <geometry>
                 <cylinder radius="${gripper_dia*0.5}" length="0.030"/>
@@ -35,7 +35,8 @@
         <collision>
                 <!-- move gripper_body frame to center of gripper and rotate same as arm_ee_link -->
-            <origin xyz="0.030 0.00 0.00" rpy="0 0 0.0"/>
+            <origin xyz="0.0 0.0 0.0" rpy="0.0 0.0 0.0"/>
             <geometry>
-                <cylinder radius="${gripper_dia + gripper_collision_value}" length="0.04"/>
+                <!--cylinder radius="${gripper_dia + gripper_collision_value}" length="0.04"/-->
+                <cylinder radius="${gripper_dia}" length="0.04"/>
             </geometry>
         </collision>
@@ -48,9 +49,9 @@
     </joint>
     <link name="${name}_body">
-		<xacro:box_inertial x="0.002" y="0.04" z="0.26" mass="0.57307">
-        	<origin xyz="0.0 0.0 0.0" rpy="0 0 0" />
+        <xacro:box_inertial x="0.002" y="0.04" z="0.26" mass="0.57307">
+            <origin xyz="0.0 0.0 0.0" rpy="0.0 0.0 0.0" />
       	</xacro:box_inertial>
         <visual>
-            <origin xyz="0.0 0 0.0" rpy="0 0 0"/>
+            <origin xyz="0.0 0.0 0.0" rpy="0.0 0.0 0.0"/>
             <geometry>
                 <mesh filename="package://raw_description/meshes/schmaltz_gripper/schmaltz_gripper.STL" scale="0.001 0.001 0.001"/>
@@ -62,5 +63,5 @@
         <collision>
                 <!-- move gripper_body frame to center of gripper and rotate same as arm_ee_link -->
-            <origin xyz="0.00 0.0 0.08" rpy="0.0 0 0.0"/>
+            <origin xyz="0.0 0.0 0.0" rpy="0.0 0.0 0.0"/>   <!-- 0.00 0.0 0.08 -->
             <geometry>
                 <cylinder radius="${gripper_dia + gripper_collision_value}" length="${gripper_length + gripper_collision_value}"/>
@@ -71,5 +72,5 @@
         <parent link="${name}_frame"/>
         <child link="${name}"/>
-        <origin xyz=" 0.215 0.0 0.03" rpy="3.1415 0 0"/> # pz = 0 -> 0.03 ,  0.0 -> 3.1415
+        <origin xyz=" 0.215 0.0 0.03" rpy="3.1415 0 0"/> <!-- pz = 0 -> 0.03 , roll: 0.0 -> 3.1415 -->
     </joint>
     <link name="${name}">
