Commit message: add scaling factor into stl file

File: raw_description/urdf/schmaltz_gripper/gripper.urdf.xacro (robot description, xacro)
@@ -55,5 +55,5 @@
             <origin xyz="0.0 0.0 0.0" rpy="0.0 0.0 0.0"/>
             <geometry>
-                <mesh filename="package://raw_description/meshes/schmaltz_gripper/schmaltz_gripper.STL" scale="0.001 0.001 0.001"/>
+                <mesh filename="package://raw_description/meshes/schmaltz_gripper/schmaltz_gripper.STL"/>
             </geometry>
             <material name="silver">
