Commit message: change stl file formate

File: raw_description/urdf/kinect_camera/kinect_camera.urdf.xacro (robot description, xacro)
@@ -30,7 +30,5 @@
                 <box size="${kinect_camera_length} ${kinect_camera_width} ${kinect_camera_height}"/> <!-- lwh-->
             </geometry>
-            <material name="silver">
-                <color rgba="0.8 0.8 0.8 1"/>
-            </material>
+            <material name="IPA/LightGrey" />
         </visual>
         <collision>

File: raw_description/urdf/schmaltz_gripper/gripper.urdf.xacro (robot description, xacro)
@@ -29,7 +29,5 @@
                 <cylinder radius="${gripper_dia*0.5}" length="0.030"/>
             </geometry>
-            <material name="silver">
-                <color rgba="0.8 0.8 0.8 1"/>
-            </material>
+            <material name="IPA/LightGrey" />
         </visual>
         <collision>
@@ -55,9 +53,7 @@
             <origin xyz="0.0 0.0 0.0" rpy="0.0 0.0 0.0"/>
             <geometry>
-                <mesh filename="package://raw_description/meshes/schmaltz_gripper/schmaltz_gripper.STL"/>
+                <mesh filename="package://raw_description/meshes/schmaltz_gripper/schmaltz_gripper.stl"/>
             </geometry>
-            <material name="silver">
-                <color rgba="0.8 0.8 0.8 1"/>
-            </material>
+            <material name="IPA/LightGrey" />
         </visual>
         <collision>
@@ -77,7 +73,5 @@
         <visual>
             <xacro:sphere_geometry radius="${gripper_collision_value}"/>
-            <material name="white">
-                <color rgba="1 1 1 0.5"/>
-            </material>
+            <material name="IPA/LightGrey" />
         </visual>
         <collision>
