Commit message: dummy stl/dae files

File: raw_description/urdf/raw4_base/base.urdf.xacro (robot description, xacro)
@@ -35,6 +35,6 @@
         <origin xyz="0 0 0.25" rpy="0 0 0" />
         <geometry>
-          <!--mesh filename="package://raw_description/meshes/base/raw_base_short.dae"/-->
-          <box size="1.2 0.75 0.1"/>
+          <mesh filename="package://raw_description/meshes/raw4_base/raw4_base.dae"/>
+          <!-- <box size="1.2 0.75 0.1"/> -->
         </geometry>
         <material name="Grey">
@@ -45,6 +45,6 @@
         <origin xyz="0 0 0.25" rpy="0 0 0" />
         <geometry>
-          <!-- mesh filename="package://raw_description/meshes/base/raw_base_short.stl"/-->
-          <box size="1.2 0.75 0.1"/>
+          <mesh filename="package://raw_description/meshes/raw4_base/raw4_base.stl"/>
+          <!-- <box size="1.2 0.75 0.1"/> -->
         </geometry>
       </collision>

Commit message: adapted wheel offsets

File: raw_description/urdf/raw4_base/base.urdf.xacro (robot description, xacro)
@@ -7,8 +7,8 @@
   <!-- properties -->
   <xacro:property name="caster_offset_x" value="0.350" />  <!--modify here-->
-  <xacro:property name="caster_offset_y_bl" value="0.190" />
-  <xacro:property name="caster_offset_y_br" value="-0.190" />
-  <xacro:property name="caster_offset_y_fl" value="0.190" />
-  <xacro:property name="caster_offset_y_fr" value="-0.190" />
+  <xacro:property name="caster_offset_y_bl" value="0.188" />
+  <xacro:property name="caster_offset_y_br" value="-0.188" />
+  <xacro:property name="caster_offset_y_fl" value="0.188" />
+  <xacro:property name="caster_offset_y_fr" value="-0.188" />
   <xacro:property name="caster_offset_z" value="0.08" />
   <xacro:property name="base_mass" value="43.1" />
