Commit message: adjusted folder structure

File: raw_description/urdf/raw3_base_long/base.urdf.xacro (robot description, xacro)
@@ -2,5 +2,5 @@
 <robot xmlns:xacro="http://www.ros.org/wiki/xacro">
   <xacro:include filename="$(find cob_description)/urdf/common.xacro"/>
-  <xacro:include filename="$(find raw_description)/urdf/base_long/base.gazebo.xacro" />
+  <xacro:include filename="$(find raw_description)/urdf/raw3_base_long/base.gazebo.xacro" />
   <!-- drive_wheel module -->
   <xacro:include filename="$(find cob_description)/urdf/drive_wheel/drive_wheel.urdf.xacro" />
@@ -36,5 +36,5 @@
         <origin xyz="0 0 0" rpy="0 0 0"/>
         <geometry>
-          <mesh filename="package://raw_description/meshes/base/raw_battery.stl"/>
+          <mesh filename="package://raw_description/meshes/raw3_base/raw3_battery.stl"/>
         </geometry>
         <material name="Gazebo/Black" />
@@ -44,5 +44,5 @@
         <geometry>
           <box size="${battery_size_x} ${battery_size_y} ${battery_size_z}" />
-          <!--mesh filename="package://raw_description/meshes/base/raw_battery.stl"/-->
+          <!--mesh filename="package://raw_description/meshes/raw3_base/raw3_battery.stl"/-->
         </geometry>
        </collision>
@@ -65,5 +65,5 @@
         <origin xyz="0 0 0.209" rpy="0 0 0" />
         <geometry>
-          <mesh filename="package://raw_description/meshes/base/raw_base_long.dae"/>
+          <mesh filename="package://raw_description/meshes/raw3_base/raw3_base_long.dae"/>
         </geometry>
       </visual>
@@ -71,5 +71,5 @@
         <origin xyz="0 0 0.209" rpy="0 0 0" />
         <geometry>
-          <mesh filename="package://raw_description/meshes/base/raw_base_long.stl"/>
+          <mesh filename="package://raw_description/meshes/raw2_base/raw3_base_long.stl"/>
           <!--box size="1.04 0.58 0.31" /-->
         </geometry>

File: raw_description/urdf/raw3_base_short/base.urdf.xacro (robot description, xacro)
@@ -2,5 +2,5 @@
 <robot xmlns:xacro="http://www.ros.org/wiki/xacro">
   <xacro:include filename="$(find cob_description)/urdf/common.xacro"/>
-  <xacro:include filename="$(find raw_description)/urdf/base_short/base.gazebo.xacro" />
+  <xacro:include filename="$(find raw_description)/urdf/raw3_base_short/base.gazebo.xacro" />
   <!-- drive_wheel module -->
   <xacro:include filename="$(find cob_description)/urdf/drive_wheel/drive_wheel.urdf.xacro" />
@@ -69,5 +69,5 @@
         <origin xyz="0 0 0.209" rpy="0 0 0" />
         <geometry>
-          <mesh filename="package://raw_description/meshes/base/raw_base_short.dae"/>
+          <mesh filename="package://raw_description/meshes/raw3_base/raw3_base_short.dae"/>
         </geometry>
       </visual>
@@ -75,5 +75,5 @@
         <origin xyz="0 0 0.209" rpy="0 0 0" />
         <geometry>
-          <mesh filename="package://raw_description/meshes/base/raw_base_short.stl"/>
+          <mesh filename="package://raw_description/meshes/raw3_base/raw3_base_short.stl"/>
           <!--box size="0.758 0.573 0.096"/-->
         </geometry>

File: raw_description/urdf/raw4_base/base.urdf.xacro (robot description, xacro)
@@ -2,5 +2,5 @@
 <robot xmlns:xacro="http://www.ros.org/wiki/xacro">
   <xacro:include filename="$(find cob_description)/urdf/common.xacro"/>
-  <xacro:include filename="$(find raw_description)/urdf/raw4_base/raw4_base.gazebo.xacro" />
+  <xacro:include filename="$(find raw_description)/urdf/raw4_base/base.gazebo.xacro" />
   <!-- drive_wheel module -->
   <xacro:include filename="$(find cob_description)/urdf/drive_wheel/drive_wheel.urdf.xacro" />

Commit message: fix mesh path

File: raw_description/urdf/raw3_base_long/base.urdf.xacro (robot description, xacro)
@@ -71,5 +71,5 @@
         <origin xyz="0 0 0.209" rpy="0 0 0" />
         <geometry>
-          <mesh filename="package://raw_description/meshes/raw2_base/raw3_base_long.stl"/>
+          <mesh filename="package://raw_description/meshes/raw3_base/raw3_base_long.stl"/>
           <!--box size="1.04 0.58 0.31" /-->
         </geometry>
