Commit message: fake inertia for pg70

File: cob_description/urdf/pg70/pg70.urdf.xacro (robot description, xacro)
@@ -40,9 +40,5 @@
     </xacro:unless>
     <link name="${name}_palm_link">
-      <inertial>
-        <origin xyz="0 0 0" rpy="0 0 0"/>
-        <mass value="1"/>
-        <inertia ixx="0.01" ixy="0" ixz="0" iyy="0.01" iyz="0" izz="0.01" />
-      </inertial>
+      <xacro:default_inertial/>
       <visual>
         <geometry>
@@ -65,9 +61,5 @@
     </joint>
     <link name="${name}_finger_left_link">
-      <inertial>
-        <origin xyz="0 0 0" rpy="0 0 0"/>
-        <mass value="1"/>
-        <inertia ixx="0.01" ixy="0" ixz="0" iyy="0.01" iyz="0" izz="0.01" />
-      </inertial>
+      <xacro:default_inertial/>
       <visual>
         <geometry>
@@ -96,9 +88,5 @@
     </joint>
     <link name="${name}_finger_right_link">
-      <inertial>
-        <origin xyz="0 0 0" rpy="0 0 0"/>
-        <mass value="1"/>
-        <inertia ixx="0.01" ixy="0" ixz="0" iyy="0.01" iyz="0" izz="0.01" />
-      </inertial>
+      <xacro:default_inertial/>
       <visual>
         <geometry>

Commit message: changed the origin of the left and right finger joints to avoid collision

File: cob_description/urdf/pg70/pg70.urdf.xacro (robot description, xacro)
@@ -54,5 +54,5 @@
     </link>
     <joint name="${name}_finger_left_joint" type="prismatic" >
-      <origin xyz="0 0 0.0789" rpy="0 0 0"/>
+      <origin xyz="0 0.0055 0.0789" rpy="0 0 0"/>
       <parent link="${name}_palm_link" />
       <child link="${name}_finger_left_link" />
@@ -80,5 +80,5 @@
     </link>
     <joint name="${name}_finger_right_joint" type="prismatic" >
-      <origin xyz="0 0 0.0789" rpy="-0 0 0"/>
+      <origin xyz="0 -0.0055 0.0789" rpy="-0 0 0"/>
       <parent link="${name}_palm_link" />
       <child link="${name}_finger_right_link" />
