Commit message: add a planar move plugin for raw-mini (no mecanum)

File: raw_description/urdf/base_mini/base.gazebo.xacro (robot description, xacro)
@@ -9,19 +9,12 @@
   </xacro:macro>
   <xacro:macro name="base_gazebo" params="name">
-    <gazebo reference="${name}_link">
-      <gravity>true</gravity>
-      <self_collide>false</self_collide>
-      <sensor name='${name}_contact_sensor' type='contact'>
-        <always_on>true</always_on>
-        <update_rate>100.0</update_rate>
-        <contact>
-          <collision>${name}_link_collision</collision>
-          <topic>${name}_bumper</topic>
-        </contact>
-        <plugin name="${name}_gazebo_ros_bumper_controller" filename="libgazebo_ros_bumper.so">
-          <frameName>world</frameName>
-          <bumperTopicName>${name}_bumper</bumperTopicName>
-        </plugin>
-      </sensor>
+    <gazebo>
+      <plugin name="object_controller" filename="libgazebo_ros_planar_move.so">
+        <commandTopic>cmd_vel</commandTopic>
+        <odometryTopic>odom</odometryTopic>
+        <odometryFrame>odom</odometryFrame>
+        <odometryRate>20.0</odometryRate>
+        <robotBaseFrame>${name}_footprint</robotBaseFrame>
+      </plugin>
     </gazebo>
     <gazebo>
@@ -32,5 +25,5 @@
         <topicName>${name}_pose_ground_truth</topicName>
         <frameName>map</frameName>
-        <xyzOffsets>25.7 25.7 0</xyzOffsets>  <!-- initialize odometry for fake localization-->
+        <xyzOffsets>25.7 25.7 0</xyzOffsets>        <!-- initialize odometry for fake localization-->
         <rpyOffsets>0 0 0</rpyOffsets>
         <gaussianNoise>0.01</gaussianNoise>

File: raw_description/urdf/base_mini/base.urdf.xacro (robot description, xacro)
@@ -58,3 +58,4 @@
     </xacro:mecanum_wheel>
   </xacro:macro>
+  <xacro:base_gazebo name="base"/>
 </robot>
