Commit message: Updated config for raw-mini

File: raw_description/urdf/base_mini/base.urdf.xacro (robot description, xacro)
@@ -6,10 +6,10 @@
   <xacro:include filename="$(find cob_description)/urdf/drive_wheel/drive_wheel.urdf.xacro" />
   <!-- properties -->
-  <xacro:property name="caster_offset_x" value="0.228" />  <!--modify here-->
-  <xacro:property name="caster_offset_y_bl" value="0.134" />
-  <xacro:property name="caster_offset_y_br" value="-0.184" />
-  <xacro:property name="caster_offset_y_fl" value="0.184" />
-  <xacro:property name="caster_offset_y_fr" value="-0.134" />
-  <xacro:property name="caster_offset_z" value="0.08" />
+  <xacro:property name="caster_offset_x" value="0.092" />  <!--modify here-->
+  <xacro:property name="caster_offset_y_bl" value="0.115" />
+  <xacro:property name="caster_offset_y_br" value="-0.115" />
+  <xacro:property name="caster_offset_y_fl" value="0.115" />
+  <xacro:property name="caster_offset_y_fr" value="-0.115" />
+  <xacro:property name="caster_offset_z" value="0.05" />
   <xacro:property name="battery_offset_x" value="0.0" />
   <xacro:property name="battery_offset_y" value="-0.008" />

Commit message: use updated meshes

File: raw_description/urdf/base_mini/base.urdf.xacro (robot description, xacro)
@@ -4,12 +4,9 @@
   <xacro:include filename="$(find raw_description)/urdf/base_mini/base.gazebo.xacro" />
   <!-- drive_wheel module -->
-  <xacro:include filename="$(find cob_description)/urdf/drive_wheel/drive_wheel.urdf.xacro" />
+  <xacro:include filename="$(find raw_description)/urdf/mecanum_wheel/mecanum_wheel.urdf.xacro" />
   <!-- properties -->
-  <xacro:property name="caster_offset_x" value="0.092" />  <!--modify here-->
-  <xacro:property name="caster_offset_y_bl" value="0.115" />
-  <xacro:property name="caster_offset_y_br" value="-0.115" />
-  <xacro:property name="caster_offset_y_fl" value="0.115" />
-  <xacro:property name="caster_offset_y_fr" value="-0.115" />
-  <xacro:property name="caster_offset_z" value="0.05" />
+  <xacro:property name="caster_offset_x" value="0.115" />
+  <xacro:property name="caster_offset_y" value="0.09" />
+  <xacro:property name="caster_offset_z" value="0.00" />
   <xacro:property name="battery_offset_x" value="0.0" />
   <xacro:property name="battery_offset_y" value="-0.008" />
@@ -23,5 +20,5 @@
     <link name="${name}_footprint"/>
     <joint name="${name}_footprint_joint" type="fixed">
-      <origin xyz="0 0 0" rpy="0 0 0" />
+      <origin xyz="0 0 0.05" rpy="0 0 0" />
       <parent link="${name}_footprint"/>
       <child link="${name}_link" />
@@ -31,17 +28,16 @@
         <origin xyz="0 0 0" />
         <mass value="${base_mass}" />
-        <inertia ixx="9.64" ixy="-0.02" ixz="0.44"
-                 iyy="11.33" iyz="-0.007" izz="3.07" />
+        <inertia ixx="9.64" ixy="-0.02" ixz="0.44" iyy="11.33" iyz="-0.007" izz="3.07" />
       </inertial>
       <visual>
-        <origin xyz="0 0 0.209" rpy="0 0 0" />
+        <origin xyz="0 0 0" rpy="0 0 0" />
         <geometry>
-          <mesh filename="package://raw_description/meshes/base/raw_base_short.dae"/>
+          <mesh filename="package://raw_description/meshes/base/raw_mini_base.dae"/>
         </geometry>
       </visual>
       <collision>
-        <origin xyz="0 0 0.209" rpy="0 0 0" />
+        <origin xyz="0 0 0" rpy="0 0 0" />
         <geometry>
-          <mesh filename="package://raw_description/meshes/base/raw_base_short.stl"/>
+          <mesh filename="package://raw_description/meshes/base/raw_mini_base.dae"/>
           <!--box size="0.758 0.573 0.096"/-->
         </geometry>
@@ -49,16 +45,16 @@
     </link>
     <!-- arrangement of the four drive_wheel modules -->
-    <xacro:drive_wheel parent="${name}_link" suffix="fl" >
-      <origin xyz="${caster_offset_x} ${caster_offset_y_fl} ${caster_offset_z}" rpy="0 0 0" />
-    </xacro:drive_wheel>
-    <xacro:drive_wheel parent="${name}_link" suffix="fr" >
-      <origin xyz="${caster_offset_x} ${caster_offset_y_fr} ${caster_offset_z}" rpy="0 0 0" />
-    </xacro:drive_wheel>
-    <xacro:drive_wheel parent="${name}_link" suffix="bl" >
-      <origin xyz="${-caster_offset_x} ${caster_offset_y_bl} ${caster_offset_z}" rpy=" 0 0 0" />
-    </xacro:drive_wheel>
-    <xacro:drive_wheel parent="${name}_link" suffix="br"  >
-      <origin xyz="${-caster_offset_x} ${caster_offset_y_br} ${caster_offset_z}" rpy="0 0 0" />
-    </xacro:drive_wheel>
+    <xacro:mecanum_wheel parent="${name}_link" suffix="fl">
+      <origin xyz="${caster_offset_x} ${caster_offset_y} ${caster_offset_z}" rpy="${M_PI/2} 0 0" />
+    </xacro:mecanum_wheel>
+    <xacro:mecanum_wheel parent="${name}_link" suffix="fr">
+      <origin xyz="${caster_offset_x} ${-caster_offset_y} ${caster_offset_z}" rpy="${-M_PI/2} 0 0" />
+    </xacro:mecanum_wheel>
+    <xacro:mecanum_wheel parent="${name}_link" suffix="bl">
+      <origin xyz="${-caster_offset_x} ${caster_offset_y} ${caster_offset_z}" rpy="${M_PI/2} 0 0" />
+    </xacro:mecanum_wheel>
+    <xacro:mecanum_wheel parent="${name}_link" suffix="br">
+      <origin xyz="${-caster_offset_x} ${-caster_offset_y} ${caster_offset_z}" rpy="${-M_PI/2} 0 0" />
+    </xacro:mecanum_wheel>
   </xacro:macro>
 </robot>

Commit message: remove unneeded values

File: raw_description/urdf/base_mini/base.urdf.xacro (robot description, xacro)
@@ -9,13 +9,6 @@
   <xacro:property name="caster_offset_y" value="0.09" />
   <xacro:property name="caster_offset_z" value="0.00" />
-  <xacro:property name="battery_offset_x" value="0.0" />
-  <xacro:property name="battery_offset_y" value="-0.008" />
-  <xacro:property name="battery_offset_z" value="0.065" />
-  <xacro:property name="base_mass" value="43.1" />
-  <xacro:property name="battery_mass" value="40" />
-  <xacro:property name="battery_size_x" value="0.5" />
-  <xacro:property name="battery_size_y" value="0.148" />
-  <xacro:property name="battery_size_z" value="0.26" />
-  <xacro:macro name="raw_base" params="name">
+  <xacro:property name="base_mass" value="2" />
+  <xacro:macro name="raw_mini_base" params="name">
     <link name="${name}_footprint"/>
     <joint name="${name}_footprint_joint" type="fixed">
@@ -25,9 +18,7 @@
     </joint>
     <link name="${name}_link">
-      <inertial>
+      <xacro:box_inertial x="0.3" y="0.2" z="0.15" mass="${base_mass}">
         <origin xyz="0 0 0" />
-        <mass value="${base_mass}" />
-        <inertia ixx="9.64" ixy="-0.02" ixz="0.44" iyy="11.33" iyz="-0.007" izz="3.07" />
-      </inertial>
+      </xacro:box_inertial>
       <visual>
         <origin xyz="0 0 0" rpy="0 0 0" />
